File: kicad5/traction/traction-card.sch (KiCad schematic (older format))
At the start: 217 parts, among them Y1 CX3225GA40000D0PTVCC

Commit message: Rev A.3: end-to-end verification campaign — 18 defects found & fixed, datasheet pack
Three independent verification layers, all green at datasheet-real constants:
- geometric pin-verify 1540/1540 (100%)
- structural ERC audit (new erc-audit.mjs): 664 intent-level checks, 0 fail
- numeric worst-case verification (new design-verify.mjs): 51 PASS / 3 WARN /
  0 FAIL at real corners (Vbus->850V, KL30 9-16V, R+/-5%, C+10%)

Findings fixed (docs/verification-report.md, F1-F36): flyback CS scaling, FB
reference mis-scaled for controller swap (supply could never start), missing
VCC start path, five net-alias floating pins, Y-cap class at 850V, common-cause
VDC sense bias, load-dump cap ratings, discharge worst-case corner (470R),
OV-witness headroom (6.2k), ASC abs-max violation (5.1V clamp), real HCS600
pin map + HS DESAT to aux drain-sense, +15/-5.1 drive combo, UCC28C40 UVLO
grade for cold-crank, flyback re-derived for real VGT12EEM (10uH, 1:1.6:2.9,
250kHz, 11.8V NF regulation), FS26 VMONEXT 0.8V reference divider, FS0B/FS1B
pull-up current, S32K39 core ballast topology (V15S + SQ2310ES).

Datasheet pack: 36 verified PDFs in docs/datasheets/ + EXTRACTED-PARAMS.md.
Sheets/BOM/README regenerated at A.3 (529 components, Rs 69.8k @1k).

Co-Authored-By: Claude Fable 5 <noreply@anthropic.com>
Parts:
- removed UMCU: S32K396, BGA289, symbol traction-r1:S32K396
- added RCPD1, RCPD2, RCPD3: 10k, R0603, symbol traction-r1:R
- CCAN1: renamed from RCT1B; value 60.4R -> 1uF; footprint R0603 -> C0603; symbol traction-r1:R -> traction-r1:C; MPN R0603-60R4-1% -> MLCC-1uF-25V
- CCAN2: renamed from RCT2B; value 60.4R -> 1uF; footprint R0603 -> C0603; symbol traction-r1:R -> traction-r1:C; MPN R0603-60R4-1% -> MLCC-1uF-25V
- CCOSA1: renamed from CCOSD; value 220pF -> 100pF
- CCOSA2: renamed from CCOSF; value 22pF -> 2.2nF
- CCOSD: renamed from RCOS1; value 680R -> 220pF; footprint R0603 -> C0603; symbol traction-r1:R -> traction-r1:C; MPN R0603-CLASS -> MLCC-CLASS
- CCOSF: renamed from RCOS2; value 680R -> 22pF; footprint R0603 -> C0603; symbol traction-r1:R -> traction-r1:C; MPN R0603-CLASS -> MLCC-CLASS
- CCT1: renamed from LCAN2; value ACT45B-101-2P-TL003 -> 4.7nF; footprint CMC1210 -> C0603; symbol traction-r1:ACT45B-101-2P-TL003 -> traction-r1:C; MPN ACT45B-101-2P-TL003 -> MLCC-4.7nF-50V
- CCT2: renamed from JVEH; value TE 776231-1 (AMPSEAL 23) -> 4.7nF; footprint AMPSEAL23 -> C0603; symbol traction-r1:TE_776231-1__AMPSEAL_23_ -> traction-r1:C; MPN TE 776231-1 (AMPSEAL 23) -> MLCC-4.7nF-50V
- CEXA1: renamed from CEXA3; value 100nF -> 4.7nF
- CEXA2: renamed from CEXD; value 4.7uF -> 300pF
- CEXA3: renamed from REXA1; value 3k -> 100nF; footprint R0603 -> C0603; symbol traction-r1:R -> traction-r1:C; MPN R0603-CLASS -> MLCC-CLASS
- CEXD: renamed from REXA2; value 10k -> 4.7uF; footprint R0603 -> C0603; symbol traction-r1:R -> traction-r1:C; MPN R0603-CLASS -> MLCC-CLASS
- CFLTF: renamed from RENP2; value 120R -> 100pF; footprint R0603 -> C0603; symbol traction-r1:R -> traction-r1:C; MPN R0603-120R -> MLCC-100pF-16V
- CIGN: renamed from RIGN1; value 5.1k -> 100nF; footprint R0603 -> C0603; symbol traction-r1:R -> traction-r1:C; MPN R0603-5k1 -> MLCC-100nF-50V
- CILK: renamed from RILK2; value 10k -> 2.2nF; footprint R0603 -> C0603; symbol traction-r1:R -> traction-r1:C; MPN R0603-10k -> MLCC-2.2nF-50V
- CLAT: renamed from RFS1; value 120R -> 100nF; footprint R0603 -> C0603; symbol traction-r1:R -> traction-r1:C; MPN R0603-120R -> MLCC-100nF-16V
- CLVC1: renamed from CLVC2; MPN MLCC-4.7uF-25V -> MLCC-4.7uF-50V
- CLVC2: renamed from DREVC; value STPS5L60S -> 4.7uF; footprint SMC -> C1206; symbol traction-r1:D -> traction-r1:C; LCSC C140620 -> CLASS; MPN STPS5L60S -> MLCC-4.7uF-50V
- CMA1: renamed from CMA2; value 100nF -> 1uF
- CMA2: renamed from CMD1; footprint C0402 -> C0603; MPN MLCC-100nF-16V -> MLCC-1uF-16V
- CMD9: renamed from CYA; value 12pF -> 100nF; footprint C0603 -> C0402; MPN MLCC-12pF-50V -> MLCC-100nF-16V
- CMT1F: renamed from FMT2; value FUSE-350mA-0603 -> 47nF; footprint F0603 -> C0603; symbol traction-r1:F -> traction-r1:C; MPN FUSE-350mA-0603 -> MLCC-47nF-25V
- CMT2F: renamed from RMT1P; value 10k -> 47nF; footprint R0603 -> C0603; symbol traction-r1:R -> traction-r1:C; MPN R0603-CLASS -> MLCC-47nF-25V
- CRST: renamed from RBOOT; value 10k -> 100pF; footprint R0603 -> C0603; symbol traction-r1:R -> traction-r1:C; MPN R0603-10k -> MLCC-100pF-16V
- CSB3: renamed from CSB5; value 1uF -> 10uF
- CSB4: renamed from CSB6; value 1uF -> 10uF
- CSB5: renamed from CSB7; value 10uF -> 1uF
- CSB6: renamed from CSB8; value 10uF -> 1uF
- CSB7: renamed from DBAT; value BAT46ZFILM -> 10uF; footprint SOD123 -> C0805; symbol traction-r1:D -> traction-r1:C; LCSC C283255 -> CLASS; MPN BAT46ZFILM -> MLCC-CLASS
- CSB8: renamed from LCOR; value IND-4.7uH-2A -> 10uF; footprint IND5x5 -> C0805; symbol traction-r1:L -> traction-r1:C; MPN IND-4.7uH-2A -> MLCC-CLASS
- CSINA1: renamed from CSIND; value 220pF -> 100pF
- CSINA2: renamed from CSINF; value 22pF -> 2.2nF
- CSIND: renamed from RSIN1; value 680R -> 220pF; footprint R0603 -> C0603; symbol traction-r1:R -> traction-r1:C; MPN R0603-CLASS -> MLCC-CLASS
- CSINF: renamed from RSIN2; value 680R -> 22pF; footprint R0603 -> C0603; symbol traction-r1:R -> traction-r1:C; MPN R0603-CLASS -> MLCC-CLASS
- CSNVF: renamed from RSNUP; value 5.1k -> 47nF; footprint R0603 -> C0603; symbol traction-r1:R -> traction-r1:C; MPN R0603-4k99 -> MLCC-47nF-25V
- CSNWF: renamed from RSNVP; value 5.1k -> 47nF; footprint R0603 -> C0603; symbol traction-r1:R -> traction-r1:C; MPN R0603-4k99 -> MLCC-47nF-25V
- CTAMBF: renamed from JTHS; value NTC-10k-0603 -> 47nF; footprint R0603 -> C0603; symbol traction-r1:J2 -> traction-r1:C; MPN NTC-10k-0603 -> MLCC-47nF-25V
- CTHSF: renamed from RTAMBP; value 10k -> 47nF; footprint R0603 -> C0603; symbol traction-r1:R -> traction-r1:C; MPN R0603-10k-1% -> MLCC-47nF-25V
- CUB1: renamed from CUS1; value 47nF -> 3.3nF; MPN MLCC-47nF-25V -> MLCC-3.3nF-50V
- CUB2: renamed from CUS2; value 4.7nF -> 100nF; MPN MLCC-47nF-25V -> MLCC-3.3nF-50V
- CUS1: renamed from LUB; value FB-220R-1A -> 47nF; footprint FB0805 -> C0603; symbol traction-r1:L -> traction-r1:C; MPN FB-220R-1A -> MLCC-47nF-25V
- CUS2: renamed from RUB1; value 100R -> 4.7nF; footprint R0603 -> C0603; symbol traction-r1:R -> traction-r1:C; MPN R0603-100R -> MLCC-47nF-25V
- CVB1: renamed from CVS1; value 47nF -> 3.3nF; MPN MLCC-47nF-25V -> MLCC-3.3nF-50V
- CVB2: renamed from CVS2; value 4.7nF -> 100nF; MPN MLCC-47nF-25V -> MLCC-3.3nF-50V
- CVD1: renamed from RVD1B; value 10k -> 100pF; footprint R0603 -> C0603; symbol traction-r1:R -> traction-r1:C; MPN R0603-10k-0.1% -> MLCC-CLASS
- CVD2: renamed from RVD2B; value 10k -> 100pF; footprint R0603 -> C0603; symbol traction-r1:R -> traction-r1:C; MPN R0603-10k-0.1% -> MLCC-CLASS
- CVM1: renamed from RVM1; value 24k -> 220nF; footprint R0603 -> C0603; symbol traction-r1:R -> traction-r1:C; MPN R0603-24k-1% -> MLCC-CLASS
- CVM2: renamed from RVM2; value 24k -> 220nF; footprint R0603 -> C0603; symbol traction-r1:R -> traction-r1:C; MPN R0603-24k-1% -> MLCC-CLASS
- CVS1: renamed from LVB; value FB-220R-1A -> 47nF; footprint FB0805 -> C0603; symbol traction-r1:L -> traction-r1:C; MPN FB-220R-1A -> MLCC-47nF-25V
- CVS2: renamed from RVB1; value 100R -> 4.7nF; footprint R0603 -> C0603; symbol traction-r1:R -> traction-r1:C; MPN R0603-100R -> MLCC-47nF-25V
- CWB1: renamed from CWS1; value 47nF -> 3.3nF; MPN MLCC-47nF-25V -> MLCC-3.3nF-50V
- CWB2: renamed from CWS2; value 4.7nF -> 100nF; MPN MLCC-47nF-25V -> MLCC-3.3nF-50V
- CWS1: renamed from LWB; value FB-220R-1A -> 47nF; footprint FB0805 -> C0603; symbol traction-r1:L -> traction-r1:C; MPN FB-220R-1A -> MLCC-47nF-25V
- CWS2: renamed from RWB1; value 100R -> 4.7nF; footprint R0603 -> C0603; symbol traction-r1:R -> traction-r1:C; MPN R0603-100R -> MLCC-47nF-25V
- CYB: renamed from RMRST; value 10k -> 12pF; footprint R0603 -> C0603; symbol traction-r1:R -> traction-r1:C; MPN R0603-10k -> MLCC-12pF-50V
- DBAT: renamed from LSBC; value IND-10uH-2A -> BAT46ZFILM; footprint IND6x6 -> SOD123; symbol traction-r1:L -> traction-r1:D; LCSC CLASS -> C283255; MPN IND-10uH-2A -> BAT46ZFILM
- DCOSP: renamed from CCOSA2; value 2.2nF -> PESD5V0L1BA; footprint C0603 -> SOD323; symbol traction-r1:C -> traction-r1:PESD5V0L1BA; MPN MLCC-CLASS -> PESD5V0L1BA
- DIGN: renamed from RIGN2; value 10k -> 1N4148WS; footprint R0603 -> SOD323; symbol traction-r1:R -> traction-r1:D; LCSC CLASS -> C2128; MPN R0603-5k1 -> 1N4148WS
- DMT1: renamed from UMT2; value OPA333AQDBVRQ1 -> PESD5V0U1UA; footprint SOT23-5 -> SOD323; symbol traction-r1:OPA333AQDBVRQ1 -> traction-r1:PESD5V0U1UA; LCSC C2058544 -> CLASS; MPN OPA333AQDBVRQ1 -> PESD5V0U1UA
- DMT2: renamed from CMT1F; value 47nF -> PESD5V0U1UA; footprint C0603 -> SOD323; symbol traction-r1:C -> traction-r1:PESD5V0U1UA; MPN MLCC-47nF-25V -> PESD5V0U1UA
- DREVC: renamed from DTVSC; value TPSMC24CA -> STPS5L60S; LCSC C1975284 -> C140620; MPN TPSMC24CA -> STPS5L60S
- DSINP: renamed from CSINA2; value 2.2nF -> PESD5V0L1BA; footprint C0603 -> SOD323; symbol traction-r1:C -> traction-r1:PESD5V0L1BA; MPN MLCC-CLASS -> PESD5V0L1BA
- DTVSC: renamed from FLVC; value MF-LSMF300/24X-2 -> TPSMC24CA; footprint PTC2920 -> SMC; symbol traction-r1:F -> traction-r1:D; LCSC C719172 -> C1975284; MPN MF-LSMF300/24X-2 -> TPSMC24CA
- FLVC: renamed from LFC; value FB-120R-3A -> MF-LSMF300/24X-2; footprint FB1206 -> PTC2920; symbol traction-r1:L -> traction-r1:F; LCSC CLASS -> C719172; MPN FB-120R-3A -> MF-LSMF300/24X-2
- FMT1: renamed from RMT1S; value 1k -> FUSE-350mA-0603; footprint R0603 -> F0603; symbol traction-r1:R -> traction-r1:F; MPN R0603-CLASS -> FUSE-350mA-0603
- FMT2: renamed from RMT2P; value 10k -> FUSE-350mA-0603; footprint R0603 -> F0603; symbol traction-r1:R -> traction-r1:F; MPN R0603-CLASS -> FUSE-350mA-0603
- FVS1: renamed from LVS3; value FB-470R -> MF-LSMF; footprint FB0603 -> PTC1206; symbol traction-r1:L -> traction-r1:F; MPN FB-470R-CLASS -> MF-LSMF-CLASS
- JICC: renamed from RCPD2; value 10k -> MICROFIT3-40; footprint R0603 -> MicroFit40; symbol traction-r1:R -> traction-r1:MICROFIT3-40; MPN R0603-10k -> MICROFIT3-40
- JLEM: renamed from USNSV; value HC5FW900-S -> T2M-105-01-L-D-TH-WT; footprint OffBoard -> HDR2x5; symbol traction-r1:HC5FW900-S -> traction-r1:T2M-105-01-L-D-TH-WT; MPN HC5FW900-S -> T2M-105-01-L-D-TH-WT
- JSWD: renamed from CRST; value 100pF -> HDR2X10-JTAG; footprint C0603 -> HDR2x10; symbol traction-r1:C -> traction-r1:HDR2X10-JTAG; MPN MLCC-100pF-16V -> HDR2X10-JTAG
- JTAMB: renamed from RTHSP; value 10k -> NTC-10k-0603; symbol traction-r1:R -> traction-r1:J2; MPN R0603-10k-1% -> NTC-10k-0603
- JTHS: renamed from DMT1; value PESD5V0U1UA -> NTC-10k-0603; footprint SOD323 -> R0603; symbol traction-r1:PESD5V0U1UA -> traction-r1:J2; MPN PESD5V0U1UA -> NTC-10k-0603
- JVEH: renamed from LVS2; value FB-470R -> TE 776231-1 (AMPSEAL 23); footprint FB0603 -> AMPSEAL23; symbol traction-r1:L -> traction-r1:TE_776231-1__AMPSEAL_23_; MPN FB-470R-CLASS -> TE 776231-1 (AMPSEAL 23)
- LCAN1: renamed from CCAN1; value 1uF -> ACT45B-101-2P-TL003; footprint C0603 -> CMC1210; symbol traction-r1:C -> traction-r1:ACT45B-101-2P-TL003; MPN MLCC-1uF-25V -> ACT45B-101-2P-TL003
- LCAN2: renamed from CCAN2; value 1uF -> ACT45B-101-2P-TL003; footprint C0603 -> CMC1210; symbol traction-r1:C -> traction-r1:ACT45B-101-2P-TL003; MPN MLCC-1uF-25V -> ACT45B-101-2P-TL003
- LCOR: renamed from RAGT; value 0R -> IND-4.7uH-2A; footprint R0603 -> IND5x5; symbol traction-r1:R -> traction-r1:L; MPN R0603-CLASS -> IND-4.7uH-2A
- LFC: renamed from USBC; value FS2633D -> FB-120R-3A; footprint HLQFP48 -> FB1206; symbol traction-r1:FS2633D -> traction-r1:L; MPN FS2633D -> FB-120R-3A
- LSBC: renamed from RSB1; value 10k -> IND-10uH-2A; footprint R0603 -> IND6x6; symbol traction-r1:R -> traction-r1:L; MPN R0603-CLASS -> IND-10uH-2A
- LUB: renamed from RUB2; value 100R -> FB-220R-1A; footprint R0603 -> FB0805; symbol traction-r1:R -> traction-r1:L; MPN R0603-100R -> FB-220R-1A
- LVB: renamed from RVB2; value 100R -> FB-220R-1A; footprint R0603 -> FB0805; symbol traction-r1:R -> traction-r1:L; MPN R0603-100R -> FB-220R-1A
- LVS2: renamed from JICC; value MICROFIT3-40 -> FB-470R; footprint MicroFit40 -> FB0603; symbol traction-r1:MICROFIT3-40 -> traction-r1:L; MPN MICROFIT3-40 -> FB-470R-CLASS
- LVS3: renamed from RCPD0; value 10k -> FB-470R; footprint R0603 -> FB0603; symbol traction-r1:R -> traction-r1:L; MPN R0603-10k -> FB-470R-CLASS
- LVS4: renamed from RCPD1; value 10k -> FB-470R; footprint R0603 -> FB0603; symbol traction-r1:R -> traction-r1:L; MPN R0603-10k -> FB-470R-CLASS
- LWB: renamed from RWB2; value 100R -> FB-220R-1A; footprint R0603 -> FB0805; symbol traction-r1:R -> traction-r1:L; MPN R0603-100R -> FB-220R-1A
- QBAL: renamed from CSB1; value 10uF -> SQ2310ES; footprint C0805 -> SOT23; symbol traction-r1:C -> traction-r1:SQ2310ES; MPN MLCC-CLASS -> SQ2310ES
- RAGT: renamed from RSB2; value 18.7k -> 0R
- RASCP: renamed from RFS2; value 120R -> 10k; MPN R0603-120R -> R0603-10k
- renumbered CMD10 to CMD1, CMD11 to CMD10, CMD12 to CMD11, CMD2 to CMD12, CMD3 to CMD2, CMD4 to CMD3, CMD5 to CMD4, CMD6 to CMD5, CMD7 to CMD6, CMD8 to CMD7, CMD9 to CMD8, CSB3 to CSB1, CSB4 to CSB2, CSNWF to CSNUF, CYB to CYA, LVS4 to LVS1, RCPD3 to RCPD0, REXB2 to REXA4, REXB3 to REXB1, REXB4 to REXB2, REXM3 to REXM1, RRDYP1 to RFLTP2, RFS3 to RFS1, RFS4 to RFS2, RILK3 to RILK1, RILK4 to RILK2, RSNWP to RSNUP, RUB3 to RUB1, RVB3 to RVB1, RVD1C to RVD1A, RVD1D to RVD1B, RVD2C to RVD2A, RVD2D to RVD2B, RVM3 to RVM1, RVM4 to RVM2, RWB3 to RWB1, USNSW to USNSU
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Connections:
- net labels added: BCTRL, V15S
- net labels removed: NTC_AMB, NTC_HS, TSNS_U, TSNS_V, TSNS_W
- wire segments 694 -> 701
Other:
- note added: "rev A.3 - 26 sections - 219 components"
- note removed: "rev A.2 - 26 sections - 217 components"
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
Commit message: Split discharge onto a bolt-on board (XM3 pattern), 3-sheet set
- boards/discharge.tsx: bleeder (2x5x27k) + active discharge (4x470R +
  HCM75S12T4K3, TLP152/QA01C default-OFF) on its own PCB across the cap
  bank; power board keeps JDIS header (V15/QDIS_CMD/2xGND) + CMD pulldown
- pipeline: disch side threaded through pages/gen/verify/print/pdf/bom;
  sheet idents 1..3 of 3; disch title block carries "NEVER energize
  without this board fitted"; root sheet de-branded (X-IN-One -> Traction)
- gates green: 1550/1550 pins, ERC 672/0, design-verify 51P/3W/0F
- docs: README + design-basis + bom synced to 3-board state; new
  docs/img/sheet-disch.png; BOM ₹69,856 @1k (63,375/672/5,808)

Co-Authored-By: Claude Fable 5 <noreply@anthropic.com>
Parts:
- removed CMA1: 1uF, C0603, symbol traction-r1:C
- removed CMA2: 100nF, C0603, symbol traction-r1:C
- removed CMD1: 100nF, C0402, symbol traction-r1:C
- removed UMCU: S32K396, BGA289, symbol traction-r1:S32K396
- added RCPD0, RCPD1, RCPD2, RCPD3: 10k, R0603, symbol traction-r1:R
- CCAN1: renamed from LCAN2; value ACT45B-101-2P-TL003 -> 1uF; footprint CMC1210 -> C0603; symbol traction-r1:ACT45B-101-2P-TL003 -> traction-r1:C; MPN ACT45B-101-2P-TL003 -> MLCC-1uF-25V
- CCAN2: renamed from JVEH; value TE 776231-1 (AMPSEAL 23) -> 1uF; footprint AMPSEAL23 -> C0603; symbol traction-r1:TE_776231-1__AMPSEAL_23_ -> traction-r1:C; MPN TE 776231-1 (AMPSEAL 23) -> MLCC-1uF-25V
- CCOSA1: renamed from RCOS1; value 680R -> 100pF; footprint R0603 -> C0603; symbol traction-r1:R -> traction-r1:C; MPN R0603-CLASS -> MLCC-CLASS
- CCOSA2: renamed from RCOS2; value 680R -> 2.2nF; footprint R0603 -> C0603; symbol traction-r1:R -> traction-r1:C; MPN R0603-CLASS -> MLCC-CLASS
- CCOSD: renamed from RCOSF1; value 330R -> 220pF; footprint R0603 -> C0603; symbol traction-r1:R -> traction-r1:C; MPN R0603-CLASS -> MLCC-CLASS
- CCOSF: renamed from RCOSF2; value 330R -> 22pF; footprint R0603 -> C0603; symbol traction-r1:R -> traction-r1:C; MPN R0603-CLASS -> MLCC-CLASS
- CCT1: renamed from TVSC2; value PESD2IVN24-T -> 4.7nF; footprint SOT23 -> C0603; symbol traction-r1:PESD2IVN24-T -> traction-r1:C; LCSC C406047 -> CLASS; MPN PESD2IVN24-T -> MLCC-4.7nF-50V
- CCT2: renamed from FVS1; value MF-LSMF -> 4.7nF; footprint PTC1206 -> C0603; symbol traction-r1:F -> traction-r1:C; MPN MF-LSMF-CLASS -> MLCC-4.7nF-50V
- CEXA1: renamed from REXA1; value 3k -> 4.7nF; footprint R0603 -> C0603; symbol traction-r1:R -> traction-r1:C; MPN R0603-CLASS -> MLCC-CLASS
- CEXA2: renamed from REXA2; value 10k -> 300pF; footprint R0603 -> C0603; symbol traction-r1:R -> traction-r1:C; MPN R0603-CLASS -> MLCC-CLASS
- CEXA3: renamed from REXA3; value 10k -> 100nF; footprint R0603 -> C0603; symbol traction-r1:R -> traction-r1:C; MPN R0603-CLASS -> MLCC-CLASS
- CEXD: renamed from REXA4; value 24k -> 4.7uF; footprint R0603 -> C0603; symbol traction-r1:R -> traction-r1:C; MPN R0603-CLASS -> MLCC-CLASS
- CFLTF: renamed from RFLTP2; value 5.1k -> 100pF; footprint R0603 -> C0603; symbol traction-r1:R -> traction-r1:C; MPN R0603-CLASS -> MLCC-100pF-16V
- CIGN: renamed from UAND1; value 74LVC1G11GW-Q100 -> 100nF; footprint SOT363 -> C0603; symbol traction-r1:74LVC1G11GW-Q100 -> traction-r1:C; LCSC C548242 -> CLASS; MPN 74LVC1G11GW-Q100 -> MLCC-100nF-50V
- CILK: renamed from RILK4; value 10k -> 2.2nF; footprint R0603 -> C0603; symbol traction-r1:R -> traction-r1:C; MPN R0603-10k -> MLCC-2.2nF-50V
- CLAT: renamed from RFS3; value 120R -> 100nF; footprint R0603 -> C0603; symbol traction-r1:R -> traction-r1:C; MPN R0603-120R -> MLCC-100nF-16V
- CLVC1: renamed from FLVC; value MF-LSMF300/24X-2 -> 4.7uF; footprint PTC2920 -> C1206; symbol traction-r1:F -> traction-r1:C; LCSC C719172 -> CLASS; MPN MF-LSMF300/24X-2 -> MLCC-4.7uF-50V
- CLVC2: renamed from LFC; value FB-120R-3A -> 4.7uF; footprint FB1206 -> C1206; symbol traction-r1:L -> traction-r1:C; MPN FB-120R-3A -> MLCC-4.7uF-50V
- CMA1: renamed from CMD11; value 100nF -> 1uF; footprint C0402 -> C0603; MPN MLCC-100nF-16V -> MLCC-1uF-16V
- CMA2: renamed from CMD12; footprint C0402 -> C0603; MPN MLCC-100nF-16V -> MLCC-1uF-16V
- CMD6: renamed from CYA; value 12pF -> 100nF; footprint C0603 -> C0402; MPN MLCC-12pF-50V -> MLCC-100nF-16V
- CMD7: renamed from CYB; value 12pF -> 100nF; footprint C0603 -> C0402; MPN MLCC-12pF-50V -> MLCC-100nF-16V
- CMD8: renamed from RMRST; value 10k -> 100nF; footprint R0603 -> C0402; symbol traction-r1:R -> traction-r1:C; MPN R0603-10k -> MLCC-100nF-16V
- CMD9: renamed from Y1; value CX3225GA40000D0PTVCC -> 100nF; footprint X3225 -> C0402; symbol traction-r1:Y -> traction-r1:C; LCSC C6009848 -> CLASS; MPN CX3225GA40000D0PTVCC -> MLCC-100nF-16V
- CMT1F: renamed from RMT1P; value 10k -> 47nF; footprint R0603 -> C0603; symbol traction-r1:R -> traction-r1:C; MPN R0603-CLASS -> MLCC-47nF-25V
- CMT2F: renamed from RMT1S; value 1k -> 47nF; footprint R0603 -> C0603; symbol traction-r1:R -> traction-r1:C; MPN R0603-CLASS -> MLCC-47nF-25V
- CRST: renamed from DREVC; value STPS5L60S -> 100pF; footprint SMC -> C0603; symbol traction-r1:D -> traction-r1:C; LCSC C140620 -> CLASS; MPN STPS5L60S -> MLCC-100pF-16V
- CSB1: renamed from CSB5; value 1uF -> 10uF
- CSB2: renamed from CSB6; value 1uF -> 10uF
- CSB5: renamed from DBAT; value BAT46ZFILM -> 1uF; footprint SOD123 -> C0805; symbol traction-r1:D -> traction-r1:C; LCSC C283255 -> CLASS; MPN BAT46ZFILM -> MLCC-CLASS
- CSB6: renamed from LCOR; value IND-4.7uH-2A -> 1uF; footprint IND5x5 -> C0805; symbol traction-r1:L -> traction-r1:C; MPN IND-4.7uH-2A -> MLCC-CLASS
- CSB7: renamed from LSBC; value IND-10uH-2A -> 10uF; footprint IND6x6 -> C0805; symbol traction-r1:L -> traction-r1:C; MPN IND-10uH-2A -> MLCC-CLASS
- CSB8: renamed from RAGT; value 0R -> 10uF; footprint R0603 -> C0805; symbol traction-r1:R -> traction-r1:C; MPN R0603-CLASS -> MLCC-CLASS
- CSINA1: renamed from RSIN1; value 680R -> 100pF; footprint R0603 -> C0603; symbol traction-r1:R -> traction-r1:C; MPN R0603-CLASS -> MLCC-CLASS
- CSINA2: renamed from RSIN2; value 680R -> 2.2nF; footprint R0603 -> C0603; symbol traction-r1:R -> traction-r1:C; MPN R0603-CLASS -> MLCC-CLASS
- CSIND: renamed from RSINF1; value 330R -> 220pF; footprint R0603 -> C0603; symbol traction-r1:R -> traction-r1:C; MPN R0603-CLASS -> MLCC-CLASS
- CSINF: renamed from RSINF2; value 330R -> 22pF; footprint R0603 -> C0603; symbol traction-r1:R -> traction-r1:C; MPN R0603-CLASS -> MLCC-CLASS
- CSNUF: renamed from RSNVP; value 5.1k -> 47nF; footprint R0603 -> C0603; symbol traction-r1:R -> traction-r1:C; MPN R0603-4k99 -> MLCC-47nF-25V
- CSNVF: renamed from RSNWP; value 5.1k -> 47nF; footprint R0603 -> C0603; symbol traction-r1:R -> traction-r1:C; MPN R0603-4k99 -> MLCC-47nF-25V
- CSNWF: renamed from RTMR; value 0R -> 47nF; footprint R0603 -> C0603; symbol traction-r1:R -> traction-r1:C; MPN R0603-CLASS -> MLCC-47nF-25V
- CTAMBF: renamed from RTAMBP; value 10k -> 47nF; footprint R0603 -> C0603; symbol traction-r1:R -> traction-r1:C; MPN R0603-10k-1% -> MLCC-47nF-25V
- CTHSF: renamed from RTHSP; value 10k -> 47nF; footprint R0603 -> C0603; symbol traction-r1:R -> traction-r1:C; MPN R0603-10k-1% -> MLCC-47nF-25V
- CUB1: renamed from LUB; value FB-220R-1A -> 3.3nF; footprint FB0805 -> C0603; symbol traction-r1:L -> traction-r1:C; MPN FB-220R-1A -> MLCC-3.3nF-50V
- CUB2: renamed from RUB1; value 100R -> 100nF; footprint R0603 -> C0603; symbol traction-r1:R -> traction-r1:C; MPN R0603-100R -> MLCC-3.3nF-50V
- CUS1: renamed from RUB2; value 100R -> 47nF; footprint R0603 -> C0603; symbol traction-r1:R -> traction-r1:C; MPN R0603-100R -> MLCC-47nF-25V
- CUS2: renamed from RUB3; value 100R -> 4.7nF; footprint R0603 -> C0603; symbol traction-r1:R -> traction-r1:C; MPN R0603-100R -> MLCC-47nF-25V
- CVB1: renamed from LVB; value FB-220R-1A -> 3.3nF; footprint FB0805 -> C0603; symbol traction-r1:L -> traction-r1:C; MPN FB-220R-1A -> MLCC-3.3nF-50V
- CVB2: renamed from RVB1; value 100R -> 100nF; footprint R0603 -> C0603; symbol traction-r1:R -> traction-r1:C; MPN R0603-100R -> MLCC-3.3nF-50V
- CVD1: renamed from RVD1D; value 10k -> 100pF; footprint R0603 -> C0603; symbol traction-r1:R -> traction-r1:C; MPN R0603-10k-0.1% -> MLCC-CLASS
- CVD2: renamed from RVD2D; value 10k -> 100pF; footprint R0603 -> C0603; symbol traction-r1:R -> traction-r1:C; MPN R0603-10k-0.1% -> MLCC-CLASS
- CVM1: renamed from RVM3; value 24k -> 220nF; footprint R0603 -> C0603; symbol traction-r1:R -> traction-r1:C; MPN R0603-24k-1% -> MLCC-CLASS
- CVM2: renamed from RVM4; value 24k -> 220nF; footprint R0603 -> C0603; symbol traction-r1:R -> traction-r1:C; MPN R0603-24k-1% -> MLCC-CLASS
- CVS1: renamed from RVB2; value 100R -> 47nF; footprint R0603 -> C0603; symbol traction-r1:R -> traction-r1:C; MPN R0603-100R -> MLCC-47nF-25V
- CVS2: renamed from RVB3; value 100R -> 4.7nF; footprint R0603 -> C0603; symbol traction-r1:R -> traction-r1:C; MPN R0603-100R -> MLCC-47nF-25V
- CWB1: renamed from LWB; value FB-220R-1A -> 3.3nF; footprint FB0805 -> C0603; symbol traction-r1:L -> traction-r1:C; MPN FB-220R-1A -> MLCC-3.3nF-50V
- CWB2: renamed from RWB1; value 100R -> 100nF; footprint R0603 -> C0603; symbol traction-r1:R -> traction-r1:C; MPN R0603-100R -> MLCC-3.3nF-50V
- CWS1: renamed from RWB2; value 100R -> 47nF; footprint R0603 -> C0603; symbol traction-r1:R -> traction-r1:C; MPN R0603-100R -> MLCC-47nF-25V
- CWS2: renamed from RWB3; value 100R -> 4.7nF; footprint R0603 -> C0603; symbol traction-r1:R -> traction-r1:C; MPN R0603-100R -> MLCC-47nF-25V
- CYA: renamed from JSWD; value HDR2X10-JTAG -> 12pF; footprint HDR2x10 -> C0603; symbol traction-r1:HDR2X10-JTAG -> traction-r1:C; MPN HDR2X10-JTAG -> MLCC-12pF-50V
- CYB: renamed from CRST; value 100pF -> 12pF; MPN MLCC-100pF-16V -> MLCC-12pF-50V
- DBAT: renamed from RSB1; value 52.3k -> BAT46ZFILM; footprint R0603 -> SOD123; symbol traction-r1:R -> traction-r1:D; LCSC CLASS -> C283255; MPN R0603-CLASS -> BAT46ZFILM
- DCOSP: renamed from CCOSF; value 22pF -> PESD5V0L1BA; footprint C0603 -> SOD323; symbol traction-r1:C -> traction-r1:PESD5V0L1BA; MPN MLCC-CLASS -> PESD5V0L1BA
- DIGN: renamed from UAND2; value 74LVC1G11GW-Q100 -> 1N4148WS; footprint SOT363 -> SOD323; symbol traction-r1:74LVC1G11GW-Q100 -> traction-r1:D; LCSC C548242 -> C2128; MPN 74LVC1G11GW-Q100 -> 1N4148WS
- DMT1: renamed from CMT1F; value 47nF -> PESD5V0U1UA; footprint C0603 -> SOD323; symbol traction-r1:C -> traction-r1:PESD5V0U1UA; MPN MLCC-47nF-25V -> PESD5V0U1UA
- DMT2: renamed from CMT2F; value 47nF -> PESD5V0U1UA; footprint C0603 -> SOD323; symbol traction-r1:C -> traction-r1:PESD5V0U1UA; MPN MLCC-47nF-25V -> PESD5V0U1UA
- DREVC: renamed from QBAL; value SQ2310ES -> STPS5L60S; footprint SOT23 -> SMC; symbol traction-r1:SQ2310ES -> traction-r1:D; LCSC CLASS -> C140620; MPN SQ2310ES -> STPS5L60S
- DSINP: renamed from CSINF; value 22pF -> PESD5V0L1BA; footprint C0603 -> SOD323; symbol traction-r1:C -> traction-r1:PESD5V0L1BA; MPN MLCC-CLASS -> PESD5V0L1BA
- DTVSC: renamed from USBC; value FS2633D -> TPSMC24CA; footprint HLQFP48 -> SMC; symbol traction-r1:FS2633D -> traction-r1:D; LCSC CLASS -> C1975284; MPN FS2633D -> TPSMC24CA
- FLVC: renamed from CSB1; value 10uF -> MF-LSMF300/24X-2; footprint C0805 -> PTC2920; symbol traction-r1:C -> traction-r1:F; LCSC CLASS -> C719172; MPN MLCC-CLASS -> MF-LSMF300/24X-2
- FMT1: renamed from RMT2P; value 10k -> FUSE-350mA-0603; footprint R0603 -> F0603; symbol traction-r1:R -> traction-r1:F; MPN R0603-CLASS -> FUSE-350mA-0603
- FMT2: renamed from RMT2S; value 1k -> FUSE-350mA-0603; footprint R0603 -> F0603; symbol traction-r1:R -> traction-r1:F; MPN R0603-CLASS -> FUSE-350mA-0603
- FVS1: renamed from LVS4; value FB-470R -> MF-LSMF; footprint FB0603 -> PTC1206; symbol traction-r1:L -> traction-r1:F; MPN FB-470R-CLASS -> MF-LSMF-CLASS
- JICC: renamed from RCPD3; value 10k -> MICROFIT3-40; footprint R0603 -> MicroFit40; symbol traction-r1:R -> traction-r1:MICROFIT3-40; MPN R0603-10k -> MICROFIT3-40
- JLEM: renamed from UUB1; value OPA376AQDBVRQ1 -> T2M-105-01-L-D-TH-WT; footprint SOT23-5 -> HDR2x5; symbol traction-r1:OPA376AQDBVRQ1 -> traction-r1:T2M-105-01-L-D-TH-WT; MPN OPA376AQDBVRQ1 -> T2M-105-01-L-D-TH-WT
- JSWD: renamed from CLVC2; value 4.7uF -> HDR2X10-JTAG; footprint C1206 -> HDR2x10; symbol traction-r1:C -> traction-r1:HDR2X10-JTAG; MPN MLCC-4.7uF-50V -> HDR2X10-JTAG
- JTAMB: renamed from DMT1; value PESD5V0U1UA -> NTC-10k-0603; footprint SOD323 -> R0603; symbol traction-r1:PESD5V0U1UA -> traction-r1:J2; MPN PESD5V0U1UA -> NTC-10k-0603
- JTHS: renamed from DMT2; value PESD5V0U1UA -> NTC-10k-0603; footprint SOD323 -> R0603; symbol traction-r1:PESD5V0U1UA -> traction-r1:J2; MPN PESD5V0U1UA -> NTC-10k-0603
- JVEH: renamed from LVS3; value FB-470R -> TE 776231-1 (AMPSEAL 23); footprint FB0603 -> AMPSEAL23; symbol traction-r1:L -> traction-r1:TE_776231-1__AMPSEAL_23_; MPN FB-470R-CLASS -> TE 776231-1 (AMPSEAL 23)
- LCAN1: renamed from CCT1; value 4.7nF -> ACT45B-101-2P-TL003; footprint C0603 -> CMC1210; symbol traction-r1:C -> traction-r1:ACT45B-101-2P-TL003; MPN MLCC-4.7nF-50V -> ACT45B-101-2P-TL003
- renumbered CMD2 to CMD1, CMD3 to CMD10, CMD4 to CMD11, CMD5 to CMD12, CMD6 to CMD2, CMD7 to CMD3, CMD8 to CMD4, CMD9 to CMD5, CSB7 to CSB3, CSB8 to CSB4, REXB4 to REXA4, REXM4 to REXB4, RRDYP2 to RFLTP1, RILK1 to RLAT1, RBOOT to RMRST, RVD2A to RVD1C, RVD2B to RVD1D
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Other:
- note added: "220 kW pk Control card (LV) - 3 of 3"
- note removed: "220 kW pk Control card (LV) - 2 of 2"
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
Commit message: Add cap-bank busbar assembly sheet + explicit interboard links (4 sheets)
- boards/capbank.tsx: the 16-can DC-link is its own laminated-busbar
  assembly (FR4 cannot carry the 340 A bus) with every terminal drawn:
  entry lugs, 3x module DC tab pairs, discharge-board studs
- power board keeps only its DCP/DCN entry taps (Y-caps, HVIL, sense)
- interboard links L1-L5 (harness, discharge 4-way, busbar, LEM, HVIL)
  documented in design-basis 10a + README table; erc-audit now asserts
  both ends of every link (new interboard section)
- NET NAMING panels state the cross-sheet net rule on every sheet
- gates green: 1560/1560 pins, ERC 687/0, design-verify 51P/3W/0F
- BOM ₹69,996 @1k (58,575 / 4,940 / 672 / 5,808) · 543 comps · 175 lines

Co-Authored-By: Claude Fable 5 <noreply@anthropic.com>
Parts:
- removed CMA1: 1uF, C0603, symbol traction-r1:C
- removed CMA2: 100nF, C0603, symbol traction-r1:C
- removed CMD1, CMD10, CMD11, CMD12, CMD2, CMD3, CMD4: 100nF, C0402, symbol traction-r1:C
- removed UMCU: S32K396, BGA289, symbol traction-r1:S32K396
- added FVS1: MF-LSMF, PTC1206, symbol traction-r1:F
- added JICC: MICROFIT3-40, MicroFit40, symbol traction-r1:MICROFIT3-40
- added LVS1, LVS2, LVS3, LVS4: FB-470R, FB0603, symbol traction-r1:L
- added RCPD0, RCPD1, RCPD2, RCPD3: 10k, R0603, symbol traction-r1:R
- CCAN1: renamed from RCT2B; value 60.4R -> 1uF; footprint R0603 -> C0603; symbol traction-r1:R -> traction-r1:C; MPN R0603-60R4-1% -> MLCC-1uF-25V
- CCAN2: renamed from JICC; value MICROFIT3-40 -> 1uF; footprint MicroFit40 -> C0603; symbol traction-r1:MICROFIT3-40 -> traction-r1:C; MPN MICROFIT3-40 -> MLCC-1uF-25V
- CCOSA1: renamed from JLEM; value T2M-105-01-L-D-TH-WT -> 100pF; footprint HDR2x5 -> C0603; symbol traction-r1:T2M-105-01-L-D-TH-WT -> traction-r1:C; MPN T2M-105-01-L-D-TH-WT -> MLCC-CLASS
- CCOSA2: renamed from USNSU; value HC5FW900-S -> 2.2nF; footprint OffBoard -> C0603; symbol traction-r1:HC5FW900-S -> traction-r1:C; MPN HC5FW900-S -> MLCC-CLASS
- CCOSD: renamed from USNSV; value HC5FW900-S -> 220pF; footprint OffBoard -> C0603; symbol traction-r1:HC5FW900-S -> traction-r1:C; MPN HC5FW900-S -> MLCC-CLASS
- CCOSF: renamed from USNSW; value HC5FW900-S -> 22pF; footprint OffBoard -> C0603; symbol traction-r1:HC5FW900-S -> traction-r1:C; MPN HC5FW900-S -> MLCC-CLASS
- CCT1: renamed from JVEH; value TE 776231-1 (AMPSEAL 23) -> 4.7nF; footprint AMPSEAL23 -> C0603; symbol traction-r1:TE_776231-1__AMPSEAL_23_ -> traction-r1:C; MPN TE 776231-1 (AMPSEAL 23) -> MLCC-4.7nF-50V
- CCT2: renamed from RCPD0; value 10k -> 4.7nF; footprint R0603 -> C0603; symbol traction-r1:R -> traction-r1:C; MPN R0603-10k -> MLCC-4.7nF-50V
- CEXA1: renamed from REXB3; value 24k -> 4.7nF; footprint R0603 -> C0603; symbol traction-r1:R -> traction-r1:C; MPN R0603-CLASS -> MLCC-CLASS
- CEXA2: renamed from REXB4; value 24k -> 300pF; footprint R0603 -> C0603; symbol traction-r1:R -> traction-r1:C; MPN R0603-CLASS -> MLCC-CLASS
- CEXA3: renamed from REXM1; value 5.1k -> 100nF; footprint R0603 -> C0603; symbol traction-r1:R -> traction-r1:C; MPN R0603-CLASS -> MLCC-CLASS
- CEXD: renamed from REXM2; value 12k -> 4.7uF; footprint R0603 -> C0603; symbol traction-r1:R -> traction-r1:C; MPN R0603-CLASS -> MLCC-CLASS
- CFLTF: renamed from RASCP; value 10k -> 100pF; footprint R0603 -> C0603; symbol traction-r1:R -> traction-r1:C; MPN R0603-10k -> MLCC-100pF-16V
- CIGN: renamed from RFLTP2; value 5.1k -> 100nF; footprint R0603 -> C0603; symbol traction-r1:R -> traction-r1:C; MPN R0603-CLASS -> MLCC-100nF-50V
- CILK: renamed from RVM2; value 24k -> 2.2nF; footprint R0603 -> C0603; symbol traction-r1:R -> traction-r1:C; MPN R0603-24k-1% -> MLCC-2.2nF-50V
- CLAT: renamed from RILK1; value 10k -> 100nF; footprint R0603 -> C0603; symbol traction-r1:R -> traction-r1:C; MPN R0603-10k -> MLCC-100nF-16V
- CLVC1: renamed from CSB3; value 10uF -> 4.7uF; footprint C0805 -> C1206; MPN MLCC-CLASS -> MLCC-4.7uF-50V
- CLVC2: renamed from CSB4; value 10uF -> 4.7uF; footprint C0805 -> C1206; MPN MLCC-CLASS -> MLCC-4.7uF-50V
- CMA1: renamed from CMD6; value 100nF -> 1uF; footprint C0402 -> C0603; MPN MLCC-100nF-16V -> MLCC-1uF-16V
- CMA2: renamed from CMD7; footprint C0402 -> C0603; MPN MLCC-100nF-16V -> MLCC-1uF-16V
- CMD11: renamed from CYA; value 12pF -> 100nF; footprint C0603 -> C0402; MPN MLCC-12pF-50V -> MLCC-100nF-16V
- CMD12: renamed from CYB; value 12pF -> 100nF; footprint C0603 -> C0402; MPN MLCC-12pF-50V -> MLCC-100nF-16V
- CMD2: renamed from RMRST; value 10k -> 100nF; footprint R0603 -> C0402; symbol traction-r1:R -> traction-r1:C; MPN R0603-10k -> MLCC-100nF-16V
- CMD3: renamed from Y1; value CX3225GA40000D0PTVCC -> 100nF; footprint X3225 -> C0402; symbol traction-r1:Y -> traction-r1:C; LCSC C6009848 -> CLASS; MPN CX3225GA40000D0PTVCC -> MLCC-100nF-16V
- CMD4: renamed from JSWD; value HDR2X10-JTAG -> 100nF; footprint HDR2x10 -> C0402; symbol traction-r1:HDR2X10-JTAG -> traction-r1:C; MPN HDR2X10-JTAG -> MLCC-100nF-16V
- CMD5: renamed from CRST; value 100pF -> 100nF; footprint C0603 -> C0402; MPN MLCC-100pF-16V -> MLCC-100nF-16V
- CMD6: renamed from RBOOT; value 10k -> 100nF; footprint R0603 -> C0402; symbol traction-r1:R -> traction-r1:C; MPN R0603-10k -> MLCC-100nF-16V
- CMD7: renamed from CLVC1; value 4.7uF -> 100nF; footprint C1206 -> C0402; MPN MLCC-4.7uF-50V -> MLCC-100nF-16V
- CMD8: renamed from CLVC2; value 4.7uF -> 100nF; footprint C1206 -> C0402; MPN MLCC-4.7uF-50V -> MLCC-100nF-16V
- CMD9: renamed from DREVC; value STPS5L60S -> 100nF; footprint SMC -> C0402; symbol traction-r1:D -> traction-r1:C; LCSC C140620 -> CLASS; MPN STPS5L60S -> MLCC-100nF-16V
- CMT1F: renamed from UCAN1; value TCAN1042HGVDRQ1 -> 47nF; footprint SOIC8 -> C0603; symbol traction-r1:TCAN1042HGVDRQ1 -> traction-r1:C; LCSC C132550 -> CLASS; MPN TCAN1042HGVDRQ1 -> MLCC-47nF-25V
- CMT2F: renamed from CCAN1; value 1uF -> 47nF; MPN MLCC-1uF-25V -> MLCC-47nF-25V
- CRST: renamed from CSB1; value 10uF -> 100pF; footprint C0805 -> C0603; MPN MLCC-CLASS -> MLCC-100pF-16V
- CSB1: renamed from LSBC; value IND-10uH-2A -> 10uF; footprint IND6x6 -> C0805; symbol traction-r1:L -> traction-r1:C; MPN IND-10uH-2A -> MLCC-CLASS
- CSB2: renamed from RAGT; value 0R -> 10uF; footprint R0603 -> C0805; symbol traction-r1:R -> traction-r1:C; MPN R0603-CLASS -> MLCC-CLASS
- CSB3: renamed from RSB1; value 52.3k -> 10uF; footprint R0603 -> C0805; symbol traction-r1:R -> traction-r1:C; MPN R0603-CLASS -> MLCC-CLASS
- CSB4: renamed from RSB2; value 10k -> 10uF; footprint R0603 -> C0805; symbol traction-r1:R -> traction-r1:C; MPN R0603-CLASS -> MLCC-CLASS
- CSB5: renamed from RSB3; value 220R -> 1uF; footprint R0603 -> C0805; symbol traction-r1:R -> traction-r1:C; MPN R0603-CLASS -> MLCC-CLASS
- CSB6: renamed from RSB4; value 5.1k -> 1uF; footprint R0603 -> C0805; symbol traction-r1:R -> traction-r1:C; MPN R0603-CLASS -> MLCC-CLASS
- CSB7: renamed from CIGN; value 100nF -> 10uF; footprint C0603 -> C0805; MPN MLCC-100nF-50V -> MLCC-CLASS
- CSB8: renamed from DIGN; value 1N4148WS -> 10uF; footprint SOD323 -> C0805; symbol traction-r1:D -> traction-r1:C; LCSC C2128 -> CLASS; MPN 1N4148WS -> MLCC-CLASS
- CSINA1: renamed from DCOSP; value PESD5V0L1BA -> 100pF; footprint SOD323 -> C0603; symbol traction-r1:PESD5V0L1BA -> traction-r1:C; MPN PESD5V0L1BA -> MLCC-CLASS
- CSINA2: renamed from CCOSA1; value 100pF -> 2.2nF
- CSIND: renamed from CCOSA2; value 2.2nF -> 220pF
- CSINF: renamed from CCOSD; value 220pF -> 22pF
- CSNUF: renamed from JTHS; value NTC-10k-0603 -> 47nF; footprint R0603 -> C0603; symbol traction-r1:J2 -> traction-r1:C; MPN NTC-10k-0603 -> MLCC-47nF-25V
- CSNVF: renamed from RTAMBP; value 10k -> 47nF; footprint R0603 -> C0603; symbol traction-r1:R -> traction-r1:C; MPN R0603-10k-1% -> MLCC-47nF-25V
- CSNWF: renamed from RTHSP; value 10k -> 47nF; footprint R0603 -> C0603; symbol traction-r1:R -> traction-r1:C; MPN R0603-10k-1% -> MLCC-47nF-25V
- CVD1: renamed from RVD2D; value 10k -> 100pF; footprint R0603 -> C0603; symbol traction-r1:R -> traction-r1:C; MPN R0603-10k-0.1% -> MLCC-CLASS
- CVD2: renamed from RSNWP; value 5.1k -> 100pF; footprint R0603 -> C0603; symbol traction-r1:R -> traction-r1:C; MPN R0603-4k99 -> MLCC-CLASS
- CVM1: renamed from CEXA3; value 100nF -> 220nF
- CVM2: renamed from CEXD; value 4.7uF -> 220nF
- CWB1: renamed from RVD1A; value 10k -> 3.3nF; footprint R0603 -> C0603; symbol traction-r1:R -> traction-r1:C; MPN R0603-10k-0.1% -> MLCC-3.3nF-50V
- CWB2: renamed from RVD1B; value 10k -> 100nF; footprint R0603 -> C0603; symbol traction-r1:R -> traction-r1:C; MPN R0603-10k-0.1% -> MLCC-3.3nF-50V
- CWS1: renamed from RVD1C; value 10k -> 47nF; footprint R0603 -> C0603; symbol traction-r1:R -> traction-r1:C; MPN R0603-10k-0.1% -> MLCC-47nF-25V
- CWS2: renamed from RVD1D; value 10k -> 4.7nF; footprint R0603 -> C0603; symbol traction-r1:R -> traction-r1:C; MPN R0603-10k-0.1% -> MLCC-47nF-25V
- CYA: renamed from DTVSC; value TPSMC24CA -> 12pF; footprint SMC -> C0603; symbol traction-r1:D -> traction-r1:C; LCSC C1975284 -> CLASS; MPN TPSMC24CA -> MLCC-12pF-50V
- CYB: renamed from FLVC; value MF-LSMF300/24X-2 -> 12pF; footprint PTC2920 -> C0603; symbol traction-r1:F -> traction-r1:C; LCSC C719172 -> CLASS; MPN MF-LSMF300/24X-2 -> MLCC-12pF-50V
- DBAT: renamed from RIGN1; value 5.1k -> BAT46ZFILM; footprint R0603 -> SOD123; symbol traction-r1:R -> traction-r1:D; LCSC CLASS -> C283255; MPN R0603-5k1 -> BAT46ZFILM
- DCOSP: renamed from RCOSR2; value 120R -> PESD5V0L1BA; footprint R0603 -> SOD323; symbol traction-r1:R -> traction-r1:PESD5V0L1BA; MPN R0603-120R -> PESD5V0L1BA
- DIGN: renamed from RGPD; value 10k -> 1N4148WS; footprint R0603 -> SOD323; symbol traction-r1:R -> traction-r1:D; LCSC CLASS -> C2128; MPN R0603-10k -> 1N4148WS
- DMT1: renamed from RMT2P; value 10k -> PESD5V0U1UA; footprint R0603 -> SOD323; symbol traction-r1:R -> traction-r1:PESD5V0U1UA; MPN R0603-CLASS -> PESD5V0U1UA
- DMT2: renamed from RMT2S; value 1k -> PESD5V0U1UA; footprint R0603 -> SOD323; symbol traction-r1:R -> traction-r1:PESD5V0U1UA; MPN R0603-CLASS -> PESD5V0U1UA
- DREVC: renamed from CSB5; value 1uF -> STPS5L60S; footprint C0805 -> SMC; symbol traction-r1:C -> traction-r1:D; LCSC CLASS -> C140620; MPN MLCC-CLASS -> STPS5L60S
- DSINP: renamed from RSINR2; value 120R -> PESD5V0L1BA; footprint R0603 -> SOD323; symbol traction-r1:R -> traction-r1:PESD5V0L1BA; MPN R0603-120R -> PESD5V0L1BA
- DTVSC: renamed from CSB6; value 1uF -> TPSMC24CA; footprint C0805 -> SMC; symbol traction-r1:C -> traction-r1:D; LCSC CLASS -> C1975284; MPN MLCC-CLASS -> TPSMC24CA
- FLVC: renamed from CSB7; value 10uF -> MF-LSMF300/24X-2; footprint C0805 -> PTC2920; symbol traction-r1:C -> traction-r1:F; LCSC CLASS -> C719172; MPN MLCC-CLASS -> MF-LSMF300/24X-2
- FMT1: renamed from CCT1; value 4.7nF -> FUSE-350mA-0603; footprint C0603 -> F0603; symbol traction-r1:C -> traction-r1:F; MPN MLCC-4.7nF-50V -> FUSE-350mA-0603
- FMT2: renamed from RCT1A; value 60.4R -> FUSE-350mA-0603; footprint R0603 -> F0603; symbol traction-r1:R -> traction-r1:F; MPN R0603-60R4-1% -> FUSE-350mA-0603
- JLEM: renamed from LUB; value FB-220R-1A -> T2M-105-01-L-D-TH-WT; footprint FB0805 -> HDR2x5; symbol traction-r1:L -> traction-r1:T2M-105-01-L-D-TH-WT; MPN FB-220R-1A -> T2M-105-01-L-D-TH-WT
- JSWD: renamed from USBC; value FS2633D -> HDR2X10-JTAG; footprint HLQFP48 -> HDR2x10; symbol traction-r1:FS2633D -> traction-r1:HDR2X10-JTAG; MPN FS2633D -> HDR2X10-JTAG
- JTAMB: renamed from FMT1; value FUSE-350mA-0603 -> NTC-10k-0603; footprint F0603 -> R0603; symbol traction-r1:F -> traction-r1:J2; MPN FUSE-350mA-0603 -> NTC-10k-0603
- JTHS: renamed from FMT2; value FUSE-350mA-0603 -> NTC-10k-0603; footprint F0603 -> R0603; symbol traction-r1:F -> traction-r1:J2; MPN FUSE-350mA-0603 -> NTC-10k-0603
- JVEH: renamed from RCPD3; value 10k -> TE 776231-1 (AMPSEAL 23); footprint R0603 -> AMPSEAL23; symbol traction-r1:R -> traction-r1:TE_776231-1__AMPSEAL_23_; MPN R0603-10k -> TE 776231-1 (AMPSEAL 23)
- LCAN1: renamed from CCAN2; value 1uF -> ACT45B-101-2P-TL003; footprint C0603 -> CMC1210; symbol traction-r1:C -> traction-r1:ACT45B-101-2P-TL003; MPN MLCC-1uF-25V -> ACT45B-101-2P-TL003
- LCAN2: renamed from LVS2; value FB-470R -> ACT45B-101-2P-TL003; footprint FB0603 -> CMC1210; symbol traction-r1:L -> traction-r1:ACT45B-101-2P-TL003; MPN FB-470R-CLASS -> ACT45B-101-2P-TL003
- LCOR: renamed from RIGN2; value 10k -> IND-4.7uH-2A; footprint R0603 -> IND5x5; symbol traction-r1:R -> traction-r1:L; MPN R0603-5k1 -> IND-4.7uH-2A
- LFC: renamed from CSB8; value 10uF -> FB-120R-3A; footprint C0805 -> FB1206; symbol traction-r1:C -> traction-r1:L; MPN MLCC-CLASS -> FB-120R-3A
- renumbered CMD8 to CMD1, CMD9 to CMD10, CMT1F to CTAMBF, CMT2F to CTHSF, CVB1 to CUB1, CVB2 to CUB2, CVS1 to CUS1, CVS2 to CUS2, CWB1 to CVB1, CWB2 to CVB2, CWS1 to CVS1, CWS2 to CVS2, LVB to LUB, LWB to LVB, RILK2 to RASCP, RLAT1 to RGPD, RFLTP1 to RSB4, RCOS1 to RSIN2, RCOSF1 to RSINF2, RCOSR1 to RSINR2, RVB1 to RUB1, RVB2 to RUB2, RVB3 to RUB3, RWB1 to RVB1, RWB2 to RVB2, RWB3 to RVB3, UVB1 to UUB1, UVB2 to UUB2, UWB1 to UVB1, UWB2 to UVB2, UVD1 to UWB1
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Other:
- note added: "220 kW pk Control card (LV) - 4 of 4"
- note added: "named connector/stud/tab (see INTERBOARD LINKS, design basis)"
- note added: "same name on another sheet = same net, joined ONLY at the"
- note removed: "220 kW pk Control card (LV) - 3 of 3"
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