File: kicad5/traction/traction-card.sch (KiCad schematic (older format))
At the start: 219 parts, among them Y1 CX3225GA40000D0PTVCC

Commit message: Rev A.4: answer external design review — 10 confirmed defects fixed (F37-F46)
Every claim verified against primary datasheets before any edit; three
claims rebutted with evidence (850V/0.1% divider corner, GEN3-exact
resolver monitors, discharge math matches). Fixed:

- F37 VGT12EEM secondary phasing: rectifier moved to pin 8 (dot); the
  drawn wiring was forward-mode ~35V into +22V-abs gates. Pins 6/7 NC'd
  (no internal winding). Aux (NF) was already correct.
- F38 flyback drain clamp: SMBJ85A (forward every OFF interval, 94.4V
  min breakdown vs 80V FET) -> US1M + SMAJ13A winding clamp; drain
  <=60V at clamped load dump
- F39 DESAT clamp: BAT64-04 series pair correctly oriented DESAT->VCC2
  (was VCC2 injected into DESAT via a wrong common-cathode symbol)
- F40 ASC latch: real SN74LVC1G74 DCU pins; 1k/10k network (was
  120R/120R = 2.5V "low" and 42mA MCU clear)
- F41 KL15: 47k/10k+100nF ADC sense (was raw 13.3V into PTA25)
- F42 VDC receivers offset +0.5V (buffered) - AMC1311 fail-safe now
  distinguishable from a dead bus
- F44 VBAT_H/L actually sourced (FVBH/FVBL polyfuses off NRC)
- F45 real package pins everywhere: 74LVC1G11 (had NO VCC pin), 1G32,
  NCV4276C (OUT=5), TPS55340 RTE16 (+SS cap +FREQ R), BUK9Y14 LFPAK56,
  ALM2402 PWP14 (+VCC_O, SHDN via 10k pullup), QA01C SIP-7, PESD as
  real 2/3-terminal parts, FS26 full LQFP-48+EP with VDIG/VBOS/
  bootstraps/DEBUG strap and DS unused-pin terminations; S32K396
  explicitly symbolic (no package table in DS - bind at layout)
- F46 hardware fault latch: FLT_HS/LS diode-OR -> LVC1G74 -> DRV_EN;
  any DESAT latches all six channels off until MCU clears
- NSI6611ASC-Q1SWR full ordering code (ASC variant)

erc-audit gains a rev-A.4 lock-in section (763 checks, 0 fail);
design-verify adds F37-F46 corner rows (60 PASS/3 WARN/0 FAIL);
pin-verify 1663/1663; card void gate 9->12% (49-pin FS26 monolith);
BOM Rs.70,059 @1k, 579 components, 180 lines. design-basis 11a
documents the full review response including the rege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
Parts:
- removed CMA1: 1uF, C0603, symbol traction-r1:C
- removed CMA2: 100nF, C0603, symbol traction-r1:C
- removed CMD1, CMD10, CMD11, CMD12, CMD2, CMD3, CMD4, CMD5: 100nF, C0402, symbol traction-r1:C
- removed UMCU: S32K396, BGA289, symbol traction-r1:S32K396
- added CCAN1, CCAN2: 1uF, C0603, symbol traction-r1:C
- added CCT1, CCT2: 4.7nF, C0603, symbol traction-r1:C
- added CMT1F, CMT2F: 47nF, C0603, symbol traction-r1:C
- added FMT1, FMT2: FUSE-350mA-0603, F0603, symbol traction-r1:F
- added FVS1: MF-LSMF, PTC1206, symbol traction-r1:F
- added JICC: MICROFIT3-40, MicroFit40, symbol traction-r1:MICROFIT3-40
- added JVEH: TE 776231-1 (AMPSEAL 23), AMPSEAL23, symbol traction-r1:TE_776231-1__AMPSEAL_23_
- added LCAN1, LCAN2: ACT45B-101-2P-TL003, CMC1210, symbol traction-r1:ACT45B-101-2P-TL003
- added LVS1, LVS2, LVS3, LVS4: FB-470R, FB0603, symbol traction-r1:L
- added RCPD0, RCPD1, RCPD2, RCPD3, RMT1P, RMT2P: 10k, R0603, symbol traction-r1:R
- added RCT1A, RCT1B, RCT2A, RCT2B: 60.4R, R0603, symbol traction-r1:R
- added RMT1S, RMT2S: 1k, R0603, symbol traction-r1:R
- added TVSC1, TVSC2: PESD2IVN24-T, SOT23, symbol traction-r1:PESD2IVN24-T
- added TVSM1, TVSM2: PESD5V0L1BA, SOD323, symbol traction-r1:R
- added UCAN1, UCAN2: TCAN1042HGVDRQ1, SOIC8, symbol traction-r1:TCAN1042HGVDRQ1
- added UMT2: OPA333AQDBVRQ1, SOT23-5, symbol traction-r1:OPA333AQDBVRQ1
- CAND1: renamed from RILK4; value 10k -> 100nF; footprint R0603 -> C0603; symbol traction-r1:R -> traction-r1:C; MPN R0603-10k -> MLCC-CLASS
- CAND2: renamed from UVMB1; value OPA348AQDBVRQ1 -> 100nF; footprint SOT23-5 -> C0603; symbol traction-r1:OPA348AQDBVRQ1 -> traction-r1:C; LCSC C2877787 -> CLASS; MPN OPA348AQDBVRQ1 -> MLCC-CLASS
- CBTC: renamed from RSB2; value 10k -> 100nF; footprint R0603 -> C0603; symbol traction-r1:R -> traction-r1:C; MPN R0603-CLASS -> MLCC-CLASS
- CBTP: renamed from RSB3; value 220R -> 100nF; footprint R0603 -> C0603; symbol traction-r1:R -> traction-r1:C; MPN R0603-CLASS -> MLCC-CLASS
- CCOSA1: renamed from RVB2; value 100R -> 100pF; footprint R0603 -> C0603; symbol traction-r1:R -> traction-r1:C; MPN R0603-100R -> MLCC-CLASS
- CCOSA2: renamed from RVB3; value 100R -> 2.2nF; footprint R0603 -> C0603; symbol traction-r1:R -> traction-r1:C; MPN R0603-100R -> MLCC-CLASS
- CCOSD: renamed from UWB1; value OPA376AQDBVRQ1 -> 220pF; footprint SOT23-5 -> C0603; symbol traction-r1:OPA376AQDBVRQ1 -> traction-r1:C; MPN OPA376AQDBVRQ1 -> MLCC-CLASS
- CCOSF: renamed from UWB2; value OPA376AQDBVRQ1 -> 22pF; footprint SOT23-5 -> C0603; symbol traction-r1:OPA376AQDBVRQ1 -> traction-r1:C; MPN OPA376AQDBVRQ1 -> MLCC-CLASS
- CEXA1: renamed from CCOSF; value 22pF -> 4.7nF
- CEXA2: renamed from RCOS1; value 680R -> 300pF; footprint R0603 -> C0603; symbol traction-r1:R -> traction-r1:C; MPN R0603-CLASS -> MLCC-CLASS
- CEXA3: renamed from RCOS2; value 680R -> 100nF; footprint R0603 -> C0603; symbol traction-r1:R -> traction-r1:C; MPN R0603-CLASS -> MLCC-CLASS
- CEXD: renamed from RCOSF1; value 330R -> 4.7uF; footprint R0603 -> C0603; symbol traction-r1:R -> traction-r1:C; MPN R0603-CLASS -> MLCC-CLASS
- CFLTF: renamed from UVMB2; value OPA348AQDBVRQ1 -> 100pF; footprint SOT23-5 -> C0603; symbol traction-r1:OPA348AQDBVRQ1 -> traction-r1:C; LCSC C2877787 -> CLASS; MPN OPA348AQDBVRQ1 -> MLCC-100pF-16V
- CIGN: renamed from RFS2; value 120R -> 100nF; footprint R0603 -> C0603; symbol traction-r1:R -> traction-r1:C; MPN R0603-120R -> MLCC-100nF-50V
- CIGNS: renamed from RFS3; value 120R -> 100nF; footprint R0603 -> C0603; symbol traction-r1:R -> traction-r1:C; MPN R0603-120R -> MLCC-CLASS
- CILK: renamed from DSINP; value PESD5V0L1BA -> 2.2nF; footprint SOD323 -> C0603; symbol traction-r1:PESD5V0L1BA -> traction-r1:C; MPN PESD5V0L1BA -> MLCC-2.2nF-50V
- CLAT: renamed from REXA2; value 10k -> 100nF; footprint R0603 -> C0603; symbol traction-r1:R -> traction-r1:C; MPN R0603-CLASS -> MLCC-100nF-16V
- CLAT2: renamed from CVM1; value 220nF -> 100nF
- CLVC1: renamed from CSB4; value 10uF -> 4.7uF; footprint C0805 -> C1206; MPN MLCC-CLASS -> MLCC-4.7uF-50V
- CLVC2: renamed from CSB5; value 1uF -> 4.7uF; footprint C0805 -> C1206; MPN MLCC-CLASS -> MLCC-4.7uF-50V
- CMA1: renamed from CMD7; value 100nF -> 1uF; footprint C0402 -> C0603; MPN MLCC-100nF-16V -> MLCC-1uF-16V
- CMA2: renamed from CMD8; footprint C0402 -> C0603; MPN MLCC-100nF-16V -> MLCC-1uF-16V
- CMD10: renamed from CYA; value 12pF -> 100nF; footprint C0603 -> C0402; MPN MLCC-12pF-50V -> MLCC-100nF-16V
- CMD11: renamed from CYB; value 12pF -> 100nF; footprint C0603 -> C0402; MPN MLCC-12pF-50V -> MLCC-100nF-16V
- CMD12: renamed from RMRST; value 10k -> 100nF; footprint R0603 -> C0402; symbol traction-r1:R -> traction-r1:C; MPN R0603-10k -> MLCC-100nF-16V
- CMD2: renamed from Y1; value CX3225GA40000D0PTVCC -> 100nF; footprint X3225 -> C0402; symbol traction-r1:Y -> traction-r1:C; LCSC C6009848 -> CLASS; MPN CX3225GA40000D0PTVCC -> MLCC-100nF-16V
- CMD3: renamed from JSWD; value HDR2X10-JTAG -> 100nF; footprint HDR2x10 -> C0402; symbol traction-r1:HDR2X10-JTAG -> traction-r1:C; MPN HDR2X10-JTAG -> MLCC-100nF-16V
- CMD4: renamed from CRST; value 100pF -> 100nF; footprint C0603 -> C0402; MPN MLCC-100pF-16V -> MLCC-100nF-16V
- CMD5: renamed from RBOOT; value 10k -> 100nF; footprint R0603 -> C0402; symbol traction-r1:R -> traction-r1:C; MPN R0603-10k -> MLCC-100nF-16V
- CMD6: renamed from CLVC1; value 4.7uF -> 100nF; footprint C1206 -> C0402; MPN MLCC-4.7uF-50V -> MLCC-100nF-16V
- CMD7: renamed from CLVC2; value 4.7uF -> 100nF; footprint C1206 -> C0402; MPN MLCC-4.7uF-50V -> MLCC-100nF-16V
- CMD8: renamed from DREVC; value STPS5L60S -> 100nF; footprint SMC -> C0402; symbol traction-r1:D -> traction-r1:C; LCSC C140620 -> CLASS; MPN STPS5L60S -> MLCC-100nF-16V
- CMD9: renamed from DTVSC; value TPSMC24CA -> 100nF; footprint SMC -> C0402; symbol traction-r1:D -> traction-r1:C; LCSC C1975284 -> CLASS; MPN TPSMC24CA -> MLCC-100nF-16V
- COF1: renamed from RMT1S; value 1k -> 100nF; footprint R0603 -> C0603; symbol traction-r1:R -> traction-r1:C; MPN R0603-CLASS -> MLCC-CLASS
- COR1: renamed from REXM3; value 5.1k -> 100nF; footprint R0603 -> C0603; symbol traction-r1:R -> traction-r1:C; MPN R0603-CLASS -> MLCC-CLASS
- COR2: renamed from REXM4; value 24k -> 100nF; footprint R0603 -> C0603; symbol traction-r1:R -> traction-r1:C; MPN R0603-CLASS -> MLCC-CLASS
- CRST: renamed from CSB2; value 10uF -> 100pF; footprint C0805 -> C0603; MPN MLCC-CLASS -> MLCC-100pF-16V
- CSB1: renamed from RSB4; value 5.1k -> 10uF; footprint R0603 -> C0805; symbol traction-r1:R -> traction-r1:C; MPN R0603-CLASS -> MLCC-CLASS
- CSB2: renamed from CIGN; value 100nF -> 10uF; footprint C0603 -> C0805; MPN MLCC-100nF-50V -> MLCC-CLASS
- CSB3: renamed from DIGN; value 1N4148WS -> 10uF; footprint SOD323 -> C0805; symbol traction-r1:D -> traction-r1:C; LCSC C2128 -> CLASS; MPN 1N4148WS -> MLCC-CLASS
- CSB4: renamed from RIGN1; value 5.1k -> 10uF; footprint R0603 -> C0805; symbol traction-r1:R -> traction-r1:C; MPN R0603-5k1 -> MLCC-CLASS
- CSB5: renamed from RIGN2; value 10k -> 1uF; footprint R0603 -> C0805; symbol traction-r1:R -> traction-r1:C; MPN R0603-5k1 -> MLCC-CLASS
- CSB6: renamed from UAND1; value 74LVC1G11GW-Q100 -> 1uF; footprint SOT363 -> C0805; symbol traction-r1:74LVC1G11GW-Q100 -> traction-r1:C; LCSC C548242 -> CLASS; MPN 74LVC1G11GW-Q100 -> MLCC-CLASS
- CSB7: renamed from UAND2; value 74LVC1G11GW-Q100 -> 10uF; footprint SOT363 -> C0805; symbol traction-r1:74LVC1G11GW-Q100 -> traction-r1:C; LCSC C548242 -> CLASS; MPN 74LVC1G11GW-Q100 -> MLCC-CLASS
- CSB8: renamed from CFLTF; value 100pF -> 10uF; footprint C0603 -> C0805; MPN MLCC-100pF-16V -> MLCC-CLASS
- CSINA1: renamed from RUB1; value 100R -> 100pF; footprint R0603 -> C0603; symbol traction-r1:R -> traction-r1:C; MPN R0603-100R -> MLCC-CLASS
- CSINA2: renamed from RUB2; value 100R -> 2.2nF; footprint R0603 -> C0603; symbol traction-r1:R -> traction-r1:C; MPN R0603-100R -> MLCC-CLASS
- CSIND: renamed from RUB3; value 100R -> 220pF; footprint R0603 -> C0603; symbol traction-r1:R -> traction-r1:C; MPN R0603-100R -> MLCC-CLASS
- CSINF: renamed from UVB1; value OPA376AQDBVRQ1 -> 22pF; footprint SOT23-5 -> C0603; symbol traction-r1:OPA376AQDBVRQ1 -> traction-r1:C; MPN OPA376AQDBVRQ1 -> MLCC-CLASS
- CSNUF: renamed from CCT2; value 4.7nF -> 47nF; MPN MLCC-4.7nF-50V -> MLCC-47nF-25V
- CSNVF: renamed from RCT2A; value 60.4R -> 47nF; footprint R0603 -> C0603; symbol traction-r1:R -> traction-r1:C; MPN R0603-60R4-1% -> MLCC-47nF-25V
- CSNWF: renamed from RCT2B; value 60.4R -> 47nF; footprint R0603 -> C0603; symbol traction-r1:R -> traction-r1:C; MPN R0603-60R4-1% -> MLCC-47nF-25V
- CTAMBF: renamed from LVS3; value FB-470R -> 47nF; footprint FB0603 -> C0603; symbol traction-r1:L -> traction-r1:C; MPN FB-470R-CLASS -> MLCC-47nF-25V
- CTHSF: renamed from LVS4; value FB-470R -> 47nF; footprint FB0603 -> C0603; symbol traction-r1:L -> traction-r1:C; MPN FB-470R-CLASS -> MLCC-47nF-25V
- CUB1: renamed from RVD1C; value 10k -> 3.3nF; footprint R0603 -> C0603; symbol traction-r1:R -> traction-r1:C; MPN R0603-10k-0.1% -> MLCC-3.3nF-50V
- CUB2: renamed from RVD1D; value 10k -> 100nF; footprint R0603 -> C0603; symbol traction-r1:R -> traction-r1:C; MPN R0603-10k-0.1% -> MLCC-3.3nF-50V
- CUS1: renamed from UVD2; value OPA376AQDBVRQ1 -> 47nF; footprint SOT23-5 -> C0603; symbol traction-r1:OPA376AQDBVRQ1 -> traction-r1:C; MPN OPA376AQDBVRQ1 -> MLCC-47nF-25V
- CUS2: renamed from CVD2; value 100pF -> 4.7nF; MPN MLCC-CLASS -> MLCC-47nF-25V
- CVB1: renamed from CSNWF; value 47nF -> 3.3nF; MPN MLCC-47nF-25V -> MLCC-3.3nF-50V
- CVB2: renamed from RSNUP; value 5.1k -> 100nF; footprint R0603 -> C0603; symbol traction-r1:R -> traction-r1:C; MPN R0603-4k99 -> MLCC-3.3nF-50V
- CVBOS: renamed from RENP1; value 1k -> 1uF; footprint R0603 -> C0603; symbol traction-r1:R -> traction-r1:C; MPN R0603-1k -> MLCC-CLASS
- CVD1: renamed from RMT2P; value 10k -> 100pF; footprint R0603 -> C0603; symbol traction-r1:R -> traction-r1:C; MPN R0603-CLASS -> MLCC-CLASS
- CVD2: renamed from RCT1B; value 60.4R -> 100pF; footprint R0603 -> C0603; symbol traction-r1:R -> traction-r1:C; MPN R0603-60R4-1% -> MLCC-CLASS
- CVDIG: renamed from RENP2; value 1k -> 1uF; footprint R0603 -> C0603; symbol traction-r1:R -> traction-r1:C; MPN R0603-1k -> MLCC-CLASS
- CVM1: renamed from RSINF1; value 330R -> 220nF; footprint R0603 -> C0603; symbol traction-r1:R -> traction-r1:C; MPN R0603-CLASS -> MLCC-CLASS
- CVM2: renamed from RSINF2; value 330R -> 220nF; footprint R0603 -> C0603; symbol traction-r1:R -> traction-r1:C; MPN R0603-CLASS -> MLCC-CLASS
- CVS1: renamed from RSNVP; value 5.1k -> 47nF; footprint R0603 -> C0603; symbol traction-r1:R -> traction-r1:C; MPN R0603-4k99 -> MLCC-47nF-25V
- CVS2: renamed from RSNWP; value 5.1k -> 4.7nF; footprint R0603 -> C0603; symbol traction-r1:R -> traction-r1:C; MPN R0603-4k99 -> MLCC-47nF-25V
- CWB1: renamed from RTHSP; value 10k -> 3.3nF; footprint R0603 -> C0603; symbol traction-r1:R -> traction-r1:C; MPN R0603-10k-1% -> MLCC-3.3nF-50V
- CWB2: renamed from DMT1; value PESD5V0U1UA -> 100nF; footprint SOD323 -> C0603; symbol traction-r1:PESD5V0U1UA -> traction-r1:C; MPN PESD5V0U1UA -> MLCC-3.3nF-50V
- CWS1: renamed from DMT2; value PESD5V0U1UA -> 47nF; footprint SOD323 -> C0603; symbol traction-r1:PESD5V0U1UA -> traction-r1:C; MPN PESD5V0U1UA -> MLCC-47nF-25V
- CWS2: renamed from UMT1; value OPA333AQDBVRQ1 -> 4.7nF; footprint SOT23-5 -> C0603; symbol traction-r1:OPA333AQDBVRQ1 -> traction-r1:C; LCSC C2058544 -> CLASS; MPN OPA333AQDBVRQ1 -> MLCC-47nF-25V
- CYA: renamed from FLVC; value MF-LSMF300/24X-2 -> 12pF; footprint PTC2920 -> C0603; symbol traction-r1:F -> traction-r1:C; LCSC C719172 -> CLASS; MPN MF-LSMF300/24X-2 -> MLCC-12pF-50V
- renumbered CMD9 to CMD1
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Connections:
- net labels added: ASC_CLR_M, CORBT, EXSD, FLT_CLR_N, FLT_CMB_N, FLT_OK, IGN_D, PREBT, SBC_DBG, VBOS, VDIG, VOFD, VOFS
- net labels removed: PGOOD
- wire segments 701 -> 776
- no-connect marks 0 -> 2
Other:
- note added: "rev A.4 - 26 sections - 244 components"
- note removed: "rev A.3 - 26 sections - 219 components"
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
Commit message: Rev A.4.1: second review round — 5 confirmed defects fixed (F47-F51)
- F47 AMC1311 real pins 2=IN/3=SHTDN (both VDC channels had them
  swapped: analog inputs grounded, SHTDN on the divider tap)
- F48 FS26 TRKIN is the VREF regulator's input supply -> VPRE
  (was grounded as an "unused tracker input"; VREF5 had no source)
- F49 TPS55340 pin 5 is SYNC (7V abs), not a second VIN -> DGND
- F50 FS26 caps to DS minimums: CVBOS 4.7uF, CSB6 4.7uF, CSB5 2.2uF
  (VREF COUT 1.1-3.3uF eff - third value found in the same audit)
- F51 V15 protective post-regulator NCV4276C-ADJ 40V/0.4A: boost
  pass-through (24V jump start / ~33V clamped load dump) can no longer
  reach the QA01C 13.5-16.5V window; boost output renamed V15B
- ASC/fault-latch interplay documented per NSI6611 DS (ASC overrides
  input side; DESAT + VCC2-UVLO outrank ASC)
- all five PDFs regenerate from one release (stale standalone A.3
  exports superseded); ERC gains A.4.1 assertions

Gates: 1674/1674 pins, ERC 769/0, design-verify 64P/3W/0F,
BOM Rs.70,074 @1k, 583 components, 184 lines.

Co-Authored-By: Claude Fable 5 <noreply@anthropic.com>
Parts:
- removed CMA1: 1uF, C0603, symbol traction-r1:C
- removed CMA2: 100nF, C0603, symbol traction-r1:C
- removed CMD1: 100nF, C0402, symbol traction-r1:C
- removed UMCU: S32K396, BGA289, symbol traction-r1:S32K396
- added RCPD0, RCPD1, RCPD2, RCPD3: 10k, R0603, symbol traction-r1:R
- CAND1: renamed from DFLT1; value 1N4148WS -> 100nF; footprint SOD323 -> C0603; symbol traction-r1:D -> traction-r1:C; LCSC C2128 -> CLASS; MPN 1N4148WS -> MLCC-CLASS
- CAND2: renamed from DFLT2; value 1N4148WS -> 100nF; footprint SOD323 -> C0603; symbol traction-r1:D -> traction-r1:C; LCSC C2128 -> CLASS; MPN 1N4148WS -> MLCC-CLASS
- CBTC: renamed from CSB3; value 10uF -> 100nF; footprint C0805 -> C0603
- CBTP: renamed from CSB4; value 10uF -> 100nF; footprint C0805 -> C0603
- CCAN1: renamed from LCAN2; value ACT45B-101-2P-TL003 -> 1uF; footprint CMC1210 -> C0603; symbol traction-r1:ACT45B-101-2P-TL003 -> traction-r1:C; MPN ACT45B-101-2P-TL003 -> MLCC-1uF-25V
- CCAN2: renamed from JVEH; value TE 776231-1 (AMPSEAL 23) -> 1uF; footprint AMPSEAL23 -> C0603; symbol traction-r1:TE_776231-1__AMPSEAL_23_ -> traction-r1:C; MPN TE 776231-1 (AMPSEAL 23) -> MLCC-1uF-25V
- CCOSA1: renamed from RCOS1; value 680R -> 100pF; footprint R0603 -> C0603; symbol traction-r1:R -> traction-r1:C; MPN R0603-CLASS -> MLCC-CLASS
- CCOSA2: renamed from RCOS2; value 680R -> 2.2nF; footprint R0603 -> C0603; symbol traction-r1:R -> traction-r1:C; MPN R0603-CLASS -> MLCC-CLASS
- CCOSD: renamed from RCOSF1; value 330R -> 220pF; footprint R0603 -> C0603; symbol traction-r1:R -> traction-r1:C; MPN R0603-CLASS -> MLCC-CLASS
- CCOSF: renamed from RCOSF2; value 330R -> 22pF; footprint R0603 -> C0603; symbol traction-r1:R -> traction-r1:C; MPN R0603-CLASS -> MLCC-CLASS
- CCT1: renamed from TVSC2; value PESD2IVN24-T -> 4.7nF; footprint SOT23 -> C0603; symbol traction-r1:PESD2IVN24-T -> traction-r1:C; LCSC C406047 -> CLASS; MPN PESD2IVN24-T -> MLCC-4.7nF-50V
- CCT2: renamed from FVS1; value MF-LSMF -> 4.7nF; footprint PTC1206 -> C0603; symbol traction-r1:F -> traction-r1:C; MPN MF-LSMF-CLASS -> MLCC-4.7nF-50V
- CEXA1: renamed from REXA1; value 3k -> 4.7nF; footprint R0603 -> C0603; symbol traction-r1:R -> traction-r1:C; MPN R0603-CLASS -> MLCC-CLASS
- CEXA2: renamed from REXA2; value 10k -> 300pF; footprint R0603 -> C0603; symbol traction-r1:R -> traction-r1:C; MPN R0603-CLASS -> MLCC-CLASS
- CEXA3: renamed from REXA3; value 10k -> 100nF; footprint R0603 -> C0603; symbol traction-r1:R -> traction-r1:C; MPN R0603-CLASS -> MLCC-CLASS
- CEXD: renamed from REXA4; value 24k -> 4.7uF; footprint R0603 -> C0603; symbol traction-r1:R -> traction-r1:C; MPN R0603-CLASS -> MLCC-CLASS
- CFLTF: renamed from RENP1; value 1k -> 100pF; footprint R0603 -> C0603; symbol traction-r1:R -> traction-r1:C; MPN R0603-1k -> MLCC-100pF-16V
- CIGN: renamed from RIGN2; value 10k -> 100nF; footprint R0603 -> C0603; symbol traction-r1:R -> traction-r1:C; MPN R0603-5k1 -> MLCC-100nF-50V
- CIGNS: renamed from RIGNS1; value 47k -> 100nF; footprint R0603 -> C0603; symbol traction-r1:R -> traction-r1:C; MPN R0603-CLASS -> MLCC-CLASS
- CILK: renamed from RILK4; value 10k -> 2.2nF; footprint R0603 -> C0603; symbol traction-r1:R -> traction-r1:C; MPN R0603-10k -> MLCC-2.2nF-50V
- CLAT: renamed from RFS3; value 1k -> 100nF; footprint R0603 -> C0603; symbol traction-r1:R -> traction-r1:C; MPN R0603-120R -> MLCC-100nF-16V
- CLAT2: renamed from RENP2; value 1k -> 100nF; footprint R0603 -> C0603; symbol traction-r1:R -> traction-r1:C; MPN R0603-1k -> MLCC-CLASS
- CLVC1: renamed from FLVC; value MF-LSMF300/24X-2 -> 4.7uF; footprint PTC2920 -> C1206; symbol traction-r1:F -> traction-r1:C; LCSC C719172 -> CLASS; MPN MF-LSMF300/24X-2 -> MLCC-4.7uF-50V
- CLVC2: renamed from FVBH; value MF-LSMF300/24X-2 -> 4.7uF; footprint PTC2920 -> C1206; symbol traction-r1:F -> traction-r1:C; LCSC C719172 -> CLASS; MPN MF-LSMF300/24X-2 -> MLCC-4.7uF-50V
- CMA1: renamed from CMD11; value 100nF -> 1uF; footprint C0402 -> C0603; MPN MLCC-100nF-16V -> MLCC-1uF-16V
- CMA2: renamed from CMD12; footprint C0402 -> C0603; MPN MLCC-100nF-16V -> MLCC-1uF-16V
- CMD6: renamed from CYA; value 12pF -> 100nF; footprint C0603 -> C0402; MPN MLCC-12pF-50V -> MLCC-100nF-16V
- CMD7: renamed from CYB; value 12pF -> 100nF; footprint C0603 -> C0402; MPN MLCC-12pF-50V -> MLCC-100nF-16V
- CMD8: renamed from RMRST; value 10k -> 100nF; footprint R0603 -> C0402; symbol traction-r1:R -> traction-r1:C; MPN R0603-10k -> MLCC-100nF-16V
- CMD9: renamed from Y1; value CX3225GA40000D0PTVCC -> 100nF; footprint X3225 -> C0402; symbol traction-r1:Y -> traction-r1:C; LCSC C6009848 -> CLASS; MPN CX3225GA40000D0PTVCC -> MLCC-100nF-16V
- CMT1F: renamed from RMT1P; value 10k -> 47nF; footprint R0603 -> C0603; symbol traction-r1:R -> traction-r1:C; MPN R0603-CLASS -> MLCC-47nF-25V
- CMT2F: renamed from RMT1S; value 1k -> 47nF; footprint R0603 -> C0603; symbol traction-r1:R -> traction-r1:C; MPN R0603-CLASS -> MLCC-47nF-25V
- COF1: renamed from RVD1A; value 10k -> 100nF; footprint R0603 -> C0603; symbol traction-r1:R -> traction-r1:C; MPN R0603-10k-0.1% -> MLCC-CLASS
- COR1: renamed from RILK2; value 10k -> 100nF; footprint R0603 -> C0603; symbol traction-r1:R -> traction-r1:C; MPN R0603-10k -> MLCC-CLASS
- COR2: renamed from RILK3; value 10k -> 100nF; footprint R0603 -> C0603; symbol traction-r1:R -> traction-r1:C; MPN R0603-10k -> MLCC-CLASS
- CRST: renamed from DREVC; value STPS5L60S -> 100pF; footprint SMC -> C0603; symbol traction-r1:D -> traction-r1:C; LCSC C140620 -> CLASS; MPN STPS5L60S -> MLCC-100pF-16V
- CSB1: renamed from CSB5; value 1uF -> 10uF
- CSB2: renamed from CSB6; value 1uF -> 10uF
- CSB5: renamed from CVBOS; value 1uF -> 2.2uF; footprint C0603 -> C0805
- CSB6: renamed from CVDIG; value 1uF -> 4.7uF; footprint C0603 -> C0805
- CSB7: renamed from DBAT; value BAT46ZFILM -> 10uF; footprint SOD123 -> C0805; symbol traction-r1:D -> traction-r1:C; LCSC C283255 -> CLASS; MPN BAT46ZFILM -> MLCC-CLASS
- CSB8: renamed from LCOR; value IND-4.7uH-2A -> 10uF; footprint IND5x5 -> C0805; symbol traction-r1:L -> traction-r1:C; MPN IND-4.7uH-2A -> MLCC-CLASS
- CSINA1: renamed from RSIN1; value 680R -> 100pF; footprint R0603 -> C0603; symbol traction-r1:R -> traction-r1:C; MPN R0603-CLASS -> MLCC-CLASS
- CSINA2: renamed from RSIN2; value 680R -> 2.2nF; footprint R0603 -> C0603; symbol traction-r1:R -> traction-r1:C; MPN R0603-CLASS -> MLCC-CLASS
- CSIND: renamed from RSINF1; value 330R -> 220pF; footprint R0603 -> C0603; symbol traction-r1:R -> traction-r1:C; MPN R0603-CLASS -> MLCC-CLASS
- CSINF: renamed from RSINF2; value 330R -> 22pF; footprint R0603 -> C0603; symbol traction-r1:R -> traction-r1:C; MPN R0603-CLASS -> MLCC-CLASS
- CSNUF: renamed from RSNVP; value 5.1k -> 47nF; footprint R0603 -> C0603; symbol traction-r1:R -> traction-r1:C; MPN R0603-4k99 -> MLCC-47nF-25V
- CSNVF: renamed from RSNWP; value 5.1k -> 47nF; footprint R0603 -> C0603; symbol traction-r1:R -> traction-r1:C; MPN R0603-4k99 -> MLCC-47nF-25V
- CSNWF: renamed from RTMR; value 0R -> 47nF; footprint R0603 -> C0603; symbol traction-r1:R -> traction-r1:C; MPN R0603-CLASS -> MLCC-47nF-25V
- CTAMBF: renamed from RTAMBP; value 10k -> 47nF; footprint R0603 -> C0603; symbol traction-r1:R -> traction-r1:C; MPN R0603-10k-1% -> MLCC-47nF-25V
- CTHSF: renamed from RTHSP; value 10k -> 47nF; footprint R0603 -> C0603; symbol traction-r1:R -> traction-r1:C; MPN R0603-10k-1% -> MLCC-47nF-25V
- CUB1: renamed from LUB; value FB-220R-1A -> 3.3nF; footprint FB0805 -> C0603; symbol traction-r1:L -> traction-r1:C; MPN FB-220R-1A -> MLCC-3.3nF-50V
- CUB2: renamed from RUB1; value 100R -> 100nF; footprint R0603 -> C0603; symbol traction-r1:R -> traction-r1:C; MPN R0603-100R -> MLCC-3.3nF-50V
- CUS1: renamed from RUB2; value 100R -> 47nF; footprint R0603 -> C0603; symbol traction-r1:R -> traction-r1:C; MPN R0603-100R -> MLCC-47nF-25V
- CUS2: renamed from RUB3; value 100R -> 4.7nF; footprint R0603 -> C0603; symbol traction-r1:R -> traction-r1:C; MPN R0603-100R -> MLCC-47nF-25V
- CVB1: renamed from LVB; value FB-220R-1A -> 3.3nF; footprint FB0805 -> C0603; symbol traction-r1:L -> traction-r1:C; MPN FB-220R-1A -> MLCC-3.3nF-50V
- CVB2: renamed from RVB1; value 100R -> 100nF; footprint R0603 -> C0603; symbol traction-r1:R -> traction-r1:C; MPN R0603-100R -> MLCC-3.3nF-50V
- CVBOS: renamed from LSBC; value IND-10uH-2A -> 4.7uF; footprint IND6x6 -> C0603; symbol traction-r1:L -> traction-r1:C; MPN IND-10uH-2A -> MLCC-CLASS
- CVD1: renamed from RVD1B; value 10k -> 100pF; footprint R0603 -> C0603; symbol traction-r1:R -> traction-r1:C; MPN R0603-10k-0.1% -> MLCC-CLASS
- CVD2: renamed from RVD2D; value 10k -> 100pF; footprint R0603 -> C0603; symbol traction-r1:R -> traction-r1:C; MPN R0603-10k-0.1% -> MLCC-CLASS
- CVDIG: renamed from RAGT; value 0R -> 1uF; footprint R0603 -> C0603; symbol traction-r1:R -> traction-r1:C; MPN R0603-CLASS -> MLCC-CLASS
- CVM1: renamed from RVM3; value 24k -> 220nF; footprint R0603 -> C0603; symbol traction-r1:R -> traction-r1:C; MPN R0603-24k-1% -> MLCC-CLASS
- CVM2: renamed from RVM4; value 24k -> 220nF; footprint R0603 -> C0603; symbol traction-r1:R -> traction-r1:C; MPN R0603-24k-1% -> MLCC-CLASS
- CVS1: renamed from RVB2; value 100R -> 47nF; footprint R0603 -> C0603; symbol traction-r1:R -> traction-r1:C; MPN R0603-100R -> MLCC-47nF-25V
- CVS2: renamed from RVB3; value 100R -> 4.7nF; footprint R0603 -> C0603; symbol traction-r1:R -> traction-r1:C; MPN R0603-100R -> MLCC-47nF-25V
- CWB1: renamed from LWB; value FB-220R-1A -> 3.3nF; footprint FB0805 -> C0603; symbol traction-r1:L -> traction-r1:C; MPN FB-220R-1A -> MLCC-3.3nF-50V
- CWB2: renamed from RWB1; value 100R -> 100nF; footprint R0603 -> C0603; symbol traction-r1:R -> traction-r1:C; MPN R0603-100R -> MLCC-3.3nF-50V
- CWS1: renamed from RWB2; value 100R -> 47nF; footprint R0603 -> C0603; symbol traction-r1:R -> traction-r1:C; MPN R0603-100R -> MLCC-47nF-25V
- CWS2: renamed from RWB3; value 100R -> 4.7nF; footprint R0603 -> C0603; symbol traction-r1:R -> traction-r1:C; MPN R0603-100R -> MLCC-47nF-25V
- CYA: renamed from JSWD; value HDR2X10-JTAG -> 12pF; footprint HDR2x10 -> C0603; symbol traction-r1:HDR2X10-JTAG -> traction-r1:C; MPN HDR2X10-JTAG -> MLCC-12pF-50V
- CYB: renamed from CRST; value 100pF -> 12pF; MPN MLCC-100pF-16V -> MLCC-12pF-50V
- DBAT: renamed from RDBG; value 10k -> BAT46ZFILM; footprint R0603 -> SOD123; symbol traction-r1:R -> traction-r1:D; LCSC CLASS -> C283255; MPN R0603-CLASS -> BAT46ZFILM
- DCOSP: renamed from CCOSF; value 22pF -> PESD2IVN24-T; footprint C0603 -> SOT23; symbol traction-r1:C -> traction-r1:PESD2IVN24-T; LCSC CLASS -> C406047; MPN MLCC-CLASS -> PESD2IVN24-T
- DFLT1: renamed from RFLTC; value 10k -> 1N4148WS; footprint R0603 -> SOD323; symbol traction-r1:R -> traction-r1:D; LCSC CLASS -> C2128; MPN R0603-CLASS -> 1N4148WS
- DFLT2: renamed from RFLTP1; value 5.1k -> 1N4148WS; footprint R0603 -> SOD323; symbol traction-r1:R -> traction-r1:D; LCSC CLASS -> C2128; MPN R0603-CLASS -> 1N4148WS
- DIGN: renamed from RIGNS2; value 10k -> 1N4148WS; footprint R0603 -> SOD323; symbol traction-r1:R -> traction-r1:D; LCSC CLASS -> C2128; MPN R0603-CLASS -> 1N4148WS
- DREVC: renamed from FVBL; value MF-LSMF300/24X-2 -> STPS5L60S; footprint PTC2920 -> SMC; symbol traction-r1:F -> traction-r1:D; LCSC C719172 -> C140620; MPN MF-LSMF300/24X-2 -> STPS5L60S
- DSINP: renamed from CSINF; value 22pF -> PESD2IVN24-T; footprint C0603 -> SOT23; symbol traction-r1:C -> traction-r1:PESD2IVN24-T; LCSC CLASS -> C406047; MPN MLCC-CLASS -> PESD2IVN24-T
- DTVSC: renamed from LFC; value FB-120R-3A -> TPSMC24CA; footprint FB1206 -> SMC; symbol traction-r1:L -> traction-r1:D; LCSC CLASS -> C1975284; MPN FB-120R-3A -> TPSMC24CA
- renumbered CMD2 to CMD1, CMD3 to CMD10, CMD4 to CMD11, CMD5 to CMD12, CMD6 to CMD2, CMD7 to CMD3, CMD8 to CMD4, CMD9 to CMD5, CSB7 to CSB3, CSB8 to CSB4, REXB4 to REXA4, REXM4 to REXB4, RRDYP1 to RFLTP1, RRDYP2 to RFLTP2, RBOOT to RMRST, RVD2A to RVD1C, RVD2B to RVD1D
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Other:
- note added: "rev A.4.1 - 26 sections - 244 components"
- note removed: "rev A.4 - 26 sections - 244 components"
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
Commit message: Rev A.4.2: third review round — 6 confirmed defects fixed (F52-F57)
- F52 FS26 buck passives to Table-106 selections: LCOR 2.2uH
  (CORE_LSEL_OTP=0x02; 4.7uH matched no listed value), V15S COUT
  2x22uF (~32uF eff vs 20-100 spec), CBTC 47nF, CBTP 22nF per
  CBOOT_PRE, VPRE COUT 2x22uF, CIN 22uF; effective-capacitance rows
  (bias/tol/temp derating) added to design-verify. VREF5 judged as a
  rail (CSB5+CMA1+CMA2 ~2.2uF eff, inside 1.1-3.3) per reviewer.
- F53 ACT45B CAN chokes: real windings are pins 1-4 and 2-3 (TDK
  circuit diagram) - both ports had transceiver CANH coupled onto
  external CANL; remapped, ERC asserts end-to-end pairing
- F54 ULDO15 completed: 220pF feed-forward across the 49.9k leg
  (fz 14.5kHz, onsemi 11-18kHz window), COUT 22uF
- F55 UEXD (ALM2402, 18V abs/16V rec) off raw VBATC -> behind ULDOEX
  12.1V (NCV4276C-ADJ); 24V jump start can no longer reach it
- F56 flyback switch BUK9Y14-80E (logic-level, VGS +/-10V DC) was
  outside abs-max at the 11.8V drive, masked by a 5.6V zener that
  conducted ~0.29A through every ON interval (~0.4W each). Now
  BUK7Y14-80E (standard-level +/-20V, same LFPAK56); zener repurposed
  to a dark 15V protective clamp
- F57 ordering code NCV4276CDTADJRKG (DT/ADJ were transposed)
- ASC-with-VCC1-open qualification documented (DESAT unavailable;
  double-fault given KL30-held V5GD) + IGN_SNS ADC disposition

Gates: 1691/1691 pins, ERC 779/0, design-verify 73P/3W/0F,
BOM Rs.70,090 @1k, 590 components, 192 lines.

Co-Authored-By: Claude Fable 5 <noreply@anthropic.com>
Parts:
- removed UMCU: S32K396, BGA289, symbol traction-r1:S32K396
- added JICC: MICROFIT3-40, MicroFit40, symbol traction-r1:MICROFIT3-40
- added LVS3, LVS4: FB-470R, FB0603, symbol traction-r1:L
- added RCPD0, RCPD1, RCPD2, RCPD3: 10k, R0603, symbol traction-r1:R
- CAND1: renamed from CFLTF; value 100pF -> 100nF; MPN MLCC-100pF-16V -> MLCC-CLASS
- CBTC: renamed from CBTP; value 100nF -> 47nF
- CBTP: renamed from CSB1; value 10uF -> 22nF; footprint C0805 -> C0603
- CCAN2: renamed from LVS2; value FB-470R -> 1uF; footprint FB0603 -> C0603; symbol traction-r1:L -> traction-r1:C; MPN FB-470R-CLASS -> MLCC-1uF-25V
- CCOSA1: renamed from RCOSF2; value 330R -> 100pF; footprint R0603 -> C0603; symbol traction-r1:R -> traction-r1:C; MPN R0603-CLASS -> MLCC-CLASS
- CCOSA2: renamed from RCOSR1; value 120R -> 2.2nF; footprint R0603 -> C0603; symbol traction-r1:R -> traction-r1:C; MPN R0603-120R -> MLCC-CLASS
- CCOSD: renamed from RCOSR2; value 120R -> 220pF; footprint R0603 -> C0603; symbol traction-r1:R -> traction-r1:C; MPN R0603-120R -> MLCC-CLASS
- CCOSF: renamed from JLEM; value T2M-105-01-L-D-TH-WT -> 22pF; footprint HDR2x5 -> C0603; symbol traction-r1:T2M-105-01-L-D-TH-WT -> traction-r1:C; MPN T2M-105-01-L-D-TH-WT -> MLCC-CLASS
- CCT2: renamed from LVS3; value FB-470R -> 4.7nF; footprint FB0603 -> C0603; symbol traction-r1:L -> traction-r1:C; MPN FB-470R-CLASS -> MLCC-4.7nF-50V
- CEXA1: renamed from CEXD; value 4.7uF -> 4.7nF
- CEXA2: renamed from REXA1; value 3k -> 300pF; footprint R0603 -> C0603; symbol traction-r1:R -> traction-r1:C; MPN R0603-CLASS -> MLCC-CLASS
- CEXA3: renamed from REXA2; value 10k -> 100nF; footprint R0603 -> C0603; symbol traction-r1:R -> traction-r1:C; MPN R0603-CLASS -> MLCC-CLASS
- CEXD: renamed from REXA3; value 10k -> 4.7uF; footprint R0603 -> C0603; symbol traction-r1:R -> traction-r1:C; MPN R0603-CLASS -> MLCC-CLASS
- CFLTF: renamed from DFLT1; value 1N4148WS -> 100pF; footprint SOD323 -> C0603; symbol traction-r1:D -> traction-r1:C; LCSC C2128 -> CLASS; MPN 1N4148WS -> MLCC-100pF-16V
- CIGN: renamed from DIGN; value 1N4148WS -> 100nF; footprint SOD323 -> C0603; symbol traction-r1:D -> traction-r1:C; LCSC C2128 -> CLASS; MPN 1N4148WS -> MLCC-100nF-50V
- CIGNS: renamed from RIGN1; value 5.1k -> 100nF; footprint R0603 -> C0603; symbol traction-r1:R -> traction-r1:C; MPN R0603-5k1 -> MLCC-CLASS
- CILK: renamed from RILK2; value 10k -> 2.2nF; footprint R0603 -> C0603; symbol traction-r1:R -> traction-r1:C; MPN R0603-10k -> MLCC-2.2nF-50V
- CLAT: renamed from RFS1; value 1k -> 100nF; footprint R0603 -> C0603; symbol traction-r1:R -> traction-r1:C; MPN R0603-120R -> MLCC-100nF-16V
- CLAT2: renamed from DFLT2; value 1N4148WS -> 100nF; footprint SOD323 -> C0603; symbol traction-r1:D -> traction-r1:C; LCSC C2128 -> CLASS; MPN 1N4148WS -> MLCC-CLASS
- CLDE: renamed from REXA4; value 24k -> 22uF; footprint R0603 -> C0603; symbol traction-r1:R -> traction-r1:C; MPN R0603-CLASS -> MLCC-CLASS
- CLDEC: renamed from REXB1; value 24k -> 270pF; footprint R0603 -> C0603; symbol traction-r1:R -> traction-r1:C; MPN R0603-CLASS -> MLCC-CLASS
- CLVC2: renamed from DREVC; value STPS5L60S -> 22uF; footprint SMC -> C1206; symbol traction-r1:D -> traction-r1:C; LCSC C140620 -> CLASS; MPN STPS5L60S -> MLCC-4.7uF-50V
- CMA1: renamed from CMA2; value 100nF -> 1uF
- CMA2: renamed from CMD1; footprint C0402 -> C0603; MPN MLCC-100nF-16V -> MLCC-1uF-16V
- CMD9: renamed from CYA; value 12pF -> 100nF; footprint C0603 -> C0402; MPN MLCC-12pF-50V -> MLCC-100nF-16V
- CMT1F: renamed from RMT2S; value 1k -> 47nF; footprint R0603 -> C0603; symbol traction-r1:R -> traction-r1:C; MPN R0603-CLASS -> MLCC-47nF-25V
- CMT2F: renamed from TVSM1; value PESD5V0L1BA -> 47nF; footprint SOD323 -> C0603; symbol traction-r1:R -> traction-r1:C; MPN PESD5V0L1BA -> MLCC-47nF-25V
- COF1: renamed from RVD1D; value 10k -> 100nF; footprint R0603 -> C0603; symbol traction-r1:R -> traction-r1:C; MPN R0603-10k-0.1% -> MLCC-CLASS
- COR1: renamed from CILK; value 2.2nF -> 100nF; MPN MLCC-2.2nF-50V -> MLCC-CLASS
- COR2: renamed from RILK1; value 10k -> 100nF; footprint R0603 -> C0603; symbol traction-r1:R -> traction-r1:C; MPN R0603-10k -> MLCC-CLASS
- CRST: renamed from RBOOT; value 10k -> 100pF; footprint R0603 -> C0603; symbol traction-r1:R -> traction-r1:C; MPN R0603-10k -> MLCC-100pF-16V
- CSB1: renamed from CSB2; value 10uF -> 22uF
- CSB2: renamed from CSB3; value 10uF -> 22uF
- CSB3: renamed from CSB4; value 10uF -> 22uF
- CSB3B: renamed from CSB5; value 2.2uF -> 22uF; footprint C0805 -> C0603
- CSB4: renamed from CSB6; value 4.7uF -> 10uF
- CSB5: renamed from CSB7; value 10uF -> 2.2uF
- CSB6: renamed from CSB8; value 10uF -> 4.7uF
- CSB7: renamed from CVBOS; value 4.7uF -> 10uF; footprint C0603 -> C0805
- CSB8: renamed from CVDIG; value 1uF -> 10uF; footprint C0603 -> C0805
- CSINA1: renamed from RSINF2; value 330R -> 100pF; footprint R0603 -> C0603; symbol traction-r1:R -> traction-r1:C; MPN R0603-CLASS -> MLCC-CLASS
- CSINA2: renamed from RSINR1; value 120R -> 2.2nF; footprint R0603 -> C0603; symbol traction-r1:R -> traction-r1:C; MPN R0603-120R -> MLCC-CLASS
- CSIND: renamed from RSINR2; value 120R -> 220pF; footprint R0603 -> C0603; symbol traction-r1:R -> traction-r1:C; MPN R0603-120R -> MLCC-CLASS
- CSINF: renamed from DCOSP; value PESD2IVN24-T -> 22pF; footprint SOT23 -> C0603; symbol traction-r1:PESD2IVN24-T -> traction-r1:C; LCSC C406047 -> CLASS; MPN PESD2IVN24-T -> MLCC-CLASS
- CSNWF: renamed from JTAMB; value NTC-10k-0603 -> 47nF; footprint R0603 -> C0603; symbol traction-r1:J2 -> traction-r1:C; MPN NTC-10k-0603 -> MLCC-47nF-25V
- CTAMBF: renamed from UMT2; value OPA333AQDBVRQ1 -> 47nF; footprint SOT23-5 -> C0603; symbol traction-r1:OPA333AQDBVRQ1 -> traction-r1:C; LCSC C2058544 -> CLASS; MPN OPA333AQDBVRQ1 -> MLCC-47nF-25V
- CUB1: renamed from RUB3; value 100R -> 3.3nF; footprint R0603 -> C0603; symbol traction-r1:R -> traction-r1:C; MPN R0603-100R -> MLCC-3.3nF-50V
- CUB2: renamed from UVB1; value OPA376AQDBVRQ1 -> 100nF; footprint SOT23-5 -> C0603; symbol traction-r1:OPA376AQDBVRQ1 -> traction-r1:C; MPN OPA376AQDBVRQ1 -> MLCC-3.3nF-50V
- CUS1: renamed from UVB2; value OPA376AQDBVRQ1 -> 47nF; footprint SOT23-5 -> C0603; symbol traction-r1:OPA376AQDBVRQ1 -> traction-r1:C; MPN OPA376AQDBVRQ1 -> MLCC-47nF-25V
- CUS2: renamed from CVB1; value 3.3nF -> 4.7nF; MPN MLCC-3.3nF-50V -> MLCC-47nF-25V
- CVB1: renamed from RVB3; value 100R -> 3.3nF; footprint R0603 -> C0603; symbol traction-r1:R -> traction-r1:C; MPN R0603-100R -> MLCC-3.3nF-50V
- CVB2: renamed from UWB1; value OPA376AQDBVRQ1 -> 100nF; footprint SOT23-5 -> C0603; symbol traction-r1:OPA376AQDBVRQ1 -> traction-r1:C; MPN OPA376AQDBVRQ1 -> MLCC-3.3nF-50V
- CVBOS: renamed from DBAT; value BAT46ZFILM -> 4.7uF; footprint SOD123 -> C0603; symbol traction-r1:D -> traction-r1:C; LCSC C283255 -> CLASS; MPN BAT46ZFILM -> MLCC-CLASS
- CVD1: renamed from UVD2; value OPA376AQDBVRQ1 -> 100pF; footprint SOT23-5 -> C0603; symbol traction-r1:OPA376AQDBVRQ1 -> traction-r1:C; MPN OPA376AQDBVRQ1 -> MLCC-CLASS
- CVD2: renamed from CSNWF; value 47nF -> 100pF; MPN MLCC-47nF-25V -> MLCC-CLASS
- CVDIG: renamed from LCOR; value IND-4.7uH-2A -> 1uF; footprint IND5x5 -> C0603; symbol traction-r1:L -> traction-r1:C; MPN IND-4.7uH-2A -> MLCC-CLASS
- CVM1: renamed from RVM1; value 24k -> 220nF; footprint R0603 -> C0603; symbol traction-r1:R -> traction-r1:C; MPN R0603-24k-1% -> MLCC-CLASS
- CVM2: renamed from RVM2; value 24k -> 220nF; footprint R0603 -> C0603; symbol traction-r1:R -> traction-r1:C; MPN R0603-24k-1% -> MLCC-CLASS
- CVS1: renamed from UWB2; value OPA376AQDBVRQ1 -> 47nF; footprint SOT23-5 -> C0603; symbol traction-r1:OPA376AQDBVRQ1 -> traction-r1:C; MPN OPA376AQDBVRQ1 -> MLCC-47nF-25V
- CVS2: renamed from CWB1; value 3.3nF -> 4.7nF; MPN MLCC-3.3nF-50V -> MLCC-47nF-25V
- CWB1: renamed from RWB3; value 100R -> 3.3nF; footprint R0603 -> C0603; symbol traction-r1:R -> traction-r1:C; MPN R0603-100R -> MLCC-3.3nF-50V
- CWB2: renamed from UVD1; value OPA376AQDBVRQ1 -> 100nF; footprint SOT23-5 -> C0603; symbol traction-r1:OPA376AQDBVRQ1 -> traction-r1:C; MPN OPA376AQDBVRQ1 -> MLCC-3.3nF-50V
- CWS1: renamed from UVOF; value OPA376AQDBVRQ1 -> 47nF; footprint SOT23-5 -> C0603; symbol traction-r1:OPA376AQDBVRQ1 -> traction-r1:C; MPN OPA376AQDBVRQ1 -> MLCC-47nF-25V
- CWS2: renamed from COF1; value 100nF -> 4.7nF; MPN MLCC-CLASS -> MLCC-47nF-25V
- CYB: renamed from RMRST; value 10k -> 12pF; footprint R0603 -> C0603; symbol traction-r1:R -> traction-r1:C; MPN R0603-10k -> MLCC-12pF-50V
- DBAT: renamed from LSBC; value IND-10uH-2A -> BAT46ZFILM; footprint IND6x6 -> SOD123; symbol traction-r1:L -> traction-r1:D; LCSC CLASS -> C283255; MPN IND-10uH-2A -> BAT46ZFILM
- DCOSP: renamed from RCOSF1; value 330R -> PESD2IVN24-T; footprint R0603 -> SOT23; symbol traction-r1:R -> traction-r1:PESD2IVN24-T; LCSC CLASS -> C406047; MPN R0603-CLASS -> PESD2IVN24-T
- DFLT1: renamed from RENP1; value 1k -> 1N4148WS; footprint R0603 -> SOD323; symbol traction-r1:R -> traction-r1:D; LCSC CLASS -> C2128; MPN R0603-1k -> 1N4148WS
- DFLT2: renamed from RENP2; value 1k -> 1N4148WS; footprint R0603 -> SOD323; symbol traction-r1:R -> traction-r1:D; LCSC CLASS -> C2128; MPN R0603-1k -> 1N4148WS
- DIGN: renamed from RIGN2; value 10k -> 1N4148WS; footprint R0603 -> SOD323; symbol traction-r1:R -> traction-r1:D; LCSC CLASS -> C2128; MPN R0603-5k1 -> 1N4148WS
- DREVC: renamed from DTVSC; value TPSMC24CA -> STPS5L60S; LCSC C1975284 -> C140620; MPN TPSMC24CA -> STPS5L60S
- DSINP: renamed from RSINF1; value 330R -> PESD2IVN24-T; footprint R0603 -> SOT23; symbol traction-r1:R -> traction-r1:PESD2IVN24-T; LCSC CLASS -> C406047; MPN R0603-CLASS -> PESD2IVN24-T
- DTVSC: renamed from FLVC; value MF-LSMF300/24X-2 -> TPSMC24CA; footprint PTC2920 -> SMC; symbol traction-r1:F -> traction-r1:D; LCSC C719172 -> C1975284; MPN MF-LSMF300/24X-2 -> TPSMC24CA
- FMT1: renamed from TVSM2; value PESD5V0L1BA -> FUSE-350mA-0603; footprint SOD323 -> F0603; symbol traction-r1:R -> traction-r1:F; MPN PESD5V0L1BA -> FUSE-350mA-0603
- FMT2: renamed from LCAN1; value ACT45B-101-2P-TL003 -> FUSE-350mA-0603; footprint CMC1210 -> F0603; symbol traction-r1:ACT45B-101-2P-TL003 -> traction-r1:F; MPN ACT45B-101-2P-TL003 -> FUSE-350mA-0603
- FVBL: renamed from LFC; value FB-120R-3A -> MF-LSMF300/24X-2; footprint FB1206 -> PTC2920; symbol traction-r1:L -> traction-r1:F; LCSC CLASS -> C719172; MPN FB-120R-3A -> MF-LSMF300/24X-2
- FVS1: renamed from RCPD1; value 10k -> MF-LSMF; footprint R0603 -> PTC1206; symbol traction-r1:R -> traction-r1:F; MPN R0603-10k -> MF-LSMF-CLASS
- JLEM: renamed from CUB2; value 100nF -> T2M-105-01-L-D-TH-WT; footprint C0603 -> HDR2x5; symbol traction-r1:C -> traction-r1:T2M-105-01-L-D-TH-WT; MPN MLCC-3.3nF-50V -> T2M-105-01-L-D-TH-WT
- JSWD: renamed from CRST; value 100pF -> HDR2X10-JTAG; footprint C0603 -> HDR2x10; symbol traction-r1:C -> traction-r1:HDR2X10-JTAG; MPN MLCC-100pF-16V -> HDR2X10-JTAG
- JTAMB: renamed from CMT2F; value 47nF -> NTC-10k-0603; footprint C0603 -> R0603; symbol traction-r1:C -> traction-r1:J2; MPN MLCC-47nF-25V -> NTC-10k-0603
- JTHS: renamed from FMT1; value FUSE-350mA-0603 -> NTC-10k-0603; footprint F0603 -> R0603; symbol traction-r1:F -> traction-r1:J2; MPN FUSE-350mA-0603 -> NTC-10k-0603
- renumbered CLAT2 to CAND2, CCAN2 to CCAN1, CCT2 to CCT1, CLVC2 to CLVC1, CMD10 to CMD1, CMD11 to CMD10, CMD12 to CMD11, CMD2 to CMD12, CMD3 to CMD2, CMD4 to CMD3, CMD5 to CMD4, CMD6 to CMD5, CMD7 to CMD6, CMD8 to CMD7, CMD9 to CMD8, CTAMBF to CSNUF, CTHSF to CSNVF, CMT1F to CTHSF, CYB to CYA, FVBH to FLVC, FVBL to FVBH, LCAN2 to LCAN1, RCT2A to RCT1A, RCT2B to RCT1B, RSB2 to RDBG, REXM4 to REXB3, RFS3 to RFS1, RILK3 to RILK1, RILK4 to RILK2, RVD2B to RVD1A, RVD2C to RVD1B, RVD2D to RVD1C, RVM3 to RVM1, RVM4 to RVM2, TVSC2 to TVSC1, UCAN2 to UCAN1
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Connections:
- net labels added: VEXD, VEXVA
- wire segments 776 -> 791
Other:
- note added: "rev A.4.2 - 26 sections - 250 components"
- note removed: "rev A.4.1 - 26 sections - 244 components"
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