File: kicad5/traction/traction-card.sch (KiCad schematic (older format))
At the start: 250 parts, among them Y1 CX3225GA40000D0PTVCC

Commit message: Rev A.4.3: fourth review round — LCOR reconciled, UB15 compensation (F58-F59)
- F58: LCOR netlist value became 2.2uH in A.4.2 but the parts-db class
  MPN kept printing IND-4.7uH-2A on the sheet and BOM - an assembler
  would fit the old part. MPN/desc now carry 2.2uH + the OTP pairing;
  value, sheet, BOM and CORE_LSEL_OTP=0x02 agree end-to-end.
- F59: TPS55340 COMP had only 10nF to ground (no zero; ~0deg screening
  phase margin in the CCM model). Series R3/C4 = 2k/100nF per TI
  8.2.1.2.11 + 470pF HF pole cap; RHPZ ~450kHz not limiting; measured
  Bode stays a bench gate.
- Narrative corrections per review: CBOOT_PRE 100nF was legal (Rev 6.1
  allows 22-100nF; 22nF kept as typ) - F52 log softened; VCC1 loss
  reclassified as a single initiating failure (UGDL open output) whose
  outcome is three-phase-open with ASC still commandable.

Gates: 1695/1695 pins, ERC 782/0, design-verify 75P/3W/0F,
BOM Rs.70,091 @1k, 592 components, 193 lines.

Co-Authored-By: Claude Fable 5 <noreply@anthropic.com>
Parts:
- removed CMA1: 1uF, C0603, symbol traction-r1:C
- removed UMCU: S32K396, BGA289, symbol traction-r1:S32K396
- added RCPD2, RCPD3: 10k, R0603, symbol traction-r1:R
- CAND1: renamed from CFLTF; value 100pF -> 100nF; MPN MLCC-100pF-16V -> MLCC-CLASS
- CBTC: renamed from CSB1; value 22uF -> 47nF; footprint C0805 -> C0603
- CBTP: renamed from CSB2; value 22uF -> 22nF; footprint C0805 -> C0603
- CCAN1: renamed from RCT1A; value 60.4R -> 1uF; footprint R0603 -> C0603; symbol traction-r1:R -> traction-r1:C; MPN R0603-60R4-1% -> MLCC-1uF-25V
- CCAN2: renamed from RCT2A; value 60.4R -> 1uF; footprint R0603 -> C0603; symbol traction-r1:R -> traction-r1:C; MPN R0603-60R4-1% -> MLCC-1uF-25V
- CCOSA1: renamed from CCOSD; value 220pF -> 100pF
- CCOSA2: renamed from CCOSF; value 22pF -> 2.2nF
- CCOSD: renamed from RCOS1; value 680R -> 220pF; footprint R0603 -> C0603; symbol traction-r1:R -> traction-r1:C; MPN R0603-CLASS -> MLCC-CLASS
- CCOSF: renamed from RCOS2; value 680R -> 22pF; footprint R0603 -> C0603; symbol traction-r1:R -> traction-r1:C; MPN R0603-CLASS -> MLCC-CLASS
- CCT1: renamed from RCT1B; value 60.4R -> 4.7nF; footprint R0603 -> C0603; symbol traction-r1:R -> traction-r1:C; MPN R0603-60R4-1% -> MLCC-4.7nF-50V
- CCT2: renamed from RCT2B; value 60.4R -> 4.7nF; footprint R0603 -> C0603; symbol traction-r1:R -> traction-r1:C; MPN R0603-60R4-1% -> MLCC-4.7nF-50V
- CEXA1: renamed from CEXA3; value 100nF -> 4.7nF
- CEXA2: renamed from CEXD; value 4.7uF -> 300pF
- CEXA3: renamed from CLDE; value 22uF -> 100nF
- CEXD: renamed from CLDEC; value 270pF -> 4.7uF
- CFLTF: renamed from DFLT1; value 1N4148WS -> 100pF; footprint SOD323 -> C0603; symbol traction-r1:D -> traction-r1:C; LCSC C2128 -> CLASS; MPN 1N4148WS -> MLCC-100pF-16V
- CIGN: renamed from DIGN; value 1N4148WS -> 100nF; footprint SOD323 -> C0603; symbol traction-r1:D -> traction-r1:C; LCSC C2128 -> CLASS; MPN 1N4148WS -> MLCC-100nF-50V
- CIGNS: renamed from RIGN1; value 5.1k -> 100nF; footprint R0603 -> C0603; symbol traction-r1:R -> traction-r1:C; MPN R0603-5k1 -> MLCC-CLASS
- CILK: renamed from RILK2; value 10k -> 2.2nF; footprint R0603 -> C0603; symbol traction-r1:R -> traction-r1:C; MPN R0603-10k -> MLCC-2.2nF-50V
- CLAT: renamed from RFS1; value 1k -> 100nF; footprint R0603 -> C0603; symbol traction-r1:R -> traction-r1:C; MPN R0603-120R -> MLCC-100nF-16V
- CLAT2: renamed from DFLT2; value 1N4148WS -> 100nF; footprint SOD323 -> C0603; symbol traction-r1:D -> traction-r1:C; LCSC C2128 -> CLASS; MPN 1N4148WS -> MLCC-CLASS
- CLDE: renamed from REXA1; value 3k -> 22uF; footprint R0603 -> C0603; symbol traction-r1:R -> traction-r1:C; MPN R0603-CLASS -> MLCC-CLASS
- CLDEC: renamed from REXA2; value 10k -> 270pF; footprint R0603 -> C0603; symbol traction-r1:R -> traction-r1:C; MPN R0603-CLASS -> MLCC-CLASS
- CLVC1: renamed from DREVC; value STPS5L60S -> 4.7uF; footprint SMC -> C1206; symbol traction-r1:D -> traction-r1:C; LCSC C140620 -> CLASS; MPN STPS5L60S -> MLCC-4.7uF-50V
- CLVC2: renamed from DTVSC; value TPSMC24CA -> 22uF; footprint SMC -> C1206; symbol traction-r1:D -> traction-r1:C; LCSC C1975284 -> CLASS; MPN TPSMC24CA -> MLCC-4.7uF-50V
- CMA1: renamed from CMD1; value 100nF -> 1uF; footprint C0402 -> C0603; MPN MLCC-100nF-16V -> MLCC-1uF-16V
- CMA2: renamed from CMD10; footprint C0402 -> C0603; MPN MLCC-100nF-16V -> MLCC-1uF-16V
- CMD8: renamed from CYA; value 12pF -> 100nF; footprint C0603 -> C0402; MPN MLCC-12pF-50V -> MLCC-100nF-16V
- CMD9: renamed from CYB; value 12pF -> 100nF; footprint C0603 -> C0402; MPN MLCC-12pF-50V -> MLCC-100nF-16V
- CMT1F: renamed from FMT1; value FUSE-350mA-0603 -> 47nF; footprint F0603 -> C0603; symbol traction-r1:F -> traction-r1:C; MPN FUSE-350mA-0603 -> MLCC-47nF-25V
- CMT2F: renamed from FMT2; value FUSE-350mA-0603 -> 47nF; footprint F0603 -> C0603; symbol traction-r1:F -> traction-r1:C; MPN FUSE-350mA-0603 -> MLCC-47nF-25V
- COF1: renamed from ROF1; value 9.1k -> 100nF; footprint R0603 -> C0603; symbol traction-r1:R -> traction-r1:C; MPN R0603-CLASS -> MLCC-CLASS
- COR1: renamed from CILK; value 2.2nF -> 100nF; MPN MLCC-2.2nF-50V -> MLCC-CLASS
- COR2: renamed from RILK1; value 10k -> 100nF; footprint R0603 -> C0603; symbol traction-r1:R -> traction-r1:C; MPN R0603-10k -> MLCC-CLASS
- CRST: renamed from CLVC1; value 4.7uF -> 100pF; footprint C1206 -> C0603; MPN MLCC-4.7uF-50V -> MLCC-100pF-16V
- CSB2: renamed from CSB3B; footprint C0603 -> C0805
- CSB3: renamed from CSB4; value 10uF -> 22uF
- CSB3B: renamed from CSB5; value 2.2uF -> 22uF; footprint C0805 -> C0603
- CSB4: renamed from CSB6; value 4.7uF -> 10uF
- CSB5: renamed from CSB7; value 10uF -> 2.2uF
- CSB6: renamed from CSB8; value 10uF -> 4.7uF
- CSB7: renamed from CVBOS; value 4.7uF -> 10uF; footprint C0603 -> C0805
- CSB8: renamed from CVDIG; value 1uF -> 10uF; footprint C0603 -> C0805
- CSINA1: renamed from CSIND; value 220pF -> 100pF
- CSINA2: renamed from CSINF; value 22pF -> 2.2nF
- CSIND: renamed from RSIN1; value 680R -> 220pF; footprint R0603 -> C0603; symbol traction-r1:R -> traction-r1:C; MPN R0603-CLASS -> MLCC-CLASS
- CSINF: renamed from RSIN2; value 680R -> 22pF; footprint R0603 -> C0603; symbol traction-r1:R -> traction-r1:C; MPN R0603-CLASS -> MLCC-CLASS
- CSNVF: renamed from RSNUP; value 5.1k -> 47nF; footprint R0603 -> C0603; symbol traction-r1:R -> traction-r1:C; MPN R0603-4k99 -> MLCC-47nF-25V
- CSNWF: renamed from RSNVP; value 5.1k -> 47nF; footprint R0603 -> C0603; symbol traction-r1:R -> traction-r1:C; MPN R0603-4k99 -> MLCC-47nF-25V
- CTAMBF: renamed from JTAMB; value NTC-10k-0603 -> 47nF; footprint R0603 -> C0603; symbol traction-r1:J2 -> traction-r1:C; MPN NTC-10k-0603 -> MLCC-47nF-25V
- CTHSF: renamed from JTHS; value NTC-10k-0603 -> 47nF; footprint R0603 -> C0603; symbol traction-r1:J2 -> traction-r1:C; MPN NTC-10k-0603 -> MLCC-47nF-25V
- CUB1: renamed from CUS1; value 47nF -> 3.3nF; MPN MLCC-47nF-25V -> MLCC-3.3nF-50V
- CUB2: renamed from CUS2; value 4.7nF -> 100nF; MPN MLCC-47nF-25V -> MLCC-3.3nF-50V
- CUS1: renamed from LUB; value FB-220R-1A -> 47nF; footprint FB0805 -> C0603; symbol traction-r1:L -> traction-r1:C; MPN FB-220R-1A -> MLCC-47nF-25V
- CUS2: renamed from RUB1; value 100R -> 4.7nF; footprint R0603 -> C0603; symbol traction-r1:R -> traction-r1:C; MPN R0603-100R -> MLCC-47nF-25V
- CVB1: renamed from CVS1; value 47nF -> 3.3nF; MPN MLCC-47nF-25V -> MLCC-3.3nF-50V
- CVB2: renamed from CVS2; value 4.7nF -> 100nF; MPN MLCC-47nF-25V -> MLCC-3.3nF-50V
- CVBOS: renamed from DBAT; value BAT46ZFILM -> 4.7uF; footprint SOD123 -> C0603; symbol traction-r1:D -> traction-r1:C; LCSC C283255 -> CLASS; MPN BAT46ZFILM -> MLCC-CLASS
- CVD1: renamed from ROF2; value 1k -> 100pF; footprint R0603 -> C0603; symbol traction-r1:R -> traction-r1:C; MPN R0603-CLASS -> MLCC-CLASS
- CVD2: renamed from RVD2B; value 10k -> 100pF; footprint R0603 -> C0603; symbol traction-r1:R -> traction-r1:C; MPN R0603-10k-0.1% -> MLCC-CLASS
- CVDIG: renamed from LCOR; value IND-4.7uH-2A -> 1uF; footprint IND5x5 -> C0603; symbol traction-r1:L -> traction-r1:C; MPN IND-4.7uH-2A -> MLCC-CLASS
- CVM1: renamed from RVM1; value 24k -> 220nF; footprint R0603 -> C0603; symbol traction-r1:R -> traction-r1:C; MPN R0603-24k-1% -> MLCC-CLASS
- CVM2: renamed from RVM2; value 24k -> 220nF; footprint R0603 -> C0603; symbol traction-r1:R -> traction-r1:C; MPN R0603-24k-1% -> MLCC-CLASS
- CVS1: renamed from LVB; value FB-220R-1A -> 47nF; footprint FB0805 -> C0603; symbol traction-r1:L -> traction-r1:C; MPN FB-220R-1A -> MLCC-47nF-25V
- CVS2: renamed from RVB1; value 100R -> 4.7nF; footprint R0603 -> C0603; symbol traction-r1:R -> traction-r1:C; MPN R0603-100R -> MLCC-47nF-25V
- CWB1: renamed from CWS1; value 47nF -> 3.3nF; MPN MLCC-47nF-25V -> MLCC-3.3nF-50V
- CWB2: renamed from CWS2; value 4.7nF -> 100nF; MPN MLCC-47nF-25V -> MLCC-3.3nF-50V
- CWS1: renamed from LWB; value FB-220R-1A -> 47nF; footprint FB0805 -> C0603; symbol traction-r1:L -> traction-r1:C; MPN FB-220R-1A -> MLCC-47nF-25V
- CWS2: renamed from RWB1; value 100R -> 4.7nF; footprint R0603 -> C0603; symbol traction-r1:R -> traction-r1:C; MPN R0603-100R -> MLCC-47nF-25V
- CYA: renamed from RMRST; value 10k -> 12pF; footprint R0603 -> C0603; symbol traction-r1:R -> traction-r1:C; MPN R0603-10k -> MLCC-12pF-50V
- CYB: renamed from Y1; value CX3225GA40000D0PTVCC -> 12pF; footprint X3225 -> C0603; symbol traction-r1:Y -> traction-r1:C; LCSC C6009848 -> CLASS; MPN CX3225GA40000D0PTVCC -> MLCC-12pF-50V
- DBAT: renamed from LSBC; value IND-10uH-2A -> BAT46ZFILM; footprint IND6x6 -> SOD123; symbol traction-r1:L -> traction-r1:D; LCSC CLASS -> C283255; MPN IND-10uH-2A -> BAT46ZFILM
- DCOSP: renamed from CCOSA2; value 2.2nF -> PESD2IVN24-T; footprint C0603 -> SOT23; symbol traction-r1:C -> traction-r1:PESD2IVN24-T; LCSC CLASS -> C406047; MPN MLCC-CLASS -> PESD2IVN24-T
- DFLT1: renamed from RENP1; value 1k -> 1N4148WS; footprint R0603 -> SOD323; symbol traction-r1:R -> traction-r1:D; LCSC CLASS -> C2128; MPN R0603-1k -> 1N4148WS
- DFLT2: renamed from RENP2; value 1k -> 1N4148WS; footprint R0603 -> SOD323; symbol traction-r1:R -> traction-r1:D; LCSC CLASS -> C2128; MPN R0603-1k -> 1N4148WS
- DIGN: renamed from RIGN2; value 10k -> 1N4148WS; footprint R0603 -> SOD323; symbol traction-r1:R -> traction-r1:D; LCSC CLASS -> C2128; MPN R0603-5k1 -> 1N4148WS
- DREVC: renamed from FLVC; value MF-LSMF300/24X-2 -> STPS5L60S; footprint PTC2920 -> SMC; symbol traction-r1:F -> traction-r1:D; LCSC C719172 -> C140620; MPN MF-LSMF300/24X-2 -> STPS5L60S
- DSINP: renamed from CSINA2; value 2.2nF -> PESD2IVN24-T; footprint C0603 -> SOT23; symbol traction-r1:C -> traction-r1:PESD2IVN24-T; LCSC CLASS -> C406047; MPN MLCC-CLASS -> PESD2IVN24-T
- DTVSC: renamed from FVBH; value MF-LSMF300/24X-2 -> TPSMC24CA; footprint PTC2920 -> SMC; symbol traction-r1:F -> traction-r1:D; LCSC C719172 -> C1975284; MPN MF-LSMF300/24X-2 -> TPSMC24CA
- FMT1: renamed from RMT1P; value 10k -> FUSE-350mA-0603; footprint R0603 -> F0603; symbol traction-r1:R -> traction-r1:F; MPN R0603-CLASS -> FUSE-350mA-0603
- FMT2: renamed from RMT1S; value 1k -> FUSE-350mA-0603; footprint R0603 -> F0603; symbol traction-r1:R -> traction-r1:F; MPN R0603-CLASS -> FUSE-350mA-0603
- FVBH: renamed from LFC; value FB-120R-3A -> MF-LSMF300/24X-2; footprint FB1206 -> PTC2920; symbol traction-r1:L -> traction-r1:F; LCSC CLASS -> C719172; MPN FB-120R-3A -> MF-LSMF300/24X-2
- FVBL: renamed from QBAL; value SQ2310ES -> MF-LSMF300/24X-2; footprint SOT23 -> PTC2920; symbol traction-r1:SQ2310ES -> traction-r1:F; LCSC CLASS -> C719172; MPN SQ2310ES -> MF-LSMF300/24X-2
- FVS1: renamed from LVS2; value FB-470R -> MF-LSMF; footprint FB0603 -> PTC1206; symbol traction-r1:L -> traction-r1:F; MPN FB-470R-CLASS -> MF-LSMF-CLASS
- JICC: renamed from RCPD1; value 10k -> MICROFIT3-40; footprint R0603 -> MicroFit40; symbol traction-r1:R -> traction-r1:MICROFIT3-40; MPN R0603-10k -> MICROFIT3-40
- JLEM: renamed from USNSV; value HC5FW900-S -> T2M-105-01-L-D-TH-WT; footprint OffBoard -> HDR2x5; symbol traction-r1:HC5FW900-S -> traction-r1:T2M-105-01-L-D-TH-WT; MPN HC5FW900-S -> T2M-105-01-L-D-TH-WT
- JSWD: renamed from RBOOT; value 10k -> HDR2X10-JTAG; footprint R0603 -> HDR2x10; symbol traction-r1:R -> traction-r1:HDR2X10-JTAG; MPN R0603-10k -> HDR2X10-JTAG
- JTAMB: renamed from RTAMBP; value 10k -> NTC-10k-0603; symbol traction-r1:R -> traction-r1:J2; MPN R0603-10k-1% -> NTC-10k-0603
- JTHS: renamed from RTHSP; value 10k -> NTC-10k-0603; symbol traction-r1:R -> traction-r1:J2; MPN R0603-10k-1% -> NTC-10k-0603
- JVEH: renamed from LVS1; value FB-470R -> TE 776231-1 (AMPSEAL 23); footprint FB0603 -> AMPSEAL23; symbol traction-r1:L -> traction-r1:TE_776231-1__AMPSEAL_23_; MPN FB-470R-CLASS -> TE 776231-1 (AMPSEAL 23)
- LCAN1: renamed from UCAN1; value TCAN1042HGVDRQ1 -> ACT45B-101-2P-TL003; footprint SOIC8 -> CMC1210; symbol traction-r1:TCAN1042HGVDRQ1 -> traction-r1:ACT45B-101-2P-TL003; LCSC C132550 -> CLASS; MPN TCAN1042HGVDRQ1 -> ACT45B-101-2P-TL003
- LCAN2: renamed from UCAN2; value TCAN1042HGVDRQ1 -> ACT45B-101-2P-TL003; footprint SOIC8 -> CMC1210; symbol traction-r1:TCAN1042HGVDRQ1 -> traction-r1:ACT45B-101-2P-TL003; LCSC C132550 -> CLASS; MPN TCAN1042HGVDRQ1 -> ACT45B-101-2P-TL003
- LCOR: renamed from RAGT; value 0R -> IND-2.2uH-4A; footprint R0603 -> IND5x5; symbol traction-r1:R -> traction-r1:L; MPN R0603-CLASS -> IND-2.2uH-4A
- LFC: renamed from USBC; value FS2633D -> FB-120R-3A; footprint HLQFP48 -> FB1206; symbol traction-r1:FS2633D -> traction-r1:L; MPN FS2633D -> FB-120R-3A
- LSBC: renamed from RDBG; value 10k -> IND-10uH-2A; footprint R0603 -> IND6x6; symbol traction-r1:R -> traction-r1:L; MPN R0603-CLASS -> IND-10uH-2A
- LUB: renamed from RUB2; value 100R -> FB-220R-1A; footprint R0603 -> FB0805; symbol traction-r1:R -> traction-r1:L; MPN R0603-100R -> FB-220R-1A
- LVB: renamed from RVB2; value 100R -> FB-220R-1A; footprint R0603 -> FB0805; symbol traction-r1:R -> traction-r1:L; MPN R0603-100R -> FB-220R-1A
- LVS3: renamed from JICC; value MICROFIT3-40 -> FB-470R; footprint MicroFit40 -> FB0603; symbol traction-r1:MICROFIT3-40 -> traction-r1:L; MPN MICROFIT3-40 -> FB-470R-CLASS
- LVS4: renamed from RCPD0; value 10k -> FB-470R; footprint R0603 -> FB0603; symbol traction-r1:R -> traction-r1:L; MPN R0603-10k -> FB-470R-CLASS
- LWB: renamed from RWB2; value 100R -> FB-220R-1A; footprint R0603 -> FB0805; symbol traction-r1:R -> traction-r1:L; MPN R0603-100R -> FB-220R-1A
- QBAL: renamed from CBTC; value 47nF -> SQ2310ES; footprint C0603 -> SOT23; symbol traction-r1:C -> traction-r1:SQ2310ES; MPN MLCC-CLASS -> SQ2310ES
- RAGT: renamed from RSB1; value 52.3k -> 0R
- RASCP: renamed from RFS2; MPN R0603-120R -> R0603-10k
- RBOOT: renamed from CLVC2; value 22uF -> 10k; footprint C1206 -> R0603; symbol traction-r1:C -> traction-r1:R; MPN MLCC-4.7uF-50V -> R0603-10k
- RCOS1: renamed from RCOSF1; value 330R -> 680R
- RCOS2: renamed from RCOSF2; value 330R -> 680R
- RCOSF1: renamed from RCOSR1; value 120R -> 330R; MPN R0603-120R -> R0603-CLASS
- RCOSF2: renamed from RCOSR2; value 120R -> 330R; MPN R0603-120R -> R0603-CLASS
- RCOSR1: renamed from JLEM; value T2M-105-01-L-D-TH-WT -> 120R; footprint HDR2x5 -> R0603; symbol traction-r1:T2M-105-01-L-D-TH-WT -> traction-r1:R; MPN T2M-105-01-L-D-TH-WT -> R0603-120R
- RCOSR2: renamed from USNSU; value HC5FW900-S -> 120R; footprint OffBoard -> R0603; symbol traction-r1:HC5FW900-S -> traction-r1:R; MPN HC5FW900-S -> R0603-120R
- RCT1A: renamed from LCAN2; value ACT45B-101-2P-TL003 -> 60.4R; footprint CMC1210 -> R0603; symbol traction-r1:ACT45B-101-2P-TL003 -> traction-r1:R; MPN ACT45B-101-2P-TL003 -> R0603-60R4-1%
- RCT1B: renamed from TVSC2; value PESD2IVN24-T -> 60.4R; footprint SOT23 -> R0603; symbol traction-r1:PESD2IVN24-T -> traction-r1:R; LCSC C406047 -> CLASS; MPN PESD2IVN24-T -> R0603-60R4-1%
- RCT2A: renamed from JVEH; value TE 776231-1 (AMPSEAL 23) -> 60.4R; footprint AMPSEAL23 -> R0603; symbol traction-r1:TE_776231-1__AMPSEAL_23_ -> traction-r1:R; MPN TE 776231-1 (AMPSEAL 23) -> R0603-60R4-1%
- RCT2B: renamed from FVS1; value MF-LSMF -> 60.4R; footprint PTC1206 -> R0603; symbol traction-r1:F -> traction-r1:R; MPN MF-LSMF-CLASS -> R0603-60R4-1%
- RENP1: renamed from RFLTC; value 10k -> 1k; MPN R0603-CLASS -> R0603-1k
- RENP2: renamed from RFLTP1; value 5.1k -> 1k; MPN R0603-CLASS -> R0603-1k
- REXA1: renamed from REXA3; value 10k -> 3k
- REXA2: renamed from REXA4; value 24k -> 10k
- REXA3: renamed from REXB1; value 24k -> 10k
- REXB3: renamed from REXM1; value 5.1k -> 24k
- REXB4: renamed from REXM2; value 12k -> 24k
- REXM2: renamed from REXM4; value 24k -> 12k
- REXM3: renamed from RLDE1; value 38.3k -> 5.1k
- REXM4: renamed from RLDE2; value 10k -> 24k
- RFLTC: renamed from RFLTP2; value 5.1k -> 10k
- RFLTP1: renamed from RGPD; value 10k -> 5.1k; MPN R0603-10k -> R0603-CLASS
- RFLTP2: renamed from RLAT2; value 10k -> 5.1k; MPN R0603-10k -> R0603-CLASS
- RFS2: renamed from RFS4; value 1k -> 10k
- RFS3: renamed from RLAT1; value 10k -> 1k; MPN R0603-10k -> R0603-120R
- RFS4: renamed from UOR1; value 74LVC1G32GW-Q100 -> 1k; footprint SOT353 -> R0603; symbol traction-r1:74LVC1G32GW-Q100 -> traction-r1:R; LCSC C548334 -> CLASS; MPN 74LVC1G32GW-Q100 -> R0603-120R
- RGPD: renamed from RRDYP1; value 5.1k -> 10k; MPN R0603-CLASS -> R0603-10k
- RIGN1: renamed from RIGNS1; value 47k -> 5.1k; MPN R0603-CLASS -> R0603-5k1
- RIGN2: renamed from RIGNS2; MPN R0603-CLASS -> R0603-5k1
- RIGNS1: renamed from UAND1; value 74LVC1G11GW-Q100 -> 47k; footprint SOT363 -> R0603; symbol traction-r1:74LVC1G11GW-Q100 -> traction-r1:R; LCSC C548242 -> CLASS; MPN 74LVC1G11GW-Q100 -> R0603-CLASS
- RIGNS2: renamed from UAND2; value 74LVC1G11GW-Q100 -> 10k; footprint SOT363 -> R0603; symbol traction-r1:74LVC1G11GW-Q100 -> traction-r1:R; LCSC C548242 -> CLASS; MPN 74LVC1G11GW-Q100 -> R0603-CLASS
- RILK3: renamed from UVMB1; value OPA348AQDBVRQ1 -> 10k; footprint SOT23-5 -> R0603; symbol traction-r1:OPA348AQDBVRQ1 -> traction-r1:R; LCSC C2877787 -> CLASS; MPN OPA348AQDBVRQ1 -> R0603-10k
- RILK4: renamed from UVMB2; value OPA348AQDBVRQ1 -> 10k; footprint SOT23-5 -> R0603; symbol traction-r1:OPA348AQDBVRQ1 -> traction-r1:R; LCSC C2877787 -> CLASS; MPN OPA348AQDBVRQ1 -> R0603-10k
- RLAT1: renamed from UOR2; value 74LVC1G32GW-Q100 -> 10k; footprint SOT353 -> R0603; symbol traction-r1:74LVC1G32GW-Q100 -> traction-r1:R; LCSC C548334 -> CLASS; MPN 74LVC1G32GW-Q100 -> R0603-10k
- RLAT2: renamed from RRDYP2; value 5.1k -> 10k; MPN R0603-CLASS -> R0603-10k
- RLDE1: renamed from RSDN; value 10k -> 38.3k
- RLDE2: renamed from DSINP; value PESD2IVN24-T -> 10k; footprint SOT23 -> R0603; symbol traction-r1:PESD2IVN24-T -> traction-r1:R; LCSC C406047 -> CLASS; MPN PESD2IVN24-T -> R0603-CLASS
- RMRST: renamed from JSWD; value HDR2X10-JTAG -> 10k; footprint HDR2x10 -> R0603; symbol traction-r1:HDR2X10-JTAG -> traction-r1:R; MPN HDR2X10-JTAG -> R0603-10k
- RMT2P: renamed from TVSM1; value PESD5V0L1BA -> 10k; footprint SOD323 -> R0603; MPN PESD5V0L1BA -> R0603-CLASS
- RMT2S: renamed from TVSM2; value PESD5V0L1BA -> 1k; footprint SOD323 -> R0603; MPN PESD5V0L1BA -> R0603-CLASS
- ROF1: renamed from RVD1A; value 10k -> 9.1k; MPN R0603-10k-0.1% -> R0603-CLASS
- ROF2: renamed from RVD1B; value 10k -> 1k; MPN R0603-10k-0.1% -> R0603-CLASS
- RRDYP1: renamed from ULAT; value SN74LVC1G74DCUR -> 5.1k; footprint VSSOP8 -> R0603; symbol traction-r1:SN74LVC1G74DCUR -> traction-r1:R; LCSC C70285 -> CLASS; MPN SN74LVC1G74DCUR -> R0603-CLASS
- RRDYP2: renamed from CLAT; value 100nF -> 5.1k; footprint C0603 -> R0603; symbol traction-r1:C -> traction-r1:R; MPN MLCC-100nF-16V -> R0603-CLASS
- RSB1: renamed from RSB3; value 220R -> 52.3k
- RSB2: renamed from RSB4; value 5.1k -> 10k
- RSB3: renamed from CIGN; value 100nF -> 220R; footprint C0603 -> R0603; symbol traction-r1:C -> traction-r1:R; MPN MLCC-100nF-50V -> R0603-CLASS
- RSB4: renamed from CIGNS; value 100nF -> 5.1k; footprint C0603 -> R0603; symbol traction-r1:C -> traction-r1:R; MPN MLCC-CLASS -> R0603-CLASS
- RSDN: renamed from CSINA1; value 100pF -> 10k; footprint C0603 -> R0603; symbol traction-r1:C -> traction-r1:R; MPN MLCC-CLASS -> R0603-CLASS
- RSIN1: renamed from RSINF1; value 330R -> 680R
- RSIN2: renamed from RSINF2; value 330R -> 680R
- RSINF1: renamed from RSINR1; value 120R -> 330R; MPN R0603-120R -> R0603-CLASS
- RSINF2: renamed from RSINR2; value 120R -> 330R; MPN R0603-120R -> R0603-CLASS
- RSINR1: renamed from DCOSP; value PESD2IVN24-T -> 120R; footprint SOT23 -> R0603; symbol traction-r1:PESD2IVN24-T -> traction-r1:R; LCSC C406047 -> CLASS; MPN PESD2IVN24-T -> R0603-120R
- RSINR2: renamed from CCOSA1; value 100pF -> 120R; footprint C0603 -> R0603; symbol traction-r1:C -> traction-r1:R; MPN MLCC-CLASS -> R0603-120R
- RSNVP: renamed from RTMR; value 0R -> 5.1k; MPN R0603-CLASS -> R0603-4k99
- RSNWP: renamed from CTAMBF; value 47nF -> 5.1k; footprint C0603 -> R0603; symbol traction-r1:C -> traction-r1:R; MPN MLCC-47nF-25V -> R0603-4k99
- RTAMBP: renamed from UMT1; value OPA333AQDBVRQ1 -> 10k; footprint SOT23-5 -> R0603; symbol traction-r1:OPA333AQDBVRQ1 -> traction-r1:R; LCSC C2058544 -> CLASS; MPN OPA333AQDBVRQ1 -> R0603-10k-1%
- RTHSP: renamed from UMT2; value OPA333AQDBVRQ1 -> 10k; footprint SOT23-5 -> R0603; symbol traction-r1:OPA333AQDBVRQ1 -> traction-r1:R; LCSC C2058544 -> CLASS; MPN OPA333AQDBVRQ1 -> R0603-10k-1%
- RTMR: renamed from CTHSF; value 47nF -> 0R; footprint C0603 -> R0603; symbol traction-r1:C -> traction-r1:R; MPN MLCC-47nF-25V -> R0603-CLASS
- RUB2: renamed from UVB1; value OPA376AQDBVRQ1 -> 100R; footprint SOT23-5 -> R0603; symbol traction-r1:OPA376AQDBVRQ1 -> traction-r1:R; MPN OPA376AQDBVRQ1 -> R0603-100R
- RUB3: renamed from UVB2; value OPA376AQDBVRQ1 -> 100R; footprint SOT23-5 -> R0603; symbol traction-r1:OPA376AQDBVRQ1 -> traction-r1:R; MPN OPA376AQDBVRQ1 -> R0603-100R
- RVB2: renamed from UWB1; value OPA376AQDBVRQ1 -> 100R; footprint SOT23-5 -> R0603; symbol traction-r1:OPA376AQDBVRQ1 -> traction-r1:R; MPN OPA376AQDBVRQ1 -> R0603-100R
- RVB3: renamed from UWB2; value OPA376AQDBVRQ1 -> 100R; footprint SOT23-5 -> R0603; symbol traction-r1:OPA376AQDBVRQ1 -> traction-r1:R; MPN OPA376AQDBVRQ1 -> R0603-100R
- RVD1C: renamed from UVD2; value OPA376AQDBVRQ1 -> 10k; footprint SOT23-5 -> R0603; symbol traction-r1:OPA376AQDBVRQ1 -> traction-r1:R; MPN OPA376AQDBVRQ1 -> R0603-10k-0.1%
- RVD1D: renamed from CVD2; value 100pF -> 10k; footprint C0603 -> R0603; symbol traction-r1:C -> traction-r1:R; MPN MLCC-CLASS -> R0603-10k-0.1%
- RVD2C: renamed from CSNUF; value 47nF -> 10k; footprint C0603 -> R0603; symbol traction-r1:C -> traction-r1:R; MPN MLCC-47nF-25V -> R0603-10k-0.1%
- RVD2D: renamed from CSNVF; value 47nF -> 10k; footprint C0603 -> R0603; symbol traction-r1:C -> traction-r1:R; MPN MLCC-47nF-25V -> R0603-10k-0.1%
- RVM3: renamed from UEXD; value ALM2402QPWPRQ1 -> 24k; footprint HTSSOP16 -> R0603; symbol traction-r1:ALM2402QPWPRQ1 -> traction-r1:R; LCSC C544754 -> CLASS; MPN ALM2402QPWPRQ1 -> R0603-24k-1%
- RVM4: renamed from UEXF; value OPA348AQDBVRQ1 -> 24k; footprint SOT23-5 -> R0603; symbol traction-r1:OPA348AQDBVRQ1 -> traction-r1:R; LCSC C2877787 -> CLASS; MPN OPA348AQDBVRQ1 -> R0603-24k-1%
- RWB2: renamed from UVD1; value OPA376AQDBVRQ1 -> 100R; footprint SOT23-5 -> R0603; symbol traction-r1:OPA376AQDBVRQ1 -> traction-r1:R; MPN OPA376AQDBVRQ1 -> R0603-100R
- RWB3: renamed from UVOF; value OPA376AQDBVRQ1 -> 100R; footprint SOT23-5 -> R0603; symbol traction-r1:OPA376AQDBVRQ1 -> traction-r1:R; MPN OPA376AQDBVRQ1 -> R0603-100R
- TVSC1: renamed from CCAN1; value 1uF -> PESD2IVN24-T; footprint C0603 -> SOT23; symbol traction-r1:C -> traction-r1:PESD2IVN24-T; LCSC CLASS -> C406047; MPN MLCC-1uF-25V -> PESD2IVN24-T
- TVSC2: renamed from CCAN2; value 1uF -> PESD2IVN24-T; footprint C0603 -> SOT23; symbol traction-r1:C -> traction-r1:PESD2IVN24-T; LCSC CLASS -> C406047; MPN MLCC-1uF-25V -> PESD2IVN24-T
- TVSM1: renamed from LCAN1; value ACT45B-101-2P-TL003 -> PESD5V0L1BA; footprint CMC1210 -> SOD323; symbol traction-r1:ACT45B-101-2P-TL003 -> traction-r1:R; MPN ACT45B-101-2P-TL003 -> PESD5V0L1BA
- TVSM2: renamed from TVSC1; value PESD2IVN24-T -> PESD5V0L1BA; footprint SOT23 -> SOD323; symbol traction-r1:PESD2IVN24-T -> traction-r1:R; LCSC C406047 -> CLASS; MPN PESD2IVN24-T -> PESD5V0L1BA
- UAND1: renamed from ULAT2; value SN74LVC1G74DCUR -> 74LVC1G11GW-Q100; footprint VSSOP8 -> SOT363; symbol traction-r1:SN74LVC1G74DCUR -> traction-r1:74LVC1G11GW-Q100; LCSC C70285 -> C548242; MPN SN74LVC1G74DCUR -> 74LVC1G11GW-Q100
- UAND2: renamed from CAND1; value 100nF -> 74LVC1G11GW-Q100; footprint C0603 -> SOT363; symbol traction-r1:C -> traction-r1:74LVC1G11GW-Q100; LCSC CLASS -> C548242; MPN MLCC-CLASS -> 74LVC1G11GW-Q100
- UCAN1: renamed from CCT1; value 4.7nF -> TCAN1042HGVDRQ1; footprint C0603 -> SOIC8; symbol traction-r1:C -> traction-r1:TCAN1042HGVDRQ1; LCSC CLASS -> C132550; MPN MLCC-4.7nF-50V -> TCAN1042HGVDRQ1
- UCAN2: renamed from CCT2; value 4.7nF -> TCAN1042HGVDRQ1; footprint C0603 -> SOIC8; symbol traction-r1:C -> traction-r1:TCAN1042HGVDRQ1; LCSC CLASS -> C132550; MPN MLCC-4.7nF-50V -> TCAN1042HGVDRQ1
- UEXD: renamed from ULDOEX; value NCV4276CDTADJRKG -> ALM2402QPWPRQ1; footprint DPAK5 -> HTSSOP16; symbol traction-r1:NCV4276CDTADJRKG -> traction-r1:ALM2402QPWPRQ1; LCSC CLASS -> C544754; MPN NCV4276CDTADJRKG -> ALM2402QPWPRQ1
- UEXF: renamed from CEXA1; value 4.7nF -> OPA348AQDBVRQ1; footprint C0603 -> SOT23-5; symbol traction-r1:C -> traction-r1:OPA348AQDBVRQ1; LCSC CLASS -> C2877787; MPN MLCC-CLASS -> OPA348AQDBVRQ1
- ULAT: renamed from RASCP; value 10k -> SN74LVC1G74DCUR; footprint R0603 -> VSSOP8; symbol traction-r1:R -> traction-r1:SN74LVC1G74DCUR; LCSC CLASS -> C70285; MPN R0603-10k -> SN74LVC1G74DCUR
- ULAT2: renamed from CAND2; value 100nF -> SN74LVC1G74DCUR; footprint C0603 -> VSSOP8; symbol traction-r1:C -> traction-r1:SN74LVC1G74DCUR; LCSC CLASS -> C70285; MPN MLCC-CLASS -> SN74LVC1G74DCUR
- ULDOEX: renamed from CEXA2; value 300pF -> NCV4276CDTADJRKG; footprint C0603 -> DPAK5; symbol traction-r1:C -> traction-r1:NCV4276CDTADJRKG; MPN MLCC-CLASS -> NCV4276CDTADJRKG
- UMCU: renamed from CMA2; value 100nF -> S32K396; footprint C0603 -> BGA289; symbol traction-r1:C -> traction-r1:S32K396; MPN MLCC-1uF-16V -> S32K396
- UMT1: renamed from CMT1F; value 47nF -> OPA333AQDBVRQ1; footprint C0603 -> SOT23-5; symbol traction-r1:C -> traction-r1:OPA333AQDBVRQ1; LCSC CLASS -> C2058544; MPN MLCC-47nF-25V -> OPA333AQDBVRQ1
- UMT2: renamed from CMT2F; value 47nF -> OPA333AQDBVRQ1; footprint C0603 -> SOT23-5; symbol traction-r1:C -> traction-r1:OPA333AQDBVRQ1; LCSC CLASS -> C2058544; MPN MLCC-47nF-25V -> OPA333AQDBVRQ1
- UOR1: renamed from COR1; value 100nF -> 74LVC1G32GW-Q100; footprint C0603 -> SOT353; symbol traction-r1:C -> traction-r1:74LVC1G32GW-Q100; LCSC CLASS -> C548334; MPN MLCC-CLASS -> 74LVC1G32GW-Q100
- UOR2: renamed from COR2; value 100nF -> 74LVC1G32GW-Q100; footprint C0603 -> SOT353; symbol traction-r1:C -> traction-r1:74LVC1G32GW-Q100; LCSC CLASS -> C548334; MPN MLCC-CLASS -> 74LVC1G32GW-Q100
- USBC: renamed from CBTP; value 22nF -> FS2633D; footprint C0603 -> HLQFP48; symbol traction-r1:C -> traction-r1:FS2633D; MPN MLCC-CLASS -> FS2633D
- USNSV: renamed from UUB1; value OPA376AQDBVRQ1 -> HC5FW900-S; footprint SOT23-5 -> OffBoard; symbol traction-r1:OPA376AQDBVRQ1 -> traction-r1:HC5FW900-S; MPN OPA376AQDBVRQ1 -> HC5FW900-S
- USNSW: renamed from UUB2; value OPA376AQDBVRQ1 -> HC5FW900-S; footprint SOT23-5 -> OffBoard; symbol traction-r1:OPA376AQDBVRQ1 -> traction-r1:HC5FW900-S; MPN OPA376AQDBVRQ1 -> HC5FW900-S
- UUB1: renamed from CUB1; value 3.3nF -> OPA376AQDBVRQ1; footprint C0603 -> SOT23-5; symbol traction-r1:C -> traction-r1:OPA376AQDBVRQ1; MPN MLCC-3.3nF-50V -> OPA376AQDBVRQ1
- UUB2: renamed from CUB2; value 100nF -> OPA376AQDBVRQ1; footprint C0603 -> SOT23-5; symbol traction-r1:C -> traction-r1:OPA376AQDBVRQ1; MPN MLCC-3.3nF-50V -> OPA376AQDBVRQ1
- UVB1: renamed from CVB1; value 3.3nF -> OPA376AQDBVRQ1; footprint C0603 -> SOT23-5; symbol traction-r1:C -> traction-r1:OPA376AQDBVRQ1; MPN MLCC-3.3nF-50V -> OPA376AQDBVRQ1
- UVB2: renamed from CVB2; value 100nF -> OPA376AQDBVRQ1; footprint C0603 -> SOT23-5; symbol traction-r1:C -> traction-r1:OPA376AQDBVRQ1; MPN MLCC-3.3nF-50V -> OPA376AQDBVRQ1
- UVD1: renamed from COF1; value 100nF -> OPA376AQDBVRQ1; footprint C0603 -> SOT23-5; symbol traction-r1:C -> traction-r1:OPA376AQDBVRQ1; MPN MLCC-CLASS -> OPA376AQDBVRQ1
- UVD2: renamed from RVD2A; value 10k -> OPA376AQDBVRQ1; footprint R0603 -> SOT23-5; symbol traction-r1:R -> traction-r1:OPA376AQDBVRQ1; MPN R0603-10k-0.1% -> OPA376AQDBVRQ1
- UVMB1: renamed from CVM1; value 220nF -> OPA348AQDBVRQ1; footprint C0603 -> SOT23-5; symbol traction-r1:C -> traction-r1:OPA348AQDBVRQ1; LCSC CLASS -> C2877787; MPN MLCC-CLASS -> OPA348AQDBVRQ1
- UVMB2: renamed from CVM2; value 220nF -> OPA348AQDBVRQ1; footprint C0603 -> SOT23-5; symbol traction-r1:C -> traction-r1:OPA348AQDBVRQ1; LCSC CLASS -> C2877787; MPN MLCC-CLASS -> OPA348AQDBVRQ1
- UVOF: renamed from CVD1; value 100pF -> OPA376AQDBVRQ1; footprint C0603 -> SOT23-5; symbol traction-r1:C -> traction-r1:OPA376AQDBVRQ1; MPN MLCC-CLASS -> OPA376AQDBVRQ1
- UWB1: renamed from CWB1; value 3.3nF -> OPA376AQDBVRQ1; footprint C0603 -> SOT23-5; symbol traction-r1:C -> traction-r1:OPA376AQDBVRQ1; MPN MLCC-3.3nF-50V -> OPA376AQDBVRQ1
- UWB2: renamed from CWB2; value 100nF -> OPA376AQDBVRQ1; footprint C0603 -> SOT23-5; symbol traction-r1:C -> traction-r1:OPA376AQDBVRQ1; MPN MLCC-3.3nF-50V -> OPA376AQDBVRQ1
- Y1: renamed from CRST; value 100pF -> CX3225GA40000D0PTVCC; footprint C0603 -> X3225; symbol traction-r1:C -> traction-r1:Y; LCSC CLASS -> C6009848; MPN MLCC-100pF-16V -> CX3225GA40000D0PTVCC
- renumbered CLAT2 to CAND2, CMD11 to CMD1, CMD12 to CMD10, CMD2 to CMD11, CMD3 to CMD12, CMD4 to CMD2, CMD5 to CMD3, CMD6 to CMD4, CMD7 to CMD5, CMD8 to CMD6, CMD9 to CMD7, CSB3 to CSB1, CSNWF to CSNUF, FVBL to FLVC, LVS3 to LVS1, LVS4 to LVS2, RCPD2 to RCPD0, RCPD3 to RCPD1, RSB2 to RDBG, REXB2 to REXA4, REXB3 to REXB1, REXB4 to REXB2, REXM3 to REXM1, RFS3 to RFS1, RILK3 to RILK1, RILK4 to RILK2, RMT2P to RMT1P, RMT2S to RMT1S, RSNWP to RSNUP, RUB3 to RUB1, RVB3 to RVB1, RVD1C to RVD1A, RVD1D to RVD1B, RVD2C to RVD2A, RVD2D to RVD2B, RVM3 to RVM1, RVM4 to RVM2, RWB3 to RWB1, USNSW to USNSU
Other:
- note added: "rev A.4.3 - 26 sections - 250 components"
- note removed: "rev A.4.2 - 26 sections - 250 components"
- moved on the sheet: CAND1, CAND2, CBTC, CBTP, CCOSA1, CCOSA2, CEXA1, CEXA2, CEXA3, CEXD, CMA1, CMA2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

Commit message: Rev A.4.4: round five — bind class MPNs to real parts, pin FS26 OTP config
No electrical change. Procurement closure of the review's remaining
generic identifiers, each verified against its manufacturer datasheet:

- LCOR -> Coilcraft XAL4020-222MEC (2.2uH molded, AEC-Q200; values
  read from the XAL4000 datasheet, now in docs/datasheets)
- LB15 + LSBC -> XAL4040-103MEC (one 10uH line item for both; LSBC
  pairing with FPRE_OTP=450kHz documented per the FS26 DS)
- PS5B/PS5C -> Murata MGJ2D150505SC (+5V output used) behind an
  explicit PO gate: verify reinforced-insulation characterization at
  850VDC working and the SIP-7 pin map before ordering
- RECOM R15P05S evaluated and REJECTED during binding: its 6.4kV is a
  1-second test voltage; IEC 62368-1 insulation grade is BASIC at
  250VACrms working - fails the 850V barrier rule. Rejection recorded
  in design-basis 11e and the BOM row so it cannot be substituted in.
- FS26 OTP configuration pinned as design-basis 8a table (VPRE 6.0V,
  FPRE 450kHz, CORE_LSEL=0x02, VCORE 1.5V, LDO1/2 3.3/5.0V, VMONEXT
  0.8V ref, TRK slots off, VBST disabled, WK2PD/IO2PD set) - the
  ordering step must match it; the family label alone is not evidence.

Gates unchanged: 1695/1695 pins, ERC 782/0, design-verify 75P/3W/0F,
sim-verify 18P/1W/0F. BOM Rs.70,934 @1k with real part prices.

Co-Authored-By: Claude Fable 5 <noreply@anthropic.com>
Parts:
- LCOR: value IND-2.2uH-4A -> XAL4020-222MEC; footprint IND5x5 -> XAL4020; MPN IND-2.2uH-4A -> XAL4020-222MEC
- LSBC: value IND-10uH-2A -> XAL4040-103MEC; footprint IND6x6 -> XAL4040; MPN IND-10uH-2A -> XAL4040-103MEC
Other:
- note added: "rev A.4.4 - 26 sections - 250 components"
- note removed: "rev A.4.3 - 26 sections - 250 components"
Changed lines of the file:
@@
 Title "Traction Inverter — Control Card (S32K396 + FS26, ASIL D)"
 Date "2026-09-09"
-Rev "A.4.3"
+Rev "A.4.4"
 Comp "Traction Inverter 220 kW pk - Control card (LV), sheet 4 of 4"
 Comment1 "Inverter = Power board + Cap bank busbar + bolt-on Discharge board (all HV) + Control card (LV); safe state holds with any link lost"
@@
 VEHICLE-IF   -   1 section
 Text Notes 36810 9300 0    60   ~ 0
-rev A.4.3   -   26 sections   -   250 components
+rev A.4.4   -   26 sections   -   250 components
 Wire Notes Line
 	36750 10250 41200 10250
@@
 P 3650 15450
 F 0 "LCOR" H 3650 15290 50  0000 C CNN
-F 1 "IND-2.2uH-4A" H 3650 15620 50  0000 C CNN
-F 2 "IND5x5" H 3650 15450 50  0001 C CNN
+F 1 "XAL4020-222MEC" H 3650 15620 50  0000 C CNN
+F 2 "XAL4020" H 3650 15450 50  0001 C CNN
 F 3 "~" H 3650 15450 50  0001 C CNN
 F 4 "CLASS" H 3650 15450 50  0001 C CNN "LCSC"
-F 5 "IND-2.2uH-4A" H 3650 15450 50  0001 C CNN "MPN"
+F 5 "XAL4020-222MEC" H 3650 15450 50  0001 C CNN "MPN"
 	1    3650 15450
 	1    0    0    -1
@@
 P 3650 15050
 F 0 "LSBC" H 3650 14890 50  0000 C CNN
-F 1 "IND-10uH-2A" H 3650 15220 50  0000 C CNN
-F 2 "IND6x6" H 3650 15050 50  0001 C CNN
+F 1 "XAL4040-103MEC" H 3650 15220 50  0000 C CNN
+F 2 "XAL4040" H 3650 15050 50  0001 C CNN
 F 3 "~" H 3650 15050 50  0001 C CNN
 F 4 "CLASS" H 3650 15050 50  0001 C CNN "LCSC"
-F 5 "IND-10uH-2A" H 3650 15050 50  0001 C CNN "MPN"
+F 5 "XAL4040-103MEC" H 3650 15050 50  0001 C CNN "MPN"
 	1    3650 15050
 	1    0    0    -1
