File: kicad5/traction/traction-card.sch (KiCad schematic (older format))
At the start: 250 parts, among them Y1 CX3225GA40000D0PTVCC

Commit message: Rev A.5: end-to-end documentation refresh + 3 defects the audit caught
Docs (every file rewritten to the released state, history kept as
labeled evidence):
- README: five stacked review paragraphs consolidated into one campaign
  table (F1-F62); new Simulation section with the S1-S7 results table
  and all five SVG plots; badges/stats/mermaids/DFM rows refreshed
  (UCC28C40, four-assembly build flow, 770669-1, sim badge, rev A.5)
- design-basis: gate-drive/LV sections describe the released circuit
  (UCC28C40+BUK7Y14+SMAJ13A clamp, boost->ULDO15 chain, MGJ2+QA01C
  bias set, QA01C +20/-4V note)
- dfm.md + cost-rollup.md rewritten (four assemblies, current tiers,
  76% module share, PO gates, banned-substitute rule)
- EXTRACTED-PARAMS: superseded sections replaced (BUK7Y14, winding
  dots, UCC28C40 UVLO), 10 new part sections, fresh 47-PDF archive
  index with evidence files labeled; SMAJ + TE-770669-1 datasheets
  added; wrong-part PDF from a mirror detected and discarded
- calculations/rev.mjs: single REV source imported by every generator
  (the stale-rev defect class is now structurally impossible)

Defects the audit caught and fixed:
- F60: JVEH was bound to TE 776231-1 "AMPSEAL 23" - its own TE drawing
  shows the 35-pos header (mates 776164). Rebound to 770669-1 (true
  23-pos, mates the 770680-1 plug); drawing archived.
- F61: QA01C DS row is +20/-4V (rails named V18*) - clamps verified
  for +20V; QDIS gate 19.5V vs +22 abs WARN row added.
- F62: the on-sheet ASIL-D + DISCHARGE panel had silently vanished
  from the power sheet as it grew through A.4.x. Placement now retries
  every void and extends the sheet if none fits; a power sheet without
  the panel REFUSES to build. Panel text refreshed (full DRV_EN chain,
  57s bleed, "never energize w/o the DISCHARGE BOARD fitted").

Gates: 1695/1695 pins, ERC 782/0, design-verify 75P/4W/0F, sim-verify
18P/1W/0F, BOM Rs.70,934. Power sheet 44.6x28.6 in (panel row added).

Co-Authored-By: Claude Fable 5 <noreply@ant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
Parts:
- JVEH: value TE 776231-1 (AMPSEAL 23) -> TE 770669-1 (AMPSEAL 23); symbol traction-r1:TE_776231-1__AMPSEAL_23_ -> traction-r1:TE_770669-1__AMPSEAL_23_; MPN TE 776231-1 (AMPSEAL 23) -> TE 770669-1 (AMPSEAL 23)
Other:
- note added: "rev A.5 - 26 sections - 250 components"
- note removed: "rev A.4.4 - 26 sections - 250 components"
Changed lines of the file:
@@
 Title "Traction Inverter — Control Card (S32K396 + FS26, ASIL D)"
 Date "2026-09-09"
-Rev "A.4.4"
+Rev "A.5"
 Comp "Traction Inverter 220 kW pk - Control card (LV), sheet 4 of 4"
 Comment1 "Inverter = Power board + Cap bank busbar + bolt-on Discharge board (all HV) + Control card (LV); safe state holds with any link lost"
@@
 VEHICLE-IF   -   1 section
 Text Notes 36810 9300 0    60   ~ 0
-rev A.4.4   -   26 sections   -   250 components
+rev A.5   -   26 sections   -   250 components
 Wire Notes Line
 	36750 10250 41200 10250
@@
 VEHICLE-IF / CONNECTOR
 $Comp
-L traction-r1:TE_776231-1__AMPSEAL_23_ JVEH
+L traction-r1:TE_770669-1__AMPSEAL_23_ JVEH
 U 1 1 5E000246
 P 27550 19200
 F 0 "JVEH" H 27150 18500 50  0000 R CNN
-F 1 "TE 776231-1 (AMPSEAL 23)" H 27150 19930 50  0000 R CNN
+F 1 "TE 770669-1 (AMPSEAL 23)" H 27150 19930 50  0000 R CNN
 F 2 "AMPSEAL23" H 27550 19200 50  0001 C CNN
 F 3 "~" H 27550 19200 50  0001 C CNN
 F 4 "CLASS" H 27550 19200 50  0001 C CNN "LCSC"
-F 5 "TE 776231-1 (AMPSEAL 23)" H 27550 19200 50  0001 C CNN "MPN"
+F 5 "TE 770669-1 (AMPSEAL 23)" H 27550 19200 50  0001 C CNN "MPN"
 	1    27550 19200
 	1    0    0    -1

Commit message: Rev A.6: review round 6 response, one platform / four SKUs, N7-N9
External review round 6 (46 findings, R-F01..R-F46) was verified finding by
finding and classified in docs/review-A6-disposition.md (+ .csv): 20
Confirmed, 9 Already Fixed, 6 Firmware Handled, 5 Not Applicable,
6 Improvement Recommended. Repo findings F63-F76 are in the verification log.

Hardware (+Rs31/unit, all SKUs unless noted):
- SiC gate 3.3/6.8 ohm; IGBT 1.0/1.0 ohm + 82 pF DESAT blanking (HCG600
  short-circuit rating is 6 us, not 10)
- gate-power flyback start: 2.2 k + 47 uF VDD + 18 V VDD zener (UCC28C40 has
  0.4 V UVLO hysteresis and no clamp); IGBT builds use RT 8.2 k for margin
- fault latch: 10 k / 3.3 nF delay + 15 nF clear one-shot (NSI6611 FLT clears
  only on an EN rising edge, so a fault-dominant latch would deadlock)
- bleeder 2 x 6 x 22 k; HW_ID identity (harness pin 40) and VOFS to the MCU;
  resolver shields to DGND

Platform: one set of PCBs, four SKUs (8XX SiC/IGBT, 4XX IGBT/SiC).
- SKU rows in parts-db, selected by BOM_VARIANT in bom-gen; bom-gen now fails
  on any value/MPN mismatch
- shared calculations/loss-model.mjs
- docs/firmware-contract.md: FW-01..21, safe-state matrix, regen ownership
  (section 4b)
- docs/variants.md: business case

New Road findings:
- N7: LEM HC5FW 900-S/SP1 is a reduced-insulation part, so the phase busbar
  needs a rated sleeve
- N8: TLP152 is UL1577-only; order the (V4) VDE option or an SO6L part
- N9: FW-06 overvoltage response tightened from 100 us to 20 us. With the
  battery path lost at full regen the link reaches 962 V at 100 us and 897 V
  at 20 us; design-verify now checks it

Gates: 602 comps, 1717/1717 pins, ERC 816/0, design-verify 102P/11W/0F,
sim 24P/4W/0F, BOM SiC Rs70,965 / IGBT Rs45,465 @1k.

Co-Authored-By: Claude Opus 5.5 <noreply@anthropic.com>
Parts:
- removed CMA1: 1uF, C0603, symbol traction-r1:C
- removed CMA2: 100nF, C0603, symbol traction-r1:C
- removed CMD1, CMD10: 100nF, C0402, symbol traction-r1:C
- removed UMCU: S32K396, BGA289, symbol traction-r1:S32K396
- added JICC: MICROFIT3-40, MicroFit40, symbol traction-r1:MICROFIT3-40
- added LVS1, LVS2, LVS3, LVS4: FB-470R, FB0603, symbol traction-r1:L
- added RCPD0, RCPD1, RCPD2, RCPD3, RHWP: 10k, R0603, symbol traction-r1:R
- CAND1: renamed from DFLT2; value 1N4148WS -> 100nF; footprint SOD323 -> C0603; symbol traction-r1:D -> traction-r1:C; LCSC C2128 -> CLASS; MPN 1N4148WS -> MLCC-CLASS
- CAND2: renamed from RENP1; value 1k -> 100nF; footprint R0603 -> C0603; symbol traction-r1:R -> traction-r1:C; MPN R0603-1k -> MLCC-CLASS
- CBTC: renamed from CSB3B; value 22uF -> 47nF
- CBTP: renamed from CSB4; value 10uF -> 22nF; footprint C0805 -> C0603
- CCAN1: renamed from RCT2A; value 60.4R -> 1uF; footprint R0603 -> C0603; symbol traction-r1:R -> traction-r1:C; MPN R0603-60R4-1% -> MLCC-1uF-25V
- CCAN2: renamed from LVS4; value FB-470R -> 1uF; footprint FB0603 -> C0603; symbol traction-r1:L -> traction-r1:C; MPN FB-470R-CLASS -> MLCC-1uF-25V
- CCLR: renamed from RENP2; value 1k -> 15nF; footprint R0603 -> C0603; symbol traction-r1:R -> traction-r1:C; MPN R0603-1k -> MLCC-15nF-50V-X7R
- CCOSA1: renamed from RCOSR2; value 120R -> 100pF; footprint R0603 -> C0603; symbol traction-r1:R -> traction-r1:C; MPN R0603-120R -> MLCC-CLASS
- CCOSA2: renamed from JLEM; value T2M-105-01-L-D-TH-WT -> 2.2nF; footprint HDR2x5 -> C0603; symbol traction-r1:T2M-105-01-L-D-TH-WT -> traction-r1:C; MPN T2M-105-01-L-D-TH-WT -> MLCC-CLASS
- CCOSD: renamed from USNSU; value HC5FW900-S -> 220pF; footprint OffBoard -> C0603; symbol traction-r1:HC5FW900-S -> traction-r1:C; MPN HC5FW900-S -> MLCC-CLASS
- CCOSF: renamed from USNSV; value HC5FW900-S -> 22pF; footprint OffBoard -> C0603; symbol traction-r1:HC5FW900-S -> traction-r1:C; MPN HC5FW900-S -> MLCC-CLASS
- CCT1: renamed from RCT2B; value 60.4R -> 4.7nF; footprint R0603 -> C0603; symbol traction-r1:R -> traction-r1:C; MPN R0603-60R4-1% -> MLCC-4.7nF-50V
- CCT2: renamed from JICC; value MICROFIT3-40 -> 4.7nF; footprint MicroFit40 -> C0603; symbol traction-r1:MICROFIT3-40 -> traction-r1:C; MPN MICROFIT3-40 -> MLCC-4.7nF-50V
- CEXA1: renamed from REXA4; value 24k -> 4.7nF; footprint R0603 -> C0603; symbol traction-r1:R -> traction-r1:C; MPN R0603-CLASS -> MLCC-CLASS
- CEXA2: renamed from REXB1; value 24k -> 300pF; footprint R0603 -> C0603; symbol traction-r1:R -> traction-r1:C; MPN R0603-CLASS -> MLCC-CLASS
- CEXA3: renamed from REXB2; value 24k -> 100nF; footprint R0603 -> C0603; symbol traction-r1:R -> traction-r1:C; MPN R0603-CLASS -> MLCC-CLASS
- CEXD: renamed from REXB3; value 24k -> 4.7uF; footprint R0603 -> C0603; symbol traction-r1:R -> traction-r1:C; MPN R0603-CLASS -> MLCC-CLASS
- CFLTD: renamed from RFLTC; value 10k -> 3.3nF; footprint R0603 -> C0603; symbol traction-r1:R -> traction-r1:C; MPN R0603-CLASS -> MLCC-3.3nF-50V-C0G
- CFLTF: renamed from RFLTP1; value 5.1k -> 100pF; footprint R0603 -> C0603; symbol traction-r1:R -> traction-r1:C; MPN R0603-CLASS -> MLCC-100pF-16V
- CIGN: renamed from RIGNS1; value 47k -> 100nF; footprint R0603 -> C0603; symbol traction-r1:R -> traction-r1:C; MPN R0603-CLASS -> MLCC-100nF-50V
- CIGNS: renamed from RIGNS2; value 10k -> 100nF; footprint R0603 -> C0603; symbol traction-r1:R -> traction-r1:C; MPN R0603-CLASS -> MLCC-CLASS
- CILK: renamed from RVM1; value 24k -> 2.2nF; footprint R0603 -> C0603; symbol traction-r1:R -> traction-r1:C; MPN R0603-24k-1% -> MLCC-2.2nF-50V
- CLAT: renamed from COR1; MPN MLCC-CLASS -> MLCC-100nF-16V
- CLAT2: renamed from RFLTP2; value 5.1k -> 100nF; footprint R0603 -> C0603; symbol traction-r1:R -> traction-r1:C; MPN R0603-CLASS -> MLCC-100nF-16V
- CLDE: renamed from REXB4; value 24k -> 22uF; footprint R0603 -> C0603; symbol traction-r1:R -> traction-r1:C; MPN R0603-CLASS -> MLCC-CLASS
- CLDEC: renamed from REXM1; value 5.1k -> 270pF; footprint R0603 -> C0603; symbol traction-r1:R -> traction-r1:C; MPN R0603-CLASS -> MLCC-CLASS
- CLVC1: renamed from FVBH; value MF-LSMF300/24X-2 -> 4.7uF; footprint PTC2920 -> C1206; symbol traction-r1:F -> traction-r1:C; LCSC C719172 -> CLASS; MPN MF-LSMF300/24X-2 -> MLCC-4.7uF-50V
- CLVC2: renamed from FVBL; value MF-LSMF300/24X-2 -> 22uF; footprint PTC2920 -> C1210; symbol traction-r1:F -> traction-r1:C; LCSC C719172 -> CLASS; MPN MF-LSMF300/24X-2 -> MLCC-22uF-50V
- CMA1: renamed from CMD12; value 100nF -> 1uF; footprint C0402 -> C0603; MPN MLCC-100nF-16V -> MLCC-1uF-16V
- CMA2: renamed from CMD2; footprint C0402 -> C0603
- CMD5: renamed from CYA; value 12pF -> 100nF; footprint C0603 -> C0402; MPN MLCC-12pF-50V -> MLCC-100nF-16V
- CMD6: renamed from CYB; value 12pF -> 100nF; footprint C0603 -> C0402; MPN MLCC-12pF-50V -> MLCC-100nF-16V
- CMD7: renamed from RMRST; value 10k -> 100nF; footprint R0603 -> C0402; symbol traction-r1:R -> traction-r1:C; MPN R0603-10k -> MLCC-100nF-16V
- CMD8: renamed from Y1; value CX3225GA40000D0PTVCC -> 100nF; footprint X3225 -> C0402; symbol traction-r1:Y -> traction-r1:C; LCSC C6009848 -> CLASS; MPN CX3225GA40000D0PTVCC -> MLCC-100nF-16V
- CMD9: renamed from JSWD; value HDR2X10-JTAG -> 100nF; footprint HDR2x10 -> C0402; symbol traction-r1:HDR2X10-JTAG -> traction-r1:C; MPN HDR2X10-JTAG -> MLCC-100nF-16V
- CMT1F: renamed from TVSM2; value PESD5V0L1BA -> 47nF; footprint SOD323 -> C0603; symbol traction-r1:R -> traction-r1:C; MPN PESD5V0L1BA -> MLCC-47nF-25V
- CMT2F: renamed from LCAN1; value ACT45B-101-2P-TL003 -> 47nF; footprint CMC1210 -> C0603; symbol traction-r1:ACT45B-101-2P-TL003 -> traction-r1:C; MPN ACT45B-101-2P-TL003 -> MLCC-47nF-25V
- COF1: renamed from CVD2; value 100pF -> 100nF
- COR1: renamed from CVM1; value 220nF -> 100nF
- COR2: renamed from CVM2; value 220nF -> 100nF
- CRST: renamed from DTVSC; value TPSMC24CA -> 100pF; footprint SMC -> C0603; symbol traction-r1:D -> traction-r1:C; LCSC C1975284 -> CLASS; MPN TPSMC24CA -> MLCC-100pF-16V
- CSB1: renamed from CSB5; value 2.2uF -> 22uF
- CSB2: renamed from CSB6; value 4.7uF -> 22uF
- CSB3: renamed from CSB7; value 10uF -> 22uF
- CSB3B: renamed from CSB8; value 10uF -> 22uF; footprint C0805 -> C0603
- CSB4: renamed from CVBOS; value 4.7uF -> 10uF; footprint C0603 -> C0805
- CSB5: renamed from CVDIG; value 1uF -> 2.2uF; footprint C0603 -> C0805
- CSB6: renamed from DBAT; value BAT46ZFILM -> 4.7uF; footprint SOD123 -> C0805; symbol traction-r1:D -> traction-r1:C; LCSC C283255 -> CLASS; MPN BAT46ZFILM -> MLCC-CLASS
- CSB7: renamed from LCOR; value XAL4020-222MEC -> 10uF; footprint XAL4020 -> C0805; symbol traction-r1:L -> traction-r1:C; MPN XAL4020-222MEC -> MLCC-CLASS
- CSB8: renamed from LSBC; value XAL4040-103MEC -> 10uF; footprint XAL4040 -> C0805; symbol traction-r1:L -> traction-r1:C; MPN XAL4040-103MEC -> MLCC-CLASS
- CSINA1: renamed from RSINR2; value 120R -> 100pF; footprint R0603 -> C0603; symbol traction-r1:R -> traction-r1:C; MPN R0603-120R -> MLCC-CLASS
- CSINA2: renamed from DCOSP; value PESD2IVN24-T -> 2.2nF; footprint SOT23 -> C0603; symbol traction-r1:PESD2IVN24-T -> traction-r1:C; LCSC C406047 -> CLASS; MPN PESD2IVN24-T -> MLCC-CLASS
- CSIND: renamed from CCOSA1; value 100pF -> 220pF
- CSINF: renamed from CCOSA2; value 2.2nF -> 22pF
- CSNUF: renamed from JTAMB; value NTC-10k-0603 -> 47nF; footprint R0603 -> C0603; symbol traction-r1:J2 -> traction-r1:C; MPN NTC-10k-0603 -> MLCC-47nF-25V
- CSNVF: renamed from JTHS; value NTC-10k-0603 -> 47nF; footprint R0603 -> C0603; symbol traction-r1:J2 -> traction-r1:C; MPN NTC-10k-0603 -> MLCC-47nF-25V
- CSNWF: renamed from RTAMBP; value 10k -> 47nF; footprint R0603 -> C0603; symbol traction-r1:R -> traction-r1:C; MPN R0603-10k-1% -> MLCC-47nF-25V
- CTHSF: renamed from FMT1; value FUSE-350mA-0603 -> 47nF; footprint F0603 -> C0603; symbol traction-r1:F -> traction-r1:C; MPN FUSE-350mA-0603 -> MLCC-47nF-25V
- CUB1: renamed from UVB2; value OPA376AQDBVRQ1 -> 3.3nF; footprint SOT23-5 -> C0603; symbol traction-r1:OPA376AQDBVRQ1 -> traction-r1:C; MPN OPA376AQDBVRQ1 -> MLCC-3.3nF-50V
- CUB2: renamed from CVB1; value 3.3nF -> 100nF; MPN MLCC-3.3nF-50V -> MLCC-100nF-25V
- CUS1: renamed from CVB2; value 100nF -> 47nF; MPN MLCC-3.3nF-50V -> MLCC-47nF-25V
- CUS2: renamed from CVS1; value 47nF -> 4.7nF; MPN MLCC-47nF-25V -> MLCC-4.7nF-50V
- CVB1: renamed from UWB2; value OPA376AQDBVRQ1 -> 3.3nF; footprint SOT23-5 -> C0603; symbol traction-r1:OPA376AQDBVRQ1 -> traction-r1:C; MPN OPA376AQDBVRQ1 -> MLCC-3.3nF-50V
- CVB2: renamed from CWB1; value 3.3nF -> 100nF; MPN MLCC-3.3nF-50V -> MLCC-100nF-25V
- CVBOS: renamed from RAGT; value 0R -> 4.7uF; footprint R0603 -> C0603; symbol traction-r1:R -> traction-r1:C; MPN R0603-CLASS -> MLCC-CLASS
- CVD1: renamed from RVD2A; value 10k -> 100pF; footprint R0603 -> C0603; symbol traction-r1:R -> traction-r1:C; MPN R0603-10k-0.1% -> MLCC-CLASS
- CVD2: renamed from RSNVP; value 5.1k -> 100pF; footprint R0603 -> C0603; symbol traction-r1:R -> traction-r1:C; MPN R0603-4k99 -> MLCC-CLASS
- CVDIG: renamed from RDBG; value 10k -> 1uF; footprint R0603 -> C0603; symbol traction-r1:R -> traction-r1:C; MPN R0603-CLASS -> MLCC-CLASS
- CVM1: renamed from CEXA1; value 4.7nF -> 220nF
- CVM2: renamed from CEXA2; value 300pF -> 220nF
- CVS1: renamed from CWB2; value 100nF -> 47nF; MPN MLCC-3.3nF-50V -> MLCC-47nF-25V
- CVS2: renamed from CWS1; value 47nF -> 4.7nF; MPN MLCC-47nF-25V -> MLCC-4.7nF-50V
- CWB1: renamed from UVOF; value OPA376AQDBVRQ1 -> 3.3nF; footprint SOT23-5 -> C0603; symbol traction-r1:OPA376AQDBVRQ1 -> traction-r1:C; MPN OPA376AQDBVRQ1 -> MLCC-3.3nF-50V
- CWB2: renamed from COF1; MPN MLCC-CLASS -> MLCC-100nF-25V
- CWS1: renamed from CVD1; value 100pF -> 47nF; MPN MLCC-CLASS -> MLCC-47nF-25V
- CWS2: renamed from ROF1; value 9.1k -> 4.7nF; footprint R0603 -> C0603; symbol traction-r1:R -> traction-r1:C; MPN R0603-CLASS -> MLCC-4.7nF-50V
- CYA: renamed from CRST; value 100pF -> 12pF; MPN MLCC-100pF-16V -> MLCC-12pF-50V
- CYB: renamed from RBOOT; value 10k -> 12pF; footprint R0603 -> C0603; symbol traction-r1:R -> traction-r1:C; MPN R0603-10k -> MLCC-12pF-50V
- DBAT: renamed from RSB1; value 52.3k -> BAT46ZFILM; footprint R0603 -> SOD123; symbol traction-r1:R -> traction-r1:D; LCSC CLASS -> C283255; MPN R0603-CLASS -> BAT46ZFILM
- DCLR: renamed from RGPD; value 10k -> BAT46ZFILM; footprint R0603 -> SOD123; symbol traction-r1:R -> traction-r1:D; LCSC CLASS -> C283255; MPN R0603-10k -> BAT46ZFILM
- DCOSP: renamed from RCOSR1; value 120R -> PESD2IVN24-T; footprint R0603 -> SOT23; symbol traction-r1:R -> traction-r1:PESD2IVN24-T; LCSC CLASS -> C406047; MPN R0603-120R -> PESD2IVN24-T
- DFLT1: renamed from RLAT2; value 10k -> 1N4148WS; footprint R0603 -> SOD323; symbol traction-r1:R -> traction-r1:D; LCSC CLASS -> C2128; MPN R0603-10k -> 1N4148WS
- DFLT2: renamed from RRDYP1; value 5.1k -> 1N4148WS; footprint R0603 -> SOD323; symbol traction-r1:R -> traction-r1:D; LCSC CLASS -> C2128; MPN R0603-CLASS -> 1N4148WS
- DIGN: renamed from UAND1; value 74LVC1G11GW-Q100 -> 1N4148WS; footprint SOT363 -> SOD323; symbol traction-r1:74LVC1G11GW-Q100 -> traction-r1:D; LCSC C548242 -> C2128; MPN 74LVC1G11GW-Q100 -> 1N4148WS
- DREVC: renamed from LFC; value FB-120R-3A -> STPS5L60S; footprint FB1206 -> SMC; symbol traction-r1:L -> traction-r1:D; LCSC CLASS -> C140620; MPN FB-120R-3A -> STPS5L60S
- DSINP: renamed from RSINR1; value 120R -> PESD2IVN24-T; footprint R0603 -> SOT23; symbol traction-r1:R -> traction-r1:PESD2IVN24-T; LCSC CLASS -> C406047; MPN R0603-120R -> PESD2IVN24-T
- DTVSC: renamed from QBAL; value SQ2310ES -> TPSMC24CA; footprint SOT23 -> SMC; symbol traction-r1:SQ2310ES -> traction-r1:D; LCSC CLASS -> C1975284; MPN SQ2310ES -> TPSMC24CA
- FLVC: renamed from USBC; value FS2633D -> MF-LSMF300/24X-2; footprint HLQFP48 -> PTC2920; symbol traction-r1:FS2633D -> traction-r1:F; LCSC CLASS -> C719172; MPN FS2633D -> MF-LSMF300/24X-2
- FMT1: renamed from TVSC1; value PESD2IVN24-T -> FUSE-350mA-0603; footprint SOT23 -> F0603; symbol traction-r1:PESD2IVN24-T -> traction-r1:F; LCSC C406047 -> CLASS; MPN PESD2IVN24-T -> FUSE-350mA-0603
- FMT2: renamed from UCAN1; value TCAN1042HGVDRQ1 -> FUSE-350mA-0603; footprint SOIC8 -> F0603; symbol traction-r1:TCAN1042HGVDRQ1 -> traction-r1:F; LCSC C132550 -> CLASS; MPN TCAN1042HGVDRQ1 -> FUSE-350mA-0603
- FVBH: renamed from CBTC; value 47nF -> MF-LSMF300/24X-2; footprint C0603 -> PTC2920; symbol traction-r1:C -> traction-r1:F; LCSC CLASS -> C719172; MPN MLCC-CLASS -> MF-LSMF300/24X-2
- FVBL: renamed from CBTP; value 22nF -> MF-LSMF300/24X-2; footprint C0603 -> PTC2920; symbol traction-r1:C -> traction-r1:F; LCSC CLASS -> C719172; MPN MLCC-CLASS -> MF-LSMF300/24X-2
- FVS1: renamed from RCPD3; value 10k -> MF-LSMF; footprint R0603 -> PTC1206; symbol traction-r1:R -> traction-r1:F; MPN R0603-10k -> MF-LSMF-CLASS
- JLEM: renamed from CUS2; value 4.7nF -> T2M-105-01-L-D-TH-WT; footprint C0603 -> HDR2x5; symbol traction-r1:C -> traction-r1:T2M-105-01-L-D-TH-WT; MPN MLCC-47nF-25V -> T2M-105-01-L-D-TH-WT
- JSWD: renamed from DREVC; value STPS5L60S -> HDR2X10-JTAG; footprint SMC -> HDR2x10; symbol traction-r1:D -> traction-r1:HDR2X10-JTAG; LCSC C140620 -> CLASS; MPN STPS5L60S -> HDR2X10-JTAG
- JTAMB: renamed from FMT2; value FUSE-350mA-0603 -> NTC-10k-0603; footprint F0603 -> R0603; symbol traction-r1:F -> traction-r1:J2; MPN FUSE-350mA-0603 -> NTC-10k-0603
- JTHS: renamed from RMT1P; value 10k -> NTC-10k-0603; symbol traction-r1:R -> traction-r1:J2; MPN R0603-CLASS -> NTC-10k-0603
- JVEH: renamed from RCPD2; value 10k -> TE 770669-1 (AMPSEAL 23); footprint R0603 -> AMPSEAL23; symbol traction-r1:R -> traction-r1:TE_770669-1__AMPSEAL_23_; MPN R0603-10k -> TE 770669-1 (AMPSEAL 23)
- LCAN1: renamed from UCAN2; value TCAN1042HGVDRQ1 -> ACT45B-101-2P-TL003; footprint SOIC8 -> CMC1210; symbol traction-r1:TCAN1042HGVDRQ1 -> traction-r1:ACT45B-101-2P-TL003; LCSC C132550 -> CLASS; MPN TCAN1042HGVDRQ1 -> ACT45B-101-2P-TL003
- LCAN2: renamed from LVS1; value FB-470R -> ACT45B-101-2P-TL003; footprint FB0603 -> CMC1210; symbol traction-r1:L -> traction-r1:ACT45B-101-2P-TL003; MPN FB-470R-CLASS -> ACT45B-101-2P-TL003
- LCOR: renamed from RSB2; value 10k -> XAL4020-222MEC; footprint R0603 -> XAL4020; symbol traction-r1:R -> traction-r1:L; MPN R0603-CLASS -> XAL4020-222MEC
- LFC: renamed from CSB1; value 22uF -> FB-120R-3A; footprint C0805 -> FB1206; symbol traction-r1:C -> traction-r1:L; MPN MLCC-CLASS -> FB-120R-3A
- LSBC: renamed from RSB3; value 220R -> XAL4040-103MEC; footprint R0603 -> XAL4040; symbol traction-r1:R -> traction-r1:L; MPN R0603-CLASS -> XAL4040-103MEC
- LUB: renamed from CVS2; value 4.7nF -> FB-220R-1A; footprint C0603 -> FB0805; symbol traction-r1:C -> traction-r1:L; MPN MLCC-47nF-25V -> FB-220R-1A
- LVB: renamed from CWS2; value 4.7nF -> FB-220R-1A; footprint C0603 -> FB0805; symbol traction-r1:C -> traction-r1:L; MPN MLCC-47nF-25V -> FB-220R-1A
- LWB: renamed from ROF2; value 1k -> FB-220R-1A; footprint R0603 -> FB0805; symbol traction-r1:R -> traction-r1:L; MPN R0603-CLASS -> FB-220R-1A
- QBAL: renamed from CSB2; value 22uF -> SQ2310ES; footprint C0805 -> SOT23; symbol traction-r1:C -> traction-r1:SQ2310ES; MPN MLCC-CLASS -> SQ2310ES
- RAGT: renamed from RSB4; value 5.1k -> 0R
- RASCP: renamed from COR2; value 100nF -> 10k; footprint C0603 -> R0603; symbol traction-r1:C -> traction-r1:R; MPN MLCC-CLASS -> R0603-10k
- RBOOT: renamed from FLVC; value MF-LSMF300/24X-2 -> 10k; footprint PTC2920 -> R0603; symbol traction-r1:F -> traction-r1:R; LCSC C719172 -> CLASS; MPN MF-LSMF300/24X-2 -> R0603-10k
- RCOS1: renamed from USNSW; value HC5FW900-S -> 680R; footprint OffBoard -> R0603; symbol traction-r1:HC5FW900-S -> traction-r1:R; MPN HC5FW900-S -> R0603-CLASS
- RCOS2: renamed from UUB1; value OPA376AQDBVRQ1 -> 680R; footprint SOT23-5 -> R0603; symbol traction-r1:OPA376AQDBVRQ1 -> traction-r1:R; MPN OPA376AQDBVRQ1 -> R0603-CLASS
- RCOSF1: renamed from UUB2; value OPA376AQDBVRQ1 -> 330R; footprint SOT23-5 -> R0603; symbol traction-r1:OPA376AQDBVRQ1 -> traction-r1:R; MPN OPA376AQDBVRQ1 -> R0603-CLASS
- RCOSF2: renamed from CUB1; value 3.3nF -> 330R; footprint C0603 -> R0603; symbol traction-r1:C -> traction-r1:R; MPN MLCC-3.3nF-50V -> R0603-CLASS
- renumbered CMD3 to CMD1, CMD4 to CMD10, CMD5 to CMD11, CMD6 to CMD12, CMD7 to CMD2, CMD8 to CMD3, CMD9 to CMD4, CMT2F to CTAMBF, RASCP to RFLTD, RILK1 to RFS2, RILK4 to RLAT1, RVB1 to RUB2, RVB2 to RUB3, RWB1 to RVB2, RWB2 to RVB3, RVD2D to RVD1A, UVB1 to UUB2, UWB1 to UVB2, UEXF to UVMB1, UVD2 to UVOF, UVD1 to UWB2
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Connections:
- net labels added: FLT_CLR_M, FLT_OKD, HW_ID
- wire segments 791 -> 803
Other:
- note added: "rev A.6 - 26 sections - 255 components"
- note removed: "rev A.5 - 26 sections - 250 components"
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
Commit message: Rev A.7: review round 7 response (RR01-RR10, A6-R01-R14) + cross-check
Two independent rechecks of c963794 were verified finding by finding and
classified in docs/review-A7-disposition.md (+ .csv): 17 confirmed and fixed,
1 spec gap closed, 3 firmware handled, 3 already-tracked release gates. Two
further defects were self-found (N10, N11).

Safety logic (control card):
- 74LVC3G17-Q100 Schmitt buffer between the RC timing nodes (clear one-shot,
  soft-off delay) and the LVC inputs they drove at 14,000-63,500 ns/V. The
  FS0B line goes through it too; a 100 k pull-down makes a dead buffer
  force DRV_EN low.
- FS0B/FS1B pull-ups 1 k -> 5.1 k (FS1B inside its 2 mA V_OL point).
- FAULT_OUT made sink-only (BAT46): a grounded vehicle wire can no longer
  preset ASC. A KL30 short is clamped at the latch.
- DRV_EN and ASC_CMD read-backs to the MCU for a boot self-test.
- Latches moved to Nexperia 74LVC1G74DC-Q100 (the TI part is not Q100).
- CCLR changed to C0G.

ASC entry is now break-before-make:
- A 12 nF delay (+ fast-release diode) holds the LS ASC off >= 3.4 us.
- MCU path: HS off via the eFlexPWM fault, then PWM-ASC with EN high.
- MCU-dead path: FS0B, then the delayed ASC.
- EN is never dropped for ASC: NSI6611 DS 8.12 honours DESAT over ASC only
  with EN high. The first draft's DASC diode did drop it and was removed
  after the cross-check.
- 1 k series resistor at each LS ASC pin.
- ASC opto LED resistor 470 -> 270 R (TLP152 I_FLH max 7.5 mA).

Gate supply:
- The flyback FB divider senses its own aux rectifier, so the start feed
  can no longer lock gate power out at high KL30.
- 52.3k/15k: VCC2 15.4 V nominal, 13.54-16.7 V corners.
- Boost output capacitors 25 V -> 50 V.

Models and checkers:
- IGBT and diode share the coldplate term.
- Flyback bank inductance corrected.
- SC soft-off checked at both I_STO corners (release gate).
- FW-06 as a measured budget: 15.6 us + 7.0 us all-off -> 905/542 V.
- bom-gen preflight and a JSWD pin-count check (Samtec 10-pin).
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
Parts:
- removed CMA1: 1uF, C0603, symbol traction-r1:C
- removed CMA2: 100nF, C0603, symbol traction-r1:C
- removed CMD1, CMD10, CMD11, CMD12, CMD2, CMD3, CMD4, CMD5: 100nF, C0402, symbol traction-r1:C
- removed UMCU: S32K396, BGA289, symbol traction-r1:S32K396
- added CCAN2: 1uF, C0603, symbol traction-r1:C
- added CCT2: 4.7nF, C0603, symbol traction-r1:C
- added FVS1: MF-LSMF, PTC1206, symbol traction-r1:F
- added JICC: MICROFIT3-40, MicroFit40, symbol traction-r1:MICROFIT3-40
- added JVEH: TE 770669-1 (AMPSEAL 23), AMPSEAL23, symbol traction-r1:TE_770669-1__AMPSEAL_23_
- added LVS1, LVS2, LVS3, LVS4: FB-470R, FB0603, symbol traction-r1:L
- added RCPD0, RCPD1, RCPD2, RCPD3, RHWP: 10k, R0603, symbol traction-r1:R
- added RCT2A, RCT2B: 60.4R, R0603, symbol traction-r1:R
- added TVSC2: PESD2IVN24-T, SOT23, symbol traction-r1:PESD2IVN24-T
- added UCAN2: TCAN1042HGVDRQ1, SOIC8, symbol traction-r1:TCAN1042HGVDRQ1
- CAND1: renamed from RFLTD; value 10k -> 100nF; footprint R0603 -> C0603; symbol traction-r1:R -> traction-r1:C; MPN R0603-10k -> MLCC-CLASS
- CAND2: renamed from RFLTP1; value 5.1k -> 100nF; footprint R0603 -> C0603; symbol traction-r1:R -> traction-r1:C; MPN R0603-5k1 -> MLCC-CLASS
- CBTC: renamed from CVBOS; value 4.7uF -> 47nF
- CBTP: renamed from CVDIG; value 1uF -> 22nF
- CCAN1: renamed from RCPD0; value 10k -> 1uF; footprint R0603 -> C0603; symbol traction-r1:R -> traction-r1:C; MPN R0603-10k -> MLCC-1uF-25V
- CCLR: renamed from RFLTP2; value 5.1k -> 15nF; footprint R0603 -> C0603; symbol traction-r1:R -> traction-r1:C; MPN R0603-5k1 -> MLCC-15nF-50V-C0G
- CCOSA1: renamed from CUS1; value 47nF -> 100pF; MPN MLCC-47nF-25V -> MLCC-CLASS
- CCOSA2: renamed from CUS2; value 4.7nF -> 2.2nF; MPN MLCC-4.7nF-50V -> MLCC-CLASS
- CCOSD: renamed from LUB; value FB-220R-1A -> 220pF; footprint FB0805 -> C0603; symbol traction-r1:L -> traction-r1:C; MPN FB-220R-1A -> MLCC-CLASS
- CCOSF: renamed from RUB1; value 100R -> 22pF; footprint R0603 -> C0603; symbol traction-r1:R -> traction-r1:C; MPN R0603-100R -> MLCC-CLASS
- CCT1: renamed from RCPD1; value 10k -> 4.7nF; footprint R0603 -> C0603; symbol traction-r1:R -> traction-r1:C; MPN R0603-10k -> MLCC-4.7nF-50V
- CEXA1: renamed from RLDE1; value 38.3k -> 4.7nF; footprint R0603 -> C0603; symbol traction-r1:R -> traction-r1:C; MPN R0603-CLASS -> MLCC-CLASS
- CEXA2: renamed from RLDE2; value 10k -> 300pF; footprint R0603 -> C0603; symbol traction-r1:R -> traction-r1:C; MPN R0603-CLASS -> MLCC-CLASS
- CEXA3: renamed from RSDN; value 10k -> 100nF; footprint R0603 -> C0603; symbol traction-r1:R -> traction-r1:C; MPN R0603-CLASS -> MLCC-CLASS
- CEXD: renamed from DSINP; value PESD2IVN24-T -> 4.7uF; footprint SOT23 -> C0603; symbol traction-r1:PESD2IVN24-T -> traction-r1:C; LCSC C406047 -> CLASS; MPN PESD2IVN24-T -> MLCC-CLASS
- CFLTD: renamed from RGPD; value 10k -> 3.3nF; footprint R0603 -> C0603; symbol traction-r1:R -> traction-r1:C; MPN R0603-10k -> MLCC-3.3nF-50V-C0G
- CFLTF: renamed from RLAT2; value 10k -> 100pF; footprint R0603 -> C0603; symbol traction-r1:R -> traction-r1:C; MPN R0603-10k -> MLCC-100pF-16V
- CIGN: renamed from CAND2; MPN MLCC-CLASS -> MLCC-100nF-50V
- CIGNS: renamed from CCLR; value 15nF -> 100nF; MPN MLCC-15nF-50V-X7R -> MLCC-CLASS
- CILK: renamed from CEXA3; value 100nF -> 2.2nF; MPN MLCC-CLASS -> MLCC-2.2nF-50V
- CLAT: renamed from RILK4; value 10k -> 100nF; footprint R0603 -> C0603; symbol traction-r1:R -> traction-r1:C; MPN R0603-10k -> MLCC-100nF-16V
- CLAT2: renamed from RRDYP1; value 5.1k -> 100nF; footprint R0603 -> C0603; symbol traction-r1:R -> traction-r1:C; MPN R0603-5k1 -> MLCC-100nF-16V
- CLDE: renamed from CSINA1; value 100pF -> 22uF
- CLDEC: renamed from CSINA2; value 2.2nF -> 270pF
- CLVC1: renamed from CBTP; value 22nF -> 4.7uF; footprint C0603 -> C1206; MPN MLCC-CLASS -> MLCC-4.7uF-50V
- CLVC2: renamed from CSB1; footprint C0805 -> C1210; MPN MLCC-CLASS -> MLCC-22uF-50V
- CMA1: renamed from CMD7; value 100nF -> 1uF; footprint C0402 -> C0603; MPN MLCC-100nF-16V -> MLCC-1uF-16V
- CMA2: renamed from CMD8; footprint C0402 -> C0603
- CMD10: renamed from CYA; value 12pF -> 100nF; footprint C0603 -> C0402; MPN MLCC-12pF-50V -> MLCC-100nF-16V
- CMD11: renamed from CYB; value 12pF -> 100nF; footprint C0603 -> C0402; MPN MLCC-12pF-50V -> MLCC-100nF-16V
- CMD12: renamed from RMRST; value 10k -> 100nF; footprint R0603 -> C0402; symbol traction-r1:R -> traction-r1:C; MPN R0603-10k -> MLCC-100nF-16V
- CMD2: renamed from Y1; value CX3225GA40000D0PTVCC -> 100nF; footprint X3225 -> C0402; symbol traction-r1:Y -> traction-r1:C; LCSC C6009848 -> CLASS; MPN CX3225GA40000D0PTVCC -> MLCC-100nF-16V
- CMD3: renamed from JSWD; value HDR2X10-JTAG -> 100nF; footprint HDR2x10 -> C0402; symbol traction-r1:HDR2X10-JTAG -> traction-r1:C; MPN HDR2X10-JTAG -> MLCC-100nF-16V
- CMD4: renamed from CRST; value 100pF -> 100nF; footprint C0603 -> C0402; MPN MLCC-100pF-16V -> MLCC-100nF-16V
- CMD5: renamed from RBOOT; value 10k -> 100nF; footprint R0603 -> C0402; symbol traction-r1:R -> traction-r1:C; MPN R0603-10k -> MLCC-100nF-16V
- CMD6: renamed from CLVC1; value 4.7uF -> 100nF; footprint C1206 -> C0402; MPN MLCC-4.7uF-50V -> MLCC-100nF-16V
- CMD7: renamed from CLVC2; value 22uF -> 100nF; footprint C1210 -> C0402; MPN MLCC-22uF-50V -> MLCC-100nF-16V
- CMD8: renamed from DREVC; value STPS5L60S -> 100nF; footprint SMC -> C0402; symbol traction-r1:D -> traction-r1:C; LCSC C140620 -> CLASS; MPN STPS5L60S -> MLCC-100nF-16V
- CMD9: renamed from DTVSC; value TPSMC24CA -> 100nF; footprint SMC -> C0402; symbol traction-r1:D -> traction-r1:C; LCSC C1975284 -> CLASS; MPN TPSMC24CA -> MLCC-100nF-16V
- CMT1F: renamed from TVSC2; value PESD2IVN24-T -> 47nF; footprint SOT23 -> C0603; symbol traction-r1:PESD2IVN24-T -> traction-r1:C; LCSC C406047 -> CLASS; MPN PESD2IVN24-T -> MLCC-47nF-25V
- CMT2F: renamed from UCAN2; value TCAN1042HGVDRQ1 -> 47nF; footprint SOIC8 -> C0603; symbol traction-r1:TCAN1042HGVDRQ1 -> traction-r1:C; LCSC C132550 -> CLASS; MPN TCAN1042HGVDRQ1 -> MLCC-47nF-25V
- COF1: renamed from RSNVP; value 5.1k -> 100nF; footprint R0603 -> C0603; symbol traction-r1:R -> traction-r1:C; MPN R0603-5k1-1% -> MLCC-CLASS
- COR1: renamed from CEXA1; value 4.7nF -> 100nF
- COR2: renamed from CEXA2; value 300pF -> 100nF
- CRST: renamed from USBC; value FS2633D -> 100pF; footprint HLQFP48 -> C0603; symbol traction-r1:FS2633D -> traction-r1:C; MPN FS2633D -> MLCC-100pF-16V
- CSB1: renamed from DBAT; value BAT46ZFILM -> 22uF; footprint SOD123 -> C0805; symbol traction-r1:D -> traction-r1:C; LCSC C283255 -> CLASS; MPN BAT46ZFILM -> MLCC-CLASS
- CSB2: renamed from LCOR; value XAL4020-222MEC -> 22uF; footprint XAL4020 -> C0805; symbol traction-r1:L -> traction-r1:C; MPN XAL4020-222MEC -> MLCC-CLASS
- CSB3: renamed from LSBC; value XAL4040-103MEC -> 22uF; footprint XAL4040 -> C0805; symbol traction-r1:L -> traction-r1:C; MPN XAL4040-103MEC -> MLCC-CLASS
- CSB3B: renamed from RAGT; value 0R -> 22uF; footprint R0603 -> C0603; symbol traction-r1:R -> traction-r1:C; MPN R0603-CLASS -> MLCC-CLASS
- CSB4: renamed from RDBG; value 10k -> 10uF; footprint R0603 -> C0805; symbol traction-r1:R -> traction-r1:C; MPN R0603-CLASS -> MLCC-CLASS
- CSB5: renamed from RSB1; value 52.3k -> 2.2uF; footprint R0603 -> C0805; symbol traction-r1:R -> traction-r1:C; MPN R0603-CLASS -> MLCC-CLASS
- CSB6: renamed from RSB2; value 10k -> 4.7uF; footprint R0603 -> C0805; symbol traction-r1:R -> traction-r1:C; MPN R0603-CLASS -> MLCC-CLASS
- CSB7: renamed from RSB3; value 220R -> 10uF; footprint R0603 -> C0805; symbol traction-r1:R -> traction-r1:C; MPN R0603-CLASS -> MLCC-CLASS
- CSB8: renamed from RSB4; value 5.1k -> 10uF; footprint R0603 -> C0805; symbol traction-r1:R -> traction-r1:C; MPN R0603-CLASS -> MLCC-CLASS
- CSCH: renamed from RRDYP2; value 5.1k -> 100nF; footprint R0603 -> C0603; symbol traction-r1:R -> traction-r1:C; MPN R0603-5k1 -> MLCC-100nF-16V
- CSINA1: renamed from RCOSF2; value 330R -> 100pF; footprint R0603 -> C0603; symbol traction-r1:R -> traction-r1:C; MPN R0603-CLASS -> MLCC-CLASS
- CSINA2: renamed from RCOSR1; value 120R -> 2.2nF; footprint R0603 -> C0603; symbol traction-r1:R -> traction-r1:C; MPN R0603-120R -> MLCC-CLASS
- CSIND: renamed from RCOSR2; value 120R -> 220pF; footprint R0603 -> C0603; symbol traction-r1:R -> traction-r1:C; MPN R0603-120R -> MLCC-CLASS
- CSINF: renamed from JLEM; value T2M-105-01-L-D-TH-WT -> 22pF; footprint HDR2x5 -> C0603; symbol traction-r1:T2M-105-01-L-D-TH-WT -> traction-r1:C; MPN T2M-105-01-L-D-TH-WT -> MLCC-CLASS
- CSNUF: renamed from FMT2; value FUSE-350mA-0603 -> 47nF; footprint F0603 -> C0603; symbol traction-r1:F -> traction-r1:C; MPN FUSE-350mA-0603 -> MLCC-47nF-25V
- CSNVF: renamed from RMT1P; value 10k -> 47nF; footprint R0603 -> C0603; symbol traction-r1:R -> traction-r1:C; MPN R0603-CLASS -> MLCC-47nF-25V
- CSNWF: renamed from RMT1S; value 1k -> 47nF; footprint R0603 -> C0603; symbol traction-r1:R -> traction-r1:C; MPN R0603-CLASS -> MLCC-47nF-25V
- CTAMBF: renamed from LCAN1; value ACT45B-101-2P-TL003 -> 47nF; footprint CMC1210 -> C0603; symbol traction-r1:ACT45B-101-2P-TL003 -> traction-r1:C; MPN ACT45B-101-2P-TL003 -> MLCC-47nF-25V
- CTHSF: renamed from TVSC1; value PESD2IVN24-T -> 47nF; footprint SOT23 -> C0603; symbol traction-r1:PESD2IVN24-T -> traction-r1:C; LCSC C406047 -> CLASS; MPN PESD2IVN24-T -> MLCC-47nF-25V
- CUB1: renamed from UWB1; value OPA376AQDBVRQ1 -> 3.3nF; footprint SOT23-5 -> C0603; symbol traction-r1:OPA376AQDBVRQ1 -> traction-r1:C; MPN OPA376AQDBVRQ1 -> MLCC-3.3nF-50V
- CUB2: renamed from UWB2; value OPA376AQDBVRQ1 -> 100nF; footprint SOT23-5 -> C0603; symbol traction-r1:OPA376AQDBVRQ1 -> traction-r1:C; MPN OPA376AQDBVRQ1 -> MLCC-100nF-25V
- CUS1: renamed from CWB1; value 3.3nF -> 47nF; MPN MLCC-3.3nF-50V -> MLCC-47nF-25V
- CUS2: renamed from CWB2; value 100nF -> 4.7nF; MPN MLCC-100nF-25V -> MLCC-4.7nF-50V
- CVB1: renamed from UVD1; value OPA376AQDBVRQ1 -> 3.3nF; footprint SOT23-5 -> C0603; symbol traction-r1:OPA376AQDBVRQ1 -> traction-r1:C; MPN OPA376AQDBVRQ1 -> MLCC-3.3nF-50V
- CVB2: renamed from UVOF; value OPA376AQDBVRQ1 -> 100nF; footprint SOT23-5 -> C0603; symbol traction-r1:OPA376AQDBVRQ1 -> traction-r1:C; MPN OPA376AQDBVRQ1 -> MLCC-100nF-25V
- CVBOS: renamed from CIGN; value 100nF -> 4.7uF; MPN MLCC-100nF-50V -> MLCC-CLASS
- CVD1: renamed from RSNWP; value 5.1k -> 100pF; footprint R0603 -> C0603; symbol traction-r1:R -> traction-r1:C; MPN R0603-5k1-1% -> MLCC-CLASS
- CVD2: renamed from UMT1; value OPA333AQDBVRQ1 -> 100pF; footprint SOT23-5 -> C0603; symbol traction-r1:OPA333AQDBVRQ1 -> traction-r1:C; LCSC C2058544 -> CLASS; MPN OPA333AQDBVRQ1 -> MLCC-CLASS
- CVDIG: renamed from CIGNS; value 100nF -> 1uF
- CVM1: renamed from REXA4; value 24k -> 220nF; footprint R0603 -> C0603; symbol traction-r1:R -> traction-r1:C; MPN R0603-CLASS -> MLCC-CLASS
- CVM2: renamed from REXB1; value 24k -> 220nF; footprint R0603 -> C0603; symbol traction-r1:R -> traction-r1:C; MPN R0603-CLASS -> MLCC-CLASS
- CVS1: renamed from COF1; value 100nF -> 47nF; MPN MLCC-CLASS -> MLCC-47nF-25V
- CVS2: renamed from CVD1; value 100pF -> 4.7nF; MPN MLCC-CLASS -> MLCC-4.7nF-50V
- CWB1: renamed from UVD2; value OPA376AQDBVRQ1 -> 3.3nF; footprint SOT23-5 -> C0603; symbol traction-r1:OPA376AQDBVRQ1 -> traction-r1:C; MPN OPA376AQDBVRQ1 -> MLCC-3.3nF-50V
- CWB2: renamed from CVD2; value 100pF -> 100nF; MPN MLCC-CLASS -> MLCC-100nF-25V
- CWS1: renamed from RVD2A; value 10k -> 47nF; footprint R0603 -> C0603; symbol traction-r1:R -> traction-r1:C; MPN R0603-10k-0.1% -> MLCC-47nF-25V
- CWS2: renamed from RVD2B; value 10k -> 4.7nF; footprint R0603 -> C0603; symbol traction-r1:R -> traction-r1:C; MPN R0603-10k-0.1% -> MLCC-4.7nF-50V
- CYA: renamed from FLVC; value MF-LSMF300/24X-2 -> 12pF; footprint PTC2920 -> C0603; symbol traction-r1:F -> traction-r1:C; LCSC C719172 -> CLASS; MPN MF-LSMF300/24X-2 -> MLCC-12pF-50V
- CYB: renamed from FVBH; value MF-LSMF300/24X-2 -> 12pF; footprint PTC2920 -> C0603; symbol traction-r1:F -> traction-r1:C; LCSC C719172 -> CLASS; MPN MF-LSMF300/24X-2 -> MLCC-12pF-50V
- DBAT: renamed from DIGN; value 1N4148WS -> BAT46ZFILM; footprint SOD323 -> SOD123; LCSC C2128 -> C283255; MPN 1N4148WS -> BAT46ZFILM
- DCLR: renamed from ULAT; value SN74LVC1G74DCUR -> BAT46ZFILM; footprint VSSOP8 -> SOD123; symbol traction-r1:SN74LVC1G74DCUR -> traction-r1:D; LCSC C70285 -> C283255; MPN SN74LVC1G74DCUR -> BAT46ZFILM
- DCOSP: renamed from CUB2; value 100nF -> PESD2IVN24-T; footprint C0603 -> SOT23; symbol traction-r1:C -> traction-r1:PESD2IVN24-T; LCSC CLASS -> C406047; MPN MLCC-100nF-25V -> PESD2IVN24-T
- DFLT1: renamed from CLAT; value 100nF -> 1N4148WS; footprint C0603 -> SOD323; symbol traction-r1:C -> traction-r1:D; LCSC CLASS -> C2128; MPN MLCC-100nF-16V -> 1N4148WS
- DFLT2: renamed from RASCP; value 10k -> 1N4148WS; footprint R0603 -> SOD323; symbol traction-r1:R -> traction-r1:D; LCSC CLASS -> C2128; MPN R0603-10k -> 1N4148WS
- DFO: renamed from UVMB1; value OPA348AQDBVRQ1 -> BAT46ZFILM; footprint SOT23-5 -> SOD123; symbol traction-r1:OPA348AQDBVRQ1 -> traction-r1:D; LCSC C2877787 -> C283255; MPN OPA348AQDBVRQ1 -> BAT46ZFILM
- DIGN: renamed from CFLTD; value 3.3nF -> 1N4148WS; footprint C0603 -> SOD323; symbol traction-r1:C -> traction-r1:D; LCSC CLASS -> C2128; MPN MLCC-3.3nF-50V-C0G -> 1N4148WS
- DREVC: renamed from CSB2; value 22uF -> STPS5L60S; footprint C0805 -> SMC; symbol traction-r1:C -> traction-r1:D; LCSC CLASS -> C140620; MPN MLCC-CLASS -> STPS5L60S
- DSET: renamed from UVMB2; value OPA348AQDBVRQ1 -> BAT46ZFILM; footprint SOT23-5 -> SOD123; symbol traction-r1:OPA348AQDBVRQ1 -> traction-r1:D; LCSC C2877787 -> C283255; MPN OPA348AQDBVRQ1 -> BAT46ZFILM
- DSINP: renamed from RCOSF1; value 330R -> PESD2IVN24-T; footprint R0603 -> SOT23; symbol traction-r1:R -> traction-r1:PESD2IVN24-T; LCSC CLASS -> C406047; MPN R0603-CLASS -> PESD2IVN24-T
- DTVSC: renamed from CSB3; value 22uF -> TPSMC24CA; footprint C0805 -> SMC; symbol traction-r1:C -> traction-r1:D; LCSC CLASS -> C1975284; MPN MLCC-CLASS -> TPSMC24CA
- FLVC: renamed from CSB3B; value 22uF -> MF-LSMF300/24X-2; footprint C0603 -> PTC2920; symbol traction-r1:C -> traction-r1:F; LCSC CLASS -> C719172; MPN MLCC-CLASS -> MF-LSMF300/24X-2
- FMT1: renamed from CCAN2; value 1uF -> FUSE-350mA-0603; footprint C0603 -> F0603; symbol traction-r1:C -> traction-r1:F; MPN MLCC-1uF-25V -> FUSE-350mA-0603
- FMT2: renamed from CCT2; value 4.7nF -> FUSE-350mA-0603; footprint C0603 -> F0603; symbol traction-r1:C -> traction-r1:F; MPN MLCC-4.7nF-50V -> FUSE-350mA-0603
- FVBH: renamed from CSB4; value 10uF -> MF-LSMF300/24X-2; footprint C0805 -> PTC2920; symbol traction-r1:C -> traction-r1:F; LCSC CLASS -> C719172; MPN MLCC-CLASS -> MF-LSMF300/24X-2
- FVBL: renamed from CSB5; value 2.2uF -> MF-LSMF300/24X-2; footprint C0805 -> PTC2920; symbol traction-r1:C -> traction-r1:F; LCSC CLASS -> C719172; MPN MLCC-CLASS -> MF-LSMF300/24X-2
- JLEM: renamed from CVS1; value 47nF -> T2M-105-01-L-D-TH-WT; footprint C0603 -> HDR2x5; symbol traction-r1:C -> traction-r1:T2M-105-01-L-D-TH-WT; MPN MLCC-47nF-25V -> T2M-105-01-L-D-TH-WT
- JSWD: renamed from QBAL; value SQ2310ES -> FTSH-105-01-L-DV-K; footprint SOT23 -> HDR2x5-1.27; symbol traction-r1:SQ2310ES -> traction-r1:FTSH-105-01-L-DV-K; MPN SQ2310ES -> FTSH-105-01-L-DV-K
- JTAMB: renamed from UCAN1; value TCAN1042HGVDRQ1 -> NTC-10k-0603; footprint SOIC8 -> R0603; symbol traction-r1:TCAN1042HGVDRQ1 -> traction-r1:J2; LCSC C132550 -> CLASS; MPN TCAN1042HGVDRQ1 -> NTC-10k-0603
- JTHS: renamed from CCAN1; value 1uF -> NTC-10k-0603; footprint C0603 -> R0603; symbol traction-r1:C -> traction-r1:J2; MPN MLCC-1uF-25V -> NTC-10k-0603
- LCAN1: renamed from LVS3; value FB-470R -> ACT45B-101-2P-TL003; footprint FB0603 -> CMC1210; symbol traction-r1:L -> traction-r1:ACT45B-101-2P-TL003; MPN FB-470R-CLASS -> ACT45B-101-2P-TL003
- LCAN2: renamed from RHWP; value 10k -> ACT45B-101-2P-TL003; footprint R0603 -> CMC1210; symbol traction-r1:R -> traction-r1:ACT45B-101-2P-TL003; MPN R0603-10k-1% -> ACT45B-101-2P-TL003
- LCOR: renamed from RIGN1; value 5.1k -> XAL4020-222MEC; footprint R0603 -> XAL4020; symbol traction-r1:R -> traction-r1:L; MPN R0603-5k1 -> XAL4020-222MEC
- LFC: renamed from CSB6; value 4.7uF -> FB-120R-3A; footprint C0805 -> FB1206; symbol traction-r1:C -> traction-r1:L; MPN MLCC-CLASS -> FB-120R-3A
- LSBC: renamed from RIGN2; value 10k -> XAL4040-103MEC; footprint R0603 -> XAL4040; symbol traction-r1:R -> traction-r1:L; MPN R0603-10k -> XAL4040-103MEC
- renumbered CMD9 to CMD1, RIGNS2 to RDBG, RLAT1 to RFLTD, RWB1 to RUB3
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Connections:
- net labels added: ASC_CMD_RB, DRV_EN_RB, FLT_CLR_B, FLT_OKB, FOUT_K, FS0B_B
- wire segments 803 -> 825
Other:
- note added: "rev A.7 - 26 sections - 262 components"
- note removed: "rev A.6 - 26 sections - 255 components"
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