File: kicad5/traction/traction-card.sch (KiCad schematic (older format))
At the start: 262 parts, among them Y1 CX3225GA40000D0PTVCC

Commit message: Rev A.8: review round 8 response (R7-01..07, A7-N01..05) + cross-check
Review round 8 on 2ac42ed, every finding verified and classified in
docs/review-A8-disposition.md (+ .csv); findings log F90-F105.

Hardware (+Rs18/unit: SiC Rs71,040, IGBT Rs45,540):
- UASCG 74LVC1G08-Q100: ASC_CMD = ASC latch AND no driver FLT, so a
  latched DESAT drops ASC on every path, FS1B included (R7-01/A7-N01;
  NSI6611 DS Fig. 8.11 read directly)
- USCH2 74LVC3G17-Q100 buffers both latch presets and drives QDIS_CMD;
  FLT diode-OR now BAT46 for the Schmitt threshold (R7-02, R7-03, N12)
- ZSET BZT52-B5V6 to ground replaces the clamp into V5A; RENP2 removed
  (A7-N04; B5V6 keeps a 35 V load dump under the 6.5 V V_I abs max)
- RASCL = RQDL = 261 R: both TLP152 LEDs 10.3-14.8 mA, inside 10-15 mA
- dead-state pulls: RFCB on FLT_CMB_B, RASCP moved to ASC_Q
- CFLTF2 100 pF on FLT_LS_N; discharge header V15-GND-CMD-GND

Firmware contract: FW-15 always clears the ASC latch; FW-16 runs on
measured no-HV/standstill conditions (stored-pass arming otherwise),
handles the FS_GPIO1 flyback OR and injects FLT from the MCU pins;
FW-08b; FS1B_TDELAY = 0, TDUR = 100 ms; FAULT_OUT outcomes stated.

Tooling: ERC locks by net, pin number and first-match MPN per SKU
(864 checks, each new one mutation-tested); computed judges replace
fixed PASS rows; S4 static junction path + static-plate bound; VCC2
FB-sense per corner; bom-gen publishes atomically, rounds ext prices.

Gates: pins 1782/1782, ERC 864/0, design-verify 108P/14W/0F,
sim-verify 23P/6W/0F, marine 81P/19W/0F.

Co-Authored-By: Claude Opus 5.5 <noreply@anthropic.com>
Parts:
- added JICC: MICROFIT3-40, MicroFit40, symbol traction-r1:MICROFIT3-40
- added RCPD0, RCPD1, RCPD2, RCPD3, RHWP: 10k, R0603, symbol traction-r1:R
- CAND2: renamed from CCLR; value 15nF -> 100nF; MPN MLCC-15nF-50V-C0G -> MLCC-CLASS
- CASCG: renamed from RFS1; value 1k -> 100nF; footprint R0603 -> C0603; symbol traction-r1:R -> traction-r1:C; MPN R0603-1k -> MLCC-100nF-16V
- CCAN1: renamed from UCAN2; value TCAN1042HGVDRQ1 -> 1uF; footprint SOIC8 -> C0603; symbol traction-r1:TCAN1042HGVDRQ1 -> traction-r1:C; LCSC C132550 -> CLASS; MPN TCAN1042HGVDRQ1 -> MLCC-1uF-25V
- CCAN2: renamed from LVS1; value FB-470R -> 1uF; footprint FB0603 -> C0603; symbol traction-r1:L -> traction-r1:C; MPN FB-470R-CLASS -> MLCC-1uF-25V
- CCLR: renamed from CFLTD; value 3.3nF -> 15nF; MPN MLCC-3.3nF-50V-C0G -> MLCC-15nF-50V-C0G
- CCOSA1: renamed from RCOSF1; value 330R -> 100pF; footprint R0603 -> C0603; symbol traction-r1:R -> traction-r1:C; MPN R0603-CLASS -> MLCC-CLASS
- CCOSA2: renamed from RCOSF2; value 330R -> 2.2nF; footprint R0603 -> C0603; symbol traction-r1:R -> traction-r1:C; MPN R0603-CLASS -> MLCC-CLASS
- CCOSD: renamed from RCOSR1; value 120R -> 220pF; footprint R0603 -> C0603; symbol traction-r1:R -> traction-r1:C; MPN R0603-120R -> MLCC-CLASS
- CCOSF: renamed from RCOSR2; value 120R -> 22pF; footprint R0603 -> C0603; symbol traction-r1:R -> traction-r1:C; MPN R0603-120R -> MLCC-CLASS
- CCT1: renamed from CCAN2; value 1uF -> 4.7nF; MPN MLCC-1uF-25V -> MLCC-4.7nF-50V
- CCT2: renamed from LVS2; value FB-470R -> 4.7nF; footprint FB0603 -> C0603; symbol traction-r1:L -> traction-r1:C; MPN FB-470R-CLASS -> MLCC-4.7nF-50V
- CEXA1: renamed from REXA1; value 3k -> 4.7nF; footprint R0603 -> C0603; symbol traction-r1:R -> traction-r1:C; MPN R0603-CLASS -> MLCC-CLASS
- CEXA2: renamed from REXA2; value 10k -> 300pF; footprint R0603 -> C0603; symbol traction-r1:R -> traction-r1:C; MPN R0603-CLASS -> MLCC-CLASS
- CEXA3: renamed from REXA3; value 10k -> 100nF; footprint R0603 -> C0603; symbol traction-r1:R -> traction-r1:C; MPN R0603-CLASS -> MLCC-CLASS
- CEXD: renamed from REXA4; value 24k -> 4.7uF; footprint R0603 -> C0603; symbol traction-r1:R -> traction-r1:C; MPN R0603-CLASS -> MLCC-CLASS
- CFLTD: renamed from CFLTF; value 100pF -> 3.3nF; MPN MLCC-100pF-16V -> MLCC-3.3nF-50V-C0G
- CFLTF: renamed from CLAT2; value 100nF -> 100pF; MPN MLCC-100nF-16V -> MLCC-100pF-16V
- CFLTF2: renamed from CSCH; value 100nF -> 100pF; MPN MLCC-100nF-16V -> MLCC-100pF-16V
- CILK: renamed from UVMB2; value OPA348AQDBVRQ1 -> 2.2nF; footprint SOT23-5 -> C0603; symbol traction-r1:OPA348AQDBVRQ1 -> traction-r1:C; LCSC C2877787 -> CLASS; MPN OPA348AQDBVRQ1 -> MLCC-2.2nF-50V
- CLAT: renamed from RFS2; value 10k -> 100nF; footprint R0603 -> C0603; symbol traction-r1:R -> traction-r1:C; MPN R0603-10k -> MLCC-100nF-16V
- CLAT2: renamed from DCLR; value BAT46ZFILM -> 100nF; footprint SOD123 -> C0603; symbol traction-r1:D -> traction-r1:C; LCSC C283255 -> CLASS; MPN BAT46ZFILM -> MLCC-100nF-16V
- CLDE: renamed from REXB1; value 24k -> 22uF; footprint R0603 -> C0603; symbol traction-r1:R -> traction-r1:C; MPN R0603-CLASS -> MLCC-CLASS
- CLDEC: renamed from REXB2; value 24k -> 270pF; footprint R0603 -> C0603; symbol traction-r1:R -> traction-r1:C; MPN R0603-CLASS -> MLCC-CLASS
- CMT1F: renamed from RMT2P; value 10k -> 47nF; footprint R0603 -> C0603; symbol traction-r1:R -> traction-r1:C; MPN R0603-CLASS -> MLCC-47nF-25V
- CMT2F: renamed from RMT2S; value 1k -> 47nF; footprint R0603 -> C0603; symbol traction-r1:R -> traction-r1:C; MPN R0603-CLASS -> MLCC-47nF-25V
- COF1: renamed from RVD1C; value 10k -> 100nF; footprint R0603 -> C0603; symbol traction-r1:R -> traction-r1:C; MPN R0603-10k-0.1% -> MLCC-CLASS
- COR1: renamed from RILK4; value 10k -> 100nF; footprint R0603 -> C0603; symbol traction-r1:R -> traction-r1:C; MPN R0603-10k -> MLCC-CLASS
- COR2: renamed from UVMB1; value OPA348AQDBVRQ1 -> 100nF; footprint SOT23-5 -> C0603; symbol traction-r1:OPA348AQDBVRQ1 -> traction-r1:C; LCSC C2877787 -> CLASS; MPN OPA348AQDBVRQ1 -> MLCC-CLASS
- CSCH: renamed from DFLT1; value 1N4148WS -> 100nF; footprint SOD323 -> C0603; symbol traction-r1:D -> traction-r1:C; LCSC C2128 -> CLASS; MPN 1N4148WS -> MLCC-100nF-16V
- CSCH2: renamed from DFLT2; value 1N4148WS -> 100nF; footprint SOD323 -> C0603; symbol traction-r1:D -> traction-r1:C; LCSC C2128 -> CLASS; MPN 1N4148WS -> MLCC-100nF-16V
- CSINA1: renamed from RSINF1; value 330R -> 100pF; footprint R0603 -> C0603; symbol traction-r1:R -> traction-r1:C; MPN R0603-CLASS -> MLCC-CLASS
- CSINA2: renamed from RSINF2; value 330R -> 2.2nF; footprint R0603 -> C0603; symbol traction-r1:R -> traction-r1:C; MPN R0603-CLASS -> MLCC-CLASS
- CSIND: renamed from RSINR1; value 120R -> 220pF; footprint R0603 -> C0603; symbol traction-r1:R -> traction-r1:C; MPN R0603-120R -> MLCC-CLASS
- CSINF: renamed from RSINR2; value 120R -> 22pF; footprint R0603 -> C0603; symbol traction-r1:R -> traction-r1:C; MPN R0603-120R -> MLCC-CLASS
- CSNUF: renamed from RTMR; value 0R -> 47nF; footprint R0603 -> C0603; symbol traction-r1:R -> traction-r1:C; MPN R0603-CLASS -> MLCC-47nF-25V
- CTAMBF: renamed from UMT1; value OPA333AQDBVRQ1 -> 47nF; footprint SOT23-5 -> C0603; symbol traction-r1:OPA333AQDBVRQ1 -> traction-r1:C; LCSC C2058544 -> CLASS; MPN OPA333AQDBVRQ1 -> MLCC-47nF-25V
- CTHSF: renamed from UMT2; value OPA333AQDBVRQ1 -> 47nF; footprint SOT23-5 -> C0603; symbol traction-r1:OPA333AQDBVRQ1 -> traction-r1:C; LCSC C2058544 -> CLASS; MPN OPA333AQDBVRQ1 -> MLCC-47nF-25V
- CUB1: renamed from RUB2; value 100R -> 3.3nF; footprint R0603 -> C0603; symbol traction-r1:R -> traction-r1:C; MPN R0603-100R -> MLCC-3.3nF-50V
- CUB2: renamed from RUB3; value 100R -> 100nF; footprint R0603 -> C0603; symbol traction-r1:R -> traction-r1:C; MPN R0603-100R -> MLCC-100nF-25V
- CUS1: renamed from UVB1; value OPA376AQDBVRQ1 -> 47nF; footprint SOT23-5 -> C0603; symbol traction-r1:OPA376AQDBVRQ1 -> traction-r1:C; MPN OPA376AQDBVRQ1 -> MLCC-47nF-25V
- CUS2: renamed from UVB2; value OPA376AQDBVRQ1 -> 4.7nF; footprint SOT23-5 -> C0603; symbol traction-r1:OPA376AQDBVRQ1 -> traction-r1:C; MPN OPA376AQDBVRQ1 -> MLCC-4.7nF-50V
- CVB1: renamed from RVB2; value 100R -> 3.3nF; footprint R0603 -> C0603; symbol traction-r1:R -> traction-r1:C; MPN R0603-100R -> MLCC-3.3nF-50V
- CVB2: renamed from RVB3; value 100R -> 100nF; footprint R0603 -> C0603; symbol traction-r1:R -> traction-r1:C; MPN R0603-100R -> MLCC-100nF-25V
- CVD1: renamed from RVD1D; value 10k -> 100pF; footprint R0603 -> C0603; symbol traction-r1:R -> traction-r1:C; MPN R0603-10k-0.1% -> MLCC-CLASS
- CVD2: renamed from CSNVF; value 47nF -> 100pF; MPN MLCC-47nF-25V -> MLCC-CLASS
- CVM1: renamed from UEXD; value ALM2402QPWPRQ1 -> 220nF; footprint HTSSOP16 -> C0603; symbol traction-r1:ALM2402QPWPRQ1 -> traction-r1:C; LCSC C544754 -> CLASS; MPN ALM2402QPWPRQ1 -> MLCC-CLASS
- CVM2: renamed from UEXF; value OPA348AQDBVRQ1 -> 220nF; footprint SOT23-5 -> C0603; symbol traction-r1:OPA348AQDBVRQ1 -> traction-r1:C; LCSC C2877787 -> CLASS; MPN OPA348AQDBVRQ1 -> MLCC-CLASS
- CVS1: renamed from UWB1; value OPA376AQDBVRQ1 -> 47nF; footprint SOT23-5 -> C0603; symbol traction-r1:OPA376AQDBVRQ1 -> traction-r1:C; MPN OPA376AQDBVRQ1 -> MLCC-47nF-25V
- CVS2: renamed from UWB2; value OPA376AQDBVRQ1 -> 4.7nF; footprint SOT23-5 -> C0603; symbol traction-r1:OPA376AQDBVRQ1 -> traction-r1:C; MPN OPA376AQDBVRQ1 -> MLCC-4.7nF-50V
- CWB1: renamed from RWB2; value 100R -> 3.3nF; footprint R0603 -> C0603; symbol traction-r1:R -> traction-r1:C; MPN R0603-100R -> MLCC-3.3nF-50V
- CWB2: renamed from RWB3; value 100R -> 100nF; footprint R0603 -> C0603; symbol traction-r1:R -> traction-r1:C; MPN R0603-100R -> MLCC-100nF-25V
- CWS1: renamed from UVD1; value OPA376AQDBVRQ1 -> 47nF; footprint SOT23-5 -> C0603; symbol traction-r1:OPA376AQDBVRQ1 -> traction-r1:C; MPN OPA376AQDBVRQ1 -> MLCC-47nF-25V
- CWS2: renamed from UVOF; value OPA376AQDBVRQ1 -> 4.7nF; footprint SOT23-5 -> C0603; symbol traction-r1:OPA376AQDBVRQ1 -> traction-r1:C; MPN OPA376AQDBVRQ1 -> MLCC-4.7nF-50V
- DCLR: renamed from RDRB; value 10k -> BAT46ZFILM; footprint R0603 -> SOD123; symbol traction-r1:R -> traction-r1:D; LCSC CLASS -> C283255; MPN R0603-10k -> BAT46ZFILM
- DCOSP: renamed from RCOS2; value 680R -> PESD2IVN24-T; footprint R0603 -> SOT23; symbol traction-r1:R -> traction-r1:PESD2IVN24-T; LCSC CLASS -> C406047; MPN R0603-CLASS -> PESD2IVN24-T
- DFLT1: renamed from RENP1; value 5.1k -> BAT46ZFILM; footprint R0603 -> SOD123; symbol traction-r1:R -> traction-r1:D; LCSC CLASS -> C283255; MPN R0603-5k1 -> BAT46ZFILM
- DFLT2: renamed from RENP2; value 5.1k -> BAT46ZFILM; footprint R0603 -> SOD123; symbol traction-r1:R -> traction-r1:D; LCSC CLASS -> C283255; MPN R0603-5k1 -> BAT46ZFILM
- DFO: renamed from RFS3; value 1k -> BAT46ZFILM; footprint R0603 -> SOD123; symbol traction-r1:R -> traction-r1:D; LCSC CLASS -> C283255; MPN R0603-1k -> BAT46ZFILM
- DSINP: renamed from RSIN2; value 680R -> PESD2IVN24-T; footprint R0603 -> SOT23; symbol traction-r1:R -> traction-r1:PESD2IVN24-T; LCSC CLASS -> C406047; MPN R0603-CLASS -> PESD2IVN24-T
- FMT1: renamed from TVSM1; value PESD5V0L1BA -> FUSE-350mA-0603; footprint SOD323 -> F0603; symbol traction-r1:R -> traction-r1:F; MPN PESD5V0L1BA -> FUSE-350mA-0603
- FMT2: renamed from TVSM2; value PESD5V0L1BA -> FUSE-350mA-0603; footprint SOD323 -> F0603; symbol traction-r1:R -> traction-r1:F; MPN PESD5V0L1BA -> FUSE-350mA-0603
- FVS1: renamed from RCPD0; value 10k -> MF-LSMF; footprint R0603 -> PTC1206; symbol traction-r1:R -> traction-r1:F; MPN R0603-10k -> MF-LSMF-CLASS
- JLEM: renamed from CUB1; value 3.3nF -> T2M-105-01-L-D-TH-WT; footprint C0603 -> HDR2x5; symbol traction-r1:C -> traction-r1:T2M-105-01-L-D-TH-WT; MPN MLCC-3.3nF-50V -> T2M-105-01-L-D-TH-WT
- JTAMB: renamed from CMT1F; value 47nF -> NTC-10k-0603; footprint C0603 -> R0603; symbol traction-r1:C -> traction-r1:J2; MPN MLCC-47nF-25V -> NTC-10k-0603
- JTHS: renamed from CMT2F; value 47nF -> NTC-10k-0603; footprint C0603 -> R0603; symbol traction-r1:C -> traction-r1:J2; MPN MLCC-47nF-25V -> NTC-10k-0603
- JVEH: renamed from JICC; value MICROFIT3-40 -> TE 770669-1 (AMPSEAL 23); footprint MicroFit40 -> AMPSEAL23; symbol traction-r1:MICROFIT3-40 -> traction-r1:TE_770669-1__AMPSEAL_23_; MPN MICROFIT3-40 -> TE 770669-1 (AMPSEAL 23)
- LCAN1: renamed from RCT1B; value 60.4R -> ACT45B-101-2P-TL003; footprint R0603 -> CMC1210; symbol traction-r1:R -> traction-r1:ACT45B-101-2P-TL003; MPN R0603-60R4-1% -> ACT45B-101-2P-TL003
- LCAN2: renamed from RCT2B; value 60.4R -> ACT45B-101-2P-TL003; footprint R0603 -> CMC1210; symbol traction-r1:R -> traction-r1:ACT45B-101-2P-TL003; MPN R0603-60R4-1% -> ACT45B-101-2P-TL003
- LUB: renamed from CVB1; value 3.3nF -> FB-220R-1A; footprint C0603 -> FB0805; symbol traction-r1:C -> traction-r1:L; MPN MLCC-3.3nF-50V -> FB-220R-1A
- LVB: renamed from CWB1; value 3.3nF -> FB-220R-1A; footprint C0603 -> FB0805; symbol traction-r1:C -> traction-r1:L; MPN MLCC-3.3nF-50V -> FB-220R-1A
- LVS1: renamed from RCPD1; value 10k -> FB-470R; footprint R0603 -> FB0603; symbol traction-r1:R -> traction-r1:L; MPN R0603-10k -> FB-470R-CLASS
- LVS2: renamed from RCPD2; value 10k -> FB-470R; footprint R0603 -> FB0603; symbol traction-r1:R -> traction-r1:L; MPN R0603-10k -> FB-470R-CLASS
- LVS3: renamed from RCPD3; value 10k -> FB-470R; footprint R0603 -> FB0603; symbol traction-r1:R -> traction-r1:L; MPN R0603-10k -> FB-470R-CLASS
- LVS4: renamed from RHWP; value 10k -> FB-470R; footprint R0603 -> FB0603; symbol traction-r1:R -> traction-r1:L; MPN R0603-10k-1% -> FB-470R-CLASS
- LWB: renamed from COF1; value 100nF -> FB-220R-1A; footprint C0603 -> FB0805; symbol traction-r1:C -> traction-r1:L; MPN MLCC-CLASS -> FB-220R-1A
- RARB: renamed from RFS4; value 1k -> 10k; MPN R0603-1k -> R0603-10k
- renumbered CAND2 to CAND1, CTAMBF to CSNVF, CTHSF to CSNWF, RLAT1 to RASCP, RCT2A to RCT1B, REXM4 to REXB2, RGPD to RFLTD, RRDYP1 to RFLTP2, RVD2A to RVD1A, RVD2B to RVD1B, RVD2C to RVD1C, RVD2D to RVD1D
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Connections:
- net labels added: ASC_Q, ASC_SET_B, FLT_CMB_B, QDIS_M
- wire segments 825 -> 846
Other:
- note added: "rev A.8 - 26 sections - 268 components"
- note removed: "rev A.7 - 26 sections - 262 components"
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
Commit message: Rev A.9: review round 9 response (A8-01..03, A8-N01..N03) + cross-check
Review round 9 on 0da9014, every finding verified and classified in
docs/review-A9-disposition.md (+ .csv, 34 items); findings log F106-F119.

Hardware (+Rs29/unit: SiC Rs71,069, IGBT Rs45,569):
- PSASC/PSQD bound to the real QA01C-18 sheet (+18/-3 V; F61 had read
  the base QA01C, +20/-4 V): envelope 16.9-20.9 V, ASC entry 7.52 us,
  FW-06 end-point 906 V; discharge gate divider RQDG 1.5k (Vgs 13.4-18.1 V)
- FLT/RDY pull-ups and the diode-OR pull-up moved to V5GD (the drivers'
  VCC1; FLT/RDY abs max = VCC1), V5GD read by the MCU on PTB5
- HARNESS40 re-laid: VBAT and V5GD touch only ground in both row-by-row
  and odd/even dual-row numbering; connector family chosen at layout
- self-found: the power board's LV side ran on unswitched KL30
  (~150 mA parked) - card-side P-FET switch DMP6023LEQ on V5A with a
  slew network; resolver LDO enabled by V5A; parking drain <= 43 uA
- RFS4 = ROHM ESR03 anti-surge; CASC/CQD 50 V

Firmware contract: FW-16 energy-limited eligibility (read < 3 V or QDIS
for 2 tau); V_DC invalid while V5GD is out of window; DESATs to NVM;
BACKUP_SAFETY_PATH_FS1B = 0; motor/vehicle release rule for SPO energy.

Gates: pins 1804/1804, ERC 883/0 (new locks mutation-tested),
design-verify 116P/14W/0F, sim-verify 23P/6W/0F, marine 81P/19W/0F.

Co-Authored-By: Claude Opus 5.5 <noreply@anthropic.com>
Parts:
- added JICC: HARNESS-2x20, MicroFit40, symbol traction-r1:HARNESS-2x20-CLASS
- added LVS2, LVS3, LVS4: FB-470R, FB0603, symbol traction-r1:L
- added RCPD0, RCPD1, RCPD2, RCPD3, RHWP: 10k, R0603, symbol traction-r1:R
- CAND1: renamed from CSCH; MPN MLCC-100nF-16V -> MLCC-CLASS
- CAND2: renamed from CSCH2; MPN MLCC-100nF-16V -> MLCC-CLASS
- CASCG: renamed from RLAT1; value 10k -> 100nF; footprint R0603 -> C0603; symbol traction-r1:R -> traction-r1:C; MPN R0603-10k -> MLCC-100nF-16V
- CBTC: renamed from CSB5; value 2.2uF -> 47nF; footprint C0805 -> C0603
- CBTP: renamed from CSB6; value 4.7uF -> 22nF; footprint C0805 -> C0603
- CCAN1: renamed from RCT2A; value 60.4R -> 1uF; footprint R0603 -> C0603; symbol traction-r1:R -> traction-r1:C; MPN R0603-60R4-1% -> MLCC-1uF-25V
- CCAN2: renamed from LVS4; value FB-470R -> 1uF; footprint FB0603 -> C0603; symbol traction-r1:L -> traction-r1:C; MPN FB-470R-CLASS -> MLCC-1uF-25V
- CCLR: renamed from DCLR; value BAT46ZFILM -> 15nF; footprint SOD123 -> C0603; symbol traction-r1:D -> traction-r1:C; LCSC C283255 -> CLASS; MPN BAT46ZFILM -> MLCC-15nF-50V-C0G
- CCOSA1: renamed from RCOSR2; value 120R -> 100pF; footprint R0603 -> C0603; symbol traction-r1:R -> traction-r1:C; MPN R0603-120R -> MLCC-CLASS
- CCOSA2: renamed from JLEM; value T2M-105-01-L-D-TH-WT -> 2.2nF; footprint HDR2x5 -> C0603; symbol traction-r1:T2M-105-01-L-D-TH-WT -> traction-r1:C; MPN T2M-105-01-L-D-TH-WT -> MLCC-CLASS
- CCOSD: renamed from USNSU; value HC5FW900-S -> 220pF; footprint OffBoard -> C0603; symbol traction-r1:HC5FW900-S -> traction-r1:C; MPN HC5FW900-S -> MLCC-CLASS
- CCOSF: renamed from USNSV; value HC5FW900-S -> 22pF; footprint OffBoard -> C0603; symbol traction-r1:HC5FW900-S -> traction-r1:C; MPN HC5FW900-S -> MLCC-CLASS
- CCT1: renamed from RCT2B; value 60.4R -> 4.7nF; footprint R0603 -> C0603; symbol traction-r1:R -> traction-r1:C; MPN R0603-60R4-1% -> MLCC-4.7nF-50V
- CCT2: renamed from JICC; value MICROFIT3-40 -> 4.7nF; footprint MicroFit40 -> C0603; symbol traction-r1:MICROFIT3-40 -> traction-r1:C; MPN MICROFIT3-40 -> MLCC-4.7nF-50V
- CEXA1: renamed from REXA4; value 24k -> 4.7nF; footprint R0603 -> C0603; symbol traction-r1:R -> traction-r1:C; MPN R0603-CLASS -> MLCC-CLASS
- CEXA2: renamed from REXB1; value 24k -> 300pF; footprint R0603 -> C0603; symbol traction-r1:R -> traction-r1:C; MPN R0603-CLASS -> MLCC-CLASS
- CEXA3: renamed from REXB2; value 24k -> 100nF; footprint R0603 -> C0603; symbol traction-r1:R -> traction-r1:C; MPN R0603-CLASS -> MLCC-CLASS
- CEXD: renamed from REXB3; value 24k -> 4.7uF; footprint R0603 -> C0603; symbol traction-r1:R -> traction-r1:C; MPN R0603-CLASS -> MLCC-CLASS
- CFLTD: renamed from DFLT1; value BAT46ZFILM -> 3.3nF; footprint SOD123 -> C0603; symbol traction-r1:D -> traction-r1:C; LCSC C283255 -> CLASS; MPN BAT46ZFILM -> MLCC-3.3nF-50V-C0G
- CFLTF: renamed from DFLT2; value BAT46ZFILM -> 100pF; footprint SOD123 -> C0603; symbol traction-r1:D -> traction-r1:C; LCSC C283255 -> CLASS; MPN BAT46ZFILM -> MLCC-100pF-16V
- CFLTF2: renamed from RDRB; value 10k -> 100pF; footprint R0603 -> C0603; symbol traction-r1:R -> traction-r1:C; MPN R0603-10k -> MLCC-100pF-16V
- CIGN: renamed from UAND1; value 74LVC1G11GW-Q100 -> 100nF; footprint SOT363 -> C0603; symbol traction-r1:74LVC1G11GW-Q100 -> traction-r1:C; LCSC C548242 -> CLASS; MPN 74LVC1G11GW-Q100 -> MLCC-100nF-50V
- CIGNS: renamed from UAND2; value 74LVC1G11GW-Q100 -> 100nF; footprint SOT363 -> C0603; symbol traction-r1:74LVC1G11GW-Q100 -> traction-r1:C; LCSC C548242 -> CLASS; MPN 74LVC1G11GW-Q100 -> MLCC-CLASS
- CILK: renamed from RVM1; value 24k -> 2.2nF; footprint R0603 -> C0603; symbol traction-r1:R -> traction-r1:C; MPN R0603-24k-1% -> MLCC-2.2nF-50V
- CLAT: renamed from ZSET; value BZT52-B5V6 -> 100nF; footprint SOD123 -> C0603; symbol traction-r1:D -> traction-r1:C; MPN BZT52-B5V6 -> MLCC-100nF-16V
- CLAT2: renamed from RENP1; value 5.1k -> 100nF; footprint R0603 -> C0603; symbol traction-r1:R -> traction-r1:C; MPN R0603-5k1 -> MLCC-100nF-16V
- CLDE: renamed from REXB4; value 24k -> 22uF; footprint R0603 -> C0603; symbol traction-r1:R -> traction-r1:C; MPN R0603-CLASS -> MLCC-CLASS
- CLDEC: renamed from REXM1; value 5.1k -> 270pF; footprint R0603 -> C0603; symbol traction-r1:R -> traction-r1:C; MPN R0603-CLASS -> MLCC-CLASS
- CLVC1: renamed from DREVC; value STPS5L60S -> 4.7uF; footprint SMC -> C1206; symbol traction-r1:D -> traction-r1:C; LCSC C140620 -> CLASS; MPN STPS5L60S -> MLCC-4.7uF-50V
- CLVC2: renamed from DTVSC; value TPSMC24CA -> 22uF; footprint SMC -> C1210; symbol traction-r1:D -> traction-r1:C; LCSC C1975284 -> CLASS; MPN TPSMC24CA -> MLCC-22uF-50V
- CLVSM: renamed from FLVC; value MF-LSMF300/24X-2 -> 100nF; footprint PTC2920 -> C0603; symbol traction-r1:F -> traction-r1:C; LCSC C719172 -> CLASS; MPN MF-LSMF300/24X-2 -> MLCC-100nF-50V
- CMT1F: renamed from TVSM2; value PESD5V0L1BA -> 47nF; footprint SOD323 -> C0603; symbol traction-r1:R -> traction-r1:C; MPN PESD5V0L1BA -> MLCC-47nF-25V
- CMT2F: renamed from LCAN1; value ACT45B-101-2P-TL003 -> 47nF; footprint CMC1210 -> C0603; symbol traction-r1:ACT45B-101-2P-TL003 -> traction-r1:C; MPN ACT45B-101-2P-TL003 -> MLCC-47nF-25V
- COF1: renamed from CVD2; value 100pF -> 100nF
- COR1: renamed from CVM1; value 220nF -> 100nF
- COR2: renamed from CVM2; value 220nF -> 100nF
- CSB1: renamed from CSB7; value 10uF -> 22uF
- CSB2: renamed from CSB8; value 10uF -> 22uF
- CSB3: renamed from CVBOS; value 4.7uF -> 22uF; footprint C0603 -> C0805
- CSB3B: renamed from CVDIG; value 1uF -> 22uF
- CSB4: renamed from DBAT; value BAT46ZFILM -> 10uF; footprint SOD123 -> C0805; symbol traction-r1:D -> traction-r1:C; LCSC C283255 -> CLASS; MPN BAT46ZFILM -> MLCC-CLASS
- CSB5: renamed from LCOR; value XAL4020-222MEC -> 2.2uF; footprint XAL4020 -> C0805; symbol traction-r1:L -> traction-r1:C; MPN XAL4020-222MEC -> MLCC-CLASS
- CSB6: renamed from LSBC; value XAL4040-103MEC -> 4.7uF; footprint XAL4040 -> C0805; symbol traction-r1:L -> traction-r1:C; MPN XAL4040-103MEC -> MLCC-CLASS
- CSB7: renamed from RAGT; value 0R -> 10uF; footprint R0603 -> C0805; symbol traction-r1:R -> traction-r1:C; MPN R0603-CLASS -> MLCC-CLASS
- CSB8: renamed from RDBG; value 10k -> 10uF; footprint R0603 -> C0805; symbol traction-r1:R -> traction-r1:C; MPN R0603-CLASS -> MLCC-CLASS
- CSCH: renamed from RFCB; value 100k -> 100nF; footprint R0603 -> C0603; symbol traction-r1:R -> traction-r1:C; MPN R0603-100k -> MLCC-100nF-16V
- CSCH2: renamed from RFLTC; value 10k -> 100nF; footprint R0603 -> C0603; symbol traction-r1:R -> traction-r1:C; MPN R0603-CLASS -> MLCC-100nF-16V
- CSINA1: renamed from RSINR2; value 120R -> 100pF; footprint R0603 -> C0603; symbol traction-r1:R -> traction-r1:C; MPN R0603-120R -> MLCC-CLASS
- CSINA2: renamed from DCOSP; value PESD2IVN24-T -> 2.2nF; footprint SOT23 -> C0603; symbol traction-r1:PESD2IVN24-T -> traction-r1:C; LCSC C406047 -> CLASS; MPN PESD2IVN24-T -> MLCC-CLASS
- CSIND: renamed from CCOSA1; value 100pF -> 220pF
- CSINF: renamed from CCOSA2; value 2.2nF -> 22pF
- CSNUF: renamed from JTAMB; value NTC-10k-0603 -> 47nF; footprint R0603 -> C0603; symbol traction-r1:J2 -> traction-r1:C; MPN NTC-10k-0603 -> MLCC-47nF-25V
- CSNVF: renamed from JTHS; value NTC-10k-0603 -> 47nF; footprint R0603 -> C0603; symbol traction-r1:J2 -> traction-r1:C; MPN NTC-10k-0603 -> MLCC-47nF-25V
- CSNWF: renamed from RTAMBP; value 10k -> 47nF; footprint R0603 -> C0603; symbol traction-r1:R -> traction-r1:C; MPN R0603-10k-1% -> MLCC-47nF-25V
- CTHSF: renamed from FMT1; value FUSE-350mA-0603 -> 47nF; footprint F0603 -> C0603; symbol traction-r1:F -> traction-r1:C; MPN FUSE-350mA-0603 -> MLCC-47nF-25V
- CUB1: renamed from UVB2; value OPA376AQDBVRQ1 -> 3.3nF; footprint SOT23-5 -> C0603; symbol traction-r1:OPA376AQDBVRQ1 -> traction-r1:C; MPN OPA376AQDBVRQ1 -> MLCC-3.3nF-50V
- CUB2: renamed from CVB1; value 3.3nF -> 100nF; MPN MLCC-3.3nF-50V -> MLCC-100nF-25V
- CUS1: renamed from CVB2; value 100nF -> 47nF; MPN MLCC-100nF-25V -> MLCC-47nF-25V
- CUS2: renamed from CVS1; value 47nF -> 4.7nF; MPN MLCC-47nF-25V -> MLCC-4.7nF-50V
- CVB1: renamed from UWB2; value OPA376AQDBVRQ1 -> 3.3nF; footprint SOT23-5 -> C0603; symbol traction-r1:OPA376AQDBVRQ1 -> traction-r1:C; MPN OPA376AQDBVRQ1 -> MLCC-3.3nF-50V
- CVB2: renamed from CWB1; value 3.3nF -> 100nF; MPN MLCC-3.3nF-50V -> MLCC-100nF-25V
- CVBOS: renamed from RSB1; value 52.3k -> 4.7uF; footprint R0603 -> C0603; symbol traction-r1:R -> traction-r1:C; MPN R0603-CLASS -> MLCC-CLASS
- CVD1: renamed from RVD2A; value 10k -> 100pF; footprint R0603 -> C0603; symbol traction-r1:R -> traction-r1:C; MPN R0603-10k-0.1% -> MLCC-CLASS
- CVD2: renamed from RSNVP; value 5.1k -> 100pF; footprint R0603 -> C0603; symbol traction-r1:R -> traction-r1:C; MPN R0603-5k1-1% -> MLCC-CLASS
- CVDIG: renamed from RSB2; value 10k -> 1uF; footprint R0603 -> C0603; symbol traction-r1:R -> traction-r1:C; MPN R0603-CLASS -> MLCC-CLASS
- CVM1: renamed from CEXA1; value 4.7nF -> 220nF
- CVM2: renamed from CEXA2; value 300pF -> 220nF
- CVS1: renamed from CWB2; value 100nF -> 47nF; MPN MLCC-100nF-25V -> MLCC-47nF-25V
- CVS2: renamed from CWS1; value 47nF -> 4.7nF; MPN MLCC-47nF-25V -> MLCC-4.7nF-50V
- CWB1: renamed from UVOF; value OPA376AQDBVRQ1 -> 3.3nF; footprint SOT23-5 -> C0603; symbol traction-r1:OPA376AQDBVRQ1 -> traction-r1:C; MPN OPA376AQDBVRQ1 -> MLCC-3.3nF-50V
- CWB2: renamed from COF1; MPN MLCC-CLASS -> MLCC-100nF-25V
- CWS1: renamed from CVD1; value 100pF -> 47nF; MPN MLCC-CLASS -> MLCC-47nF-25V
- CWS2: renamed from ROF1; value 9.1k -> 4.7nF; footprint R0603 -> C0603; symbol traction-r1:R -> traction-r1:C; MPN R0603-CLASS -> MLCC-4.7nF-50V
- DBAT: renamed from RSB3; value 220R -> BAT46ZFILM; footprint R0603 -> SOD123; symbol traction-r1:R -> traction-r1:D; LCSC CLASS -> C283255; MPN R0603-CLASS -> BAT46ZFILM
- DCLR: renamed from RFLTD; value 10k -> BAT46ZFILM; footprint R0603 -> SOD123; symbol traction-r1:R -> traction-r1:D; LCSC CLASS -> C283255; MPN R0603-10k -> BAT46ZFILM
- DCOSP: renamed from RCOSR1; value 120R -> PESD2IVN24-T; footprint R0603 -> SOT23; symbol traction-r1:R -> traction-r1:PESD2IVN24-T; LCSC CLASS -> C406047; MPN R0603-120R -> PESD2IVN24-T
- DFLT1: renamed from RFLTP1; value 5.1k -> BAT46ZFILM; footprint R0603 -> SOD123; symbol traction-r1:R -> traction-r1:D; LCSC CLASS -> C283255; MPN R0603-5k1 -> BAT46ZFILM
- DFLT2: renamed from RFLTP2; value 5.1k -> BAT46ZFILM; footprint R0603 -> SOD123; symbol traction-r1:R -> traction-r1:D; LCSC CLASS -> C283255; MPN R0603-5k1 -> BAT46ZFILM
- DFO: renamed from UOR1; value 74LVC1G32GW-Q100 -> BAT46ZFILM; footprint SOT353 -> SOD123; symbol traction-r1:74LVC1G32GW-Q100 -> traction-r1:D; LCSC C548334 -> C283255; MPN 74LVC1G32GW-Q100 -> BAT46ZFILM
- DIGN: renamed from ULAT2; value 74LVC1G74DC-Q100 -> 1N4148WS; footprint VSSOP8 -> SOD323; symbol traction-r1:74LVC1G74DC-Q100 -> traction-r1:D; LCSC CLASS -> C2128; MPN 74LVC1G74DC-Q100 -> 1N4148WS
- DREVC: renamed from FVBH; value MF-LSMF300/24X-2 -> STPS5L60S; footprint PTC2920 -> SMC; symbol traction-r1:F -> traction-r1:D; LCSC C719172 -> C140620; MPN MF-LSMF300/24X-2 -> STPS5L60S
- DSINP: renamed from RSINR1; value 120R -> PESD2IVN24-T; footprint R0603 -> SOT23; symbol traction-r1:R -> traction-r1:PESD2IVN24-T; LCSC CLASS -> C406047; MPN R0603-120R -> PESD2IVN24-T
- DTVSC: renamed from FVBL; value MF-LSMF300/24X-2 -> TPSMC24CA; footprint PTC2920 -> SMC; symbol traction-r1:F -> traction-r1:D; LCSC C719172 -> C1975284; MPN MF-LSMF300/24X-2 -> TPSMC24CA
- FLVC: renamed from LFC; value FB-120R-3A -> MF-LSMF300/24X-2; footprint FB1206 -> PTC2920; symbol traction-r1:L -> traction-r1:F; LCSC CLASS -> C719172; MPN FB-120R-3A -> MF-LSMF300/24X-2
- FMT1: renamed from TVSC1; value PESD2IVN24-T -> FUSE-350mA-0603; footprint SOT23 -> F0603; symbol traction-r1:PESD2IVN24-T -> traction-r1:F; LCSC C406047 -> CLASS; MPN PESD2IVN24-T -> FUSE-350mA-0603
- renumbered CMT2F to CTAMBF, RGPD to RDRB, RILK3 to RLAT1, RVB1 to RUB2, RVB2 to RUB3, RWB1 to RVB2, RWB2 to RVB3, RVD2D to RVD1A, UVB1 to UUB2, UWB1 to UVB2, UEXF to UVMB1, UVD2 to UVOF, UVD1 to UWB2
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Connections:
- net labels added: LVS_D, LVS_G, LVS_M, V5GD, V5GD_SNS, VBSW
- wire segments 846 -> 868
Other:
- note added: "rev A.9 - 26 sections - 277 components"
- note removed: "rev A.8 - 26 sections - 268 components"
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
Commit message: Rev A.10: schematic rechecks of A.9 (A9-S01, S9-01, S9-02)
Two schematic-only rechecks of 7235337 kept every A.9 correction;
dispositioned in docs/review-A10-disposition.md (+ .csv); F120-F122.

- RDY_HS/RDY_LS now reach UAND1/UAND2 through a third 74LVC3G17-Q100
  (USCH3, RRDB dead-state pull-down): the open-drain lines rose at
  ~20-100 ns/V against the 74LVC1G11's 10 ns/V limit (A9-S01; reverses
  the round-7/8 "state-benign" rejection)
- RASCG = ROHM ESR03EZPF2201 (0.27 W at 85 C): it carries up to 0.12 W
  for as long as ASC is held; 2.2 k kept for the ASC timing (S9-01)
- discharge sheet note 66k bleeder; gate divider stated as 13.3-18.2 V
  (a divider, not a clamp); A9 disposition quotes the final harness map

+Rs11/unit (SiC Rs71,080, IGBT Rs45,580).
Gates: pins 1815/1815, ERC 891/0 (new locks mutation-tested),
design-verify 118P/14W/0F, sim-verify 23P/6W/0F, marine 81P/19W/0F.

Co-Authored-By: Claude Opus 5.5 <noreply@anthropic.com>
Parts:
- added RCPD2, RCPD3, RHWP: 10k, R0603, symbol traction-r1:R
- CAND2: renamed from CCLR; value 15nF -> 100nF; MPN MLCC-15nF-50V-C0G -> MLCC-CLASS
- CASCG: renamed from RARB; value 10k -> 100nF; footprint R0603 -> C0603; symbol traction-r1:R -> traction-r1:C; MPN R0603-10k -> MLCC-100nF-16V
- CCAN1: renamed from RCT1B; value 60.4R -> 1uF; footprint R0603 -> C0603; symbol traction-r1:R -> traction-r1:C; MPN R0603-60R4-1% -> MLCC-1uF-25V
- CCAN2: renamed from RCT2B; value 60.4R -> 1uF; footprint R0603 -> C0603; symbol traction-r1:R -> traction-r1:C; MPN R0603-60R4-1% -> MLCC-1uF-25V
- CCLR: renamed from CFLTD; value 3.3nF -> 15nF; MPN MLCC-3.3nF-50V-C0G -> MLCC-15nF-50V-C0G
- CCOSA1: renamed from CCOSF; value 22pF -> 100pF
- CCOSA2: renamed from RCOS1; value 680R -> 2.2nF; footprint R0603 -> C0603; symbol traction-r1:R -> traction-r1:C; MPN R0603-CLASS -> MLCC-CLASS
- CCOSD: renamed from RCOS2; value 680R -> 220pF; footprint R0603 -> C0603; symbol traction-r1:R -> traction-r1:C; MPN R0603-CLASS -> MLCC-CLASS
- CCOSF: renamed from RCOSF1; value 330R -> 22pF; footprint R0603 -> C0603; symbol traction-r1:R -> traction-r1:C; MPN R0603-CLASS -> MLCC-CLASS
- CCT1: renamed from LCAN2; value ACT45B-101-2P-TL003 -> 4.7nF; footprint CMC1210 -> C0603; symbol traction-r1:ACT45B-101-2P-TL003 -> traction-r1:C; MPN ACT45B-101-2P-TL003 -> MLCC-4.7nF-50V
- CCT2: renamed from JVEH; value TE 770669-1 (AMPSEAL 23) -> 4.7nF; footprint AMPSEAL23 -> C0603; symbol traction-r1:TE_770669-1__AMPSEAL_23_ -> traction-r1:C; MPN TE 770669-1 (AMPSEAL 23) -> MLCC-4.7nF-50V
- CEXA1: renamed from CEXD; value 4.7uF -> 4.7nF
- CEXA2: renamed from CLDE; value 22uF -> 300pF
- CEXA3: renamed from CLDEC; value 270pF -> 100nF
- CEXD: renamed from REXA1; value 3k -> 4.7uF; footprint R0603 -> C0603; symbol traction-r1:R -> traction-r1:C; MPN R0603-CLASS -> MLCC-CLASS
- CFLTD: renamed from CFLTF; value 100pF -> 3.3nF; MPN MLCC-100pF-16V -> MLCC-3.3nF-50V-C0G
- CFLTF2: renamed from CLAT2; value 100nF -> 100pF; MPN MLCC-100nF-16V -> MLCC-100pF-16V
- CILK: renamed from RILK3; value 10k -> 2.2nF; footprint R0603 -> C0603; symbol traction-r1:R -> traction-r1:C; MPN R0603-10k -> MLCC-2.2nF-50V
- CLAT: renamed from RASCP; value 10k -> 100nF; footprint R0603 -> C0603; symbol traction-r1:R -> traction-r1:C; MPN R0603-10k -> MLCC-100nF-16V
- CLDE: renamed from REXA2; value 10k -> 22uF; footprint R0603 -> C0603; symbol traction-r1:R -> traction-r1:C; MPN R0603-CLASS -> MLCC-CLASS
- CLDEC: renamed from REXA3; value 10k -> 270pF; footprint R0603 -> C0603; symbol traction-r1:R -> traction-r1:C; MPN R0603-CLASS -> MLCC-CLASS
- CMT1F: renamed from FMT2; value FUSE-350mA-0603 -> 47nF; footprint F0603 -> C0603; symbol traction-r1:F -> traction-r1:C; MPN FUSE-350mA-0603 -> MLCC-47nF-25V
- CMT2F: renamed from RMT1P; value 10k -> 47nF; footprint R0603 -> C0603; symbol traction-r1:R -> traction-r1:C; MPN R0603-CLASS -> MLCC-47nF-25V
- COF1: renamed from ROF2; value 1k -> 100nF; footprint R0603 -> C0603; symbol traction-r1:R -> traction-r1:C; MPN R0603-CLASS -> MLCC-CLASS
- COR1: renamed from RILK1; value 10k -> 100nF; footprint R0603 -> C0603; symbol traction-r1:R -> traction-r1:C; MPN R0603-10k -> MLCC-CLASS
- COR2: renamed from RILK2; value 10k -> 100nF; footprint R0603 -> C0603; symbol traction-r1:R -> traction-r1:C; MPN R0603-10k -> MLCC-CLASS
- CSCH2: renamed from DCLR; value BAT46ZFILM -> 100nF; footprint SOD123 -> C0603; symbol traction-r1:D -> traction-r1:C; LCSC C283255 -> CLASS; MPN BAT46ZFILM -> MLCC-100nF-16V
- CSCH3: renamed from DFLT1; value BAT46ZFILM -> 100nF; footprint SOD123 -> C0603; symbol traction-r1:D -> traction-r1:C; LCSC C283255 -> CLASS; MPN BAT46ZFILM -> MLCC-100nF-16V
- CSINA1: renamed from CSINF; value 22pF -> 100pF
- CSINA2: renamed from RSIN1; value 680R -> 2.2nF; footprint R0603 -> C0603; symbol traction-r1:R -> traction-r1:C; MPN R0603-CLASS -> MLCC-CLASS
- CSIND: renamed from RSIN2; value 680R -> 220pF; footprint R0603 -> C0603; symbol traction-r1:R -> traction-r1:C; MPN R0603-CLASS -> MLCC-CLASS
- CSINF: renamed from RSINF1; value 330R -> 22pF; footprint R0603 -> C0603; symbol traction-r1:R -> traction-r1:C; MPN R0603-CLASS -> MLCC-CLASS
- CSNUF: renamed from RSNUP; value 5.1k -> 47nF; footprint R0603 -> C0603; symbol traction-r1:R -> traction-r1:C; MPN R0603-5k1-1% -> MLCC-47nF-25V
- CSNVF: renamed from RSNVP; value 5.1k -> 47nF; footprint R0603 -> C0603; symbol traction-r1:R -> traction-r1:C; MPN R0603-5k1-1% -> MLCC-47nF-25V
- CSNWF: renamed from RSNWP; value 5.1k -> 47nF; footprint R0603 -> C0603; symbol traction-r1:R -> traction-r1:C; MPN R0603-5k1-1% -> MLCC-47nF-25V
- CTAMBF: renamed from JTHS; value NTC-10k-0603 -> 47nF; footprint R0603 -> C0603; symbol traction-r1:J2 -> traction-r1:C; MPN NTC-10k-0603 -> MLCC-47nF-25V
- CTHSF: renamed from RTAMBP; value 10k -> 47nF; footprint R0603 -> C0603; symbol traction-r1:R -> traction-r1:C; MPN R0603-10k-1% -> MLCC-47nF-25V
- CUB1: renamed from CUS2; value 4.7nF -> 3.3nF; MPN MLCC-4.7nF-50V -> MLCC-3.3nF-50V
- CUB2: renamed from LUB; value FB-220R-1A -> 100nF; footprint FB0805 -> C0603; symbol traction-r1:L -> traction-r1:C; MPN FB-220R-1A -> MLCC-100nF-25V
- CUS1: renamed from RUB1; value 100R -> 47nF; footprint R0603 -> C0603; symbol traction-r1:R -> traction-r1:C; MPN R0603-100R -> MLCC-47nF-25V
- CUS2: renamed from RUB2; value 100R -> 4.7nF; footprint R0603 -> C0603; symbol traction-r1:R -> traction-r1:C; MPN R0603-100R -> MLCC-4.7nF-50V
- CVB1: renamed from CVS2; value 4.7nF -> 3.3nF; MPN MLCC-4.7nF-50V -> MLCC-3.3nF-50V
- CVB2: renamed from LVB; value FB-220R-1A -> 100nF; footprint FB0805 -> C0603; symbol traction-r1:L -> traction-r1:C; MPN FB-220R-1A -> MLCC-100nF-25V
- CVD1: renamed from RVD1A; value 10k -> 100pF; footprint R0603 -> C0603; symbol traction-r1:R -> traction-r1:C; MPN R0603-10k-0.1% -> MLCC-CLASS
- CVD2: renamed from RVD2C; value 10k -> 100pF; footprint R0603 -> C0603; symbol traction-r1:R -> traction-r1:C; MPN R0603-10k-0.1% -> MLCC-CLASS
- CVM1: renamed from RVM2; value 24k -> 220nF; footprint R0603 -> C0603; symbol traction-r1:R -> traction-r1:C; MPN R0603-24k-1% -> MLCC-CLASS
- CVM2: renamed from RVM3; value 24k -> 220nF; footprint R0603 -> C0603; symbol traction-r1:R -> traction-r1:C; MPN R0603-24k-1% -> MLCC-CLASS
- CVS1: renamed from RVB1; value 100R -> 47nF; footprint R0603 -> C0603; symbol traction-r1:R -> traction-r1:C; MPN R0603-100R -> MLCC-47nF-25V
- CVS2: renamed from RVB2; value 100R -> 4.7nF; footprint R0603 -> C0603; symbol traction-r1:R -> traction-r1:C; MPN R0603-100R -> MLCC-4.7nF-50V
- CWB1: renamed from CWS2; value 4.7nF -> 3.3nF; MPN MLCC-4.7nF-50V -> MLCC-3.3nF-50V
- CWB2: renamed from LWB; value FB-220R-1A -> 100nF; footprint FB0805 -> C0603; symbol traction-r1:L -> traction-r1:C; MPN FB-220R-1A -> MLCC-100nF-25V
- CWS1: renamed from RWB1; value 100R -> 47nF; footprint R0603 -> C0603; symbol traction-r1:R -> traction-r1:C; MPN R0603-100R -> MLCC-47nF-25V
- CWS2: renamed from RWB2; value 100R -> 4.7nF; footprint R0603 -> C0603; symbol traction-r1:R -> traction-r1:C; MPN R0603-100R -> MLCC-4.7nF-50V
- DCOSP: renamed from CCOSD; value 220pF -> PESD2IVN24-T; footprint C0603 -> SOT23; symbol traction-r1:C -> traction-r1:PESD2IVN24-T; LCSC CLASS -> C406047; MPN MLCC-CLASS -> PESD2IVN24-T
- DFLT1: renamed from RDRB; value 10k -> BAT46ZFILM; footprint R0603 -> SOD123; symbol traction-r1:R -> traction-r1:D; LCSC CLASS -> C283255; MPN R0603-10k -> BAT46ZFILM
- DFLT2: renamed from RENP1; value 5.1k -> BAT46ZFILM; footprint R0603 -> SOD123; symbol traction-r1:R -> traction-r1:D; LCSC CLASS -> C283255; MPN R0603-5k1 -> BAT46ZFILM
- DFO: renamed from RFS1; value 1k -> BAT46ZFILM; footprint R0603 -> SOD123; symbol traction-r1:R -> traction-r1:D; LCSC CLASS -> C283255; MPN R0603-1k -> BAT46ZFILM
- DSINP: renamed from CSIND; value 220pF -> PESD2IVN24-T; footprint C0603 -> SOT23; symbol traction-r1:C -> traction-r1:PESD2IVN24-T; LCSC CLASS -> C406047; MPN MLCC-CLASS -> PESD2IVN24-T
- FMT1: renamed from RMT1S; value 1k -> FUSE-350mA-0603; footprint R0603 -> F0603; symbol traction-r1:R -> traction-r1:F; MPN R0603-CLASS -> FUSE-350mA-0603
- FMT2: renamed from RMT2P; value 10k -> FUSE-350mA-0603; footprint R0603 -> F0603; symbol traction-r1:R -> traction-r1:F; MPN R0603-CLASS -> FUSE-350mA-0603
- FVS1: renamed from LVS3; value FB-470R -> MF-LSMF; footprint FB0603 -> PTC1206; symbol traction-r1:L -> traction-r1:F; MPN FB-470R-CLASS -> MF-LSMF-CLASS
- JICC: renamed from RCPD2; value 10k -> HARNESS-2x20; footprint R0603 -> MicroFit40; symbol traction-r1:R -> traction-r1:HARNESS-2x20-CLASS; MPN R0603-10k -> HARNESS-2x20-CLASS
- JLEM: renamed from USNSW; value HC5FW900-S -> T2M-105-01-L-D-TH-WT; footprint OffBoard -> HDR2x5; symbol traction-r1:HC5FW900-S -> traction-r1:T2M-105-01-L-D-TH-WT; MPN HC5FW900-S -> T2M-105-01-L-D-TH-WT
- JTAMB: renamed from RTHSP; value 10k -> NTC-10k-0603; symbol traction-r1:R -> traction-r1:J2; MPN R0603-10k-1% -> NTC-10k-0603
- JTHS: renamed from UMT1; value OPA333AQDBVRQ1 -> NTC-10k-0603; footprint SOT23-5 -> R0603; symbol traction-r1:OPA333AQDBVRQ1 -> traction-r1:J2; LCSC C2058544 -> CLASS; MPN OPA333AQDBVRQ1 -> NTC-10k-0603
- JVEH: renamed from LVS2; value FB-470R -> TE 770669-1 (AMPSEAL 23); footprint FB0603 -> AMPSEAL23; symbol traction-r1:L -> traction-r1:TE_770669-1__AMPSEAL_23_; MPN FB-470R-CLASS -> TE 770669-1 (AMPSEAL 23)
- LCAN1: renamed from CCAN1; value 1uF -> ACT45B-101-2P-TL003; footprint C0603 -> CMC1210; symbol traction-r1:C -> traction-r1:ACT45B-101-2P-TL003; MPN MLCC-1uF-25V -> ACT45B-101-2P-TL003
- LCAN2: renamed from CCAN2; value 1uF -> ACT45B-101-2P-TL003; footprint C0603 -> CMC1210; symbol traction-r1:C -> traction-r1:ACT45B-101-2P-TL003; MPN MLCC-1uF-25V -> ACT45B-101-2P-TL003
- LUB: renamed from RUB3; value 100R -> FB-220R-1A; footprint R0603 -> FB0805; symbol traction-r1:R -> traction-r1:L; MPN R0603-100R -> FB-220R-1A
- LVB: renamed from RVB3; value 100R -> FB-220R-1A; footprint R0603 -> FB0805; symbol traction-r1:R -> traction-r1:L; MPN R0603-100R -> FB-220R-1A
- LVS2: renamed from JICC; value HARNESS-2x20 -> FB-470R; footprint MicroFit40 -> FB0603; symbol traction-r1:HARNESS-2x20-CLASS -> traction-r1:L; MPN HARNESS-2x20-CLASS -> FB-470R-CLASS
- LVS3: renamed from RCPD0; value 10k -> FB-470R; footprint R0603 -> FB0603; symbol traction-r1:R -> traction-r1:L; MPN R0603-10k -> FB-470R-CLASS
- LVS4: renamed from RCPD1; value 10k -> FB-470R; footprint R0603 -> FB0603; symbol traction-r1:R -> traction-r1:L; MPN R0603-10k -> FB-470R-CLASS
- LWB: renamed from RWB3; value 100R -> FB-220R-1A; footprint R0603 -> FB0805; symbol traction-r1:R -> traction-r1:L; MPN R0603-100R -> FB-220R-1A
- RASCP: renamed from RFS3; value 1k -> 10k; MPN R0603-1k -> R0603-10k
- RCOS1: renamed from RCOSF2; value 330R -> 680R
- RCOS2: renamed from RCOSR1; value 120R -> 680R; MPN R0603-120R -> R0603-CLASS
- RCOSF1: renamed from RCOSR2; value 120R -> 330R; MPN R0603-120R -> R0603-CLASS
- RCOSF2: renamed from JLEM; value T2M-105-01-L-D-TH-WT -> 330R; footprint HDR2x5 -> R0603; symbol traction-r1:T2M-105-01-L-D-TH-WT -> traction-r1:R; MPN T2M-105-01-L-D-TH-WT -> R0603-CLASS
- RCOSR1: renamed from USNSU; value HC5FW900-S -> 120R; footprint OffBoard -> R0603; symbol traction-r1:HC5FW900-S -> traction-r1:R; MPN HC5FW900-S -> R0603-120R
- RCOSR2: renamed from USNSV; value HC5FW900-S -> 120R; footprint OffBoard -> R0603; symbol traction-r1:HC5FW900-S -> traction-r1:R; MPN HC5FW900-S -> R0603-120R
- RCPD1: renamed from RHWP; MPN R0603-10k-1% -> R0603-10k
- RCT1A: renamed from TVSC2; value PESD2IVN24-T -> 60.4R; footprint SOT23 -> R0603; symbol traction-r1:PESD2IVN24-T -> traction-r1:R; LCSC C406047 -> CLASS; MPN PESD2IVN24-T -> R0603-60R4-1%
- renumbered CAND2 to CAND1, CFLTF2 to CFLTF, CSCH to CLAT2, CSCH2 to CSCH, DFLT2 to DCLR, LVS4 to LVS1, RFS2 to RARB, RCPD3 to RCPD0, REXB3 to REXA4, REXB4 to REXB1, RLAT1 to RFS2, RQDM to RGPD, RILK4 to RILK1, RSCH to RRDB, RVD1D to RVD1A, RVD2A to RVD1D, RVD2D to RVD2A, RVM4 to RVM1
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Connections:
- net labels added: RDY_HS_B, RDY_LS_B
- wire segments 868 -> 879
- no-connect marks 2 -> 3
Other:
- note added: "rev A.10 - 26 sections - 280 components"
- note removed: "rev A.9 - 26 sections - 277 components"
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