File: kicad5/traction/traction-card.sch (KiCad schematic (older format))
At the start: 280 parts, among them Y1 CX3225GA40000D0PTVCC

Commit message: Rev A.11: review round 12 response (R1-F01..F28, R2-F01..F35) + datasheet archive
Two whole-system reviews of 4544715 (28 + 35 findings), dispositioned line by
line in docs/review-A11-disposition.md (+ CSV). Twelve real findings fixed
(F123-F134); the rest are tracked gates, firmware-owned, wording or out of the
schematic release's scope. No power-stage, capacitor or topology change.

Hardware / contract:
- SS6 release rule (a) is an energy inequality: winding energy 1.5*L*I^2 plus the
  back-EMF work during the decay, closed-form screen while E < V0, diode-bridge
  simulation otherwise; screening rows (WARN) per SKU
- Resolver exciter rewired as a textbook MFB (1.5 nF / 220 pF): the drawn network
  had the feedback pair swapped, |H(10 kHz)| 0.18 -> 1.85; SWG given its 47 pF load
- V_DC bias: "MGJ2D150505SC" was not an existing order code and no MGJ2 is
  reinforced above 150 Vrms -> TI UCC12050 per channel (V_IOWM 1200 Vrms /
  1697 VDC) behind its own NCV4276C from V15
- Hall: 100 k pull-downs drawn (claimed since A.4); LEM HC5FW drawn with its
  real terminals (1 V_ref, 2 V_out, 3 Gnd, 4 U_C, E1-E4)
- Resolver inputs 10 k / 10 k with rescaled, symmetric filter caps: a wire shorted
  to KL30 injected 23 mA into an SDADC pin against the 3 mA limit
- LV-entry TVS bound explicitly as TPSMC24CA-VR (24 V stand-off, AEC-Q101): the
  classic part the notes described conducts at a 24 V jump start; the OEM's
  load-dump source resistance becomes gate 23
- CSB5 1 uF 0805 (VREF5 inside the FS26 window), ALM2402 as HTSSOP14-PWP,
  on-board NTCs RTAMB/RTHS, kicad5-verify empty-set guard
- Contract wording: FW-05 in instantaneous amperes with a validity window, the
  "BMS limit 0" row split from "contactor open", NVM logging queued behind the
  safe action, FW-02 tau check demoted to plausibility (EOL measurement in dfm),
  FW-18 "unknown, never safe", S6 double-update stated; stale pin-40 / LQFP-176 /
  "inside 6 us" / ALT-field texts corrected; CAN termination DNP option

Doc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
Parts:
- removed CMA1: 1uF, C0603, symbol traction-r1:C
- removed CMA2: 100nF, C0603, symbol traction-r1:C
- removed CMD1, CMD10, CMD11, CMD12: 100nF, C0402, symbol traction-r1:C
- removed UMCU: S32K396, BGA289, symbol traction-r1:S32K396
- added CCT2: 4.7nF, C0603, symbol traction-r1:C
- added FVS1: MF-LSMF, PTC1206, symbol traction-r1:F
- added JICC: HARNESS-2x20, MicroFit40, symbol traction-r1:HARNESS-2x20-CLASS
- added JVEH: TE 770669-1 (AMPSEAL 23), AMPSEAL23, symbol traction-r1:TE_770669-1__AMPSEAL_23_
- added LVS1, LVS2, LVS3, LVS4: FB-470R, FB0603, symbol traction-r1:L
- added RCPD0, RCPD1, RCPD2, RCPD3, RHWP: 10k, R0603, symbol traction-r1:R
- added RCT2A, RCT2B: 60.4R, R0603, symbol traction-r1:R
- CAND1: renamed from CSCH; MPN MLCC-100nF-16V -> MLCC-CLASS
- CAND2: renamed from CSCH2; MPN MLCC-100nF-16V -> MLCC-CLASS
- CASCG: renamed from RFS3; value 1k -> 100nF; footprint R0603 -> C0603; symbol traction-r1:R -> traction-r1:C; MPN R0603-1k -> MLCC-100nF-16V
- CBTC: renamed from CSB5; value 2.2uF -> 47nF; footprint C0805 -> C0603
- CBTP: renamed from CSB6; value 4.7uF -> 22nF; footprint C0805 -> C0603
- CCAN1: renamed from LVS3; value FB-470R -> 1uF; footprint FB0603 -> C0603; symbol traction-r1:L -> traction-r1:C; MPN FB-470R-CLASS -> MLCC-1uF-25V
- CCAN2: renamed from RHWP; value 10k -> 1uF; footprint R0603 -> C0603; symbol traction-r1:R -> traction-r1:C; MPN R0603-10k-1% -> MLCC-1uF-25V
- CCLR: renamed from CSCH3; value 100nF -> 15nF; MPN MLCC-100nF-16V -> MLCC-15nF-50V-C0G
- CCOSA1: renamed from JLEM; value T2M-105-01-L-D-TH-WT -> 22pF; footprint HDR2x5 -> C0603; symbol traction-r1:T2M-105-01-L-D-TH-WT -> traction-r1:C; MPN T2M-105-01-L-D-TH-WT -> MLCC-CLASS
- CCOSA2: renamed from USNSU; value HC5FW900-S -> 100pF; footprint OffBoard -> C0603; symbol traction-r1:HC5FW900-S -> traction-r1:C; MPN HC5FW900-S -> MLCC-CLASS
- CCOSA3: renamed from USNSV; value HC5FW900-S -> 22pF; footprint OffBoard -> C0603; symbol traction-r1:HC5FW900-S -> traction-r1:C; MPN HC5FW900-S -> MLCC-CLASS
- CCOSD: renamed from USNSW; value HC5FW900-S -> 47pF; footprint OffBoard -> C0603; symbol traction-r1:HC5FW900-S -> traction-r1:C; MPN HC5FW900-S -> MLCC-CLASS
- CCOSF1: renamed from UUB1; value OPA376AQDBVRQ1 -> 22pF; footprint SOT23-5 -> C0603; symbol traction-r1:OPA376AQDBVRQ1 -> traction-r1:C; MPN OPA376AQDBVRQ1 -> MLCC-CLASS
- CCOSF2: renamed from UUB2; value OPA376AQDBVRQ1 -> 22pF; footprint SOT23-5 -> C0603; symbol traction-r1:OPA376AQDBVRQ1 -> traction-r1:C; MPN OPA376AQDBVRQ1 -> MLCC-CLASS
- CCT1: renamed from LVS4; value FB-470R -> 4.7nF; footprint FB0603 -> C0603; symbol traction-r1:L -> traction-r1:C; MPN FB-470R-CLASS -> MLCC-4.7nF-50V
- CEXA1: renamed from REXA2; value 10k -> 220pF; footprint R0603 -> C0603; symbol traction-r1:R -> traction-r1:C; MPN R0603-CLASS -> MLCC-CLASS
- CEXA2: renamed from REXA3; value 10k -> 1.5nF; footprint R0603 -> C0603; symbol traction-r1:R -> traction-r1:C; MPN R0603-CLASS -> MLCC-CLASS
- CEXA3: renamed from REXA4; value 24k -> 100nF; footprint R0603 -> C0603; symbol traction-r1:R -> traction-r1:C; MPN R0603-CLASS -> MLCC-CLASS
- CEXA4: renamed from REXB1; value 24k -> 47pF; footprint R0603 -> C0603; symbol traction-r1:R -> traction-r1:C; MPN R0603-CLASS -> MLCC-CLASS
- CEXD: renamed from REXB2; value 24k -> 4.7uF; footprint R0603 -> C0603; symbol traction-r1:R -> traction-r1:C; MPN R0603-CLASS -> MLCC-CLASS
- CFLTD: renamed from DCLR; value BAT46ZFILM -> 3.3nF; footprint SOD123 -> C0603; symbol traction-r1:D -> traction-r1:C; LCSC C283255 -> CLASS; MPN BAT46ZFILM -> MLCC-3.3nF-50V-C0G
- CFLTF: renamed from DFLT1; value BAT46ZFILM -> 100pF; footprint SOD123 -> C0603; symbol traction-r1:D -> traction-r1:C; LCSC C283255 -> CLASS; MPN BAT46ZFILM -> MLCC-100pF-16V
- CFLTF2: renamed from DFLT2; value BAT46ZFILM -> 100pF; footprint SOD123 -> C0603; symbol traction-r1:D -> traction-r1:C; LCSC C283255 -> CLASS; MPN BAT46ZFILM -> MLCC-100pF-16V
- CIGN: renamed from UAND1; value 74LVC1G11GW-Q100 -> 100nF; footprint SOT363 -> C0603; symbol traction-r1:74LVC1G11GW-Q100 -> traction-r1:C; LCSC C548242 -> CLASS; MPN 74LVC1G11GW-Q100 -> MLCC-100nF-50V
- CIGNS: renamed from UAND2; value 74LVC1G11GW-Q100 -> 100nF; footprint SOT363 -> C0603; symbol traction-r1:74LVC1G11GW-Q100 -> traction-r1:C; LCSC C548242 -> CLASS; MPN 74LVC1G11GW-Q100 -> MLCC-CLASS
- CILK: renamed from CVM1; value 220nF -> 2.2nF; MPN MLCC-CLASS -> MLCC-2.2nF-50V
- CLAT: renamed from RFS4; value 1k -> 100nF; footprint R0603 -> C0603; symbol traction-r1:R -> traction-r1:C; MPN ESR03EZPF1001 -> MLCC-100nF-16V
- CLAT2: renamed from RDRB; value 10k -> 100nF; footprint R0603 -> C0603; symbol traction-r1:R -> traction-r1:C; MPN R0603-10k -> MLCC-100nF-16V
- CLDE: renamed from REXB3; value 24k -> 22uF; footprint R0603 -> C0603; symbol traction-r1:R -> traction-r1:C; MPN R0603-CLASS -> MLCC-CLASS
- CLDEC: renamed from REXB4; value 24k -> 270pF; footprint R0603 -> C0603; symbol traction-r1:R -> traction-r1:C; MPN R0603-CLASS -> MLCC-CLASS
- CLVC1: renamed from FVBL; value MF-LSMF300/24X-2 -> 4.7uF; footprint PTC2920 -> C1206; symbol traction-r1:F -> traction-r1:C; LCSC C719172 -> CLASS; MPN MF-LSMF300/24X-2 -> MLCC-4.7uF-50V
- CLVC2: renamed from LFC; value FB-120R-3A -> 22uF; footprint FB1206 -> C1210; symbol traction-r1:L -> traction-r1:C; MPN FB-120R-3A -> MLCC-22uF-50V
- CLVSM: renamed from RLVSD; value 4.7k -> 100nF; footprint R0603 -> C0603; symbol traction-r1:R -> traction-r1:C; MPN R0603-4k7 -> MLCC-100nF-50V
- CMA1: renamed from CMD3; value 100nF -> 1uF; footprint C0402 -> C0603; MPN MLCC-100nF-16V -> MLCC-1uF-16V
- CMA2: renamed from CMD4; footprint C0402 -> C0603
- CMD3: renamed from CYA; value 12pF -> 100nF; footprint C0603 -> C0402; MPN MLCC-12pF-50V -> MLCC-100nF-16V
- CMD4: renamed from CYB; value 12pF -> 100nF; footprint C0603 -> C0402; MPN MLCC-12pF-50V -> MLCC-100nF-16V
- CMD5: renamed from RMRST; value 10k -> 100nF; footprint R0603 -> C0402; symbol traction-r1:R -> traction-r1:C; MPN R0603-10k -> MLCC-100nF-16V
- CMD6: renamed from Y1; value CX3225GA40000D0PTVCC -> 100nF; footprint X3225 -> C0402; symbol traction-r1:Y -> traction-r1:C; LCSC C6009848 -> CLASS; MPN CX3225GA40000D0PTVCC -> MLCC-100nF-16V
- CMD7: renamed from JSWD; value FTSH-105-01-L-DV-K -> 100nF; footprint HDR2x5-1.27 -> C0402; symbol traction-r1:FTSH-105-01-L-DV-K -> traction-r1:C; MPN FTSH-105-01-L-DV-K -> MLCC-100nF-16V
- CMD8: renamed from CRST; value 100pF -> 100nF; footprint C0603 -> C0402; MPN MLCC-100pF-16V -> MLCC-100nF-16V
- CMD9: renamed from RBOOT; value 10k -> 100nF; footprint R0603 -> C0402; symbol traction-r1:R -> traction-r1:C; MPN R0603-10k -> MLCC-100nF-16V
- CMT1F: renamed from RCT1A; value 60.4R -> 47nF; footprint R0603 -> C0603; symbol traction-r1:R -> traction-r1:C; MPN R0603-60R4-1% -> MLCC-47nF-25V
- CMT2F: renamed from RCT1B; value 60.4R -> 47nF; footprint R0603 -> C0603; symbol traction-r1:R -> traction-r1:C; MPN R0603-60R4-1% -> MLCC-47nF-25V
- COF1: renamed from CSNVF; value 47nF -> 100nF; MPN MLCC-47nF-25V -> MLCC-CLASS
- COR1: renamed from UVMB1; value OPA348AQDBVRQ1 -> 100nF; footprint SOT23-5 -> C0603; symbol traction-r1:OPA348AQDBVRQ1 -> traction-r1:C; LCSC C2877787 -> CLASS; MPN OPA348AQDBVRQ1 -> MLCC-CLASS
- COR2: renamed from UVMB2; value OPA348AQDBVRQ1 -> 100nF; footprint SOT23-5 -> C0603; symbol traction-r1:OPA348AQDBVRQ1 -> traction-r1:C; LCSC C2877787 -> CLASS; MPN OPA348AQDBVRQ1 -> MLCC-CLASS
- CRST: renamed from DREVC; value STPS5L60S -> 100pF; footprint SMC -> C0603; symbol traction-r1:D -> traction-r1:C; LCSC C140620 -> CLASS; MPN STPS5L60S -> MLCC-100pF-16V
- CSB1: renamed from CSB7; value 10uF -> 22uF
- CSB2: renamed from CSB8; value 10uF -> 22uF
- CSB3: renamed from CVBOS; value 4.7uF -> 22uF; footprint C0603 -> C0805
- CSB3B: renamed from CVDIG; value 1uF -> 22uF
- CSB4: renamed from DBAT; value BAT46ZFILM -> 10uF; footprint SOD123 -> C0805; symbol traction-r1:D -> traction-r1:C; LCSC C283255 -> CLASS; MPN BAT46ZFILM -> MLCC-CLASS
- CSB5: renamed from LCOR; value XAL4020-222MEC -> 1uF; footprint XAL4020 -> C0805; symbol traction-r1:L -> traction-r1:C; MPN XAL4020-222MEC -> MLCC-1uF-16V-X7R-0805
- CSB6: renamed from LSBC; value XAL4040-103MEC -> 4.7uF; footprint XAL4040 -> C0805; symbol traction-r1:L -> traction-r1:C; MPN XAL4040-103MEC -> MLCC-CLASS
- CSB7: renamed from RAGT; value 0R -> 10uF; footprint R0603 -> C0805; symbol traction-r1:R -> traction-r1:C; MPN R0603-CLASS -> MLCC-CLASS
- CSB8: renamed from RDBG; value 10k -> 10uF; footprint R0603 -> C0805; symbol traction-r1:R -> traction-r1:C; MPN R0603-CLASS -> MLCC-CLASS
- CSCH: renamed from RENP1; value 5.1k -> 100nF; footprint R0603 -> C0603; symbol traction-r1:R -> traction-r1:C; MPN R0603-5k1 -> MLCC-100nF-16V
- CSCH2: renamed from RFCB; value 100k -> 100nF; footprint R0603 -> C0603; symbol traction-r1:R -> traction-r1:C; MPN R0603-100k -> MLCC-100nF-16V
- CSCH3: renamed from RFLTC; value 10k -> 100nF; footprint R0603 -> C0603; symbol traction-r1:R -> traction-r1:C; MPN R0603-10k -> MLCC-100nF-16V
- CSINA1: renamed from RSINR1; value 120R -> 22pF; footprint R0603 -> C0603; symbol traction-r1:R -> traction-r1:C; MPN R0603-120R -> MLCC-CLASS
- CSINA2: renamed from RSINR2; value 120R -> 100pF; footprint R0603 -> C0603; symbol traction-r1:R -> traction-r1:C; MPN R0603-120R -> MLCC-CLASS
- CSINA3: renamed from DCOSP; value PESD2IVN24-T -> 22pF; footprint SOT23 -> C0603; symbol traction-r1:PESD2IVN24-T -> traction-r1:C; LCSC C406047 -> CLASS; MPN PESD2IVN24-T -> MLCC-CLASS
- CSIND: renamed from CCOSA1; value 100pF -> 47pF
- CSINF1: renamed from CCOSA2; value 2.2nF -> 22pF
- CSINF2: renamed from CCOSD; value 220pF -> 22pF
- CSNWF: renamed from FMT1; value FUSE-350mA-0603 -> 47nF; footprint F0603 -> C0603; symbol traction-r1:F -> traction-r1:C; MPN FUSE-350mA-0603 -> MLCC-47nF-25V
- CTAMBF: renamed from RMT2S; value 1k -> 47nF; footprint R0603 -> C0603; symbol traction-r1:R -> traction-r1:C; MPN R0603-CLASS -> MLCC-47nF-25V
- CTHSF: renamed from TVSM1; value PESD5V0L1BA -> 47nF; footprint SOD323 -> C0603; symbol traction-r1:R -> traction-r1:C; MPN PESD5V0L1BA -> MLCC-47nF-25V
- CUB1: renamed from CVS1; value 47nF -> 3.3nF; MPN MLCC-47nF-25V -> MLCC-3.3nF-50V
- CUB2: renamed from CVS2; value 4.7nF -> 100nF; MPN MLCC-4.7nF-50V -> MLCC-100nF-25V
- CUS1: renamed from LVB; value FB-220R-1A -> 47nF; footprint FB0805 -> C0603; symbol traction-r1:L -> traction-r1:C; MPN FB-220R-1A -> MLCC-47nF-25V
- CUS2: renamed from RVB1; value 100R -> 4.7nF; footprint R0603 -> C0603; symbol traction-r1:R -> traction-r1:C; MPN R0603-100R -> MLCC-4.7nF-50V
- CVB1: renamed from CWS2; value 4.7nF -> 3.3nF; MPN MLCC-4.7nF-50V -> MLCC-3.3nF-50V
- CVB2: renamed from LWB; value FB-220R-1A -> 100nF; footprint FB0805 -> C0603; symbol traction-r1:L -> traction-r1:C; MPN FB-220R-1A -> MLCC-100nF-25V
- CVBOS: renamed from RSB1; value 52.3k -> 4.7uF; footprint R0603 -> C0603; symbol traction-r1:R -> traction-r1:C; MPN R0603-CLASS -> MLCC-CLASS
- CVD1: renamed from CSNWF; value 47nF -> 100pF; MPN MLCC-47nF-25V -> MLCC-CLASS
- CVD2: renamed from JTHS; value NTC-10k-0603 -> 100pF; footprint R0603 -> C0603; symbol traction-r1:J2 -> traction-r1:C; MPN NTC-10k-0603 -> MLCC-CLASS
- CVDIG: renamed from RSB2; value 10k -> 1uF; footprint R0603 -> C0603; symbol traction-r1:R -> traction-r1:C; MPN R0603-CLASS -> MLCC-CLASS
- CVM1: renamed from UEXF; value OPA348AQDBVRQ1 -> 220nF; footprint SOT23-5 -> C0603; symbol traction-r1:OPA348AQDBVRQ1 -> traction-r1:C; LCSC C2877787 -> CLASS; MPN OPA348AQDBVRQ1 -> MLCC-CLASS
- CVM2: renamed from ULDOEX; value NCV4276CDTADJRKG -> 220nF; footprint DPAK5 -> C0603; symbol traction-r1:NCV4276CDTADJRKG -> traction-r1:C; MPN NCV4276CDTADJRKG -> MLCC-CLASS
- CVS1: renamed from RWB1; value 100R -> 47nF; footprint R0603 -> C0603; symbol traction-r1:R -> traction-r1:C; MPN R0603-100R -> MLCC-47nF-25V
- CVS2: renamed from RWB2; value 100R -> 4.7nF; footprint R0603 -> C0603; symbol traction-r1:R -> traction-r1:C; MPN R0603-100R -> MLCC-4.7nF-50V
- CWB1: renamed from RVD1A; value 10k -> 3.3nF; footprint R0603 -> C0603; symbol traction-r1:R -> traction-r1:C; MPN R0603-10k-0.1% -> MLCC-3.3nF-50V
- CWB2: renamed from RVD1B; value 10k -> 100nF; footprint R0603 -> C0603; symbol traction-r1:R -> traction-r1:C; MPN R0603-10k-0.1% -> MLCC-100nF-25V
- CWS1: renamed from RVD1C; value 10k -> 47nF; footprint R0603 -> C0603; symbol traction-r1:R -> traction-r1:C; MPN R0603-10k-0.1% -> MLCC-47nF-25V
- CWS2: renamed from RVD1D; value 10k -> 4.7nF; footprint R0603 -> C0603; symbol traction-r1:R -> traction-r1:C; MPN R0603-10k-0.1% -> MLCC-4.7nF-50V
- CYA: renamed from QLVN; value 2N7002 -> 12pF; footprint SOT23 -> C0603; symbol traction-r1:2N7002 -> traction-r1:C; LCSC C8545 -> CLASS; MPN 2N7002 -> MLCC-12pF-50V
- CYB: renamed from QLVS; value DMP6023LEQ-13 -> 12pF; footprint SOT223 -> C0603; symbol traction-r1:DMP6023LEQ-13 -> traction-r1:C; MPN DMP6023LEQ-13 -> MLCC-12pF-50V
- DBAT: renamed from RSB3; value 220R -> BAT46ZFILM; footprint R0603 -> SOD123; symbol traction-r1:R -> traction-r1:D; LCSC CLASS -> C283255; MPN R0603-CLASS -> BAT46ZFILM
- DCLR: renamed from RFLTD; value 10k -> BAT46ZFILM; footprint R0603 -> SOD123; symbol traction-r1:R -> traction-r1:D; LCSC CLASS -> C283255; MPN R0603-10k -> BAT46ZFILM
- DCOSP: renamed from RCOSR2; value 120R -> PESD2IVN24-T; footprint R0603 -> SOT23; symbol traction-r1:R -> traction-r1:PESD2IVN24-T; LCSC CLASS -> C406047; MPN R0603-120R -> PESD2IVN24-T
- DFLT1: renamed from RFLTP1; value 5.1k -> BAT46ZFILM; footprint R0603 -> SOD123; symbol traction-r1:R -> traction-r1:D; LCSC CLASS -> C283255; MPN R0603-5k1 -> BAT46ZFILM
- DFLT2: renamed from RFLTP2; value 5.1k -> BAT46ZFILM; footprint R0603 -> SOD123; symbol traction-r1:R -> traction-r1:D; LCSC CLASS -> C283255; MPN R0603-5k1 -> BAT46ZFILM
- DFO: renamed from RLAT1; value 10k -> BAT46ZFILM; footprint R0603 -> SOD123; symbol traction-r1:R -> traction-r1:D; LCSC CLASS -> C283255; MPN R0603-10k -> BAT46ZFILM
- DIGN: renamed from ULAT2; value 74LVC1G74DC-Q100 -> 1N4148WS; footprint VSSOP8 -> SOD323; symbol traction-r1:74LVC1G74DC-Q100 -> traction-r1:D; LCSC CLASS -> C2128; MPN 74LVC1G74DC-Q100 -> 1N4148WS
- DREVC: renamed from RLVSG; value 10k -> STPS5L60S; footprint R0603 -> SMC; symbol traction-r1:R -> traction-r1:D; LCSC CLASS -> C140620; MPN R0603-10k -> STPS5L60S
- DSINP: renamed from RSINF2; value 330R -> PESD2IVN24-T; footprint R0603 -> SOT23; symbol traction-r1:R -> traction-r1:PESD2IVN24-T; LCSC CLASS -> C406047; MPN R0603-CLASS -> PESD2IVN24-T
- DTVSC: renamed from RLVSM; value 1k -> TPSMC24CA-VR; footprint R0603 -> SMC; symbol traction-r1:R -> traction-r1:D; LCSC CLASS -> C1975284; MPN R0603-1k -> TPSMC24CA-VR
- FLVC: renamed from ZLVS; value BZT52-C15 -> MF-LSMF300/24X-2; footprint SOD123 -> PTC2920; symbol traction-r1:D -> traction-r1:F; LCSC CLASS -> C719172; MPN BZT52-C15 -> MF-LSMF300/24X-2
- FMT1: renamed from LCAN2; value ACT45B-101-2P-TL003 -> FUSE-350mA-0603; footprint CMC1210 -> F0603; symbol traction-r1:ACT45B-101-2P-TL003 -> traction-r1:F; MPN ACT45B-101-2P-TL003 -> FUSE-350mA-0603
- FMT2: renamed from TVSC2; value PESD2IVN24-T -> FUSE-350mA-0603; footprint SOT23 -> F0603; symbol traction-r1:PESD2IVN24-T -> traction-r1:F; LCSC C406047 -> CLASS; MPN PESD2IVN24-T -> FUSE-350mA-0603
- FVBH: renamed from QBAL; value SQ2310ES -> MF-LSMF300/24X-2; footprint SOT23 -> PTC2920; symbol traction-r1:SQ2310ES -> traction-r1:F; LCSC CLASS -> C719172; MPN SQ2310ES -> MF-LSMF300/24X-2
- FVBL: renamed from USBC; value FS2633D -> MF-LSMF300/24X-2; footprint HLQFP48 -> PTC2920; symbol traction-r1:FS2633D -> traction-r1:F; LCSC CLASS -> C719172; MPN FS2633D -> MF-LSMF300/24X-2
- JLEM: renamed from RUB2; value 100R -> T2M-105-01-L-D-TH-WT; footprint R0603 -> HDR2x5; symbol traction-r1:R -> traction-r1:T2M-105-01-L-D-TH-WT; MPN R0603-100R -> T2M-105-01-L-D-TH-WT
- JSWD: renamed from CLVSM; value 100nF -> FTSH-105-01-L-DV-K; footprint C0603 -> HDR2x5-1.27; symbol traction-r1:C -> traction-r1:FTSH-105-01-L-DV-K; MPN MLCC-100nF-50V -> FTSH-105-01-L-DV-K
- LCAN1: renamed from FVS1; value MF-LSMF -> ACT45B-101-2P-TL003; footprint PTC1206 -> CMC1210; symbol traction-r1:F -> traction-r1:ACT45B-101-2P-TL003; MPN MF-LSMF-CLASS -> ACT45B-101-2P-TL003
- LCAN2: renamed from RCPD1; value 10k -> ACT45B-101-2P-TL003; footprint R0603 -> CMC1210; symbol traction-r1:R -> traction-r1:ACT45B-101-2P-TL003; MPN R0603-10k -> ACT45B-101-2P-TL003
- LCOR: renamed from RSB4; value 5.1k -> XAL4020-222MEC; footprint R0603 -> XAL4020; symbol traction-r1:R -> traction-r1:L; MPN R0603-CLASS -> XAL4020-222MEC
- LFC: renamed from CBTC; value 47nF -> FB-120R-3A; footprint C0603 -> FB1206; symbol traction-r1:C -> traction-r1:L; MPN MLCC-CLASS -> FB-120R-3A
- LSBC: renamed from CIGN; value 100nF -> XAL4040-103MEC; footprint C0603 -> XAL4040; symbol traction-r1:C -> traction-r1:L; MPN MLCC-100nF-50V -> XAL4040-103MEC
- LUB: renamed from RVB2; value 100R -> FB-220R-1A; footprint R0603 -> FB0805; symbol traction-r1:R -> traction-r1:L; MPN R0603-100R -> FB-220R-1A
- LVB: renamed from RWB3; value 100R -> FB-220R-1A; footprint R0603 -> FB0805; symbol traction-r1:R -> traction-r1:L; MPN R0603-100R -> FB-220R-1A
- LWB: renamed from UVD2; value OPA376AQDBVRQ1 -> FB-220R-1A; footprint SOT23-5 -> FB0805; symbol traction-r1:OPA376AQDBVRQ1 -> traction-r1:L; MPN OPA376AQDBVRQ1 -> FB-220R-1A
- QBAL: renamed from CSB3B; value 22uF -> SQ2310ES; footprint C0603 -> SOT23; symbol traction-r1:C -> traction-r1:SQ2310ES; MPN MLCC-CLASS -> SQ2310ES
- QLVN: renamed from FLVC; value MF-LSMF300/24X-2 -> 2N7002; footprint PTC2920 -> SOT23; symbol traction-r1:F -> traction-r1:2N7002; LCSC C719172 -> C8545; MPN MF-LSMF300/24X-2 -> 2N7002
- QLVS: renamed from FVBH; value MF-LSMF300/24X-2 -> DMP6023LEQ-13; footprint PTC2920 -> SOT223; symbol traction-r1:F -> traction-r1:DMP6023LEQ-13; LCSC C719172 -> CLASS; MPN MF-LSMF300/24X-2 -> DMP6023LEQ-13
- RAGT: renamed from CIGNS; value 100nF -> 0R; footprint C0603 -> R0603; symbol traction-r1:C -> traction-r1:R; MPN MLCC-CLASS -> R0603-CLASS
- RARB: renamed from ZSET; value BZT52-B5V6 -> 10k; footprint SOD123 -> R0603; symbol traction-r1:D -> traction-r1:R; MPN BZT52-B5V6 -> R0603-10k
- RASCP: renamed from UOR1; value 74LVC1G32GW-Q100 -> 10k; footprint SOT353 -> R0603; symbol traction-r1:74LVC1G32GW-Q100 -> traction-r1:R; LCSC C548334 -> CLASS; MPN 74LVC1G32GW-Q100 -> R0603-10k
- renumbered CMD5 to CMD1, CMD6 to CMD10, CMD7 to CMD11, CMD8 to CMD12, CMD9 to CMD2, CMT1F to CSNUF, CMT2F to CSNVF, RGPD to RDRB, REXM4 to REXA4, RRDYP2 to RFLTP1, RILK1 to RLAT1, RCOSR1 to RSINR2
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Connections:
- wire segments 879 -> 907
Other:
- note added: "rev A.11 - 26 sections - 288 components"
- note removed: "rev A.10 - 26 sections - 280 components"
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
Commit message: Rev A.12: round 13 rechecks (F135-F139), pin freeze (F140), barrier + orderability closure (F141-F142), Marine A.12, firmware
- Rechecks of 30ae0a2: §6 winding-energy rule at every speed; resolver 12 k series + 220 pF C_AAF
  (injection 2.92 mA with the MCU unpowered); verifier counts distinct assemblies; TPS55340-Q1 real
  ratings (38/40 V); NCV4276C thermal on the datasheet pad.
- MCU pin freeze: all 289 S32K396 balls bound from SPF-91122 rev C anchored on the DS supply balls
  (calculations/mcu-ballmap.json, docs/mcu-pin-manifest.md); seven port corrections; FS26 pins verified;
  ERC pin-freeze lock.
- Barrier closure: VOW3120-X017T optos and UCC14141-Q1 biases (shared IsoBias18 cell, single-output
  18.0 V) replace TLP152/QA01C-18; LED resistors 270 R; VY1 Y-caps; Samtec IPL1/IPD1 harness;
  Faratronic 4XX can; SQP10 discharge resistors; UCC12051-Q1 on the AVL.
- Tooling: ERC open-pin helper + HARNESS40 parser scoped to its block; kicad5-verify assembly-set guard.
- Marine ported to A.12 (86 PASS / 22 WARN / 0 FAIL); firmware/ (C11, 178 tests / 1209 checks).
- Docs: README, design-basis §6a/§8/§11l, dfm, variants, cost-rollup, EXTRACTED-PARAMS §27-30 +
  seven archived datasheets, review-A12-disposition (+CSV), regenerated sheets/PDFs/BOMs/previews.

ERC 933/0 · design-verify 123/19/0 · sim 23/6/0 · sheets 2027/2027.

Co-Authored-By: Claude Fable 5.1 <noreply@anthropic.com>
Parts:
- removed CMA1: 1uF, C0603, symbol traction-r1:C
- removed CMA2: 100nF, C0603, symbol traction-r1:C
- removed CMD1, CMD10, CMD11, CMD12, CMD2, CMD3, CMD4, CMD5, CMD6, CMD7, CMD8, CMD9: 100nF, C0402, symbol traction-r1:C
- removed CYA, CYB: 12pF, C0603, symbol traction-r1:C
- removed RMRST: 10k, R0603, symbol traction-r1:R
- removed UMCU: S32K396, BGA289, symbol traction-r1:S32K396
- added CCAN2: 1uF, C0603, symbol traction-r1:C
- added CCT2: 4.7nF, C0603, symbol traction-r1:C
- added FVS1: MF-LSMF, PTC1206, symbol traction-r1:F
- added JICC: IPL1-120-01-L-D-K, HDR2x20-2.54, symbol traction-r1:IPL1-120-01-L-D-K
- added JVEH: TE 770669-1 (AMPSEAL 23), AMPSEAL23, symbol traction-r1:TE_770669-1__AMPSEAL_23_
- added LVS1, LVS2, LVS3, LVS4: FB-470R, FB0603, symbol traction-r1:L
- added RCPD0, RCPD1, RCPD2, RCPD3, RHWP: 10k, R0603, symbol traction-r1:R
- added RCT2A, RCT2B: 60.4R, R0603, symbol traction-r1:R
- added TVSC2: PESD2IVN24-T, SOT23, symbol traction-r1:PESD2IVN24-T
- added UCAN2: TCAN1042HGVDRQ1, SOIC8, symbol traction-r1:TCAN1042HGVDRQ1
- CAND1: renamed from RFLTP1; value 5.1k -> 100nF; footprint R0603 -> C0603; symbol traction-r1:R -> traction-r1:C; MPN R0603-5k1 -> MLCC-CLASS
- CAND2: renamed from RFLTP2; value 5.1k -> 100nF; footprint R0603 -> C0603; symbol traction-r1:R -> traction-r1:C; MPN R0603-5k1 -> MLCC-CLASS
- CASCG: renamed from RILK3; value 10k -> 100nF; footprint R0603 -> C0603; symbol traction-r1:R -> traction-r1:C; MPN R0603-10k -> MLCC-100nF-16V
- CBTC: renamed from RSB1; value 52.3k -> 47nF; footprint R0603 -> C0603; symbol traction-r1:R -> traction-r1:C; MPN R0603-CLASS -> MLCC-CLASS
- CBTP: renamed from RSB2; value 10k -> 22nF; footprint R0603 -> C0603; symbol traction-r1:R -> traction-r1:C; MPN R0603-CLASS -> MLCC-CLASS
- CCAN1: renamed from RCPD0; value 10k -> 1uF; footprint R0603 -> C0603; symbol traction-r1:R -> traction-r1:C; MPN R0603-10k -> MLCC-1uF-25V
- CCLR: renamed from RGPD; value 10k -> 15nF; footprint R0603 -> C0603; symbol traction-r1:R -> traction-r1:C; MPN R0603-10k -> MLCC-15nF-50V-C0G
- CCOSA1: renamed from CUB1; value 3.3nF -> 22pF; MPN MLCC-3.3nF-50V -> MLCC-CLASS
- CCOSA2: renamed from CUB2; value 100nF -> 220pF; MPN MLCC-100nF-25V -> MLCC-CLASS
- CCOSA3: renamed from CUS1; value 47nF -> 22pF; MPN MLCC-47nF-25V -> MLCC-CLASS
- CCOSD: renamed from CUS2; value 4.7nF -> 47pF; MPN MLCC-4.7nF-50V -> MLCC-CLASS
- CCOSF1: renamed from LUB; value FB-220R-1A -> 22pF; footprint FB0805 -> C0603; symbol traction-r1:L -> traction-r1:C; MPN FB-220R-1A -> MLCC-CLASS
- CCOSF2: renamed from RUB0; value 100k -> 22pF; footprint R0603 -> C0603; symbol traction-r1:R -> traction-r1:C; MPN R0603-100k -> MLCC-CLASS
- CCT1: renamed from RCPD1; value 10k -> 4.7nF; footprint R0603 -> C0603; symbol traction-r1:R -> traction-r1:C; MPN R0603-10k -> MLCC-4.7nF-50V
- CEXA1: renamed from REXM4; value 24k -> 220pF; footprint R0603 -> C0603; symbol traction-r1:R -> traction-r1:C; MPN R0603-CLASS -> MLCC-CLASS
- CEXA2: renamed from RLDE1; value 38.3k -> 1.5nF; footprint R0603 -> C0603; symbol traction-r1:R -> traction-r1:C; MPN R0603-CLASS -> MLCC-CLASS
- CEXA3: renamed from RLDE2; value 10k -> 100nF; footprint R0603 -> C0603; symbol traction-r1:R -> traction-r1:C; MPN R0603-CLASS -> MLCC-CLASS
- CEXA4: renamed from RSDN; value 10k -> 47pF; footprint R0603 -> C0603; symbol traction-r1:R -> traction-r1:C; MPN R0603-CLASS -> MLCC-CLASS
- CEXD: renamed from DSINP; value PESD2IVN24-T -> 4.7uF; footprint SOT23 -> C0603; symbol traction-r1:PESD2IVN24-T -> traction-r1:C; LCSC C406047 -> CLASS; MPN PESD2IVN24-T -> MLCC-CLASS
- CFLTD: renamed from RLAT2; value 10k -> 3.3nF; footprint R0603 -> C0603; symbol traction-r1:R -> traction-r1:C; MPN R0603-10k -> MLCC-3.3nF-50V-C0G
- CFLTF: renamed from RQDM; value 10k -> 100pF; footprint R0603 -> C0603; symbol traction-r1:R -> traction-r1:C; MPN R0603-10k -> MLCC-100pF-16V
- CFLTF2: renamed from RRDB; value 100k -> 100pF; footprint R0603 -> C0603; symbol traction-r1:R -> traction-r1:C; MPN R0603-100k -> MLCC-100pF-16V
- CIGN: renamed from CFLTF2; value 100pF -> 100nF; MPN MLCC-100pF-16V -> MLCC-100nF-50V
- CIGNS: renamed from CLAT2; MPN MLCC-100nF-16V -> MLCC-CLASS
- CILK: renamed from CEXA3; value 100nF -> 2.2nF; MPN MLCC-CLASS -> MLCC-2.2nF-50V
- CLAT: renamed from RILK4; value 10k -> 100nF; footprint R0603 -> C0603; symbol traction-r1:R -> traction-r1:C; MPN R0603-10k -> MLCC-100nF-16V
- CLAT2: renamed from RRDYP1; value 5.1k -> 100nF; footprint R0603 -> C0603; symbol traction-r1:R -> traction-r1:C; MPN R0603-5k1 -> MLCC-100nF-16V
- CLDE: renamed from CSINA1; value 22pF -> 22uF
- CLDEC: renamed from CSINA2; value 100pF -> 270pF
- CLVC1: renamed from CSB2; value 22uF -> 4.7uF; footprint C0805 -> C1206; MPN MLCC-CLASS -> MLCC-4.7uF-50V
- CLVC2: renamed from CSB3; footprint C0805 -> C1210; MPN MLCC-CLASS -> MLCC-22uF-50V
- CLVSM: renamed from CSB3B; value 22uF -> 100nF; MPN MLCC-CLASS -> MLCC-100nF-50V
- CMA1: renamed from JSWD; value FTSH-105-01-L-DV-K -> 1uF; footprint HDR2x5-1.27 -> C0603; symbol traction-r1:FTSH-105-01-L-DV-K -> traction-r1:C; MPN FTSH-105-01-L-DV-K -> MLCC-1uF-16V
- CMA2: renamed from CRST; value 100pF -> 100nF; MPN MLCC-100pF-16V -> MLCC-100nF-16V
- CMD1: renamed from RBOOT; value 10k -> 100nF; footprint R0603 -> C0402; symbol traction-r1:R -> traction-r1:C; MPN R0603-10k -> MLCC-100nF-16V
- CMD10: renamed from QLVN; value 2N7002 -> 100nF; footprint SOT23 -> C0402; symbol traction-r1:2N7002 -> traction-r1:C; LCSC C8545 -> CLASS; MPN 2N7002 -> MLCC-100nF-16V
- CMD11: renamed from QLVS; value DMP6023LEQ-13 -> 100nF; footprint SOT223 -> C0402; symbol traction-r1:DMP6023LEQ-13 -> traction-r1:C; MPN DMP6023LEQ-13 -> MLCC-100nF-16V
- CMD12: renamed from CLVC1; value 4.7uF -> 100nF; footprint C1206 -> C0402; MPN MLCC-4.7uF-50V -> MLCC-100nF-16V
- CMD2: renamed from CLVC2; value 22uF -> 100nF; footprint C1210 -> C0402; MPN MLCC-22uF-50V -> MLCC-100nF-16V
- CMD3: renamed from CLVSM; footprint C0603 -> C0402; MPN MLCC-100nF-50V -> MLCC-100nF-16V
- CMD4: renamed from DREVC; value STPS5L60S -> 100nF; footprint SMC -> C0402; symbol traction-r1:D -> traction-r1:C; LCSC C140620 -> CLASS; MPN STPS5L60S -> MLCC-100nF-16V
- CMD5: renamed from DTVSC; value TPSMC24CA-VR -> 100nF; footprint SMC -> C0402; symbol traction-r1:D -> traction-r1:C; LCSC C1975284 -> CLASS; MPN TPSMC24CA-VR -> MLCC-100nF-16V
- CMD6: renamed from FLVC; value MF-LSMF300/24X-2 -> 100nF; footprint PTC2920 -> C0402; symbol traction-r1:F -> traction-r1:C; LCSC C719172 -> CLASS; MPN MF-LSMF300/24X-2 -> MLCC-100nF-16V
- CMD7: renamed from FVBH; value MF-LSMF300/24X-2 -> 100nF; footprint PTC2920 -> C0402; symbol traction-r1:F -> traction-r1:C; LCSC C719172 -> CLASS; MPN MF-LSMF300/24X-2 -> MLCC-100nF-16V
- CMD8: renamed from FVBL; value MF-LSMF300/24X-2 -> 100nF; footprint PTC2920 -> C0402; symbol traction-r1:F -> traction-r1:C; LCSC C719172 -> CLASS; MPN MF-LSMF300/24X-2 -> MLCC-100nF-16V
- CMD9: renamed from LFC; value FB-120R-3A -> 100nF; footprint FB1206 -> C0402; symbol traction-r1:L -> traction-r1:C; MPN FB-120R-3A -> MLCC-100nF-16V
- CMT1F: renamed from TVSC2; value PESD2IVN24-T -> 47nF; footprint SOT23 -> C0603; symbol traction-r1:PESD2IVN24-T -> traction-r1:C; LCSC C406047 -> CLASS; MPN PESD2IVN24-T -> MLCC-47nF-25V
- CMT2F: renamed from UCAN2; value TCAN1042HGVDRQ1 -> 47nF; footprint SOIC8 -> C0603; symbol traction-r1:TCAN1042HGVDRQ1 -> traction-r1:C; LCSC C132550 -> CLASS; MPN TCAN1042HGVDRQ1 -> MLCC-47nF-25V
- COF1: renamed from RSNVP; value 5.1k -> 100nF; footprint R0603 -> C0603; symbol traction-r1:R -> traction-r1:C; MPN R0603-5k1-1% -> MLCC-CLASS
- COR1: renamed from CEXA1; value 220pF -> 100nF
- COR2: renamed from CEXA2; value 1.5nF -> 100nF
- CRST: renamed from USBC; value FS2633D -> 100pF; footprint HLQFP48 -> C0603; symbol traction-r1:FS2633D -> traction-r1:C; MPN FS2633D -> MLCC-100pF-16V
- CSB1: renamed from RSB3; value 220R -> 22uF; footprint R0603 -> C0805; symbol traction-r1:R -> traction-r1:C; MPN R0603-CLASS -> MLCC-CLASS
- CSB2: renamed from RSB4; value 5.1k -> 22uF; footprint R0603 -> C0805; symbol traction-r1:R -> traction-r1:C; MPN R0603-CLASS -> MLCC-CLASS
- CSB3: renamed from CIGN; value 100nF -> 22uF; footprint C0603 -> C0805; MPN MLCC-100nF-50V -> MLCC-CLASS
- CSB3B: renamed from CIGNS; value 100nF -> 22uF
- CSB4: renamed from DIGN; value 1N4148WS -> 10uF; footprint SOD323 -> C0805; symbol traction-r1:D -> traction-r1:C; LCSC C2128 -> CLASS; MPN 1N4148WS -> MLCC-CLASS
- CSB5: renamed from RIGN1; value 5.1k -> 1uF; footprint R0603 -> C0805; symbol traction-r1:R -> traction-r1:C; MPN R0603-5k1 -> MLCC-1uF-16V-X7R-0805
- CSB6: renamed from RIGN2; value 10k -> 4.7uF; footprint R0603 -> C0805; symbol traction-r1:R -> traction-r1:C; MPN R0603-10k -> MLCC-CLASS
- CSB7: renamed from RIGNS1; value 47k -> 10uF; footprint R0603 -> C0805; symbol traction-r1:R -> traction-r1:C; MPN R0603-CLASS -> MLCC-CLASS
- CSB8: renamed from RIGNS2; value 10k -> 10uF; footprint R0603 -> C0805; symbol traction-r1:R -> traction-r1:C; MPN R0603-CLASS -> MLCC-CLASS
- CSCH: renamed from RRDYP2; value 5.1k -> 100nF; footprint R0603 -> C0603; symbol traction-r1:R -> traction-r1:C; MPN R0603-5k1 -> MLCC-100nF-16V
- CSCH2: renamed from RSCH; value 100k -> 100nF; footprint R0603 -> C0603; symbol traction-r1:R -> traction-r1:C; MPN R0603-100k -> MLCC-100nF-16V
- CSCH3: renamed from RV5GP; value 47k -> 100nF; footprint R0603 -> C0603; symbol traction-r1:R -> traction-r1:C; MPN R0603-47k -> MLCC-100nF-16V
- CSINA2: renamed from RCOS1; value 10k -> 220pF; footprint R0603 -> C0603; symbol traction-r1:R -> traction-r1:C; MPN R0603-CLASS -> MLCC-CLASS
- CSINA3: renamed from RCOS2; value 10k -> 22pF; footprint R0603 -> C0603; symbol traction-r1:R -> traction-r1:C; MPN R0603-CLASS -> MLCC-CLASS
- CSIND: renamed from RCOSF1; value 10k -> 47pF; footprint R0603 -> C0603; symbol traction-r1:R -> traction-r1:C; MPN R0603-CLASS -> MLCC-CLASS
- CSINF1: renamed from RCOSF2; value 10k -> 22pF; footprint R0603 -> C0603; symbol traction-r1:R -> traction-r1:C; MPN R0603-CLASS -> MLCC-CLASS
- CSINF2: renamed from RCOSR1; value 120R -> 22pF; footprint R0603 -> C0603; symbol traction-r1:R -> traction-r1:C; MPN R0603-120R -> MLCC-CLASS
- CSNUF: renamed from FMT2; value FUSE-350mA-0603 -> 47nF; footprint F0603 -> C0603; symbol traction-r1:F -> traction-r1:C; MPN FUSE-350mA-0603 -> MLCC-47nF-25V
- CSNVF: renamed from RMT1P; value 10k -> 47nF; footprint R0603 -> C0603; symbol traction-r1:R -> traction-r1:C; MPN R0603-CLASS -> MLCC-47nF-25V
- CSNWF: renamed from RMT1S; value 1k -> 47nF; footprint R0603 -> C0603; symbol traction-r1:R -> traction-r1:C; MPN R0603-CLASS -> MLCC-47nF-25V
- CTAMBF: renamed from LCAN1; value ACT45B-101-2P-TL003 -> 47nF; footprint CMC1210 -> C0603; symbol traction-r1:ACT45B-101-2P-TL003 -> traction-r1:C; MPN ACT45B-101-2P-TL003 -> MLCC-47nF-25V
- CTHSF: renamed from TVSC1; value PESD2IVN24-T -> 47nF; footprint SOT23 -> C0603; symbol traction-r1:PESD2IVN24-T -> traction-r1:C; LCSC C406047 -> CLASS; MPN PESD2IVN24-T -> MLCC-47nF-25V
- CUB1: renamed from RVB2; value 100R -> 3.3nF; footprint R0603 -> C0603; symbol traction-r1:R -> traction-r1:C; MPN R0603-100R -> MLCC-3.3nF-50V
- CUB2: renamed from RVB3; value 100R -> 100nF; footprint R0603 -> C0603; symbol traction-r1:R -> traction-r1:C; MPN R0603-100R -> MLCC-100nF-25V
- CUS1: renamed from UWB1; value OPA376AQDBVRQ1 -> 47nF; footprint SOT23-5 -> C0603; symbol traction-r1:OPA376AQDBVRQ1 -> traction-r1:C; MPN OPA376AQDBVRQ1 -> MLCC-47nF-25V
- CUS2: renamed from UWB2; value OPA376AQDBVRQ1 -> 4.7nF; footprint SOT23-5 -> C0603; symbol traction-r1:OPA376AQDBVRQ1 -> traction-r1:C; MPN OPA376AQDBVRQ1 -> MLCC-4.7nF-50V
- CVB1: renamed from RWB2; value 100R -> 3.3nF; footprint R0603 -> C0603; symbol traction-r1:R -> traction-r1:C; MPN R0603-100R -> MLCC-3.3nF-50V
- CVB2: renamed from RWB3; value 100R -> 100nF; footprint R0603 -> C0603; symbol traction-r1:R -> traction-r1:C; MPN R0603-100R -> MLCC-100nF-25V
- CVBOS: renamed from UAND1; value 74LVC1G11GW-Q100 -> 4.7uF; footprint SOT363 -> C0603; symbol traction-r1:74LVC1G11GW-Q100 -> traction-r1:C; LCSC C548242 -> CLASS; MPN 74LVC1G11GW-Q100 -> MLCC-CLASS
- CVD1: renamed from RSNWP; value 5.1k -> 100pF; footprint R0603 -> C0603; symbol traction-r1:R -> traction-r1:C; MPN R0603-5k1-1% -> MLCC-CLASS
- CVD2: renamed from UMT1; value OPA333AQDBVRQ1 -> 100pF; footprint SOT23-5 -> C0603; symbol traction-r1:OPA333AQDBVRQ1 -> traction-r1:C; LCSC C2058544 -> CLASS; MPN OPA333AQDBVRQ1 -> MLCC-CLASS
- CVDIG: renamed from UAND2; value 74LVC1G11GW-Q100 -> 1uF; footprint SOT363 -> C0603; symbol traction-r1:74LVC1G11GW-Q100 -> traction-r1:C; LCSC C548242 -> CLASS; MPN 74LVC1G11GW-Q100 -> MLCC-CLASS
- CVM1: renamed from REXA3; value 10k -> 220nF; footprint R0603 -> C0603; symbol traction-r1:R -> traction-r1:C; MPN R0603-CLASS -> MLCC-CLASS
- CVM2: renamed from REXA4; value 24k -> 220nF; footprint R0603 -> C0603; symbol traction-r1:R -> traction-r1:C; MPN R0603-CLASS -> MLCC-CLASS
- CVS1: renamed from UVD1; value OPA376AQDBVRQ1 -> 47nF; footprint SOT23-5 -> C0603; symbol traction-r1:OPA376AQDBVRQ1 -> traction-r1:C; MPN OPA376AQDBVRQ1 -> MLCC-47nF-25V
- CVS2: renamed from UVOF; value OPA376AQDBVRQ1 -> 4.7nF; footprint SOT23-5 -> C0603; symbol traction-r1:OPA376AQDBVRQ1 -> traction-r1:C; MPN OPA376AQDBVRQ1 -> MLCC-4.7nF-50V
- CWB1: renamed from RVD1D; value 10k -> 3.3nF; footprint R0603 -> C0603; symbol traction-r1:R -> traction-r1:C; MPN R0603-10k-0.1% -> MLCC-3.3nF-50V
- CWB2: renamed from UVD2; value OPA376AQDBVRQ1 -> 100nF; footprint SOT23-5 -> C0603; symbol traction-r1:OPA376AQDBVRQ1 -> traction-r1:C; MPN OPA376AQDBVRQ1 -> MLCC-100nF-25V
- CWS1: renamed from CVD2; value 100pF -> 47nF; MPN MLCC-CLASS -> MLCC-47nF-25V
- CWS2: renamed from RVD2A; value 10k -> 4.7nF; footprint R0603 -> C0603; symbol traction-r1:R -> traction-r1:C; MPN R0603-10k-0.1% -> MLCC-4.7nF-50V
- CYA: renamed from RLVSD; value 4.7k -> 12pF; footprint R0603 -> C0603; symbol traction-r1:R -> traction-r1:C; MPN R0603-4k7 -> MLCC-12pF-50V
- CYB: renamed from RLVSG; value 10k -> 12pF; footprint R0603 -> C0603; symbol traction-r1:R -> traction-r1:C; MPN R0603-10k -> MLCC-12pF-50V
- DBAT: renamed from ULAT2; value 74LVC1G74DC-Q100 -> BAT46ZFILM; footprint VSSOP8 -> SOD123; symbol traction-r1:74LVC1G74DC-Q100 -> traction-r1:D; LCSC CLASS -> C283255; MPN 74LVC1G74DC-Q100 -> BAT46ZFILM
- DCLR: renamed from RV5GS; value 47k -> BAT46ZFILM; footprint R0603 -> SOD123; symbol traction-r1:R -> traction-r1:D; LCSC CLASS -> C283255; MPN R0603-47k -> BAT46ZFILM
- DCOSP: renamed from UUB2; value OPA376AQDBVRQ1 -> PESD2IVN24-T; footprint SOT23-5 -> SOT23; symbol traction-r1:OPA376AQDBVRQ1 -> traction-r1:PESD2IVN24-T; LCSC CLASS -> C406047; MPN OPA376AQDBVRQ1 -> PESD2IVN24-T
- DFLT1: renamed from UASCG; value 74LVC1G08GW-Q100 -> BAT46ZFILM; footprint SOT353 -> SOD123; symbol traction-r1:74LVC1G08GW-Q100 -> traction-r1:D; LCSC CLASS -> C283255; MPN 74LVC1G08GW-Q100 -> BAT46ZFILM
- DFLT2: renamed from ULAT; value 74LVC1G74DC-Q100 -> BAT46ZFILM; footprint VSSOP8 -> SOD123; symbol traction-r1:74LVC1G74DC-Q100 -> traction-r1:D; LCSC CLASS -> C283255; MPN 74LVC1G74DC-Q100 -> BAT46ZFILM
- DFO: renamed from UVMB1; value OPA348AQDBVRQ1 -> BAT46ZFILM; footprint SOT23-5 -> SOD123; symbol traction-r1:OPA348AQDBVRQ1 -> traction-r1:D; LCSC C2877787 -> C283255; MPN OPA348AQDBVRQ1 -> BAT46ZFILM
- DIGN: renamed from CSCH; value 100nF -> 1N4148WS; footprint C0603 -> SOD323; symbol traction-r1:C -> traction-r1:D; LCSC CLASS -> C2128; MPN MLCC-100nF-16V -> 1N4148WS
- DREVC: renamed from CSB4; value 10uF -> STPS5L60S; footprint C0805 -> SMC; symbol traction-r1:C -> traction-r1:D; LCSC CLASS -> C140620; MPN MLCC-CLASS -> STPS5L60S
- DSINP: renamed from CCOSF1; value 22pF -> PESD2IVN24-T; footprint C0603 -> SOT23; symbol traction-r1:C -> traction-r1:PESD2IVN24-T; LCSC CLASS -> C406047; MPN MLCC-CLASS -> PESD2IVN24-T
- DTVSC: renamed from CSB5; value 1uF -> TPSMC24CA-VR; footprint C0805 -> SMC; symbol traction-r1:C -> traction-r1:D; LCSC CLASS -> C1975284; MPN MLCC-1uF-16V-X7R-0805 -> TPSMC24CA-VR
- FLVC: renamed from CSB6; value 4.7uF -> MF-LSMF300/24X-2; footprint C0805 -> PTC2920; symbol traction-r1:C -> traction-r1:F; LCSC CLASS -> C719172; MPN MLCC-CLASS -> MF-LSMF300/24X-2
- FMT1: renamed from CCAN2; value 1uF -> FUSE-350mA-0603; footprint C0603 -> F0603; symbol traction-r1:C -> traction-r1:F; MPN MLCC-1uF-25V -> FUSE-350mA-0603
- FMT2: renamed from CCT2; value 4.7nF -> FUSE-350mA-0603; footprint C0603 -> F0603; symbol traction-r1:C -> traction-r1:F; MPN MLCC-4.7nF-50V -> FUSE-350mA-0603
- FVBH: renamed from CSB7; value 10uF -> MF-LSMF300/24X-2; footprint C0805 -> PTC2920; symbol traction-r1:C -> traction-r1:F; LCSC CLASS -> C719172; MPN MLCC-CLASS -> MF-LSMF300/24X-2
- FVBL: renamed from CSB8; value 10uF -> MF-LSMF300/24X-2; footprint C0805 -> PTC2920; symbol traction-r1:C -> traction-r1:F; LCSC CLASS -> C719172; MPN MLCC-CLASS -> MF-LSMF300/24X-2
- JLEM: renamed from CVB2; value 100nF -> T2M-105-01-L-D-TH-WT; footprint C0603 -> HDR2x5; symbol traction-r1:C -> traction-r1:T2M-105-01-L-D-TH-WT; MPN MLCC-100nF-25V -> T2M-105-01-L-D-TH-WT
- JSWD: renamed from QBAL; value SQ2310ES -> FTSH-105-01-L-DV-K; footprint SOT23 -> HDR2x5-1.27; symbol traction-r1:SQ2310ES -> traction-r1:FTSH-105-01-L-DV-K; MPN SQ2310ES -> FTSH-105-01-L-DV-K
- LCAN1: renamed from LVS3; value FB-470R -> ACT45B-101-2P-TL003; footprint FB0603 -> CMC1210; symbol traction-r1:L -> traction-r1:ACT45B-101-2P-TL003; MPN FB-470R-CLASS -> ACT45B-101-2P-TL003
- LCAN2: renamed from RHWP; value 10k -> ACT45B-101-2P-TL003; footprint R0603 -> CMC1210; symbol traction-r1:R -> traction-r1:ACT45B-101-2P-TL003; MPN R0603-10k-1% -> ACT45B-101-2P-TL003
- LCOR: renamed from USCH; value 74LVC3G17DC-Q100 -> XAL4020-222MEC; footprint VSSOP8 -> XAL4020; symbol traction-r1:74LVC3G17DC-Q100 -> traction-r1:L; MPN 74LVC3G17DC-Q100 -> XAL4020-222MEC
- LFC: renamed from CVBOS; value 4.7uF -> FB-120R-3A; footprint C0603 -> FB1206; symbol traction-r1:C -> traction-r1:L; MPN MLCC-CLASS -> FB-120R-3A
- LSBC: renamed from USCH2; value 74LVC3G17DC-Q100 -> XAL4040-103MEC; footprint VSSOP8 -> XAL4040; symbol traction-r1:74LVC3G17DC-Q100 -> traction-r1:L; MPN 74LVC3G17DC-Q100 -> XAL4040-103MEC
- LUB: renamed from CWB1; value 3.3nF -> FB-220R-1A; footprint C0603 -> FB0805; symbol traction-r1:C -> traction-r1:L; MPN MLCC-3.3nF-50V -> FB-220R-1A
- renumbered CCOSF2 to CSINA1, RARB to RFLTC, RASCP to RFLTD, RLAT1 to RQDM
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Connections:
- wire segments 907 -> 955
Other:
- note added: "rev A.12 - 26 sections - 288 components"
- note removed: "rev A.11 - 26 sections - 288 components"
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