File: kicad5/traction/traction-card.sch (KiCad schematic (older format))
At the start: 288 parts, among them Y1 CX3225GA40000D0PTVCC

Commit message: Rev A.13: round 14 — three reviews of cfd35a7 (F143-F158): MCU map vs NXP netlist, fail-closed firmware, terminal-fault protection
- Pin freeze reopened and closed: H5 is V15 (1.5 V, was on VREF5) and J7 is V25 (regulator output,
  was grounded); whole map re-derived against NXP's GEN3 net report NET-91122_C (U513, 244 balls) —
  every supply ball and 164/165 port names agree; HW_ID/NTC_A/MT2_SIG/ASC_REQ moved to netlist-confirmed
  balls (B5/T15/D5/U4); KiCad symbol numbered by physical ball, mutation-tested; CNMOS 1 nF.
- Firmware (214 tests / 1622 checks, ASan/UBSan, target-check): DESAT hold for every caller, 64-bit
  monotonic clock, keep_hv from rule (b) reliance at any speed, IMCR placeholders = build error,
  config-matches vs protection-locked, arming-evidence record (fail closed), torque feasibility witness,
  stuck-channel detection, stuck-on discharge detection; board map regenerated.
- Analog: excitation monitor 18 k/42.2 k/84.5 k + 220 pF C_AAF; exciter SMCJ8.5CA + MF-MSMF020 per line;
  motor-temp SMAJ5.0A + 0438.375WRA; bias-LDO 47 R ballast, UCC12051-Q1 primary; UCC14141-Q1 VDE cert.
- Docs: contract FW-22..FW-26 + keep_hv; design-basis §11m; variants/cost/dfm/README; disposition + CSV;
  EXTRACTED §31/§32 + archived datasheets; report-template defect fixed; Marine at A.13 (86/22/0).

ERC 945/0 · design-verify 130/23/0 · sim 23/6/0 · sheets 2045/2045 · BOM 8XX SiC ₹72,492.

Co-Authored-By: Claude Fable 5.1 <noreply@anthropic.com>
Parts:
- removed CMA1: 1uF, C0603, symbol traction-r1:C
- removed UMCU: S32K396EHT1MJBST, MAPBGA289, symbol traction-r1:S32K396EHT1MJBST
- added JICC: IPL1-120-01-L-D-K, HDR2x20-2.54, symbol traction-r1:IPL1-120-01-L-D-K
- added LVS2, LVS3, LVS4: FB-470R, FB0603, symbol traction-r1:L
- added RCPD0, RCPD1, RCPD2, RCPD3, RHWP: 10k, R0603, symbol traction-r1:R
- CAND1: renamed from CFLTF; value 100pF -> 100nF; MPN MLCC-100pF-16V -> MLCC-CLASS
- CAND2: renamed from CFLTF2; value 100pF -> 100nF; MPN MLCC-100pF-16V -> MLCC-CLASS
- CASCG: renamed from RASCP; value 10k -> 100nF; footprint R0603 -> C0603; symbol traction-r1:R -> traction-r1:C; MPN R0603-10k -> MLCC-100nF-16V
- CBAL: renamed from CSB2; value 22uF -> 1nF; footprint C0805 -> C0603; MPN MLCC-CLASS -> MLCC-1nF-50V-C0G
- CBTC: renamed from CSB3; value 22uF -> 47nF; footprint C0805 -> C0603
- CBTP: renamed from CSB3B; value 22uF -> 22nF
- CCAN1: renamed from RCT2A; value 60.4R -> 1uF; footprint R0603 -> C0603; symbol traction-r1:R -> traction-r1:C; MPN R0603-60R4-1% -> MLCC-1uF-25V
- CCAN2: renamed from LVS4; value FB-470R -> 1uF; footprint FB0603 -> C0603; symbol traction-r1:L -> traction-r1:C; MPN FB-470R-CLASS -> MLCC-1uF-25V
- CCLR: renamed from CLAT2; value 100nF -> 15nF; MPN MLCC-100nF-16V -> MLCC-15nF-50V-C0G
- CCOSA1: renamed from RCOSF2; value 12k -> 22pF; footprint R0603 -> C0603; symbol traction-r1:R -> traction-r1:C; MPN R0603-CLASS -> MLCC-CLASS
- CCOSA2: renamed from RCOSR1; value 120R -> 220pF; footprint R0603 -> C0603; symbol traction-r1:R -> traction-r1:C; MPN R0603-120R -> MLCC-CLASS
- CCOSA3: renamed from RCOSR2; value 120R -> 22pF; footprint R0603 -> C0603; symbol traction-r1:R -> traction-r1:C; MPN R0603-120R -> MLCC-CLASS
- CCOSD: renamed from JLEM; value T2M-105-01-L-D-TH-WT -> 47pF; footprint HDR2x5 -> C0603; symbol traction-r1:T2M-105-01-L-D-TH-WT -> traction-r1:C; MPN T2M-105-01-L-D-TH-WT -> MLCC-CLASS
- CCOSF1: renamed from USNSU; value HC5FW900-S -> 22pF; footprint OffBoard -> C0603; symbol traction-r1:HC5FW900-S -> traction-r1:C; MPN HC5FW900-S -> MLCC-CLASS
- CCOSF2: renamed from USNSV; value HC5FW900-S -> 22pF; footprint OffBoard -> C0603; symbol traction-r1:HC5FW900-S -> traction-r1:C; MPN HC5FW900-S -> MLCC-CLASS
- CCT1: renamed from RCT2B; value 60.4R -> 4.7nF; footprint R0603 -> C0603; symbol traction-r1:R -> traction-r1:C; MPN R0603-60R4-1% -> MLCC-4.7nF-50V
- CCT2: renamed from JICC; value IPL1-120-01-L-D-K -> 4.7nF; footprint HDR2x20-2.54 -> C0603; symbol traction-r1:IPL1-120-01-L-D-K -> traction-r1:C; MPN IPL1-120-01-L-D-K -> MLCC-4.7nF-50V
- CEXA1: renamed from CEXD; value 4.7uF -> 220pF
- CEXA2: renamed from CLDE; value 22uF -> 1.5nF
- CEXA3: renamed from CLDEC; value 270pF -> 100nF
- CEXA4: renamed from REXA1; value 3k -> 47pF; footprint R0603 -> C0603; symbol traction-r1:R -> traction-r1:C; MPN R0603-CLASS -> MLCC-CLASS
- CEXD: renamed from REXA2; value 10k -> 4.7uF; footprint R0603 -> C0603; symbol traction-r1:R -> traction-r1:C; MPN R0603-CLASS -> MLCC-CLASS
- CEXM: renamed from REXA3; value 10k -> 220pF; footprint R0603 -> C0603; symbol traction-r1:R -> traction-r1:C; MPN R0603-CLASS -> MLCC-220pF-50V-C0G
- CFLTD: renamed from CSCH; value 100nF -> 3.3nF; MPN MLCC-100nF-16V -> MLCC-3.3nF-50V-C0G
- CFLTF: renamed from CSCH2; value 100nF -> 100pF; MPN MLCC-100nF-16V -> MLCC-100pF-16V
- CFLTF2: renamed from CSCH3; value 100nF -> 100pF; MPN MLCC-100nF-16V -> MLCC-100pF-16V
- CIGN: renamed from RIGN2; value 10k -> 100nF; footprint R0603 -> C0603; symbol traction-r1:R -> traction-r1:C; MPN R0603-10k -> MLCC-100nF-50V
- CIGNS: renamed from RIGNS1; value 47k -> 100nF; footprint R0603 -> C0603; symbol traction-r1:R -> traction-r1:C; MPN R0603-CLASS -> MLCC-CLASS
- CILK: renamed from RILK4; value 10k -> 2.2nF; footprint R0603 -> C0603; symbol traction-r1:R -> traction-r1:C; MPN R0603-10k -> MLCC-2.2nF-50V
- CLAT: renamed from RFS1; value 1k -> 100nF; footprint R0603 -> C0603; symbol traction-r1:R -> traction-r1:C; MPN R0603-1k -> MLCC-100nF-16V
- CLAT2: renamed from DCLR; value BAT46ZFILM -> 100nF; footprint SOD123 -> C0603; symbol traction-r1:D -> traction-r1:C; LCSC C283255 -> CLASS; MPN BAT46ZFILM -> MLCC-100nF-16V
- CLDE: renamed from REXA4; value 24k -> 22uF; footprint R0603 -> C0603; symbol traction-r1:R -> traction-r1:C; MPN R0603-CLASS -> MLCC-CLASS
- CLDEC: renamed from REXB1; value 24k -> 270pF; footprint R0603 -> C0603; symbol traction-r1:R -> traction-r1:C; MPN R0603-CLASS -> MLCC-CLASS
- CLVC1: renamed from DREVC; value STPS5L60S -> 4.7uF; footprint SMC -> C1206; symbol traction-r1:D -> traction-r1:C; LCSC C140620 -> CLASS; MPN STPS5L60S -> MLCC-4.7uF-50V
- CLVC2: renamed from DTVSC; value TPSMC24CA-VR -> 22uF; footprint SMC -> C1210; symbol traction-r1:D -> traction-r1:C; LCSC C1975284 -> CLASS; MPN TPSMC24CA-VR -> MLCC-22uF-50V
- CLVSM: renamed from FLVC; value MF-LSMF300/24X-2 -> 100nF; footprint PTC2920 -> C0603; symbol traction-r1:F -> traction-r1:C; LCSC C719172 -> CLASS; MPN MF-LSMF300/24X-2 -> MLCC-100nF-50V
- CMA1: renamed from CMD1; value 100nF -> 1uF; footprint C0402 -> C0603; MPN MLCC-100nF-16V -> MLCC-1uF-16V
- CMA2: renamed from CMD10; footprint C0402 -> C0603
- CMD8: renamed from CYA; value 12pF -> 100nF; footprint C0603 -> C0402; MPN MLCC-12pF-50V -> MLCC-100nF-16V
- CMD9: renamed from CYB; value 12pF -> 100nF; footprint C0603 -> C0402; MPN MLCC-12pF-50V -> MLCC-100nF-16V
- CMT1F: renamed from TVSM2; value PESD5V0L1BA -> 47nF; footprint SOD323 -> C0603; symbol traction-r1:R -> traction-r1:C; MPN PESD5V0L1BA -> MLCC-47nF-25V
- CMT2F: renamed from LCAN1; value ACT45B-101-2P-TL003 -> 47nF; footprint CMC1210 -> C0603; symbol traction-r1:ACT45B-101-2P-TL003 -> traction-r1:C; MPN ACT45B-101-2P-TL003 -> MLCC-47nF-25V
- COF1: renamed from CVD2; value 100pF -> 100nF
- COR1: renamed from RILK2; value 10k -> 100nF; footprint R0603 -> C0603; symbol traction-r1:R -> traction-r1:C; MPN R0603-10k -> MLCC-CLASS
- COR2: renamed from RILK3; value 10k -> 100nF; footprint R0603 -> C0603; symbol traction-r1:R -> traction-r1:C; MPN R0603-10k -> MLCC-CLASS
- CRST: renamed from QLVS; value DMP6023LEQ-13 -> 100pF; footprint SOT223 -> C0603; symbol traction-r1:DMP6023LEQ-13 -> traction-r1:C; MPN DMP6023LEQ-13 -> MLCC-100pF-16V
- CSB1: renamed from CSB4; value 10uF -> 22uF
- CSB2: renamed from CSB5; value 1uF -> 22uF; MPN MLCC-1uF-16V-X7R-0805 -> MLCC-CLASS
- CSB3: renamed from CSB6; value 4.7uF -> 22uF
- CSB3B: renamed from CSB7; value 10uF -> 22uF; footprint C0805 -> C0603
- CSB5: renamed from CVBOS; value 4.7uF -> 1uF; footprint C0603 -> C0805; MPN MLCC-CLASS -> MLCC-1uF-16V-X7R-0805
- CSB6: renamed from CVDIG; value 1uF -> 4.7uF; footprint C0603 -> C0805
- CSB7: renamed from DBAT; value BAT46ZFILM -> 10uF; footprint SOD123 -> C0805; symbol traction-r1:D -> traction-r1:C; LCSC C283255 -> CLASS; MPN BAT46ZFILM -> MLCC-CLASS
- CSB8: renamed from LCOR; value XAL4020-222MEC -> 10uF; footprint XAL4020 -> C0805; symbol traction-r1:L -> traction-r1:C; MPN XAL4020-222MEC -> MLCC-CLASS
- CSCH: renamed from DFLT1; value BAT46ZFILM -> 100nF; footprint SOD123 -> C0603; symbol traction-r1:D -> traction-r1:C; LCSC C283255 -> CLASS; MPN BAT46ZFILM -> MLCC-100nF-16V
- CSCH2: renamed from DFLT2; value BAT46ZFILM -> 100nF; footprint SOD123 -> C0603; symbol traction-r1:D -> traction-r1:C; LCSC C283255 -> CLASS; MPN BAT46ZFILM -> MLCC-100nF-16V
- CSCH3: renamed from RDRB; value 10k -> 100nF; footprint R0603 -> C0603; symbol traction-r1:R -> traction-r1:C; MPN R0603-10k -> MLCC-100nF-16V
- CSINA1: renamed from RSINF2; value 12k -> 22pF; footprint R0603 -> C0603; symbol traction-r1:R -> traction-r1:C; MPN R0603-CLASS -> MLCC-CLASS
- CSINA2: renamed from RSINR1; value 120R -> 220pF; footprint R0603 -> C0603; symbol traction-r1:R -> traction-r1:C; MPN R0603-120R -> MLCC-CLASS
- CSINA3: renamed from RSINR2; value 120R -> 22pF; footprint R0603 -> C0603; symbol traction-r1:R -> traction-r1:C; MPN R0603-120R -> MLCC-CLASS
- CSIND: renamed from DCOSP; value PESD2IVN24-T -> 47pF; footprint SOT23 -> C0603; symbol traction-r1:PESD2IVN24-T -> traction-r1:C; LCSC C406047 -> CLASS; MPN PESD2IVN24-T -> MLCC-CLASS
- CSINF2: renamed from CCOSA2; value 220pF -> 22pF
- CSNUF: renamed from RTAMB; value 10k -> 47nF; footprint R0603 -> C0603; symbol traction-r1:R -> traction-r1:C; MPN NTC-10k-0603 -> MLCC-47nF-25V
- CSNVF: renamed from RTAMBP; value 10k -> 47nF; footprint R0603 -> C0603; symbol traction-r1:R -> traction-r1:C; MPN R0603-10k-1% -> MLCC-47nF-25V
- CSNWF: renamed from RTHS; value 10k -> 47nF; footprint R0603 -> C0603; symbol traction-r1:R -> traction-r1:C; MPN NTC-10k-0603 -> MLCC-47nF-25V
- CTHSF: renamed from FMT1; value FUSE-350mA-0603 -> 47nF; footprint F0603 -> C0603; symbol traction-r1:F -> traction-r1:C; MPN FUSE-350mA-0603 -> MLCC-47nF-25V
- CUB1: renamed from UVB1; value OPA376AQDBVRQ1 -> 3.3nF; footprint SOT23-5 -> C0603; symbol traction-r1:OPA376AQDBVRQ1 -> traction-r1:C; MPN OPA376AQDBVRQ1 -> MLCC-3.3nF-50V
- CUB2: renamed from UVB2; value OPA376AQDBVRQ1 -> 100nF; footprint SOT23-5 -> C0603; symbol traction-r1:OPA376AQDBVRQ1 -> traction-r1:C; MPN OPA376AQDBVRQ1 -> MLCC-100nF-25V
- CUS1: renamed from CVB1; value 3.3nF -> 47nF; MPN MLCC-3.3nF-50V -> MLCC-47nF-25V
- CUS2: renamed from CVB2; value 100nF -> 4.7nF; MPN MLCC-100nF-25V -> MLCC-4.7nF-50V
- CV25: renamed from RMRST; value 10k -> 220nF; footprint R0603 -> C0603; symbol traction-r1:R -> traction-r1:C; MPN R0603-10k -> MLCC-220nF-10V-X7R
- CVB1: renamed from UWB1; value OPA376AQDBVRQ1 -> 3.3nF; footprint SOT23-5 -> C0603; symbol traction-r1:OPA376AQDBVRQ1 -> traction-r1:C; MPN OPA376AQDBVRQ1 -> MLCC-3.3nF-50V
- CVB2: renamed from UWB2; value OPA376AQDBVRQ1 -> 100nF; footprint SOT23-5 -> C0603; symbol traction-r1:OPA376AQDBVRQ1 -> traction-r1:C; MPN OPA376AQDBVRQ1 -> MLCC-100nF-25V
- CVBOS: renamed from LSBC; value XAL4040-103MEC -> 4.7uF; footprint XAL4040 -> C0603; symbol traction-r1:L -> traction-r1:C; MPN XAL4040-103MEC -> MLCC-CLASS
- CVD1: renamed from RVD2A; value 10k -> 100pF; footprint R0603 -> C0603; symbol traction-r1:R -> traction-r1:C; MPN R0603-10k-0.1% -> MLCC-CLASS
- CVD2: renamed from RSNVP; value 5.1k -> 100pF; footprint R0603 -> C0603; symbol traction-r1:R -> traction-r1:C; MPN R0603-5k1-1% -> MLCC-CLASS
- CVDIG: renamed from RAGT; value 0R -> 1uF; footprint R0603 -> C0603; symbol traction-r1:R -> traction-r1:C; MPN R0603-CLASS -> MLCC-CLASS
- CVM1: renamed from RVM3; value 24k -> 220nF; footprint R0603 -> C0603; symbol traction-r1:R -> traction-r1:C; MPN R0603-24k-1% -> MLCC-CLASS
- CVM2: renamed from RVM4; value 24k -> 220nF; footprint R0603 -> C0603; symbol traction-r1:R -> traction-r1:C; MPN R0603-24k-1% -> MLCC-CLASS
- CVS1: renamed from CWB1; value 3.3nF -> 47nF; MPN MLCC-3.3nF-50V -> MLCC-47nF-25V
- CVS2: renamed from CWB2; value 100nF -> 4.7nF; MPN MLCC-100nF-25V -> MLCC-4.7nF-50V
- CWB1: renamed from UVD1; value OPA376AQDBVRQ1 -> 3.3nF; footprint SOT23-5 -> C0603; symbol traction-r1:OPA376AQDBVRQ1 -> traction-r1:C; MPN OPA376AQDBVRQ1 -> MLCC-3.3nF-50V
- CWB2: renamed from UVOF; value OPA376AQDBVRQ1 -> 100nF; footprint SOT23-5 -> C0603; symbol traction-r1:OPA376AQDBVRQ1 -> traction-r1:C; MPN OPA376AQDBVRQ1 -> MLCC-100nF-25V
- CWS1: renamed from COF1; value 100nF -> 47nF; MPN MLCC-CLASS -> MLCC-47nF-25V
- CWS2: renamed from CVD1; value 100pF -> 4.7nF; MPN MLCC-CLASS -> MLCC-4.7nF-50V
- CYA: renamed from Y1; value CX3225GA40000D0PTVCC -> 12pF; footprint X3225 -> C0603; symbol traction-r1:Y -> traction-r1:C; LCSC C6009848 -> CLASS; MPN CX3225GA40000D0PTVCC -> MLCC-12pF-50V
- CYB: renamed from JSWD; value FTSH-105-01-L-DV-K -> 12pF; footprint HDR2x5-1.27 -> C0603; symbol traction-r1:FTSH-105-01-L-DV-K -> traction-r1:C; MPN FTSH-105-01-L-DV-K -> MLCC-12pF-50V
- DBAT: renamed from RDBG; value 10k -> BAT46ZFILM; footprint R0603 -> SOD123; symbol traction-r1:R -> traction-r1:D; LCSC CLASS -> C283255; MPN R0603-CLASS -> BAT46ZFILM
- DCLR: renamed from RENP1; value 5.1k -> BAT46ZFILM; footprint R0603 -> SOD123; symbol traction-r1:R -> traction-r1:D; LCSC CLASS -> C283255; MPN R0603-5k1 -> BAT46ZFILM
- DCOSP: renamed from RCOSF1; value 12k -> PESD2IVN24-T; footprint R0603 -> SOT23; symbol traction-r1:R -> traction-r1:PESD2IVN24-T; LCSC CLASS -> C406047; MPN R0603-CLASS -> PESD2IVN24-T
- DFLT1: renamed from RFCB; value 100k -> BAT46ZFILM; footprint R0603 -> SOD123; symbol traction-r1:R -> traction-r1:D; LCSC CLASS -> C283255; MPN R0603-100k -> BAT46ZFILM
- DFLT2: renamed from RFLTC; value 10k -> BAT46ZFILM; footprint R0603 -> SOD123; symbol traction-r1:R -> traction-r1:D; LCSC CLASS -> C283255; MPN R0603-10k -> BAT46ZFILM
- DFO: renamed from RFS2; value 10k -> BAT46ZFILM; footprint R0603 -> SOD123; symbol traction-r1:R -> traction-r1:D; LCSC CLASS -> C283255; MPN R0603-10k -> BAT46ZFILM
- DIGN: renamed from RIGNS2; value 10k -> 1N4148WS; footprint R0603 -> SOD323; symbol traction-r1:R -> traction-r1:D; LCSC CLASS -> C2128; MPN R0603-CLASS -> 1N4148WS
- DREVC: renamed from FVBH; value MF-LSMF300/24X-2 -> STPS5L60S; footprint PTC2920 -> SMC; symbol traction-r1:F -> traction-r1:D; LCSC C719172 -> C140620; MPN MF-LSMF300/24X-2 -> STPS5L60S
- DSINP: renamed from RSINF1; value 12k -> PESD2IVN24-T; footprint R0603 -> SOT23; symbol traction-r1:R -> traction-r1:PESD2IVN24-T; LCSC CLASS -> C406047; MPN R0603-CLASS -> PESD2IVN24-T
- DTVSC: renamed from FVBL; value MF-LSMF300/24X-2 -> TPSMC24CA-VR; footprint PTC2920 -> SMC; symbol traction-r1:F -> traction-r1:D; LCSC C719172 -> C1975284; MPN MF-LSMF300/24X-2 -> TPSMC24CA-VR
- FEXN: renamed from REXB2; value 24k -> MF-MSMF020; footprint R0603 -> 1206; symbol traction-r1:R -> traction-r1:F; MPN R0603-CLASS -> MF-MSMF020
- FEXP: renamed from REXB3; value 24k -> MF-MSMF020; footprint R0603 -> 1206; symbol traction-r1:R -> traction-r1:F; MPN R0603-CLASS -> MF-MSMF020
- FLVC: renamed from LFC; value FB-120R-3A -> MF-LSMF300/24X-2; footprint FB1206 -> PTC2920; symbol traction-r1:L -> traction-r1:F; LCSC CLASS -> C719172; MPN FB-120R-3A -> MF-LSMF300/24X-2
- FMT1: renamed from TVSC1; value PESD2IVN24-T -> 0438.375WRA; footprint SOT23 -> F0603; symbol traction-r1:PESD2IVN24-T -> traction-r1:F; LCSC C406047 -> CLASS; MPN PESD2IVN24-T -> 0438.375WRA
- FMT2: renamed from UCAN1; value TCAN1042HGVDRQ1 -> 0438.375WRA; footprint SOIC8 -> F0603; symbol traction-r1:TCAN1042HGVDRQ1 -> traction-r1:F; LCSC C132550 -> CLASS; MPN TCAN1042HGVDRQ1 -> 0438.375WRA
- FVBH: renamed from RLVSD; value 4.7k -> MF-LSMF300/24X-2; footprint R0603 -> PTC2920; symbol traction-r1:R -> traction-r1:F; LCSC CLASS -> C719172; MPN R0603-4k7 -> MF-LSMF300/24X-2
- FVBL: renamed from RLVSG; value 10k -> MF-LSMF300/24X-2; footprint R0603 -> PTC2920; symbol traction-r1:R -> traction-r1:F; LCSC CLASS -> C719172; MPN R0603-10k -> MF-LSMF300/24X-2
- FVS1: renamed from RCPD3; value 10k -> MF-LSMF; footprint R0603 -> PTC1206; symbol traction-r1:R -> traction-r1:F; MPN R0603-10k -> MF-LSMF-CLASS
- JLEM: renamed from CUS2; value 4.7nF -> T2M-105-01-L-D-TH-WT; footprint C0603 -> HDR2x5; symbol traction-r1:C -> traction-r1:T2M-105-01-L-D-TH-WT; MPN MLCC-4.7nF-50V -> T2M-105-01-L-D-TH-WT
- JSWD: renamed from QLVN; value 2N7002 -> FTSH-105-01-L-DV-K; footprint SOT23 -> HDR2x5-1.27; symbol traction-r1:2N7002 -> traction-r1:FTSH-105-01-L-DV-K; LCSC C8545 -> CLASS; MPN 2N7002 -> FTSH-105-01-L-DV-K
- JVEH: renamed from RCPD2; value 10k -> TE 770669-1 (AMPSEAL 23); footprint R0603 -> AMPSEAL23; symbol traction-r1:R -> traction-r1:TE_770669-1__AMPSEAL_23_; MPN R0603-10k -> TE 770669-1 (AMPSEAL 23)
- LCAN1: renamed from UCAN2; value TCAN1042HGVDRQ1 -> ACT45B-101-2P-TL003; footprint SOIC8 -> CMC1210; symbol traction-r1:TCAN1042HGVDRQ1 -> traction-r1:ACT45B-101-2P-TL003; LCSC C132550 -> CLASS; MPN TCAN1042HGVDRQ1 -> ACT45B-101-2P-TL003
- LCAN2: renamed from LVS1; value FB-470R -> ACT45B-101-2P-TL003; footprint FB0603 -> CMC1210; symbol traction-r1:L -> traction-r1:ACT45B-101-2P-TL003; MPN FB-470R-CLASS -> ACT45B-101-2P-TL003
- LCOR: renamed from RSB1; value 52.3k -> XAL4020-222MEC; footprint R0603 -> XAL4020; symbol traction-r1:R -> traction-r1:L; MPN R0603-CLASS -> XAL4020-222MEC
- LFC: renamed from RLVSM; value 1k -> FB-120R-3A; footprint R0603 -> FB1206; symbol traction-r1:R -> traction-r1:L; MPN R0603-1k -> FB-120R-3A
- LSBC: renamed from RSB2; value 10k -> XAL4040-103MEC; footprint R0603 -> XAL4040; symbol traction-r1:R -> traction-r1:L; MPN R0603-CLASS -> XAL4040-103MEC
- LUB: renamed from CVS1; value 47nF -> FB-220R-1A; footprint C0603 -> FB0805; symbol traction-r1:C -> traction-r1:L; MPN MLCC-47nF-25V -> FB-220R-1A
- LVB: renamed from CWS1; value 47nF -> FB-220R-1A; footprint C0603 -> FB0805; symbol traction-r1:C -> traction-r1:L; MPN MLCC-47nF-25V -> FB-220R-1A
- LVS1: renamed from RHWP; value 10k -> FB-470R; footprint R0603 -> FB0603; symbol traction-r1:R -> traction-r1:L; MPN R0603-10k-1% -> FB-470R-CLASS
- LWB: renamed from ROF1; value 9.1k -> FB-220R-1A; footprint R0603 -> FB0805; symbol traction-r1:R -> traction-r1:L; MPN R0603-CLASS -> FB-220R-1A
- QBAL: renamed from CBTP; value 22nF -> SQ2310ES; footprint C0603 -> SOT23; symbol traction-r1:C -> traction-r1:SQ2310ES; MPN MLCC-CLASS -> SQ2310ES
- QLVN: renamed from CLVC2; value 22uF -> 2N7002; footprint C1210 -> SOT23; symbol traction-r1:C -> traction-r1:2N7002; LCSC CLASS -> C8545; MPN MLCC-22uF-50V -> 2N7002
- QLVS: renamed from CLVSM; value 100nF -> DMP6023LEQ-13; footprint C0603 -> SOT223; symbol traction-r1:C -> traction-r1:DMP6023LEQ-13; MPN MLCC-100nF-50V -> DMP6023LEQ-13
- RAGT: renamed from RSB3; value 220R -> 0R
- RARB: renamed from RFS3; value 1k -> 10k; MPN R0603-1k -> R0603-10k
- RASCP: renamed from RFS4; value 1k -> 10k; MPN ESR03EZPF1001 -> R0603-10k
- RBOOT: renamed from CLVC1; value 4.7uF -> 10k; footprint C1206 -> R0603; symbol traction-r1:C -> traction-r1:R; MPN MLCC-4.7uF-50V -> R0603-10k
- RCOS1: renamed from USNSW; value HC5FW900-S -> 12k; footprint OffBoard -> R0603; symbol traction-r1:HC5FW900-S -> traction-r1:R; MPN HC5FW900-S -> R0603-CLASS
- RCOS2: renamed from UUB1; value OPA376AQDBVRQ1 -> 12k; footprint SOT23-5 -> R0603; symbol traction-r1:OPA376AQDBVRQ1 -> traction-r1:R; MPN OPA376AQDBVRQ1 -> R0603-CLASS
- RCOSF1: renamed from UUB2; value OPA376AQDBVRQ1 -> 12k; footprint SOT23-5 -> R0603; symbol traction-r1:OPA376AQDBVRQ1 -> traction-r1:R; MPN OPA376AQDBVRQ1 -> R0603-CLASS
- RCOSF2: renamed from CUB1; value 3.3nF -> 12k; footprint C0603 -> R0603; symbol traction-r1:C -> traction-r1:R; MPN MLCC-3.3nF-50V -> R0603-CLASS
- RCOSR1: renamed from CUB2; value 100nF -> 120R; footprint C0603 -> R0603; symbol traction-r1:C -> traction-r1:R; MPN MLCC-100nF-25V -> R0603-120R
- RCOSR2: renamed from CUS1; value 47nF -> 120R; footprint C0603 -> R0603; symbol traction-r1:C -> traction-r1:R; MPN MLCC-47nF-25V -> R0603-120R
- RCT1A: renamed from JVEH; value TE 770669-1 (AMPSEAL 23) -> 60.4R; footprint AMPSEAL23 -> R0603; symbol traction-r1:TE_770669-1__AMPSEAL_23_ -> traction-r1:R; MPN TE 770669-1 (AMPSEAL 23) -> R0603-60R4-1%
- RCT1B: renamed from FVS1; value MF-LSMF -> 60.4R; footprint PTC1206 -> R0603; symbol traction-r1:F -> traction-r1:R; MPN MF-LSMF-CLASS -> R0603-60R4-1%
- RCT2A: renamed from RCPD0; value 10k -> 60.4R; MPN R0603-10k -> R0603-60R4-1%
- RCT2B: renamed from RCPD1; value 10k -> 60.4R; MPN R0603-10k -> R0603-60R4-1%
- RDBG: renamed from RSB4; value 5.1k -> 10k
- REXA1: renamed from REXB4; value 24k -> 3k
- REXA2: renamed from REXM1; value 5.1k -> 10k
- REXA3: renamed from REXM2; value 12k -> 10k
- REXA4: renamed from REXM3; value 5.1k -> 24k
- REXB2: renamed from RLDE1; value 38.3k -> 24k
- REXB3: renamed from RLDE2; value 10k -> 24k
- REXB4: renamed from RSDN; value 10k -> 24k
- REXM1: renamed from DSINP; value PESD2IVN24-T -> 18k; footprint SOT23 -> R0603; symbol traction-r1:PESD2IVN24-T -> traction-r1:R; LCSC C406047 -> CLASS; MPN PESD2IVN24-T -> R0603-18k-1%
- REXM2: renamed from CSINA1; value 22pF -> 42.2k; footprint C0603 -> R0603; symbol traction-r1:C -> traction-r1:R; MPN MLCC-CLASS -> R0603-42k2-1%
- REXM3: renamed from CSINA2; value 220pF -> 18k; footprint C0603 -> R0603; symbol traction-r1:C -> traction-r1:R; MPN MLCC-CLASS -> R0603-18k-1%
- REXM4: renamed from CSINA3; value 22pF -> 84.5k; footprint C0603 -> R0603; symbol traction-r1:C -> traction-r1:R; MPN MLCC-CLASS -> R0603-84k5-1%
- RFCB: renamed from RFLTP2; value 5.1k -> 100k; MPN R0603-5k1 -> R0603-100k
- RFLTP1: renamed from RQDM; value 10k -> 5.1k; MPN R0603-10k -> R0603-5k1
- RFLTP2: renamed from RRDB; value 100k -> 5.1k; MPN R0603-100k -> R0603-5k1
- RFS1: renamed from RLAT1; value 10k -> 1k; MPN R0603-10k -> R0603-1k
- RFS2: renamed from ZSET; value BZT52-B5V6 -> 10k; footprint SOD123 -> R0603; symbol traction-r1:D -> traction-r1:R; MPN BZT52-B5V6 -> R0603-10k
- RFS3: renamed from UOR1; value 74LVC1G32GW-Q100 -> 1k; footprint SOT353 -> R0603; symbol traction-r1:74LVC1G32GW-Q100 -> traction-r1:R; LCSC C548334 -> CLASS; MPN 74LVC1G32GW-Q100 -> R0603-1k
- RFS4: renamed from UOR2; value 74LVC1G32GW-Q100 -> 1k; footprint SOT353 -> R0603; symbol traction-r1:74LVC1G32GW-Q100 -> traction-r1:R; LCSC C548334 -> CLASS; MPN 74LVC1G32GW-Q100 -> ESR03EZPF1001
- RGPD: renamed from RRDYP1; value 5.1k -> 10k; MPN R0603-5k1 -> R0603-10k
- RIGN1: renamed from UAND1; value 74LVC1G11GW-Q100 -> 5.1k; footprint SOT363 -> R0603; symbol traction-r1:74LVC1G11GW-Q100 -> traction-r1:R; LCSC C548242 -> CLASS; MPN 74LVC1G11GW-Q100 -> R0603-5k1
- RIGN2: renamed from UAND2; value 74LVC1G11GW-Q100 -> 10k; footprint SOT363 -> R0603; symbol traction-r1:74LVC1G11GW-Q100 -> traction-r1:R; LCSC C548242 -> CLASS; MPN 74LVC1G11GW-Q100 -> R0603-10k
- RIGNS1: renamed from ULAT2; value 74LVC1G74DC-Q100 -> 47k; footprint VSSOP8 -> R0603; symbol traction-r1:74LVC1G74DC-Q100 -> traction-r1:R; MPN 74LVC1G74DC-Q100 -> R0603-CLASS
- RIGNS2: renamed from USCH; value 74LVC3G17DC-Q100 -> 10k; footprint VSSOP8 -> R0603; symbol traction-r1:74LVC3G17DC-Q100 -> traction-r1:R; MPN 74LVC3G17DC-Q100 -> R0603-CLASS
- RILK1: renamed from UVMB1; value OPA348AQDBVRQ1 -> 10k; footprint SOT23-5 -> R0603; symbol traction-r1:OPA348AQDBVRQ1 -> traction-r1:R; LCSC C2877787 -> CLASS; MPN OPA348AQDBVRQ1 -> R0603-10k
- RILK2: renamed from UVMB2; value OPA348AQDBVRQ1 -> 10k; footprint SOT23-5 -> R0603; symbol traction-r1:OPA348AQDBVRQ1 -> traction-r1:R; LCSC C2877787 -> CLASS; MPN OPA348AQDBVRQ1 -> R0603-10k
- RILK3: renamed from CVM1; value 220nF -> 10k; footprint C0603 -> R0603; symbol traction-r1:C -> traction-r1:R; MPN MLCC-CLASS -> R0603-10k
- RILK4: renamed from CVM2; value 220nF -> 10k; footprint C0603 -> R0603; symbol traction-r1:C -> traction-r1:R; MPN MLCC-CLASS -> R0603-10k
- RLAT1: renamed from COR1; value 100nF -> 10k; footprint C0603 -> R0603; symbol traction-r1:C -> traction-r1:R; MPN MLCC-CLASS -> R0603-10k
- RLAT2: renamed from RRDYP2; value 5.1k -> 10k; MPN R0603-5k1 -> R0603-10k
- RLDE1: renamed from CSIND; value 47pF -> 38.3k; footprint C0603 -> R0603; symbol traction-r1:C -> traction-r1:R; MPN MLCC-CLASS -> R0603-CLASS
- RLDE2: renamed from CSINF1; value 22pF -> 10k; footprint C0603 -> R0603; symbol traction-r1:C -> traction-r1:R; MPN MLCC-CLASS -> R0603-CLASS
- RLVSD: renamed from ZLVS; value BZT52-C15 -> 4.7k; footprint SOD123 -> R0603; symbol traction-r1:D -> traction-r1:R; MPN BZT52-C15 -> R0603-4k7
- RLVSG: renamed from QBAL; value SQ2310ES -> 10k; footprint SOT23 -> R0603; symbol traction-r1:SQ2310ES -> traction-r1:R; MPN SQ2310ES -> R0603-10k
- RLVSM: renamed from USBC; value FS2633D -> 1k; footprint HLQFP48 -> R0603; symbol traction-r1:FS2633D -> traction-r1:R; MPN FS2633D -> R0603-1k
- RMRST: renamed from CRST; value 100pF -> 10k; footprint C0603 -> R0603; symbol traction-r1:C -> traction-r1:R; MPN MLCC-100pF-16V -> R0603-10k
- RMT1P: renamed from CCAN1; value 1uF -> 10k; footprint C0603 -> R0603; symbol traction-r1:C -> traction-r1:R; MPN MLCC-1uF-25V -> R0603-CLASS
- RMT1S: renamed from CCT1; value 4.7nF -> 1k; footprint C0603 -> R0603; symbol traction-r1:C -> traction-r1:R; MPN MLCC-4.7nF-50V -> R0603-CLASS
- RMT2P: renamed from RCT1A; value 60.4R -> 10k; MPN R0603-60R4-1% -> R0603-CLASS
- RMT2S: renamed from RCT1B; value 60.4R -> 1k; MPN R0603-60R4-1% -> R0603-CLASS
- ROF1: renamed from RVD2B; value 10k -> 9.1k; MPN R0603-10k-0.1% -> R0603-CLASS
- ROF2: renamed from RVD2C; value 10k -> 1k; MPN R0603-10k-0.1% -> R0603-CLASS
- RQDM: renamed from RSCH; value 100k -> 10k; MPN R0603-100k -> R0603-10k
- RRDB: renamed from RV5GP; value 47k -> 100k; MPN R0603-47k -> R0603-100k
- RRDYP1: renamed from RV5GS; value 47k -> 5.1k; MPN R0603-47k -> R0603-5k1
- RRDYP2: renamed from UASCG; value 74LVC1G08GW-Q100 -> 5.1k; footprint SOT353 -> R0603; symbol traction-r1:74LVC1G08GW-Q100 -> traction-r1:R; MPN 74LVC1G08GW-Q100 -> R0603-5k1
- RSB1: renamed from CIGN; value 100nF -> 52.3k; footprint C0603 -> R0603; symbol traction-r1:C -> traction-r1:R; MPN MLCC-100nF-50V -> R0603-CLASS
- RSB2: renamed from CIGNS; value 100nF -> 10k; footprint C0603 -> R0603; symbol traction-r1:C -> traction-r1:R; MPN MLCC-CLASS -> R0603-CLASS
- RSB3: renamed from DIGN; value 1N4148WS -> 220R; footprint SOD323 -> R0603; symbol traction-r1:D -> traction-r1:R; LCSC C2128 -> CLASS; MPN 1N4148WS -> R0603-CLASS
- RSB4: renamed from RIGN1; MPN R0603-5k1 -> R0603-CLASS
- RSCH: renamed from ULAT; value 74LVC1G74DC-Q100 -> 100k; footprint VSSOP8 -> R0603; symbol traction-r1:74LVC1G74DC-Q100 -> traction-r1:R; MPN 74LVC1G74DC-Q100 -> R0603-100k
- RSDN: renamed from CSINF2; value 22pF -> 10k; footprint C0603 -> R0603; symbol traction-r1:C -> traction-r1:R; MPN MLCC-CLASS -> R0603-CLASS
- RSIN1: renamed from CCOSA3; value 22pF -> 12k; footprint C0603 -> R0603; symbol traction-r1:C -> traction-r1:R; MPN MLCC-CLASS -> R0603-CLASS
- RSIN2: renamed from CCOSD; value 47pF -> 12k; footprint C0603 -> R0603; symbol traction-r1:C -> traction-r1:R; MPN MLCC-CLASS -> R0603-CLASS
- RSINF1: renamed from CCOSF1; value 22pF -> 12k; footprint C0603 -> R0603; symbol traction-r1:C -> traction-r1:R; MPN MLCC-CLASS -> R0603-CLASS
- RSINF2: renamed from CCOSF2; value 22pF -> 12k; footprint C0603 -> R0603; symbol traction-r1:C -> traction-r1:R; MPN MLCC-CLASS -> R0603-CLASS
- RSINR1: renamed from RCOS1; value 12k -> 120R; MPN R0603-CLASS -> R0603-120R
- RSINR2: renamed from RCOS2; value 12k -> 120R; MPN R0603-CLASS -> R0603-120R
- RSNUP: renamed from RTHSP; value 10k -> 5.1k; MPN R0603-10k-1% -> R0603-5k1-1%
- RSNVP: renamed from UMT1; value OPA333AQDBVRQ1 -> 5.1k; footprint SOT23-5 -> R0603; symbol traction-r1:OPA333AQDBVRQ1 -> traction-r1:R; LCSC C2058544 -> CLASS; MPN OPA333AQDBVRQ1 -> R0603-5k1-1%
- RSNWP: renamed from UMT2; value OPA333AQDBVRQ1 -> 5.1k; footprint SOT23-5 -> R0603; symbol traction-r1:OPA333AQDBVRQ1 -> traction-r1:R; LCSC C2058544 -> CLASS; MPN OPA333AQDBVRQ1 -> R0603-5k1-1%
- RTAMB: renamed from FMT2; value FUSE-350mA-0603 -> 10k; footprint F0603 -> R0603; symbol traction-r1:F -> traction-r1:R; MPN FUSE-350mA-0603 -> NTC-10k-0603
- RTAMBP: renamed from RMT1P; MPN R0603-CLASS -> R0603-10k-1%
- RTHS: renamed from RMT1S; value 1k -> 10k; MPN R0603-CLASS -> NTC-10k-0603
- RTHSP: renamed from RMT2P; MPN R0603-CLASS -> R0603-10k-1%
- RTMR: renamed from CMT1F; value 47nF -> 0R; footprint C0603 -> R0603; symbol traction-r1:C -> traction-r1:R; MPN MLCC-47nF-25V -> R0603-CLASS
- RUB0: renamed from CVS2; value 4.7nF -> 100k; footprint C0603 -> R0603; symbol traction-r1:C -> traction-r1:R; MPN MLCC-4.7nF-50V -> R0603-100k
- RUB1: renamed from LVB; value FB-220R-1A -> 100R; footprint FB0805 -> R0603; symbol traction-r1:L -> traction-r1:R; MPN FB-220R-1A -> R0603-100R
- RUB2: renamed from RVB0; value 100k -> 100R; MPN R0603-100k -> R0603-100R
- RV5GP: renamed from CASCG; value 100nF -> 47k; footprint C0603 -> R0603; symbol traction-r1:C -> traction-r1:R; MPN MLCC-100nF-16V -> R0603-47k
- RV5GS: renamed from CLAT; value 100nF -> 47k; footprint C0603 -> R0603; symbol traction-r1:C -> traction-r1:R; MPN MLCC-100nF-16V -> R0603-47k
- RVB0: renamed from CWS2; value 4.7nF -> 100k; footprint C0603 -> R0603; symbol traction-r1:C -> traction-r1:R; MPN MLCC-4.7nF-50V -> R0603-100k
- RVB1: renamed from LWB; value FB-220R-1A -> 100R; footprint FB0805 -> R0603; symbol traction-r1:L -> traction-r1:R; MPN FB-220R-1A -> R0603-100R
- RVB2: renamed from RWB0; value 100k -> 100R; MPN R0603-100k -> R0603-100R
- RVD1B: renamed from CSNUF; value 47nF -> 10k; footprint C0603 -> R0603; symbol traction-r1:C -> traction-r1:R; MPN MLCC-47nF-25V -> R0603-10k-0.1%
- RVD1C: renamed from CSNVF; value 47nF -> 10k; footprint C0603 -> R0603; symbol traction-r1:C -> traction-r1:R; MPN MLCC-47nF-25V -> R0603-10k-0.1%
- RVD1D: renamed from CSNWF; value 47nF -> 10k; footprint C0603 -> R0603; symbol traction-r1:C -> traction-r1:R; MPN MLCC-47nF-25V -> R0603-10k-0.1%
- RVD2A: renamed from RSNWP; value 5.1k -> 10k; MPN R0603-5k1-1% -> R0603-10k-0.1%
- RVD2B: renamed from RTMR; value 0R -> 10k; MPN R0603-CLASS -> R0603-10k-0.1%
- RVD2C: renamed from CTAMBF; value 47nF -> 10k; footprint C0603 -> R0603; symbol traction-r1:C -> traction-r1:R; MPN MLCC-47nF-25V -> R0603-10k-0.1%
- RVD2D: renamed from CTHSF; value 47nF -> 10k; footprint C0603 -> R0603; symbol traction-r1:C -> traction-r1:R; MPN MLCC-47nF-25V -> R0603-10k-0.1%
- RVM1: renamed from UEXD; value ALM2402QPWPRQ1 -> 24k; footprint HTSSOP14-PWP -> R0603; symbol traction-r1:ALM2402QPWPRQ1 -> traction-r1:R; LCSC C544754 -> CLASS; MPN ALM2402QPWPRQ1 -> R0603-24k-1%
- RVM2: renamed from UEXF; value OPA348AQDBVRQ1 -> 24k; footprint SOT23-5 -> R0603; symbol traction-r1:OPA348AQDBVRQ1 -> traction-r1:R; LCSC C2877787 -> CLASS; MPN OPA348AQDBVRQ1 -> R0603-24k-1%
- RVM3: renamed from ULDOEX; value NCV4276CDTADJRKG -> 24k; footprint DPAK5 -> R0603; symbol traction-r1:NCV4276CDTADJRKG -> traction-r1:R; MPN NCV4276CDTADJRKG -> R0603-24k-1%
- RVM4: renamed from CEXA1; value 220pF -> 24k; footprint C0603 -> R0603; symbol traction-r1:C -> traction-r1:R; MPN MLCC-CLASS -> R0603-24k-1%
- RWB0: renamed from ROF2; value 1k -> 100k; MPN R0603-CLASS -> R0603-100k
- RWB1: renamed from RVD1A; value 10k -> 100R; MPN R0603-10k-0.1% -> R0603-100R
- RWB2: renamed from RVD1B; value 10k -> 100R; MPN R0603-10k-0.1% -> R0603-100R
- RWB3: renamed from RVD1C; value 10k -> 100R; MPN R0603-10k-0.1% -> R0603-100R
- TVSC1: renamed from CCAN2; value 1uF -> PESD2IVN24-T; footprint C0603 -> SOT23; symbol traction-r1:C -> traction-r1:PESD2IVN24-T; LCSC CLASS -> C406047; MPN MLCC-1uF-25V -> PESD2IVN24-T
- TVSC2: renamed from LVS2; value FB-470R -> PESD2IVN24-T; footprint FB0603 -> SOT23; symbol traction-r1:L -> traction-r1:PESD2IVN24-T; LCSC CLASS -> C406047; MPN FB-470R-CLASS -> PESD2IVN24-T
- TVSEN: renamed from RSIN1; value 12k -> SMCJ8.5CA; footprint R0603 -> SMC; symbol traction-r1:R -> traction-r1:D_21; MPN R0603-CLASS -> SMCJ8.5CA
- TVSEP: renamed from RSIN2; value 12k -> SMCJ8.5CA; footprint R0603 -> SMC; symbol traction-r1:R -> traction-r1:D_21; MPN R0603-CLASS -> SMCJ8.5CA
- TVSM1: renamed from LCAN2; value ACT45B-101-2P-TL003 -> SMAJ5.0A; footprint CMC1210 -> SMA; symbol traction-r1:ACT45B-101-2P-TL003 -> traction-r1:D_21; MPN ACT45B-101-2P-TL003 -> SMAJ5.0A
- TVSM2: renamed from TVSC2; value PESD2IVN24-T -> SMAJ5.0A; footprint SOT23 -> SMA; symbol traction-r1:PESD2IVN24-T -> traction-r1:D_21; LCSC C406047 -> CLASS; MPN PESD2IVN24-T -> SMAJ5.0A
- UAND1: renamed from USCH2; value 74LVC3G17DC-Q100 -> 74LVC1G11GW-Q100; footprint VSSOP8 -> SOT363; symbol traction-r1:74LVC3G17DC-Q100 -> traction-r1:74LVC1G11GW-Q100; LCSC CLASS -> C548242; MPN 74LVC3G17DC-Q100 -> 74LVC1G11GW-Q100
- UAND2: renamed from USCH3; value 74LVC3G17DC-Q100 -> 74LVC1G11GW-Q100; footprint VSSOP8 -> SOT363; symbol traction-r1:74LVC3G17DC-Q100 -> traction-r1:74LVC1G11GW-Q100; LCSC CLASS -> C548242; MPN 74LVC3G17DC-Q100 -> 74LVC1G11GW-Q100
- UASCG: renamed from DFO; value BAT46ZFILM -> 74LVC1G08GW-Q100; footprint SOD123 -> SOT353; symbol traction-r1:D -> traction-r1:74LVC1G08GW-Q100; LCSC C283255 -> CLASS; MPN BAT46ZFILM -> 74LVC1G08GW-Q100
- UCAN1: renamed from CCT2; value 4.7nF -> TCAN1042HGVDRQ1; footprint C0603 -> SOIC8; symbol traction-r1:C -> traction-r1:TCAN1042HGVDRQ1; LCSC CLASS -> C132550; MPN MLCC-4.7nF-50V -> TCAN1042HGVDRQ1
- UCAN2: renamed from LVS3; value FB-470R -> TCAN1042HGVDRQ1; footprint FB0603 -> SOIC8; symbol traction-r1:L -> traction-r1:TCAN1042HGVDRQ1; LCSC CLASS -> C132550; MPN FB-470R-CLASS -> TCAN1042HGVDRQ1
- UEXD: renamed from CEXA2; value 1.5nF -> ALM2402QPWPRQ1; footprint C0603 -> HTSSOP14-PWP; symbol traction-r1:C -> traction-r1:ALM2402QPWPRQ1; LCSC CLASS -> C544754; MPN MLCC-CLASS -> ALM2402QPWPRQ1
- UEXF: renamed from CEXA3; value 100nF -> OPA348AQDBVRQ1; footprint C0603 -> SOT23-5; symbol traction-r1:C -> traction-r1:OPA348AQDBVRQ1; LCSC CLASS -> C2877787; MPN MLCC-CLASS -> OPA348AQDBVRQ1
- ULAT: renamed from RARB; value 10k -> 74LVC1G74DC-Q100; footprint R0603 -> VSSOP8; symbol traction-r1:R -> traction-r1:74LVC1G74DC-Q100; MPN R0603-10k -> 74LVC1G74DC-Q100
- ULAT2: renamed from CAND1; value 100nF -> 74LVC1G74DC-Q100; footprint C0603 -> VSSOP8; symbol traction-r1:C -> traction-r1:74LVC1G74DC-Q100; MPN MLCC-CLASS -> 74LVC1G74DC-Q100
- ULDOEX: renamed from CEXA4; value 47pF -> NCV4276CDTADJRKG; footprint C0603 -> DPAK5; symbol traction-r1:C -> traction-r1:NCV4276CDTADJRKG; MPN MLCC-CLASS -> NCV4276CDTADJRKG
- UMCU: renamed from CMA2; value 100nF -> S32K396EHT1MJBST; footprint C0603 -> MAPBGA289; symbol traction-r1:C -> traction-r1:S32K396EHT1MJBST; MPN MLCC-100nF-16V -> S32K396EHT1MJBST
- UMT1: renamed from RMT2S; value 1k -> OPA333AQDBVRQ1; footprint R0603 -> SOT23-5; symbol traction-r1:R -> traction-r1:OPA333AQDBVRQ1; LCSC CLASS -> C2058544; MPN R0603-CLASS -> OPA333AQDBVRQ1
- UMT2: renamed from TVSM1; value PESD5V0L1BA -> OPA333AQDBVRQ1; footprint SOD323 -> SOT23-5; symbol traction-r1:R -> traction-r1:OPA333AQDBVRQ1; LCSC CLASS -> C2058544; MPN PESD5V0L1BA -> OPA333AQDBVRQ1
- UOR1: renamed from CILK; value 2.2nF -> 74LVC1G32GW-Q100; footprint C0603 -> SOT353; symbol traction-r1:C -> traction-r1:74LVC1G32GW-Q100; LCSC CLASS -> C548334; MPN MLCC-2.2nF-50V -> 74LVC1G32GW-Q100
- UOR2: renamed from RILK1; value 10k -> 74LVC1G32GW-Q100; footprint R0603 -> SOT353; symbol traction-r1:R -> traction-r1:74LVC1G32GW-Q100; LCSC CLASS -> C548334; MPN R0603-10k -> 74LVC1G32GW-Q100
- USBC: renamed from CSB1; value 22uF -> FS2633D; footprint C0805 -> HLQFP48; symbol traction-r1:C -> traction-r1:FS2633D; MPN MLCC-CLASS -> FS2633D
- USCH: renamed from CAND2; value 100nF -> 74LVC3G17DC-Q100; footprint C0603 -> VSSOP8; symbol traction-r1:C -> traction-r1:74LVC3G17DC-Q100; MPN MLCC-CLASS -> 74LVC3G17DC-Q100
- USCH2: renamed from CCLR; value 15nF -> 74LVC3G17DC-Q100; footprint C0603 -> VSSOP8; symbol traction-r1:C -> traction-r1:74LVC3G17DC-Q100; MPN MLCC-15nF-50V-C0G -> 74LVC3G17DC-Q100
- USCH3: renamed from CFLTD; value 3.3nF -> 74LVC3G17DC-Q100; footprint C0603 -> VSSOP8; symbol traction-r1:C -> traction-r1:74LVC3G17DC-Q100; MPN MLCC-3.3nF-50V-C0G -> 74LVC3G17DC-Q100
- USNSU: renamed from LUB; value FB-220R-1A -> HC5FW900-S; footprint FB0805 -> OffBoard; symbol traction-r1:L -> traction-r1:HC5FW900-S; MPN FB-220R-1A -> HC5FW900-S
- USNSV: renamed from RUB0; value 100k -> HC5FW900-S; footprint R0603 -> OffBoard; symbol traction-r1:R -> traction-r1:HC5FW900-S; MPN R0603-100k -> HC5FW900-S
- USNSW: renamed from RUB1; value 100R -> HC5FW900-S; footprint R0603 -> OffBoard; symbol traction-r1:R -> traction-r1:HC5FW900-S; MPN R0603-100R -> HC5FW900-S
- UUB1: renamed from RUB2; value 100R -> OPA376AQDBVRQ1; footprint R0603 -> SOT23-5; symbol traction-r1:R -> traction-r1:OPA376AQDBVRQ1; MPN R0603-100R -> OPA376AQDBVRQ1
- UUB2: renamed from RUB3; value 100R -> OPA376AQDBVRQ1; footprint R0603 -> SOT23-5; symbol traction-r1:R -> traction-r1:OPA376AQDBVRQ1; MPN R0603-100R -> OPA376AQDBVRQ1
- UVB1: renamed from RVB2; value 100R -> OPA376AQDBVRQ1; footprint R0603 -> SOT23-5; symbol traction-r1:R -> traction-r1:OPA376AQDBVRQ1; MPN R0603-100R -> OPA376AQDBVRQ1
- UVB2: renamed from RVB3; value 100R -> OPA376AQDBVRQ1; footprint R0603 -> SOT23-5; symbol traction-r1:R -> traction-r1:OPA376AQDBVRQ1; MPN R0603-100R -> OPA376AQDBVRQ1
- UVD1: renamed from RVD1D; value 10k -> OPA376AQDBVRQ1; footprint R0603 -> SOT23-5; symbol traction-r1:R -> traction-r1:OPA376AQDBVRQ1; MPN R0603-10k-0.1% -> OPA376AQDBVRQ1
- UVD2: renamed from RSNUP; value 5.1k -> OPA376AQDBVRQ1; footprint R0603 -> SOT23-5; symbol traction-r1:R -> traction-r1:OPA376AQDBVRQ1; MPN R0603-5k1-1% -> OPA376AQDBVRQ1
- UVMB1: renamed from RVM1; value 24k -> OPA348AQDBVRQ1; footprint R0603 -> SOT23-5; symbol traction-r1:R -> traction-r1:OPA348AQDBVRQ1; LCSC CLASS -> C2877787; MPN R0603-24k-1% -> OPA348AQDBVRQ1
- UVMB2: renamed from RVM2; value 24k -> OPA348AQDBVRQ1; footprint R0603 -> SOT23-5; symbol traction-r1:R -> traction-r1:OPA348AQDBVRQ1; LCSC CLASS -> C2877787; MPN R0603-24k-1% -> OPA348AQDBVRQ1
- UWB1: renamed from RWB2; value 100R -> OPA376AQDBVRQ1; footprint R0603 -> SOT23-5; symbol traction-r1:R -> traction-r1:OPA376AQDBVRQ1; MPN R0603-100R -> OPA376AQDBVRQ1
- UWB2: renamed from RWB3; value 100R -> OPA376AQDBVRQ1; footprint R0603 -> SOT23-5; symbol traction-r1:R -> traction-r1:OPA376AQDBVRQ1; MPN R0603-100R -> OPA376AQDBVRQ1
- Y1: renamed from RBOOT; value 10k -> CX3225GA40000D0PTVCC; footprint R0603 -> X3225; symbol traction-r1:R -> traction-r1:Y; LCSC CLASS -> C6009848; MPN R0603-10k -> CX3225GA40000D0PTVCC
- ZLVS: renamed from CBTC; value 47nF -> BZT52-C15; footprint C0603 -> SOD123; symbol traction-r1:C -> traction-r1:D; MPN MLCC-CLASS -> BZT52-C15
- ZSET: renamed from COR2; value 100nF -> BZT52-B5V6; footprint C0603 -> SOD123; symbol traction-r1:C -> traction-r1:D; MPN MLCC-CLASS -> BZT52-B5V6
- renumbered CMD11 to CMD1, CMD12 to CMD10, CMD2 to CMD11, CMD3 to CMD12, CMD4 to CMD2, CMD5 to CMD3, CMD6 to CMD4, CMD7 to CMD5, CMD8 to CMD6, CMD9 to CMD7, CSB8 to CSB4, CCOSA1 to CSINF1, CMT2F to CTAMBF, RFLTD to RDRB, RFLTP1 to RENP1, REXM4 to REXB1, RGPD to RFLTC, RLAT2 to RFLTD, RVB1 to RUB3, RWB1 to RVB3, RVD2D to RVD1A, UVD2 to UVOF
Connections:
- net labels added: V25, VREX_NC, VREX_PC
- wire segments 955 -> 969
Other:
- note added: "rev A.13 - 26 sections - 295 components"
- note removed: "rev A.12 - 26 sections - 288 components"
- moved on the sheet: CAND1, CAND2, CBAL, CBTC, CBTP, CCAN2, CCLR, CEXA1, CEXA2, CEXA3, CFLTD, CFLTF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
