File: kicad5/traction/traction-power.sch (KiCad schematic (older format))
At the start: 309 parts

Commit message: Rev A.3: end-to-end verification campaign — 18 defects found & fixed, datasheet pack
Three independent verification layers, all green at datasheet-real constants:
- geometric pin-verify 1540/1540 (100%)
- structural ERC audit (new erc-audit.mjs): 664 intent-level checks, 0 fail
- numeric worst-case verification (new design-verify.mjs): 51 PASS / 3 WARN /
  0 FAIL at real corners (Vbus->850V, KL30 9-16V, R+/-5%, C+10%)

Findings fixed (docs/verification-report.md, F1-F36): flyback CS scaling, FB
reference mis-scaled for controller swap (supply could never start), missing
VCC start path, five net-alias floating pins, Y-cap class at 850V, common-cause
VDC sense bias, load-dump cap ratings, discharge worst-case corner (470R),
OV-witness headroom (6.2k), ASC abs-max violation (5.1V clamp), real HCS600
pin map + HS DESAT to aux drain-sense, +15/-5.1 drive combo, UCC28C40 UVLO
grade for cold-crank, flyback re-derived for real VGT12EEM (10uH, 1:1.6:2.9,
250kHz, 11.8V NF regulation), FS26 VMONEXT 0.8V reference divider, FS0B/FS1B
pull-up current, S32K39 core ballast topology (V15S + SQ2310ES).

Datasheet pack: 36 verified PDFs in docs/datasheets/ + EXTRACTED-PARAMS.md.
Sheets/BOM/README regenerated at A.3 (529 components, Rs 69.8k @1k).

Co-Authored-By: Claude Fable 5 <noreply@anthropic.com>
Parts:
- added RPD9: 10k, R0603, symbol traction-r1:R
- C5B1: renamed from PS5B; value ISO5V-RFC-6K -> 1uF; footprint SIP7 -> C0603; symbol traction-r1:ISO5V-RFC-6K -> traction-r1:C; MPN ISO5V-RFC-6K -> MLCC-1uF-25V
- C5B2: renamed from C5B1; value 1uF -> 100nF
- C5C1: renamed from C5B2; value 100nF -> 1uF
- C5G1: renamed from C5G2; value 10uF -> 1uF
- C5G2: renamed from UB15; value TPS55340QRTERQ1 -> 10uF; footprint WQFN16 -> C1206; symbol traction-r1:TPS55340QRTERQ1 -> traction-r1:C; LCSC C2070860 -> CLASS; MPN TPS55340QRTERQ1 -> MLCC-10uF-25V
- CB15C: renamed from CB15I; value 10uF -> 10nF; footprint C1206 -> C0603; MPN MLCC-10uF-25V -> MLCC-CLASS
- CB15I: renamed from CB15O1; value 22uF -> 10uF; MPN MLCC-22uF-25V -> MLCC-10uF-50V
- CB15O2: renamed from DB15; value SS34 -> 22uF; footprint SMA -> C1210; symbol traction-r1:D -> traction-r1:C; MPN SS34 -> MLCC-22uF-25V
- CFHCT: value 3.3nF -> 680pF
- CFLA: renamed from UFL; value UCC28C43DR -> 4.7uF; footprint SOP8 -> C1206; symbol traction-r1:UCC28C43DR -> traction-r1:C; LCSC C111694 -> CLASS; MPN UCC28C43DR -> MLCC-4.7uF-50V
- CFLCF: renamed from CFLA; value 4.7uF -> 47pF; footprint C1206 -> C0603; MPN MLCC-4.7uF-50V -> MLCC-CLASS
- CFLCO: renamed from CFLCF; value 47pF -> 22nF
- CFLCT: renamed from CFLCO; value 22nF -> 680pF
- CFLSI: renamed from CFLCT; value 3.3nF -> 100pF
- CFLSN: renamed from CFLSI; footprint C0603 -> C1206; MPN MLCC-CLASS -> MLCC-100pF-500V
- CFLVR: renamed from CFLSN; value 100pF -> 100nF; footprint C1206 -> C0603; MPN MLCC-100pF-500V -> MLCC-CLASS
- CLVH1: renamed from CLVH2; MPN MLCC-4.7uF-25V -> MLCC-4.7uF-50V
- CLVH2: renamed from DRH; value NRVBAF360T3G -> 4.7uF; footprint SMA-flat -> C1206; symbol traction-r1:D -> traction-r1:C; MPN NRVBAF360T3G -> MLCC-4.7uF-50V
- CLVL1: renamed from CLVL2; MPN MLCC-4.7uF-25V -> MLCC-4.7uF-50V
- CLVL2: renamed from DRL; value NRVBAF360T3G -> 4.7uF; footprint SMA-flat -> C1206; symbol traction-r1:D -> traction-r1:C; MPN NRVBAF360T3G -> MLCC-4.7uF-50V
- CVBDF: renamed from RVDDL; value 6.65k -> 1nF; footprint R0603 -> C0603; symbol traction-r1:R -> traction-r1:C; MPN R0603-6k65-0.1% -> MLCC-1nF-50V
- CVDDF: renamed from ZFLG; value BZT52-C5V6 -> 1nF; footprint SOD123 -> C0603; symbol traction-r1:D -> traction-r1:C; MPN BZT52-C5V6 -> MLCC-1nF-50V
- CY1, CY2: MPN Y2-4.7nF-CD -> Y1-4.7nF-500VAC
- DB15: renamed from LB15; value IND-10uH-3A -> SS34; footprint IND6x6 -> SMA; symbol traction-r1:L -> traction-r1:D; MPN IND-10uH-3A -> SS34
- DFLA: renamed from CFLVR; value 100nF -> US1M; footprint C0603 -> SMA; symbol traction-r1:C -> traction-r1:D; LCSC CLASS -> C412437; MPN MLCC-CLASS -> US1M
- DFLG: renamed from DFLA; value US1M -> PMEG4010EH; footprint SMA -> SOD123; LCSC C412437 -> C282566; MPN US1M -> PMEG4010EH
- DFLSN: renamed from DFLG; value PMEG4010EH -> SMBJ85A; footprint SOD123 -> SMB; LCSC C282566 -> CLASS; MPN PMEG4010EH -> SMBJ85A
- DRH: renamed from DTVH; value TPSMC24CA -> NRVBAF360T3G; footprint SMC -> SMA-flat; LCSC C1975284 -> CLASS; MPN TPSMC24CA -> NRVBAF360T3G
- DRL: renamed from DTVL; value TPSMC24CA -> NRVBAF360T3G; footprint SMC -> SMA-flat; LCSC C1975284 -> CLASS; MPN TPSMC24CA -> NRVBAF360T3G
- DTVH: renamed from FH1; value MF-LSMF300/24X-2 -> TPSMC24CA; footprint PTC2920 -> SMC; symbol traction-r1:F -> traction-r1:D; LCSC C719172 -> C1975284; MPN MF-LSMF300/24X-2 -> TPSMC24CA
- DTVL: renamed from FL1; value MF-LSMF300/24X-2 -> TPSMC24CA; footprint PTC2920 -> SMC; symbol traction-r1:F -> traction-r1:D; LCSC C719172 -> C1975284; MPN MF-LSMF300/24X-2 -> TPSMC24CA
- FH1: renamed from LFH1; value FB-120R-3A -> MF-LSMF300/24X-2; footprint FB1206 -> PTC2920; symbol traction-r1:L -> traction-r1:F; LCSC CLASS -> C719172; MPN FB-120R-3A -> MF-LSMF300/24X-2
- FL1: renamed from LFL1; value FB-120R-3A -> MF-LSMF300/24X-2; footprint FB1206 -> PTC2920; symbol traction-r1:L -> traction-r1:F; LCSC CLASS -> C719172; MPN FB-120R-3A -> MF-LSMF300/24X-2
- JIC: renamed from RPD0; value 10k -> MICROFIT3-40; footprint R0603 -> MicroFit40; symbol traction-r1:R -> traction-r1:MICROFIT3-40; MPN R0603-10k -> MICROFIT3-40
- LB15: renamed from RB15F1; value 110k -> IND-10uH-3A; footprint R0603 -> IND6x6; symbol traction-r1:R -> traction-r1:L; MPN R0603-1% -> IND-10uH-3A
- LFH1: renamed from CLVL1; value 4.7uF -> FB-120R-3A; footprint C1206 -> FB1206; symbol traction-r1:C -> traction-r1:L; MPN MLCC-4.7uF-25V -> FB-120R-3A
- LFL1: renamed from UGDL; value NCV4276CDT50RKG -> FB-120R-3A; footprint DPAK -> FB1206; symbol traction-r1:NCV4276CDT50RKG -> traction-r1:L; MPN NCV4276CDT50RKG -> FB-120R-3A
- PS5B: renamed from RVBD6; value 470k -> ISO5V-RFC-6K; footprint R1206 -> SIP7; symbol traction-r1:R -> traction-r1:ISO5V-RFC-6K; MPN R1206-470k-TF -> ISO5V-RFC-6K
- PS5C: renamed from RVBDL; value 6.65k -> ISO5V-RFC-6K; footprint R0603 -> SIP7; symbol traction-r1:R -> traction-r1:ISO5V-RFC-6K; MPN R0603-6k65-0.1% -> ISO5V-RFC-6K
- QFL: renamed from ZFHG; value BZT52-C5V6 -> BUK9Y14-80E; footprint SOD123 -> LFPAK56; symbol traction-r1:D -> traction-r1:BUK9Y14-80E; LCSC CLASS -> C86732; MPN BZT52-C5V6 -> BUK9Y14-80E
- QFLE1: renamed from QFL; value BUK9Y14-80E -> 2N7002; footprint LFPAK56 -> SOT23; symbol traction-r1:BUK9Y14-80E -> traction-r1:2N7002; LCSC C86732 -> C8545; MPN BUK9Y14-80E -> 2N7002
- RASCG: value 100R -> 2.2k; MPN R0603-100R -> R0603-2k2
- RB15F1: renamed from RB15F2; value 9.53k -> 110k
- RB15F2: renamed from JIC; value MICROFIT3-40 -> 9.53k; footprint MicroFit40 -> R0603; symbol traction-r1:MICROFIT3-40 -> traction-r1:R; MPN MICROFIT3-40 -> R0603-1%
- RDIS1, RDIS2, RDIS3, RDIS4: value 560R -> 470R; MPN WW-560R-10W-AX -> WW-470R-10W-AX
- RFHCS: value 33m -> 330m; footprint R1206 -> R1210; MPN R1206-0R1-3x -> R1210-0R33-0.75W
- RFHFB1: value 18k -> 56k
- RFHG: renamed from RFHFB3; value 1.3k -> 10R; MPN R0603-1% -> R0603-CLASS
- RFHGO: renamed from RFHG; value 10R -> 20R
- RFHGS: renamed from RFHGO; value 20R -> 51k
- RFHRT: renamed from RFHGS; value 51k -> 10k
- RFHSI: renamed from RFHRT; value 10k -> 100R
- RFHSN: renamed from RFHSI; footprint R0603 -> R0805; MPN R0603-CLASS -> R0805-100R
- RFHST: renamed from RFHSN; value 100R -> 4.7k; footprint R0805 -> R0603; MPN R0805-100R -> R0603-CLASS
- RFLCS: renamed from DFLSN; value SMBJ85A -> 330m; footprint SMB -> R1210; symbol traction-r1:D -> traction-r1:R; MPN SMBJ85A -> R1210-0R33-0.75W
- RFLEN: renamed from RFLCS; value 33m -> 100k; footprint R1206 -> R0603; MPN R1206-0R1-3x -> R0603-CLASS
- RFLFB1: renamed from RFLEN; value 100k -> 56k; MPN R0603-CLASS -> R0603-1%
- RFLFB2: renamed from RFLFB1; value 18k -> 15k
- RFLG: renamed from RFLFB2; value 15k -> 10R; MPN R0603-1% -> R0603-CLASS
- RFLGO: renamed from RFLFB3; value 1.3k -> 20R; MPN R0603-1% -> R0603-CLASS
- RFLGS: renamed from RFLG; value 10R -> 51k
- RFLRT: renamed from RFLGO; value 20R -> 10k
- RFLSI: renamed from RFLGS; value 51k -> 100R
- RFLSN: renamed from RFLRT; value 10k -> 100R; footprint R0603 -> R0805; MPN R0603-CLASS -> R0805-100R
- RFLST: renamed from RFLSI; value 100R -> 4.7k
- RVBD1: renamed from UIVB; value AMC1311BDWVR -> 470k; footprint SOIC8W -> R1206; symbol traction-r1:AMC1311BDWVR -> traction-r1:R; LCSC C456277 -> CLASS; MPN AMC1311BDWVR -> R1206-470k-TF
- RVBD2: renamed from CVBDF; value 1nF -> 470k; footprint C0603 -> R1206; symbol traction-r1:C -> traction-r1:R; MPN MLCC-1nF-50V -> R1206-470k-TF
- RVBDL: renamed from RVBD5; value 470k -> 6.2k; footprint R1206 -> R0603; MPN R1206-470k-TF -> R0603-6k2-0.1%
- RVDD1: renamed from UIVDC; value AMC1311BDWVR -> 470k; footprint SOIC8W -> R1206; symbol traction-r1:AMC1311BDWVR -> traction-r1:R; LCSC C456277 -> CLASS; MPN AMC1311BDWVR -> R1206-470k-TF
- RVDD2: renamed from CVDDF; value 1nF -> 470k; footprint C0603 -> R1206; symbol traction-r1:C -> traction-r1:R; MPN MLCC-1nF-50V -> R1206-470k-TF
- RVDDL: renamed from RVDD5; value 470k -> 6.2k; footprint R1206 -> R0603; MPN R1206-470k-TF -> R0603-6k2-0.1%
- TFL1: renamed from QFLE2; value 2N7002 -> VGT12EEM-200S1A4; footprint SOT23 -> XfmrEE12; symbol traction-r1:2N7002 -> traction-r1:VGT12EEM-200S1A4; LCSC C8545 -> CLASS; MPN 2N7002 -> VGT12EEM-200S1A4
- UB15: renamed from CB15C; value 10nF -> TPS55340QRTERQ1; footprint C0603 -> WQFN16; symbol traction-r1:C -> traction-r1:TPS55340QRTERQ1; LCSC CLASS -> C2070860; MPN MLCC-CLASS -> TPS55340QRTERQ1
- UFH: value UCC28C43DR -> UCC28C40DR; symbol traction-r1:UCC28C43DR -> traction-r1:UCC28C40DR; LCSC C111694 -> CLASS; MPN UCC28C43DR -> UCC28C40DR
- UFL: renamed from TFL3; value VGT12EEM-200S1A4 -> UCC28C40DR; footprint XfmrEE12 -> SOP8; symbol traction-r1:VGT12EEM-200S1A4 -> traction-r1:UCC28C40DR; MPN VGT12EEM-200S1A4 -> UCC28C40DR
- UGDL: renamed from C5G1; value 1uF -> NCV4276CDT50RKG; footprint C1206 -> DPAK; symbol traction-r1:C -> traction-r1:NCV4276CDT50RKG; MPN MLCC-10uF-25V -> NCV4276CDT50RKG
- UIVB: renamed from RVDD6; value 470k -> AMC1311BDWVR; footprint R1206 -> SOIC8W; symbol traction-r1:R -> traction-r1:AMC1311BDWVR; LCSC CLASS -> C456277; MPN R1206-470k-TF -> AMC1311BDWVR
- UIVDC: renamed from RFLST; value 4.7k -> AMC1311BDWVR; footprint R0603 -> SOIC8W; symbol traction-r1:R -> traction-r1:AMC1311BDWVR; LCSC CLASS -> C456277; MPN R0603-CLASS -> AMC1311BDWVR
- ZASC: renamed from CLVH1; value 4.7uF -> BZT52-C5V1; footprint C1206 -> SOD123; symbol traction-r1:C -> traction-r1:D; MPN MLCC-4.7uF-25V -> BZT52-C5V1
- ZFHG: renamed from RFHST; value 4.7k -> BZT52-C5V6; footprint R0603 -> SOD123; symbol traction-r1:R -> traction-r1:D; MPN R0603-CLASS -> BZT52-C5V6
- ZFLG: renamed from RFLSN; value 100R -> BZT52-C5V6; footprint R0805 -> SOD123; symbol traction-r1:R -> traction-r1:D; MPN R0805-100R -> BZT52-C5V6
- ZUHV, ZULV, ZVHV, ZVLV, ZWHV, ZWLV: value BZT52-C4V3 -> BZT52-C5V1; MPN BZT52-C4V3 -> BZT52-C5V1
- renumbered CB15O2 to CB15O1, QFLE1 to QFLE2, RPD1 to RPD0, RPD10 to RPD1, RPD2 to RPD10, RPD3 to RPD2, RPD4 to RPD3, RPD5 to RPD4, RPD6 to RPD5, RPD7 to RPD6, RPD8 to RPD7, RPD9 to RPD8, RVBD1 to RVBD3, RVBD2 to RVBD4, RVBD3 to RVBD5, RVBD4 to RVBD6, RVDD1 to RVDD3, RVDD2 to RVDD4, RVDD3 to RVDD5, RVDD4 to RVDD6, TFL1 to TFL2, TFL2 to TFL3
Connections:
- net labels added: DSH_U, DSH_V, DSH_W, V5ISO2
- net labels removed: FFB2_H, FFB2_L, NT_UB, NT_VB, NT_WB, W_UH_B, W_UL_B, W_VH_B, W_VL_B, W_WH_B, W_WL_B
- wire segments 829 -> 839
Other:
- note added: "ACTIVE QDIS + 4x 470R 10W = 1.88k: 1.6 s to 60 V"
- note added: "E = 116 J @850 V - 32 J/res worst (>=100 J rated)"
- note added: "rev A.3 - 26 sections - 310 components"
- note removed: "ACTIVE QDIS + 4x 560R 10W = 2.24k: 1.9 s to 60 V"
- note removed: "E = 116 J @850 V - 29 J/res pulse (>=100 J rated)"
- note removed: "rev A.2 - 26 sections - 309 components"
- moved on the sheet: C5B2, C5C1, C5G1, CASC, CB15C, CB15I, CB15O1, CDC1, CDC10, CDC11, CDC12, CDC13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

Commit message: Split discharge onto a bolt-on board (XM3 pattern), 3-sheet set
- boards/discharge.tsx: bleeder (2x5x27k) + active discharge (4x470R +
  HCM75S12T4K3, TLP152/QA01C default-OFF) on its own PCB across the cap
  bank; power board keeps JDIS header (V15/QDIS_CMD/2xGND) + CMD pulldown
- pipeline: disch side threaded through pages/gen/verify/print/pdf/bom;
  sheet idents 1..3 of 3; disch title block carries "NEVER energize
  without this board fitted"; root sheet de-branded (X-IN-One -> Traction)
- gates green: 1550/1550 pins, ERC 672/0, design-verify 51P/3W/0F
- docs: README + design-basis + bom synced to 3-board state; new
  docs/img/sheet-disch.png; BOM ₹69,856 @1k (63,375/672/5,808)

Co-Authored-By: Claude Fable 5 <noreply@anthropic.com>
Parts:
- removed CB15C: 10nF, C0603, symbol traction-r1:C
- removed CB15I: 10uF, C1210, symbol traction-r1:C
- removed CB15O1, CB15O2: 22uF, C1210, symbol traction-r1:C
- removed DB15: SS34, SMA, symbol traction-r1:D
- removed JIC: MICROFIT3-40, MicroFit40, symbol traction-r1:MICROFIT3-40
- removed LB15: IND-10uH-3A, IND6x6, symbol traction-r1:L
- removed RB15F1: 110k, R0603, symbol traction-r1:R
- removed RB15F2: 9.53k, R0603, symbol traction-r1:R
- removed RPD0, RPD1, RPD10, RPD2, RPD3, RPD4, RPD5, RPD6, RPD7, RPD8, RPD9: 10k, R0603, symbol traction-r1:R
- C5B1: renamed from UIVDC; value AMC1311BDWVR -> 1uF; footprint SOIC8W -> C0603; symbol traction-r1:AMC1311BDWVR -> traction-r1:C; LCSC C456277 -> CLASS; MPN AMC1311BDWVR -> MLCC-1uF-25V
- C5B2: renamed from CVDDF; value 1nF -> 100nF; MPN MLCC-1nF-50V -> MLCC-1uF-25V
- C5C1: renamed from RVDD1; value 470k -> 1uF; footprint R1206 -> C0603; symbol traction-r1:R -> traction-r1:C; MPN R1206-470k-TF -> MLCC-1uF-25V
- C5G1: renamed from PSASC; value QA01C-18 -> 1uF; footprint SIP7 -> C1206; symbol traction-r1:QA01C-18 -> traction-r1:C; MPN QA01C-18 -> MLCC-10uF-25V
- C5G2: renamed from UASC; value TLP152 -> 10uF; footprint SO6 -> C1206; symbol traction-r1:TLP152 -> traction-r1:C; LCSC C17255258 -> CLASS; MPN TLP152 -> MLCC-10uF-25V
- CASC: renamed from RVDD4; value 470k -> 100nF; footprint R1206 -> C0603; symbol traction-r1:R -> traction-r1:C; MPN R1206-470k-TF -> MLCC-100nF-25V
- CB15C: renamed from RASCG; value 2.2k -> 10nF; footprint R0603 -> C0603; symbol traction-r1:R -> traction-r1:C; MPN R0603-2k2 -> MLCC-CLASS
- CB15I: renamed from RASCL; value 470R -> 10uF; footprint R0603 -> C1210; symbol traction-r1:R -> traction-r1:C; MPN R0603-470R -> MLCC-10uF-50V
- CB15O1: renamed from RASCPD; value 10k -> 22uF; footprint R0603 -> C1210; symbol traction-r1:R -> traction-r1:C; MPN R0603-10k -> MLCC-22uF-25V
- CB15O2: renamed from ZASC; value BZT52-C5V1 -> 22uF; footprint SOD123 -> C1210; symbol traction-r1:D -> traction-r1:C; MPN BZT52-C5V1 -> MLCC-22uF-25V
- CFHA: renamed from DWLR; value US1M -> 4.7uF; footprint SMA -> C1206; symbol traction-r1:D -> traction-r1:C; LCSC C412437 -> CLASS; MPN US1M -> MLCC-4.7uF-50V
- CFHCF: renamed from DWLS1; value US1M -> 47pF; footprint SMA -> C0603; symbol traction-r1:D -> traction-r1:C; LCSC C412437 -> CLASS; MPN US1M -> MLCC-CLASS
- CFHCO: renamed from DWLS2; value US1M -> 22nF; footprint SMA -> C0603; symbol traction-r1:D -> traction-r1:C; LCSC C412437 -> CLASS; MPN US1M -> MLCC-CLASS
- CFHCT: renamed from DWLZ1; value BZT52-C18 -> 680pF; footprint SOD123 -> C0603; symbol traction-r1:D -> traction-r1:C; MPN BZT52-C18 -> MLCC-CLASS
- CFHSI: renamed from DWLZ2; value BZT52-C5V1 -> 100pF; footprint SOD123 -> C0603; symbol traction-r1:D -> traction-r1:C; MPN BZT52-C5V1 -> MLCC-CLASS
- CFHSN: renamed from RWLBL; value 5.1k -> 100pF; footprint R0805 -> C1206; symbol traction-r1:R -> traction-r1:C; MPN R0805-4k99 -> MLCC-100pF-500V
- CFHVR: renamed from RWLDS; value 100R -> 100nF; footprint R0805 -> C0603; symbol traction-r1:R -> traction-r1:C; MPN R0805-100R -> MLCC-CLASS
- CFLA: renamed from DFHSN; value SMBJ85A -> 4.7uF; footprint SMB -> C1206; symbol traction-r1:D -> traction-r1:C; MPN SMBJ85A -> MLCC-4.7uF-50V
- CFLCF: renamed from RFHCS; value 330m -> 47pF; footprint R1210 -> C0603; symbol traction-r1:R -> traction-r1:C; MPN R1210-0R33-0.75W -> MLCC-CLASS
- CFLCO: renamed from RFHEN; value 100k -> 22nF; footprint R0603 -> C0603; symbol traction-r1:R -> traction-r1:C; MPN R0603-CLASS -> MLCC-CLASS
- CFLCT: renamed from RFHFB1; value 56k -> 680pF; footprint R0603 -> C0603; symbol traction-r1:R -> traction-r1:C; MPN R0603-1% -> MLCC-CLASS
- CFLSI: renamed from RFHFB2; value 15k -> 100pF; footprint R0603 -> C0603; symbol traction-r1:R -> traction-r1:C; MPN R0603-1% -> MLCC-CLASS
- CFLSN: renamed from RFHG; value 10R -> 100pF; footprint R0603 -> C1206; symbol traction-r1:R -> traction-r1:C; MPN R0603-CLASS -> MLCC-100pF-500V
- CFLVR: renamed from RFHGO; value 20R -> 100nF; footprint R0603 -> C0603; symbol traction-r1:R -> traction-r1:C; MPN R0603-CLASS -> MLCC-CLASS
- CLVH1: renamed from CVBDF; value 1nF -> 4.7uF; footprint C0603 -> C1206; MPN MLCC-1nF-50V -> MLCC-4.7uF-50V
- CLVH2: renamed from RVBD1; value 470k -> 4.7uF; footprint R1206 -> C1206; symbol traction-r1:R -> traction-r1:C; MPN R1206-470k-TF -> MLCC-4.7uF-50V
- CLVL1: renamed from RVBD6; value 470k -> 4.7uF; footprint R1206 -> C1206; symbol traction-r1:R -> traction-r1:C; MPN R1206-470k-TF -> MLCC-4.7uF-50V
- CLVL2: renamed from RVBDL; value 6.2k -> 4.7uF; footprint R0603 -> C1206; symbol traction-r1:R -> traction-r1:C; MPN R0603-6k2-0.1% -> MLCC-4.7uF-50V
- CUHB1: renamed from RBLD9; value 27k -> 100nF; footprint R2512 -> C0603; symbol traction-r1:R -> traction-r1:C; MPN R2512-27k-2W -> MLCC-100nF-50V
- CUHB2: renamed from PSQD; value QA01C-18 -> 4.7uF; footprint SIP7 -> C1206; symbol traction-r1:QA01C-18 -> traction-r1:C; MPN QA01C-18 -> MLCC-4.7uF-50V
- CUHBL: renamed from QDIS; value HCM75S12T4K3 -> 47pF; footprint TO247-4L -> C0603; symbol traction-r1:HCM75S12T4K3 -> traction-r1:C; MPN HCM75S12T4K3 -> MLCC-47pF-100V
- CUHE1: renamed from UQD; value TLP152 -> 10uF; footprint SO6 -> C1206; symbol traction-r1:TLP152 -> traction-r1:C; LCSC C17255258 -> CLASS; MPN TLP152 -> MLCC-10uF-25V
- CUHV1: renamed from CQD; value 100nF -> 4.7uF; footprint C0603 -> C1206; MPN MLCC-100nF-25V -> MLCC-4.7uF-50V
- CUSN: renamed from RBLD2; value 27k -> 1uF; footprint R2512 -> FilmP27.5; symbol traction-r1:R -> traction-r1:C; MPN R2512-27k-2W -> FILM-1uF-1200V
- CUTF: renamed from RBLD3; value 27k -> 2.2nF; footprint R2512 -> C0603; symbol traction-r1:R -> traction-r1:C; MPN R2512-27k-2W -> MLCC-2.2nF-50V
- CVBDF: renamed from RFLFB1; value 56k -> 1nF; footprint R0603 -> C0603; symbol traction-r1:R -> traction-r1:C; MPN R0603-1% -> MLCC-1nF-50V
- CVDDF: renamed from CFLCT; value 680pF -> 1nF; MPN MLCC-CLASS -> MLCC-1nF-50V
- CVHB1: renamed from DULS1; value US1M -> 100nF; footprint SMA -> C0603; symbol traction-r1:D -> traction-r1:C; LCSC C412437 -> CLASS; MPN US1M -> MLCC-100nF-50V
- CVHB2: renamed from DULS2; value US1M -> 4.7uF; footprint SMA -> C1206; symbol traction-r1:D -> traction-r1:C; LCSC C412437 -> CLASS; MPN US1M -> MLCC-4.7uF-50V
- CVHBL: renamed from DULZ1; value BZT52-C18 -> 47pF; footprint SOD123 -> C0603; symbol traction-r1:D -> traction-r1:C; MPN BZT52-C18 -> MLCC-47pF-100V
- CVHE1: renamed from DULZ2; value BZT52-C5V1 -> 10uF; footprint SOD123 -> C1206; symbol traction-r1:D -> traction-r1:C; MPN BZT52-C5V1 -> MLCC-10uF-25V
- CVHV1: renamed from RULBL; value 5.1k -> 4.7uF; footprint R0805 -> C1206; symbol traction-r1:R -> traction-r1:C; MPN R0805-4k99 -> MLCC-4.7uF-50V
- CVSN: renamed from UULG; value NSI6611A-Q1 -> 1uF; footprint SOIC16W -> FilmP27.5; symbol traction-r1:NSI6611A-Q1 -> traction-r1:C; LCSC C7470934 -> CLASS; MPN NSI6611A-Q1 -> FILM-1uF-1200V
- CVTF: renamed from CULB1; value 100nF -> 2.2nF; MPN MLCC-100nF-50V -> MLCC-2.2nF-50V
- CWHB1: renamed from DVLS1; value US1M -> 100nF; footprint SMA -> C0603; symbol traction-r1:D -> traction-r1:C; LCSC C412437 -> CLASS; MPN US1M -> MLCC-100nF-50V
- CWHB2: renamed from DVLS2; value US1M -> 4.7uF; footprint SMA -> C1206; symbol traction-r1:D -> traction-r1:C; LCSC C412437 -> CLASS; MPN US1M -> MLCC-4.7uF-50V
- CWHBL: renamed from DVLZ1; value BZT52-C18 -> 47pF; footprint SOD123 -> C0603; symbol traction-r1:D -> traction-r1:C; MPN BZT52-C18 -> MLCC-47pF-100V
- CWHE1: renamed from DVLZ2; value BZT52-C5V1 -> 10uF; footprint SOD123 -> C1206; symbol traction-r1:D -> traction-r1:C; MPN BZT52-C5V1 -> MLCC-10uF-25V
- CWHV1: renamed from RVLBL; value 5.1k -> 4.7uF; footprint R0805 -> C1206; symbol traction-r1:R -> traction-r1:C; MPN R0805-4k99 -> MLCC-4.7uF-50V
- CWSN: renamed from UVLG; value NSI6611A-Q1 -> 1uF; footprint SOIC16W -> FilmP27.5; symbol traction-r1:NSI6611A-Q1 -> traction-r1:C; LCSC C7470934 -> CLASS; MPN NSI6611A-Q1 -> FILM-1uF-1200V
- CWTF: renamed from CVLB1; value 100nF -> 2.2nF; MPN MLCC-100nF-50V -> MLCC-2.2nF-50V
- DB15: renamed from CLVH1; value 4.7uF -> SS34; footprint C1206 -> SMA; symbol traction-r1:C -> traction-r1:D; MPN MLCC-4.7uF-50V -> SS34
- DFHA: renamed from RWLGS; value 10k -> US1M; footprint R0805 -> SMA; symbol traction-r1:R -> traction-r1:D; LCSC CLASS -> C412437; MPN R0805-10k -> US1M
- DFHG: renamed from RWLMC; value 0R -> PMEG4010EH; footprint R0805 -> SOD123; symbol traction-r1:R -> traction-r1:D; LCSC CLASS -> C282566; MPN R0805-0R -> PMEG4010EH
- DFHSN: renamed from RWLOFF; value 1R -> SMBJ85A; footprint R2512 -> SMB; symbol traction-r1:R -> traction-r1:D; MPN R2512-1R0-2W -> SMBJ85A
- DFLA: renamed from RFHGS; value 51k -> US1M; footprint R0603 -> SMA; symbol traction-r1:R -> traction-r1:D; LCSC CLASS -> C412437; MPN R0603-CLASS -> US1M
- DFLG: renamed from RFHRT; value 10k -> PMEG4010EH; footprint R0603 -> SOD123; symbol traction-r1:R -> traction-r1:D; LCSC CLASS -> C282566; MPN R0603-CLASS -> PMEG4010EH
- DFLSN: renamed from RFHSI; value 100R -> SMBJ85A; footprint R0603 -> SMB; symbol traction-r1:R -> traction-r1:D; MPN R0603-CLASS -> SMBJ85A
- DRH: renamed from RVBD2; value 470k -> NRVBAF360T3G; footprint R1206 -> SMA-flat; symbol traction-r1:R -> traction-r1:D; MPN R1206-470k-TF -> NRVBAF360T3G
- DRL: renamed from PS5B; value ISO5V-RFC-6K -> NRVBAF360T3G; footprint SIP7 -> SMA-flat; symbol traction-r1:ISO5V-RFC-6K -> traction-r1:D; MPN ISO5V-RFC-6K -> NRVBAF360T3G
- DTVH: renamed from RVBD3; value 470k -> TPSMC24CA; footprint R1206 -> SMC; symbol traction-r1:R -> traction-r1:D; LCSC CLASS -> C1975284; MPN R1206-470k-TF -> TPSMC24CA
- DTVL: renamed from PS5C; value ISO5V-RFC-6K -> TPSMC24CA; footprint SIP7 -> SMC; symbol traction-r1:ISO5V-RFC-6K -> traction-r1:D; LCSC CLASS -> C1975284; MPN ISO5V-RFC-6K -> TPSMC24CA
- DUHR: renamed from RDIS1; value 470R -> US1M; footprint AxialWW10W -> SMA; symbol traction-r1:R -> traction-r1:D; LCSC CLASS -> C412437; MPN WW-470R-10W-AX -> US1M
- DUHS1: renamed from RDIS2; value 470R -> US1M; footprint AxialWW10W -> SMA; symbol traction-r1:R -> traction-r1:D; LCSC CLASS -> C412437; MPN WW-470R-10W-AX -> US1M
- DUHS2: renamed from RDIS3; value 470R -> US1M; footprint AxialWW10W -> SMA; symbol traction-r1:R -> traction-r1:D; LCSC CLASS -> C412437; MPN WW-470R-10W-AX -> US1M
- DUHSB: renamed from RBLD7; value 27k -> BAT64-04; footprint R2512 -> SOT23; symbol traction-r1:R -> traction-r1:BAT64-04; MPN R2512-27k-2W -> BAT64-04
- DUHZ1: renamed from RDIS4; value 470R -> BZT52-C18; footprint AxialWW10W -> SOD123; symbol traction-r1:R -> traction-r1:D; MPN WW-470R-10W-AX -> BZT52-C18
- DUHZ2: renamed from RQDG; value 47R -> BZT52-C5V1; footprint R0603 -> SOD123; symbol traction-r1:R -> traction-r1:D; MPN R0603-47R -> BZT52-C5V1
- DUTP: renamed from RBLD4; value 27k -> PESD5V0U1UA; footprint R2512 -> SOD323; symbol traction-r1:R -> traction-r1:D; MPN R2512-27k-2W -> PESD5V0U1UA
- DVHR: renamed from RULDS; value 100R -> US1M; footprint R0805 -> SMA; symbol traction-r1:R -> traction-r1:D; LCSC CLASS -> C412437; MPN R0805-100R -> US1M
- DVHS1: renamed from RULGS; value 10k -> US1M; footprint R0805 -> SMA; symbol traction-r1:R -> traction-r1:D; LCSC CLASS -> C412437; MPN R0805-10k -> US1M
- DVHS2: renamed from RULMC; value 0R -> US1M; footprint R0805 -> SMA; symbol traction-r1:R -> traction-r1:D; LCSC CLASS -> C412437; MPN R0805-0R -> US1M
- DVHSB: renamed from CULV1; value 4.7uF -> BAT64-04; footprint C1206 -> SOT23; symbol traction-r1:C -> traction-r1:BAT64-04; MPN MLCC-4.7uF-50V -> BAT64-04
- DVHZ1: renamed from RULOFF; value 1R -> BZT52-C18; footprint R2512 -> SOD123; symbol traction-r1:R -> traction-r1:D; MPN R2512-1R0-2W -> BZT52-C18
- DVHZ2: renamed from RULON; value 1.5R -> BZT52-C5V1; footprint R2512 -> SOD123; symbol traction-r1:R -> traction-r1:D; MPN R2512-1R5-2W -> BZT52-C5V1
- DVTP: renamed from CULB2; value 4.7uF -> PESD5V0U1UA; footprint C1206 -> SOD323; symbol traction-r1:C -> traction-r1:D; MPN MLCC-4.7uF-50V -> PESD5V0U1UA
- DWHR: renamed from RVLDS; value 100R -> US1M; footprint R0805 -> SMA; symbol traction-r1:R -> traction-r1:D; LCSC CLASS -> C412437; MPN R0805-100R -> US1M
- renumbered CUHB1 to CULB1, CUHB2 to CULB2, CUHBL to CULBL, CUHE1 to CULE1, CUHV1 to CULV1, CVHB1 to CVLB1, CVHB2 to CVLB2, CVHBL to CVLBL, CVHE1 to CVLE1, CVHV1 to CVLV1, CWHB1 to CWLB1, CWHB2 to CWLB2, CWHBL to CWLBL, CWHE1 to CWLE1, CWHV1 to CWLV1, DUHR to DULR, DUHS1 to DULS1, DUHS2 to DULS2, DUHSB to DULSB, DUHZ1 to DULZ1, DUHZ2 to DULZ2, DVHR to DVLR, DVHS1 to DVLS1, DVHS2 to DVLS2, DVHSB to DVLSB, DVHZ1 to DVLZ1, DVHZ2 to DVLZ2, DWHR to DWLR, DWHS1 to DWLS1, DWHS2 to DWLS2, DWHSB to DWLSB, DWHZ1 to DWLZ1, DWHZ2 to DWLZ2, RUHBL to RULBL, RUHDS to RULDS, RUHGS to RULGS, RUHMC to RULMC, RUHOFF to RULOFF, RUHON to RULON, RUHPD to RULPD, RVHBL to RVLBL, RVHDS to RVLDS, RVHGS to RVLGS, RVHMC to RVLMC, RVHOFF to RVLOFF, RVHON to RVLON, RVHPD to RVLPD, RWHBL to RWLBL, RWHDS to RWLDS, RWHGS to RWLGS, RWHMC to RWLMC, RWHOFF to RWLOFF, RWHON to RWLON, RWHPD to RWLPD, UUHG to UULG, UVHG to UVLG, UWHG to UWLG, ZUHV to ZULV, ZVHV to ZVLV, ZWHV to ZWLV
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Connections:
- net labels removed: BL01, BL02, BL03, BL04, BL11, BL12, BL13, BL14, DIS1, DIS2, DIS3, G_QDIS, QDA, QDVO, QD_D, V18Q
- wire segments 839 -> 794
Other:
- note added: "220 kW pk Power (HV) - 1 of 3"
- note added: "DC-LINK - 2 sections"
- note added: "DC-LINK / DISCH-IF"
- note added: "rev A.3 - 25 sections - 290 components"
- note removed: "220 kW pk Power (HV) - 1 of 2"
- note removed: "DC-LINK - 3 sections"
- note removed: "DC-LINK / BLEED"
- note removed: "DC-LINK / DISCHARGE"
- note removed: "rev A.3 - 26 sections - 310 components"
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
Commit message: Add cap-bank busbar assembly sheet + explicit interboard links (4 sheets)
- boards/capbank.tsx: the 16-can DC-link is its own laminated-busbar
  assembly (FR4 cannot carry the 340 A bus) with every terminal drawn:
  entry lugs, 3x module DC tab pairs, discharge-board studs
- power board keeps only its DCP/DCN entry taps (Y-caps, HVIL, sense)
- interboard links L1-L5 (harness, discharge 4-way, busbar, LEM, HVIL)
  documented in design-basis 10a + README table; erc-audit now asserts
  both ends of every link (new interboard section)
- NET NAMING panels state the cross-sheet net rule on every sheet
- gates green: 1560/1560 pins, ERC 687/0, design-verify 51P/3W/0F
- BOM ₹69,996 @1k (58,575 / 4,940 / 672 / 5,808) · 543 comps · 175 lines

Co-Authored-By: Claude Fable 5 <noreply@anthropic.com>
Parts:
- removed DB15: SS34, SMA, symbol traction-r1:D
- removed JIC: MICROFIT3-40, MicroFit40, symbol traction-r1:MICROFIT3-40
- removed LB15: IND-10uH-3A, IND6x6, symbol traction-r1:L
- removed RB15F1: 110k, R0603, symbol traction-r1:R
- removed RB15F2: 9.53k, R0603, symbol traction-r1:R
- removed RPD0, RPD1, RPD10, RPD2, RPD3, RPD4, RPD5, RPD6, RPD7, RPD8, RPD9: 10k, R0603, symbol traction-r1:R
- C5B1: renamed from RVDD3; value 470k -> 1uF; footprint R1206 -> C0603; symbol traction-r1:R -> traction-r1:C; MPN R1206-470k-TF -> MLCC-1uF-25V
- C5B2: renamed from RVDD4; value 470k -> 100nF; footprint R1206 -> C0603; symbol traction-r1:R -> traction-r1:C; MPN R1206-470k-TF -> MLCC-1uF-25V
- C5C1: renamed from RVDD5; value 470k -> 1uF; footprint R1206 -> C0603; symbol traction-r1:R -> traction-r1:C; MPN R1206-470k-TF -> MLCC-1uF-25V
- C5G1: renamed from RASCL; value 470R -> 1uF; footprint R0603 -> C1206; symbol traction-r1:R -> traction-r1:C; MPN R0603-470R -> MLCC-10uF-25V
- C5G2: renamed from RASCPD; value 10k -> 10uF; footprint R0603 -> C1206; symbol traction-r1:R -> traction-r1:C; MPN R0603-10k -> MLCC-10uF-25V
- CASC: renamed from UIVB; value AMC1311BDWVR -> 100nF; footprint SOIC8W -> C0603; symbol traction-r1:AMC1311BDWVR -> traction-r1:C; LCSC C456277 -> CLASS; MPN AMC1311BDWVR -> MLCC-100nF-25V
- CB15C: renamed from CLVH1; value 4.7uF -> 10nF; footprint C1206 -> C0603; MPN MLCC-4.7uF-50V -> MLCC-CLASS
- CB15I: renamed from CLVH2; value 4.7uF -> 10uF; footprint C1206 -> C1210; MPN MLCC-4.7uF-50V -> MLCC-10uF-50V
- CB15O1: renamed from DRH; value NRVBAF360T3G -> 22uF; footprint SMA-flat -> C1210; symbol traction-r1:D -> traction-r1:C; MPN NRVBAF360T3G -> MLCC-22uF-25V
- CB15O2: renamed from DTVH; value TPSMC24CA -> 22uF; footprint SMC -> C1210; symbol traction-r1:D -> traction-r1:C; LCSC C1975284 -> CLASS; MPN TPSMC24CA -> MLCC-22uF-25V
- CFHA: renamed from DWLZ2; value BZT52-C5V1 -> 4.7uF; footprint SOD123 -> C1206; symbol traction-r1:D -> traction-r1:C; MPN BZT52-C5V1 -> MLCC-4.7uF-50V
- CFHCF: renamed from RWLBL; value 5.1k -> 47pF; footprint R0805 -> C0603; symbol traction-r1:R -> traction-r1:C; MPN R0805-4k99 -> MLCC-CLASS
- CFHCO: renamed from RWLDS; value 100R -> 22nF; footprint R0805 -> C0603; symbol traction-r1:R -> traction-r1:C; MPN R0805-100R -> MLCC-CLASS
- CFHCT: renamed from RWLGS; value 10k -> 680pF; footprint R0805 -> C0603; symbol traction-r1:R -> traction-r1:C; MPN R0805-10k -> MLCC-CLASS
- CFHSI: renamed from RWLMC; value 0R -> 100pF; footprint R0805 -> C0603; symbol traction-r1:R -> traction-r1:C; MPN R0805-0R -> MLCC-CLASS
- CFHSN: renamed from RWLOFF; value 1R -> 100pF; footprint R2512 -> C1206; symbol traction-r1:R -> traction-r1:C; MPN R2512-1R0-2W -> MLCC-100pF-500V
- CFHVR: renamed from RWLON; value 1.5R -> 100nF; footprint R2512 -> C0603; symbol traction-r1:R -> traction-r1:C; MPN R2512-1R5-2W -> MLCC-CLASS
- CFLA: renamed from RFHFB2; value 15k -> 4.7uF; footprint R0603 -> C1206; symbol traction-r1:R -> traction-r1:C; MPN R0603-1% -> MLCC-4.7uF-50V
- CFLCF: renamed from RFHG; value 10R -> 47pF; footprint R0603 -> C0603; symbol traction-r1:R -> traction-r1:C; MPN R0603-CLASS -> MLCC-CLASS
- CFLCO: renamed from RFHGO; value 20R -> 22nF; footprint R0603 -> C0603; symbol traction-r1:R -> traction-r1:C; MPN R0603-CLASS -> MLCC-CLASS
- CFLCT: renamed from RFHGS; value 51k -> 680pF; footprint R0603 -> C0603; symbol traction-r1:R -> traction-r1:C; MPN R0603-CLASS -> MLCC-CLASS
- CFLSI: renamed from RFHRT; value 10k -> 100pF; footprint R0603 -> C0603; symbol traction-r1:R -> traction-r1:C; MPN R0603-CLASS -> MLCC-CLASS
- CFLSN: renamed from RFHSI; value 100R -> 100pF; footprint R0603 -> C1206; symbol traction-r1:R -> traction-r1:C; MPN R0603-CLASS -> MLCC-100pF-500V
- CFLVR: renamed from RFHSN; value 100R -> 100nF; footprint R0805 -> C0603; symbol traction-r1:R -> traction-r1:C; MPN R0805-100R -> MLCC-CLASS
- CLVH1: renamed from RVBD4; value 470k -> 4.7uF; footprint R1206 -> C1206; symbol traction-r1:R -> traction-r1:C; MPN R1206-470k-TF -> MLCC-4.7uF-50V
- CLVH2: renamed from RVBD5; value 470k -> 4.7uF; footprint R1206 -> C1206; symbol traction-r1:R -> traction-r1:C; MPN R1206-470k-TF -> MLCC-4.7uF-50V
- CLVL1: renamed from C5B1; value 1uF -> 4.7uF; footprint C0603 -> C1206; MPN MLCC-1uF-25V -> MLCC-4.7uF-50V
- CLVL2: renamed from C5B2; value 100nF -> 4.7uF; footprint C0603 -> C1206; MPN MLCC-1uF-25V -> MLCC-4.7uF-50V
- CUHB1: renamed from CDC3; value 20uF -> 100nF; footprint FilmCan37.5 -> C0603; LCSC C2840809 -> CLASS; MPN C3D1M206KFSA382 -> MLCC-100nF-50V
- CUHB2: renamed from CDC4; value 20uF -> 4.7uF; footprint FilmCan37.5 -> C1206; LCSC C2840809 -> CLASS; MPN C3D1M206KFSA382 -> MLCC-4.7uF-50V
- CUHBL: renamed from CDC5; value 20uF -> 47pF; footprint FilmCan37.5 -> C0603; LCSC C2840809 -> CLASS; MPN C3D1M206KFSA382 -> MLCC-47pF-100V
- CUHE1: renamed from CDC6; value 20uF -> 10uF; footprint FilmCan37.5 -> C1206; LCSC C2840809 -> CLASS; MPN C3D1M206KFSA382 -> MLCC-10uF-25V
- CUHV1: renamed from CDC7; value 20uF -> 4.7uF; footprint FilmCan37.5 -> C1206; LCSC C2840809 -> CLASS; MPN C3D1M206KFSA382 -> MLCC-4.7uF-50V
- CULB1: renamed from CUHV1; value 4.7uF -> 100nF; footprint C1206 -> C0603; MPN MLCC-4.7uF-50V -> MLCC-100nF-50V
- CULB2: renamed from DUHR; value US1M -> 4.7uF; footprint SMA -> C1206; symbol traction-r1:D -> traction-r1:C; LCSC C412437 -> CLASS; MPN US1M -> MLCC-4.7uF-50V
- CULBL: renamed from DUHS1; value US1M -> 47pF; footprint SMA -> C0603; symbol traction-r1:D -> traction-r1:C; LCSC C412437 -> CLASS; MPN US1M -> MLCC-47pF-100V
- CULE1: renamed from DUHS2; value US1M -> 10uF; footprint SMA -> C1206; symbol traction-r1:D -> traction-r1:C; LCSC C412437 -> CLASS; MPN US1M -> MLCC-10uF-25V
- CULV1: renamed from DUHZ1; value BZT52-C18 -> 4.7uF; footprint SOD123 -> C1206; symbol traction-r1:D -> traction-r1:C; MPN BZT52-C18 -> MLCC-4.7uF-50V
- CUSN: renamed from CDC11; value 20uF -> 1uF; footprint FilmCan37.5 -> FilmP27.5; LCSC C2840809 -> CLASS; MPN C3D1M206KFSA382 -> FILM-1uF-1200V
- CUTF: renamed from CDC12; value 20uF -> 2.2nF; footprint FilmCan37.5 -> C0603; LCSC C2840809 -> CLASS; MPN C3D1M206KFSA382 -> MLCC-2.2nF-50V
- CVBDF: renamed from RFLGS; value 51k -> 1nF; footprint R0603 -> C0603; symbol traction-r1:R -> traction-r1:C; MPN R0603-CLASS -> MLCC-1nF-50V
- CVDDF: renamed from DFLA; value US1M -> 1nF; footprint SMA -> C0603; symbol traction-r1:D -> traction-r1:C; LCSC C412437 -> CLASS; MPN US1M -> MLCC-1nF-50V
- CVHB1: renamed from RULBL; value 5.1k -> 100nF; footprint R0805 -> C0603; symbol traction-r1:R -> traction-r1:C; MPN R0805-4k99 -> MLCC-100nF-50V
- CVHB2: renamed from RULDS; value 100R -> 4.7uF; footprint R0805 -> C1206; symbol traction-r1:R -> traction-r1:C; MPN R0805-100R -> MLCC-4.7uF-50V
- CVHBL: renamed from RULGS; value 10k -> 47pF; footprint R0805 -> C0603; symbol traction-r1:R -> traction-r1:C; MPN R0805-10k -> MLCC-47pF-100V
- CVHE1: renamed from RULMC; value 0R -> 10uF; footprint R0805 -> C1206; symbol traction-r1:R -> traction-r1:C; MPN R0805-0R -> MLCC-10uF-25V
- CVHV1: renamed from RULOFF; value 1R -> 4.7uF; footprint R2512 -> C1206; symbol traction-r1:R -> traction-r1:C; MPN R2512-1R0-2W -> MLCC-4.7uF-50V
- CVLB1: renamed from CVHV1; value 4.7uF -> 100nF; footprint C1206 -> C0603; MPN MLCC-4.7uF-50V -> MLCC-100nF-50V
- CVLB2: renamed from DVHR; value US1M -> 4.7uF; footprint SMA -> C1206; symbol traction-r1:D -> traction-r1:C; LCSC C412437 -> CLASS; MPN US1M -> MLCC-4.7uF-50V
- CVLBL: renamed from DVHS1; value US1M -> 47pF; footprint SMA -> C0603; symbol traction-r1:D -> traction-r1:C; LCSC C412437 -> CLASS; MPN US1M -> MLCC-47pF-100V
- CVLE1: renamed from DVHS2; value US1M -> 10uF; footprint SMA -> C1206; symbol traction-r1:D -> traction-r1:C; LCSC C412437 -> CLASS; MPN US1M -> MLCC-10uF-25V
- CVLV1: renamed from DVHZ1; value BZT52-C18 -> 4.7uF; footprint SOD123 -> C1206; symbol traction-r1:D -> traction-r1:C; MPN BZT52-C18 -> MLCC-4.7uF-50V
- CVSN: renamed from CULE1; value 10uF -> 1uF; footprint C1206 -> FilmP27.5; MPN MLCC-10uF-25V -> FILM-1uF-1200V
- CVTF: renamed from CULV1; value 4.7uF -> 2.2nF; footprint C1206 -> C0603; MPN MLCC-4.7uF-50V -> MLCC-2.2nF-50V
- CWHB1: renamed from RVLBL; value 5.1k -> 100nF; footprint R0805 -> C0603; symbol traction-r1:R -> traction-r1:C; MPN R0805-4k99 -> MLCC-100nF-50V
- CWHB2: renamed from RVLDS; value 100R -> 4.7uF; footprint R0805 -> C1206; symbol traction-r1:R -> traction-r1:C; MPN R0805-100R -> MLCC-4.7uF-50V
- CWHBL: renamed from RVLGS; value 10k -> 47pF; footprint R0805 -> C0603; symbol traction-r1:R -> traction-r1:C; MPN R0805-10k -> MLCC-47pF-100V
- CWHE1: renamed from RVLMC; value 0R -> 10uF; footprint R0805 -> C1206; symbol traction-r1:R -> traction-r1:C; MPN R0805-0R -> MLCC-10uF-25V
- CWHV1: renamed from RVLOFF; value 1R -> 4.7uF; footprint R2512 -> C1206; symbol traction-r1:R -> traction-r1:C; MPN R2512-1R0-2W -> MLCC-4.7uF-50V
- CWLB1: renamed from CWHV1; value 4.7uF -> 100nF; footprint C1206 -> C0603; MPN MLCC-4.7uF-50V -> MLCC-100nF-50V
- CWLB2: renamed from DWHR; value US1M -> 4.7uF; footprint SMA -> C1206; symbol traction-r1:D -> traction-r1:C; LCSC C412437 -> CLASS; MPN US1M -> MLCC-4.7uF-50V
- CWLBL: renamed from DWHS1; value US1M -> 47pF; footprint SMA -> C0603; symbol traction-r1:D -> traction-r1:C; LCSC C412437 -> CLASS; MPN US1M -> MLCC-47pF-100V
- CWLE1: renamed from DWHS2; value US1M -> 10uF; footprint SMA -> C1206; symbol traction-r1:D -> traction-r1:C; LCSC C412437 -> CLASS; MPN US1M -> MLCC-10uF-25V
- CWLV1: renamed from DWHZ1; value BZT52-C18 -> 4.7uF; footprint SOD123 -> C1206; symbol traction-r1:D -> traction-r1:C; MPN BZT52-C18 -> MLCC-4.7uF-50V
- CWSN: renamed from CVLE1; value 10uF -> 1uF; footprint C1206 -> FilmP27.5; MPN MLCC-10uF-25V -> FILM-1uF-1200V
- CWTF: renamed from CVLV1; value 4.7uF -> 2.2nF; footprint C1206 -> C0603; MPN MLCC-4.7uF-50V -> MLCC-2.2nF-50V
- DB15: renamed from FH1; value MF-LSMF300/24X-2 -> SS34; footprint PTC2920 -> SMA; symbol traction-r1:F -> traction-r1:D; LCSC C719172 -> CLASS; MPN MF-LSMF300/24X-2 -> SS34
- DFHA: renamed from RWLPD; value 1M -> US1M; footprint R1206 -> SMA; symbol traction-r1:R -> traction-r1:D; LCSC CLASS -> C412437; MPN HV73-1M-1206 -> US1M
- DFHG: renamed from ZWLV; value BZT52-C5V1 -> PMEG4010EH; LCSC CLASS -> C282566; MPN BZT52-C5V1 -> PMEG4010EH
- DFHSN: renamed from QFH; value BUK9Y14-80E -> SMBJ85A; footprint LFPAK56 -> SMB; symbol traction-r1:BUK9Y14-80E -> traction-r1:D; LCSC C86732 -> CLASS; MPN BUK9Y14-80E -> SMBJ85A
- DFLA: renamed from RFHST; value 4.7k -> US1M; footprint R0603 -> SMA; symbol traction-r1:R -> traction-r1:D; LCSC CLASS -> C412437; MPN R0603-CLASS -> US1M
- DFLG: renamed from ZFHG; value BZT52-C5V6 -> PMEG4010EH; LCSC CLASS -> C282566; MPN BZT52-C5V6 -> PMEG4010EH
- DFLSN: renamed from QFL; value BUK9Y14-80E -> SMBJ85A; footprint LFPAK56 -> SMB; symbol traction-r1:BUK9Y14-80E -> traction-r1:D; LCSC C86732 -> CLASS; MPN BUK9Y14-80E -> SMBJ85A
- DRH: renamed from RVBD6; value 470k -> NRVBAF360T3G; footprint R1206 -> SMA-flat; symbol traction-r1:R -> traction-r1:D; MPN R1206-470k-TF -> NRVBAF360T3G
- DRL: renamed from C5C1; value 1uF -> NRVBAF360T3G; footprint C0603 -> SMA-flat; symbol traction-r1:C -> traction-r1:D; MPN MLCC-1uF-25V -> NRVBAF360T3G
- DTVH: renamed from RVBDL; value 6.2k -> TPSMC24CA; footprint R0603 -> SMC; symbol traction-r1:R -> traction-r1:D; LCSC CLASS -> C1975284; MPN R0603-6k2-0.1% -> TPSMC24CA
- DTVL: renamed from PSASC; value QA01C-18 -> TPSMC24CA; footprint SIP7 -> SMC; symbol traction-r1:QA01C-18 -> traction-r1:D; LCSC CLASS -> C1975284; MPN QA01C-18 -> TPSMC24CA
- DUHR: renamed from CDC8; value 20uF -> US1M; footprint FilmCan37.5 -> SMA; symbol traction-r1:C -> traction-r1:D; LCSC C2840809 -> C412437; MPN C3D1M206KFSA382 -> US1M
- DUHS1: renamed from CDC9; value 20uF -> US1M; footprint FilmCan37.5 -> SMA; symbol traction-r1:C -> traction-r1:D; LCSC C2840809 -> C412437; MPN C3D1M206KFSA382 -> US1M
- DUHS2: renamed from JDIS; value HDR-1x4-2.54 -> US1M; footprint HDR1x4 -> SMA; symbol traction-r1:HDR-1x4-2.54 -> traction-r1:D; LCSC CLASS -> C412437; MPN HDR-1x4-2.54 -> US1M
- DUHSB: renamed from CDC16; value 20uF -> BAT64-04; footprint FilmCan37.5 -> SOT23; symbol traction-r1:C -> traction-r1:BAT64-04; LCSC C2840809 -> CLASS; MPN C3D1M206KFSA382 -> BAT64-04
- DUHZ1: renamed from MODU; value HCS600FH120D3C1 -> BZT52-C18; footprint EconoDUAL3 -> SOD123; symbol traction-r1:HCS600FH120D3C1 -> traction-r1:D; MPN HCS600FH120D3C1 -> BZT52-C18
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Connections:
- wire segments 794 -> 762
Other:
- note added: "+ 10 more"
- note added: "220 kW pk Power (HV) - 1 of 4"
- note added: "DC-LINK - 1 section"
- note added: "named connector/stud/tab (see INTERBOARD LINKS, design basis)"
- note added: "rev A.3 - 24 sections - 274 components"
- note added: "same name on another sheet = same net, joined ONLY at the"
- note removed: "--- DISCHARGE ---"
- note removed: "220 kW pk Power (HV) - 1 of 3"
- note removed: "6 3x hall + sum(I)=0 plausibility (torque path)"
- note removed: "7 2x isolated VDC senses, >5% mismatch = fault"
- note removed: "8 DESAT per switch, ~1.5 us blanking, latching"
- note removed: "9 HVIL open = VDDIO/2 signature -> discharge"
- note removed: "ACTIVE QDIS + 4x 470R 10W = 1.88k: 1.6 s to 60 V"
- note removed: "DC-LINK - 2 sections"
- note removed: "DC-LINK / LINK-BANK"
- note removed: "E = 116 J @850 V - 32 J/res worst (>=100 J rated)"
- note removed: "PASSIVE 10x 27k 2512-2W (5s x 2p = 67.5k): 58 s to 60 V"
- note removed: "RULE: never energize without the bleeder fitted"
- note removed: "VERIFY: MCU fires QDIS, watches BOTH VDC channels"
- note removed: "rev A.3 - 25 sections - 290 components"
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