File: kicad5/traction/traction-power.sch (KiCad schematic (older format))
At the start: 274 parts

Commit message: Rev A.4: answer external design review — 10 confirmed defects fixed (F37-F46)
Every claim verified against primary datasheets before any edit; three
claims rebutted with evidence (850V/0.1% divider corner, GEN3-exact
resolver monitors, discharge math matches). Fixed:

- F37 VGT12EEM secondary phasing: rectifier moved to pin 8 (dot); the
  drawn wiring was forward-mode ~35V into +22V-abs gates. Pins 6/7 NC'd
  (no internal winding). Aux (NF) was already correct.
- F38 flyback drain clamp: SMBJ85A (forward every OFF interval, 94.4V
  min breakdown vs 80V FET) -> US1M + SMAJ13A winding clamp; drain
  <=60V at clamped load dump
- F39 DESAT clamp: BAT64-04 series pair correctly oriented DESAT->VCC2
  (was VCC2 injected into DESAT via a wrong common-cathode symbol)
- F40 ASC latch: real SN74LVC1G74 DCU pins; 1k/10k network (was
  120R/120R = 2.5V "low" and 42mA MCU clear)
- F41 KL15: 47k/10k+100nF ADC sense (was raw 13.3V into PTA25)
- F42 VDC receivers offset +0.5V (buffered) - AMC1311 fail-safe now
  distinguishable from a dead bus
- F44 VBAT_H/L actually sourced (FVBH/FVBL polyfuses off NRC)
- F45 real package pins everywhere: 74LVC1G11 (had NO VCC pin), 1G32,
  NCV4276C (OUT=5), TPS55340 RTE16 (+SS cap +FREQ R), BUK9Y14 LFPAK56,
  ALM2402 PWP14 (+VCC_O, SHDN via 10k pullup), QA01C SIP-7, PESD as
  real 2/3-terminal parts, FS26 full LQFP-48+EP with VDIG/VBOS/
  bootstraps/DEBUG strap and DS unused-pin terminations; S32K396
  explicitly symbolic (no package table in DS - bind at layout)
- F46 hardware fault latch: FLT_HS/LS diode-OR -> LVC1G74 -> DRV_EN;
  any DESAT latches all six channels off until MCU clears
- NSI6611ASC-Q1SWR full ordering code (ASC variant)

erc-audit gains a rev-A.4 lock-in section (763 checks, 0 fail);
design-verify adds F37-F46 corner rows (60 PASS/3 WARN/0 FAIL);
pin-verify 1663/1663; card void gate 9->12% (49-pin FS26 monolith);
BOM Rs.70,059 @1k, 579 components, 180 lines. design-basis 11a
documents the full review response including the rege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
Parts:
- added RPD0, RPD1, RPD10, RPD2, RPD3, RPD4, RPD5, RPD6, RPD7, RPD8, RPD9: 10k, R0603, symbol traction-r1:R
- C5B1: renamed from RASCPD; value 10k -> 1uF; footprint R0603 -> C0603; symbol traction-r1:R -> traction-r1:C; MPN R0603-10k -> MLCC-1uF-25V
- C5B2: renamed from ZASC; value BZT52-C5V1 -> 100nF; footprint SOD123 -> C0603; symbol traction-r1:D -> traction-r1:C; MPN BZT52-C5V1 -> MLCC-1uF-25V
- C5C1: renamed from CLVH1; value 4.7uF -> 1uF; footprint C1206 -> C0603; MPN MLCC-4.7uF-50V -> MLCC-1uF-25V
- C5G1: renamed from LB15; value IND-10uH-3A -> 1uF; footprint IND6x6 -> C1206; symbol traction-r1:L -> traction-r1:C; MPN IND-10uH-3A -> MLCC-10uF-25V
- C5G2: renamed from RB15F1; value 110k -> 10uF; footprint R0603 -> C1206; symbol traction-r1:R -> traction-r1:C; MPN R0603-1% -> MLCC-10uF-25V
- CASC: renamed from DTVH; value TPSMC24CA -> 100nF; footprint SMC -> C0603; symbol traction-r1:D -> traction-r1:C; LCSC C1975284 -> CLASS; MPN TPSMC24CA -> MLCC-100nF-25V
- CB15C: renamed from RPD0; value 10k -> 10nF; footprint R0603 -> C0603; symbol traction-r1:R -> traction-r1:C; MPN R0603-10k -> MLCC-CLASS
- CB15I: renamed from RPD1; value 10k -> 10uF; footprint R0603 -> C1210; symbol traction-r1:R -> traction-r1:C; MPN R0603-10k -> MLCC-10uF-50V
- CB15O1: renamed from RPD10; value 10k -> 22uF; footprint R0603 -> C1210; symbol traction-r1:R -> traction-r1:C; MPN R0603-10k -> MLCC-22uF-25V
- CB15O2: renamed from RPD2; value 10k -> 22uF; footprint R0603 -> C1210; symbol traction-r1:R -> traction-r1:C; MPN R0603-10k -> MLCC-22uF-25V
- CB15S: renamed from RPD3; value 10k -> 47nF; footprint R0603 -> C0603; symbol traction-r1:R -> traction-r1:C; MPN R0603-10k -> MLCC-CLASS
- CFHA: renamed from CFHVR; value 100nF -> 4.7uF; footprint C0603 -> C1206; MPN MLCC-CLASS -> MLCC-4.7uF-50V
- CFHCF: renamed from DFHA; value US1M -> 47pF; footprint SMA -> C0603; symbol traction-r1:D -> traction-r1:C; LCSC C412437 -> CLASS; MPN US1M -> MLCC-CLASS
- CFHCO: renamed from DFHG; value PMEG4010EH -> 22nF; footprint SOD123 -> C0603; symbol traction-r1:D -> traction-r1:C; LCSC C282566 -> CLASS; MPN PMEG4010EH -> MLCC-CLASS
- CFHCT: renamed from DFHSN; value SMBJ85A -> 680pF; footprint SMB -> C0603; symbol traction-r1:D -> traction-r1:C; MPN SMBJ85A -> MLCC-CLASS
- CFHSI: renamed from RFHCS; value 330m -> 100pF; footprint R1210 -> C0603; symbol traction-r1:R -> traction-r1:C; MPN R1210-0R33-0.75W -> MLCC-CLASS
- CFHSN: renamed from RFHEN; value 100k -> 100pF; footprint R0603 -> C1206; symbol traction-r1:R -> traction-r1:C; MPN R0603-CLASS -> MLCC-100pF-500V
- CFHVR: renamed from RFHFB1; value 56k -> 100nF; footprint R0603 -> C0603; symbol traction-r1:R -> traction-r1:C; MPN R0603-1% -> MLCC-CLASS
- CFLA: renamed from DFLA; value US1M -> 4.7uF; footprint SMA -> C1206; symbol traction-r1:D -> traction-r1:C; LCSC C412437 -> CLASS; MPN US1M -> MLCC-4.7uF-50V
- CFLCF: renamed from DFLG; value PMEG4010EH -> 47pF; footprint SOD123 -> C0603; symbol traction-r1:D -> traction-r1:C; LCSC C282566 -> CLASS; MPN PMEG4010EH -> MLCC-CLASS
- CFLCO: renamed from DFLSN; value SMBJ85A -> 22nF; footprint SMB -> C0603; symbol traction-r1:D -> traction-r1:C; MPN SMBJ85A -> MLCC-CLASS
- CFLCT: renamed from RFLCS; value 330m -> 680pF; footprint R1210 -> C0603; symbol traction-r1:R -> traction-r1:C; MPN R1210-0R33-0.75W -> MLCC-CLASS
- CFLSI: renamed from RFLEN; value 100k -> 100pF; footprint R0603 -> C0603; symbol traction-r1:R -> traction-r1:C; MPN R0603-CLASS -> MLCC-CLASS
- CFLSN: renamed from RFLFB1; value 56k -> 100pF; footprint R0603 -> C1206; symbol traction-r1:R -> traction-r1:C; MPN R0603-1% -> MLCC-100pF-500V
- CFLVR: renamed from RFLFB2; value 15k -> 100nF; footprint R0603 -> C0603; symbol traction-r1:R -> traction-r1:C; MPN R0603-1% -> MLCC-CLASS
- CLVH1: renamed from DRL; value NRVBAF360T3G -> 4.7uF; footprint SMA-flat -> C1206; symbol traction-r1:D -> traction-r1:C; MPN NRVBAF360T3G -> MLCC-4.7uF-50V
- CLVH2: renamed from DTVL; value TPSMC24CA -> 4.7uF; footprint SMC -> C1206; symbol traction-r1:D -> traction-r1:C; LCSC C1975284 -> CLASS; MPN TPSMC24CA -> MLCC-4.7uF-50V
- CLVL1: renamed from C5G2; value 10uF -> 4.7uF; MPN MLCC-10uF-25V -> MLCC-4.7uF-50V
- CLVL2: renamed from UB15; value TPS55340QRTERQ1 -> 4.7uF; footprint WQFN16 -> C1206; symbol traction-r1:TPS55340QRTERQ1 -> traction-r1:C; LCSC C2070860 -> CLASS; MPN TPS55340QRTERQ1 -> MLCC-4.7uF-50V
- CUHB1: renamed from UUHG; value NSI6611A-Q1 -> 100nF; footprint SOIC16W -> C0603; symbol traction-r1:NSI6611A-Q1 -> traction-r1:C; LCSC C7470934 -> CLASS; MPN NSI6611A-Q1 -> MLCC-100nF-50V
- CUHB2: renamed from CUHB1; value 100nF -> 4.7uF; footprint C0603 -> C1206; MPN MLCC-100nF-50V -> MLCC-4.7uF-50V
- CUHBL: renamed from CUHB2; value 4.7uF -> 47pF; footprint C1206 -> C0603; MPN MLCC-4.7uF-50V -> MLCC-47pF-100V
- CUHE1: renamed from CUHBL; value 47pF -> 10uF; footprint C0603 -> C1206; MPN MLCC-47pF-100V -> MLCC-10uF-25V
- CUHIN: renamed from CUHE1; value 10uF -> 100nF; footprint C1206 -> C0603; MPN MLCC-10uF-25V -> MLCC-CLASS
- CULIN: renamed from CULV1; value 4.7uF -> 100nF; footprint C1206 -> C0603; MPN MLCC-4.7uF-50V -> MLCC-CLASS
- CULV1: renamed from DULR; value US1M -> 4.7uF; footprint SMA -> C1206; symbol traction-r1:D -> traction-r1:C; LCSC C412437 -> CLASS; MPN US1M -> MLCC-4.7uF-50V
- CVBDF: renamed from PS5B; value ISO5V-RFC-6K -> 1nF; footprint SIP7 -> C0603; symbol traction-r1:ISO5V-RFC-6K -> traction-r1:C; MPN ISO5V-RFC-6K -> MLCC-1nF-50V
- CVDDF: renamed from UIVB; value AMC1311BDWVR -> 1nF; footprint SOIC8W -> C0603; symbol traction-r1:AMC1311BDWVR -> traction-r1:C; LCSC C456277 -> CLASS; MPN AMC1311BDWVR -> MLCC-1nF-50V
- CVHB1: renamed from CVHB2; value 4.7uF -> 100nF; footprint C1206 -> C0603; MPN MLCC-4.7uF-50V -> MLCC-100nF-50V
- CVHB2: renamed from CVHBL; value 47pF -> 4.7uF; footprint C0603 -> C1206; MPN MLCC-47pF-100V -> MLCC-4.7uF-50V
- CVHBL: renamed from CVHE1; value 10uF -> 47pF; footprint C1206 -> C0603; MPN MLCC-10uF-25V -> MLCC-47pF-100V
- CVHE1: renamed from CVHV1; value 4.7uF -> 10uF; MPN MLCC-4.7uF-50V -> MLCC-10uF-25V
- CVHIN: renamed from DVHR; value US1M -> 100nF; footprint SMA -> C0603; symbol traction-r1:D -> traction-r1:C; LCSC C412437 -> CLASS; MPN US1M -> MLCC-CLASS
- CVHV1: renamed from DVHS1; value US1M -> 4.7uF; footprint SMA -> C1206; symbol traction-r1:D -> traction-r1:C; LCSC C412437 -> CLASS; MPN US1M -> MLCC-4.7uF-50V
- CVLB1: renamed from CVLBL; value 47pF -> 100nF; MPN MLCC-47pF-100V -> MLCC-100nF-50V
- CVLB2: renamed from CVLE1; value 10uF -> 4.7uF; MPN MLCC-10uF-25V -> MLCC-4.7uF-50V
- CVLBL: renamed from CVLV1; value 4.7uF -> 47pF; footprint C1206 -> C0603; MPN MLCC-4.7uF-50V -> MLCC-47pF-100V
- CVLE1: renamed from DVLR; value US1M -> 10uF; footprint SMA -> C1206; symbol traction-r1:D -> traction-r1:C; LCSC C412437 -> CLASS; MPN US1M -> MLCC-10uF-25V
- CVLIN: renamed from DVLS1; value US1M -> 100nF; footprint SMA -> C0603; symbol traction-r1:D -> traction-r1:C; LCSC C412437 -> CLASS; MPN US1M -> MLCC-CLASS
- CVLV1: renamed from DVLS2; value US1M -> 4.7uF; footprint SMA -> C1206; symbol traction-r1:D -> traction-r1:C; LCSC C412437 -> CLASS; MPN US1M -> MLCC-4.7uF-50V
- CVSN: renamed from DVTP; value PESD5V0U1UA -> 1uF; footprint SOD323 -> FilmP27.5; symbol traction-r1:D -> traction-r1:C; MPN PESD5V0U1UA -> FILM-1uF-1200V
- CVTF: renamed from JMV; value STUD-M8 -> 2.2nF; footprint StudM8 -> C0603; symbol traction-r1:TERM_1 -> traction-r1:C; MPN STUD-M8 -> MLCC-2.2nF-50V
- CWHB1: renamed from CWHE1; value 10uF -> 100nF; footprint C1206 -> C0603; MPN MLCC-10uF-25V -> MLCC-100nF-50V
- CWHBL: renamed from DWHR; value US1M -> 47pF; footprint SMA -> C0603; symbol traction-r1:D -> traction-r1:C; LCSC C412437 -> CLASS; MPN US1M -> MLCC-47pF-100V
- CWHE1: renamed from DWHS1; value US1M -> 10uF; footprint SMA -> C1206; symbol traction-r1:D -> traction-r1:C; LCSC C412437 -> CLASS; MPN US1M -> MLCC-10uF-25V
- CWHIN: renamed from DWHS2; value US1M -> 100nF; footprint SMA -> C0603; symbol traction-r1:D -> traction-r1:C; LCSC C412437 -> CLASS; MPN US1M -> MLCC-CLASS
- CWHV1: renamed from DWHZ1; value BZT52-C18 -> 4.7uF; footprint SOD123 -> C1206; symbol traction-r1:D -> traction-r1:C; MPN BZT52-C18 -> MLCC-4.7uF-50V
- CWLB1: renamed from CWLV1; value 4.7uF -> 100nF; footprint C1206 -> C0603; MPN MLCC-4.7uF-50V -> MLCC-100nF-50V
- CWLB2: renamed from DWLR; value US1M -> 4.7uF; footprint SMA -> C1206; symbol traction-r1:D -> traction-r1:C; LCSC C412437 -> CLASS; MPN US1M -> MLCC-4.7uF-50V
- CWLBL: renamed from DWLS1; value US1M -> 47pF; footprint SMA -> C0603; symbol traction-r1:D -> traction-r1:C; LCSC C412437 -> CLASS; MPN US1M -> MLCC-47pF-100V
- CWLE1: renamed from DWLS2; value US1M -> 10uF; footprint SMA -> C1206; symbol traction-r1:D -> traction-r1:C; LCSC C412437 -> CLASS; MPN US1M -> MLCC-10uF-25V
- CWLIN: renamed from DWLZ1; value BZT52-C18 -> 100nF; footprint SOD123 -> C0603; symbol traction-r1:D -> traction-r1:C; MPN BZT52-C18 -> MLCC-CLASS
- CWLV1: renamed from DWLZ2; value BZT52-C5V1 -> 4.7uF; footprint SOD123 -> C1206; symbol traction-r1:D -> traction-r1:C; MPN BZT52-C5V1 -> MLCC-4.7uF-50V
- CWSN: renamed from RWTS; value 100R -> 1uF; footprint R0603 -> FilmP27.5; symbol traction-r1:R -> traction-r1:C; MPN R0603-100R -> FILM-1uF-1200V
- CWTF: renamed from DWHSB; value BAT64-04 -> 2.2nF; footprint SOT23 -> C0603; symbol traction-r1:BAT64-04 -> traction-r1:C; MPN BAT64-04 -> MLCC-2.2nF-50V
- DB15: renamed from RPD4; value 10k -> SS34; footprint R0603 -> SMA; symbol traction-r1:R -> traction-r1:D; MPN R0603-10k -> SS34
- DFHA: renamed from RFHFB2; value 15k -> US1M; footprint R0603 -> SMA; symbol traction-r1:R -> traction-r1:D; LCSC CLASS -> C412437; MPN R0603-1% -> US1M
- DFHG: renamed from RFHG; value 10R -> PMEG4010EH; footprint R0603 -> SOD123; symbol traction-r1:R -> traction-r1:D; LCSC CLASS -> C282566; MPN R0603-CLASS -> PMEG4010EH
- DFHSN: renamed from RFHGO; value 20R -> US1M; footprint R0603 -> SMA; symbol traction-r1:R -> traction-r1:D; LCSC CLASS -> C412437; MPN R0603-CLASS -> US1M
- DFLA: renamed from RFLG; value 10R -> US1M; footprint R0603 -> SMA; symbol traction-r1:R -> traction-r1:D; LCSC CLASS -> C412437; MPN R0603-CLASS -> US1M
- DFLG: renamed from RFLGO; value 20R -> PMEG4010EH; footprint R0603 -> SOD123; symbol traction-r1:R -> traction-r1:D; LCSC CLASS -> C282566; MPN R0603-CLASS -> PMEG4010EH
- DFLSN: renamed from RFLGS; value 51k -> US1M; footprint R0603 -> SMA; symbol traction-r1:R -> traction-r1:D; LCSC CLASS -> C412437; MPN R0603-CLASS -> US1M
- DRH: renamed from FL1; value MF-LSMF300/24X-2 -> NRVBAF360T3G; footprint PTC2920 -> SMA-flat; symbol traction-r1:F -> traction-r1:D; LCSC C719172 -> CLASS; MPN MF-LSMF300/24X-2 -> NRVBAF360T3G
- DRL: renamed from CB15C; value 10nF -> NRVBAF360T3G; footprint C0603 -> SMA-flat; symbol traction-r1:C -> traction-r1:D; MPN MLCC-CLASS -> NRVBAF360T3G
- DTVH: renamed from LFL1; value FB-120R-3A -> TPSMC24CA; footprint FB1206 -> SMC; symbol traction-r1:L -> traction-r1:D; LCSC CLASS -> C1975284; MPN FB-120R-3A -> TPSMC24CA
- DTVL: renamed from CB15I; value 10uF -> TPSMC24CA; footprint C1210 -> SMC; symbol traction-r1:C -> traction-r1:D; LCSC CLASS -> C1975284; MPN MLCC-10uF-50V -> TPSMC24CA
- DUHSB: renamed from DUHZ1; value BZT52-C18 -> BAT64-04; footprint SOD123 -> SOT23; MPN BZT52-C18 -> BAT64-04
- DUHZ1: renamed from DUHZ2; value BZT52-C5V1 -> BZT52-C18; MPN BZT52-C5V1 -> BZT52-C18
- DUHZ2: renamed from RUHBL; value 5.1k -> BZT52-C5V1; footprint R0805 -> SOD123; symbol traction-r1:R -> traction-r1:D; MPN R0805-4k99 -> BZT52-C5V1
- DULS2: renamed from DULZ1; value BZT52-C18 -> US1M; footprint SOD123 -> SMA; LCSC CLASS -> C412437; MPN BZT52-C18 -> US1M
- DULSB: renamed from DULZ2; value BZT52-C5V1 -> BAT64-04; footprint SOD123 -> SOT23; MPN BZT52-C5V1 -> BAT64-04
- DULZ1: renamed from RULBL; value 5.1k -> BZT52-C18; footprint R0805 -> SOD123; symbol traction-r1:R -> traction-r1:D; MPN R0805-4k99 -> BZT52-C18
- DULZ2: renamed from RULDS; value 100R -> BZT52-C5V1; footprint R0805 -> SOD123; symbol traction-r1:R -> traction-r1:D; MPN R0805-100R -> BZT52-C5V1
- DVHS1: renamed from DVHZ1; value BZT52-C18 -> US1M; footprint SOD123 -> SMA; LCSC CLASS -> C412437; MPN BZT52-C18 -> US1M
- DVHS2: renamed from DVHZ2; value BZT52-C5V1 -> US1M; footprint SOD123 -> SMA; LCSC CLASS -> C412437; MPN BZT52-C5V1 -> US1M
- DVHSB: renamed from RVHBL; value 5.1k -> BAT64-04; footprint R0805 -> SOT23; symbol traction-r1:R -> traction-r1:D; MPN R0805-4k99 -> BAT64-04
- DVHZ1: renamed from RVHDS; value 100R -> BZT52-C18; footprint R0805 -> SOD123; symbol traction-r1:R -> traction-r1:D; MPN R0805-100R -> BZT52-C18
- DVHZ2: renamed from RVHGS; value 10k -> BZT52-C5V1; footprint R0805 -> SOD123; symbol traction-r1:R -> traction-r1:D; MPN R0805-10k -> BZT52-C5V1
- DVLR: renamed from DVLZ1; value BZT52-C18 -> US1M; footprint SOD123 -> SMA; LCSC CLASS -> C412437; MPN BZT52-C18 -> US1M
- DVLS1: renamed from DVLZ2; value BZT52-C5V1 -> US1M; footprint SOD123 -> SMA; LCSC CLASS -> C412437; MPN BZT52-C5V1 -> US1M
- DVLS2: renamed from RVLBL; value 5.1k -> US1M; footprint R0805 -> SMA; symbol traction-r1:R -> traction-r1:D; LCSC CLASS -> C412437; MPN R0805-4k99 -> US1M
- DVLSB: renamed from RVLDS; value 100R -> BAT64-04; footprint R0805 -> SOT23; symbol traction-r1:R -> traction-r1:D; MPN R0805-100R -> BAT64-04
- DVLZ1: renamed from RVLGS; value 10k -> BZT52-C18; footprint R0805 -> SOD123; symbol traction-r1:R -> traction-r1:D; MPN R0805-10k -> BZT52-C18
- DVLZ2: renamed from RVLMC; value 0R -> BZT52-C5V1; footprint R0805 -> SOD123; symbol traction-r1:R -> traction-r1:D; MPN R0805-0R -> BZT52-C5V1
- DVTP: renamed from RVTS; value 100R -> PESD5V0U1UA; footprint R0603 -> SOD323; symbol traction-r1:R -> traction-r1:D; MPN R0603-100R -> PESD5V0U1UA
- DWHR: renamed from DWHZ2; value BZT52-C5V1 -> US1M; footprint SOD123 -> SMA; LCSC CLASS -> C412437; MPN BZT52-C5V1 -> US1M
- DWHS1: renamed from RWHBL; value 5.1k -> US1M; footprint R0805 -> SMA; symbol traction-r1:R -> traction-r1:D; LCSC CLASS -> C412437; MPN R0805-4k99 -> US1M
- DWHS2: renamed from RWHDS; value 100R -> US1M; footprint R0805 -> SMA; symbol traction-r1:R -> traction-r1:D; LCSC CLASS -> C412437; MPN R0805-100R -> US1M
- DWHSB: renamed from RWHGS; value 10k -> BAT64-04; footprint R0805 -> SOT23; symbol traction-r1:R -> traction-r1:D; MPN R0805-10k -> BAT64-04
- DWHZ1: renamed from RWHMC; value 0R -> BZT52-C18; footprint R0805 -> SOD123; symbol traction-r1:R -> traction-r1:D; MPN R0805-0R -> BZT52-C18
- DWHZ2: renamed from RWHOFF; value 1R -> BZT52-C5V1; footprint R2512 -> SOD123; symbol traction-r1:R -> traction-r1:D; MPN R2512-1R0-2W -> BZT52-C5V1
- DWLR: renamed from RWLBL; value 5.1k -> US1M; footprint R0805 -> SMA; symbol traction-r1:R -> traction-r1:D; LCSC CLASS -> C412437; MPN R0805-4k99 -> US1M
- DWLS1: renamed from RWLDS; value 100R -> US1M; footprint R0805 -> SMA; symbol traction-r1:R -> traction-r1:D; LCSC CLASS -> C412437; MPN R0805-100R -> US1M
- DWLS2: renamed from RWLGS; value 10k -> US1M; footprint R0805 -> SMA; symbol traction-r1:R -> traction-r1:D; LCSC CLASS -> C412437; MPN R0805-10k -> US1M
- DWLSB: renamed from RWLMC; value 0R -> BAT64-04; footprint R0805 -> SOT23; symbol traction-r1:R -> traction-r1:D; MPN R0805-0R -> BAT64-04
- DWLZ1: renamed from RWLOFF; value 1R -> BZT52-C18; footprint R2512 -> SOD123; symbol traction-r1:R -> traction-r1:D; MPN R2512-1R0-2W -> BZT52-C18
- DWLZ2: renamed from RWLON; value 1.5R -> BZT52-C5V1; footprint R2512 -> SOD123; symbol traction-r1:R -> traction-r1:D; MPN R2512-1R5-2W -> BZT52-C5V1
- DWTP: renamed from UWHG; value NSI6611A-Q1 -> PESD5V0U1UA; footprint SOIC16W -> SOD323; symbol traction-r1:NSI6611A-Q1 -> traction-r1:D; LCSC C7470934 -> CLASS; MPN NSI6611A-Q1 -> PESD5V0U1UA
- FH1: renamed from UGDL; value NCV4276CDT50RKG -> MF-LSMF300/24X-2; footprint DPAK -> PTC2920; symbol traction-r1:NCV4276CDT50RKG -> traction-r1:F; LCSC CLASS -> C719172; MPN NCV4276CDT50RKG -> MF-LSMF300/24X-2
- FL1: renamed from CB15O1; value 22uF -> MF-LSMF300/24X-2; footprint C1210 -> PTC2920; symbol traction-r1:C -> traction-r1:F; LCSC CLASS -> C719172; MPN MLCC-22uF-25V -> MF-LSMF300/24X-2
- JIC: renamed from RPD9; value 10k -> MICROFIT3-40; footprint R0603 -> MicroFit40; symbol traction-r1:R -> traction-r1:MICROFIT3-40; MPN R0603-10k -> MICROFIT3-40
- JMV: renamed from DVHSB; value BAT64-04 -> STUD-M8; footprint SOT23 -> StudM8; symbol traction-r1:BAT64-04 -> traction-r1:TERM_1; MPN BAT64-04 -> STUD-M8
- JMW: renamed from CWHB1; value 100nF -> STUD-M8; footprint C0603 -> StudM8; symbol traction-r1:C -> traction-r1:TERM_1; MPN MLCC-100nF-50V -> STUD-M8
- LB15: renamed from RPD5; value 10k -> IND-10uH-3A; footprint R0603 -> IND6x6; symbol traction-r1:R -> traction-r1:L; MPN R0603-10k -> IND-10uH-3A
- LFH1: renamed from C5G1; value 1uF -> FB-120R-3A; footprint C1206 -> FB1206; symbol traction-r1:C -> traction-r1:L; MPN MLCC-10uF-25V -> FB-120R-3A
- LFL1: renamed from CB15O2; value 22uF -> FB-120R-3A; footprint C1210 -> FB1206; symbol traction-r1:C -> traction-r1:L; MPN MLCC-22uF-25V -> FB-120R-3A
- MODV: renamed from CVTF; value 2.2nF -> HCS600FH120D3C1; footprint C0603 -> EconoDUAL3; symbol traction-r1:C -> traction-r1:HCS600FH120D3C1; MPN MLCC-2.2nF-50V -> HCS600FH120D3C1
- MODW: renamed from JMW; value STUD-M8 -> HCS600FH120D3C1; footprint StudM8 -> EconoDUAL3; symbol traction-r1:TERM_1 -> traction-r1:HCS600FH120D3C1; MPN STUD-M8 -> HCS600FH120D3C1
- PS5B: renamed from RASCG; value 2.2k -> ISO5V-RFC-6K; footprint R0603 -> SIP7; symbol traction-r1:R -> traction-r1:ISO5V-RFC-6K; MPN R0603-2k2 -> ISO5V-RFC-6K
- PS5C: renamed from RASCL; value 470R -> ISO5V-RFC-6K; footprint R0603 -> SIP7; symbol traction-r1:R -> traction-r1:ISO5V-RFC-6K; MPN R0603-470R -> ISO5V-RFC-6K
- PSASC: renamed from CLVH2; value 4.7uF -> QA01C-18; footprint C1206 -> SIP7; symbol traction-r1:C -> traction-r1:QA01C-18; MPN MLCC-4.7uF-50V -> QA01C-18
- QFH: renamed from UFH; value UCC28C40DR -> BUK9Y14-80E; footprint SOP8 -> LFPAK56; symbol traction-r1:UCC28C40DR -> traction-r1:BUK9Y14-80E; LCSC CLASS -> C86732; MPN UCC28C40DR -> BUK9Y14-80E
- QFHE1: renamed from CFHA; value 4.7uF -> 2N7002; footprint C1206 -> SOT23; symbol traction-r1:C -> traction-r1:2N7002; LCSC CLASS -> C8545; MPN MLCC-4.7uF-50V -> 2N7002
- QFHE2: renamed from CFHCF; value 47pF -> 2N7002; footprint C0603 -> SOT23; symbol traction-r1:C -> traction-r1:2N7002; LCSC CLASS -> C8545; MPN MLCC-CLASS -> 2N7002
- QFL: renamed from CFLA; value 4.7uF -> BUK9Y14-80E; footprint C1206 -> LFPAK56; symbol traction-r1:C -> traction-r1:BUK9Y14-80E; LCSC CLASS -> C86732; MPN MLCC-4.7uF-50V -> BUK9Y14-80E
- QFLE1: renamed from CFLCF; value 47pF -> 2N7002; footprint C0603 -> SOT23; symbol traction-r1:C -> traction-r1:2N7002; LCSC CLASS -> C8545; MPN MLCC-CLASS -> 2N7002
- QFLE2: renamed from CFLCO; value 22nF -> 2N7002; footprint C0603 -> SOT23; symbol traction-r1:C -> traction-r1:2N7002; LCSC CLASS -> C8545; MPN MLCC-CLASS -> 2N7002
- RASCG: renamed from FH1; value MF-LSMF300/24X-2 -> 2.2k; footprint PTC2920 -> R0603; symbol traction-r1:F -> traction-r1:R; LCSC C719172 -> CLASS; MPN MF-LSMF300/24X-2 -> R0603-2k2
- RASCL: renamed from LFH1; value FB-120R-3A -> 470R; footprint FB1206 -> R0603; symbol traction-r1:L -> traction-r1:R; MPN FB-120R-3A -> R0603-470R
- RASCPD: renamed from CLVL1; value 4.7uF -> 10k; footprint C1206 -> R0603; symbol traction-r1:C -> traction-r1:R; MPN MLCC-4.7uF-50V -> R0603-10k
- RB15F1: renamed from RPD6; value 10k -> 110k; MPN R0603-10k -> R0603-1%
- RB15F2: renamed from RPD7; value 10k -> 9.53k; MPN R0603-10k -> R0603-1%
- RB15Q: renamed from RPD8; value 10k -> 80.6k; MPN R0603-10k -> R0603-CLASS
- RFHCS: renamed from RFHGS; value 51k -> 330m; footprint R0603 -> R1210; MPN R0603-CLASS -> R1210-0R33-0.75W
- RFHEN: renamed from RFHRT; value 10k -> 100k
- RFHFB1: renamed from RFHSI; value 100R -> 56k; MPN R0603-CLASS -> R0603-1%
- RFHFB2: renamed from RFHSN; value 100R -> 15k; footprint R0805 -> R0603; MPN R0805-100R -> R0603-1%
- RFHG: renamed from RFHST; value 4.7k -> 10R
- RFHGO: renamed from ZFHG; value BZT52-C5V6 -> 20R; footprint SOD123 -> R0603; symbol traction-r1:D -> traction-r1:R; MPN BZT52-C5V6 -> R0603-CLASS
- RFHGS: renamed from QFL; value BUK9Y14-80E -> 51k; footprint LFPAK56 -> R0603; symbol traction-r1:BUK9Y14-80E -> traction-r1:R; LCSC C86732 -> CLASS; MPN BUK9Y14-80E -> R0603-CLASS
- RFHRT: renamed from QFLE1; value 2N7002 -> 10k; footprint SOT23 -> R0603; symbol traction-r1:2N7002 -> traction-r1:R; LCSC C8545 -> CLASS; MPN 2N7002 -> R0603-CLASS
- RFHSI: renamed from QFLE2; value 2N7002 -> 100R; footprint SOT23 -> R0603; symbol traction-r1:2N7002 -> traction-r1:R; LCSC C8545 -> CLASS; MPN 2N7002 -> R0603-CLASS
- RFHSN: renamed from TFL1; value VGT12EEM-200S1A4 -> 100R; footprint XfmrEE12 -> R0805; symbol traction-r1:VGT12EEM-200S1A4 -> traction-r1:R; MPN VGT12EEM-200S1A4 -> R0805-100R
- RFHST: renamed from TFL2; value VGT12EEM-200S1A4 -> 4.7k; footprint XfmrEE12 -> R0603; symbol traction-r1:VGT12EEM-200S1A4 -> traction-r1:R; MPN VGT12EEM-200S1A4 -> R0603-CLASS
- RFLCS: renamed from RFLRT; value 10k -> 330m; footprint R0603 -> R1210; MPN R0603-CLASS -> R1210-0R33-0.75W
- RFLEN: renamed from RFLSI; value 100R -> 100k
- RFLFB1: renamed from RFLSN; value 100R -> 56k; footprint R0805 -> R0603; MPN R0805-100R -> R0603-1%
- RFLFB2: renamed from RFLST; value 4.7k -> 15k; MPN R0603-CLASS -> R0603-1%
- RFLG: renamed from ZFLG; value BZT52-C5V6 -> 10R; footprint SOD123 -> R0603; symbol traction-r1:D -> traction-r1:R; MPN BZT52-C5V6 -> R0603-CLASS
- RFLGO: renamed from UIVDC; value AMC1311BDWVR -> 20R; footprint SOIC8W -> R0603; symbol traction-r1:AMC1311BDWVR -> traction-r1:R; LCSC C456277 -> CLASS; MPN AMC1311BDWVR -> R0603-CLASS
- RFLGS: renamed from CVDDF; value 1nF -> 51k; footprint C0603 -> R0603; symbol traction-r1:C -> traction-r1:R; MPN MLCC-1nF-50V -> R0603-CLASS
- RFLRT: renamed from RVDD1; value 470k -> 10k; footprint R1206 -> R0603; MPN R1206-470k-TF -> R0603-CLASS
- RFLSI: renamed from RVDD2; value 470k -> 100R; footprint R1206 -> R0603; MPN R1206-470k-TF -> R0603-CLASS
- RFLSN: renamed from RVDD3; value 470k -> 100R; footprint R1206 -> R0805; MPN R1206-470k-TF -> R0805-100R
- RFLST: renamed from RVDD4; value 470k -> 4.7k; footprint R1206 -> R0603; MPN R1206-470k-TF -> R0603-CLASS
- RGDLE: renamed from RB15F2; value 9.53k -> 100k; MPN R0603-1% -> R0603-CLASS
- RUHBL: renamed from RUHDS; value 100R -> 5.1k; MPN R0805-100R -> R0805-4k99
- RUHDS: renamed from RUHGS; value 10k -> 100R; MPN R0805-10k -> R0805-100R
- RUHGS: renamed from RUHMC; value 0R -> 10k; MPN R0805-0R -> R0805-10k
- RUHMC: renamed from RUHOFF; value 1R -> 0R; footprint R2512 -> R0805; MPN R2512-1R0-2W -> R0805-0R
- RUHOFF: renamed from RUHON; value 1.5R -> 1R; MPN R2512-1R5-2W -> R2512-1R0-2W
- RUHON: renamed from RUHPD; value 1M -> 1.5R; footprint R1206 -> R2512; MPN HV73-1M-1206 -> R2512-1R5-2W
- RUHPD: renamed from ZUHV; value BZT52-C5V1 -> 1M; footprint SOD123 -> R1206; symbol traction-r1:D -> traction-r1:R; MPN BZT52-C5V1 -> HV73-1M-1206
- RULBL: renamed from RULGS; value 10k -> 5.1k; MPN R0805-10k -> R0805-4k99
- RULDS: renamed from RULMC; value 0R -> 100R; MPN R0805-0R -> R0805-100R
- RULGS: renamed from RULOFF; value 1R -> 10k; footprint R2512 -> R0805; MPN R2512-1R0-2W -> R0805-10k
- RULMC: renamed from RULON; value 1.5R -> 0R; footprint R2512 -> R0805; MPN R2512-1R5-2W -> R0805-0R
- RULOFF: renamed from RULPD; value 1M -> 1R; footprint R1206 -> R2512; MPN HV73-1M-1206 -> R2512-1R0-2W
- RULON: renamed from ZULV; value BZT52-C5V1 -> 1.5R; footprint SOD123 -> R2512; symbol traction-r1:D -> traction-r1:R; MPN BZT52-C5V1 -> R2512-1R5-2W
- RULPD: renamed from MODV; value HCS600FH120D3C1 -> 1M; footprint EconoDUAL3 -> R1206; symbol traction-r1:HCS600FH120D3C1 -> traction-r1:R; MPN HCS600FH120D3C1 -> HV73-1M-1206
- RVBD1: renamed from PS5C; value ISO5V-RFC-6K -> 470k; footprint SIP7 -> R1206; symbol traction-r1:ISO5V-RFC-6K -> traction-r1:R; MPN ISO5V-RFC-6K -> R1206-470k-TF
- RVBD2: renamed from C5B1; value 1uF -> 470k; footprint C0603 -> R1206; symbol traction-r1:C -> traction-r1:R; MPN MLCC-1uF-25V -> R1206-470k-TF
- RVBD3: renamed from C5B2; value 100nF -> 470k; footprint C0603 -> R1206; symbol traction-r1:C -> traction-r1:R; MPN MLCC-1uF-25V -> R1206-470k-TF
- renumbered CWHV1 to CWHB2, DULS1 to DULR, DULS2 to DULS1, DVHS2 to DVHR, RVBD1 to RVDD2, RVBD2 to RVDD3, RVBD3 to RVDD4, RVBD4 to RVDD5, RVBD5 to RVDD6
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Connections:
- net labels added: B15FQ, B15SS, FCL_H, FCL_L, GDL_ON
- wire segments 762 -> 790
Other:
- note added: "+ 12 more"
- note added: "rev A.4 - 24 sections - 285 components"
- note removed: "+ 10 more"
- note removed: "4 FS1B strap -> LS ASC latch (HS strapped OFF)"
- note removed: "5 flyback EN = MCU OR FS26-GPIO1 (ASC gate power)"
- note removed: "rev A.3 - 24 sections - 274 components"
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
Commit message: Rev A.4.1: second review round — 5 confirmed defects fixed (F47-F51)
- F47 AMC1311 real pins 2=IN/3=SHTDN (both VDC channels had them
  swapped: analog inputs grounded, SHTDN on the divider tap)
- F48 FS26 TRKIN is the VREF regulator's input supply -> VPRE
  (was grounded as an "unused tracker input"; VREF5 had no source)
- F49 TPS55340 pin 5 is SYNC (7V abs), not a second VIN -> DGND
- F50 FS26 caps to DS minimums: CVBOS 4.7uF, CSB6 4.7uF, CSB5 2.2uF
  (VREF COUT 1.1-3.3uF eff - third value found in the same audit)
- F51 V15 protective post-regulator NCV4276C-ADJ 40V/0.4A: boost
  pass-through (24V jump start / ~33V clamped load dump) can no longer
  reach the QA01C 13.5-16.5V window; boost output renamed V15B
- ASC/fault-latch interplay documented per NSI6611 DS (ASC overrides
  input side; DESAT + VCC2-UVLO outrank ASC)
- all five PDFs regenerate from one release (stale standalone A.3
  exports superseded); ERC gains A.4.1 assertions

Gates: 1674/1674 pins, ERC 769/0, design-verify 64P/3W/0F,
BOM Rs.70,074 @1k, 583 components, 184 lines.

Co-Authored-By: Claude Fable 5 <noreply@anthropic.com>
Parts:
- added RPD6, RPD7, RPD8, RPD9: 10k, R0603, symbol traction-r1:R
- CB15C: renamed from CB15I; value 10uF -> 10nF; footprint C1210 -> C0603; MPN MLCC-10uF-50V -> MLCC-CLASS
- CB15I: renamed from CB15O1; value 22uF -> 10uF; MPN MLCC-22uF-25V -> MLCC-10uF-50V
- CB15O2: renamed from CB15S; value 47nF -> 22uF; footprint C0603 -> C1210; MPN MLCC-CLASS -> MLCC-22uF-25V
- CB15S: renamed from DB15; value SS34 -> 47nF; footprint SMA -> C0603; symbol traction-r1:D -> traction-r1:C; MPN SS34 -> MLCC-CLASS
- CLD15: renamed from LB15; value IND-10uH-3A -> 4.7uF; footprint IND6x6 -> C0603; symbol traction-r1:L -> traction-r1:C; MPN IND-10uH-3A -> MLCC-CLASS
- DB15: renamed from RB15F1; value 110k -> SS34; footprint R0603 -> SMA; symbol traction-r1:R -> traction-r1:D; MPN R0603-1% -> SS34
- JIC: renamed from RPD2; value 10k -> MICROFIT3-40; footprint R0603 -> MicroFit40; symbol traction-r1:R -> traction-r1:MICROFIT3-40; MPN R0603-10k -> MICROFIT3-40
- LB15: renamed from RB15F2; value 9.53k -> IND-10uH-3A; footprint R0603 -> IND6x6; symbol traction-r1:R -> traction-r1:L; MPN R0603-1% -> IND-10uH-3A
- RB15F1: renamed from RB15Q; value 80.6k -> 110k; MPN R0603-CLASS -> R0603-1%
- RB15F2: renamed from JIC; value MICROFIT3-40 -> 9.53k; footprint MicroFit40 -> R0603; symbol traction-r1:MICROFIT3-40 -> traction-r1:R; MPN MICROFIT3-40 -> R0603-1%
- RB15Q: renamed from RPD0; value 10k -> 80.6k; MPN R0603-10k -> R0603-CLASS
- RLD1: renamed from RPD1; value 10k -> 49.9k; MPN R0603-10k -> R0603-CLASS
- RLD2: renamed from RPD10; MPN R0603-10k -> R0603-CLASS
- ULDO15: renamed from CB15C; value 10nF -> NCV4276CADJDTRKG; footprint C0603 -> DPAK5; symbol traction-r1:C -> traction-r1:NCV4276CADJDTRKG; MPN MLCC-CLASS -> NCV4276CADJDTRKG
- renumbered CB15O2 to CB15O1, RPD3 to RPD0, RPD4 to RPD1, RPD5 to RPD10, RPD6 to RPD2, RPD7 to RPD3, RPD8 to RPD4, RPD9 to RPD5
Connections:
- net labels added: V15B, V15VA
- wire segments 790 -> 801
Other:
- note added: "rev A.4.1 - 24 sections - 289 components"
- note removed: "rev A.4 - 24 sections - 285 components"
- moved on the sheet: CB15C, CB15I, CB15O1, CB15O2, CLD15, RB15F1, RB15Q, RLD1, RLD2, RPD0, RPD1, RPD10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

Commit message: Rev A.4.2: third review round — 6 confirmed defects fixed (F52-F57)
- F52 FS26 buck passives to Table-106 selections: LCOR 2.2uH
  (CORE_LSEL_OTP=0x02; 4.7uH matched no listed value), V15S COUT
  2x22uF (~32uF eff vs 20-100 spec), CBTC 47nF, CBTP 22nF per
  CBOOT_PRE, VPRE COUT 2x22uF, CIN 22uF; effective-capacitance rows
  (bias/tol/temp derating) added to design-verify. VREF5 judged as a
  rail (CSB5+CMA1+CMA2 ~2.2uF eff, inside 1.1-3.3) per reviewer.
- F53 ACT45B CAN chokes: real windings are pins 1-4 and 2-3 (TDK
  circuit diagram) - both ports had transceiver CANH coupled onto
  external CANL; remapped, ERC asserts end-to-end pairing
- F54 ULDO15 completed: 220pF feed-forward across the 49.9k leg
  (fz 14.5kHz, onsemi 11-18kHz window), COUT 22uF
- F55 UEXD (ALM2402, 18V abs/16V rec) off raw VBATC -> behind ULDOEX
  12.1V (NCV4276C-ADJ); 24V jump start can no longer reach it
- F56 flyback switch BUK9Y14-80E (logic-level, VGS +/-10V DC) was
  outside abs-max at the 11.8V drive, masked by a 5.6V zener that
  conducted ~0.29A through every ON interval (~0.4W each). Now
  BUK7Y14-80E (standard-level +/-20V, same LFPAK56); zener repurposed
  to a dark 15V protective clamp
- F57 ordering code NCV4276CDTADJRKG (DT/ADJ were transposed)
- ASC-with-VCC1-open qualification documented (DESAT unavailable;
  double-fault given KL30-held V5GD) + IGN_SNS ADC disposition

Gates: 1691/1691 pins, ERC 779/0, design-verify 73P/3W/0F,
BOM Rs.70,090 @1k, 590 components, 192 lines.

Co-Authored-By: Claude Fable 5 <noreply@anthropic.com>
Parts:
- added RPD9: 10k, R0603, symbol traction-r1:R
- CLD15: value 4.7uF -> 22uF
- CLDC: renamed from DB15; value SS34 -> 220pF; footprint SMA -> C0603; symbol traction-r1:D -> traction-r1:C; MPN SS34 -> MLCC-CLASS
- DB15: renamed from LB15; value IND-10uH-3A -> SS34; footprint IND6x6 -> SMA; symbol traction-r1:L -> traction-r1:D; MPN IND-10uH-3A -> SS34
- JIC: renamed from RPD0; value 10k -> MICROFIT3-40; footprint R0603 -> MicroFit40; symbol traction-r1:R -> traction-r1:MICROFIT3-40; MPN R0603-10k -> MICROFIT3-40
- LB15: renamed from RB15F1; value 110k -> IND-10uH-3A; footprint R0603 -> IND6x6; symbol traction-r1:R -> traction-r1:L; MPN R0603-1% -> IND-10uH-3A
- QFH, QFL: value BUK9Y14-80E -> BUK7Y14-80E; symbol traction-r1:BUK9Y14-80E -> traction-r1:BUK7Y14-80E; MPN BUK9Y14-80E -> BUK7Y14-80E
- RB15F1: renamed from RB15F2; value 9.53k -> 110k
- RB15F2: renamed from RB15Q; value 80.6k -> 9.53k; MPN R0603-CLASS -> R0603-1%
- RB15Q: renamed from RLD1; value 49.9k -> 80.6k
- RLD1: renamed from RLD2; value 10k -> 49.9k
- RLD2: renamed from JIC; value MICROFIT3-40 -> 10k; footprint MicroFit40 -> R0603; symbol traction-r1:MICROFIT3-40 -> traction-r1:R; MPN MICROFIT3-40 -> R0603-CLASS
- ULDO15: value NCV4276CADJDTRKG -> NCV4276CDTADJRKG; symbol traction-r1:NCV4276CADJDTRKG -> traction-r1:NCV4276CDTADJRKG; MPN NCV4276CADJDTRKG -> NCV4276CDTADJRKG
- ZFHG, ZFLG: value BZT52-C5V6 -> BZT52-C15; MPN BZT52-C5V6 -> BZT52-C15
- renumbered RPD1 to RPD0, RPD10 to RPD1, RPD2 to RPD10, RPD3 to RPD2, RPD4 to RPD3, RPD5 to RPD4, RPD6 to RPD5, RPD7 to RPD6, RPD8 to RPD7, RPD9 to RPD8
Connections:
- wire segments 801 -> 803
Other:
- note added: "rev A.4.2 - 24 sections - 290 components"
- note removed: "+ 12 more"
- note removed: "1 lockstep S32K396 (ASIL-D core) runs torque path"
- note removed: "2 FS26 Q&A watchdog + monitors -> FS0B (no SW)"
- note removed: "3 FS0B AND MCU_EN -> all 6 driver EN = 3-ph open"
- note removed: "ASIL-D SAFETY CONCEPT + DC-LINK DISCHARGE VERIFICATION"
- note removed: "rev A.4.1 - 24 sections - 289 components"
- note removed: "safe state = 3-phase-open (ASC above overspeed); discharge vs ECE R100 / ISO 6469"
- moved on the sheet: CB15C, CB15I, CB15S, CLD15, RB15F1, RB15F2, RB15Q, RLD1, RPD0, RPD1, RPD10, RPD2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

Commit message: Rev A.4.3: fourth review round — LCOR reconciled, UB15 compensation (F58-F59)
- F58: LCOR netlist value became 2.2uH in A.4.2 but the parts-db class
  MPN kept printing IND-4.7uH-2A on the sheet and BOM - an assembler
  would fit the old part. MPN/desc now carry 2.2uH + the OTP pairing;
  value, sheet, BOM and CORE_LSEL_OTP=0x02 agree end-to-end.
- F59: TPS55340 COMP had only 10nF to ground (no zero; ~0deg screening
  phase margin in the CCM model). Series R3/C4 = 2k/100nF per TI
  8.2.1.2.11 + 470pF HF pole cap; RHPZ ~450kHz not limiting; measured
  Bode stays a bench gate.
- Narrative corrections per review: CBOOT_PRE 100nF was legal (Rev 6.1
  allows 22-100nF; 22nF kept as typ) - F52 log softened; VCC1 loss
  reclassified as a single initiating failure (UGDL open output) whose
  outcome is three-phase-open with ASC still commandable.

Gates: 1695/1695 pins, ERC 782/0, design-verify 75P/3W/0F,
BOM Rs.70,091 @1k, 592 components, 193 lines.

Co-Authored-By: Claude Fable 5 <noreply@anthropic.com>
Parts:
- added RPD8, RPD9: 10k, R0603, symbol traction-r1:R
- CB15C: value 10nF -> 470pF
- CB15CC: renamed from CB15I; value 10uF -> 100nF; footprint C1210 -> C0603; MPN MLCC-10uF-50V -> MLCC-CLASS
- CB15I: renamed from CB15O1; value 22uF -> 10uF; MPN MLCC-22uF-25V -> MLCC-10uF-50V
- CB15O2: renamed from CB15S; value 47nF -> 22uF; footprint C0603 -> C1210; MPN MLCC-CLASS -> MLCC-22uF-25V
- CB15S: renamed from CLD15; value 22uF -> 47nF
- CLD15: renamed from CLDC; value 220pF -> 22uF
- CLDC: renamed from DB15; value SS34 -> 220pF; footprint SMA -> C0603; symbol traction-r1:D -> traction-r1:C; MPN SS34 -> MLCC-CLASS
- DB15: renamed from LB15; value IND-10uH-3A -> SS34; footprint IND6x6 -> SMA; symbol traction-r1:L -> traction-r1:D; MPN IND-10uH-3A -> SS34
- JIC: renamed from RPD1; value 10k -> MICROFIT3-40; footprint R0603 -> MicroFit40; symbol traction-r1:R -> traction-r1:MICROFIT3-40; MPN R0603-10k -> MICROFIT3-40
- LB15: renamed from RB15F1; value 110k -> IND-10uH-3A; footprint R0603 -> IND6x6; symbol traction-r1:R -> traction-r1:L; MPN R0603-1% -> IND-10uH-3A
- RB15C: renamed from RB15F2; value 9.53k -> 2k; MPN R0603-1% -> R0603-CLASS
- RB15F1: renamed from RB15Q; value 80.6k -> 110k; MPN R0603-CLASS -> R0603-1%
- RB15F2: renamed from RLD1; value 49.9k -> 9.53k; MPN R0603-CLASS -> R0603-1%
- RB15Q: renamed from RLD2; value 10k -> 80.6k
- RLD1: renamed from JIC; value MICROFIT3-40 -> 49.9k; footprint MicroFit40 -> R0603; symbol traction-r1:MICROFIT3-40 -> traction-r1:R; MPN MICROFIT3-40 -> R0603-CLASS
- RLD2: renamed from RPD0; MPN R0603-10k -> R0603-CLASS
- renumbered CB15O2 to CB15O1, RPD10 to RPD0, RPD2 to RPD1, RPD3 to RPD10, RPD4 to RPD2, RPD5 to RPD3, RPD6 to RPD4, RPD7 to RPD5, RPD8 to RPD6, RPD9 to RPD7
Connections:
- net labels added: B15CZ
- wire segments 803 -> 807
Other:
- note added: "rev A.4.3 - 24 sections - 292 components"
- note removed: "rev A.4.2 - 24 sections - 290 components"
- moved on the sheet: CB15CC, CB15I, CB15O1, CB15O2, RB15C, RB15F1, RB15F2, RLD2, RPD0, RPD1, RPD10, RPD2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

Commit message: Rev A.4.4: round five — bind class MPNs to real parts, pin FS26 OTP config
No electrical change. Procurement closure of the review's remaining
generic identifiers, each verified against its manufacturer datasheet:

- LCOR -> Coilcraft XAL4020-222MEC (2.2uH molded, AEC-Q200; values
  read from the XAL4000 datasheet, now in docs/datasheets)
- LB15 + LSBC -> XAL4040-103MEC (one 10uH line item for both; LSBC
  pairing with FPRE_OTP=450kHz documented per the FS26 DS)
- PS5B/PS5C -> Murata MGJ2D150505SC (+5V output used) behind an
  explicit PO gate: verify reinforced-insulation characterization at
  850VDC working and the SIP-7 pin map before ordering
- RECOM R15P05S evaluated and REJECTED during binding: its 6.4kV is a
  1-second test voltage; IEC 62368-1 insulation grade is BASIC at
  250VACrms working - fails the 850V barrier rule. Rejection recorded
  in design-basis 11e and the BOM row so it cannot be substituted in.
- FS26 OTP configuration pinned as design-basis 8a table (VPRE 6.0V,
  FPRE 450kHz, CORE_LSEL=0x02, VCORE 1.5V, LDO1/2 3.3/5.0V, VMONEXT
  0.8V ref, TRK slots off, VBST disabled, WK2PD/IO2PD set) - the
  ordering step must match it; the family label alone is not evidence.

Gates unchanged: 1695/1695 pins, ERC 782/0, design-verify 75P/3W/0F,
sim-verify 18P/1W/0F. BOM Rs.70,934 @1k with real part prices.

Co-Authored-By: Claude Fable 5 <noreply@anthropic.com>
Parts:
- LB15: value IND-10uH-3A -> XAL4040-103MEC; footprint IND6x6 -> XAL4040; MPN IND-10uH-3A -> XAL4040-103MEC
- PS5B, PS5C: value ISO5V-RFC-6K -> MGJ2D150505SC; symbol traction-r1:ISO5V-RFC-6K -> traction-r1:MGJ2D150505SC; MPN ISO5V-RFC-6K -> MGJ2D150505SC
Other:
- note added: "rev A.4.4 - 24 sections - 292 components"
- note removed: "rev A.4.3 - 24 sections - 292 components"
Changed lines of the file:
@@
 Title "Traction Inverter 220 kW — Power board (3x EconoDUAL 3 SiC)"
 Date "2026-09-09"
-Rev "A.4.3"
+Rev "A.4.4"
 Comp "Traction Inverter 220 kW pk - Power (HV), sheet 1 of 4"
 Comment1 "Inverter = Power board + Cap bank busbar + bolt-on Discharge board (all HV) + Control card (LV); safe state holds with any link lost"
@@
 DC-LINK   -   1 section
 Text Notes 29110 22000 0    60   ~ 0
-rev A.4.3   -   24 sections   -   292 components
+rev A.4.4   -   24 sections   -   292 components
 Wire Notes Line
 	34650 18100 39100 18100
@@
 HV-SENSING / ISO-BIAS
 $Comp
-L traction-r1:ISO5V-RFC-6K PS5B
+L traction-r1:MGJ2D150505SC PS5B
 U 1 1 5E0000EB
 P 30400 13050
 F 0 "PS5B" H 30000 12750 50  0000 R CNN
-F 1 "ISO5V-RFC-6K" H 30000 13380 50  0000 R CNN
+F 1 "MGJ2D150505SC" H 30000 13380 50  0000 R CNN
 F 2 "SIP7" H 30400 13050 50  0001 C CNN
 F 3 "~" H 30400 13050 50  0001 C CNN
 F 4 "CLASS" H 30400 13050 50  0001 C CNN "LCSC"
-F 5 "ISO5V-RFC-6K" H 30400 13050 50  0001 C CNN "MPN"
+F 5 "MGJ2D150505SC" H 30400 13050 50  0001 C CNN "MPN"
 	1    30400 13050
 	1    0    0    -1
@@
 DGND
 $Comp
-L traction-r1:ISO5V-RFC-6K PS5C
+L traction-r1:MGJ2D150505SC PS5C
 U 1 1 5E0000EC
 P 30400 14800
 F 0 "PS5C" H 30000 14500 50  0000 R CNN
-F 1 "ISO5V-RFC-6K" H 30000 15130 50  0000 R CNN
+F 1 "MGJ2D150505SC" H 30000 15130 50  0000 R CNN
 F 2 "SIP7" H 30400 14800 50  0001 C CNN
 F 3 "~" H 30400 14800 50  0001 C CNN
 F 4 "CLASS" H 30400 14800 50  0001 C CNN "LCSC"
-F 5 "ISO5V-RFC-6K" H 30400 14800 50  0001 C CNN "MPN"
+F 5 "MGJ2D150505SC" H 30400 14800 50  0001 C CNN "MPN"
 	1    30400 14800
 	1    0    0    -1
@@
 P 40250 12150
 F 0 "LB15" H 40250 11990 50  0000 C CNN
-F 1 "IND-10uH-3A" H 40250 12320 50  0000 C CNN
-F 2 "IND6x6" H 40250 12150 50  0001 C CNN
+F 1 "XAL4040-103MEC" H 40250 12320 50  0000 C CNN
+F 2 "XAL4040" H 40250 12150 50  0001 C CNN
 F 3 "~" H 40250 12150 50  0001 C CNN
 F 4 "CLASS" H 40250 12150 50  0001 C CNN "LCSC"
-F 5 "IND-10uH-3A" H 40250 12150 50  0001 C CNN "MPN"
+F 5 "XAL4040-103MEC" H 40250 12150 50  0001 C CNN "MPN"
 	1    40250 12150
 	1    0    0    -1
