File: kicad5/traction/traction-power.sch (KiCad schematic (older format))
At the start: 292 parts

Commit message: Rev A.5: end-to-end documentation refresh + 3 defects the audit caught
Docs (every file rewritten to the released state, history kept as
labeled evidence):
- README: five stacked review paragraphs consolidated into one campaign
  table (F1-F62); new Simulation section with the S1-S7 results table
  and all five SVG plots; badges/stats/mermaids/DFM rows refreshed
  (UCC28C40, four-assembly build flow, 770669-1, sim badge, rev A.5)
- design-basis: gate-drive/LV sections describe the released circuit
  (UCC28C40+BUK7Y14+SMAJ13A clamp, boost->ULDO15 chain, MGJ2+QA01C
  bias set, QA01C +20/-4V note)
- dfm.md + cost-rollup.md rewritten (four assemblies, current tiers,
  76% module share, PO gates, banned-substitute rule)
- EXTRACTED-PARAMS: superseded sections replaced (BUK7Y14, winding
  dots, UCC28C40 UVLO), 10 new part sections, fresh 47-PDF archive
  index with evidence files labeled; SMAJ + TE-770669-1 datasheets
  added; wrong-part PDF from a mirror detected and discarded
- calculations/rev.mjs: single REV source imported by every generator
  (the stale-rev defect class is now structurally impossible)

Defects the audit caught and fixed:
- F60: JVEH was bound to TE 776231-1 "AMPSEAL 23" - its own TE drawing
  shows the 35-pos header (mates 776164). Rebound to 770669-1 (true
  23-pos, mates the 770680-1 plug); drawing archived.
- F61: QA01C DS row is +20/-4V (rails named V18*) - clamps verified
  for +20V; QDIS gate 19.5V vs +22 abs WARN row added.
- F62: the on-sheet ASIL-D + DISCHARGE panel had silently vanished
  from the power sheet as it grew through A.4.x. Placement now retries
  every void and extends the sheet if none fits; a power sheet without
  the panel REFUSES to build. Panel text refreshed (full DRV_EN chain,
  57s bleed, "never energize w/o the DISCHARGE BOARD fitted").

Gates: 1695/1695 pins, ERC 782/0, design-verify 75P/4W/0F, sim-verify
18P/1W/0F, BOM Rs.70,934. Power sheet 44.6x28.6 in (panel row added).

Co-Authored-By: Claude Fable 5 <noreply@ant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
Other:
- note added: "--- DISCHARGE ---"
- note added: "1 lockstep S32K396 (ASIL-D core) runs torque path"
- note added: "2 FS26 Q&A watchdog + monitors -> FS0B (no SW)"
- note added: "3 FS0B&MCU_EN&RDY&FLT-latch -> DRV_EN = 3-ph open"
- note added: "4 FS1B strap -> LS ASC latch (HS strapped OFF)"
- note added: "5 flyback EN = MCU OR FS26-GPIO1 (ASC gate power)"
- note added: "6 3x hall + sum(I)=0 plausibility (torque path)"
- note added: "7 2x isolated VDC senses, >5% mismatch = fault"
- note added: "8 DESAT per switch, ~1.5 us blanking, latching"
- note added: "9 HVIL open = VDDIO/2 signature -> discharge"
- note added: "ACTIVE QDIS + 4x 470R 10W = 1.88k: 1.6 s to 60 V"
- note added: "ASIL-D SAFETY CONCEPT + DC-LINK DISCHARGE VERIFICATION"
- note added: "E = 116 J @850 V - 32 J/res worst (>=100 J rated)"
- note added: "PASSIVE 10x 27k 2512-2W (5s x 2p = 67.5k): 57 s to 60 V"
- note added: "RULE: never energize w/o the DISCHARGE BOARD fitted"
- note added: "VERIFY: MCU fires QDIS, watches BOTH VDC channels"
- note added: "rev A.5 - 24 sections - 292 components"
- note added: "safe state = 3-phase-open (ASC above overspeed); discharge vs ECE R100 / ISO 6469"
- note removed: "rev A.4.4 - 24 sections - 292 components"
Changed lines of the file:
@@
 EELAYER 30 0
 EELAYER END
-$Descr User 44600 22800
+$Descr User 44600 28550
 encoding utf-8
 Sheet 1 1
 Title "Traction Inverter 220 kW — Power board (3x EconoDUAL 3 SiC)"
 Date "2026-09-09"
-Rev "A.4.4"
+Rev "A.5"
 Comp "Traction Inverter 220 kW pk - Power (HV), sheet 1 of 4"
 Comment1 "Inverter = Power board + Cap bank busbar + bolt-on Discharge board (all HV) + Control card (LV); safe state holds with any link lost"
@@
 DC-LINK   -   1 section
 Text Notes 29110 22000 0    60   ~ 0
-rev A.4.4   -   24 sections   -   292 components
+rev A.5   -   24 sections   -   292 components
 Wire Notes Line
 	34650 18100 39100 18100
@@
 named connector/stud/tab (see INTERBOARD LINKS, design basis)
 Wire Notes Line
+	1400 22900 10050 22900
+Wire Notes Line
+	10050 22900 10050 26700
+Wire Notes Line
+	10050 26700 1400 26700
+Wire Notes Line
+	1400 26700 1400 22900
+Text Notes 1460 23060 0    79   ~ 16
+ASIL-D SAFETY CONCEPT + DC-LINK DISCHARGE VERIFICATION
+Text Notes 1460 23320 0    60   ~ 0
+safe state = 3-phase-open (ASC above overspeed); discharge vs ECE R100 / ISO 6469
+Text Notes 1450 23750 0    60   ~ 0
+1 lockstep S32K396 (ASIL-D core) runs torque path
+Text Notes 1450 24050 0    60   ~ 0
+2 FS26 Q&A watchdog + monitors -> FS0B (no SW)
+Text Notes 1450 24350 0    60   ~ 0
+3 FS0B&MCU_EN&RDY&FLT-latch -> DRV_EN = 3-ph open
+Text Notes 1450 24650 0    60   ~ 0
+4 FS1B strap -> LS ASC latch (HS strapped OFF)
+Text Notes 1450 24950 0    60   ~ 0
+5 flyback EN = MCU OR FS26-GPIO1 (ASC gate power)
+Text Notes 1450 25250 0    60   ~ 0
+6 3x hall + sum(I)=0 plausibility (torque path)
+Text Notes 1450 25550 0    60   ~ 0
+7 2x isolated VDC senses, >5% mismatch = fault
+Text Notes 1450 25850 0    60   ~ 0
+8 DESAT per switch, ~1.5 us blanking, latching
+Text Notes 5650 23750 0    60   ~ 0
+9 HVIL open = VDDIO/2 signature -> discharge
+Text Notes 5650 24050 0    60   ~ 0
+--- DISCHARGE ---
+Text Notes 5650 24350 0    60   ~ 0
+PASSIVE 10x 27k 2512-2W (5s x 2p = 67.5k): 57 s to 60 V
+Text Notes 5650 24650 0    60   ~ 0
+ACTIVE QDIS + 4x 470R 10W = 1.88k: 1.6 s to 60 V
+Text Notes 5650 24950 0    60   ~ 0
+E = 116 J @850 V - 32 J/res worst (>=100 J rated)
+Text Notes 5650 25250 0    60   ~ 0
+VERIFY: MCU fires QDIS, watches BOTH VDC channels
+Text Notes 5650 25550 0    60   ~ 0
+RULE: never energize w/o the DISCHARGE BOARD fitted
+Wire Notes Line
 	500 500 4100 500

Commit message: Rev A.6: review round 6 response, one platform / four SKUs, N7-N9
External review round 6 (46 findings, R-F01..R-F46) was verified finding by
finding and classified in docs/review-A6-disposition.md (+ .csv): 20
Confirmed, 9 Already Fixed, 6 Firmware Handled, 5 Not Applicable,
6 Improvement Recommended. Repo findings F63-F76 are in the verification log.

Hardware (+Rs31/unit, all SKUs unless noted):
- SiC gate 3.3/6.8 ohm; IGBT 1.0/1.0 ohm + 82 pF DESAT blanking (HCG600
  short-circuit rating is 6 us, not 10)
- gate-power flyback start: 2.2 k + 47 uF VDD + 18 V VDD zener (UCC28C40 has
  0.4 V UVLO hysteresis and no clamp); IGBT builds use RT 8.2 k for margin
- fault latch: 10 k / 3.3 nF delay + 15 nF clear one-shot (NSI6611 FLT clears
  only on an EN rising edge, so a fault-dominant latch would deadlock)
- bleeder 2 x 6 x 22 k; HW_ID identity (harness pin 40) and VOFS to the MCU;
  resolver shields to DGND

Platform: one set of PCBs, four SKUs (8XX SiC/IGBT, 4XX IGBT/SiC).
- SKU rows in parts-db, selected by BOM_VARIANT in bom-gen; bom-gen now fails
  on any value/MPN mismatch
- shared calculations/loss-model.mjs
- docs/firmware-contract.md: FW-01..21, safe-state matrix, regen ownership
  (section 4b)
- docs/variants.md: business case

New Road findings:
- N7: LEM HC5FW 900-S/SP1 is a reduced-insulation part, so the phase busbar
  needs a rated sleeve
- N8: TLP152 is UL1577-only; order the (V4) VDE option or an SO6L part
- N9: FW-06 overvoltage response tightened from 100 us to 20 us. With the
  battery path lost at full regen the link reaches 962 V at 100 us and 897 V
  at 20 us; design-verify now checks it

Gates: 602 comps, 1717/1717 pins, ERC 816/0, design-verify 102P/11W/0F,
sim 24P/4W/0F, BOM SiC Rs70,965 / IGBT Rs45,465 @1k.

Co-Authored-By: Claude Opus 5.5 <noreply@anthropic.com>
Parts:
- added RPD7, RPD8, RPD9: 10k, R0603, symbol traction-r1:R
- C5B2: renamed from PSASC; value QA01C-18 -> 100nF; footprint SIP7 -> C0603; symbol traction-r1:QA01C-18 -> traction-r1:C; MPN QA01C-18 -> MLCC-100nF-25V
- C5C1: renamed from UASC; value TLP152 -> 1uF; footprint SO6 -> C0603; symbol traction-r1:TLP152 -> traction-r1:C; LCSC C17255258 -> CLASS; MPN TLP152 -> MLCC-1uF-25V
- C5G1: renamed from RGDLE; value 100k -> 1uF; footprint R0603 -> C0805; symbol traction-r1:R -> traction-r1:C; MPN R0603-CLASS -> MLCC-1uF-50V
- C5G2: renamed from UB15; value TPS55340QRTERQ1 -> 10uF; footprint WQFN16 -> C1206; symbol traction-r1:TPS55340QRTERQ1 -> traction-r1:C; LCSC C2070860 -> CLASS; MPN TPS55340QRTERQ1 -> MLCC-10uF-25V
- CASC: renamed from RASCL; value 470R -> 100nF; footprint R0603 -> C0603; symbol traction-r1:R -> traction-r1:C; MPN R0603-470R -> MLCC-100nF-25V
- CB15C: renamed from CB15I; value 10uF -> 470pF; footprint C1210 -> C0603; MPN MLCC-10uF-50V -> MLCC-CLASS
- CB15CC: renamed from CB15O1; value 22uF -> 100nF; footprint C1210 -> C0603; MPN MLCC-22uF-25V -> MLCC-CLASS
- CB15I: renamed from CB15O2; value 22uF -> 10uF; MPN MLCC-22uF-25V -> MLCC-10uF-50V
- CB15O1: renamed from CB15S; value 47nF -> 22uF; footprint C0603 -> C1210; MPN MLCC-CLASS -> MLCC-22uF-25V
- CB15O2: renamed from CLD15; footprint C0603 -> C1210; MPN MLCC-CLASS -> MLCC-22uF-25V
- CB15S: renamed from CLDC; value 220pF -> 47nF
- CFHA: value 4.7uF -> 47uF; footprint C1206 -> C1210; MPN MLCC-4.7uF-50V -> MLCC-47uF-25V-X7R
- CFLA: renamed from CFLCF; value 47pF -> 47uF; footprint C0603 -> C1210; MPN MLCC-CLASS -> MLCC-47uF-25V-X7R
- CFLCF: renamed from CFLCO; value 22nF -> 47pF
- CFLCO: renamed from CFLCT; value 680pF -> 22nF
- CFLCT: renamed from CFLSI; value 100pF -> 680pF
- CFLSI: renamed from CFLSN; footprint C1206 -> C0603; MPN MLCC-100pF-500V -> MLCC-CLASS
- CFLSN: renamed from CFLVR; value 100nF -> 100pF; footprint C0603 -> C1206; MPN MLCC-CLASS -> MLCC-100pF-500V
- CFLVR: renamed from DFLA; value US1M -> 100nF; footprint SMA -> C0603; symbol traction-r1:D -> traction-r1:C; LCSC C412437 -> CLASS; MPN US1M -> MLCC-CLASS
- CLD15: renamed from DB15; value SS34 -> 22uF; footprint SMA -> C0603; symbol traction-r1:D -> traction-r1:C; MPN SS34 -> MLCC-CLASS
- CLDC: renamed from LB15; value XAL4040-103MEC -> 220pF; footprint XAL4040 -> C0603; symbol traction-r1:L -> traction-r1:C; MPN XAL4040-103MEC -> MLCC-CLASS
- CLVH1: renamed from DRH; value NRVBAF360T3G -> 4.7uF; footprint SMA-flat -> C1206; symbol traction-r1:D -> traction-r1:C; MPN NRVBAF360T3G -> MLCC-4.7uF-50V
- CLVH2: renamed from DTVH; value TPSMC24CA -> 4.7uF; footprint SMC -> C1206; symbol traction-r1:D -> traction-r1:C; LCSC C1975284 -> CLASS; MPN TPSMC24CA -> MLCC-4.7uF-50V
- CLVL1: renamed from DRL; value NRVBAF360T3G -> 4.7uF; footprint SMA-flat -> C1206; symbol traction-r1:D -> traction-r1:C; MPN NRVBAF360T3G -> MLCC-4.7uF-50V
- CLVL2: renamed from DTVL; value TPSMC24CA -> 4.7uF; footprint SMC -> C1206; symbol traction-r1:D -> traction-r1:C; LCSC C1975284 -> CLASS; MPN TPSMC24CA -> MLCC-4.7uF-50V
- CVBDF: renamed from RVBD2; value 470k -> 1nF; footprint R1206 -> C0603; symbol traction-r1:R -> traction-r1:C; MPN R1206-470k-TF -> MLCC-1nF-50V
- CVDDF: renamed from RVDD2; value 470k -> 1nF; footprint R1206 -> C0603; symbol traction-r1:R -> traction-r1:C; MPN R1206-470k-TF -> MLCC-1nF-50V
- DB15: renamed from RB15C; value 2k -> SS34; footprint R0603 -> SMA; symbol traction-r1:R -> traction-r1:D; MPN R0603-CLASS -> SS34
- DFHVZ: renamed from RFHCS; value 330m -> BZT52-C18; footprint R1210 -> SOD123; symbol traction-r1:R -> traction-r1:D; MPN R1210-0R33-0.75W -> BZT52-C18
- DFLA: renamed from DFLG; value PMEG4010EH -> US1M; footprint SOD123 -> SMA; LCSC C282566 -> C412437; MPN PMEG4010EH -> US1M
- DFLG: renamed from DFLSN; value US1M -> PMEG4010EH; footprint SMA -> SOD123; LCSC C412437 -> C282566; MPN US1M -> PMEG4010EH
- DFLSN: renamed from RFLCS; value 330m -> US1M; footprint R1210 -> SMA; symbol traction-r1:R -> traction-r1:D; LCSC CLASS -> C412437; MPN R1210-0R33-0.75W -> US1M
- DFLVZ: renamed from RFLEN; value 100k -> BZT52-C18; footprint R0603 -> SOD123; symbol traction-r1:R -> traction-r1:D; MPN R0603-CLASS -> BZT52-C18
- DRH: renamed from FH1; value MF-LSMF300/24X-2 -> NRVBAF360T3G; footprint PTC2920 -> SMA-flat; symbol traction-r1:F -> traction-r1:D; LCSC C719172 -> CLASS; MPN MF-LSMF300/24X-2 -> NRVBAF360T3G
- DRL: renamed from FL1; value MF-LSMF300/24X-2 -> NRVBAF360T3G; footprint PTC2920 -> SMA-flat; symbol traction-r1:F -> traction-r1:D; LCSC C719172 -> CLASS; MPN MF-LSMF300/24X-2 -> NRVBAF360T3G
- DTVH: renamed from LFH1; value FB-120R-3A -> TPSMC24CA; footprint FB1206 -> SMC; symbol traction-r1:L -> traction-r1:D; LCSC CLASS -> C1975284; MPN FB-120R-3A -> TPSMC24CA
- DTVL: renamed from LFL1; value FB-120R-3A -> TPSMC24CA; footprint FB1206 -> SMC; symbol traction-r1:L -> traction-r1:D; LCSC CLASS -> C1975284; MPN FB-120R-3A -> TPSMC24CA
- FH1: renamed from CLVL1; value 4.7uF -> MF-LSMF300/24X-2; footprint C1206 -> PTC2920; symbol traction-r1:C -> traction-r1:F; LCSC CLASS -> C719172; MPN MLCC-4.7uF-50V -> MF-LSMF300/24X-2
- FL1: renamed from UGDL; value NCV4276CDT50RKG -> MF-LSMF300/24X-2; footprint DPAK -> PTC2920; symbol traction-r1:NCV4276CDT50RKG -> traction-r1:F; LCSC CLASS -> C719172; MPN NCV4276CDT50RKG -> MF-LSMF300/24X-2
- JIC: renamed from RPD1; value 10k -> MICROFIT3-40; footprint R0603 -> MicroFit40; symbol traction-r1:R -> traction-r1:MICROFIT3-40; MPN R0603-10k -> MICROFIT3-40
- LB15: renamed from RB15F1; value 110k -> XAL4040-103MEC; footprint R0603 -> XAL4040; symbol traction-r1:R -> traction-r1:L; MPN R0603-1% -> XAL4040-103MEC
- LFH1: renamed from CLVL2; value 4.7uF -> FB-120R-3A; footprint C1206 -> FB1206; symbol traction-r1:C -> traction-r1:L; MPN MLCC-4.7uF-50V -> FB-120R-3A
- LFL1: renamed from C5G1; value 1uF -> FB-120R-3A; footprint C1206 -> FB1206; symbol traction-r1:C -> traction-r1:L; MPN MLCC-10uF-25V -> FB-120R-3A
- PS5B: renamed from C5B1; value 1uF -> MGJ2D150505SC; footprint C0603 -> SIP7; symbol traction-r1:C -> traction-r1:MGJ2D150505SC; MPN MLCC-1uF-25V -> MGJ2D150505SC
- PS5C: renamed from C5B2; value 100nF -> MGJ2D150505SC; footprint C0603 -> SIP7; symbol traction-r1:C -> traction-r1:MGJ2D150505SC; MPN MLCC-1uF-25V -> MGJ2D150505SC
- PSASC: renamed from CASC; value 100nF -> QA01C-18; footprint C0603 -> SIP7; symbol traction-r1:C -> traction-r1:QA01C-18; MPN MLCC-100nF-25V -> QA01C-18
- QFL: renamed from QFLE1; value 2N7002 -> BUK7Y14-80E; footprint SOT23 -> LFPAK56; symbol traction-r1:2N7002 -> traction-r1:BUK7Y14-80E; LCSC C8545 -> C86732; MPN 2N7002 -> BUK7Y14-80E
- QFLE2: renamed from TFL1; value VGT12EEM-200S1A4 -> 2N7002; footprint XfmrEE12 -> SOT23; symbol traction-r1:VGT12EEM-200S1A4 -> traction-r1:2N7002; LCSC CLASS -> C8545; MPN VGT12EEM-200S1A4 -> 2N7002
- RASCG: renamed from RASCPD; value 10k -> 2.2k; MPN R0603-10k -> R0603-2k2
- RASCL: renamed from ZASC; value BZT52-C5V1 -> 470R; footprint SOD123 -> R0603; symbol traction-r1:D -> traction-r1:R; MPN BZT52-C5V1 -> R0603-470R
- RASCPD: renamed from CLVH1; value 4.7uF -> 10k; footprint C1206 -> R0603; symbol traction-r1:C -> traction-r1:R; MPN MLCC-4.7uF-50V -> R0603-10k
- RB15C: renamed from RB15F2; value 9.53k -> 2k; MPN R0603-1% -> R0603-CLASS
- RB15F1: renamed from RB15Q; value 80.6k -> 110k; MPN R0603-CLASS -> R0603-1%
- RB15F2: renamed from RLD1; value 49.9k -> 9.53k; MPN R0603-CLASS -> R0603-1%
- RB15Q: renamed from RLD2; value 10k -> 80.6k
- RFHCS: renamed from RFHEN; value 100k -> 330m; footprint R0603 -> R1210; MPN R0603-CLASS -> R1210-0R33-0.75W
- RFHEN: renamed from RFHFB1; value 56k -> 100k; MPN R0603-1% -> R0603-CLASS
- RFHFB1: renamed from RFHFB2; value 15k -> 56k
- RFHFB2: renamed from RFHG; value 10R -> 15k; MPN R0603-CLASS -> R0603-1%
- RFHG: renamed from RFHGO; value 20R -> 10R
- RFHGO: renamed from RFHGS; value 51k -> 20R
- RFHGS: renamed from RFHRT; value 10k -> 51k
- RFHRT: renamed from RFHSI; value 100R -> 10k
- RFHSI: renamed from RFHSN; footprint R0805 -> R0603; MPN R0805-100R -> R0603-CLASS
- RFHSN: renamed from RFHST; value 4.7k -> 100R; footprint R0603 -> R0805; MPN R0603-CLASS -> R0805-100R
- RFHST: renamed from ZFHG; value BZT52-C15 -> 2.2k; footprint SOD123 -> R1206; symbol traction-r1:D -> traction-r1:R; MPN BZT52-C15 -> R1206-2k2
- RFLCS: renamed from RFLFB1; value 56k -> 330m; footprint R0603 -> R1210; MPN R0603-1% -> R1210-0R33-0.75W
- RFLEN: renamed from RFLFB2; value 15k -> 100k; MPN R0603-1% -> R0603-CLASS
- RFLFB1: renamed from RFLG; value 10R -> 56k; MPN R0603-CLASS -> R0603-1%
- RFLFB2: renamed from RFLGO; value 20R -> 15k; MPN R0603-CLASS -> R0603-1%
- RFLG: renamed from RFLGS; value 51k -> 10R
- RFLGO: renamed from RFLRT; value 10k -> 20R
- RFLGS: renamed from RFLSI; value 100R -> 51k
- RFLRT: renamed from RFLSN; value 100R -> 10k; footprint R0805 -> R0603; MPN R0805-100R -> R0603-CLASS
- RFLSI: renamed from RFLST; value 4.7k -> 100R
- RFLSN: renamed from ZFLG; value BZT52-C15 -> 100R; footprint SOD123 -> R0805; symbol traction-r1:D -> traction-r1:R; MPN BZT52-C15 -> R0805-100R
- RFLST: renamed from ZFLSN; value SMAJ13A -> 2.2k; footprint SMA -> R1206; symbol traction-r1:D -> traction-r1:R; MPN SMAJ13A -> R1206-2k2
- RGDLE: renamed from ULDO15; value NCV4276CDTADJRKG -> 100k; footprint DPAK5 -> R0603; symbol traction-r1:NCV4276CDTADJRKG -> traction-r1:R; MPN NCV4276CDTADJRKG -> R0603-CLASS
- RHWID: renamed from RPD10; MPN R0603-10k -> R0603-10k-1%
- RLD1: renamed from JIC; value MICROFIT3-40 -> 49.9k; footprint MicroFit40 -> R0603; symbol traction-r1:MICROFIT3-40 -> traction-r1:R; MPN MICROFIT3-40 -> R0603-CLASS
- RLD2: renamed from RPD0; MPN R0603-10k -> R0603-CLASS
- RUHBL, RULBL, RVHBL, RVLBL, RWHBL, RWLBL: MPN R0805-4k99 -> R0805-5k1
- RUHOFF, RULOFF, RVHOFF, RVLOFF, RWHOFF, RWLOFF: value 1R -> 6.8R; MPN R2512-1R0-2W -> R2512-6R8-2W
- RUHON, RULON, RVHON, RVLON, RWHON, RWLON: value 1.5R -> 3.3R; MPN R2512-1R5-2W -> R2512-3R3-2W
- RVBD5: renamed from RVBDL; value 6.2k -> 470k; footprint R0603 -> R1206; MPN R0603-6k2-0.1% -> R1206-470k-TF
- RVBD6: renamed from PS5B; value MGJ2D150505SC -> 470k; footprint SIP7 -> R1206; symbol traction-r1:MGJ2D150505SC -> traction-r1:R; MPN MGJ2D150505SC -> R1206-470k-TF
- RVBDL: renamed from PS5C; value MGJ2D150505SC -> 6.2k; footprint SIP7 -> R0603; symbol traction-r1:MGJ2D150505SC -> traction-r1:R; MPN MGJ2D150505SC -> R0603-6k2-0.1%
- RVDD5: renamed from RVDDL; value 6.2k -> 470k; footprint R0603 -> R1206; MPN R0603-6k2-0.1% -> R1206-470k-TF
- RVDD6: renamed from UIVB; value AMC1311BDWVR -> 470k; footprint SOIC8W -> R1206; symbol traction-r1:AMC1311BDWVR -> traction-r1:R; LCSC C456277 -> CLASS; MPN AMC1311BDWVR -> R1206-470k-TF
- RVDDL: renamed from CVBDF; value 1nF -> 6.2k; footprint C0603 -> R0603; symbol traction-r1:C -> traction-r1:R; MPN MLCC-1nF-50V -> R0603-6k2-0.1%
- TFL3: renamed from UFL; value UCC28C40DR -> VGT12EEM-200S1A4; footprint SOP8 -> XfmrEE12; symbol traction-r1:UCC28C40DR -> traction-r1:VGT12EEM-200S1A4; MPN UCC28C40DR -> VGT12EEM-200S1A4
- UASC: renamed from RASCG; value 2.2k -> TLP152; footprint R0603 -> SO6; symbol traction-r1:R -> traction-r1:TLP152; LCSC CLASS -> C17255258; MPN R0603-2k2 -> TLP152
- UB15: renamed from CB15C; value 470pF -> TPS55340QRTERQ1; footprint C0603 -> WQFN16; symbol traction-r1:C -> traction-r1:TPS55340QRTERQ1; LCSC CLASS -> C2070860; MPN MLCC-CLASS -> TPS55340QRTERQ1
- UFL: renamed from CFLA; value 4.7uF -> UCC28C40DR; footprint C1206 -> SOP8; symbol traction-r1:C -> traction-r1:UCC28C40DR; MPN MLCC-4.7uF-50V -> UCC28C40DR
- UGDL: renamed from C5G2; value 10uF -> NCV4276CDT50RKG; footprint C1206 -> DPAK; symbol traction-r1:C -> traction-r1:NCV4276CDT50RKG; MPN MLCC-10uF-25V -> NCV4276CDT50RKG
- UIVB: renamed from RVBD1; value 470k -> AMC1311BDWVR; footprint R1206 -> SOIC8W; symbol traction-r1:R -> traction-r1:AMC1311BDWVR; LCSC CLASS -> C456277; MPN R1206-470k-TF -> AMC1311BDWVR
- UIVDC: renamed from RVDD1; value 470k -> AMC1311BDWVR; footprint R1206 -> SOIC8W; symbol traction-r1:R -> traction-r1:AMC1311BDWVR; LCSC CLASS -> C456277; MPN R1206-470k-TF -> AMC1311BDWVR
- ULDO15: renamed from CB15CC; value 100nF -> NCV4276CDTADJRKG; footprint C0603 -> DPAK5; symbol traction-r1:C -> traction-r1:NCV4276CDTADJRKG; MPN MLCC-CLASS -> NCV4276CDTADJRKG
- ZASC: renamed from CLVH2; value 4.7uF -> BZT52-C5V1; footprint C1206 -> SOD123; symbol traction-r1:C -> traction-r1:D; MPN MLCC-4.7uF-50V -> BZT52-C5V1
- ZFHG: renamed from ZFHSN; value SMAJ13A -> BZT52-C15; footprint SMA -> SOD123; MPN SMAJ13A -> BZT52-C15
- ZFHSN: renamed from QFL; value BUK7Y14-80E -> SMAJ13A; footprint LFPAK56 -> SMA; symbol traction-r1:BUK7Y14-80E -> traction-r1:D; LCSC C86732 -> CLASS; MPN BUK7Y14-80E -> SMAJ13A
- ZFLG: renamed from UIVDC; value AMC1311BDWVR -> BZT52-C15; footprint SOIC8W -> SOD123; symbol traction-r1:AMC1311BDWVR -> traction-r1:D; LCSC C456277 -> CLASS; MPN AMC1311BDWVR -> BZT52-C15
- ZFLSN: renamed from CVDDF; value 1nF -> SMAJ13A; footprint C0603 -> SMA; symbol traction-r1:C -> traction-r1:D; MPN MLCC-1nF-50V -> SMAJ13A
- renumbered C5C1 to C5B1, QFLE2 to QFLE1, RPD2 to RPD0, RPD3 to RPD1, RPD4 to RPD10, RPD5 to RPD2, RPD6 to RPD3, RPD7 to RPD4, RPD8 to RPD5, RPD9 to RPD6, RVBD3 to RVBD1, RVBD4 to RVBD2, RVBD5 to RVBD3, RVBD6 to RVBD4, RVDD3 to RVDD1, RVDD4 to RVDD2, RVDD5 to RVDD3, RVDD6 to RVDD4, TFL2 to TFL1, TFL3 to TFL2
Connections:
- net labels added: HW_ID
- wire segments 807 -> 813
Other:
- note added: "7 2x iso VDC senses >5% = fault, VOFS monitored"
- note added: "8 DESAT per switch (SiC <=1.9 us detect), latching"
- note added: "9 HVIL open = VDDIO/2 signature -> torque off (FW)"
- note added: "E = 116 J @850 V - 32 J/res worst; 4XX: 220R/15k"
- note added: "PASSIVE 12x 22k 2512-2W (6s x 2p = 66k): 56 s to 60 V"
- note added: "rev A.6 - 24 sections - 295 components"
- note removed: "7 2x isolated VDC senses, >5% mismatch = fault"
- note removed: "8 DESAT per switch, ~1.5 us blanking, latching"
- note removed: "9 HVIL open = VDDIO/2 signature -> discharge"
- note removed: "E = 116 J @850 V - 32 J/res worst (>=100 J rated)"
- note removed: "PASSIVE 10x 27k 2512-2W (5s x 2p = 67.5k): 57 s to 60 V"
- note removed: "rev A.5 - 24 sections - 292 components"
- moved on the sheet: C5B1, CB15C, CB15CC, CB15I, CB15O1, CB15O2, CB15S, CFLA, CFLCF, CFLCO, CFLCT, CFLSI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

Commit message: Rev A.7: review round 7 response (RR01-RR10, A6-R01-R14) + cross-check
Two independent rechecks of c963794 were verified finding by finding and
classified in docs/review-A7-disposition.md (+ .csv): 17 confirmed and fixed,
1 spec gap closed, 3 firmware handled, 3 already-tracked release gates. Two
further defects were self-found (N10, N11).

Safety logic (control card):
- 74LVC3G17-Q100 Schmitt buffer between the RC timing nodes (clear one-shot,
  soft-off delay) and the LVC inputs they drove at 14,000-63,500 ns/V. The
  FS0B line goes through it too; a 100 k pull-down makes a dead buffer
  force DRV_EN low.
- FS0B/FS1B pull-ups 1 k -> 5.1 k (FS1B inside its 2 mA V_OL point).
- FAULT_OUT made sink-only (BAT46): a grounded vehicle wire can no longer
  preset ASC. A KL30 short is clamped at the latch.
- DRV_EN and ASC_CMD read-backs to the MCU for a boot self-test.
- Latches moved to Nexperia 74LVC1G74DC-Q100 (the TI part is not Q100).
- CCLR changed to C0G.

ASC entry is now break-before-make:
- A 12 nF delay (+ fast-release diode) holds the LS ASC off >= 3.4 us.
- MCU path: HS off via the eFlexPWM fault, then PWM-ASC with EN high.
- MCU-dead path: FS0B, then the delayed ASC.
- EN is never dropped for ASC: NSI6611 DS 8.12 honours DESAT over ASC only
  with EN high. The first draft's DASC diode did drop it and was removed
  after the cross-check.
- 1 k series resistor at each LS ASC pin.
- ASC opto LED resistor 470 -> 270 R (TLP152 I_FLH max 7.5 mA).

Gate supply:
- The flyback FB divider senses its own aux rectifier, so the start feed
  can no longer lock gate power out at high KL30.
- 52.3k/15k: VCC2 15.4 V nominal, 13.54-16.7 V corners.
- Boost output capacitors 25 V -> 50 V.

Models and checkers:
- IGBT and diode share the coldplate term.
- Flyback bank inductance corrected.
- SC soft-off checked at both I_STO corners (release gate).
- FW-06 as a measured budget: 15.6 us + 7.0 us all-off -> 905/542 V.
- bom-gen preflight and a JSWD pin-count check (Samtec 10-pin).
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
Parts:
- added RPD0, RPD1, RPD10, RPD2, RPD3, RPD4, RPD5, RPD6, RPD7, RPD8, RPD9: 10k, R0603, symbol traction-r1:R
- C5B1: renamed from ZASC; value BZT52-C5V1 -> 1uF; footprint SOD123 -> C0603; symbol traction-r1:D -> traction-r1:C; MPN BZT52-C5V1 -> MLCC-1uF-25V
- C5B2: renamed from CLVH1; value 4.7uF -> 100nF; footprint C1206 -> C0603; MPN MLCC-4.7uF-50V -> MLCC-100nF-25V
- C5C1: renamed from CLVH2; value 4.7uF -> 1uF; footprint C1206 -> C0603; MPN MLCC-4.7uF-50V -> MLCC-1uF-25V
- C5G1: renamed from CLD15; value 22uF -> 1uF; footprint C0603 -> C0805; MPN MLCC-CLASS -> MLCC-1uF-50V
- C5G2: renamed from CLDC; value 220pF -> 10uF; footprint C0603 -> C1206; MPN MLCC-CLASS -> MLCC-10uF-25V
- CASC: renamed from FH1; value MF-LSMF300/24X-2 -> 100nF; footprint PTC2920 -> C0603; symbol traction-r1:F -> traction-r1:C; LCSC C719172 -> CLASS; MPN MF-LSMF300/24X-2 -> MLCC-100nF-25V
- CASCD: renamed from LFH1; value FB-120R-3A -> 12nF; footprint FB1206 -> C0603; symbol traction-r1:L -> traction-r1:C; MPN FB-120R-3A -> MLCC-12nF-50V-C0G
- CB15C: renamed from RB15F1; value 110k -> 470pF; footprint R0603 -> C0603; symbol traction-r1:R -> traction-r1:C; MPN R0603-1% -> MLCC-CLASS
- CB15CC: renamed from RB15F2; value 9.53k -> 100nF; footprint R0603 -> C0603; symbol traction-r1:R -> traction-r1:C; MPN R0603-1% -> MLCC-CLASS
- CB15I: renamed from RB15Q; value 80.6k -> 10uF; footprint R0603 -> C1210; symbol traction-r1:R -> traction-r1:C; MPN R0603-CLASS -> MLCC-10uF-50V
- CB15O1: renamed from RLD1; value 49.9k -> 22uF; footprint R0603 -> C1210; symbol traction-r1:R -> traction-r1:C; MPN R0603-CLASS -> MLCC-22uF-50V
- CB15O2: renamed from RLD2; value 10k -> 22uF; footprint R0603 -> C1210; symbol traction-r1:R -> traction-r1:C; MPN R0603-CLASS -> MLCC-22uF-50V
- CB15S: renamed from JIC; value MICROFIT3-40 -> 47nF; footprint MicroFit40 -> C0603; symbol traction-r1:MICROFIT3-40 -> traction-r1:C; MPN MICROFIT3-40 -> MLCC-CLASS
- CFHA: renamed from CFHCT; value 680pF -> 47uF; footprint C0603 -> C1210; MPN MLCC-CLASS -> MLCC-47uF-25V-X7R
- CFHCF: renamed from CFHSI; value 100pF -> 47pF
- CFHCO: renamed from CFHSN; value 100pF -> 22nF; footprint C1206 -> C0603; MPN MLCC-100pF-500V -> MLCC-CLASS
- CFHCT: renamed from CFHVR; value 100nF -> 680pF
- CFHFS: renamed from DFHA; value US1M -> 100nF; footprint SMA -> C0603; symbol traction-r1:D -> traction-r1:C; LCSC C412437 -> CLASS; MPN US1M -> MLCC-100nF-50V-SOFT
- CFHSI: renamed from DFHG; value PMEG4010EH -> 100pF; footprint SOD123 -> C0603; symbol traction-r1:D -> traction-r1:C; LCSC C282566 -> CLASS; MPN PMEG4010EH -> MLCC-CLASS
- CFHSN: renamed from DFHSN; value US1M -> 100pF; footprint SMA -> C1206; symbol traction-r1:D -> traction-r1:C; LCSC C412437 -> CLASS; MPN US1M -> MLCC-100pF-500V
- CFHVR: renamed from DFHVZ; value BZT52-C18 -> 100nF; footprint SOD123 -> C0603; symbol traction-r1:D -> traction-r1:C; MPN BZT52-C18 -> MLCC-CLASS
- CFLA: renamed from CFLVR; value 100nF -> 47uF; footprint C0603 -> C1210; MPN MLCC-CLASS -> MLCC-47uF-25V-X7R
- CFLCF: renamed from DFLA; value US1M -> 47pF; footprint SMA -> C0603; symbol traction-r1:D -> traction-r1:C; LCSC C412437 -> CLASS; MPN US1M -> MLCC-CLASS
- CFLCO: renamed from DFLG; value PMEG4010EH -> 22nF; footprint SOD123 -> C0603; symbol traction-r1:D -> traction-r1:C; LCSC C282566 -> CLASS; MPN PMEG4010EH -> MLCC-CLASS
- CFLCT: renamed from DFLSN; value US1M -> 680pF; footprint SMA -> C0603; symbol traction-r1:D -> traction-r1:C; LCSC C412437 -> CLASS; MPN US1M -> MLCC-CLASS
- CFLFS: renamed from DFLVZ; value BZT52-C18 -> 100nF; footprint SOD123 -> C0603; symbol traction-r1:D -> traction-r1:C; MPN BZT52-C18 -> MLCC-100nF-50V-SOFT
- CFLSI: renamed from RFLCS; value 330m -> 100pF; footprint R1210 -> C0603; symbol traction-r1:R -> traction-r1:C; MPN R1210-0R33-0.75W -> MLCC-CLASS
- CFLSN: renamed from RFLEN; value 100k -> 100pF; footprint R0603 -> C1206; symbol traction-r1:R -> traction-r1:C; MPN R0603-CLASS -> MLCC-100pF-500V
- CFLVR: renamed from RFLFB1; value 56k -> 100nF; footprint R0603 -> C0603; symbol traction-r1:R -> traction-r1:C; MPN R0603-1% -> MLCC-CLASS
- CLD15: renamed from RHWID; value 10k -> 22uF; footprint R0603 -> C0603; symbol traction-r1:R -> traction-r1:C; MPN R0603-10k-1% -> MLCC-CLASS
- CLDC: renamed from RPD0; value 10k -> 220pF; footprint R0603 -> C0603; symbol traction-r1:R -> traction-r1:C; MPN R0603-10k -> MLCC-CLASS
- CLVH1: renamed from LFL1; value FB-120R-3A -> 4.7uF; footprint FB1206 -> C1206; symbol traction-r1:L -> traction-r1:C; MPN FB-120R-3A -> MLCC-4.7uF-50V
- CLVH2: renamed from UGDL; value NCV4276CDT50RKG -> 4.7uF; footprint DPAK -> C1206; symbol traction-r1:NCV4276CDT50RKG -> traction-r1:C; MPN NCV4276CDT50RKG -> MLCC-4.7uF-50V
- CLVL1: renamed from ULDO15; value NCV4276CDTADJRKG -> 4.7uF; footprint DPAK5 -> C1206; symbol traction-r1:NCV4276CDTADJRKG -> traction-r1:C; MPN NCV4276CDTADJRKG -> MLCC-4.7uF-50V
- CLVL2: renamed from CB15C; value 470pF -> 4.7uF; footprint C0603 -> C1206; MPN MLCC-CLASS -> MLCC-4.7uF-50V
- CVBDF: renamed from PS5C; value MGJ2D150505SC -> 1nF; footprint SIP7 -> C0603; symbol traction-r1:MGJ2D150505SC -> traction-r1:C; MPN MGJ2D150505SC -> MLCC-1nF-50V
- CVHB1: renamed from CVHB2; value 4.7uF -> 100nF; footprint C1206 -> C0603; MPN MLCC-4.7uF-50V -> MLCC-100nF-50V
- CVHB2: renamed from CVHBL; value 47pF -> 4.7uF; footprint C0603 -> C1206; MPN MLCC-47pF-100V -> MLCC-4.7uF-50V
- CVHBL: renamed from CVHE1; value 10uF -> 47pF; footprint C1206 -> C0603; MPN MLCC-10uF-25V -> MLCC-47pF-100V
- CVHE1: renamed from CVHIN; value 100nF -> 10uF; footprint C0603 -> C1206; MPN MLCC-CLASS -> MLCC-10uF-25V
- CVHIN: renamed from CVHV1; value 4.7uF -> 100nF; footprint C1206 -> C0603; MPN MLCC-4.7uF-50V -> MLCC-CLASS
- CVHV1: renamed from DVHR; value US1M -> 4.7uF; footprint SMA -> C1206; symbol traction-r1:D -> traction-r1:C; LCSC C412437 -> CLASS; MPN US1M -> MLCC-4.7uF-50V
- CVLB1: renamed from CVLB2; value 4.7uF -> 100nF; footprint C1206 -> C0603; MPN MLCC-4.7uF-50V -> MLCC-100nF-50V
- CVLB2: renamed from CVLBL; value 47pF -> 4.7uF; footprint C0603 -> C1206; MPN MLCC-47pF-100V -> MLCC-4.7uF-50V
- CVLBL: renamed from CVLE1; value 10uF -> 47pF; footprint C1206 -> C0603; MPN MLCC-10uF-25V -> MLCC-47pF-100V
- CVLE1: renamed from CVLIN; value 100nF -> 10uF; footprint C0603 -> C1206; MPN MLCC-CLASS -> MLCC-10uF-25V
- CVLIN: renamed from CVLV1; value 4.7uF -> 100nF; footprint C1206 -> C0603; MPN MLCC-4.7uF-50V -> MLCC-CLASS
- CVLV1: renamed from DVLR; value US1M -> 4.7uF; footprint SMA -> C1206; symbol traction-r1:D -> traction-r1:C; LCSC C412437 -> CLASS; MPN US1M -> MLCC-4.7uF-50V
- CVSN: renamed from CVTF; value 2.2nF -> 1uF; footprint C0603 -> FilmP27.5; MPN MLCC-2.2nF-50V -> FILM-1uF-1200V
- CVTF: renamed from DVTP; value PESD5V0U1UA -> 2.2nF; footprint SOD323 -> C0603; symbol traction-r1:D -> traction-r1:C; MPN PESD5V0U1UA -> MLCC-2.2nF-50V
- CWHB1: renamed from CWHBL; value 47pF -> 100nF; MPN MLCC-47pF-100V -> MLCC-100nF-50V
- CWHB2: renamed from CWHE1; value 10uF -> 4.7uF; MPN MLCC-10uF-25V -> MLCC-4.7uF-50V
- CWHBL: renamed from CWHIN; value 100nF -> 47pF; MPN MLCC-CLASS -> MLCC-47pF-100V
- CWHE1: renamed from CWHV1; value 4.7uF -> 10uF; MPN MLCC-4.7uF-50V -> MLCC-10uF-25V
- CWHIN: renamed from DWHR; value US1M -> 100nF; footprint SMA -> C0603; symbol traction-r1:D -> traction-r1:C; LCSC C412437 -> CLASS; MPN US1M -> MLCC-CLASS
- CWHV1: renamed from DWHS1; value US1M -> 4.7uF; footprint SMA -> C1206; symbol traction-r1:D -> traction-r1:C; LCSC C412437 -> CLASS; MPN US1M -> MLCC-4.7uF-50V
- CWLB1: renamed from CWLBL; value 47pF -> 100nF; MPN MLCC-47pF-100V -> MLCC-100nF-50V
- CWLB2: renamed from CWLE1; value 10uF -> 4.7uF; MPN MLCC-10uF-25V -> MLCC-4.7uF-50V
- CWLBL: renamed from CWLIN; value 100nF -> 47pF; MPN MLCC-CLASS -> MLCC-47pF-100V
- CWLE1: renamed from CWLV1; value 4.7uF -> 10uF; MPN MLCC-4.7uF-50V -> MLCC-10uF-25V
- CWLIN: renamed from DWLR; value US1M -> 100nF; footprint SMA -> C0603; symbol traction-r1:D -> traction-r1:C; LCSC C412437 -> CLASS; MPN US1M -> MLCC-CLASS
- CWLV1: renamed from DWLS1; value US1M -> 4.7uF; footprint SMA -> C1206; symbol traction-r1:D -> traction-r1:C; LCSC C412437 -> CLASS; MPN US1M -> MLCC-4.7uF-50V
- CWSN: renamed from DWTP; value PESD5V0U1UA -> 1uF; footprint SOD323 -> FilmP27.5; symbol traction-r1:D -> traction-r1:C; MPN PESD5V0U1UA -> FILM-1uF-1200V
- CWTF: renamed from JMW; value STUD-M8 -> 2.2nF; footprint StudM8 -> C0603; symbol traction-r1:TERM_1 -> traction-r1:C; MPN STUD-M8 -> MLCC-2.2nF-50V
- DASCR: renamed from CLVL1; value 4.7uF -> 1N4148WS; footprint C1206 -> SOD323; symbol traction-r1:C -> traction-r1:D; LCSC CLASS -> C2128; MPN MLCC-4.7uF-50V -> 1N4148WS
- DB15: renamed from RPD1; value 10k -> SS34; footprint R0603 -> SMA; symbol traction-r1:R -> traction-r1:D; MPN R0603-10k -> SS34
- DFHA: renamed from RFHCS; value 330m -> US1M; footprint R1210 -> SMA; symbol traction-r1:R -> traction-r1:D; LCSC CLASS -> C412437; MPN R1210-0R33-0.75W -> US1M
- DFHFS: renamed from RFHEN; value 100k -> 1N4148WS; footprint R0603 -> SOD323; symbol traction-r1:R -> traction-r1:D; LCSC CLASS -> C2128; MPN R0603-CLASS -> 1N4148WS
- DFHG: renamed from RFHFB1; value 56k -> PMEG4010EH; footprint R0603 -> SOD123; symbol traction-r1:R -> traction-r1:D; LCSC CLASS -> C282566; MPN R0603-1% -> PMEG4010EH
- DFHSN: renamed from RFHFB2; value 15k -> US1M; footprint R0603 -> SMA; symbol traction-r1:R -> traction-r1:D; LCSC CLASS -> C412437; MPN R0603-1% -> US1M
- DFHVZ: renamed from RFHG; value 10R -> BZT52-C18; footprint R0603 -> SOD123; symbol traction-r1:R -> traction-r1:D; MPN R0603-CLASS -> BZT52-C18
- DFLA: renamed from RFLFB2; value 15k -> US1M; footprint R0603 -> SMA; symbol traction-r1:R -> traction-r1:D; LCSC CLASS -> C412437; MPN R0603-1% -> US1M
- DFLFS: renamed from RFLG; value 10R -> 1N4148WS; footprint R0603 -> SOD323; symbol traction-r1:R -> traction-r1:D; LCSC CLASS -> C2128; MPN R0603-CLASS -> 1N4148WS
- DFLG: renamed from RFLGO; value 20R -> PMEG4010EH; footprint R0603 -> SOD123; symbol traction-r1:R -> traction-r1:D; LCSC CLASS -> C282566; MPN R0603-CLASS -> PMEG4010EH
- DFLSN: renamed from RFLGS; value 51k -> US1M; footprint R0603 -> SMA; symbol traction-r1:R -> traction-r1:D; LCSC CLASS -> C412437; MPN R0603-CLASS -> US1M
- DFLVZ: renamed from RFLRT; value 10k -> BZT52-C18; footprint R0603 -> SOD123; symbol traction-r1:R -> traction-r1:D; MPN R0603-CLASS -> BZT52-C18
- DRH: renamed from C5G1; value 1uF -> NRVBAF360T3G; footprint C0805 -> SMA-flat; symbol traction-r1:C -> traction-r1:D; MPN MLCC-1uF-50V -> NRVBAF360T3G
- DRL: renamed from CB15CC; value 100nF -> NRVBAF360T3G; footprint C0603 -> SMA-flat; symbol traction-r1:C -> traction-r1:D; MPN MLCC-CLASS -> NRVBAF360T3G
- DTVH: renamed from C5G2; value 10uF -> TPSMC24CA; footprint C1206 -> SMC; symbol traction-r1:C -> traction-r1:D; LCSC CLASS -> C1975284; MPN MLCC-10uF-25V -> TPSMC24CA
- DTVL: renamed from CB15I; value 10uF -> TPSMC24CA; footprint C1210 -> SMC; symbol traction-r1:C -> traction-r1:D; LCSC CLASS -> C1975284; MPN MLCC-10uF-50V -> TPSMC24CA
- DVHS2: renamed from DVHSB; value BAT64-04 -> US1M; footprint SOT23 -> SMA; LCSC CLASS -> C412437; MPN BAT64-04 -> US1M
- DVHSB: renamed from DVHZ1; value BZT52-C18 -> BAT64-04; footprint SOD123 -> SOT23; MPN BZT52-C18 -> BAT64-04
- DVHZ1: renamed from DVHZ2; value BZT52-C5V1 -> BZT52-C18; MPN BZT52-C5V1 -> BZT52-C18
- DVHZ2: renamed from RVHBL; value 5.1k -> BZT52-C5V1; footprint R0805 -> SOD123; symbol traction-r1:R -> traction-r1:D; MPN R0805-5k1 -> BZT52-C5V1
- DVLS2: renamed from DVLSB; value BAT64-04 -> US1M; footprint SOT23 -> SMA; LCSC CLASS -> C412437; MPN BAT64-04 -> US1M
- DVLSB: renamed from DVLZ1; value BZT52-C18 -> BAT64-04; footprint SOD123 -> SOT23; MPN BZT52-C18 -> BAT64-04
- DVLZ1: renamed from DVLZ2; value BZT52-C5V1 -> BZT52-C18; MPN BZT52-C5V1 -> BZT52-C18
- DVLZ2: renamed from RVLBL; value 5.1k -> BZT52-C5V1; footprint R0805 -> SOD123; symbol traction-r1:R -> traction-r1:D; MPN R0805-5k1 -> BZT52-C5V1
- DVTP: renamed from JMV; value STUD-M8 -> PESD5V0U1UA; footprint StudM8 -> SOD323; symbol traction-r1:TERM_1 -> traction-r1:D; MPN STUD-M8 -> PESD5V0U1UA
- DWHS1: renamed from DWHSB; value BAT64-04 -> US1M; footprint SOT23 -> SMA; LCSC CLASS -> C412437; MPN BAT64-04 -> US1M
- DWHS2: renamed from DWHZ1; value BZT52-C18 -> US1M; footprint SOD123 -> SMA; LCSC CLASS -> C412437; MPN BZT52-C18 -> US1M
- DWHSB: renamed from DWHZ2; value BZT52-C5V1 -> BAT64-04; footprint SOD123 -> SOT23; MPN BZT52-C5V1 -> BAT64-04
- DWHZ1: renamed from RWHBL; value 5.1k -> BZT52-C18; footprint R0805 -> SOD123; symbol traction-r1:R -> traction-r1:D; MPN R0805-5k1 -> BZT52-C18
- DWHZ2: renamed from RWHDS; value 100R -> BZT52-C5V1; footprint R0805 -> SOD123; symbol traction-r1:R -> traction-r1:D; MPN R0805-100R -> BZT52-C5V1
- DWLS1: renamed from DWLSB; value BAT64-04 -> US1M; footprint SOT23 -> SMA; LCSC CLASS -> C412437; MPN BAT64-04 -> US1M
- DWLS2: renamed from DWLZ1; value BZT52-C18 -> US1M; footprint SOD123 -> SMA; LCSC CLASS -> C412437; MPN BZT52-C18 -> US1M
- DWLSB: renamed from DWLZ2; value BZT52-C5V1 -> BAT64-04; footprint SOD123 -> SOT23; MPN BZT52-C5V1 -> BAT64-04
- DWLZ1: renamed from RWLBL; value 5.1k -> BZT52-C18; footprint R0805 -> SOD123; symbol traction-r1:R -> traction-r1:D; MPN R0805-5k1 -> BZT52-C18
- DWLZ2: renamed from RWLDS; value 100R -> BZT52-C5V1; footprint R0805 -> SOD123; symbol traction-r1:R -> traction-r1:D; MPN R0805-100R -> BZT52-C5V1
- DWTP: renamed from RWTS; value 100R -> PESD5V0U1UA; footprint R0603 -> SOD323; symbol traction-r1:R -> traction-r1:D; MPN R0603-100R -> PESD5V0U1UA
- FH1: renamed from RGDLE; value 100k -> MF-LSMF300/24X-2; footprint R0603 -> PTC2920; symbol traction-r1:R -> traction-r1:F; LCSC CLASS -> C719172; MPN R0603-CLASS -> MF-LSMF300/24X-2
- FL1: renamed from CB15O1; value 22uF -> MF-LSMF300/24X-2; footprint C1210 -> PTC2920; symbol traction-r1:C -> traction-r1:F; LCSC CLASS -> C719172; MPN MLCC-22uF-25V -> MF-LSMF300/24X-2
- JIC: renamed from RPD8; value 10k -> MICROFIT3-40; footprint R0603 -> MicroFit40; symbol traction-r1:R -> traction-r1:MICROFIT3-40; MPN R0603-10k -> MICROFIT3-40
- JMV: renamed from RVTS; value 100R -> STUD-M8; footprint R0603 -> StudM8; symbol traction-r1:R -> traction-r1:TERM_1; MPN R0603-100R -> STUD-M8
- JMW: renamed from UWHG; value NSI6611ASC-Q1SWR -> STUD-M8; footprint SOIC16W -> StudM8; symbol traction-r1:NSI6611ASC-Q1SWR -> traction-r1:TERM_1; LCSC C7470934 -> CLASS; MPN NSI6611ASC-Q1SWR -> STUD-M8
- LB15: renamed from RPD10; value 10k -> XAL4040-103MEC; footprint R0603 -> XAL4040; symbol traction-r1:R -> traction-r1:L; MPN R0603-10k -> XAL4040-103MEC
- LFH1: renamed from UB15; value TPS55340QRTERQ1 -> FB-120R-3A; footprint WQFN16 -> FB1206; symbol traction-r1:TPS55340QRTERQ1 -> traction-r1:L; LCSC C2070860 -> CLASS; MPN TPS55340QRTERQ1 -> FB-120R-3A
- LFL1: renamed from CB15O2; value 22uF -> FB-120R-3A; footprint C1210 -> FB1206; symbol traction-r1:C -> traction-r1:L; MPN MLCC-22uF-25V -> FB-120R-3A
- MODV: renamed from CVSN; value 1uF -> HCS600FH120D3C1; footprint FilmP27.5 -> EconoDUAL3; symbol traction-r1:C -> traction-r1:HCS600FH120D3C1; MPN FILM-1uF-1200V -> HCS600FH120D3C1
- MODW: renamed from CWTF; value 2.2nF -> HCS600FH120D3C1; footprint C0603 -> EconoDUAL3; symbol traction-r1:C -> traction-r1:HCS600FH120D3C1; MPN MLCC-2.2nF-50V -> HCS600FH120D3C1
- PS5B: renamed from RASCL; value 470R -> MGJ2D150505SC; footprint R0603 -> SIP7; symbol traction-r1:R -> traction-r1:MGJ2D150505SC; MPN R0603-470R -> MGJ2D150505SC
- PS5C: renamed from RASCPD; value 10k -> MGJ2D150505SC; footprint R0603 -> SIP7; symbol traction-r1:R -> traction-r1:MGJ2D150505SC; MPN R0603-10k -> MGJ2D150505SC
- PSASC: renamed from DRH; value NRVBAF360T3G -> QA01C-18; footprint SMA-flat -> SIP7; symbol traction-r1:D -> traction-r1:QA01C-18; MPN NRVBAF360T3G -> QA01C-18
- QFH: renamed from TFH1; value VGT12EEM-200S1A4 -> BUK7Y14-80E; footprint XfmrEE12 -> LFPAK56; symbol traction-r1:VGT12EEM-200S1A4 -> traction-r1:BUK7Y14-80E; LCSC CLASS -> C86732; MPN VGT12EEM-200S1A4 -> BUK7Y14-80E
- QFHE1: renamed from TFH2; value VGT12EEM-200S1A4 -> 2N7002; footprint XfmrEE12 -> SOT23; symbol traction-r1:VGT12EEM-200S1A4 -> traction-r1:2N7002; LCSC CLASS -> C8545; MPN VGT12EEM-200S1A4 -> 2N7002
- QFHE2: renamed from TFH3; value VGT12EEM-200S1A4 -> 2N7002; footprint XfmrEE12 -> SOT23; symbol traction-r1:VGT12EEM-200S1A4 -> traction-r1:2N7002; LCSC CLASS -> C8545; MPN VGT12EEM-200S1A4 -> 2N7002
- renumbered CVBDF to CVDDF, DVHS1 to DVHR, DVHS2 to DVHS1, DVLS1 to DVLR, DVLS2 to DVLS1, DWHS2 to DWHR, DWLS2 to DWLR, RVBD1 to RVDD1, RVBD2 to RVDD2, RVBD3 to RVDD3, RVBD4 to RVDD4, RVBD5 to RVDD5, RVBD6 to RVDD6, RVBDL to RVDDL, UIVB to UIVDC
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Connections:
- net labels added: ASCP_UL, ASCP_VL, ASCP_WL, FFD_H, FFD_L, FFS_H, FFS_L
- wire segments 813 -> 835
Other:
- note added: "rev A.7 - 24 sections - 306 components"
- note removed: "rev A.6 - 24 sections - 295 components"
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