File: kicad5/traction/traction-power.sch (KiCad schematic (older format))
At the start: 313 parts, among them U5LB NCV4276CDT50RKG, U5LC NCV4276CDT50RKG

Commit message: Rev A.12: round 13 rechecks (F135-F139), pin freeze (F140), barrier + orderability closure (F141-F142), Marine A.12, firmware
- Rechecks of 30ae0a2: §6 winding-energy rule at every speed; resolver 12 k series + 220 pF C_AAF
  (injection 2.92 mA with the MCU unpowered); verifier counts distinct assemblies; TPS55340-Q1 real
  ratings (38/40 V); NCV4276C thermal on the datasheet pad.
- MCU pin freeze: all 289 S32K396 balls bound from SPF-91122 rev C anchored on the DS supply balls
  (calculations/mcu-ballmap.json, docs/mcu-pin-manifest.md); seven port corrections; FS26 pins verified;
  ERC pin-freeze lock.
- Barrier closure: VOW3120-X017T optos and UCC14141-Q1 biases (shared IsoBias18 cell, single-output
  18.0 V) replace TLP152/QA01C-18; LED resistors 270 R; VY1 Y-caps; Samtec IPL1/IPD1 harness;
  Faratronic 4XX can; SQP10 discharge resistors; UCC12051-Q1 on the AVL.
- Tooling: ERC open-pin helper + HARNESS40 parser scoped to its block; kicad5-verify assembly-set guard.
- Marine ported to A.12 (86 PASS / 22 WARN / 0 FAIL); firmware/ (C11, 178 tests / 1209 checks).
- Docs: README, design-basis §6a/§8/§11l, dfm, variants, cost-rollup, EXTRACTED-PARAMS §27-30 +
  seven archived datasheets, review-A12-disposition (+CSV), regenerated sheets/PDFs/BOMs/previews.

ERC 933/0 · design-verify 123/19/0 · sim 23/6/0 · sheets 2027/2027.

Co-Authored-By: Claude Fable 5.1 <noreply@anthropic.com>
Parts:
- added RPD10, RPD2, RPD3, RPD4, RPD5, RPD6, RPD7, RPD8, RPD9: 10k, R0603, symbol traction-r1:R
- C5G1: renamed from CB15O2; value 22uF -> 1uF; footprint C1210 -> C0805; MPN MLCC-22uF-50V -> MLCC-1uF-50V
- C5G2: renamed from CB15S; value 47nF -> 10uF; footprint C0603 -> C1206; MPN MLCC-CLASS -> MLCC-10uF-25V
- CASCF: renamed from DASCR; value 1N4148WS -> 330pF; footprint SOD323 -> C0603; symbol traction-r1:D -> traction-r1:C; LCSC C2128 -> CLASS; MPN 1N4148WS -> MLCC-330pF-50V-C0G
- CASCI1: renamed from RASCG; value 2.2k -> 10uF; footprint R0603 -> C1206; symbol traction-r1:R -> traction-r1:C; MPN ESR03EZPF2201 -> MLCC-10uF-25V-X7R
- CASCI2: renamed from RASCL; value 261R -> 10uF; footprint R0603 -> C1206; symbol traction-r1:R -> traction-r1:C; MPN R0603-261R-1% -> MLCC-10uF-25V-X7R
- CASCIB: renamed from RASCPD; value 10k -> 100nF; footprint R0603 -> C0603; symbol traction-r1:R -> traction-r1:C; MPN R0603-10k -> MLCC-100nF-50V
- CASCO: renamed from ZASC; value BZT52-C5V1 -> 10uF; footprint SOD123 -> C1210; symbol traction-r1:D -> traction-r1:C; MPN BZT52-C5V1 -> MLCC-10uF-50V
- CB15C: renamed from LB15; value XAL4040-103MEC -> 470pF; footprint XAL4040 -> C0603; symbol traction-r1:L -> traction-r1:C; MPN XAL4040-103MEC -> MLCC-CLASS
- CB15CC: renamed from RB15C; value 2k -> 100nF; footprint R0603 -> C0603; symbol traction-r1:R -> traction-r1:C; MPN R0603-CLASS -> MLCC-CLASS
- CB15I: renamed from RB15F1; value 110k -> 10uF; footprint R0603 -> C1210; symbol traction-r1:R -> traction-r1:C; MPN R0603-1% -> MLCC-10uF-50V
- CB15O1: renamed from RB15F2; value 9.53k -> 22uF; footprint R0603 -> C1210; symbol traction-r1:R -> traction-r1:C; MPN R0603-1% -> MLCC-22uF-50V
- CB15O2: renamed from RB15Q; value 80.6k -> 22uF; footprint R0603 -> C1210; symbol traction-r1:R -> traction-r1:C; MPN R0603-CLASS -> MLCC-22uF-50V
- CB15S: renamed from RLD1; value 49.9k -> 47nF; footprint R0603 -> C0603; symbol traction-r1:R -> traction-r1:C; MPN R0603-CLASS -> MLCC-CLASS
- CLD15: renamed from RLD2; value 10k -> 22uF; footprint R0603 -> C0603; symbol traction-r1:R -> traction-r1:C; MPN R0603-CLASS -> MLCC-CLASS
- CLDC: renamed from JIC; value HARNESS-2x20 -> 220pF; footprint MicroFit40 -> C0603; symbol traction-r1:HARNESS-2x20-CLASS -> traction-r1:C; MPN HARNESS-2x20-CLASS -> MLCC-CLASS
- CLVH1: renamed from DTVL; value TPSMC24CA-VR -> 4.7uF; footprint SMC -> C1206; symbol traction-r1:D -> traction-r1:C; LCSC C1975284 -> CLASS; MPN TPSMC24CA-VR -> MLCC-4.7uF-50V
- CLVH2: renamed from FL1; value MF-LSMF300/24X-2 -> 4.7uF; footprint PTC2920 -> C1206; symbol traction-r1:F -> traction-r1:C; LCSC C719172 -> CLASS; MPN MF-LSMF300/24X-2 -> MLCC-4.7uF-50V
- CLVL1: renamed from RGDLE; value 100k -> 4.7uF; footprint R0603 -> C1206; symbol traction-r1:R -> traction-r1:C; MPN R0603-CLASS -> MLCC-4.7uF-50V
- CLVL2: renamed from UB15; value TPS55340QRTERQ1 -> 4.7uF; footprint WQFN16 -> C1206; symbol traction-r1:TPS55340QRTERQ1 -> traction-r1:C; LCSC C2070860 -> CLASS; MPN TPS55340QRTERQ1 -> MLCC-4.7uF-50V
- CY1, CY2: MPN Y1-4.7nF-500VAC -> VY1472M63Y5UQ6TV0
- DASCR: renamed from CLVH1; value 4.7uF -> 1N4148WS; footprint C1206 -> SOD323; symbol traction-r1:C -> traction-r1:D; LCSC CLASS -> C2128; MPN MLCC-4.7uF-50V -> 1N4148WS
- DB15: renamed from RHWID; value 10k -> SS34; footprint R0603 -> SMA; symbol traction-r1:R -> traction-r1:D; MPN R0603-10k-1% -> SS34
- DRH: renamed from LFL1; value FB-120R-3A -> NRVBAF360T3G; footprint FB1206 -> SMA-flat; symbol traction-r1:L -> traction-r1:D; MPN FB-120R-3A -> NRVBAF360T3G
- DRL: renamed from ULDO15; value NCV4276CDTADJRKG -> NRVBAF360T3G; footprint DPAK5 -> SMA-flat; symbol traction-r1:NCV4276CDTADJRKG -> traction-r1:D; MPN NCV4276CDTADJRKG -> NRVBAF360T3G
- DTVH: renamed from UGDL; value NCV4276CDT50RKG -> TPSMC24CA-VR; footprint DPAK -> SMC; symbol traction-r1:NCV4276CDT50RKG -> traction-r1:D; LCSC CLASS -> C1975284; MPN NCV4276CDT50RKG -> TPSMC24CA-VR
- DTVL: renamed from CB15C; value 470pF -> TPSMC24CA-VR; footprint C0603 -> SMC; symbol traction-r1:C -> traction-r1:D; LCSC CLASS -> C1975284; MPN MLCC-CLASS -> TPSMC24CA-VR
- FH1: renamed from C5G1; value 1uF -> MF-LSMF300/24X-2; footprint C0805 -> PTC2920; symbol traction-r1:C -> traction-r1:F; LCSC CLASS -> C719172; MPN MLCC-1uF-50V -> MF-LSMF300/24X-2
- FL1: renamed from CB15CC; value 100nF -> MF-LSMF300/24X-2; footprint C0603 -> PTC2920; symbol traction-r1:C -> traction-r1:F; LCSC CLASS -> C719172; MPN MLCC-CLASS -> MF-LSMF300/24X-2
- JIC: renamed from RPD6; value 10k -> IPL1-120-01-L-D-K; footprint R0603 -> HDR2x20-2.54; symbol traction-r1:R -> traction-r1:IPL1-120-01-L-D-K; MPN R0603-10k -> IPL1-120-01-L-D-K
- LB15: renamed from RPD0; value 10k -> XAL4040-103MEC; footprint R0603 -> XAL4040; symbol traction-r1:R -> traction-r1:L; MPN R0603-10k -> XAL4040-103MEC
- LFH1: renamed from C5G2; value 10uF -> FB-120R-3A; footprint C1206 -> FB1206; symbol traction-r1:C -> traction-r1:L; MPN MLCC-10uF-25V -> FB-120R-3A
- LFL1: renamed from CB15I; value 10uF -> FB-120R-3A; footprint C1210 -> FB1206; symbol traction-r1:C -> traction-r1:L; MPN MLCC-10uF-50V -> FB-120R-3A
- PSASC: value QA01C-18 -> UCC14141QDWNRQ1; footprint SIP7 -> DWN36; symbol traction-r1:QA01C-18 -> traction-r1:UCC14141QDWNRQ1; MPN QA01C-18 -> UCC14141QDWNRQ1
- RASCE1: renamed from CLVH2; value 4.7uF -> 10k; footprint C1206 -> R0603; symbol traction-r1:C -> traction-r1:R; MPN MLCC-4.7uF-50V -> R0603-10k
- RASCE2: renamed from DRH; value NRVBAF360T3G -> 4.7k; footprint SMA-flat -> R0603; symbol traction-r1:D -> traction-r1:R; MPN NRVBAF360T3G -> R0603-4k7
- RASCF1: renamed from DTVH; value TPSMC24CA-VR -> 62k; footprint SMC -> R0603; symbol traction-r1:D -> traction-r1:R; LCSC C1975284 -> CLASS; MPN TPSMC24CA-VR -> R0603-62k-1%
- RASCF2: renamed from FH1; value MF-LSMF300/24X-2 -> 10k; footprint PTC2920 -> R0603; symbol traction-r1:F -> traction-r1:R; LCSC C719172 -> CLASS; MPN MF-LSMF300/24X-2 -> R0603-10k-1%
- RASCG: renamed from LFH1; value FB-120R-3A -> 2.2k; footprint FB1206 -> R0603; symbol traction-r1:L -> traction-r1:R; MPN FB-120R-3A -> ESR03EZPF2201
- RASCL: renamed from CLVL1; value 4.7uF -> 270R; footprint C1206 -> R0603; symbol traction-r1:C -> traction-r1:R; MPN MLCC-4.7uF-50V -> R0603-270R-1%
- RASCPD: renamed from CLVL2; value 4.7uF -> 10k; footprint C1206 -> R0603; symbol traction-r1:C -> traction-r1:R; MPN MLCC-4.7uF-50V -> R0603-10k
- RB15C: renamed from RPD1; value 10k -> 2k; MPN R0603-10k -> R0603-CLASS
- RB15F1: renamed from RPD10; value 10k -> 110k; MPN R0603-10k -> R0603-1%
- RB15F2: renamed from RPD2; value 10k -> 9.53k; MPN R0603-10k -> R0603-1%
- RB15Q: renamed from RPD3; value 10k -> 80.6k; MPN R0603-10k -> R0603-CLASS
- RGDLE: renamed from CLD15; value 22uF -> 100k; footprint C0603 -> R0603; symbol traction-r1:C -> traction-r1:R; MPN MLCC-CLASS -> R0603-CLASS
- RHWID: renamed from RPD7; MPN R0603-10k -> R0603-10k-1%
- RLD1: renamed from RPD4; value 10k -> 49.9k; MPN R0603-10k -> R0603-CLASS
- RLD2: renamed from RPD5; MPN R0603-10k -> R0603-CLASS
- UASC: value TLP152 -> VOW3120-X017T; footprint SO6 -> SMD8W; symbol traction-r1:TLP152 -> traction-r1:VOW3120-X017T; LCSC C17255258 -> CLASS; MPN TLP152 -> VOW3120-X017T
- UB15: renamed from CLDC; value 220pF -> TPS55340QRTERQ1; footprint C0603 -> WQFN16; symbol traction-r1:C -> traction-r1:TPS55340QRTERQ1; LCSC CLASS -> C2070860; MPN MLCC-CLASS -> TPS55340QRTERQ1
- UGDL: renamed from CB15O1; value 22uF -> NCV4276CDT50RKG; footprint C1210 -> DPAK; symbol traction-r1:C -> traction-r1:NCV4276CDT50RKG; MPN MLCC-22uF-50V -> NCV4276CDT50RKG
- ULDO15: renamed from DB15; value SS34 -> NCV4276CDTADJRKG; footprint SMA -> DPAK5; symbol traction-r1:D -> traction-r1:NCV4276CDTADJRKG; MPN SS34 -> NCV4276CDTADJRKG
- ZASC: renamed from DRL; value NRVBAF360T3G -> BZT52-C5V1; footprint SMA-flat -> SOD123; MPN NRVBAF360T3G -> BZT52-C5V1
- renumbered RPD8 to RPD0, RPD9 to RPD1
Connections:
- net labels added: ENA_ASC, FB_ASC
- wire segments 875 -> 923
Other:
- note added: "rev A.12 - 24 sections - 322 components"
- note removed: "rev A.11 - 24 sections - 313 components"
- moved on the sheet: C5G1, C5G2, CASC, CASCD, CB15C, CLVH2, FH1, FL1, LFH1, LFL1, RB15C, RB15F1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
