File: kicad5/traction/traction-power.sch (KiCad schematic (older format))
At the start: 322 parts, among them U5LB NCV4276CDT50RKG, U5LC NCV4276CDT50RKG

Commit message: Rev A.13: round 14 — three reviews of cfd35a7 (F143-F158): MCU map vs NXP netlist, fail-closed firmware, terminal-fault protection
- Pin freeze reopened and closed: H5 is V15 (1.5 V, was on VREF5) and J7 is V25 (regulator output,
  was grounded); whole map re-derived against NXP's GEN3 net report NET-91122_C (U513, 244 balls) —
  every supply ball and 164/165 port names agree; HW_ID/NTC_A/MT2_SIG/ASC_REQ moved to netlist-confirmed
  balls (B5/T15/D5/U4); KiCad symbol numbered by physical ball, mutation-tested; CNMOS 1 nF.
- Firmware (214 tests / 1622 checks, ASan/UBSan, target-check): DESAT hold for every caller, 64-bit
  monotonic clock, keep_hv from rule (b) reliance at any speed, IMCR placeholders = build error,
  config-matches vs protection-locked, arming-evidence record (fail closed), torque feasibility witness,
  stuck-channel detection, stuck-on discharge detection; board map regenerated.
- Analog: excitation monitor 18 k/42.2 k/84.5 k + 220 pF C_AAF; exciter SMCJ8.5CA + MF-MSMF020 per line;
  motor-temp SMAJ5.0A + 0438.375WRA; bias-LDO 47 R ballast, UCC12051-Q1 primary; UCC14141-Q1 VDE cert.
- Docs: contract FW-22..FW-26 + keep_hv; design-basis §11m; variants/cost/dfm/README; disposition + CSV;
  EXTRACTED §31/§32 + archived datasheets; report-template defect fixed; Marine at A.13 (86/22/0).

ERC 945/0 · design-verify 130/23/0 · sim 23/6/0 · sheets 2045/2045 · BOM 8XX SiC ₹72,492.

Co-Authored-By: Claude Fable 5.1 <noreply@anthropic.com>
Parts:
- added RPD8, RPD9: 10k, R0603, symbol traction-r1:R
- C5G1: renamed from RGDLE; value 100k -> 1uF; footprint R0603 -> C0805; symbol traction-r1:R -> traction-r1:C; MPN R0603-CLASS -> MLCC-1uF-50V
- C5G2: renamed from UB15; value TPS55340QRTERQ1 -> 10uF; footprint WQFN16 -> C1206; symbol traction-r1:TPS55340QRTERQ1 -> traction-r1:C; LCSC C2070860 -> CLASS; MPN TPS55340QRTERQ1 -> MLCC-10uF-25V
- CASC: renamed from CASCF; value 330pF -> 100nF; MPN MLCC-330pF-50V-C0G -> MLCC-100nF-50V
- CASCD: renamed from CASCI1; value 10uF -> 12nF; footprint C1206 -> C0603; MPN MLCC-10uF-25V-X7R -> MLCC-12nF-50V-C0G
- CASCF: renamed from CASCI2; value 10uF -> 330pF; footprint C1206 -> C0603; MPN MLCC-10uF-25V-X7R -> MLCC-330pF-50V-C0G
- CASCI1: renamed from CASCIB; value 100nF -> 10uF; footprint C0603 -> C1206; MPN MLCC-100nF-50V -> MLCC-10uF-25V-X7R
- CASCI2: renamed from CASCO; footprint C1210 -> C1206; MPN MLCC-10uF-50V -> MLCC-10uF-25V-X7R
- CASCIB: renamed from DASCR; value 1N4148WS -> 100nF; footprint SOD323 -> C0603; symbol traction-r1:D -> traction-r1:C; LCSC C2128 -> CLASS; MPN 1N4148WS -> MLCC-100nF-50V
- CASCO: renamed from RASCE1; value 10k -> 10uF; footprint R0603 -> C1210; symbol traction-r1:R -> traction-r1:C; MPN R0603-10k -> MLCC-10uF-50V
- CB15C: renamed from CB15I; value 10uF -> 470pF; footprint C1210 -> C0603; MPN MLCC-10uF-50V -> MLCC-CLASS
- CB15CC: renamed from CB15O1; value 22uF -> 100nF; footprint C1210 -> C0603; MPN MLCC-22uF-50V -> MLCC-CLASS
- CB15I: renamed from CB15O2; value 22uF -> 10uF; MPN MLCC-22uF-50V -> MLCC-10uF-50V
- CB15O1: renamed from CB15S; value 47nF -> 22uF; footprint C0603 -> C1210; MPN MLCC-CLASS -> MLCC-22uF-50V
- CB15O2: renamed from CLD15; footprint C0603 -> C1210; MPN MLCC-CLASS -> MLCC-22uF-50V
- CB15S: renamed from CLDC; value 220pF -> 47nF
- CLD15: renamed from DB15; value SS34 -> 22uF; footprint SMA -> C0603; symbol traction-r1:D -> traction-r1:C; MPN SS34 -> MLCC-CLASS
- CLDC: renamed from LB15; value XAL4040-103MEC -> 220pF; footprint XAL4040 -> C0603; symbol traction-r1:L -> traction-r1:C; MPN XAL4040-103MEC -> MLCC-CLASS
- CLVH1: renamed from DRH; value NRVBAF360T3G -> 4.7uF; footprint SMA-flat -> C1206; symbol traction-r1:D -> traction-r1:C; MPN NRVBAF360T3G -> MLCC-4.7uF-50V
- CLVH2: renamed from DTVH; value TPSMC24CA-VR -> 4.7uF; footprint SMC -> C1206; symbol traction-r1:D -> traction-r1:C; LCSC C1975284 -> CLASS; MPN TPSMC24CA-VR -> MLCC-4.7uF-50V
- CLVL1: renamed from DRL; value NRVBAF360T3G -> 4.7uF; footprint SMA-flat -> C1206; symbol traction-r1:D -> traction-r1:C; MPN NRVBAF360T3G -> MLCC-4.7uF-50V
- CLVL2: renamed from DTVL; value TPSMC24CA-VR -> 4.7uF; footprint SMC -> C1206; symbol traction-r1:D -> traction-r1:C; LCSC C1975284 -> CLASS; MPN TPSMC24CA-VR -> MLCC-4.7uF-50V
- DASCR: renamed from RASCE2; value 4.7k -> 1N4148WS; footprint R0603 -> SOD323; symbol traction-r1:R -> traction-r1:D; LCSC CLASS -> C2128; MPN R0603-4k7 -> 1N4148WS
- DB15: renamed from RB15C; value 2k -> SS34; footprint R0603 -> SMA; symbol traction-r1:R -> traction-r1:D; MPN R0603-CLASS -> SS34
- DRH: renamed from FH1; value MF-LSMF300/24X-2 -> NRVBAF360T3G; footprint PTC2920 -> SMA-flat; symbol traction-r1:F -> traction-r1:D; LCSC C719172 -> CLASS; MPN MF-LSMF300/24X-2 -> NRVBAF360T3G
- DRL: renamed from FL1; value MF-LSMF300/24X-2 -> NRVBAF360T3G; footprint PTC2920 -> SMA-flat; symbol traction-r1:F -> traction-r1:D; LCSC C719172 -> CLASS; MPN MF-LSMF300/24X-2 -> NRVBAF360T3G
- DTVH: renamed from LFH1; value FB-120R-3A -> TPSMC24CA-VR; footprint FB1206 -> SMC; symbol traction-r1:L -> traction-r1:D; LCSC CLASS -> C1975284; MPN FB-120R-3A -> TPSMC24CA-VR
- DTVL: renamed from LFL1; value FB-120R-3A -> TPSMC24CA-VR; footprint FB1206 -> SMC; symbol traction-r1:L -> traction-r1:D; LCSC CLASS -> C1975284; MPN FB-120R-3A -> TPSMC24CA-VR
- FH1: renamed from CLVL1; value 4.7uF -> MF-LSMF300/24X-2; footprint C1206 -> PTC2920; symbol traction-r1:C -> traction-r1:F; LCSC CLASS -> C719172; MPN MLCC-4.7uF-50V -> MF-LSMF300/24X-2
- FL1: renamed from UGDL; value NCV4276CDT50RKG -> MF-LSMF300/24X-2; footprint DPAK -> PTC2920; symbol traction-r1:NCV4276CDT50RKG -> traction-r1:F; LCSC CLASS -> C719172; MPN NCV4276CDT50RKG -> MF-LSMF300/24X-2
- JIC: renamed from RPD0; value 10k -> IPL1-120-01-L-D-K; footprint R0603 -> HDR2x20-2.54; symbol traction-r1:R -> traction-r1:IPL1-120-01-L-D-K; MPN R0603-10k -> IPL1-120-01-L-D-K
- LB15: renamed from RB15F1; value 110k -> XAL4040-103MEC; footprint R0603 -> XAL4040; symbol traction-r1:R -> traction-r1:L; MPN R0603-1% -> XAL4040-103MEC
- LFH1: renamed from CLVL2; value 4.7uF -> FB-120R-3A; footprint C1206 -> FB1206; symbol traction-r1:C -> traction-r1:L; MPN MLCC-4.7uF-50V -> FB-120R-3A
- LFL1: renamed from C5G1; value 1uF -> FB-120R-3A; footprint C0805 -> FB1206; symbol traction-r1:C -> traction-r1:L; MPN MLCC-1uF-50V -> FB-120R-3A
- PS5B, PS5C: value UCC12050DVER -> UCC12051QDVERQ1; symbol traction-r1:UCC12050DVER -> traction-r1:UCC12051QDVERQ1; MPN UCC12050DVER -> UCC12051QDVERQ1
- PSASC: renamed from CASC; value 100nF -> UCC14141QDWNRQ1; footprint C0603 -> DWN36; symbol traction-r1:C -> traction-r1:UCC14141QDWNRQ1; MPN MLCC-100nF-50V -> UCC14141QDWNRQ1
- R5LB: renamed from PSASC; value UCC14141QDWNRQ1 -> 47R; footprint DWN36 -> R2512; symbol traction-r1:UCC14141QDWNRQ1 -> traction-r1:R; MPN UCC14141QDWNRQ1 -> R2512-47R-1%-1W
- R5LC: renamed from UASC; value VOW3120-X017T -> 47R; footprint SMD8W -> R2512; symbol traction-r1:VOW3120-X017T -> traction-r1:R; MPN VOW3120-X017T -> R2512-47R-1%-1W
- RASCE1: renamed from RASCF1; value 62k -> 10k; MPN R0603-62k-1% -> R0603-10k
- RASCE2: renamed from RASCF2; value 10k -> 4.7k; MPN R0603-10k-1% -> R0603-4k7
- RASCF1: renamed from RASCG; value 2.2k -> 62k; MPN ESR03EZPF2201 -> R0603-62k-1%
- RASCF2: renamed from RASCL; value 270R -> 10k; MPN R0603-270R-1% -> R0603-10k-1%
- RASCG: renamed from RASCPD; value 10k -> 2.2k; MPN R0603-10k -> ESR03EZPF2201
- RASCL: renamed from ZASC; value BZT52-C5V1 -> 270R; footprint SOD123 -> R0603; symbol traction-r1:D -> traction-r1:R; MPN BZT52-C5V1 -> R0603-270R-1%
- RASCPD: renamed from CLVH1; value 4.7uF -> 10k; footprint C1206 -> R0603; symbol traction-r1:C -> traction-r1:R; MPN MLCC-4.7uF-50V -> R0603-10k
- RB15C: renamed from RB15F2; value 9.53k -> 2k; MPN R0603-1% -> R0603-CLASS
- RB15F1: renamed from RB15Q; value 80.6k -> 110k; MPN R0603-CLASS -> R0603-1%
- RB15F2: renamed from RLD1; value 49.9k -> 9.53k; MPN R0603-CLASS -> R0603-1%
- RB15Q: renamed from RLD2; value 10k -> 80.6k
- RGDLE: renamed from ULDO15; value NCV4276CDTADJRKG -> 100k; footprint DPAK5 -> R0603; symbol traction-r1:NCV4276CDTADJRKG -> traction-r1:R; MPN NCV4276CDTADJRKG -> R0603-CLASS
- RHWID: renamed from RPD1; MPN R0603-10k -> R0603-10k-1%
- RLD1: renamed from JIC; value IPL1-120-01-L-D-K -> 49.9k; footprint HDR2x20-2.54 -> R0603; symbol traction-r1:IPL1-120-01-L-D-K -> traction-r1:R; MPN IPL1-120-01-L-D-K -> R0603-CLASS
- RLD2: renamed from RHWID; MPN R0603-10k-1% -> R0603-CLASS
- UASC: renamed from CASCD; value 12nF -> VOW3120-X017T; footprint C0603 -> SMD8W; symbol traction-r1:C -> traction-r1:VOW3120-X017T; MPN MLCC-12nF-50V-C0G -> VOW3120-X017T
- UB15: renamed from CB15C; value 470pF -> TPS55340QRTERQ1; footprint C0603 -> WQFN16; symbol traction-r1:C -> traction-r1:TPS55340QRTERQ1; LCSC CLASS -> C2070860; MPN MLCC-CLASS -> TPS55340QRTERQ1
- UGDL: renamed from C5G2; value 10uF -> NCV4276CDT50RKG; footprint C1206 -> DPAK; symbol traction-r1:C -> traction-r1:NCV4276CDT50RKG; MPN MLCC-10uF-25V -> NCV4276CDT50RKG
- ULDO15: renamed from CB15CC; value 100nF -> NCV4276CDTADJRKG; footprint C0603 -> DPAK5; symbol traction-r1:C -> traction-r1:NCV4276CDTADJRKG; MPN MLCC-CLASS -> NCV4276CDTADJRKG
- ZASC: renamed from CLVH2; value 4.7uF -> BZT52-C5V1; footprint C1206 -> SOD123; symbol traction-r1:C -> traction-r1:D; MPN MLCC-4.7uF-50V -> BZT52-C5V1
- renumbered RPD10 to RPD0, RPD2 to RPD1, RPD3 to RPD10, RPD4 to RPD2, RPD5 to RPD3, RPD6 to RPD4, RPD7 to RPD5, RPD8 to RPD6, RPD9 to RPD7
Connections:
- net labels added: V15LB, V15LC
- wire segments 923 -> 927
Other:
- note added: "rev A.13 - 24 sections - 324 components"
- note removed: "rev A.12 - 24 sections - 322 components"
- moved on the sheet: CASC, CASCD, CASCF, CASCI1, CASCI2, CB15C, CB15CC, CB15I, CB15O1, CB15O2, CB15S, CLDC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
