File: kicad5/traction/traction-disch.sch (KiCad schematic (older format))
At the start: 24 parts

Commit message: Add cap-bank busbar assembly sheet + explicit interboard links (4 sheets)
- boards/capbank.tsx: the 16-can DC-link is its own laminated-busbar
  assembly (FR4 cannot carry the 340 A bus) with every terminal drawn:
  entry lugs, 3x module DC tab pairs, discharge-board studs
- power board keeps only its DCP/DCN entry taps (Y-caps, HVIL, sense)
- interboard links L1-L5 (harness, discharge 4-way, busbar, LEM, HVIL)
  documented in design-basis 10a + README table; erc-audit now asserts
  both ends of every link (new interboard section)
- NET NAMING panels state the cross-sheet net rule on every sheet
- gates green: 1560/1560 pins, ERC 687/0, design-verify 51P/3W/0F
- BOM ₹69,996 @1k (58,575 / 4,940 / 672 / 5,808) · 543 comps · 175 lines

Co-Authored-By: Claude Fable 5 <noreply@anthropic.com>
Parts:
- removed JCTL: HDR-1x4-2.54, HDR1x4, symbol traction-r1:HDR-1x4-2.54
- removed JDCN, JDCP: STUD-M6, StudM6, symbol traction-r1:TERM_1
- removed RBLD1, RBLD10, RBLD2, RBLD3, RBLD4, RBLD5, RBLD6: 27k, R2512, symbol traction-r1:R
- added CQD: 100nF, C0603, symbol traction-r1:C
- added QDIS: HCM75S12T4K3, TO247-4L, symbol traction-r1:HCM75S12T4K3
- added RDIS1, RDIS2, RDIS3, RDIS4: 470R, AxialWW10W, symbol traction-r1:R
- added RQDG: 47R, R0603, symbol traction-r1:R
- added RQDL: 470R, R0603, symbol traction-r1:R
- added RQDPD: 10k, R0603, symbol traction-r1:R
- added UQD: TLP152, SO6, symbol traction-r1:TLP152
- JCTL: renamed from RBLD7; value 27k -> HDR-1x4-2.54; footprint R2512 -> HDR1x4; symbol traction-r1:R -> traction-r1:HDR-1x4-2.54; MPN R2512-27k-2W -> HDR-1x4-2.54
- JDCN: renamed from RBLD8; value 27k -> STUD-M6; footprint R2512 -> StudM6; symbol traction-r1:R -> traction-r1:TERM_1; MPN R2512-27k-2W -> STUD-M6
- JDCP: renamed from RBLD9; value 27k -> STUD-M6; footprint R2512 -> StudM6; symbol traction-r1:R -> traction-r1:TERM_1; MPN R2512-27k-2W -> STUD-M6
- PSQD: renamed from RQDPD; value 10k -> QA01C-18; footprint R0603 -> SIP7; symbol traction-r1:R -> traction-r1:QA01C-18; MPN R0603-10k -> QA01C-18
- RBLD1: renamed from PSQD; value QA01C-18 -> 27k; footprint SIP7 -> R2512; symbol traction-r1:QA01C-18 -> traction-r1:R; MPN QA01C-18 -> R2512-27k-2W
- RBLD10: renamed from QDIS; value HCM75S12T4K3 -> 27k; footprint TO247-4L -> R2512; symbol traction-r1:HCM75S12T4K3 -> traction-r1:R; MPN HCM75S12T4K3 -> R2512-27k-2W
- RBLD2: renamed from UQD; value TLP152 -> 27k; footprint SO6 -> R2512; symbol traction-r1:TLP152 -> traction-r1:R; LCSC C17255258 -> CLASS; MPN TLP152 -> R2512-27k-2W
- RBLD3: renamed from CQD; value 100nF -> 27k; footprint C0603 -> R2512; symbol traction-r1:C -> traction-r1:R; MPN MLCC-100nF-25V -> R2512-27k-2W
- RBLD4: renamed from RDIS1; value 470R -> 27k; footprint AxialWW10W -> R2512; MPN WW-470R-10W-AX -> R2512-27k-2W
- RBLD5: renamed from RDIS2; value 470R -> 27k; footprint AxialWW10W -> R2512; MPN WW-470R-10W-AX -> R2512-27k-2W
- RBLD6: renamed from RDIS3; value 470R -> 27k; footprint AxialWW10W -> R2512; MPN WW-470R-10W-AX -> R2512-27k-2W
- RBLD7: renamed from RDIS4; value 470R -> 27k; footprint AxialWW10W -> R2512; MPN WW-470R-10W-AX -> R2512-27k-2W
- RBLD8: renamed from RQDG; value 47R -> 27k; footprint R0603 -> R2512; MPN R0603-47R -> R2512-27k-2W
- RBLD9: renamed from RQDL; value 470R -> 27k; footprint R0603 -> R2512; MPN R0603-470R -> R2512-27k-2W
Other:
- note added: "220 kW pk Discharge (HV, bolt-on) - 3 of 4 · rev A.3 · 3 sections · 24 components"
- note added: "DISCHARGE / ACTIVE"
- note added: "DISCHARGE / BLEED"
- note added: "DISCHARGE / ENTRY"
- note added: "NET NAMING: U<ref>_<PIN> = node at that IC pin · R<stem>_M = series-pair midpoint · R<stem>_<nm> = tap between R<stem>n/m · all others are explicit design nets · same name on another sheet = same net, joined only at the named connector/stud/tab"
- note removed: "220 kW pk Discharge (HV, bolt-on) - 2 of 3 · rev A.3 · 3 sections · 24 components"
- note removed: "NET NAMING: U<ref>_<PIN> = node at that IC pin · R<stem>_M = series-pair midpoint · R<stem>_<nm> = tap between R<stem>n/m · all others are explicit design nets"
- note removed: "disch-DISCHARGE / ACTIVE"
- note removed: "disch-DISCHARGE / BLEED"
- note removed: "disch-DISCHARGE / ENTRY"
- moved on the sheet: RBLD4, RBLD5, RBLD6, RBLD7, RBLD8, RBLD9

Commit message: Rev A.4: answer external design review — 10 confirmed defects fixed (F37-F46)
Every claim verified against primary datasheets before any edit; three
claims rebutted with evidence (850V/0.1% divider corner, GEN3-exact
resolver monitors, discharge math matches). Fixed:

- F37 VGT12EEM secondary phasing: rectifier moved to pin 8 (dot); the
  drawn wiring was forward-mode ~35V into +22V-abs gates. Pins 6/7 NC'd
  (no internal winding). Aux (NF) was already correct.
- F38 flyback drain clamp: SMBJ85A (forward every OFF interval, 94.4V
  min breakdown vs 80V FET) -> US1M + SMAJ13A winding clamp; drain
  <=60V at clamped load dump
- F39 DESAT clamp: BAT64-04 series pair correctly oriented DESAT->VCC2
  (was VCC2 injected into DESAT via a wrong common-cathode symbol)
- F40 ASC latch: real SN74LVC1G74 DCU pins; 1k/10k network (was
  120R/120R = 2.5V "low" and 42mA MCU clear)
- F41 KL15: 47k/10k+100nF ADC sense (was raw 13.3V into PTA25)
- F42 VDC receivers offset +0.5V (buffered) - AMC1311 fail-safe now
  distinguishable from a dead bus
- F44 VBAT_H/L actually sourced (FVBH/FVBL polyfuses off NRC)
- F45 real package pins everywhere: 74LVC1G11 (had NO VCC pin), 1G32,
  NCV4276C (OUT=5), TPS55340 RTE16 (+SS cap +FREQ R), BUK9Y14 LFPAK56,
  ALM2402 PWP14 (+VCC_O, SHDN via 10k pullup), QA01C SIP-7, PESD as
  real 2/3-terminal parts, FS26 full LQFP-48+EP with VDIG/VBOS/
  bootstraps/DEBUG strap and DS unused-pin terminations; S32K396
  explicitly symbolic (no package table in DS - bind at layout)
- F46 hardware fault latch: FLT_HS/LS diode-OR -> LVC1G74 -> DRV_EN;
  any DESAT latches all six channels off until MCU clears
- NSI6611ASC-Q1SWR full ordering code (ASC variant)

erc-audit gains a rev-A.4 lock-in section (763 checks, 0 fail);
design-verify adds F37-F46 corner rows (60 PASS/3 WARN/0 FAIL);
pin-verify 1663/1663; card void gate 9->12% (49-pin FS26 monolith);
BOM Rs.70,059 @1k, 579 components, 180 lines. design-basis 11a
documents the full review response including the rege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
Parts:
- removed JCTL: HDR-1x4-2.54, HDR1x4, symbol traction-r1:HDR-1x4-2.54
- removed JDCN, JDCP: STUD-M6, StudM6, symbol traction-r1:TERM_1
- removed RBLD1, RBLD10, RBLD2, RBLD3, RBLD4, RBLD5, RBLD6, RBLD7: 27k, R2512, symbol traction-r1:R
- added CQD: 100nF, C0603, symbol traction-r1:C
- added PSQD: QA01C-18, SIP7, symbol traction-r1:QA01C-18
- added QDIS: HCM75S12T4K3, TO247-4L, symbol traction-r1:HCM75S12T4K3
- added RDIS1, RDIS2, RDIS3, RDIS4: 470R, AxialWW10W, symbol traction-r1:R
- added RQDG: 47R, R0603, symbol traction-r1:R
- added RQDL: 470R, R0603, symbol traction-r1:R
- added RQDPD: 10k, R0603, symbol traction-r1:R
- added UQD: TLP152, SO6, symbol traction-r1:TLP152
- JCTL: renamed from RBLD8; value 27k -> HDR-1x4-2.54; footprint R2512 -> HDR1x4; symbol traction-r1:R -> traction-r1:HDR-1x4-2.54; MPN R2512-27k-2W -> HDR-1x4-2.54
- JDCN: renamed from RBLD9; value 27k -> STUD-M6; footprint R2512 -> StudM6; symbol traction-r1:R -> traction-r1:TERM_1; MPN R2512-27k-2W -> STUD-M6
- JDCP: renamed from PSQD; value QA01C-18 -> STUD-M6; footprint SIP7 -> StudM6; symbol traction-r1:QA01C-18 -> traction-r1:TERM_1; MPN QA01C-18 -> STUD-M6
- RBLD1: renamed from QDIS; value HCM75S12T4K3 -> 27k; footprint TO247-4L -> R2512; symbol traction-r1:HCM75S12T4K3 -> traction-r1:R; MPN HCM75S12T4K3 -> R2512-27k-2W
- RBLD10: renamed from UQD; value TLP152 -> 27k; footprint SO6 -> R2512; symbol traction-r1:TLP152 -> traction-r1:R; LCSC C17255258 -> CLASS; MPN TLP152 -> R2512-27k-2W
- RBLD2: renamed from CQD; value 100nF -> 27k; footprint C0603 -> R2512; symbol traction-r1:C -> traction-r1:R; MPN MLCC-100nF-25V -> R2512-27k-2W
- RBLD3: renamed from RDIS1; value 470R -> 27k; footprint AxialWW10W -> R2512; MPN WW-470R-10W-AX -> R2512-27k-2W
- RBLD4: renamed from RDIS2; value 470R -> 27k; footprint AxialWW10W -> R2512; MPN WW-470R-10W-AX -> R2512-27k-2W
- RBLD5: renamed from RDIS3; value 470R -> 27k; footprint AxialWW10W -> R2512; MPN WW-470R-10W-AX -> R2512-27k-2W
- RBLD6: renamed from RDIS4; value 470R -> 27k; footprint AxialWW10W -> R2512; MPN WW-470R-10W-AX -> R2512-27k-2W
- RBLD7: renamed from RQDG; value 47R -> 27k; footprint R0603 -> R2512; MPN R0603-47R -> R2512-27k-2W
- RBLD8: renamed from RQDL; value 470R -> 27k; footprint R0603 -> R2512; MPN R0603-470R -> R2512-27k-2W
- RBLD9: renamed from RQDPD; value 10k -> 27k; footprint R0603 -> R2512; MPN R0603-10k -> R2512-27k-2W
Other:
- note added: "220 kW pk Discharge (HV, bolt-on) - 3 of 4 · rev A.4 · 3 sections · 24 components"
- note removed: "220 kW pk Discharge (HV, bolt-on) - 3 of 4 · rev A.3 · 3 sections · 24 components"
- moved on the sheet: RBLD3, RBLD4, RBLD5, RBLD6, RBLD7, RBLD8, RBLD9
Changed lines of the file:
@@
 Title "Traction Inverter — Discharge board (bolt-on, XM3 pattern)"
 Date "2026-09-09"
-Rev "A.3"
+Rev "A.4"
 Comp "Traction Inverter 220 kW pk - Discharge (HV, bolt-on), sheet 3 of 4"
 Comment1 "Inverter = Power board + Cap bank busbar + bolt-on Discharge board (all HV) + Control card (LV); safe state holds with any link lost"
@@
 $EndDescr
 Text Notes 600 7100 0    60   ~ 12
-220 kW pk Discharge (HV, bolt-on) - 3 of 4   ·   rev A.3   ·   3 sections   ·   24 components
+220 kW pk Discharge (HV, bolt-on) - 3 of 4   ·   rev A.4   ·   3 sections   ·   24 components
 Text Notes 600 7400 0    50   ~ 0
 NET NAMING: U<ref>_<PIN> = node at that IC pin   ·   R<stem>_M = series-pair midpoint   ·   R<stem>_<nm> = tap between R<stem>n/m   ·   all others are explicit design nets   ·   same name on another sheet = same net, joined only at the named connector/stud/tab
@@
 $Comp
 L traction-r1:HDR-1x4-2.54 JCTL
-U 1 1 5E00012D
+U 1 1 5E000138
 P 9150 2100
 F 0 "JCTL" H 8750 1800 50  0000 R CNN
@@
 $Comp
 L traction-r1:TERM_1 JDCN
-U 1 1 5E00012E
+U 1 1 5E000139
 P 8800 1550
 F 0 "JDCN" H 8800 1390 50  0000 C CNN
@@
 $Comp
 L traction-r1:TERM_1 JDCP
-U 1 1 5E00012F
+U 1 1 5E00013A
 P 8800 1150
 F 0 "JDCP" H 8800 990 50  0000 C CNN
@@
 $Comp
 L traction-r1:R RBLD1
-U 1 1 5E000130
+U 1 1 5E00013B
 P 8300 4400
 F 0 "RBLD1" H 8300 4240 50  0000 C CNN
@@
 $Comp
 L traction-r1:R RBLD10
-U 1 1 5E000131
+U 1 1 5E00013C
 P 9800 6000
 F 0 "RBLD10" H 9800 5840 50  0000 C CNN
@@
 $Comp
 L traction-r1:R RBLD2
-U 1 1 5E000132
+U 1 1 5E00013D
 P 8300 4800
 F 0 "RBLD2" H 8300 4640 50  0000 C CNN
@@
 $Comp
 L traction-r1:R RBLD3
-U 1 1 5E000133
+U 1 1 5E00013E
 P 8300 5200
 F 0 "RBLD3" H 8300 5040 50  0000 C CNN
@@
 $Comp
 L traction-r1:R RBLD4
-U 1 1 5E000134
+U 1 1 5E00013F
 P 8300 5600
 F 0 "RBLD4" H 8300 5440 50  0000 C CNN
@@
 $Comp
 L traction-r1:R RBLD5
-U 1 1 5E000135
+U 1 1 5E000140
 P 8300 6000
 F 0 "RBLD5" H 8300 5840 50  0000 C CNN
@@
 $Comp
 L traction-r1:R RBLD6
-U 1 1 5E000136
+U 1 1 5E000141
 P 9800 4400
 F 0 "RBLD6" H 9800 4240 50  0000 C CNN
@@
 $Comp
 L traction-r1:R RBLD7
-U 1 1 5E000137
+U 1 1 5E000142
 P 9800 4800
 F 0 "RBLD7" H 9800 4640 50  0000 C CNN
@@
 $Comp
 L traction-r1:R RBLD8
-U 1 1 5E000138
+U 1 1 5E000143
 P 9800 5200
 F 0 "RBLD8" H 9800 5040 50  0000 C CNN
@@
 $Comp
 L traction-r1:R RBLD9
-U 1 1 5E000139
+U 1 1 5E000144
 P 9800 5600
 F 0 "RBLD9" H 9800 5440 50  0000 C CNN
@@
 $Comp
 L traction-r1:QA01C-18 PSQD
-U 1 1 5E00013A
+U 1 1 5E000145
 P 2850 1800
 F 0 "PSQD" H 2450 1500 50  0000 R CNN
@@
 $EndComp
 Wire Wire Line
-	3300 1700 3500 1700
-Text Label 3500 1700 0    45   ~ 0
+	2400 1700 2200 1700
+Text Label 2200 1700 2    45   ~ 0
 V18Q
 Wire Wire Line
@@
 $Comp
 L traction-r1:HCM75S12T4K3 QDIS
-U 1 1 5E00013B
+U 1 1 5E000146
 P 4850 1350
 F 0 "QDIS" H 4450 1000 50  0000 R CNN
@@
 $Comp
 L traction-r1:TLP152 UQD
-U 1 1 5E00013C
+U 1 1 5E000147
 P 2850 3550
 F 0 "UQD" H 2450 3250 50  0000 R CNN
@@
 $Comp
 L traction-r1:C CQD
-U 1 1 5E00013D
+U 1 1 5E000148
 P 2650 5850
 F 0 "CQD" H 2650 5690 50  0000 C CNN
@@
 $Comp
 L traction-r1:R RDIS1
-U 1 1 5E00013E
+U 1 1 5E000149
 P 4650 2000
 F 0 "RDIS1" H 4650 1840 50  0000 C CNN
@@
 $Comp
 L traction-r1:R RDIS2
-U 1 1 5E00013F
+U 1 1 5E00014A
 P 4650 2400
 F 0 "RDIS2" H 4650 2240 50  0000 C CNN
@@
 $Comp
 L traction-r1:R RDIS3
-U 1 1 5E000140
+U 1 1 5E00014B
 P 4650 2800
 F 0 "RDIS3" H 4650 2640 50  0000 C CNN
@@
 $Comp
 L traction-r1:R RDIS4
-U 1 1 5E000141
+U 1 1 5E00014C
 P 4650 3200
 F 0 "RDIS4" H 4650 3040 50  0000 C CNN
@@
 $Comp
 L traction-r1:R RQDG
-U 1 1 5E000142
+U 1 1 5E00014D
 P 2650 5050
 F 0 "RQDG" H 2650 4890 50  0000 C CNN
@@
 $Comp
 L traction-r1:R RQDL
-U 1 1 5E000143
+U 1 1 5E00014E
 P 2650 4650
 F 0 "RQDL" H 2650 4490 50  0000 C CNN
@@
 $Comp
 L traction-r1:R RQDPD
-U 1 1 5E000144
+U 1 1 5E00014F
 P 2650 5450
 F 0 "RQDPD" H 2650 5290 50  0000 C CNN

Commit message: Rev A.4.1: second review round — 5 confirmed defects fixed (F47-F51)
- F47 AMC1311 real pins 2=IN/3=SHTDN (both VDC channels had them
  swapped: analog inputs grounded, SHTDN on the divider tap)
- F48 FS26 TRKIN is the VREF regulator's input supply -> VPRE
  (was grounded as an "unused tracker input"; VREF5 had no source)
- F49 TPS55340 pin 5 is SYNC (7V abs), not a second VIN -> DGND
- F50 FS26 caps to DS minimums: CVBOS 4.7uF, CSB6 4.7uF, CSB5 2.2uF
  (VREF COUT 1.1-3.3uF eff - third value found in the same audit)
- F51 V15 protective post-regulator NCV4276C-ADJ 40V/0.4A: boost
  pass-through (24V jump start / ~33V clamped load dump) can no longer
  reach the QA01C 13.5-16.5V window; boost output renamed V15B
- ASC/fault-latch interplay documented per NSI6611 DS (ASC overrides
  input side; DESAT + VCC2-UVLO outrank ASC)
- all five PDFs regenerate from one release (stale standalone A.3
  exports superseded); ERC gains A.4.1 assertions

Gates: 1674/1674 pins, ERC 769/0, design-verify 64P/3W/0F,
BOM Rs.70,074 @1k, 583 components, 184 lines.

Co-Authored-By: Claude Fable 5 <noreply@anthropic.com>
Parts:
- removed JCTL: HDR-1x4-2.54, HDR1x4, symbol traction-r1:HDR-1x4-2.54
- removed JDCN, JDCP: STUD-M6, StudM6, symbol traction-r1:TERM_1
- removed RBLD1: 27k, R2512, symbol traction-r1:R
- added RDIS4: 470R, AxialWW10W, symbol traction-r1:R
- added RQDG: 47R, R0603, symbol traction-r1:R
- added RQDL: 470R, R0603, symbol traction-r1:R
- added RQDPD: 10k, R0603, symbol traction-r1:R
- CQD: renamed from RDIS4; value 470R -> 100nF; footprint AxialWW10W -> C0603; symbol traction-r1:R -> traction-r1:C; MPN WW-470R-10W-AX -> MLCC-100nF-25V
- JCTL: renamed from RBLD10; value 27k -> HDR-1x4-2.54; footprint R2512 -> HDR1x4; symbol traction-r1:R -> traction-r1:HDR-1x4-2.54; MPN R2512-27k-2W -> HDR-1x4-2.54
- JDCN: renamed from RBLD2; value 27k -> STUD-M6; footprint R2512 -> StudM6; symbol traction-r1:R -> traction-r1:TERM_1; MPN R2512-27k-2W -> STUD-M6
- JDCP: renamed from RBLD3; value 27k -> STUD-M6; footprint R2512 -> StudM6; symbol traction-r1:R -> traction-r1:TERM_1; MPN R2512-27k-2W -> STUD-M6
- PSQD: renamed from RDIS1; value 470R -> QA01C-18; footprint AxialWW10W -> SIP7; symbol traction-r1:R -> traction-r1:QA01C-18; MPN WW-470R-10W-AX -> QA01C-18
- QDIS: renamed from RDIS2; value 470R -> HCM75S12T4K3; footprint AxialWW10W -> TO247-4L; symbol traction-r1:R -> traction-r1:HCM75S12T4K3; MPN WW-470R-10W-AX -> HCM75S12T4K3
- RBLD6: renamed from PSQD; value QA01C-18 -> 27k; footprint SIP7 -> R2512; symbol traction-r1:QA01C-18 -> traction-r1:R; MPN QA01C-18 -> R2512-27k-2W
- RBLD7: renamed from QDIS; value HCM75S12T4K3 -> 27k; footprint TO247-4L -> R2512; symbol traction-r1:HCM75S12T4K3 -> traction-r1:R; MPN HCM75S12T4K3 -> R2512-27k-2W
- RBLD8: renamed from UQD; value TLP152 -> 27k; footprint SO6 -> R2512; symbol traction-r1:TLP152 -> traction-r1:R; LCSC C17255258 -> CLASS; MPN TLP152 -> R2512-27k-2W
- RBLD9: renamed from CQD; value 100nF -> 27k; footprint C0603 -> R2512; symbol traction-r1:C -> traction-r1:R; MPN MLCC-100nF-25V -> R2512-27k-2W
- RDIS1: renamed from RQDG; value 47R -> 470R; footprint R0603 -> AxialWW10W; MPN R0603-47R -> WW-470R-10W-AX
- RDIS2: renamed from RQDL; footprint R0603 -> AxialWW10W; MPN R0603-470R -> WW-470R-10W-AX
- RDIS3: renamed from RQDPD; value 10k -> 470R; footprint R0603 -> AxialWW10W; MPN R0603-10k -> WW-470R-10W-AX
- UQD: renamed from RDIS3; value 470R -> TLP152; footprint AxialWW10W -> SO6; symbol traction-r1:R -> traction-r1:TLP152; LCSC CLASS -> C17255258; MPN WW-470R-10W-AX -> TLP152
- renumbered RBLD4 to RBLD1, RBLD5 to RBLD10, RBLD6 to RBLD2, RBLD7 to RBLD3, RBLD8 to RBLD4, RBLD9 to RBLD5
Other:
- note added: "220 kW pk Discharge (HV, bolt-on) - 3 of 4 · rev A.4.1 · 3 sections · 24 components"
- note removed: "220 kW pk Discharge (HV, bolt-on) - 3 of 4 · rev A.4 · 3 sections · 24 components"
- moved on the sheet: RBLD1, RBLD10, RBLD2, RBLD3, RBLD4, RBLD5, RDIS1, RDIS2, RDIS3
Changed lines of the file:
@@
 Title "Traction Inverter — Discharge board (bolt-on, XM3 pattern)"
 Date "2026-09-09"
-Rev "A.4"
+Rev "A.4.1"
 Comp "Traction Inverter 220 kW pk - Discharge (HV, bolt-on), sheet 3 of 4"
 Comment1 "Inverter = Power board + Cap bank busbar + bolt-on Discharge board (all HV) + Control card (LV); safe state holds with any link lost"
@@
 $EndDescr
 Text Notes 600 7100 0    60   ~ 12
-220 kW pk Discharge (HV, bolt-on) - 3 of 4   ·   rev A.4   ·   3 sections   ·   24 components
+220 kW pk Discharge (HV, bolt-on) - 3 of 4   ·   rev A.4.1   ·   3 sections   ·   24 components
 Text Notes 600 7400 0    50   ~ 0
 NET NAMING: U<ref>_<PIN> = node at that IC pin   ·   R<stem>_M = series-pair midpoint   ·   R<stem>_<nm> = tap between R<stem>n/m   ·   all others are explicit design nets   ·   same name on another sheet = same net, joined only at the named connector/stud/tab
@@
 $Comp
 L traction-r1:HDR-1x4-2.54 JCTL
-U 1 1 5E000138
+U 1 1 5E00013C
 P 9150 2100
 F 0 "JCTL" H 8750 1800 50  0000 R CNN
@@
 $Comp
 L traction-r1:TERM_1 JDCN
-U 1 1 5E000139
+U 1 1 5E00013D
 P 8800 1550
 F 0 "JDCN" H 8800 1390 50  0000 C CNN
@@
 $Comp
 L traction-r1:TERM_1 JDCP
-U 1 1 5E00013A
+U 1 1 5E00013E
 P 8800 1150
 F 0 "JDCP" H 8800 990 50  0000 C CNN
@@
 $Comp
 L traction-r1:R RBLD1
-U 1 1 5E00013B
+U 1 1 5E00013F
 P 8300 4400
 F 0 "RBLD1" H 8300 4240 50  0000 C CNN
@@
 $Comp
 L traction-r1:R RBLD10
-U 1 1 5E00013C
+U 1 1 5E000140
 P 9800 6000
 F 0 "RBLD10" H 9800 5840 50  0000 C CNN
@@
 $Comp
 L traction-r1:R RBLD2
-U 1 1 5E00013D
+U 1 1 5E000141
 P 8300 4800
 F 0 "RBLD2" H 8300 4640 50  0000 C CNN
@@
 $Comp
 L traction-r1:R RBLD3
-U 1 1 5E00013E
+U 1 1 5E000142
 P 8300 5200
 F 0 "RBLD3" H 8300 5040 50  0000 C CNN
@@
 $Comp
 L traction-r1:R RBLD4
-U 1 1 5E00013F
+U 1 1 5E000143
 P 8300 5600
 F 0 "RBLD4" H 8300 5440 50  0000 C CNN
@@
 $Comp
 L traction-r1:R RBLD5
-U 1 1 5E000140
+U 1 1 5E000144
 P 8300 6000
 F 0 "RBLD5" H 8300 5840 50  0000 C CNN
@@
 $Comp
 L traction-r1:R RBLD6
-U 1 1 5E000141
+U 1 1 5E000145
 P 9800 4400
 F 0 "RBLD6" H 9800 4240 50  0000 C CNN
@@
 $Comp
 L traction-r1:R RBLD7
-U 1 1 5E000142
+U 1 1 5E000146
 P 9800 4800
 F 0 "RBLD7" H 9800 4640 50  0000 C CNN
@@
 $Comp
 L traction-r1:R RBLD8
-U 1 1 5E000143
+U 1 1 5E000147
 P 9800 5200
 F 0 "RBLD8" H 9800 5040 50  0000 C CNN
@@
 $Comp
 L traction-r1:R RBLD9
-U 1 1 5E000144
+U 1 1 5E000148
 P 9800 5600
 F 0 "RBLD9" H 9800 5440 50  0000 C CNN
@@
 $Comp
 L traction-r1:QA01C-18 PSQD
-U 1 1 5E000145
+U 1 1 5E000149
 P 2850 1800
 F 0 "PSQD" H 2450 1500 50  0000 R CNN
@@
 $Comp
 L traction-r1:HCM75S12T4K3 QDIS
-U 1 1 5E000146
+U 1 1 5E00014A
 P 4850 1350
 F 0 "QDIS" H 4450 1000 50  0000 R CNN
@@
 $Comp
 L traction-r1:TLP152 UQD
-U 1 1 5E000147
+U 1 1 5E00014B
 P 2850 3550
 F 0 "UQD" H 2450 3250 50  0000 R CNN
@@
 $Comp
 L traction-r1:C CQD
-U 1 1 5E000148
+U 1 1 5E00014C
 P 2650 5850
 F 0 "CQD" H 2650 5690 50  0000 C CNN
@@
 $Comp
 L traction-r1:R RDIS1
-U 1 1 5E000149
+U 1 1 5E00014D
 P 4650 2000
 F 0 "RDIS1" H 4650 1840 50  0000 C CNN
@@
 $Comp
 L traction-r1:R RDIS2
-U 1 1 5E00014A
+U 1 1 5E00014E
 P 4650 2400
 F 0 "RDIS2" H 4650 2240 50  0000 C CNN
@@
 $Comp
 L traction-r1:R RDIS3
-U 1 1 5E00014B
+U 1 1 5E00014F
 P 4650 2800
 F 0 "RDIS3" H 4650 2640 50  0000 C CNN
@@
 $Comp
 L traction-r1:R RDIS4
-U 1 1 5E00014C
+U 1 1 5E000150
 P 4650 3200
 F 0 "RDIS4" H 4650 3040 50  0000 C CNN
@@
 $Comp
 L traction-r1:R RQDG
-U 1 1 5E00014D
+U 1 1 5E000151
 P 2650 5050
 F 0 "RQDG" H 2650 4890 50  0000 C CNN
@@
 $Comp
 L traction-r1:R RQDL
-U 1 1 5E00014E
+U 1 1 5E000152
 P 2650 4650
 F 0 "RQDL" H 2650 4490 50  0000 C CNN
@@
 $Comp
 L traction-r1:R RQDPD
-U 1 1 5E00014F
+U 1 1 5E000153
 P 2650 5450
 F 0 "RQDPD" H 2650 5290 50  0000 C CNN
