File: kicad5/traction/traction-disch.sch (KiCad schematic (older format))
At the start: 26 parts

Commit message: Rev A.11: review round 12 response (R1-F01..F28, R2-F01..F35) + datasheet archive
Two whole-system reviews of 4544715 (28 + 35 findings), dispositioned line by
line in docs/review-A11-disposition.md (+ CSV). Twelve real findings fixed
(F123-F134); the rest are tracked gates, firmware-owned, wording or out of the
schematic release's scope. No power-stage, capacitor or topology change.

Hardware / contract:
- SS6 release rule (a) is an energy inequality: winding energy 1.5*L*I^2 plus the
  back-EMF work during the decay, closed-form screen while E < V0, diode-bridge
  simulation otherwise; screening rows (WARN) per SKU
- Resolver exciter rewired as a textbook MFB (1.5 nF / 220 pF): the drawn network
  had the feedback pair swapped, |H(10 kHz)| 0.18 -> 1.85; SWG given its 47 pF load
- V_DC bias: "MGJ2D150505SC" was not an existing order code and no MGJ2 is
  reinforced above 150 Vrms -> TI UCC12050 per channel (V_IOWM 1200 Vrms /
  1697 VDC) behind its own NCV4276C from V15
- Hall: 100 k pull-downs drawn (claimed since A.4); LEM HC5FW drawn with its
  real terminals (1 V_ref, 2 V_out, 3 Gnd, 4 U_C, E1-E4)
- Resolver inputs 10 k / 10 k with rescaled, symmetric filter caps: a wire shorted
  to KL30 injected 23 mA into an SDADC pin against the 3 mA limit
- LV-entry TVS bound explicitly as TPSMC24CA-VR (24 V stand-off, AEC-Q101): the
  classic part the notes described conducts at a 24 V jump start; the OEM's
  load-dump source resistance becomes gate 23
- CSB5 1 uF 0805 (VREF5 inside the FS26 window), ALM2402 as HTSSOP14-PWP,
  on-board NTCs RTAMB/RTHS, kicad5-verify empty-set guard
- Contract wording: FW-05 in instantaneous amperes with a validity window, the
  "BMS limit 0" row split from "contactor open", NVM logging queued behind the
  safe action, FW-02 tau check demoted to plausibility (EOL measurement in dfm),
  FW-18 "unknown, never safe", S6 double-update stated; stale pin-40 / LQFP-176 /
  "inside 6 us" / ALT-field texts corrected; CAN termination DNP option

Doc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
Parts:
- removed JCTL: HDR-1x4-2.54, HDR1x4, symbol traction-r1:HDR-1x4-2.54
- removed JDCN, JDCP: STUD-M6, StudM6, symbol traction-r1:TERM_1
- removed RBLD1, RBLD10, RBLD11, RBLD12: 22k, R2512, symbol traction-r1:R
- added RDIS1, RDIS2, RDIS3, RDIS4: 470R, AxialWW10W, symbol traction-r1:R
- added RQDG: 1.5k, R0603, symbol traction-r1:R
- added RQDL: 261R, R0603, symbol traction-r1:R
- added RQDPD: 10k, R0603, symbol traction-r1:R
- CQD: renamed from RQDPD; value 10k -> 100nF; footprint R0603 -> C0603; symbol traction-r1:R -> traction-r1:C; MPN R0603-10k -> MLCC-100nF-50V
- JCTL: renamed from RBLD2; value 22k -> HDR-1x4-2.54; footprint R2512 -> HDR1x4; symbol traction-r1:R -> traction-r1:HDR-1x4-2.54; MPN R2512-22k-2W -> HDR-1x4-2.54
- JDCN: renamed from RBLD3; value 22k -> STUD-M6; footprint R2512 -> StudM6; symbol traction-r1:R -> traction-r1:TERM_1; MPN R2512-22k-2W -> STUD-M6
- JDCP: renamed from RBLD4; value 22k -> STUD-M6; footprint R2512 -> StudM6; symbol traction-r1:R -> traction-r1:TERM_1; MPN R2512-22k-2W -> STUD-M6
- PSQD: renamed from RDIS4; value 470R -> QA01C-18; footprint AxialWW10W -> SIP7; symbol traction-r1:R -> traction-r1:QA01C-18; MPN WW-470R-10W-AX -> QA01C-18
- QDIS: renamed from RQDG; value 1.5k -> HCM75S12T4K3; footprint R0603 -> TO247-4L; symbol traction-r1:R -> traction-r1:HCM75S12T4K3; MPN R0603-1k5 -> HCM75S12T4K3
- RBLD3: renamed from PSQD; value QA01C-18 -> 22k; footprint SIP7 -> R2512; symbol traction-r1:QA01C-18 -> traction-r1:R; MPN QA01C-18 -> R2512-22k-2W
- RBLD4: renamed from QDIS; value HCM75S12T4K3 -> 22k; footprint TO247-4L -> R2512; symbol traction-r1:HCM75S12T4K3 -> traction-r1:R; MPN HCM75S12T4K3 -> R2512-22k-2W
- RBLD5: renamed from UQD; value TLP152 -> 22k; footprint SO6 -> R2512; symbol traction-r1:TLP152 -> traction-r1:R; LCSC C17255258 -> CLASS; MPN TLP152 -> R2512-22k-2W
- RBLD6: renamed from CQD; value 100nF -> 22k; footprint C0603 -> R2512; symbol traction-r1:C -> traction-r1:R; MPN MLCC-100nF-50V -> R2512-22k-2W
- RBLD7: renamed from RDIS1; value 470R -> 22k; footprint AxialWW10W -> R2512; MPN WW-470R-10W-AX -> R2512-22k-2W
- RBLD8: renamed from RDIS2; value 470R -> 22k; footprint AxialWW10W -> R2512; MPN WW-470R-10W-AX -> R2512-22k-2W
- RBLD9: renamed from RDIS3; value 470R -> 22k; footprint AxialWW10W -> R2512; MPN WW-470R-10W-AX -> R2512-22k-2W
- UQD: renamed from RQDL; value 261R -> TLP152; footprint R0603 -> SO6; symbol traction-r1:R -> traction-r1:TLP152; LCSC CLASS -> C17255258; MPN R0603-261R-1% -> TLP152
- renumbered RBLD5 to RBLD1, RBLD6 to RBLD10, RBLD7 to RBLD11, RBLD8 to RBLD12, RBLD9 to RBLD2
Other:
- note added: "220 kW pk Discharge (HV, bolt-on) - 3 of 4 · rev A.11 · 3 sections · 26 components"
- note removed: "220 kW pk Discharge (HV, bolt-on) - 3 of 4 · rev A.10 · 3 sections · 26 components"
- moved on the sheet: RBLD1, RBLD10, RBLD11, RBLD12, RBLD2, RBLD7, RBLD8, RBLD9
Changed lines of the file:
@@
 Title "Traction Inverter — Discharge board (bolt-on, XM3 pattern)"
 Date "2026-09-23"
-Rev "A.10"
+Rev "A.11"
 Comp "Traction Inverter 220 kW pk - Discharge (HV, bolt-on), sheet 3 of 4"
 Comment1 "Inverter = Power board + Cap bank busbar + bolt-on Discharge board (all HV) + Control card (LV); safe state holds with any link lost"
@@
 $EndDescr
 Text Notes 600 7600 0    60   ~ 12
-220 kW pk Discharge (HV, bolt-on) - 3 of 4   ·   rev A.10   ·   3 sections   ·   26 components
+220 kW pk Discharge (HV, bolt-on) - 3 of 4   ·   rev A.11   ·   3 sections   ·   26 components
 Text Notes 600 7900 0    50   ~ 0
 NET NAMING: U<ref>_<PIN> = node at that IC pin   ·   R<stem>_M = series-pair midpoint   ·   R<stem>_<nm> = tap between R<stem>n/m   ·   all others are explicit design nets   ·   same name on another sheet = same net, joined only at the named connector/stud/tab
@@
 $Comp
 L traction-r1:HDR-1x4-2.54 JCTL
-U 1 1 5E00014D
+U 1 1 5E000154
 P 9150 5850
 F 0 "JCTL" H 8750 5550 50  0000 R CNN
@@
 $Comp
 L traction-r1:TERM_1 JDCN
-U 1 1 5E00014E
+U 1 1 5E000155
 P 8800 5300
 F 0 "JDCN" H 8800 5140 50  0000 C CNN
@@
 $Comp
 L traction-r1:TERM_1 JDCP
-U 1 1 5E00014F
+U 1 1 5E000156
 P 8800 4900
 F 0 "JDCP" H 8800 4740 50  0000 C CNN
@@
 $Comp
 L traction-r1:R RBLD1
-U 1 1 5E000150
+U 1 1 5E000157
 P 8300 1150
 F 0 "RBLD1" H 8300 990 50  0000 C CNN
@@
 $Comp
 L traction-r1:R RBLD10
-U 1 1 5E000151
+U 1 1 5E000158
 P 9800 2350
 F 0 "RBLD10" H 9800 2190 50  0000 C CNN
@@
 $Comp
 L traction-r1:R RBLD11
-U 1 1 5E000152
+U 1 1 5E000159
 P 9800 2750
 F 0 "RBLD11" H 9800 2590 50  0000 C CNN
@@
 $Comp
 L traction-r1:R RBLD12
-U 1 1 5E000153
+U 1 1 5E00015A
 P 9800 3150
 F 0 "RBLD12" H 9800 2990 50  0000 C CNN
@@
 $Comp
 L traction-r1:R RBLD2
-U 1 1 5E000154
+U 1 1 5E00015B
 P 8300 1550
 F 0 "RBLD2" H 8300 1390 50  0000 C CNN
@@
 $Comp
 L traction-r1:R RBLD3
-U 1 1 5E000155
+U 1 1 5E00015C
 P 8300 1950
 F 0 "RBLD3" H 8300 1790 50  0000 C CNN
@@
 $Comp
 L traction-r1:R RBLD4
-U 1 1 5E000156
+U 1 1 5E00015D
 P 8300 2350
 F 0 "RBLD4" H 8300 2190 50  0000 C CNN
@@
 $Comp
 L traction-r1:R RBLD5
-U 1 1 5E000157
+U 1 1 5E00015E
 P 8300 2750
 F 0 "RBLD5" H 8300 2590 50  0000 C CNN
@@
 $Comp
 L traction-r1:R RBLD6
-U 1 1 5E000158
+U 1 1 5E00015F
 P 8300 3150
 F 0 "RBLD6" H 8300 2990 50  0000 C CNN
@@
 $Comp
 L traction-r1:R RBLD7
-U 1 1 5E000159
+U 1 1 5E000160
 P 9800 1150
 F 0 "RBLD7" H 9800 990 50  0000 C CNN
@@
 $Comp
 L traction-r1:R RBLD8
-U 1 1 5E00015A
+U 1 1 5E000161
 P 9800 1550
 F 0 "RBLD8" H 9800 1390 50  0000 C CNN
@@
 $Comp
 L traction-r1:R RBLD9
-U 1 1 5E00015B
+U 1 1 5E000162
 P 9800 1950
 F 0 "RBLD9" H 9800 1790 50  0000 C CNN
@@
 $Comp
 L traction-r1:QA01C-18 PSQD
-U 1 1 5E00015C
+U 1 1 5E000163
 P 2850 1800
 F 0 "PSQD" H 2450 1500 50  0000 R CNN
@@
 $Comp
 L traction-r1:HCM75S12T4K3 QDIS
-U 1 1 5E00015D
+U 1 1 5E000164
 P 4850 1350
 F 0 "QDIS" H 4450 1000 50  0000 R CNN
@@
 $Comp
 L traction-r1:TLP152 UQD
-U 1 1 5E00015E
+U 1 1 5E000165
 P 2850 3550
 F 0 "UQD" H 2450 3250 50  0000 R CNN
@@
 $Comp
 L traction-r1:C CQD
-U 1 1 5E00015F
+U 1 1 5E000166
 P 2650 5850
 F 0 "CQD" H 2650 5690 50  0000 C CNN
@@
 $Comp
 L traction-r1:R RDIS1
-U 1 1 5E000160
+U 1 1 5E000167
 P 4650 2000
 F 0 "RDIS1" H 4650 1840 50  0000 C CNN
@@
 $Comp
 L traction-r1:R RDIS2
-U 1 1 5E000161
+U 1 1 5E000168
 P 4650 2400
 F 0 "RDIS2" H 4650 2240 50  0000 C CNN
@@
 $Comp
 L traction-r1:R RDIS3
-U 1 1 5E000162
+U 1 1 5E000169
 P 4650 2800
 F 0 "RDIS3" H 4650 2640 50  0000 C CNN
@@
 $Comp
 L traction-r1:R RDIS4
-U 1 1 5E000163
+U 1 1 5E00016A
 P 4650 3200
 F 0 "RDIS4" H 4650 3040 50  0000 C CNN
@@
 $Comp
 L traction-r1:R RQDG
-U 1 1 5E000164
+U 1 1 5E00016B
 P 2650 5050
 F 0 "RQDG" H 2650 4890 50  0000 C CNN
@@
 $Comp
 L traction-r1:R RQDL
-U 1 1 5E000165
+U 1 1 5E00016C
 P 2650 4650
 F 0 "RQDL" H 2650 4490 50  0000 C CNN
@@
 $Comp
 L traction-r1:R RQDPD
-U 1 1 5E000166
+U 1 1 5E00016D
 P 2650 5450
 F 0 "RQDPD" H 2650 5290 50  0000 C CNN

Commit message: Rev A.12: round 13 rechecks (F135-F139), pin freeze (F140), barrier + orderability closure (F141-F142), Marine A.12, firmware
- Rechecks of 30ae0a2: §6 winding-energy rule at every speed; resolver 12 k series + 220 pF C_AAF
  (injection 2.92 mA with the MCU unpowered); verifier counts distinct assemblies; TPS55340-Q1 real
  ratings (38/40 V); NCV4276C thermal on the datasheet pad.
- MCU pin freeze: all 289 S32K396 balls bound from SPF-91122 rev C anchored on the DS supply balls
  (calculations/mcu-ballmap.json, docs/mcu-pin-manifest.md); seven port corrections; FS26 pins verified;
  ERC pin-freeze lock.
- Barrier closure: VOW3120-X017T optos and UCC14141-Q1 biases (shared IsoBias18 cell, single-output
  18.0 V) replace TLP152/QA01C-18; LED resistors 270 R; VY1 Y-caps; Samtec IPL1/IPD1 harness;
  Faratronic 4XX can; SQP10 discharge resistors; UCC12051-Q1 on the AVL.
- Tooling: ERC open-pin helper + HARNESS40 parser scoped to its block; kicad5-verify assembly-set guard.
- Marine ported to A.12 (86 PASS / 22 WARN / 0 FAIL); firmware/ (C11, 178 tests / 1209 checks).
- Docs: README, design-basis §6a/§8/§11l, dfm, variants, cost-rollup, EXTRACTED-PARAMS §27-30 +
  seven archived datasheets, review-A12-disposition (+CSV), regenerated sheets/PDFs/BOMs/previews.

ERC 933/0 · design-verify 123/19/0 · sim 23/6/0 · sheets 2027/2027.

Co-Authored-By: Claude Fable 5.1 <noreply@anthropic.com>
Parts:
- removed JCTL: HDR-1x4-2.54, HDR1x4, symbol traction-r1:HDR-1x4-2.54
- removed JDCN, JDCP: STUD-M6, StudM6, symbol traction-r1:TERM_1
- removed RBLD1, RBLD10, RBLD11, RBLD12, RBLD2, RBLD3: 22k, R2512, symbol traction-r1:R
- added CQD, CQDIB: 100nF, C0603, symbol traction-r1:C
- added CQDF: 330pF, C0603, symbol traction-r1:C
- added CQDI1, CQDI2: 10uF, C1206, symbol traction-r1:C
- added CQDO: 10uF, C1210, symbol traction-r1:C
- added RDIS1, RDIS2, RDIS3, RDIS4: 470R, AxialWW10W, symbol traction-r1:R
- added RQDE1, RQDF2, RQDPD: 10k, R0603, symbol traction-r1:R
- added RQDE2: 4.7k, R0603, symbol traction-r1:R
- added RQDF1: 62k, R0603, symbol traction-r1:R
- added RQDG: 1.5k, R0603, symbol traction-r1:R
- added RQDL: 270R, R0603, symbol traction-r1:R
- added UQD: VOW3120-X017T, SMD8W, symbol traction-r1:VOW3120-X017T
- JCTL: renamed from RBLD4; value 22k -> HDR-1x4-2.54; footprint R2512 -> HDR1x4; symbol traction-r1:R -> traction-r1:HDR-1x4-2.54; MPN R2512-22k-2W -> HDR-1x4-2.54
- JDCN: renamed from RBLD5; value 22k -> STUD-M6; footprint R2512 -> StudM6; symbol traction-r1:R -> traction-r1:TERM_1; MPN R2512-22k-2W -> STUD-M6
- JDCP: renamed from RBLD6; value 22k -> STUD-M6; footprint R2512 -> StudM6; symbol traction-r1:R -> traction-r1:TERM_1; MPN R2512-22k-2W -> STUD-M6
- PSQD: renamed from RQDL; value 261R -> UCC14141QDWNRQ1; footprint R0603 -> DWN36; symbol traction-r1:R -> traction-r1:UCC14141QDWNRQ1; MPN R0603-261R-1% -> UCC14141QDWNRQ1
- QDIS: renamed from RQDPD; value 10k -> HCM75S12T4K3; footprint R0603 -> TO247-4L; symbol traction-r1:R -> traction-r1:HCM75S12T4K3; MPN R0603-10k -> HCM75S12T4K3
- RBLD12: renamed from PSQD; value QA01C-18 -> 22k; footprint SIP7 -> R2512; symbol traction-r1:QA01C-18 -> traction-r1:R; MPN QA01C-18 -> R2512-22k-2W
- RBLD2: renamed from QDIS; value HCM75S12T4K3 -> 22k; footprint TO247-4L -> R2512; symbol traction-r1:HCM75S12T4K3 -> traction-r1:R; MPN HCM75S12T4K3 -> R2512-22k-2W
- RBLD3: renamed from UQD; value TLP152 -> 22k; footprint SO6 -> R2512; symbol traction-r1:TLP152 -> traction-r1:R; LCSC C17255258 -> CLASS; MPN TLP152 -> R2512-22k-2W
- RBLD4: renamed from CQD; value 100nF -> 22k; footprint C0603 -> R2512; symbol traction-r1:C -> traction-r1:R; MPN MLCC-100nF-50V -> R2512-22k-2W
- RBLD5: renamed from RDIS1; value 470R -> 22k; footprint AxialWW10W -> R2512; MPN WW-470R-10W-AX -> R2512-22k-2W
- RBLD6: renamed from RDIS2; value 470R -> 22k; footprint AxialWW10W -> R2512; MPN WW-470R-10W-AX -> R2512-22k-2W
- RBLD7: renamed from RDIS3; value 470R -> 22k; footprint AxialWW10W -> R2512; MPN WW-470R-10W-AX -> R2512-22k-2W
- RBLD8: renamed from RDIS4; value 470R -> 22k; footprint AxialWW10W -> R2512; MPN WW-470R-10W-AX -> R2512-22k-2W
- RBLD9: renamed from RQDG; value 1.5k -> 22k; footprint R0603 -> R2512; MPN R0603-1k5 -> R2512-22k-2W
- renumbered RBLD7 to RBLD1, RBLD8 to RBLD10, RBLD9 to RBLD11
Connections:
- net labels added: ENA_QD, FB_QD
- wire segments 59 -> 107
Other:
- note added: "220 kW pk Discharge (HV, bolt-on) - 3 of 4 · rev A.12 · 3 sections · 35 components"
- note removed: "220 kW pk Discharge (HV, bolt-on) - 3 of 4 · rev A.11 · 3 sections · 26 components"
- moved on the sheet: RBLD1, RBLD10, RBLD11, RBLD5, RBLD6, RBLD7, RBLD8, RBLD9
