File: kicad5/traction/traction-disch.sch (KiCad schematic (older format))
At the start: 35 parts

Commit message: Rev A.13: round 14 — three reviews of cfd35a7 (F143-F158): MCU map vs NXP netlist, fail-closed firmware, terminal-fault protection
- Pin freeze reopened and closed: H5 is V15 (1.5 V, was on VREF5) and J7 is V25 (regulator output,
  was grounded); whole map re-derived against NXP's GEN3 net report NET-91122_C (U513, 244 balls) —
  every supply ball and 164/165 port names agree; HW_ID/NTC_A/MT2_SIG/ASC_REQ moved to netlist-confirmed
  balls (B5/T15/D5/U4); KiCad symbol numbered by physical ball, mutation-tested; CNMOS 1 nF.
- Firmware (214 tests / 1622 checks, ASan/UBSan, target-check): DESAT hold for every caller, 64-bit
  monotonic clock, keep_hv from rule (b) reliance at any speed, IMCR placeholders = build error,
  config-matches vs protection-locked, arming-evidence record (fail closed), torque feasibility witness,
  stuck-channel detection, stuck-on discharge detection; board map regenerated.
- Analog: excitation monitor 18 k/42.2 k/84.5 k + 220 pF C_AAF; exciter SMCJ8.5CA + MF-MSMF020 per line;
  motor-temp SMAJ5.0A + 0438.375WRA; bias-LDO 47 R ballast, UCC12051-Q1 primary; UCC14141-Q1 VDE cert.
- Docs: contract FW-22..FW-26 + keep_hv; design-basis §11m; variants/cost/dfm/README; disposition + CSV;
  EXTRACTED §31/§32 + archived datasheets; report-template defect fixed; Marine at A.13 (86/22/0).

ERC 945/0 · design-verify 130/23/0 · sim 23/6/0 · sheets 2045/2045 · BOM 8XX SiC ₹72,492.

Co-Authored-By: Claude Fable 5.1 <noreply@anthropic.com>
Parts:
- removed JCTL: HDR-1x4-2.54, HDR1x4, symbol traction-r1:HDR-1x4-2.54
- removed JDCN: STUD-M6, StudM6, symbol traction-r1:TERM_1
- added RQDL: 270R, R0603, symbol traction-r1:R
- added RQDPD: 10k, R0603, symbol traction-r1:R
- CQD: renamed from CQDI1; value 10uF -> 100nF; footprint C1206 -> C0603; MPN MLCC-10uF-25V-X7R -> MLCC-100nF-50V
- CQDF: renamed from CQDI2; value 10uF -> 330pF; footprint C1206 -> C0603; MPN MLCC-10uF-25V-X7R -> MLCC-330pF-50V-C0G
- CQDI1: renamed from CQDIB; value 100nF -> 10uF; footprint C0603 -> C1206; MPN MLCC-100nF-50V -> MLCC-10uF-25V-X7R
- CQDI2: renamed from CQDO; footprint C1210 -> C1206; MPN MLCC-10uF-50V -> MLCC-10uF-25V-X7R
- CQDIB: renamed from RDIS1; value 470R -> 100nF; footprint AxialWW10W -> C0603; symbol traction-r1:R -> traction-r1:C; MPN SQP10-470RJB15 -> MLCC-100nF-50V
- CQDO: renamed from RDIS2; value 470R -> 10uF; footprint AxialWW10W -> C1210; symbol traction-r1:R -> traction-r1:C; MPN SQP10-470RJB15 -> MLCC-10uF-50V
- JCTL: renamed from JDCP; value STUD-M6 -> HDR-1x4-2.54; footprint StudM6 -> HDR1x4; symbol traction-r1:TERM_1 -> traction-r1:HDR-1x4-2.54; MPN STUD-M6 -> HDR-1x4-2.54
- JDCN: renamed from RBLD1; value 22k -> STUD-M6; footprint R2512 -> StudM6; symbol traction-r1:R -> traction-r1:TERM_1; MPN R2512-22k-2W -> STUD-M6
- JDCP: renamed from RBLD10; value 22k -> STUD-M6; footprint R2512 -> StudM6; symbol traction-r1:R -> traction-r1:TERM_1; MPN R2512-22k-2W -> STUD-M6
- PSQD: renamed from UQD; value VOW3120-X017T -> UCC14141QDWNRQ1; footprint SMD8W -> DWN36; symbol traction-r1:VOW3120-X017T -> traction-r1:UCC14141QDWNRQ1; MPN VOW3120-X017T -> UCC14141QDWNRQ1
- QDIS: renamed from CQD; value 100nF -> HCM75S12T4K3; footprint C0603 -> TO247-4L; symbol traction-r1:C -> traction-r1:HCM75S12T4K3; MPN MLCC-100nF-50V -> HCM75S12T4K3
- RBLD8: renamed from PSQD; value UCC14141QDWNRQ1 -> 22k; footprint DWN36 -> R2512; symbol traction-r1:UCC14141QDWNRQ1 -> traction-r1:R; MPN UCC14141QDWNRQ1 -> R2512-22k-2W
- RBLD9: renamed from QDIS; value HCM75S12T4K3 -> 22k; footprint TO247-4L -> R2512; symbol traction-r1:HCM75S12T4K3 -> traction-r1:R; MPN HCM75S12T4K3 -> R2512-22k-2W
- RDIS3: renamed from RQDE1; value 10k -> 470R; footprint R0603 -> AxialWW10W; MPN R0603-10k -> SQP10-470RJB15
- RDIS4: renamed from RQDE2; value 4.7k -> 470R; footprint R0603 -> AxialWW10W; MPN R0603-4k7 -> SQP10-470RJB15
- RQDE1: renamed from RQDF1; value 62k -> 10k; MPN R0603-62k-1% -> R0603-10k
- RQDE2: renamed from RQDF2; value 10k -> 4.7k; MPN R0603-10k-1% -> R0603-4k7
- RQDF1: renamed from RQDG; value 1.5k -> 62k; MPN R0603-1k5 -> R0603-62k-1%
- RQDF2: renamed from RQDL; value 270R -> 10k; MPN R0603-270R-1% -> R0603-10k-1%
- RQDG: renamed from RQDPD; value 10k -> 1.5k; MPN R0603-10k -> R0603-1k5
- UQD: renamed from CQDF; value 330pF -> VOW3120-X017T; footprint C0603 -> SMD8W; symbol traction-r1:C -> traction-r1:VOW3120-X017T; MPN MLCC-330pF-50V-C0G -> VOW3120-X017T
- renumbered RBLD11 to RBLD1, RBLD12 to RBLD10, RBLD2 to RBLD11, RBLD3 to RBLD12, RBLD4 to RBLD2, RBLD5 to RBLD3, RBLD6 to RBLD4, RBLD7 to RBLD5, RBLD8 to RBLD6, RBLD9 to RBLD7, RDIS3 to RDIS1, RDIS4 to RDIS2
Other:
- note added: "220 kW pk Discharge (HV, bolt-on) - 3 of 4 · rev A.13 · 3 sections · 35 components"
- note removed: "220 kW pk Discharge (HV, bolt-on) - 3 of 4 · rev A.12 · 3 sections · 35 components"
- moved on the sheet: CQD, CQDF, CQDI1, CQDI2, RBLD1, RBLD10, RBLD11, RBLD12, RBLD2, RBLD3, RBLD4, RBLD5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
Changed lines of the file:
@@
 Title "Traction Inverter — Discharge board (bolt-on, XM3 pattern)"
 Date "2026-09-23"
-Rev "A.12"
+Rev "A.13"
 Comp "Traction Inverter 220 kW pk - Discharge (HV, bolt-on), sheet 3 of 4"
 Comment1 "Inverter = Power board + Cap bank busbar + bolt-on Discharge board (all HV) + Control card (LV); safe state holds with any link lost"
@@
 $EndDescr
 Text Notes 600 7600 0    60   ~ 12
-220 kW pk Discharge (HV, bolt-on) - 3 of 4   ·   rev A.12   ·   3 sections   ·   35 components
+220 kW pk Discharge (HV, bolt-on) - 3 of 4   ·   rev A.13   ·   3 sections   ·   35 components
 Text Notes 600 7900 0    50   ~ 0
 NET NAMING: U<ref>_<PIN> = node at that IC pin   ·   R<stem>_M = series-pair midpoint   ·   R<stem>_<nm> = tap between R<stem>n/m   ·   all others are explicit design nets   ·   same name on another sheet = same net, joined only at the named connector/stud/tab
@@
 $Comp
 L traction-r1:HDR-1x4-2.54 JCTL
-U 1 1 5E00015D
+U 1 1 5E00015F
 P 9150 5850
 F 0 "JCTL" H 8750 5550 50  0000 R CNN
@@
 $Comp
 L traction-r1:TERM_1 JDCN
-U 1 1 5E00015E
+U 1 1 5E000160
 P 8800 5300
 F 0 "JDCN" H 8800 5140 50  0000 C CNN
@@
 $Comp
 L traction-r1:TERM_1 JDCP
-U 1 1 5E00015F
+U 1 1 5E000161
 P 8800 4900
 F 0 "JDCP" H 8800 4740 50  0000 C CNN
@@
 $Comp
 L traction-r1:R RBLD1
-U 1 1 5E000160
+U 1 1 5E000162
 P 8300 1150
 F 0 "RBLD1" H 8300 990 50  0000 C CNN
@@
 $Comp
 L traction-r1:R RBLD10
-U 1 1 5E000161
+U 1 1 5E000163
 P 9800 2350
 F 0 "RBLD10" H 9800 2190 50  0000 C CNN
@@
 $Comp
 L traction-r1:R RBLD11
-U 1 1 5E000162
+U 1 1 5E000164
 P 9800 2750
 F 0 "RBLD11" H 9800 2590 50  0000 C CNN
@@
 $Comp
 L traction-r1:R RBLD12
-U 1 1 5E000163
+U 1 1 5E000165
 P 9800 3150
 F 0 "RBLD12" H 9800 2990 50  0000 C CNN
@@
 $Comp
 L traction-r1:R RBLD2
-U 1 1 5E000164
+U 1 1 5E000166
 P 8300 1550
 F 0 "RBLD2" H 8300 1390 50  0000 C CNN
@@
 $Comp
 L traction-r1:R RBLD3
-U 1 1 5E000165
+U 1 1 5E000167
 P 8300 1950
 F 0 "RBLD3" H 8300 1790 50  0000 C CNN
@@
 $Comp
 L traction-r1:R RBLD4
-U 1 1 5E000166
+U 1 1 5E000168
 P 8300 2350
 F 0 "RBLD4" H 8300 2190 50  0000 C CNN
@@
 $Comp
 L traction-r1:R RBLD5
-U 1 1 5E000167
+U 1 1 5E000169
 P 8300 2750
 F 0 "RBLD5" H 8300 2590 50  0000 C CNN
@@
 $Comp
 L traction-r1:R RBLD6
-U 1 1 5E000168
+U 1 1 5E00016A
 P 8300 3150
 F 0 "RBLD6" H 8300 2990 50  0000 C CNN
@@
 $Comp
 L traction-r1:R RBLD7
-U 1 1 5E000169
+U 1 1 5E00016B
 P 9800 1150
 F 0 "RBLD7" H 9800 990 50  0000 C CNN
@@
 $Comp
 L traction-r1:R RBLD8
-U 1 1 5E00016A
+U 1 1 5E00016C
 P 9800 1550
 F 0 "RBLD8" H 9800 1390 50  0000 C CNN
@@
 $Comp
 L traction-r1:R RBLD9
-U 1 1 5E00016B
+U 1 1 5E00016D
 P 9800 1950
 F 0 "RBLD9" H 9800 1790 50  0000 C CNN
@@
 $Comp
 L traction-r1:UCC14141QDWNRQ1 PSQD
-U 1 1 5E00016C
+U 1 1 5E00016E
 P 1850 2050
 F 0 "PSQD" H 1400 1000 50  0000 R CNN
@@
 $Comp
 L traction-r1:HCM75S12T4K3 QDIS
-U 1 1 5E00016D
+U 1 1 5E00016F
 P 5850 1350
 F 0 "QDIS" H 5450 1000 50  0000 R CNN
@@
 $Comp
 L traction-r1:VOW3120-X017T UQD
-U 1 1 5E00016E
+U 1 1 5E000170
 P 3900 1800
 F 0 "UQD" H 3500 1500 50  0000 R CNN
@@
 $Comp
 L traction-r1:C CQD
-U 1 1 5E00016F
+U 1 1 5E000171
 P 3700 4100
 F 0 "CQD" H 3700 3940 50  0000 C CNN
@@
 $Comp
 L traction-r1:C CQDF
-U 1 1 5E000170
+U 1 1 5E000172
 P 1600 6200
 F 0 "CQDF" H 1600 6040 50  0000 C CNN
@@
 $Comp
 L traction-r1:C CQDI1
-U 1 1 5E000171
+U 1 1 5E000173
 P 1600 3400
 F 0 "CQDI1" H 1600 3240 50  0000 C CNN
@@
 $Comp
 L traction-r1:C CQDI2
-U 1 1 5E000172
+U 1 1 5E000174
 P 1600 3800
 F 0 "CQDI2" H 1600 3640 50  0000 C CNN
@@
 $Comp
 L traction-r1:C CQDIB
-U 1 1 5E000173
+U 1 1 5E000175
 P 1600 4200
 F 0 "CQDIB" H 1600 4040 50  0000 C CNN
@@
 $Comp
 L traction-r1:C CQDO
-U 1 1 5E000174
+U 1 1 5E000176
 P 1600 6600
 F 0 "CQDO" H 1600 6440 50  0000 C CNN
@@
 $Comp
 L traction-r1:R RDIS1
-U 1 1 5E000175
+U 1 1 5E000177
 P 5650 2000
 F 0 "RDIS1" H 5650 1840 50  0000 C CNN
@@
 $Comp
 L traction-r1:R RDIS2
-U 1 1 5E000176
+U 1 1 5E000178
 P 5650 2400
 F 0 "RDIS2" H 5650 2240 50  0000 C CNN
@@
 $Comp
 L traction-r1:R RDIS3
-U 1 1 5E000177
+U 1 1 5E000179
 P 5650 2800
 F 0 "RDIS3" H 5650 2640 50  0000 C CNN
@@
 $Comp
 L traction-r1:R RDIS4
-U 1 1 5E000178
+U 1 1 5E00017A
 P 5650 3200
 F 0 "RDIS4" H 5650 3040 50  0000 C CNN
@@
 $Comp
 L traction-r1:R RQDE1
-U 1 1 5E000179
+U 1 1 5E00017B
 P 1600 4600
 F 0 "RQDE1" H 1600 4440 50  0000 C CNN
@@
 $Comp
 L traction-r1:R RQDE2
-U 1 1 5E00017A
+U 1 1 5E00017C
 P 1600 5000
 F 0 "RQDE2" H 1600 4840 50  0000 C CNN
@@
 $Comp
 L traction-r1:R RQDF1
-U 1 1 5E00017B
+U 1 1 5E00017D
 P 1600 5400
 F 0 "RQDF1" H 1600 5240 50  0000 C CNN
@@
 $Comp
 L traction-r1:R RQDF2
-U 1 1 5E00017C
+U 1 1 5E00017E
 P 1600 5800
 F 0 "RQDF2" H 1600 5640 50  0000 C CNN
@@
 $Comp
 L traction-r1:R RQDG
-U 1 1 5E00017D
+U 1 1 5E00017F
 P 3700 3300
 F 0 "RQDG" H 3700 3140 50  0000 C CNN
@@
 $Comp
 L traction-r1:R RQDL
-U 1 1 5E00017E
+U 1 1 5E000180
 P 3700 2900
 F 0 "RQDL" H 3700 2740 50  0000 C CNN
@@
 $Comp
 L traction-r1:R RQDPD
-U 1 1 5E00017F
+U 1 1 5E000181
 P 3700 3700
 F 0 "RQDPD" H 3700 3540 50  0000 C CNN
