File: kicad5/traction/traction-capbank.sch (KiCad schematic (older format))
At the start: 26 parts

Commit message: Rev A.4: answer external design review — 10 confirmed defects fixed (F37-F46)
Every claim verified against primary datasheets before any edit; three
claims rebutted with evidence (850V/0.1% divider corner, GEN3-exact
resolver monitors, discharge math matches). Fixed:

- F37 VGT12EEM secondary phasing: rectifier moved to pin 8 (dot); the
  drawn wiring was forward-mode ~35V into +22V-abs gates. Pins 6/7 NC'd
  (no internal winding). Aux (NF) was already correct.
- F38 flyback drain clamp: SMBJ85A (forward every OFF interval, 94.4V
  min breakdown vs 80V FET) -> US1M + SMAJ13A winding clamp; drain
  <=60V at clamped load dump
- F39 DESAT clamp: BAT64-04 series pair correctly oriented DESAT->VCC2
  (was VCC2 injected into DESAT via a wrong common-cathode symbol)
- F40 ASC latch: real SN74LVC1G74 DCU pins; 1k/10k network (was
  120R/120R = 2.5V "low" and 42mA MCU clear)
- F41 KL15: 47k/10k+100nF ADC sense (was raw 13.3V into PTA25)
- F42 VDC receivers offset +0.5V (buffered) - AMC1311 fail-safe now
  distinguishable from a dead bus
- F44 VBAT_H/L actually sourced (FVBH/FVBL polyfuses off NRC)
- F45 real package pins everywhere: 74LVC1G11 (had NO VCC pin), 1G32,
  NCV4276C (OUT=5), TPS55340 RTE16 (+SS cap +FREQ R), BUK9Y14 LFPAK56,
  ALM2402 PWP14 (+VCC_O, SHDN via 10k pullup), QA01C SIP-7, PESD as
  real 2/3-terminal parts, FS26 full LQFP-48+EP with VDIG/VBOS/
  bootstraps/DEBUG strap and DS unused-pin terminations; S32K396
  explicitly symbolic (no package table in DS - bind at layout)
- F46 hardware fault latch: FLT_HS/LS diode-OR -> LVC1G74 -> DRV_EN;
  any DESAT latches all six channels off until MCU clears
- NSI6611ASC-Q1SWR full ordering code (ASC variant)

erc-audit gains a rev-A.4 lock-in section (763 checks, 0 fail);
design-verify adds F37-F46 corner rows (60 PASS/3 WARN/0 FAIL);
pin-verify 1663/1663; card void gate 9->12% (49-pin FS26 monolith);
BOM Rs.70,059 @1k, 579 components, 180 lines. design-basis 11a
documents the full review response including the rege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
Parts:
- removed CDC1: 20uF, FilmCan37.5, symbol traction-r1:C
- removed JCBDN, JCBDP: STUD-M6, StudM6, symbol traction-r1:TERM_1
- removed JCBEN, JCBEP: STUD-M8, StudM8, symbol traction-r1:TERM_1
- removed JCBUN, JCBUP, JCBVN, JCBVP, JCBWN, JCBWP: TAB-M6, TabM6, symbol traction-r1:TERM_1
- added CDC14, CDC15, CDC16, CDC2, CDC3, CDC4, CDC5, CDC6, CDC7, CDC8, CDC9: 20uF, FilmCan37.5, symbol traction-r1:C
- JCBDN: renamed from CDC10; value 20uF -> STUD-M6; footprint FilmCan37.5 -> StudM6; symbol traction-r1:C -> traction-r1:TERM_1; LCSC C2840809 -> CLASS; MPN C3D1M206KFSA382 -> STUD-M6
- JCBDP: renamed from CDC11; value 20uF -> STUD-M6; footprint FilmCan37.5 -> StudM6; symbol traction-r1:C -> traction-r1:TERM_1; LCSC C2840809 -> CLASS; MPN C3D1M206KFSA382 -> STUD-M6
- JCBEN: renamed from CDC12; value 20uF -> STUD-M8; footprint FilmCan37.5 -> StudM8; symbol traction-r1:C -> traction-r1:TERM_1; LCSC C2840809 -> CLASS; MPN C3D1M206KFSA382 -> STUD-M8
- JCBEP: renamed from CDC13; value 20uF -> STUD-M8; footprint FilmCan37.5 -> StudM8; symbol traction-r1:C -> traction-r1:TERM_1; LCSC C2840809 -> CLASS; MPN C3D1M206KFSA382 -> STUD-M8
- JCBUN: renamed from CDC14; value 20uF -> TAB-M6; footprint FilmCan37.5 -> TabM6; symbol traction-r1:C -> traction-r1:TERM_1; LCSC C2840809 -> CLASS; MPN C3D1M206KFSA382 -> TAB-M6
- JCBUP: renamed from CDC15; value 20uF -> TAB-M6; footprint FilmCan37.5 -> TabM6; symbol traction-r1:C -> traction-r1:TERM_1; LCSC C2840809 -> CLASS; MPN C3D1M206KFSA382 -> TAB-M6
- JCBVN: renamed from CDC16; value 20uF -> TAB-M6; footprint FilmCan37.5 -> TabM6; symbol traction-r1:C -> traction-r1:TERM_1; LCSC C2840809 -> CLASS; MPN C3D1M206KFSA382 -> TAB-M6
- JCBVP: renamed from CDC2; value 20uF -> TAB-M6; footprint FilmCan37.5 -> TabM6; symbol traction-r1:C -> traction-r1:TERM_1; LCSC C2840809 -> CLASS; MPN C3D1M206KFSA382 -> TAB-M6
- JCBWN: renamed from CDC3; value 20uF -> TAB-M6; footprint FilmCan37.5 -> TabM6; symbol traction-r1:C -> traction-r1:TERM_1; LCSC C2840809 -> CLASS; MPN C3D1M206KFSA382 -> TAB-M6
- JCBWP: renamed from CDC4; value 20uF -> TAB-M6; footprint FilmCan37.5 -> TabM6; symbol traction-r1:C -> traction-r1:TERM_1; LCSC C2840809 -> CLASS; MPN C3D1M206KFSA382 -> TAB-M6
- renumbered CDC5 to CDC1, CDC6 to CDC10, CDC7 to CDC11, CDC8 to CDC12, CDC9 to CDC13
Connections:
- net DCN: now also JCBDN.1 (P), JCBEN.1 (P), JCBUN.1 (P), JCBVN.1 (P), JCBWN.1 (P), CDC14.2, CDC15.2, CDC16.2, CDC2.2, CDC3.2, CDC4.2, CDC5.2, CDC6.2, CDC7.2, CDC8.2, CDC9.2; no longer JCBDN.2, JCBDP.2, JCBEN.2, JCBEP.2, JCBUN.2, JCBUP.2, JCBVN.2, JCBVP.2, JCBWN.2, JCBWP.2
- net DCP: now also CDC14.1, CDC15.1, CDC16.1, CDC2.1, CDC3.1, CDC4.1, CDC5.1, CDC6.1, CDC7.1, CDC8.1, CDC9.1; no longer JCBDN.1, JCBEN.1, JCBUN.1, JCBVN.1, JCBWN.1
Other:
- note added: "220 kW pk Cap bank (HV, busbar) - 2 of 4 · rev A.4 · 2 sections · 26 components"
- note removed: "220 kW pk Cap bank (HV, busbar) - 2 of 4 · rev A.3 · 2 sections · 26 components"
- moved on the sheet: CDC1, CDC10, CDC11, CDC12, CDC13
Changed lines of the file:
@@
 Title "Traction Inverter — Cap bank (busbar assembly, 320 uF)"
 Date "2026-09-09"
-Rev "A.3"
+Rev "A.4"
 Comp "Traction Inverter 220 kW pk - Cap bank (HV, busbar), sheet 2 of 4"
 Comment1 "Inverter = Power board + Cap bank busbar + bolt-on Discharge board (all HV) + Control card (LV); safe state holds with any link lost"
@@
 $EndDescr
 Text Notes 600 5100 0    60   ~ 12
-220 kW pk Cap bank (HV, busbar) - 2 of 4   ·   rev A.3   ·   2 sections   ·   26 components
+220 kW pk Cap bank (HV, busbar) - 2 of 4   ·   rev A.4   ·   2 sections   ·   26 components
 Text Notes 600 5400 0    50   ~ 0
 NET NAMING: U<ref>_<PIN> = node at that IC pin   ·   R<stem>_M = series-pair midpoint   ·   R<stem>_<nm> = tap between R<stem>n/m   ·   all others are explicit design nets   ·   same name on another sheet = same net, joined only at the named connector/stud/tab
@@
 $Comp
 L traction-r1:TERM_1 JCBDN
-U 1 1 5E000113
+U 1 1 5E00011E
 P 1250 2350
 F 0 "JCBDN" H 1250 2190 50  0000 C CNN
@@
 $Comp
 L traction-r1:TERM_1 JCBDP
-U 1 1 5E000114
+U 1 1 5E00011F
 P 1250 1950
 F 0 "JCBDP" H 1250 1790 50  0000 C CNN
@@
 $Comp
 L traction-r1:TERM_1 JCBEN
-U 1 1 5E000115
+U 1 1 5E000120
 P 1250 1550
 F 0 "JCBEN" H 1250 1390 50  0000 C CNN
@@
 $Comp
 L traction-r1:TERM_1 JCBEP
-U 1 1 5E000116
+U 1 1 5E000121
 P 1250 1150
 F 0 "JCBEP" H 1250 990 50  0000 C CNN
@@
 $Comp
 L traction-r1:TERM_1 JCBUN
-U 1 1 5E000117
+U 1 1 5E000122
 P 2150 1550
 F 0 "JCBUN" H 2150 1390 50  0000 C CNN
@@
 $Comp
 L traction-r1:TERM_1 JCBUP
-U 1 1 5E000118
+U 1 1 5E000123
 P 2150 1150
 F 0 "JCBUP" H 2150 990 50  0000 C CNN
@@
 $Comp
 L traction-r1:TERM_1 JCBVN
-U 1 1 5E000119
+U 1 1 5E000124
 P 2150 2350
 F 0 "JCBVN" H 2150 2190 50  0000 C CNN
@@
 $Comp
 L traction-r1:TERM_1 JCBVP
-U 1 1 5E00011A
+U 1 1 5E000125
 P 2150 1950
 F 0 "JCBVP" H 2150 1790 50  0000 C CNN
@@
 $Comp
 L traction-r1:TERM_1 JCBWN
-U 1 1 5E00011B
+U 1 1 5E000126
 P 2150 3150
 F 0 "JCBWN" H 2150 2990 50  0000 C CNN
@@
 $Comp
 L traction-r1:TERM_1 JCBWP
-U 1 1 5E00011C
+U 1 1 5E000127
 P 2150 2750
 F 0 "JCBWP" H 2150 2590 50  0000 C CNN
@@
 $Comp
 L traction-r1:C CDC1
-U 1 1 5E00011D
+U 1 1 5E000128
 P 4550 1150
 F 0 "CDC1" H 4550 990 50  0000 C CNN
@@
 $Comp
 L traction-r1:C CDC10
-U 1 1 5E00011E
+U 1 1 5E000129
 P 6050 1550
 F 0 "CDC10" H 6050 1390 50  0000 C CNN
@@
 $Comp
 L traction-r1:C CDC11
-U 1 1 5E00011F
+U 1 1 5E00012A
 P 6050 1950
 F 0 "CDC11" H 6050 1790 50  0000 C CNN
@@
 $Comp
 L traction-r1:C CDC12
-U 1 1 5E000120
+U 1 1 5E00012B
 P 6050 2350
 F 0 "CDC12" H 6050 2190 50  0000 C CNN
@@
 $Comp
 L traction-r1:C CDC13
-U 1 1 5E000121
+U 1 1 5E00012C
 P 6050 2750
 F 0 "CDC13" H 6050 2590 50  0000 C CNN
@@
 $Comp
 L traction-r1:C CDC14
-U 1 1 5E000122
+U 1 1 5E00012D
 P 6050 3150
 F 0 "CDC14" H 6050 2990 50  0000 C CNN
@@
 $Comp
 L traction-r1:C CDC15
-U 1 1 5E000123
+U 1 1 5E00012E
 P 6050 3550
 F 0 "CDC15" H 6050 3390 50  0000 C CNN
@@
 $Comp
 L traction-r1:C CDC16
-U 1 1 5E000124
+U 1 1 5E00012F
 P 6050 3950
 F 0 "CDC16" H 6050 3790 50  0000 C CNN
@@
 $Comp
 L traction-r1:C CDC2
-U 1 1 5E000125
+U 1 1 5E000130
 P 4550 1550
 F 0 "CDC2" H 4550 1390 50  0000 C CNN
@@
 $Comp
 L traction-r1:C CDC3
-U 1 1 5E000126
+U 1 1 5E000131
 P 4550 1950
 F 0 "CDC3" H 4550 1790 50  0000 C CNN
@@
 $Comp
 L traction-r1:C CDC4
-U 1 1 5E000127
+U 1 1 5E000132
 P 4550 2350
 F 0 "CDC4" H 4550 2190 50  0000 C CNN
@@
 $Comp
 L traction-r1:C CDC5
-U 1 1 5E000128
+U 1 1 5E000133
 P 4550 2750
 F 0 "CDC5" H 4550 2590 50  0000 C CNN
@@
 $Comp
 L traction-r1:C CDC6
-U 1 1 5E000129
+U 1 1 5E000134
 P 4550 3150
 F 0 "CDC6" H 4550 2990 50  0000 C CNN
@@
 $Comp
 L traction-r1:C CDC7
-U 1 1 5E00012A
+U 1 1 5E000135
 P 4550 3550
 F 0 "CDC7" H 4550 3390 50  0000 C CNN
@@
 $Comp
 L traction-r1:C CDC8
-U 1 1 5E00012B
+U 1 1 5E000136
 P 4550 3950
 F 0 "CDC8" H 4550 3790 50  0000 C CNN
@@
 $Comp
 L traction-r1:C CDC9
-U 1 1 5E00012C
+U 1 1 5E000137
 P 6050 1150
 F 0 "CDC9" H 6050 990 50  0000 C CNN

Commit message: Rev A.4.1: second review round — 5 confirmed defects fixed (F47-F51)
- F47 AMC1311 real pins 2=IN/3=SHTDN (both VDC channels had them
  swapped: analog inputs grounded, SHTDN on the divider tap)
- F48 FS26 TRKIN is the VREF regulator's input supply -> VPRE
  (was grounded as an "unused tracker input"; VREF5 had no source)
- F49 TPS55340 pin 5 is SYNC (7V abs), not a second VIN -> DGND
- F50 FS26 caps to DS minimums: CVBOS 4.7uF, CSB6 4.7uF, CSB5 2.2uF
  (VREF COUT 1.1-3.3uF eff - third value found in the same audit)
- F51 V15 protective post-regulator NCV4276C-ADJ 40V/0.4A: boost
  pass-through (24V jump start / ~33V clamped load dump) can no longer
  reach the QA01C 13.5-16.5V window; boost output renamed V15B
- ASC/fault-latch interplay documented per NSI6611 DS (ASC overrides
  input side; DESAT + VCC2-UVLO outrank ASC)
- all five PDFs regenerate from one release (stale standalone A.3
  exports superseded); ERC gains A.4.1 assertions

Gates: 1674/1674 pins, ERC 769/0, design-verify 64P/3W/0F,
BOM Rs.70,074 @1k, 583 components, 184 lines.

Co-Authored-By: Claude Fable 5 <noreply@anthropic.com>
Parts:
- removed JCBDN, JCBDP: STUD-M6, StudM6, symbol traction-r1:TERM_1
- removed JCBEN, JCBEP: STUD-M8, StudM8, symbol traction-r1:TERM_1
- added CDC6, CDC7, CDC8, CDC9: 20uF, FilmCan37.5, symbol traction-r1:C
- JCBDN: renamed from JCBUN; value TAB-M6 -> STUD-M6; footprint TabM6 -> StudM6; MPN TAB-M6 -> STUD-M6
- JCBDP: renamed from JCBUP; value TAB-M6 -> STUD-M6; footprint TabM6 -> StudM6; MPN TAB-M6 -> STUD-M6
- JCBEN: renamed from JCBVN; value TAB-M6 -> STUD-M8; footprint TabM6 -> StudM8; MPN TAB-M6 -> STUD-M8
- JCBEP: renamed from JCBVP; value TAB-M6 -> STUD-M8; footprint TabM6 -> StudM8; MPN TAB-M6 -> STUD-M8
- JCBVN: renamed from CDC1; value 20uF -> TAB-M6; footprint FilmCan37.5 -> TabM6; symbol traction-r1:C -> traction-r1:TERM_1; LCSC C2840809 -> CLASS; MPN C3D1M206KFSA382 -> TAB-M6
- JCBVP: renamed from CDC10; value 20uF -> TAB-M6; footprint FilmCan37.5 -> TabM6; symbol traction-r1:C -> traction-r1:TERM_1; LCSC C2840809 -> CLASS; MPN C3D1M206KFSA382 -> TAB-M6
- JCBWN: renamed from CDC11; value 20uF -> TAB-M6; footprint FilmCan37.5 -> TabM6; symbol traction-r1:C -> traction-r1:TERM_1; LCSC C2840809 -> CLASS; MPN C3D1M206KFSA382 -> TAB-M6
- JCBWP: renamed from CDC12; value 20uF -> TAB-M6; footprint FilmCan37.5 -> TabM6; symbol traction-r1:C -> traction-r1:TERM_1; LCSC C2840809 -> CLASS; MPN C3D1M206KFSA382 -> TAB-M6
- renumbered CDC13 to CDC1, CDC14 to CDC10, CDC15 to CDC11, CDC16 to CDC12, CDC2 to CDC13, CDC3 to CDC14, CDC4 to CDC15, CDC5 to CDC16, CDC6 to CDC2, CDC7 to CDC3, CDC8 to CDC4, CDC9 to CDC5, JCBWN to JCBUN, JCBWP to JCBUP
Connections:
- net DCN: now also JCBVN.1 (P), JCBWN.1 (P), CDC6.2, CDC7.2, CDC8.2, CDC9.2; no longer JCBVN.2, JCBVP.2, JCBWN.2, JCBWP.2
- net DCP: now also CDC6.1, CDC7.1, CDC8.1, CDC9.1; no longer JCBVN.1, JCBWN.1
Other:
- note added: "220 kW pk Cap bank (HV, busbar) - 2 of 4 · rev A.4.1 · 2 sections · 26 components"
- note removed: "220 kW pk Cap bank (HV, busbar) - 2 of 4 · rev A.4 · 2 sections · 26 components"
- moved on the sheet: CDC1, CDC10, CDC11, CDC12, CDC13, CDC14, CDC15, CDC16, CDC2, CDC3, CDC4, CDC5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
Changed lines of the file:
@@
 Title "Traction Inverter — Cap bank (busbar assembly, 320 uF)"
 Date "2026-09-09"
-Rev "A.4"
+Rev "A.4.1"
 Comp "Traction Inverter 220 kW pk - Cap bank (HV, busbar), sheet 2 of 4"
 Comment1 "Inverter = Power board + Cap bank busbar + bolt-on Discharge board (all HV) + Control card (LV); safe state holds with any link lost"
@@
 $EndDescr
 Text Notes 600 5100 0    60   ~ 12
-220 kW pk Cap bank (HV, busbar) - 2 of 4   ·   rev A.4   ·   2 sections   ·   26 components
+220 kW pk Cap bank (HV, busbar) - 2 of 4   ·   rev A.4.1   ·   2 sections   ·   26 components
 Text Notes 600 5400 0    50   ~ 0
 NET NAMING: U<ref>_<PIN> = node at that IC pin   ·   R<stem>_M = series-pair midpoint   ·   R<stem>_<nm> = tap between R<stem>n/m   ·   all others are explicit design nets   ·   same name on another sheet = same net, joined only at the named connector/stud/tab
@@
 $Comp
 L traction-r1:TERM_1 JCBDN
-U 1 1 5E00011E
+U 1 1 5E000122
 P 1250 2350
 F 0 "JCBDN" H 1250 2190 50  0000 C CNN
@@
 $Comp
 L traction-r1:TERM_1 JCBDP
-U 1 1 5E00011F
+U 1 1 5E000123
 P 1250 1950
 F 0 "JCBDP" H 1250 1790 50  0000 C CNN
@@
 $Comp
 L traction-r1:TERM_1 JCBEN
-U 1 1 5E000120
+U 1 1 5E000124
 P 1250 1550
 F 0 "JCBEN" H 1250 1390 50  0000 C CNN
@@
 $Comp
 L traction-r1:TERM_1 JCBEP
-U 1 1 5E000121
+U 1 1 5E000125
 P 1250 1150
 F 0 "JCBEP" H 1250 990 50  0000 C CNN
@@
 $Comp
 L traction-r1:TERM_1 JCBUN
-U 1 1 5E000122
+U 1 1 5E000126
 P 2150 1550
 F 0 "JCBUN" H 2150 1390 50  0000 C CNN
@@
 $Comp
 L traction-r1:TERM_1 JCBUP
-U 1 1 5E000123
+U 1 1 5E000127
 P 2150 1150
 F 0 "JCBUP" H 2150 990 50  0000 C CNN
@@
 $Comp
 L traction-r1:TERM_1 JCBVN
-U 1 1 5E000124
+U 1 1 5E000128
 P 2150 2350
 F 0 "JCBVN" H 2150 2190 50  0000 C CNN
@@
 $Comp
 L traction-r1:TERM_1 JCBVP
-U 1 1 5E000125
+U 1 1 5E000129
 P 2150 1950
 F 0 "JCBVP" H 2150 1790 50  0000 C CNN
@@
 $Comp
 L traction-r1:TERM_1 JCBWN
-U 1 1 5E000126
+U 1 1 5E00012A
 P 2150 3150
 F 0 "JCBWN" H 2150 2990 50  0000 C CNN
@@
 $Comp
 L traction-r1:TERM_1 JCBWP
-U 1 1 5E000127
+U 1 1 5E00012B
 P 2150 2750
 F 0 "JCBWP" H 2150 2590 50  0000 C CNN
@@
 $Comp
 L traction-r1:C CDC1
-U 1 1 5E000128
+U 1 1 5E00012C
 P 4550 1150
 F 0 "CDC1" H 4550 990 50  0000 C CNN
@@
 $Comp
 L traction-r1:C CDC10
-U 1 1 5E000129
+U 1 1 5E00012D
 P 6050 1550
 F 0 "CDC10" H 6050 1390 50  0000 C CNN
@@
 $Comp
 L traction-r1:C CDC11
-U 1 1 5E00012A
+U 1 1 5E00012E
 P 6050 1950
 F 0 "CDC11" H 6050 1790 50  0000 C CNN
@@
 $Comp
 L traction-r1:C CDC12
-U 1 1 5E00012B
+U 1 1 5E00012F
 P 6050 2350
 F 0 "CDC12" H 6050 2190 50  0000 C CNN
@@
 $Comp
 L traction-r1:C CDC13
-U 1 1 5E00012C
+U 1 1 5E000130
 P 6050 2750
 F 0 "CDC13" H 6050 2590 50  0000 C CNN
@@
 $Comp
 L traction-r1:C CDC14
-U 1 1 5E00012D
+U 1 1 5E000131
 P 6050 3150
 F 0 "CDC14" H 6050 2990 50  0000 C CNN
@@
 $Comp
 L traction-r1:C CDC15
-U 1 1 5E00012E
+U 1 1 5E000132
 P 6050 3550
 F 0 "CDC15" H 6050 3390 50  0000 C CNN
@@
 $Comp
 L traction-r1:C CDC16
-U 1 1 5E00012F
+U 1 1 5E000133
 P 6050 3950
 F 0 "CDC16" H 6050 3790 50  0000 C CNN
@@
 $Comp
 L traction-r1:C CDC2
-U 1 1 5E000130
+U 1 1 5E000134
 P 4550 1550
 F 0 "CDC2" H 4550 1390 50  0000 C CNN
@@
 $Comp
 L traction-r1:C CDC3
-U 1 1 5E000131
+U 1 1 5E000135
 P 4550 1950
 F 0 "CDC3" H 4550 1790 50  0000 C CNN
@@
 $Comp
 L traction-r1:C CDC4
-U 1 1 5E000132
+U 1 1 5E000136
 P 4550 2350
 F 0 "CDC4" H 4550 2190 50  0000 C CNN
@@
 $Comp
 L traction-r1:C CDC5
-U 1 1 5E000133
+U 1 1 5E000137
 P 4550 2750
 F 0 "CDC5" H 4550 2590 50  0000 C CNN
@@
 $Comp
 L traction-r1:C CDC6
-U 1 1 5E000134
+U 1 1 5E000138
 P 4550 3150
 F 0 "CDC6" H 4550 2990 50  0000 C CNN
@@
 $Comp
 L traction-r1:C CDC7
-U 1 1 5E000135
+U 1 1 5E000139
 P 4550 3550
 F 0 "CDC7" H 4550 3390 50  0000 C CNN
@@
 $Comp
 L traction-r1:C CDC8
-U 1 1 5E000136
+U 1 1 5E00013A
 P 4550 3950
 F 0 "CDC8" H 4550 3790 50  0000 C CNN
@@
 $Comp
 L traction-r1:C CDC9
-U 1 1 5E000137
+U 1 1 5E00013B
 P 6050 1150
 F 0 "CDC9" H 6050 990 50  0000 C CNN

Commit message: Rev A.4.2: third review round — 6 confirmed defects fixed (F52-F57)
- F52 FS26 buck passives to Table-106 selections: LCOR 2.2uH
  (CORE_LSEL_OTP=0x02; 4.7uH matched no listed value), V15S COUT
  2x22uF (~32uF eff vs 20-100 spec), CBTC 47nF, CBTP 22nF per
  CBOOT_PRE, VPRE COUT 2x22uF, CIN 22uF; effective-capacitance rows
  (bias/tol/temp derating) added to design-verify. VREF5 judged as a
  rail (CSB5+CMA1+CMA2 ~2.2uF eff, inside 1.1-3.3) per reviewer.
- F53 ACT45B CAN chokes: real windings are pins 1-4 and 2-3 (TDK
  circuit diagram) - both ports had transceiver CANH coupled onto
  external CANL; remapped, ERC asserts end-to-end pairing
- F54 ULDO15 completed: 220pF feed-forward across the 49.9k leg
  (fz 14.5kHz, onsemi 11-18kHz window), COUT 22uF
- F55 UEXD (ALM2402, 18V abs/16V rec) off raw VBATC -> behind ULDOEX
  12.1V (NCV4276C-ADJ); 24V jump start can no longer reach it
- F56 flyback switch BUK9Y14-80E (logic-level, VGS +/-10V DC) was
  outside abs-max at the 11.8V drive, masked by a 5.6V zener that
  conducted ~0.29A through every ON interval (~0.4W each). Now
  BUK7Y14-80E (standard-level +/-20V, same LFPAK56); zener repurposed
  to a dark 15V protective clamp
- F57 ordering code NCV4276CDTADJRKG (DT/ADJ were transposed)
- ASC-with-VCC1-open qualification documented (DESAT unavailable;
  double-fault given KL30-held V5GD) + IGN_SNS ADC disposition

Gates: 1691/1691 pins, ERC 779/0, design-verify 73P/3W/0F,
BOM Rs.70,090 @1k, 590 components, 192 lines.

Co-Authored-By: Claude Fable 5 <noreply@anthropic.com>
Parts:
- removed JCBDN: STUD-M6, StudM6, symbol traction-r1:TERM_1
- added CDC9: 20uF, FilmCan37.5, symbol traction-r1:C
- JCBDP: renamed from JCBEN; value STUD-M8 -> STUD-M6; footprint StudM8 -> StudM6; MPN STUD-M8 -> STUD-M6
- JCBEP: renamed from JCBUN; value TAB-M6 -> STUD-M8; footprint TabM6 -> StudM8; MPN TAB-M6 -> STUD-M8
- JCBWP: renamed from CDC1; value 20uF -> TAB-M6; footprint FilmCan37.5 -> TabM6; symbol traction-r1:C -> traction-r1:TERM_1; LCSC C2840809 -> CLASS; MPN C3D1M206KFSA382 -> TAB-M6
- renumbered CDC10 to CDC1, CDC11 to CDC10, CDC12 to CDC11, CDC13 to CDC12, CDC14 to CDC13, CDC15 to CDC14, CDC16 to CDC15, CDC2 to CDC16, CDC3 to CDC2, CDC4 to CDC3, CDC5 to CDC4, CDC6 to CDC5, CDC7 to CDC6, CDC8 to CDC7, CDC9 to CDC8, JCBDP to JCBDN, JCBEP to JCBEN, JCBUP to JCBUN, JCBVN to JCBUP, JCBVP to JCBVN, JCBWN to JCBVP, JCBWP to JCBWN
Connections:
- net DCN: now also JCBDN.1 (P), JCBEN.1 (P), JCBUN.1 (P), JCBVN.1 (P), JCBWN.1 (P), CDC9.2; no longer JCBDP.1 (P), JCBEP.1 (P), JCBUP.1 (P), JCBVP.1 (P), JCBWP.2
- net DCP: now also JCBDP.1 (P), JCBEP.1 (P), JCBUP.1 (P), JCBVP.1 (P), CDC9.1; no longer JCBDN.1 (P), JCBEN.1 (P), JCBUN.1 (P), JCBVN.1 (P), JCBWN.1 (P)
Other:
- note added: "220 kW pk Cap bank (HV, busbar) - 2 of 4 · rev A.4.2 · 2 sections · 26 components"
- note removed: "220 kW pk Cap bank (HV, busbar) - 2 of 4 · rev A.4.1 · 2 sections · 26 components"
- moved on the sheet: CDC1, CDC10, CDC11, CDC12, CDC13, CDC14, CDC15, CDC16, CDC2, CDC3, CDC4, CDC5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
Changed lines of the file:
@@
 Title "Traction Inverter — Cap bank (busbar assembly, 320 uF)"
 Date "2026-09-09"
-Rev "A.4.1"
+Rev "A.4.2"
 Comp "Traction Inverter 220 kW pk - Cap bank (HV, busbar), sheet 2 of 4"
 Comment1 "Inverter = Power board + Cap bank busbar + bolt-on Discharge board (all HV) + Control card (LV); safe state holds with any link lost"
@@
 $EndDescr
 Text Notes 600 5100 0    60   ~ 12
-220 kW pk Cap bank (HV, busbar) - 2 of 4   ·   rev A.4.1   ·   2 sections   ·   26 components
+220 kW pk Cap bank (HV, busbar) - 2 of 4   ·   rev A.4.2   ·   2 sections   ·   26 components
 Text Notes 600 5400 0    50   ~ 0
 NET NAMING: U<ref>_<PIN> = node at that IC pin   ·   R<stem>_M = series-pair midpoint   ·   R<stem>_<nm> = tap between R<stem>n/m   ·   all others are explicit design nets   ·   same name on another sheet = same net, joined only at the named connector/stud/tab
@@
 $Comp
 L traction-r1:TERM_1 JCBDN
-U 1 1 5E000122
+U 1 1 5E000123
 P 1250 2350
 F 0 "JCBDN" H 1250 2190 50  0000 C CNN
@@
 $Comp
 L traction-r1:TERM_1 JCBDP
-U 1 1 5E000123
+U 1 1 5E000124
 P 1250 1950
 F 0 "JCBDP" H 1250 1790 50  0000 C CNN
@@
 $Comp
 L traction-r1:TERM_1 JCBEN
-U 1 1 5E000124
+U 1 1 5E000125
 P 1250 1550
 F 0 "JCBEN" H 1250 1390 50  0000 C CNN
@@
 $Comp
 L traction-r1:TERM_1 JCBEP
-U 1 1 5E000125
+U 1 1 5E000126
 P 1250 1150
 F 0 "JCBEP" H 1250 990 50  0000 C CNN
@@
 $Comp
 L traction-r1:TERM_1 JCBUN
-U 1 1 5E000126
+U 1 1 5E000127
 P 2150 1550
 F 0 "JCBUN" H 2150 1390 50  0000 C CNN
@@
 $Comp
 L traction-r1:TERM_1 JCBUP
-U 1 1 5E000127
+U 1 1 5E000128
 P 2150 1150
 F 0 "JCBUP" H 2150 990 50  0000 C CNN
@@
 $Comp
 L traction-r1:TERM_1 JCBVN
-U 1 1 5E000128
+U 1 1 5E000129
 P 2150 2350
 F 0 "JCBVN" H 2150 2190 50  0000 C CNN
@@
 $Comp
 L traction-r1:TERM_1 JCBVP
-U 1 1 5E000129
+U 1 1 5E00012A
 P 2150 1950
 F 0 "JCBVP" H 2150 1790 50  0000 C CNN
@@
 $Comp
 L traction-r1:TERM_1 JCBWN
-U 1 1 5E00012A
+U 1 1 5E00012B
 P 2150 3150
 F 0 "JCBWN" H 2150 2990 50  0000 C CNN
@@
 $Comp
 L traction-r1:TERM_1 JCBWP
-U 1 1 5E00012B
+U 1 1 5E00012C
 P 2150 2750
 F 0 "JCBWP" H 2150 2590 50  0000 C CNN
@@
 $Comp
 L traction-r1:C CDC1
-U 1 1 5E00012C
+U 1 1 5E00012D
 P 4550 1150
 F 0 "CDC1" H 4550 990 50  0000 C CNN
@@
 $Comp
 L traction-r1:C CDC10
-U 1 1 5E00012D
+U 1 1 5E00012E
 P 6050 1550
 F 0 "CDC10" H 6050 1390 50  0000 C CNN
@@
 $Comp
 L traction-r1:C CDC11
-U 1 1 5E00012E
+U 1 1 5E00012F
 P 6050 1950
 F 0 "CDC11" H 6050 1790 50  0000 C CNN
@@
 $Comp
 L traction-r1:C CDC12
-U 1 1 5E00012F
+U 1 1 5E000130
 P 6050 2350
 F 0 "CDC12" H 6050 2190 50  0000 C CNN
@@
 $Comp
 L traction-r1:C CDC13
-U 1 1 5E000130
+U 1 1 5E000131
 P 6050 2750
 F 0 "CDC13" H 6050 2590 50  0000 C CNN
@@
 $Comp
 L traction-r1:C CDC14
-U 1 1 5E000131
+U 1 1 5E000132
 P 6050 3150
 F 0 "CDC14" H 6050 2990 50  0000 C CNN
@@
 $Comp
 L traction-r1:C CDC15
-U 1 1 5E000132
+U 1 1 5E000133
 P 6050 3550
 F 0 "CDC15" H 6050 3390 50  0000 C CNN
@@
 $Comp
 L traction-r1:C CDC16
-U 1 1 5E000133
+U 1 1 5E000134
 P 6050 3950
 F 0 "CDC16" H 6050 3790 50  0000 C CNN
@@
 $Comp
 L traction-r1:C CDC2
-U 1 1 5E000134
+U 1 1 5E000135
 P 4550 1550
 F 0 "CDC2" H 4550 1390 50  0000 C CNN
@@
 $Comp
 L traction-r1:C CDC3
-U 1 1 5E000135
+U 1 1 5E000136
 P 4550 1950
 F 0 "CDC3" H 4550 1790 50  0000 C CNN
@@
 $Comp
 L traction-r1:C CDC4
-U 1 1 5E000136
+U 1 1 5E000137
 P 4550 2350
 F 0 "CDC4" H 4550 2190 50  0000 C CNN
@@
 $Comp
 L traction-r1:C CDC5
-U 1 1 5E000137
+U 1 1 5E000138
 P 4550 2750
 F 0 "CDC5" H 4550 2590 50  0000 C CNN
@@
 $Comp
 L traction-r1:C CDC6
-U 1 1 5E000138
+U 1 1 5E000139
 P 4550 3150
 F 0 "CDC6" H 4550 2990 50  0000 C CNN
@@
 $Comp
 L traction-r1:C CDC7
-U 1 1 5E000139
+U 1 1 5E00013A
 P 4550 3550
 F 0 "CDC7" H 4550 3390 50  0000 C CNN
@@
 $Comp
 L traction-r1:C CDC8
-U 1 1 5E00013A
+U 1 1 5E00013B
 P 4550 3950
 F 0 "CDC8" H 4550 3790 50  0000 C CNN
@@
 $Comp
 L traction-r1:C CDC9
-U 1 1 5E00013B
+U 1 1 5E00013C
 P 6050 1150
 F 0 "CDC9" H 6050 990 50  0000 C CNN
