File: kicad5/traction/traction-capbank.sch (KiCad schematic (older format))
At the start: 26 parts

Commit message: Rev A.6: review round 6 response, one platform / four SKUs, N7-N9
External review round 6 (46 findings, R-F01..R-F46) was verified finding by
finding and classified in docs/review-A6-disposition.md (+ .csv): 20
Confirmed, 9 Already Fixed, 6 Firmware Handled, 5 Not Applicable,
6 Improvement Recommended. Repo findings F63-F76 are in the verification log.

Hardware (+Rs31/unit, all SKUs unless noted):
- SiC gate 3.3/6.8 ohm; IGBT 1.0/1.0 ohm + 82 pF DESAT blanking (HCG600
  short-circuit rating is 6 us, not 10)
- gate-power flyback start: 2.2 k + 47 uF VDD + 18 V VDD zener (UCC28C40 has
  0.4 V UVLO hysteresis and no clamp); IGBT builds use RT 8.2 k for margin
- fault latch: 10 k / 3.3 nF delay + 15 nF clear one-shot (NSI6611 FLT clears
  only on an EN rising edge, so a fault-dominant latch would deadlock)
- bleeder 2 x 6 x 22 k; HW_ID identity (harness pin 40) and VOFS to the MCU;
  resolver shields to DGND

Platform: one set of PCBs, four SKUs (8XX SiC/IGBT, 4XX IGBT/SiC).
- SKU rows in parts-db, selected by BOM_VARIANT in bom-gen; bom-gen now fails
  on any value/MPN mismatch
- shared calculations/loss-model.mjs
- docs/firmware-contract.md: FW-01..21, safe-state matrix, regen ownership
  (section 4b)
- docs/variants.md: business case

New Road findings:
- N7: LEM HC5FW 900-S/SP1 is a reduced-insulation part, so the phase busbar
  needs a rated sleeve
- N8: TLP152 is UL1577-only; order the (V4) VDE option or an SO6L part
- N9: FW-06 overvoltage response tightened from 100 us to 20 us. With the
  battery path lost at full regen the link reaches 962 V at 100 us and 897 V
  at 20 us; design-verify now checks it

Gates: 602 comps, 1717/1717 pins, ERC 816/0, design-verify 102P/11W/0F,
sim 24P/4W/0F, BOM SiC Rs70,965 / IGBT Rs45,465 @1k.

Co-Authored-By: Claude Opus 5.5 <noreply@anthropic.com>
Parts:
- removed JCBDN, JCBDP: STUD-M6, StudM6, symbol traction-r1:TERM_1
- removed JCBEN: STUD-M8, StudM8, symbol traction-r1:TERM_1
- added CDC7, CDC8, CDC9: 20uF, FilmCan37.5, symbol traction-r1:C
- JCBDN: renamed from JCBEP; value STUD-M8 -> STUD-M6; footprint StudM8 -> StudM6; MPN STUD-M8 -> STUD-M6
- JCBDP: renamed from JCBUN; value TAB-M6 -> STUD-M6; footprint TabM6 -> StudM6; MPN TAB-M6 -> STUD-M6
- JCBEN: renamed from JCBUP; value TAB-M6 -> STUD-M8; footprint TabM6 -> StudM8; MPN TAB-M6 -> STUD-M8
- JCBEP: renamed from JCBVN; value TAB-M6 -> STUD-M8; footprint TabM6 -> StudM8; MPN TAB-M6 -> STUD-M8
- JCBVP: renamed from CDC1; value 20uF -> TAB-M6; footprint FilmCan37.5 -> TabM6; symbol traction-r1:C -> traction-r1:TERM_1; LCSC C2840809 -> CLASS; MPN C3D1M206KFSA382 -> TAB-M6
- JCBWN: renamed from CDC10; value 20uF -> TAB-M6; footprint FilmCan37.5 -> TabM6; symbol traction-r1:C -> traction-r1:TERM_1; LCSC C2840809 -> CLASS; MPN C3D1M206KFSA382 -> TAB-M6
- JCBWP: renamed from CDC11; value 20uF -> TAB-M6; footprint FilmCan37.5 -> TabM6; symbol traction-r1:C -> traction-r1:TERM_1; LCSC C2840809 -> CLASS; MPN C3D1M206KFSA382 -> TAB-M6
- renumbered CDC12 to CDC1, CDC13 to CDC10, CDC14 to CDC11, CDC15 to CDC12, CDC16 to CDC13, CDC2 to CDC14, CDC3 to CDC15, CDC4 to CDC16, CDC5 to CDC2, CDC6 to CDC3, CDC7 to CDC4, CDC8 to CDC5, CDC9 to CDC6, JCBVP to JCBUN, JCBWN to JCBUP, JCBWP to JCBVN
Connections:
- net DCN: now also JCBDN.1 (P), JCBEN.1 (P), JCBUN.1 (P), JCBVN.1 (P), JCBWN.1 (P), CDC7.2, CDC8.2, CDC9.2; no longer JCBDP.1 (P), JCBEP.1 (P), JCBUP.1 (P), JCBVP.2, JCBWN.2, JCBWP.2
- net DCP: now also JCBDP.1 (P), JCBEP.1 (P), JCBUP.1 (P), CDC7.1, CDC8.1, CDC9.1; no longer JCBDN.1 (P), JCBEN.1 (P), JCBUN.1 (P), JCBVN.1 (P), JCBWN.1
Other:
- note added: "220 kW pk Cap bank (HV, busbar) - 2 of 4 · rev A.6 · 2 sections · 26 components"
- note removed: "220 kW pk Cap bank (HV, busbar) - 2 of 4 · rev A.5 · 2 sections · 26 components"
- moved on the sheet: CDC1, CDC10, CDC11, CDC12, CDC13, CDC14, CDC15, CDC16, CDC2, CDC3, CDC4, CDC5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
Changed lines of the file:
@@
 Sheet 1 1
 Title "Traction Inverter — Cap bank (busbar assembly, 320 uF)"
-Date "2026-09-09"
-Rev "A.5"
+Date "2026-09-23"
+Rev "A.6"
 Comp "Traction Inverter 220 kW pk - Cap bank (HV, busbar), sheet 2 of 4"
 Comment1 "Inverter = Power board + Cap bank busbar + bolt-on Discharge board (all HV) + Control card (LV); safe state holds with any link lost"
@@
 $EndDescr
 Text Notes 600 5100 0    60   ~ 12
-220 kW pk Cap bank (HV, busbar) - 2 of 4   ·   rev A.5   ·   2 sections   ·   26 components
+220 kW pk Cap bank (HV, busbar) - 2 of 4   ·   rev A.6   ·   2 sections   ·   26 components
 Text Notes 600 5400 0    50   ~ 0
 NET NAMING: U<ref>_<PIN> = node at that IC pin   ·   R<stem>_M = series-pair midpoint   ·   R<stem>_<nm> = tap between R<stem>n/m   ·   all others are explicit design nets   ·   same name on another sheet = same net, joined only at the named connector/stud/tab
@@
 $Comp
 L traction-r1:TERM_1 JCBDN
-U 1 1 5E000125
+U 1 1 5E000128
 P 1250 2350
 F 0 "JCBDN" H 1250 2190 50  0000 C CNN
@@
 $Comp
 L traction-r1:TERM_1 JCBDP
-U 1 1 5E000126
+U 1 1 5E000129
 P 1250 1950
 F 0 "JCBDP" H 1250 1790 50  0000 C CNN
@@
 $Comp
 L traction-r1:TERM_1 JCBEN
-U 1 1 5E000127
+U 1 1 5E00012A
 P 1250 1550
 F 0 "JCBEN" H 1250 1390 50  0000 C CNN
@@
 $Comp
 L traction-r1:TERM_1 JCBEP
-U 1 1 5E000128
+U 1 1 5E00012B
 P 1250 1150
 F 0 "JCBEP" H 1250 990 50  0000 C CNN
@@
 $Comp
 L traction-r1:TERM_1 JCBUN
-U 1 1 5E000129
+U 1 1 5E00012C
 P 2150 1550
 F 0 "JCBUN" H 2150 1390 50  0000 C CNN
@@
 $Comp
 L traction-r1:TERM_1 JCBUP
-U 1 1 5E00012A
+U 1 1 5E00012D
 P 2150 1150
 F 0 "JCBUP" H 2150 990 50  0000 C CNN
@@
 $Comp
 L traction-r1:TERM_1 JCBVN
-U 1 1 5E00012B
+U 1 1 5E00012E
 P 2150 2350
 F 0 "JCBVN" H 2150 2190 50  0000 C CNN
@@
 $Comp
 L traction-r1:TERM_1 JCBVP
-U 1 1 5E00012C
+U 1 1 5E00012F
 P 2150 1950
 F 0 "JCBVP" H 2150 1790 50  0000 C CNN
@@
 $Comp
 L traction-r1:TERM_1 JCBWN
-U 1 1 5E00012D
+U 1 1 5E000130
 P 2150 3150
 F 0 "JCBWN" H 2150 2990 50  0000 C CNN
@@
 $Comp
 L traction-r1:TERM_1 JCBWP
-U 1 1 5E00012E
+U 1 1 5E000131
 P 2150 2750
 F 0 "JCBWP" H 2150 2590 50  0000 C CNN
@@
 $Comp
 L traction-r1:C CDC1
-U 1 1 5E00012F
+U 1 1 5E000132
 P 4550 1150
 F 0 "CDC1" H 4550 990 50  0000 C CNN
@@
 $Comp
 L traction-r1:C CDC10
-U 1 1 5E000130
+U 1 1 5E000133
 P 6050 1550
 F 0 "CDC10" H 6050 1390 50  0000 C CNN
@@
 $Comp
 L traction-r1:C CDC11
-U 1 1 5E000131
+U 1 1 5E000134
 P 6050 1950
 F 0 "CDC11" H 6050 1790 50  0000 C CNN
@@
 $Comp
 L traction-r1:C CDC12
-U 1 1 5E000132
+U 1 1 5E000135
 P 6050 2350
 F 0 "CDC12" H 6050 2190 50  0000 C CNN
@@
 $Comp
 L traction-r1:C CDC13
-U 1 1 5E000133
+U 1 1 5E000136
 P 6050 2750
 F 0 "CDC13" H 6050 2590 50  0000 C CNN
@@
 $Comp
 L traction-r1:C CDC14
-U 1 1 5E000134
+U 1 1 5E000137
 P 6050 3150
 F 0 "CDC14" H 6050 2990 50  0000 C CNN
@@
 $Comp
 L traction-r1:C CDC15
-U 1 1 5E000135
+U 1 1 5E000138
 P 6050 3550
 F 0 "CDC15" H 6050 3390 50  0000 C CNN
@@
 $Comp
 L traction-r1:C CDC16
-U 1 1 5E000136
+U 1 1 5E000139
 P 6050 3950
 F 0 "CDC16" H 6050 3790 50  0000 C CNN
@@
 $Comp
 L traction-r1:C CDC2
-U 1 1 5E000137
+U 1 1 5E00013A
 P 4550 1550
 F 0 "CDC2" H 4550 1390 50  0000 C CNN
@@
 $Comp
 L traction-r1:C CDC3
-U 1 1 5E000138
+U 1 1 5E00013B
 P 4550 1950
 F 0 "CDC3" H 4550 1790 50  0000 C CNN
@@
 $Comp
 L traction-r1:C CDC4
-U 1 1 5E000139
+U 1 1 5E00013C
 P 4550 2350
 F 0 "CDC4" H 4550 2190 50  0000 C CNN
@@
 $Comp
 L traction-r1:C CDC5
-U 1 1 5E00013A
+U 1 1 5E00013D
 P 4550 2750
 F 0 "CDC5" H 4550 2590 50  0000 C CNN
@@
 $Comp
 L traction-r1:C CDC6
-U 1 1 5E00013B
+U 1 1 5E00013E
 P 4550 3150
 F 0 "CDC6" H 4550 2990 50  0000 C CNN
@@
 $Comp
 L traction-r1:C CDC7
-U 1 1 5E00013C
+U 1 1 5E00013F
 P 4550 3550
 F 0 "CDC7" H 4550 3390 50  0000 C CNN
@@
 $Comp
 L traction-r1:C CDC8
-U 1 1 5E00013D
+U 1 1 5E000140
 P 4550 3950
 F 0 "CDC8" H 4550 3790 50  0000 C CNN
@@
 $Comp
 L traction-r1:C CDC9
-U 1 1 5E00013E
+U 1 1 5E000141
 P 6050 1150
 F 0 "CDC9" H 6050 990 50  0000 C CNN

Commit message: Rev A.7: review round 7 response (RR01-RR10, A6-R01-R14) + cross-check
Two independent rechecks of c963794 were verified finding by finding and
classified in docs/review-A7-disposition.md (+ .csv): 17 confirmed and fixed,
1 spec gap closed, 3 firmware handled, 3 already-tracked release gates. Two
further defects were self-found (N10, N11).

Safety logic (control card):
- 74LVC3G17-Q100 Schmitt buffer between the RC timing nodes (clear one-shot,
  soft-off delay) and the LVC inputs they drove at 14,000-63,500 ns/V. The
  FS0B line goes through it too; a 100 k pull-down makes a dead buffer
  force DRV_EN low.
- FS0B/FS1B pull-ups 1 k -> 5.1 k (FS1B inside its 2 mA V_OL point).
- FAULT_OUT made sink-only (BAT46): a grounded vehicle wire can no longer
  preset ASC. A KL30 short is clamped at the latch.
- DRV_EN and ASC_CMD read-backs to the MCU for a boot self-test.
- Latches moved to Nexperia 74LVC1G74DC-Q100 (the TI part is not Q100).
- CCLR changed to C0G.

ASC entry is now break-before-make:
- A 12 nF delay (+ fast-release diode) holds the LS ASC off >= 3.4 us.
- MCU path: HS off via the eFlexPWM fault, then PWM-ASC with EN high.
- MCU-dead path: FS0B, then the delayed ASC.
- EN is never dropped for ASC: NSI6611 DS 8.12 honours DESAT over ASC only
  with EN high. The first draft's DASC diode did drop it and was removed
  after the cross-check.
- 1 k series resistor at each LS ASC pin.
- ASC opto LED resistor 470 -> 270 R (TLP152 I_FLH max 7.5 mA).

Gate supply:
- The flyback FB divider senses its own aux rectifier, so the start feed
  can no longer lock gate power out at high KL30.
- 52.3k/15k: VCC2 15.4 V nominal, 13.54-16.7 V corners.
- Boost output capacitors 25 V -> 50 V.

Models and checkers:
- IGBT and diode share the coldplate term.
- Flyback bank inductance corrected.
- SC soft-off checked at both I_STO corners (release gate).
- FW-06 as a measured budget: 15.6 us + 7.0 us all-off -> 905/542 V.
- bom-gen preflight and a JSWD pin-count check (Samtec 10-pin).
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
Parts:
- removed CDC1: 20uF, FilmCan37.5, symbol traction-r1:C
- removed JCBDN, JCBDP: STUD-M6, StudM6, symbol traction-r1:TERM_1
- removed JCBEN, JCBEP: STUD-M8, StudM8, symbol traction-r1:TERM_1
- removed JCBUN, JCBUP, JCBVN, JCBVP, JCBWN, JCBWP: TAB-M6, TabM6, symbol traction-r1:TERM_1
- added CDC14, CDC15, CDC16, CDC2, CDC3, CDC4, CDC5, CDC6, CDC7, CDC8, CDC9: 20uF, FilmCan37.5, symbol traction-r1:C
- JCBDN: renamed from CDC10; value 20uF -> STUD-M6; footprint FilmCan37.5 -> StudM6; symbol traction-r1:C -> traction-r1:TERM_1; LCSC C2840809 -> CLASS; MPN C3D1M206KFSA382 -> STUD-M6
- JCBDP: renamed from CDC11; value 20uF -> STUD-M6; footprint FilmCan37.5 -> StudM6; symbol traction-r1:C -> traction-r1:TERM_1; LCSC C2840809 -> CLASS; MPN C3D1M206KFSA382 -> STUD-M6
- JCBEN: renamed from CDC12; value 20uF -> STUD-M8; footprint FilmCan37.5 -> StudM8; symbol traction-r1:C -> traction-r1:TERM_1; LCSC C2840809 -> CLASS; MPN C3D1M206KFSA382 -> STUD-M8
- JCBEP: renamed from CDC13; value 20uF -> STUD-M8; footprint FilmCan37.5 -> StudM8; symbol traction-r1:C -> traction-r1:TERM_1; LCSC C2840809 -> CLASS; MPN C3D1M206KFSA382 -> STUD-M8
- JCBUN: renamed from CDC14; value 20uF -> TAB-M6; footprint FilmCan37.5 -> TabM6; symbol traction-r1:C -> traction-r1:TERM_1; LCSC C2840809 -> CLASS; MPN C3D1M206KFSA382 -> TAB-M6
- JCBUP: renamed from CDC15; value 20uF -> TAB-M6; footprint FilmCan37.5 -> TabM6; symbol traction-r1:C -> traction-r1:TERM_1; LCSC C2840809 -> CLASS; MPN C3D1M206KFSA382 -> TAB-M6
- JCBVN: renamed from CDC16; value 20uF -> TAB-M6; footprint FilmCan37.5 -> TabM6; symbol traction-r1:C -> traction-r1:TERM_1; LCSC C2840809 -> CLASS; MPN C3D1M206KFSA382 -> TAB-M6
- JCBVP: renamed from CDC2; value 20uF -> TAB-M6; footprint FilmCan37.5 -> TabM6; symbol traction-r1:C -> traction-r1:TERM_1; LCSC C2840809 -> CLASS; MPN C3D1M206KFSA382 -> TAB-M6
- JCBWN: renamed from CDC3; value 20uF -> TAB-M6; footprint FilmCan37.5 -> TabM6; symbol traction-r1:C -> traction-r1:TERM_1; LCSC C2840809 -> CLASS; MPN C3D1M206KFSA382 -> TAB-M6
- JCBWP: renamed from CDC4; value 20uF -> TAB-M6; footprint FilmCan37.5 -> TabM6; symbol traction-r1:C -> traction-r1:TERM_1; LCSC C2840809 -> CLASS; MPN C3D1M206KFSA382 -> TAB-M6
- renumbered CDC5 to CDC1, CDC6 to CDC10, CDC7 to CDC11, CDC8 to CDC12, CDC9 to CDC13
Connections:
- net DCN: now also JCBDN.1 (P), JCBEN.1 (P), JCBUN.1 (P), JCBVN.1 (P), JCBWN.1 (P), CDC14.2, CDC15.2, CDC16.2, CDC2.2, CDC3.2, CDC4.2, CDC5.2, CDC6.2, CDC7.2, CDC8.2, CDC9.2; no longer JCBDN.2, JCBDP.2, JCBEN.2, JCBEP.2, JCBUN.2, JCBUP.2, JCBVN.2, JCBVP.2, JCBWN.2, JCBWP.2
- net DCP: now also CDC14.1, CDC15.1, CDC16.1, CDC2.1, CDC3.1, CDC4.1, CDC5.1, CDC6.1, CDC7.1, CDC8.1, CDC9.1; no longer JCBDN.1, JCBEN.1, JCBUN.1, JCBVN.1, JCBWN.1
Other:
- note added: "220 kW pk Cap bank (HV, busbar) - 2 of 4 · rev A.7 · 2 sections · 26 components"
- note removed: "220 kW pk Cap bank (HV, busbar) - 2 of 4 · rev A.6 · 2 sections · 26 components"
- moved on the sheet: CDC1, CDC10, CDC11, CDC12, CDC13
Changed lines of the file:
@@
 Title "Traction Inverter — Cap bank (busbar assembly, 320 uF)"
 Date "2026-09-23"
-Rev "A.6"
+Rev "A.7"
 Comp "Traction Inverter 220 kW pk - Cap bank (HV, busbar), sheet 2 of 4"
 Comment1 "Inverter = Power board + Cap bank busbar + bolt-on Discharge board (all HV) + Control card (LV); safe state holds with any link lost"
@@
 $EndDescr
 Text Notes 600 5100 0    60   ~ 12
-220 kW pk Cap bank (HV, busbar) - 2 of 4   ·   rev A.6   ·   2 sections   ·   26 components
+220 kW pk Cap bank (HV, busbar) - 2 of 4   ·   rev A.7   ·   2 sections   ·   26 components
 Text Notes 600 5400 0    50   ~ 0
 NET NAMING: U<ref>_<PIN> = node at that IC pin   ·   R<stem>_M = series-pair midpoint   ·   R<stem>_<nm> = tap between R<stem>n/m   ·   all others are explicit design nets   ·   same name on another sheet = same net, joined only at the named connector/stud/tab
@@
 $Comp
 L traction-r1:TERM_1 JCBDN
-U 1 1 5E000128
+U 1 1 5E000133
 P 1250 2350
 F 0 "JCBDN" H 1250 2190 50  0000 C CNN
@@
 $Comp
 L traction-r1:TERM_1 JCBDP
-U 1 1 5E000129
+U 1 1 5E000134
 P 1250 1950
 F 0 "JCBDP" H 1250 1790 50  0000 C CNN
@@
 $Comp
 L traction-r1:TERM_1 JCBEN
-U 1 1 5E00012A
+U 1 1 5E000135
 P 1250 1550
 F 0 "JCBEN" H 1250 1390 50  0000 C CNN
@@
 $Comp
 L traction-r1:TERM_1 JCBEP
-U 1 1 5E00012B
+U 1 1 5E000136
 P 1250 1150
 F 0 "JCBEP" H 1250 990 50  0000 C CNN
@@
 $Comp
 L traction-r1:TERM_1 JCBUN
-U 1 1 5E00012C
+U 1 1 5E000137
 P 2150 1550
 F 0 "JCBUN" H 2150 1390 50  0000 C CNN
@@
 $Comp
 L traction-r1:TERM_1 JCBUP
-U 1 1 5E00012D
+U 1 1 5E000138
 P 2150 1150
 F 0 "JCBUP" H 2150 990 50  0000 C CNN
@@
 $Comp
 L traction-r1:TERM_1 JCBVN
-U 1 1 5E00012E
+U 1 1 5E000139
 P 2150 2350
 F 0 "JCBVN" H 2150 2190 50  0000 C CNN
@@
 $Comp
 L traction-r1:TERM_1 JCBVP
-U 1 1 5E00012F
+U 1 1 5E00013A
 P 2150 1950
 F 0 "JCBVP" H 2150 1790 50  0000 C CNN
@@
 $Comp
 L traction-r1:TERM_1 JCBWN
-U 1 1 5E000130
+U 1 1 5E00013B
 P 2150 3150
 F 0 "JCBWN" H 2150 2990 50  0000 C CNN
@@
 $Comp
 L traction-r1:TERM_1 JCBWP
-U 1 1 5E000131
+U 1 1 5E00013C
 P 2150 2750
 F 0 "JCBWP" H 2150 2590 50  0000 C CNN
@@
 $Comp
 L traction-r1:C CDC1
-U 1 1 5E000132
+U 1 1 5E00013D
 P 4550 1150
 F 0 "CDC1" H 4550 990 50  0000 C CNN
@@
 $Comp
 L traction-r1:C CDC10
-U 1 1 5E000133
+U 1 1 5E00013E
 P 6050 1550
 F 0 "CDC10" H 6050 1390 50  0000 C CNN
@@
 $Comp
 L traction-r1:C CDC11
-U 1 1 5E000134
+U 1 1 5E00013F
 P 6050 1950
 F 0 "CDC11" H 6050 1790 50  0000 C CNN
@@
 $Comp
 L traction-r1:C CDC12
-U 1 1 5E000135
+U 1 1 5E000140
 P 6050 2350
 F 0 "CDC12" H 6050 2190 50  0000 C CNN
@@
 $Comp
 L traction-r1:C CDC13
-U 1 1 5E000136
+U 1 1 5E000141
 P 6050 2750
 F 0 "CDC13" H 6050 2590 50  0000 C CNN
@@
 $Comp
 L traction-r1:C CDC14
-U 1 1 5E000137
+U 1 1 5E000142
 P 6050 3150
 F 0 "CDC14" H 6050 2990 50  0000 C CNN
@@
 $Comp
 L traction-r1:C CDC15
-U 1 1 5E000138
+U 1 1 5E000143
 P 6050 3550
 F 0 "CDC15" H 6050 3390 50  0000 C CNN
@@
 $Comp
 L traction-r1:C CDC16
-U 1 1 5E000139
+U 1 1 5E000144
 P 6050 3950
 F 0 "CDC16" H 6050 3790 50  0000 C CNN
@@
 $Comp
 L traction-r1:C CDC2
-U 1 1 5E00013A
+U 1 1 5E000145
 P 4550 1550
 F 0 "CDC2" H 4550 1390 50  0000 C CNN
@@
 $Comp
 L traction-r1:C CDC3
-U 1 1 5E00013B
+U 1 1 5E000146
 P 4550 1950
 F 0 "CDC3" H 4550 1790 50  0000 C CNN
@@
 $Comp
 L traction-r1:C CDC4
-U 1 1 5E00013C
+U 1 1 5E000147
 P 4550 2350
 F 0 "CDC4" H 4550 2190 50  0000 C CNN
@@
 $Comp
 L traction-r1:C CDC5
-U 1 1 5E00013D
+U 1 1 5E000148
 P 4550 2750
 F 0 "CDC5" H 4550 2590 50  0000 C CNN
@@
 $Comp
 L traction-r1:C CDC6
-U 1 1 5E00013E
+U 1 1 5E000149
 P 4550 3150
 F 0 "CDC6" H 4550 2990 50  0000 C CNN
@@
 $Comp
 L traction-r1:C CDC7
-U 1 1 5E00013F
+U 1 1 5E00014A
 P 4550 3550
 F 0 "CDC7" H 4550 3390 50  0000 C CNN
@@
 $Comp
 L traction-r1:C CDC8
-U 1 1 5E000140
+U 1 1 5E00014B
 P 4550 3950
 F 0 "CDC8" H 4550 3790 50  0000 C CNN
@@
 $Comp
 L traction-r1:C CDC9
-U 1 1 5E000141
+U 1 1 5E00014C
 P 6050 1150
 F 0 "CDC9" H 6050 990 50  0000 C CNN
