File: kicad5/traction/traction-capbank.sch (KiCad schematic (older format))
At the start: 26 parts

Commit message: Rev A.12: round 13 rechecks (F135-F139), pin freeze (F140), barrier + orderability closure (F141-F142), Marine A.12, firmware
- Rechecks of 30ae0a2: §6 winding-energy rule at every speed; resolver 12 k series + 220 pF C_AAF
  (injection 2.92 mA with the MCU unpowered); verifier counts distinct assemblies; TPS55340-Q1 real
  ratings (38/40 V); NCV4276C thermal on the datasheet pad.
- MCU pin freeze: all 289 S32K396 balls bound from SPF-91122 rev C anchored on the DS supply balls
  (calculations/mcu-ballmap.json, docs/mcu-pin-manifest.md); seven port corrections; FS26 pins verified;
  ERC pin-freeze lock.
- Barrier closure: VOW3120-X017T optos and UCC14141-Q1 biases (shared IsoBias18 cell, single-output
  18.0 V) replace TLP152/QA01C-18; LED resistors 270 R; VY1 Y-caps; Samtec IPL1/IPD1 harness;
  Faratronic 4XX can; SQP10 discharge resistors; UCC12051-Q1 on the AVL.
- Tooling: ERC open-pin helper + HARNESS40 parser scoped to its block; kicad5-verify assembly-set guard.
- Marine ported to A.12 (86 PASS / 22 WARN / 0 FAIL); firmware/ (C11, 178 tests / 1209 checks).
- Docs: README, design-basis §6a/§8/§11l, dfm, variants, cost-rollup, EXTRACTED-PARAMS §27-30 +
  seven archived datasheets, review-A12-disposition (+CSV), regenerated sheets/PDFs/BOMs/previews.

ERC 933/0 · design-verify 123/19/0 · sim 23/6/0 · sheets 2027/2027.

Co-Authored-By: Claude Fable 5.1 <noreply@anthropic.com>
Parts:
- removed JCBDN, JCBDP: STUD-M6, StudM6, symbol traction-r1:TERM_1
- removed JCBEN, JCBEP: STUD-M8, StudM8, symbol traction-r1:TERM_1
- removed JCBUN, JCBUP, JCBVN, JCBVP, JCBWN: TAB-M6, TabM6, symbol traction-r1:TERM_1
- added CDC16, CDC2, CDC3, CDC4, CDC5, CDC6, CDC7, CDC8, CDC9: 20uF, FilmCan37.5, symbol traction-r1:C
- JCBDN: renamed from JCBWP; value TAB-M6 -> STUD-M6; footprint TabM6 -> StudM6; MPN TAB-M6 -> STUD-M6
- JCBDP: renamed from CDC1; value 20uF -> STUD-M6; footprint FilmCan37.5 -> StudM6; symbol traction-r1:C -> traction-r1:TERM_1; LCSC C2840809 -> CLASS; MPN C3D1M206KFSA382 -> STUD-M6
- JCBEN: renamed from CDC10; value 20uF -> STUD-M8; footprint FilmCan37.5 -> StudM8; symbol traction-r1:C -> traction-r1:TERM_1; LCSC C2840809 -> CLASS; MPN C3D1M206KFSA382 -> STUD-M8
- JCBEP: renamed from CDC11; value 20uF -> STUD-M8; footprint FilmCan37.5 -> StudM8; symbol traction-r1:C -> traction-r1:TERM_1; LCSC C2840809 -> CLASS; MPN C3D1M206KFSA382 -> STUD-M8
- JCBUN: renamed from CDC12; value 20uF -> TAB-M6; footprint FilmCan37.5 -> TabM6; symbol traction-r1:C -> traction-r1:TERM_1; LCSC C2840809 -> CLASS; MPN C3D1M206KFSA382 -> TAB-M6
- JCBUP: renamed from CDC13; value 20uF -> TAB-M6; footprint FilmCan37.5 -> TabM6; symbol traction-r1:C -> traction-r1:TERM_1; LCSC C2840809 -> CLASS; MPN C3D1M206KFSA382 -> TAB-M6
- JCBVN: renamed from CDC14; value 20uF -> TAB-M6; footprint FilmCan37.5 -> TabM6; symbol traction-r1:C -> traction-r1:TERM_1; LCSC C2840809 -> CLASS; MPN C3D1M206KFSA382 -> TAB-M6
- JCBVP: renamed from CDC15; value 20uF -> TAB-M6; footprint FilmCan37.5 -> TabM6; symbol traction-r1:C -> traction-r1:TERM_1; LCSC C2840809 -> CLASS; MPN C3D1M206KFSA382 -> TAB-M6
- JCBWN: renamed from CDC16; value 20uF -> TAB-M6; footprint FilmCan37.5 -> TabM6; symbol traction-r1:C -> traction-r1:TERM_1; LCSC C2840809 -> CLASS; MPN C3D1M206KFSA382 -> TAB-M6
- JCBWP: renamed from CDC2; value 20uF -> TAB-M6; footprint FilmCan37.5 -> TabM6; symbol traction-r1:C -> traction-r1:TERM_1; LCSC C2840809 -> CLASS; MPN C3D1M206KFSA382 -> TAB-M6
- renumbered CDC3 to CDC1, CDC4 to CDC10, CDC5 to CDC11, CDC6 to CDC12, CDC7 to CDC13, CDC8 to CDC14, CDC9 to CDC15
Connections:
- net DCN: now also JCBDN.1 (P), JCBEN.1 (P), JCBUN.1 (P), JCBVN.1 (P), JCBWN.1 (P), CDC16.2, CDC2.2, CDC3.2, CDC4.2, CDC5.2, CDC6.2, CDC7.2, CDC8.2, CDC9.2; no longer JCBDP.2, JCBEN.2, JCBEP.2, JCBUN.2, JCBUP.2, JCBVN.2, JCBVP.2, JCBWN.2, JCBWP.2
- net DCP: now also CDC16.1, CDC2.1, CDC3.1, CDC4.1, CDC5.1, CDC6.1, CDC7.1, CDC8.1, CDC9.1; no longer JCBDN.1 (P), JCBEN.1, JCBUN.1, JCBVN.1, JCBWN.1
Other:
- note added: "220 kW pk Cap bank (HV, busbar) - 2 of 4 · rev A.12 · 2 sections · 26 components"
- note removed: "220 kW pk Cap bank (HV, busbar) - 2 of 4 · rev A.11 · 2 sections · 26 components"
- moved on the sheet: CDC1, CDC10, CDC11, CDC12, CDC13, CDC14, CDC15, JCBDN
Changed lines of the file:
@@
 Title "Traction Inverter — Cap bank (busbar assembly, 320 uF)"
 Date "2026-09-23"
-Rev "A.11"
+Rev "A.12"
 Comp "Traction Inverter 220 kW pk - Cap bank (HV, busbar), sheet 2 of 4"
 Comment1 "Inverter = Power board + Cap bank busbar + bolt-on Discharge board (all HV) + Control card (LV); safe state holds with any link lost"
@@
 $EndDescr
 Text Notes 600 5100 0    60   ~ 12
-220 kW pk Cap bank (HV, busbar) - 2 of 4   ·   rev A.11   ·   2 sections   ·   26 components
+220 kW pk Cap bank (HV, busbar) - 2 of 4   ·   rev A.12   ·   2 sections   ·   26 components
 Text Notes 600 5400 0    50   ~ 0
 NET NAMING: U<ref>_<PIN> = node at that IC pin   ·   R<stem>_M = series-pair midpoint   ·   R<stem>_<nm> = tap between R<stem>n/m   ·   all others are explicit design nets   ·   same name on another sheet = same net, joined only at the named connector/stud/tab
@@
 $Comp
 L traction-r1:TERM_1 JCBDN
-U 1 1 5E00013A
+U 1 1 5E000143
 P 1250 2350
 F 0 "JCBDN" H 1250 2190 50  0000 C CNN
@@
 $Comp
 L traction-r1:TERM_1 JCBDP
-U 1 1 5E00013B
+U 1 1 5E000144
 P 1250 1950
 F 0 "JCBDP" H 1250 1790 50  0000 C CNN
@@
 $Comp
 L traction-r1:TERM_1 JCBEN
-U 1 1 5E00013C
+U 1 1 5E000145
 P 1250 1550
 F 0 "JCBEN" H 1250 1390 50  0000 C CNN
@@
 $Comp
 L traction-r1:TERM_1 JCBEP
-U 1 1 5E00013D
+U 1 1 5E000146
 P 1250 1150
 F 0 "JCBEP" H 1250 990 50  0000 C CNN
@@
 $Comp
 L traction-r1:TERM_1 JCBUN
-U 1 1 5E00013E
+U 1 1 5E000147
 P 2150 1550
 F 0 "JCBUN" H 2150 1390 50  0000 C CNN
@@
 $Comp
 L traction-r1:TERM_1 JCBUP
-U 1 1 5E00013F
+U 1 1 5E000148
 P 2150 1150
 F 0 "JCBUP" H 2150 990 50  0000 C CNN
@@
 $Comp
 L traction-r1:TERM_1 JCBVN
-U 1 1 5E000140
+U 1 1 5E000149
 P 2150 2350
 F 0 "JCBVN" H 2150 2190 50  0000 C CNN
@@
 $Comp
 L traction-r1:TERM_1 JCBVP
-U 1 1 5E000141
+U 1 1 5E00014A
 P 2150 1950
 F 0 "JCBVP" H 2150 1790 50  0000 C CNN
@@
 $Comp
 L traction-r1:TERM_1 JCBWN
-U 1 1 5E000142
+U 1 1 5E00014B
 P 2150 3150
 F 0 "JCBWN" H 2150 2990 50  0000 C CNN
@@
 $Comp
 L traction-r1:TERM_1 JCBWP
-U 1 1 5E000143
+U 1 1 5E00014C
 P 2150 2750
 F 0 "JCBWP" H 2150 2590 50  0000 C CNN
@@
 $Comp
 L traction-r1:C CDC1
-U 1 1 5E000144
+U 1 1 5E00014D
 P 4550 1150
 F 0 "CDC1" H 4550 990 50  0000 C CNN
@@
 $Comp
 L traction-r1:C CDC10
-U 1 1 5E000145
+U 1 1 5E00014E
 P 6050 1550
 F 0 "CDC10" H 6050 1390 50  0000 C CNN
@@
 $Comp
 L traction-r1:C CDC11
-U 1 1 5E000146
+U 1 1 5E00014F
 P 6050 1950
 F 0 "CDC11" H 6050 1790 50  0000 C CNN
@@
 $Comp
 L traction-r1:C CDC12
-U 1 1 5E000147
+U 1 1 5E000150
 P 6050 2350
 F 0 "CDC12" H 6050 2190 50  0000 C CNN
@@
 $Comp
 L traction-r1:C CDC13
-U 1 1 5E000148
+U 1 1 5E000151
 P 6050 2750
 F 0 "CDC13" H 6050 2590 50  0000 C CNN
@@
 $Comp
 L traction-r1:C CDC14
-U 1 1 5E000149
+U 1 1 5E000152
 P 6050 3150
 F 0 "CDC14" H 6050 2990 50  0000 C CNN
@@
 $Comp
 L traction-r1:C CDC15
-U 1 1 5E00014A
+U 1 1 5E000153
 P 6050 3550
 F 0 "CDC15" H 6050 3390 50  0000 C CNN
@@
 $Comp
 L traction-r1:C CDC16
-U 1 1 5E00014B
+U 1 1 5E000154
 P 6050 3950
 F 0 "CDC16" H 6050 3790 50  0000 C CNN
@@
 $Comp
 L traction-r1:C CDC2
-U 1 1 5E00014C
+U 1 1 5E000155
 P 4550 1550
 F 0 "CDC2" H 4550 1390 50  0000 C CNN
@@
 $Comp
 L traction-r1:C CDC3
-U 1 1 5E00014D
+U 1 1 5E000156
 P 4550 1950
 F 0 "CDC3" H 4550 1790 50  0000 C CNN
@@
 $Comp
 L traction-r1:C CDC4
-U 1 1 5E00014E
+U 1 1 5E000157
 P 4550 2350
 F 0 "CDC4" H 4550 2190 50  0000 C CNN
@@
 $Comp
 L traction-r1:C CDC5
-U 1 1 5E00014F
+U 1 1 5E000158
 P 4550 2750
 F 0 "CDC5" H 4550 2590 50  0000 C CNN
@@
 $Comp
 L traction-r1:C CDC6
-U 1 1 5E000150
+U 1 1 5E000159
 P 4550 3150
 F 0 "CDC6" H 4550 2990 50  0000 C CNN
@@
 $Comp
 L traction-r1:C CDC7
-U 1 1 5E000151
+U 1 1 5E00015A
 P 4550 3550
 F 0 "CDC7" H 4550 3390 50  0000 C CNN
@@
 $Comp
 L traction-r1:C CDC8
-U 1 1 5E000152
+U 1 1 5E00015B
 P 4550 3950
 F 0 "CDC8" H 4550 3790 50  0000 C CNN
@@
 $Comp
 L traction-r1:C CDC9
-U 1 1 5E000153
+U 1 1 5E00015C
 P 6050 1150
 F 0 "CDC9" H 6050 990 50  0000 C CNN

Commit message: Rev A.13: round 14 — three reviews of cfd35a7 (F143-F158): MCU map vs NXP netlist, fail-closed firmware, terminal-fault protection
- Pin freeze reopened and closed: H5 is V15 (1.5 V, was on VREF5) and J7 is V25 (regulator output,
  was grounded); whole map re-derived against NXP's GEN3 net report NET-91122_C (U513, 244 balls) —
  every supply ball and 164/165 port names agree; HW_ID/NTC_A/MT2_SIG/ASC_REQ moved to netlist-confirmed
  balls (B5/T15/D5/U4); KiCad symbol numbered by physical ball, mutation-tested; CNMOS 1 nF.
- Firmware (214 tests / 1622 checks, ASan/UBSan, target-check): DESAT hold for every caller, 64-bit
  monotonic clock, keep_hv from rule (b) reliance at any speed, IMCR placeholders = build error,
  config-matches vs protection-locked, arming-evidence record (fail closed), torque feasibility witness,
  stuck-channel detection, stuck-on discharge detection; board map regenerated.
- Analog: excitation monitor 18 k/42.2 k/84.5 k + 220 pF C_AAF; exciter SMCJ8.5CA + MF-MSMF020 per line;
  motor-temp SMAJ5.0A + 0438.375WRA; bias-LDO 47 R ballast, UCC12051-Q1 primary; UCC14141-Q1 VDE cert.
- Docs: contract FW-22..FW-26 + keep_hv; design-basis §11m; variants/cost/dfm/README; disposition + CSV;
  EXTRACTED §31/§32 + archived datasheets; report-template defect fixed; Marine at A.13 (86/22/0).

ERC 945/0 · design-verify 130/23/0 · sim 23/6/0 · sheets 2045/2045 · BOM 8XX SiC ₹72,492.

Co-Authored-By: Claude Fable 5.1 <noreply@anthropic.com>
Parts:
- removed JCBDN, JCBDP: STUD-M6, StudM6, symbol traction-r1:TERM_1
- added CDC8, CDC9: 20uF, FilmCan37.5, symbol traction-r1:C
- JCBDN: renamed from JCBEN; value STUD-M8 -> STUD-M6; footprint StudM8 -> StudM6; MPN STUD-M8 -> STUD-M6
- JCBDP: renamed from JCBEP; value STUD-M8 -> STUD-M6; footprint StudM8 -> StudM6; MPN STUD-M8 -> STUD-M6
- JCBEN: renamed from JCBUN; value TAB-M6 -> STUD-M8; footprint TabM6 -> StudM8; MPN TAB-M6 -> STUD-M8
- JCBEP: renamed from JCBUP; value TAB-M6 -> STUD-M8; footprint TabM6 -> StudM8; MPN TAB-M6 -> STUD-M8
- JCBWN: renamed from CDC1; value 20uF -> TAB-M6; footprint FilmCan37.5 -> TabM6; symbol traction-r1:C -> traction-r1:TERM_1; LCSC C2840809 -> CLASS; MPN C3D1M206KFSA382 -> TAB-M6
- JCBWP: renamed from CDC10; value 20uF -> TAB-M6; footprint FilmCan37.5 -> TabM6; symbol traction-r1:C -> traction-r1:TERM_1; LCSC C2840809 -> CLASS; MPN C3D1M206KFSA382 -> TAB-M6
- renumbered CDC11 to CDC1, CDC12 to CDC10, CDC13 to CDC11, CDC14 to CDC12, CDC15 to CDC13, CDC16 to CDC14, CDC2 to CDC15, CDC3 to CDC16, CDC4 to CDC2, CDC5 to CDC3, CDC6 to CDC4, CDC7 to CDC5, CDC8 to CDC6, CDC9 to CDC7, JCBVN to JCBUN, JCBVP to JCBUP, JCBWN to JCBVN, JCBWP to JCBVP
Connections:
- net DCN: now also JCBWN.1 (P), CDC8.2, CDC9.2; no longer JCBWN.2, JCBWP.2
- net DCP: now also CDC8.1, CDC9.1; no longer JCBWN.1
Other:
- note added: "220 kW pk Cap bank (HV, busbar) - 2 of 4 · rev A.13 · 2 sections · 26 components"
- note removed: "220 kW pk Cap bank (HV, busbar) - 2 of 4 · rev A.12 · 2 sections · 26 components"
- moved on the sheet: CDC1, CDC10, CDC11, CDC12, CDC13, CDC14, CDC15, CDC16, CDC2, CDC3, CDC4, CDC5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
Changed lines of the file:
@@
 Title "Traction Inverter — Cap bank (busbar assembly, 320 uF)"
 Date "2026-09-23"
-Rev "A.12"
+Rev "A.13"
 Comp "Traction Inverter 220 kW pk - Cap bank (HV, busbar), sheet 2 of 4"
 Comment1 "Inverter = Power board + Cap bank busbar + bolt-on Discharge board (all HV) + Control card (LV); safe state holds with any link lost"
@@
 $EndDescr
 Text Notes 600 5100 0    60   ~ 12
-220 kW pk Cap bank (HV, busbar) - 2 of 4   ·   rev A.12   ·   2 sections   ·   26 components
+220 kW pk Cap bank (HV, busbar) - 2 of 4   ·   rev A.13   ·   2 sections   ·   26 components
 Text Notes 600 5400 0    50   ~ 0
 NET NAMING: U<ref>_<PIN> = node at that IC pin   ·   R<stem>_M = series-pair midpoint   ·   R<stem>_<nm> = tap between R<stem>n/m   ·   all others are explicit design nets   ·   same name on another sheet = same net, joined only at the named connector/stud/tab
@@
 $Comp
 L traction-r1:TERM_1 JCBDN
-U 1 1 5E000143
+U 1 1 5E000145
 P 1250 2350
 F 0 "JCBDN" H 1250 2190 50  0000 C CNN
@@
 $Comp
 L traction-r1:TERM_1 JCBDP
-U 1 1 5E000144
+U 1 1 5E000146
 P 1250 1950
 F 0 "JCBDP" H 1250 1790 50  0000 C CNN
@@
 $Comp
 L traction-r1:TERM_1 JCBEN
-U 1 1 5E000145
+U 1 1 5E000147
 P 1250 1550
 F 0 "JCBEN" H 1250 1390 50  0000 C CNN
@@
 $Comp
 L traction-r1:TERM_1 JCBEP
-U 1 1 5E000146
+U 1 1 5E000148
 P 1250 1150
 F 0 "JCBEP" H 1250 990 50  0000 C CNN
@@
 $Comp
 L traction-r1:TERM_1 JCBUN
-U 1 1 5E000147
+U 1 1 5E000149
 P 2150 1550
 F 0 "JCBUN" H 2150 1390 50  0000 C CNN
@@
 $Comp
 L traction-r1:TERM_1 JCBUP
-U 1 1 5E000148
+U 1 1 5E00014A
 P 2150 1150
 F 0 "JCBUP" H 2150 990 50  0000 C CNN
@@
 $Comp
 L traction-r1:TERM_1 JCBVN
-U 1 1 5E000149
+U 1 1 5E00014B
 P 2150 2350
 F 0 "JCBVN" H 2150 2190 50  0000 C CNN
@@
 $Comp
 L traction-r1:TERM_1 JCBVP
-U 1 1 5E00014A
+U 1 1 5E00014C
 P 2150 1950
 F 0 "JCBVP" H 2150 1790 50  0000 C CNN
@@
 $Comp
 L traction-r1:TERM_1 JCBWN
-U 1 1 5E00014B
+U 1 1 5E00014D
 P 2150 3150
 F 0 "JCBWN" H 2150 2990 50  0000 C CNN
@@
 $Comp
 L traction-r1:TERM_1 JCBWP
-U 1 1 5E00014C
+U 1 1 5E00014E
 P 2150 2750
 F 0 "JCBWP" H 2150 2590 50  0000 C CNN
@@
 $Comp
 L traction-r1:C CDC1
-U 1 1 5E00014D
+U 1 1 5E00014F
 P 4550 1150
 F 0 "CDC1" H 4550 990 50  0000 C CNN
@@
 $Comp
 L traction-r1:C CDC10
-U 1 1 5E00014E
+U 1 1 5E000150
 P 6050 1550
 F 0 "CDC10" H 6050 1390 50  0000 C CNN
@@
 $Comp
 L traction-r1:C CDC11
-U 1 1 5E00014F
+U 1 1 5E000151
 P 6050 1950
 F 0 "CDC11" H 6050 1790 50  0000 C CNN
@@
 $Comp
 L traction-r1:C CDC12
-U 1 1 5E000150
+U 1 1 5E000152
 P 6050 2350
 F 0 "CDC12" H 6050 2190 50  0000 C CNN
@@
 $Comp
 L traction-r1:C CDC13
-U 1 1 5E000151
+U 1 1 5E000153
 P 6050 2750
 F 0 "CDC13" H 6050 2590 50  0000 C CNN
@@
 $Comp
 L traction-r1:C CDC14
-U 1 1 5E000152
+U 1 1 5E000154
 P 6050 3150
 F 0 "CDC14" H 6050 2990 50  0000 C CNN
@@
 $Comp
 L traction-r1:C CDC15
-U 1 1 5E000153
+U 1 1 5E000155
 P 6050 3550
 F 0 "CDC15" H 6050 3390 50  0000 C CNN
@@
 $Comp
 L traction-r1:C CDC16
-U 1 1 5E000154
+U 1 1 5E000156
 P 6050 3950
 F 0 "CDC16" H 6050 3790 50  0000 C CNN
@@
 $Comp
 L traction-r1:C CDC2
-U 1 1 5E000155
+U 1 1 5E000157
 P 4550 1550
 F 0 "CDC2" H 4550 1390 50  0000 C CNN
@@
 $Comp
 L traction-r1:C CDC3
-U 1 1 5E000156
+U 1 1 5E000158
 P 4550 1950
 F 0 "CDC3" H 4550 1790 50  0000 C CNN
@@
 $Comp
 L traction-r1:C CDC4
-U 1 1 5E000157
+U 1 1 5E000159
 P 4550 2350
 F 0 "CDC4" H 4550 2190 50  0000 C CNN
@@
 $Comp
 L traction-r1:C CDC5
-U 1 1 5E000158
+U 1 1 5E00015A
 P 4550 2750
 F 0 "CDC5" H 4550 2590 50  0000 C CNN
@@
 $Comp
 L traction-r1:C CDC6
-U 1 1 5E000159
+U 1 1 5E00015B
 P 4550 3150
 F 0 "CDC6" H 4550 2990 50  0000 C CNN
@@
 $Comp
 L traction-r1:C CDC7
-U 1 1 5E00015A
+U 1 1 5E00015C
 P 4550 3550
 F 0 "CDC7" H 4550 3390 50  0000 C CNN
@@
 $Comp
 L traction-r1:C CDC8
-U 1 1 5E00015B
+U 1 1 5E00015D
 P 4550 3950
 F 0 "CDC8" H 4550 3790 50  0000 C CNN
@@
 $Comp
 L traction-r1:C CDC9
-U 1 1 5E00015C
+U 1 1 5E00015E
 P 6050 1150
 F 0 "CDC9" H 6050 990 50  0000 C CNN
