File: kicad/traction/traction-disch.kicad_sch (KiCad schematic)
At the start: 35 parts

Commit message: Rev A.17: round 18 — three rechecks of 4425af9 (F190-F198): diversion diodes on the amplifier node (loop passes RSX), diode cell cathode = pin 1 on all 35 diodes, exciter TVS/PTC rows at worst corners + ECU-asleep sustained short (WARN rows, layout rule, QP-RX-04 2b gate), anti-surge RSX, NCV4276C reverse current = QP-RX-05 gate + VR-33, IR-16/IR-42, firmware FW-34..36 (sample freshness, cadence-locked resolver frames, latency sign) + three self-found instances
Co-Authored-By: Claude Fable 5.1 <noreply@anthropic.com>
Other:
- note added: "220 kW pk Discharge (HV, bolt-on) - 3 of 4 · rev A.17 · 3 sections · 35 components"
- note removed: "220 kW pk Discharge (HV, bolt-on) - 3 of 4 · rev A.16 · 3 sections · 35 components"
Changed lines of the file:
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@@
 		(title "Traction Inverter — Discharge board (bolt-on, XM3 pattern)")
 		(date "2026-09-23")
-		(rev "A.16")
+		(rev "A.17")
 		(company "Traction Inverter 220 kW pk - Discharge (HV, bolt-on), sheet 3 of 4")
 		(comment 1 "Inverter = Power board + Cap bank busbar + bolt-on Discharge board (all HV) + Control card (LV); safe state holds with any link lost")
@@
 	(rectangle (start 190.5 12.7) (end 269.24 95.25) (stroke (width 0) (type dash)) (fill (type none)))
 	(rectangle (start 12.7 12.7) (end 180.34 177.8) (stroke (width 0) (type dash)) (fill (type none)))
-	(text "220 kW pk Discharge (HV, bolt-on) - 3 of 4   ·   rev A.16   ·   3 sections   ·   35 components" (exclude_from_sim no) (at 15.24 193.04 0) (effects (font (size 1.524 1.524) (bold yes)) (justify left bottom)))
+	(text "220 kW pk Discharge (HV, bolt-on) - 3 of 4   ·   rev A.17   ·   3 sections   ·   35 components" (exclude_from_sim no) (at 15.24 193.04 0) (effects (font (size 1.524 1.524) (bold yes)) (justify left bottom)))
 	(text "NET NAMING: U<ref>_<PIN> = node at that IC pin   ·   R<stem>_M = series-pair midpoint   ·   R<stem>_<nm> = tap between R<stem>n/m   ·   all others are explicit design nets   ·   same name on another sheet = same net, joined only at the named connector/stud/tab" (exclude_from_sim no) (at 15.24 200.66 0) (effects (font (size 1.27 1.27)) (justify left bottom)))
 	(text "DISCHARGE / ENTRY" (exclude_from_sim no) (at 192.024 112.014 0) (effects (font (size 2.0066 2.0066) (bold yes)) (justify left bottom)))

Commit message: Rev A.18: round 19 — three rechecks of e315bf1 (F199-F204): PTC-current row at every permitted voltage (IR-16 0.08/0.14/0.37/0.26 Ω), ≥8 A TVS energy an explicit assumption + QP-RX-04 release criterion, window criterion fixed, exciter TVS → SMDJ7.0A-HRA (coupled island holds the 7.0 V class at a parked 12 V battery / the Marine rail), shared exciter-fault model run for the Marine port (QP-MA-11, kit-loom rule), FW-35 rewritten on an SWG-anchored time origin with clock-derived resync and bounded restart
Co-Authored-By: Claude Fable 5.1 <noreply@anthropic.com>
Other:
- note added: "220 kW pk Discharge (HV, bolt-on) - 3 of 4 · rev A.18 · 3 sections · 35 components"
- note removed: "220 kW pk Discharge (HV, bolt-on) - 3 of 4 · rev A.17 · 3 sections · 35 components"
Changed lines of the file:
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@@
 		(title "Traction Inverter — Discharge board (bolt-on, XM3 pattern)")
 		(date "2026-09-23")
-		(rev "A.17")
+		(rev "A.18")
 		(company "Traction Inverter 220 kW pk - Discharge (HV, bolt-on), sheet 3 of 4")
 		(comment 1 "Inverter = Power board + Cap bank busbar + bolt-on Discharge board (all HV) + Control card (LV); safe state holds with any link lost")
@@
 	(rectangle (start 190.5 12.7) (end 269.24 95.25) (stroke (width 0) (type dash)) (fill (type none)))
 	(rectangle (start 12.7 12.7) (end 180.34 177.8) (stroke (width 0) (type dash)) (fill (type none)))
-	(text "220 kW pk Discharge (HV, bolt-on) - 3 of 4   ·   rev A.17   ·   3 sections   ·   35 components" (exclude_from_sim no) (at 15.24 193.04 0) (effects (font (size 1.524 1.524) (bold yes)) (justify left bottom)))
+	(text "220 kW pk Discharge (HV, bolt-on) - 3 of 4   ·   rev A.18   ·   3 sections   ·   35 components" (exclude_from_sim no) (at 15.24 193.04 0) (effects (font (size 1.524 1.524) (bold yes)) (justify left bottom)))
 	(text "NET NAMING: U<ref>_<PIN> = node at that IC pin   ·   R<stem>_M = series-pair midpoint   ·   R<stem>_<nm> = tap between R<stem>n/m   ·   all others are explicit design nets   ·   same name on another sheet = same net, joined only at the named connector/stud/tab" (exclude_from_sim no) (at 15.24 200.66 0) (effects (font (size 1.27 1.27)) (justify left bottom)))
 	(text "DISCHARGE / ENTRY" (exclude_from_sim no) (at 192.024 112.014 0) (effects (font (size 2.0066 2.0066) (bold yes)) (justify left bottom)))

Commit message: Rev A.19: round 20 — three rechecks of 00f6252 (F205-F207): TVS alternate to the 7.0 V class + lock, 4XX discharge alternate 470→220 Ω + lock, T-05/T-06 firmware ID, 8.5 V-era figures re-derived at the IR-16 allocations
Co-Authored-By: Claude Fable 5.1 <noreply@anthropic.com>
Other:
- note added: "220 kW pk Discharge (HV, bolt-on) - 3 of 4 · rev A.19 · 3 sections · 35 components"
- note removed: "220 kW pk Discharge (HV, bolt-on) - 3 of 4 · rev A.18 · 3 sections · 35 components"
Changed lines of the file:
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@@
 		(title "Traction Inverter — Discharge board (bolt-on, XM3 pattern)")
 		(date "2026-09-23")
-		(rev "A.18")
+		(rev "A.19")
 		(company "Traction Inverter 220 kW pk - Discharge (HV, bolt-on), sheet 3 of 4")
 		(comment 1 "Inverter = Power board + Cap bank busbar + bolt-on Discharge board (all HV) + Control card (LV); safe state holds with any link lost")
@@
 	(rectangle (start 190.5 12.7) (end 269.24 95.25) (stroke (width 0) (type dash)) (fill (type none)))
 	(rectangle (start 12.7 12.7) (end 180.34 177.8) (stroke (width 0) (type dash)) (fill (type none)))
-	(text "220 kW pk Discharge (HV, bolt-on) - 3 of 4   ·   rev A.18   ·   3 sections   ·   35 components" (exclude_from_sim no) (at 15.24 193.04 0) (effects (font (size 1.524 1.524) (bold yes)) (justify left bottom)))
+	(text "220 kW pk Discharge (HV, bolt-on) - 3 of 4   ·   rev A.19   ·   3 sections   ·   35 components" (exclude_from_sim no) (at 15.24 193.04 0) (effects (font (size 1.524 1.524) (bold yes)) (justify left bottom)))
 	(text "NET NAMING: U<ref>_<PIN> = node at that IC pin   ·   R<stem>_M = series-pair midpoint   ·   R<stem>_<nm> = tap between R<stem>n/m   ·   all others are explicit design nets   ·   same name on another sheet = same net, joined only at the named connector/stud/tab" (exclude_from_sim no) (at 15.24 200.66 0) (effects (font (size 1.27 1.27)) (justify left bottom)))
 	(text "DISCHARGE / ENTRY" (exclude_from_sim no) (at 192.024 112.014 0) (effects (font (size 2.0066 2.0066) (bold yes)) (justify left bottom)))

Commit message: Rev A.20: round 21 — three rechecks of 551c405 (F208): stale 0.29 Ω in gate ㉘ and the QP-RX-04 fixture instruction → 0.37 Ω, last 8.5 V-era figures aligned, Marine sweep cross-references at the current values
Co-Authored-By: Claude Fable 5.1 <noreply@anthropic.com>
Other:
- note added: "220 kW pk Discharge (HV, bolt-on) - 3 of 4 · rev A.20 · 3 sections · 35 components"
- note removed: "220 kW pk Discharge (HV, bolt-on) - 3 of 4 · rev A.19 · 3 sections · 35 components"
Changed lines of the file:
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@@
 		(title "Traction Inverter — Discharge board (bolt-on, XM3 pattern)")
 		(date "2026-09-23")
-		(rev "A.19")
+		(rev "A.20")
 		(company "Traction Inverter 220 kW pk - Discharge (HV, bolt-on), sheet 3 of 4")
 		(comment 1 "Inverter = Power board + Cap bank busbar + bolt-on Discharge board (all HV) + Control card (LV); safe state holds with any link lost")
@@
 	(rectangle (start 190.5 12.7) (end 269.24 95.25) (stroke (width 0) (type dash)) (fill (type none)))
 	(rectangle (start 12.7 12.7) (end 180.34 177.8) (stroke (width 0) (type dash)) (fill (type none)))
-	(text "220 kW pk Discharge (HV, bolt-on) - 3 of 4   ·   rev A.19   ·   3 sections   ·   35 components" (exclude_from_sim no) (at 15.24 193.04 0) (effects (font (size 1.524 1.524) (bold yes)) (justify left bottom)))
+	(text "220 kW pk Discharge (HV, bolt-on) - 3 of 4   ·   rev A.20   ·   3 sections   ·   35 components" (exclude_from_sim no) (at 15.24 193.04 0) (effects (font (size 1.524 1.524) (bold yes)) (justify left bottom)))
 	(text "NET NAMING: U<ref>_<PIN> = node at that IC pin   ·   R<stem>_M = series-pair midpoint   ·   R<stem>_<nm> = tap between R<stem>n/m   ·   all others are explicit design nets   ·   same name on another sheet = same net, joined only at the named connector/stud/tab" (exclude_from_sim no) (at 15.24 200.66 0) (effects (font (size 1.27 1.27)) (justify left bottom)))
 	(text "DISCHARGE / ENTRY" (exclude_from_sim no) (at 192.024 112.014 0) (effects (font (size 2.0066 2.0066) (bold yes)) (justify left bottom)))

Commit message: Rev A.21: round 22 — three rechecks of 0ff44d9 (F209) + the layout handoff (F210–F213): every KiCad symbol bound to a footprint in a shipped traction.pretty (45 verbatim KiCad-10 patterns + 18 datasheet-drawn), fp-lib-table and per-board projects in all sets, pad-per-pin KiCad proof; NCV4276C 5-lead lands, ALM2402/TPS55340 thermal-pad pins, 2-pad crystal; QP §0.2 baseline and stale IDs; docs/layout-handoff.md
Co-Authored-By: Claude Fable 5.1 <noreply@anthropic.com>
Parts:
- CQD, CQDF, CQDIB: footprint C0603 -> traction:C_0603_1608Metric
- CQDI1, CQDI2: footprint C1206 -> traction:C_1206_3216Metric
- CQDO: footprint C1210 -> traction:C_1210_3225Metric
- JCTL: footprint IPL1-104 (1x4 2.54 mm THT) -> traction:Samtec_IPL1-104_1x04
- JDCN, JDCP: footprint StudM6 -> traction:MountingHole_6.4mm_M6_Pad
- PSQD: footprint DWN36 -> traction:UCC14141-Q1_DWN36
- QDIS: footprint TO247-4L -> traction:TO-247-4_Vertical
- RBLD1, RBLD10, RBLD11, RBLD12, RBLD2, RBLD3, RBLD4, RBLD5, RBLD6, RBLD7, RBLD8, RBLD9: footprint R2512 -> traction:R_2512_6332Metric
- RDIS1, RDIS2, RDIS3, RDIS4: footprint AxialWW10W -> traction:Yageo_SQP10_P55.88
- RQDE1, RQDE2, RQDF1, RQDF2, RQDG, RQDL, RQDPD: footprint R0603 -> traction:R_0603_1608Metric
- UQD: footprint SMD8W -> traction:VOW3120_SMD8W
Other:
- note added: "220 kW pk Discharge (HV, bolt-on) - 3 of 4 · rev A.21 · 3 sections · 35 components"
- note removed: "220 kW pk Discharge (HV, bolt-on) - 3 of 4 · rev A.20 · 3 sections · 35 components"

Commit message: Rev A.22: round 23 — rechecks of 452de85 (F214–F220), the VESC program (FW-38…FW-46, Traction Tool in Qt) and the "why not done" extension (F221–F239)
Hardware: the R2R reference isolated at ball A9 (RR2R 10 Ω + 1 µF + 100 nF, S32K39 DS note 8), the SWD header on its
surface-mount Samtec land with a mounting-technology lock in the library generator, the footprint library declared
KiCad 10.0.6+ and no longer mirrored into the KiCad 5 sets; the BOM intro follows the SKU; a VREFH window row and VR-34/35.

Firmware (TI_FW_ID 0x0A0F0015, CAL layout 4, 190 fields / 91 CAL rows, 80 DTCs): FW-37 joint torque solve with a
postcondition; the VESC gap closure — FW-38 signed field update (Ed25519, anti-rollback, ISO-TP), FW-39 interlocked motor
self-commissioning, FW-40 UDS diagnostics (0x19/0x22/0x2A/0x14 over ISO 15765-2), FW-41 fault-triggered waveform capture,
FW-42 overspeed, FW-43 run-time statistics, FW-44 key-on offset adoption, FW-45 saturation-dependent inductance tables
with gain scheduling, FW-46 cogging feed-forward; twelve defects found by the closed-loop simulator bridge (F221–F232),
the 64-bit divide out of every ISR path with a link-time guard, the UDS escape single frame accepted by every service,
the root of trust reported (DID 0xFD23), the boot record, motor data and active maps as DIDs; 421 tests / 4937 checks /
0 failed on the host (-O1, -O2, ASan/UBSan, -ffp-contract=off) and on the Cortex-M7 under QEMU with the target compiler
(make qemu-test, T-59); make target-check 63 markers, make target-size with the divide guard.

Traction Tool (tool/): Qt 6 / C++17 Widgets + Qwt, offline; pages Dashboard, Live plots, Controls, Commissioning,
Parameters, Faults & alerts, Analysis, Terminal, Firmware; transports simulator bridge (tool/bridge, the real firmware
against a plant), log replay, CAN (QCanBus with ISO-TP both ways, proved against the firmware over the virtualcan bus);
the signed update end to end over both transports; the commissioning routines, the map sw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
Other:
- note added: "220 kW pk Discharge (HV, bolt-on) - 3 of 4 · rev A.22 · 3 sections · 35 components"
- note removed: "220 kW pk Discharge (HV, bolt-on) - 3 of 4 · rev A.21 · 3 sections · 35 components"
Changed lines of the file:
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@@
 		(title "Traction Inverter — Discharge board (bolt-on, XM3 pattern)")
 		(date "2026-09-23")
-		(rev "A.21")
+		(rev "A.22")
 		(company "Traction Inverter 220 kW pk - Discharge (HV, bolt-on), sheet 3 of 4")
 		(comment 1 "Inverter = Power board + Cap bank busbar + bolt-on Discharge board (all HV) + Control card (LV); safe state holds with any link lost")
@@
 	(rectangle (start 190.5 12.7) (end 269.24 95.25) (stroke (width 0) (type dash)) (fill (type none)))
 	(rectangle (start 12.7 12.7) (end 180.34 177.8) (stroke (width 0) (type dash)) (fill (type none)))
-	(text "220 kW pk Discharge (HV, bolt-on) - 3 of 4   ·   rev A.21   ·   3 sections   ·   35 components" (exclude_from_sim no) (at 15.24 193.04 0) (effects (font (size 1.524 1.524) (bold yes)) (justify left bottom)))
+	(text "220 kW pk Discharge (HV, bolt-on) - 3 of 4   ·   rev A.22   ·   3 sections   ·   35 components" (exclude_from_sim no) (at 15.24 193.04 0) (effects (font (size 1.524 1.524) (bold yes)) (justify left bottom)))
 	(text "NET NAMING: U<ref>_<PIN> = node at that IC pin   ·   R<stem>_M = series-pair midpoint   ·   R<stem>_<nm> = tap between R<stem>n/m   ·   all others are explicit design nets   ·   same name on another sheet = same net, joined only at the named connector/stud/tab" (exclude_from_sim no) (at 15.24 200.66 0) (effects (font (size 1.27 1.27)) (justify left bottom)))
 	(text "DISCHARGE / ENTRY" (exclude_from_sim no) (at 192.024 112.014 0) (effects (font (size 2.0066 2.0066) (bold yes)) (justify left bottom)))

Commit message: Rev A.23: round 24 — four rechecks of 4ed0101 (F240–F244): the SDADC reference on its supply node, acquisition freshness, the map's flux slope and the ripple limiter's exact bounds, the temperature latch, the V_DC expiry
Hardware (F240, no new part): the S32K39 data sheet's SDADC table (Rev. 3 Table 38, in our archive and our own
extracted-parameters file) requires VREFP within ±25 mV of AVDD; the round-23 disposition had judged the general +100 mV
note and called the figure absent while the references sat on the FS26 VREF, matched to the SDADC-supply LDO only within
±1 %. Every non-R2R reference group (E6/H6 SAR, E10/F13 SDADC) is now on V5A itself with VDDA_SDADC and VDD_HV_A (NXP's
GEN3 arrangement); the ratiometric loads (HW_ID and offset dividers, the seven NTC pull-ups) moved with the reference; the
R2R ladder keeps the FS26 VREF as its isolated supply through the 10 Ω branch (CR2R1 330 nF, 37 kHz); CSB5 2.2 µF holds
the FS26 window alone (1.36–2.92 µF effective); the absolute SAR scale re-budgeted at the LDO2's ±1.75 %; ERC locks, pin
freeze, manifest, handoff §4.11 island rule (≤ 20 mΩ from E12 to any VREFH ball), VR-34 closed by design, IR-26, QP-TH-06.
Pipeline at A.23: ERC 981/0/0, verify 158/18/0, sim 23/6/0, Marine 87/23/0, 21 pages / 2065 pins, KiCad proof PASS, PDFs
and BOMs regenerated (₹72,983 unchanged). The handoff §6 gives every open pre-layout decision a provisional default.

Firmware (TI_FW_ID 0x0A0F0016, CAL layout 4, 191 fields / 92 CAL rows, 82 DTCs): F241 a stopped slow ADC channel stayed
valid forever (the caller discarded the acquisition stamp) → a three-state contract new/held/expired for every slow-list
input with cal_temp_hold_ms and DTC_ADC_SLOW_STALE, every slow consumer audited (V5GD/VOFS, IGN, INTRLOK_N, VSUP, HW_ID);
F242 the inductance map must keep a positive flux slope (≥ 0.25 × L0 below every breakpoint) and the ripple limiter bounds
every piece of its interval in closed form (breakpoints alone shown insufficient by a 20 000-m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
Other:
- note added: "220 kW pk Discharge (HV, bolt-on) - 3 of 4 · rev A.23 · 3 sections · 35 components"
- note removed: "220 kW pk Discharge (HV, bolt-on) - 3 of 4 · rev A.22 · 3 sections · 35 components"
Changed lines of the file:
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@@
 		(title "Traction Inverter — Discharge board (bolt-on, XM3 pattern)")
 		(date "2026-09-23")
-		(rev "A.22")
+		(rev "A.23")
 		(company "Traction Inverter 220 kW pk - Discharge (HV, bolt-on), sheet 3 of 4")
 		(comment 1 "Inverter = Power board + Cap bank busbar + bolt-on Discharge board (all HV) + Control card (LV); safe state holds with any link lost")
@@
 	(rectangle (start 190.5 12.7) (end 269.24 95.25) (stroke (width 0) (type dash)) (fill (type none)))
 	(rectangle (start 12.7 12.7) (end 180.34 177.8) (stroke (width 0) (type dash)) (fill (type none)))
-	(text "220 kW pk Discharge (HV, bolt-on) - 3 of 4   ·   rev A.22   ·   3 sections   ·   35 components" (exclude_from_sim no) (at 15.24 193.04 0) (effects (font (size 1.524 1.524) (bold yes)) (justify left bottom)))
+	(text "220 kW pk Discharge (HV, bolt-on) - 3 of 4   ·   rev A.23   ·   3 sections   ·   35 components" (exclude_from_sim no) (at 15.24 193.04 0) (effects (font (size 1.524 1.524) (bold yes)) (justify left bottom)))
 	(text "NET NAMING: U<ref>_<PIN> = node at that IC pin   ·   R<stem>_M = series-pair midpoint   ·   R<stem>_<nm> = tap between R<stem>n/m   ·   all others are explicit design nets   ·   same name on another sheet = same net, joined only at the named connector/stud/tab" (exclude_from_sim no) (at 15.24 200.66 0) (effects (font (size 1.27 1.27)) (justify left bottom)))
 	(text "DISCHARGE / ENTRY" (exclude_from_sim no) (at 192.024 112.014 0) (effects (font (size 2.0066 2.0066) (bold yes)) (justify left bottom)))
