File: kicad/traction/traction-power.kicad_sch (KiCad schematic)
At the start: 324 parts, among them U5LB NCV4276CDT50RKG, U5LC NCV4276CDT50RKG

Commit message: Rev A.17: round 18 — three rechecks of 4425af9 (F190-F198): diversion diodes on the amplifier node (loop passes RSX), diode cell cathode = pin 1 on all 35 diodes, exciter TVS/PTC rows at worst corners + ECU-asleep sustained short (WARN rows, layout rule, QP-RX-04 2b gate), anti-surge RSX, NCV4276C reverse current = QP-RX-05 gate + VR-33, IR-16/IR-42, firmware FW-34..36 (sample freshness, cadence-locked resolver frames, latency sign) + three self-found instances
Co-Authored-By: Claude Fable 5.1 <noreply@anthropic.com>
Parts:
- DASCR, DB15, DFHA, DFHFS, DFHG, DFHSN, DFHVZ, DFLA, DFLFS, DFLG, DFLSN, DFLVZ, DRH, DRL, DTVH, DTVL, DTVSH, DUHR, DUHS1, DUHS2, DUHZ1, DUHZ2, DULR, DULS1, DULS2, DULZ1, DULZ2, DUTP, DVHR, DVHS1, DVHS2, DVHZ1, DVHZ2, DVLR, DVLS1, DVLS2, DVLZ1, DVLZ2, DVTP, DWHR, DWHS1, DWHS2, DWHZ1, DWHZ2, DWLR, DWLS1, DWLS2, DWLZ1, DWLZ2, DWTP, ZASC, ZFHG, ZFHSN, ZFLG, ZFLSN, ZUHV, ZULV, ZVHV, ZVLV, ZWHV, ZWLV: symbol traction:D -> traction:D_21
Connections:
- net ASCVO: now also DASCR.1; no longer DASCR.2
- net ASC_DRV: now also DASCR.2, ZASC.1; no longer DASCR.1, ZASC.2
- net B15SW: now also DB15.2; no longer DB15.1
- net DCN: now also ZASC.2; no longer ZASC.1
- net DGND: now also DFHVZ.2, DFLVZ.2, DTVH.2, DTVL.2, DTVSH.2; no longer DFHVZ.1, DFLVZ.1, DTVH.1, DTVL.1, DTVSH.1
- net DS1_UH: now also DUHS1.2; no longer DUHS1.1
- net DS1_UL: now also DULS1.2; no longer DULS1.1
- net DS1_VH: now also DVHS1.2; no longer DVHS1.1
- net DS1_VL: now also DVLS1.2; no longer DVLS1.1
- net DS1_WH: now also DWHS1.2; no longer DWHS1.1
- net DS1_WL: now also DWLS1.2; no longer DWLS1.1
- net DS2_UH: now also DUHS1.1, DUHS2.2; no longer DUHS1.2, DUHS2.1
- net DS2_UL: now also DULS1.1, DULS2.2; no longer DULS1.2, DULS2.1
- net DS2_VH: now also DVHS1.1, DVHS2.2; no longer DVHS1.2, DVHS2.1
- net DS2_VL: now also DVLS1.1, DVLS2.2; no longer DVLS1.2, DVLS2.1
- net DS2_WH: now also DWHS1.1, DWHS2.2; no longer DWHS1.2, DWHS2.1
- net DS2_WL: now also DWLS1.1, DWLS2.2; no longer DWLS1.2, DWLS2.1
- net DSH_U: now also DUHS2.1; no longer DUHS2.2
- net DSH_V: now also DVHS2.1; no longer DVHS2.2
- net DSH_W: now also DWHS2.1; no longer DWHS2.2
- net FAX_H: now also DFHA.2, DFHFS.2; no longer DFHA.1, DFHFS.1
- net FAX_L: now also DFLA.2, DFLFS.2; no longer DFLA.1, DFLFS.1
- net FCL_H: now also DFHSN.1, ZFHSN.1; no longer DFHSN.2, ZFHSN.2
- net FCL_L: now also DFLSN.1, ZFLSN.1; no longer DFLSN.2, ZFLSN.2
- net FCS_H: now also ZFHG.2; no longer ZFHG.1
- net FCS_L: now also ZFLG.2; no longer ZFLG.1
- net FDR_H: now also DFHG.1; no longer DFHG.2
- net FDR_L: now also DFLG.1; no longer DFLG.2
- net FFD_H: now also DFHFS.1; no longer DFHFS.2
- net FFD_L: now also DFLFS.1; no longer DFLFS.2
- net FGO_H: now also DFHG.2; no longer DFHG.1
- net FGO_L: now also DFLG.2; no longer DFLG.1
- net FG_H: now also ZFHG.1; no longer ZFHG.2
- net FG_L: now also ZFLG.1; no longer ZFLG.2
- net FHO: now also DRH.2; no longer DRH.1
- net FLO: now also DRL.2; no longer DRL.1
- net FSW_H: now also DFHSN.2; no longer DFHSN.1
- net FSW_L: now also DFLSN.2; no longer DFLSN.1
- net FVCC_H: now also DFHA.1, DFHVZ.1; no longer DFHA.2, DFHVZ.2
- net FVCC_L: now also DFLA.1, DFLVZ.1; no longer DFLA.2, DFLVZ.2
- net G_UH: now also DUHZ1.1; no longer DUHZ1.2
- net G_UL: now also DULZ1.1; no longer DULZ1.2
- net G_VH: now also DVHZ1.1; no longer DVHZ1.2
- net G_VL: now also DVLZ1.1; no longer DVLZ1.2
- net G_WH: now also DWHZ1.1; no longer DWHZ1.2
- net G_WL: now also DWLZ1.1; no longer DWLZ1.2
- net HVIL_B: now also DTVSH.1; no longer DTVSH.2
- net KS_UH: now also DUHZ2.1, ZUHV.1; no longer DUHZ2.2, ZUHV.2
- net KS_UL: now also DULZ2.1, ZULV.1; no longer DULZ2.2, ZULV.2
- net KS_VH: now also DVHZ2.1, ZVHV.1; no longer DVHZ2.2, ZVHV.2
- net KS_VL: now also DVLZ2.1, ZVLV.1; no longer DVLZ2.2, ZVLV.2
- net KS_WH: now also DWHZ2.1, ZWHV.1; no longer DWHZ2.2, ZWHV.2
- net KS_WL: now also DWLZ2.1, ZWLV.1; no longer DWLZ2.2, ZWLV.2
- net NRH: now also DRH.1, DTVH.1; no longer DRH.2, DTVH.2
- net NRL: now also DRL.1, DTVL.1; no longer DRL.2, DTVL.2
- net PHU: now also DULS2.1; no longer DULS2.2
- net PHV: now also DVLS2.1; no longer DVLS2.2
- net PHW: now also DWLS2.1; no longer DWLS2.2
- net TMOD_U: now also DUTP.2; no longer DUTP.1
- net TMOD_V: now also DVTP.2; no longer DVTP.1
- net TMOD_W: now also DWTP.2; no longer DWTP.1
- net V12H: now also ZFHSN.2; no longer ZFHSN.1
- net V12L: now also ZFLSN.2; no longer ZFLSN.1
- net V15B: now also DB15.1; no longer DB15.2
- net V5GD: now also DUTP.1, DVTP.1, DWTP.1; no longer DUTP.2, DVTP.2, DWTP.2
- net VCC_UH: now also DUHR.1; no longer DUHR.2
- net VCC_UL: now also DULR.1; no longer DULR.2
- net VCC_VH: now also DVHR.1; no longer DVHR.2
- net VCC_VL: now also DVLR.1; no longer DVLR.2
- net VCC_WH: now also DWHR.1; no longer DWHR.2
- net VCC_WL: now also DWLR.1; no longer DWLR.2
- net VEE_UH: now also ZUHV.2; no longer ZUHV.1
- net VEE_UL: now also ZULV.2; no longer ZULV.1
- net VEE_VH: now also ZVHV.2; no longer ZVHV.1
- net VEE_VL: now also ZVLV.2; no longer ZVLV.1
- net VEE_WH: now also ZWHV.2; no longer ZWHV.1
- net VEE_WL: now also ZWLV.2; no longer ZWLV.1
- net W_UH_A: now also DUHR.2; no longer DUHR.1
- net W_UL_A: now also DULR.2; no longer DULR.1
- net W_VH_A: now also DVHR.2; no longer DVHR.1
- net W_VL_A: now also DVLR.2; no longer DVLR.1
- net W_WH_A: now also DWHR.2; no longer DWHR.1
- net W_WL_A: now also DWLR.2; no longer DWLR.1
- net ZK_UH: now also DUHZ1.2, DUHZ2.2; no longer DUHZ1.1, DUHZ2.1
- net ZK_UL: now also DULZ1.2, DULZ2.2; no longer DULZ1.1, DULZ2.1
- net ZK_VH: now also DVHZ1.2, DVHZ2.2; no longer DVHZ1.1, DVHZ2.1
- net ZK_VL: now also DVLZ1.2, DVLZ2.2; no longer DVLZ1.1, DVLZ2.1
- net ZK_WH: now also DWHZ1.2, DWHZ2.2; no longer DWHZ1.1, DWHZ2.1
- net ZK_WL: now also DWLZ1.2, DWLZ2.2; no longer DWLZ1.1, DWLZ2.1
Other:
- note added: "rev A.17 - 24 sections - 324 components"
- note removed: "rev A.16 - 24 sections - 324 components"

Commit message: Rev A.18: round 19 — three rechecks of e315bf1 (F199-F204): PTC-current row at every permitted voltage (IR-16 0.08/0.14/0.37/0.26 Ω), ≥8 A TVS energy an explicit assumption + QP-RX-04 release criterion, window criterion fixed, exciter TVS → SMDJ7.0A-HRA (coupled island holds the 7.0 V class at a parked 12 V battery / the Marine rail), shared exciter-fault model run for the Marine port (QP-MA-11, kit-loom rule), FW-35 rewritten on an SWG-anchored time origin with clock-derived resync and bounded restart
Co-Authored-By: Claude Fable 5.1 <noreply@anthropic.com>
Other:
- note added: "rev A.18 - 24 sections - 324 components"
- note removed: "rev A.17 - 24 sections - 324 components"
Changed lines of the file:
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@@
 		(title "Traction Inverter 220 kW — Power board (3x EconoDUAL 3 SiC)")
 		(date "2026-09-23")
-		(rev "A.17")
+		(rev "A.18")
 		(company "Traction Inverter 220 kW pk - Power (HV), sheet 1 of 4")
 		(comment 1 "Inverter = Power board + Cap bank busbar + bolt-on Discharge board (all HV) + Control card (LV); safe state holds with any link lost")
@@
 	(text "CONTROL-IF   -   1 section" (exclude_from_sim no) (at 740.41 607.06 0) (effects (font (size 1.524 1.524)) (justify left bottom)))
 	(text "DC-LINK   -   1 section" (exclude_from_sim no) (at 740.41 614.68 0) (effects (font (size 1.524 1.524)) (justify left bottom)))
-	(text "rev A.17   -   24 sections   -   324 components" (exclude_from_sim no) (at 740.664 631.19 0) (effects (font (size 1.524 1.524)) (justify left bottom)))
+	(text "rev A.18   -   24 sections   -   324 components" (exclude_from_sim no) (at 740.664 631.19 0) (effects (font (size 1.524 1.524)) (justify left bottom)))
 	(text "NET NAMING" (exclude_from_sim no) (at 232.664 715.264 0) (effects (font (size 2.0066 2.0066) (bold yes)) (justify left bottom)))
 	(text "internal junctions are named for what they join" (exclude_from_sim no) (at 232.664 721.868 0) (effects (font (size 1.524 1.524)) (justify left bottom)))

Commit message: Rev A.19: round 20 — three rechecks of 00f6252 (F205-F207): TVS alternate to the 7.0 V class + lock, 4XX discharge alternate 470→220 Ω + lock, T-05/T-06 firmware ID, 8.5 V-era figures re-derived at the IR-16 allocations
Co-Authored-By: Claude Fable 5.1 <noreply@anthropic.com>
Other:
- note added: "rev A.19 - 24 sections - 324 components"
- note removed: "rev A.18 - 24 sections - 324 components"
Changed lines of the file:
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@@
 		(title "Traction Inverter 220 kW — Power board (3x EconoDUAL 3 SiC)")
 		(date "2026-09-23")
-		(rev "A.18")
+		(rev "A.19")
 		(company "Traction Inverter 220 kW pk - Power (HV), sheet 1 of 4")
 		(comment 1 "Inverter = Power board + Cap bank busbar + bolt-on Discharge board (all HV) + Control card (LV); safe state holds with any link lost")
@@
 	(text "CONTROL-IF   -   1 section" (exclude_from_sim no) (at 740.41 607.06 0) (effects (font (size 1.524 1.524)) (justify left bottom)))
 	(text "DC-LINK   -   1 section" (exclude_from_sim no) (at 740.41 614.68 0) (effects (font (size 1.524 1.524)) (justify left bottom)))
-	(text "rev A.18   -   24 sections   -   324 components" (exclude_from_sim no) (at 740.664 631.19 0) (effects (font (size 1.524 1.524)) (justify left bottom)))
+	(text "rev A.19   -   24 sections   -   324 components" (exclude_from_sim no) (at 740.664 631.19 0) (effects (font (size 1.524 1.524)) (justify left bottom)))
 	(text "NET NAMING" (exclude_from_sim no) (at 232.664 715.264 0) (effects (font (size 2.0066 2.0066) (bold yes)) (justify left bottom)))
 	(text "internal junctions are named for what they join" (exclude_from_sim no) (at 232.664 721.868 0) (effects (font (size 1.524 1.524)) (justify left bottom)))

Commit message: Rev A.20: round 21 — three rechecks of 551c405 (F208): stale 0.29 Ω in gate ㉘ and the QP-RX-04 fixture instruction → 0.37 Ω, last 8.5 V-era figures aligned, Marine sweep cross-references at the current values
Co-Authored-By: Claude Fable 5.1 <noreply@anthropic.com>
Other:
- note added: "rev A.20 - 24 sections - 324 components"
- note removed: "rev A.19 - 24 sections - 324 components"
Changed lines of the file:
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@@
 		(title "Traction Inverter 220 kW — Power board (3x EconoDUAL 3 SiC)")
 		(date "2026-09-23")
-		(rev "A.19")
+		(rev "A.20")
 		(company "Traction Inverter 220 kW pk - Power (HV), sheet 1 of 4")
 		(comment 1 "Inverter = Power board + Cap bank busbar + bolt-on Discharge board (all HV) + Control card (LV); safe state holds with any link lost")
@@
 	(text "CONTROL-IF   -   1 section" (exclude_from_sim no) (at 740.41 607.06 0) (effects (font (size 1.524 1.524)) (justify left bottom)))
 	(text "DC-LINK   -   1 section" (exclude_from_sim no) (at 740.41 614.68 0) (effects (font (size 1.524 1.524)) (justify left bottom)))
-	(text "rev A.19   -   24 sections   -   324 components" (exclude_from_sim no) (at 740.664 631.19 0) (effects (font (size 1.524 1.524)) (justify left bottom)))
+	(text "rev A.20   -   24 sections   -   324 components" (exclude_from_sim no) (at 740.664 631.19 0) (effects (font (size 1.524 1.524)) (justify left bottom)))
 	(text "NET NAMING" (exclude_from_sim no) (at 232.664 715.264 0) (effects (font (size 2.0066 2.0066) (bold yes)) (justify left bottom)))
 	(text "internal junctions are named for what they join" (exclude_from_sim no) (at 232.664 721.868 0) (effects (font (size 1.524 1.524)) (justify left bottom)))

Commit message: Rev A.21: round 22 — three rechecks of 0ff44d9 (F209) + the layout handoff (F210–F213): every KiCad symbol bound to a footprint in a shipped traction.pretty (45 verbatim KiCad-10 patterns + 18 datasheet-drawn), fp-lib-table and per-board projects in all sets, pad-per-pin KiCad proof; NCV4276C 5-lead lands, ALM2402/TPS55340 thermal-pad pins, 2-pad crystal; QP §0.2 baseline and stale IDs; docs/layout-handoff.md
Co-Authored-By: Claude Fable 5.1 <noreply@anthropic.com>
Parts:
- C5B1, C5C1, C5G2, C5LB2, C5LC2, CASCI1, CASCI2, CB15I, CFHSN, CFLSN, CLVH1, CLVH2, CLVL1, CLVL2, CUHB2, CUHE1, CUHV1, CULB2, CULE1, CULV1, CVHB2, CVHE1, CVHV1, CVLB2, CVLE1, CVLV1, CWHB2, CWHE1, CWHV1, CWLB2, CWLE1, CWLV1: footprint C1206 -> traction:C_1206_3216Metric
- C5B2, C5C2, CASC, CASCD, CASCF, CASCIB, CB15C, CB15CC, CB15S, CFHCF, CFHCO, CFHCT, CFHFS, CFHSI, CFHVR, CFLCF, CFLCO, CFLCT, CFLFS, CFLSI, CFLVR, CLDC, CUHB1, CUHBL, CUHIN, CULB1, CULBL, CULIN, CUTF, CVBDF, CVDDF, CVHB1, CVHBL, CVHIN, CVLB1, CVLBL, CVLIN, CVTF, CWHB1, CWHBL, CWHIN, CWLB1, CWLBL, CWLIN, CWTF: footprint C0603 -> traction:C_0603_1608Metric
- C5G1, C5LB1, C5LC1: footprint C0805 -> traction:C_0805_2012Metric
- CASCO, CB15O1, CB15O2, CFHA, CFLA, CLD15: footprint C1210 -> traction:C_1210_3225Metric
- CPET: footprint disc, 10 mm pitch (FilmBoxFP(10) land) -> traction:C_Disc_D12.5mm_W5.0mm_P10.00mm
- CUSN, CVSN, CWSN: footprint FilmP27.5 -> traction:C_Rect_L31.5mm_W17.0mm_P27.50mm_MKS4
- CY1, CY2: footprint DiscP10 -> traction:C_Disc_D16.0mm_W5.0mm_P10.00mm
- DASCR, DFHFS, DFLFS, DTVSH, DUTP, DVTP, DWTP: footprint SOD323 -> traction:D_SOD-323
- DB15, DFHA, DFHSN, DFLA, DFLSN, DUHR, DUHS1, DUHS2, DULR, DULS1, DULS2, DVHR, DVHS1, DVHS2, DVLR, DVLS1, DVLS2, DWHR, DWHS1, DWHS2, DWLR, DWLS1, DWLS2, ZFHSN, ZFLSN: footprint SMA -> traction:D_SMA
- DFHG, DFLG: footprint SOD123 -> traction:D_SOD-123F
- DFHVZ, DFLVZ, DUHZ1, DUHZ2, DULZ1, DULZ2, DVHZ1, DVHZ2, DVLZ1, DVLZ2, DWHZ1, DWHZ2, DWLZ1, DWLZ2, ZASC, ZFHG, ZFLG, ZUHV, ZULV, ZVHV, ZVLV, ZWHV, ZWLV: footprint SOD123 -> traction:D_SOD-123
- DRH, DRL: footprint SMA-flat -> traction:NRVBAF360T3G_SMA-FL
- DTVH, DTVL: footprint SMC -> traction:D_SMC
- DUHSB, DULSB, DVHSB, DVLSB, DWHSB, DWLSB, QFHE1, QFHE2, QFLE1, QFLE2: footprint SOT23 -> traction:SOT-23-3
- FH1, FL1: footprint PTC2920 -> traction:Fuse_2920_7451Metric
- JDIS: footprint IPL1-104 (1x4 2.54 mm THT) -> traction:Samtec_IPL1-104_1x04
- JHVIL: footprint IPL1-102 (1x2 2.54 mm THT) -> traction:Samtec_IPL1-102_1x02
- JHVN, JHVP, JMU, JMV, JMW: footprint StudM8 -> traction:MountingHole_8.4mm_M8_Pad
- JIC: footprint HDR2x20-2.54 -> traction:Samtec_IPL1-120_2x20
- JPE: footprint StudM6 -> traction:MountingHole_6.4mm_M6_Pad
- LB15: footprint XAL4040 -> traction:L_Coilcraft_XAL4040-XXX
- LFH1, LFL1: footprint FB1206 -> traction:L_1206_3216Metric
- MODU, MODV, MODW: footprint EconoDUAL3 -> traction:EconoDUAL3
- PS5B, PS5C, UUHG, UULG, UVHG, UVLG, UWHG, UWLG: footprint SOIC16W -> traction:SOIC-16W_7.5x10.3mm_P1.27mm
- PSASC: footprint DWN36 -> traction:UCC14141-Q1_DWN36
- QFH, QFL: footprint LFPAK56 -> traction:LFPAK56
- R5LB, R5LC, RUHOFF, RUHON, RULOFF, RULON, RVHOFF, RVHON, RVLOFF, RVLON, RWHOFF, RWHON, RWLOFF, RWLON: footprint R2512 -> traction:R_2512_6332Metric
- RASCE1, RASCE2, RASCF1, RASCF2, RASCG, RASCL, RASCPD, RB15C, RB15F1, RB15F2, RB15Q, RFHEN, RFHFB1, RFHFB2, RFHFS, RFHG, RFHGO, RFHGS, RFHRT, RFHSI, RFLEN, RFLFB1, RFLFB2, RFLFS, RFLG, RFLGO, RFLGS, RFLRT, RFLSI, RGDLE, RHVL1, RHVL2, RHWID, RLD1, RLD2, RPD0, RPD1, RPD10, RPD2, RPD3, RPD4, RPD5, RPD6, RPD7, RPD8, RPD9, RULAS, RUTS, RVBDL, RVDDL, RVLAS, RVTS, RWLAS, RWTS: footprint R0603 -> traction:R_0603_1608Metric
- RFHCS, RFLCS: footprint R1210 -> traction:R_1210_3225Metric
- RFHSN, RFLSN, RUHBL, RUHDS, RUHGS, RUHMC, RULBL, RULDS, RULGS, RULMC, RVHBL, RVHDS, RVHGS, RVHMC, RVLBL, RVLDS, RVLGS, RVLMC, RWHBL, RWHDS, RWHGS, RWHMC, RWLBL, RWLDS, RWLGS, RWLMC: footprint R0805 -> traction:R_0805_2012Metric
- RFHST, RFLST, RPET, RUHPD, RULPD, RVBD1, RVBD2, RVBD3, RVBD4, RVBD5, RVBD6, RVDD1, RVDD2, RVDD3, RVDD4, RVDD5, RVDD6, RVHPD, RVLPD, RWHPD, RWLPD: footprint R1206 -> traction:R_1206_3216Metric
- TFH1, TFH2, TFH3, TFL1, TFL2, TFL3: footprint XfmrEE12 -> traction:VGT12EEM-200S1A4
- U5LB, U5LC, UGDL: footprint DPAK -> traction:TO-252-5_TabPin3
- UASC: footprint SMD8W -> traction:VOW3120_SMD8W
- UB15: footprint WQFN16 -> traction:WQFN-16-1EP_3x3mm_P0.5mm_EP1.68x1.68mm
- UFH, UFL: footprint SOP8 -> traction:SOIC-8_3.9x4.9mm_P1.27mm
- UIVB, UIVDC: footprint SOIC8W -> traction:AMC1311B_DWV8
- ULDO15: footprint D2PAK5 -> traction:TO-263-5_TabPin3
Connections:
- net DGND: now also UB15.17 (PAD)
Other:
- note added: "rev A.21 - 24 sections - 324 components"
- note removed: "rev A.20 - 24 sections - 324 components"
- moved on the sheet: CB15C, CB15CC, CB15I, CB15O1, CB15O2, CB15S, CLD15, CLDC, DB15, LB15, RB15C, RB15F1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

Commit message: Rev A.22: round 23 — rechecks of 452de85 (F214–F220), the VESC program (FW-38…FW-46, Traction Tool in Qt) and the "why not done" extension (F221–F239)
Hardware: the R2R reference isolated at ball A9 (RR2R 10 Ω + 1 µF + 100 nF, S32K39 DS note 8), the SWD header on its
surface-mount Samtec land with a mounting-technology lock in the library generator, the footprint library declared
KiCad 10.0.6+ and no longer mirrored into the KiCad 5 sets; the BOM intro follows the SKU; a VREFH window row and VR-34/35.

Firmware (TI_FW_ID 0x0A0F0015, CAL layout 4, 190 fields / 91 CAL rows, 80 DTCs): FW-37 joint torque solve with a
postcondition; the VESC gap closure — FW-38 signed field update (Ed25519, anti-rollback, ISO-TP), FW-39 interlocked motor
self-commissioning, FW-40 UDS diagnostics (0x19/0x22/0x2A/0x14 over ISO 15765-2), FW-41 fault-triggered waveform capture,
FW-42 overspeed, FW-43 run-time statistics, FW-44 key-on offset adoption, FW-45 saturation-dependent inductance tables
with gain scheduling, FW-46 cogging feed-forward; twelve defects found by the closed-loop simulator bridge (F221–F232),
the 64-bit divide out of every ISR path with a link-time guard, the UDS escape single frame accepted by every service,
the root of trust reported (DID 0xFD23), the boot record, motor data and active maps as DIDs; 421 tests / 4937 checks /
0 failed on the host (-O1, -O2, ASan/UBSan, -ffp-contract=off) and on the Cortex-M7 under QEMU with the target compiler
(make qemu-test, T-59); make target-check 63 markers, make target-size with the divide guard.

Traction Tool (tool/): Qt 6 / C++17 Widgets + Qwt, offline; pages Dashboard, Live plots, Controls, Commissioning,
Parameters, Faults & alerts, Analysis, Terminal, Firmware; transports simulator bridge (tool/bridge, the real firmware
against a plant), log replay, CAN (QCanBus with ISO-TP both ways, proved against the firmware over the virtualcan bus);
the signed update end to end over both transports; the commissioning routines, the map sw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
Other:
- note added: "rev A.22 - 24 sections - 324 components"
- note removed: "rev A.21 - 24 sections - 324 components"
Changed lines of the file:
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@@
 		(title "Traction Inverter 220 kW — Power board (3x EconoDUAL 3 SiC)")
 		(date "2026-09-23")
-		(rev "A.21")
+		(rev "A.22")
 		(company "Traction Inverter 220 kW pk - Power (HV), sheet 1 of 4")
 		(comment 1 "Inverter = Power board + Cap bank busbar + bolt-on Discharge board (all HV) + Control card (LV); safe state holds with any link lost")
@@
 	(text "CONTROL-IF   -   1 section" (exclude_from_sim no) (at 740.41 607.06 0) (effects (font (size 1.524 1.524)) (justify left bottom)))
 	(text "DC-LINK   -   1 section" (exclude_from_sim no) (at 740.41 614.68 0) (effects (font (size 1.524 1.524)) (justify left bottom)))
-	(text "rev A.21   -   24 sections   -   324 components" (exclude_from_sim no) (at 740.664 631.19 0) (effects (font (size 1.524 1.524)) (justify left bottom)))
+	(text "rev A.22   -   24 sections   -   324 components" (exclude_from_sim no) (at 740.664 631.19 0) (effects (font (size 1.524 1.524)) (justify left bottom)))
 	(text "NET NAMING" (exclude_from_sim no) (at 232.664 715.264 0) (effects (font (size 2.0066 2.0066) (bold yes)) (justify left bottom)))
 	(text "internal junctions are named for what they join" (exclude_from_sim no) (at 232.664 721.868 0) (effects (font (size 1.524 1.524)) (justify left bottom)))

Commit message: Rev A.23: round 24 — four rechecks of 4ed0101 (F240–F244): the SDADC reference on its supply node, acquisition freshness, the map's flux slope and the ripple limiter's exact bounds, the temperature latch, the V_DC expiry
Hardware (F240, no new part): the S32K39 data sheet's SDADC table (Rev. 3 Table 38, in our archive and our own
extracted-parameters file) requires VREFP within ±25 mV of AVDD; the round-23 disposition had judged the general +100 mV
note and called the figure absent while the references sat on the FS26 VREF, matched to the SDADC-supply LDO only within
±1 %. Every non-R2R reference group (E6/H6 SAR, E10/F13 SDADC) is now on V5A itself with VDDA_SDADC and VDD_HV_A (NXP's
GEN3 arrangement); the ratiometric loads (HW_ID and offset dividers, the seven NTC pull-ups) moved with the reference; the
R2R ladder keeps the FS26 VREF as its isolated supply through the 10 Ω branch (CR2R1 330 nF, 37 kHz); CSB5 2.2 µF holds
the FS26 window alone (1.36–2.92 µF effective); the absolute SAR scale re-budgeted at the LDO2's ±1.75 %; ERC locks, pin
freeze, manifest, handoff §4.11 island rule (≤ 20 mΩ from E12 to any VREFH ball), VR-34 closed by design, IR-26, QP-TH-06.
Pipeline at A.23: ERC 981/0/0, verify 158/18/0, sim 23/6/0, Marine 87/23/0, 21 pages / 2065 pins, KiCad proof PASS, PDFs
and BOMs regenerated (₹72,983 unchanged). The handoff §6 gives every open pre-layout decision a provisional default.

Firmware (TI_FW_ID 0x0A0F0016, CAL layout 4, 191 fields / 92 CAL rows, 82 DTCs): F241 a stopped slow ADC channel stayed
valid forever (the caller discarded the acquisition stamp) → a three-state contract new/held/expired for every slow-list
input with cal_temp_hold_ms and DTC_ADC_SLOW_STALE, every slow consumer audited (V5GD/VOFS, IGN, INTRLOK_N, VSUP, HW_ID);
F242 the inductance map must keep a positive flux slope (≥ 0.25 × L0 below every breakpoint) and the ripple limiter bounds
every piece of its interval in closed form (breakpoints alone shown insufficient by a 20 000-m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
Other:
- note added: "rev A.23 - 24 sections - 324 components"
- note removed: "rev A.22 - 24 sections - 324 components"
Changed lines of the file:
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@@
 		(title "Traction Inverter 220 kW — Power board (3x EconoDUAL 3 SiC)")
 		(date "2026-09-23")
-		(rev "A.22")
+		(rev "A.23")
 		(company "Traction Inverter 220 kW pk - Power (HV), sheet 1 of 4")
 		(comment 1 "Inverter = Power board + Cap bank busbar + bolt-on Discharge board (all HV) + Control card (LV); safe state holds with any link lost")
@@
 	(text "CONTROL-IF   -   1 section" (exclude_from_sim no) (at 740.41 607.06 0) (effects (font (size 1.524 1.524)) (justify left bottom)))
 	(text "DC-LINK   -   1 section" (exclude_from_sim no) (at 740.41 614.68 0) (effects (font (size 1.524 1.524)) (justify left bottom)))
-	(text "rev A.22   -   24 sections   -   324 components" (exclude_from_sim no) (at 740.664 631.19 0) (effects (font (size 1.524 1.524)) (justify left bottom)))
+	(text "rev A.23   -   24 sections   -   324 components" (exclude_from_sim no) (at 740.664 631.19 0) (effects (font (size 1.524 1.524)) (justify left bottom)))
 	(text "NET NAMING" (exclude_from_sim no) (at 232.664 715.264 0) (effects (font (size 2.0066 2.0066) (bold yes)) (justify left bottom)))
 	(text "internal junctions are named for what they join" (exclude_from_sim no) (at 232.664 721.868 0) (effects (font (size 1.524 1.524)) (justify left bottom)))
