File: kicad5/traction-native/traction-card.sch (KiCad schematic (older format))
At the start: 301 parts, among them Y1 CX3225GA40000D0PTVCC

Commit message: Rev A.22: round 23 — rechecks of 452de85 (F214–F220), the VESC program (FW-38…FW-46, Traction Tool in Qt) and the "why not done" extension (F221–F239)
Hardware: the R2R reference isolated at ball A9 (RR2R 10 Ω + 1 µF + 100 nF, S32K39 DS note 8), the SWD header on its
surface-mount Samtec land with a mounting-technology lock in the library generator, the footprint library declared
KiCad 10.0.6+ and no longer mirrored into the KiCad 5 sets; the BOM intro follows the SKU; a VREFH window row and VR-34/35.

Firmware (TI_FW_ID 0x0A0F0015, CAL layout 4, 190 fields / 91 CAL rows, 80 DTCs): FW-37 joint torque solve with a
postcondition; the VESC gap closure — FW-38 signed field update (Ed25519, anti-rollback, ISO-TP), FW-39 interlocked motor
self-commissioning, FW-40 UDS diagnostics (0x19/0x22/0x2A/0x14 over ISO 15765-2), FW-41 fault-triggered waveform capture,
FW-42 overspeed, FW-43 run-time statistics, FW-44 key-on offset adoption, FW-45 saturation-dependent inductance tables
with gain scheduling, FW-46 cogging feed-forward; twelve defects found by the closed-loop simulator bridge (F221–F232),
the 64-bit divide out of every ISR path with a link-time guard, the UDS escape single frame accepted by every service,
the root of trust reported (DID 0xFD23), the boot record, motor data and active maps as DIDs; 421 tests / 4937 checks /
0 failed on the host (-O1, -O2, ASan/UBSan, -ffp-contract=off) and on the Cortex-M7 under QEMU with the target compiler
(make qemu-test, T-59); make target-check 63 markers, make target-size with the divide guard.

Traction Tool (tool/): Qt 6 / C++17 Widgets + Qwt, offline; pages Dashboard, Live plots, Controls, Commissioning,
Parameters, Faults & alerts, Analysis, Terminal, Firmware; transports simulator bridge (tool/bridge, the real firmware
against a plant), log replay, CAN (QCanBus with ISO-TP both ways, proved against the firmware over the virtualcan bus);
the signed update end to end over both transports; the commissioning routines, the map sw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
Parts:
- added RCPD2, RCPD3, RHWP: 10k, traction:R_0603_1608Metric, symbol traction-r1:R
- CAND1: renamed from CFLTD; value 3.3nF -> 100nF; MPN MLCC-3.3nF-50V-C0G -> MLCC-CLASS
- CAND2: renamed from CFLTF; value 100pF -> 100nF; MPN MLCC-100pF-16V -> MLCC-CLASS
- CASCG: renamed from RARB; value 10k -> 100nF; footprint traction:R_0603_1608Metric -> traction:C_0603_1608Metric; symbol traction-r1:R -> traction-r1:C; MPN R0603-10k -> MLCC-100nF-16V
- CBAL: renamed from CSB1; value 22uF -> 1nF; footprint traction:C_0805_2012Metric -> traction:C_0603_1608Metric; MPN MLCC-22uF-16V-X7R-0805 -> MLCC-1nF-50V-C0G
- CBTC: renamed from CSB2; value 22uF -> 47nF; footprint traction:C_0805_2012Metric -> traction:C_0603_1608Metric; MPN MLCC-22uF-16V-X7R-0805 -> MLCC-47nF-50V-X7R-0603
- CBTP: renamed from CSB3; value 22uF -> 22nF; footprint traction:C_0805_2012Metric -> traction:C_0603_1608Metric; MPN MLCC-22uF-10V-X7R-0805 -> MLCC-22nF-50V-X7R-0603
- CCAN1: renamed from RCT1B; value 60.4R -> 1uF; footprint traction:R_0603_1608Metric -> traction:C_0603_1608Metric; symbol traction-r1:R -> traction-r1:C; MPN R0603-60R4-1% -> MLCC-1uF-25V
- CCAN2: renamed from RCT2B; value 60.4R -> 1uF; footprint traction:R_0603_1608Metric -> traction:C_0603_1608Metric; symbol traction-r1:R -> traction-r1:C; MPN R0603-60R4-1% -> MLCC-1uF-25V
- CCLR: renamed from CFLTF2; value 100pF -> 15nF; MPN MLCC-100pF-16V -> MLCC-15nF-50V-C0G
- CCOSA1: renamed from CCOSD; value 47pF -> 22pF; MPN MLCC-47pF-50V-C0G-0603 -> MLCC-22pF-50V-C0G-0603
- CCOSA2: renamed from CCOSF1; value 22pF -> 220pF; MPN MLCC-22pF-50V-C0G-0603 -> MLCC-220pF-50V-C0G-0603
- CCOSD: renamed from RCOS1; value 12k -> 47pF; footprint traction:R_0603_1608Metric -> traction:C_0603_1608Metric; symbol traction-r1:R -> traction-r1:C; MPN R0603-CLASS -> MLCC-47pF-50V-C0G-0603
- CCOSF1: renamed from RCOS2; value 12k -> 22pF; footprint traction:R_0603_1608Metric -> traction:C_0603_1608Metric; symbol traction-r1:R -> traction-r1:C; MPN R0603-CLASS -> MLCC-22pF-50V-C0G-0603
- CCOSF2: renamed from RCOSF1; value 12k -> 22pF; footprint traction:R_0603_1608Metric -> traction:C_0603_1608Metric; symbol traction-r1:R -> traction-r1:C; MPN R0603-CLASS -> MLCC-22pF-50V-C0G-0603
- CCT1: renamed from LCAN2; value ACT45B-101-2P-TL003 -> 4.7nF; footprint traction:TDK_ACT45B -> traction:C_0603_1608Metric; symbol traction-r1:ACT45B-101-2P-TL003 -> traction-r1:C; MPN ACT45B-101-2P-TL003 -> MLCC-4.7nF-50V
- CCT2: renamed from JVEH; value TE 770669-1 (AMPSEAL 23) -> 4.7nF; footprint traction:TE_770669-1 -> traction:C_0603_1608Metric; symbol traction-r1:TE_770669-1__AMPSEAL_23_ -> traction-r1:C; MPN TE 770669-1 (AMPSEAL 23) -> MLCC-4.7nF-50V
- CEXA1: renamed from CEXA4; value 47pF -> 220pF; MPN MLCC-47pF-50V-C0G-0603 -> MLCC-220pF-50V-C0G-0603
- CEXA2: renamed from CEXD; value 4.7uF -> 1.5nF; footprint traction:C_1206_3216Metric -> traction:C_0603_1608Metric; MPN MLCC-4.7uF-25V-X7R -> MLCC-1.5nF-50V-C0G-0603
- CEXA3: renamed from CEXM; value 220pF -> 100nF; MPN MLCC-220pF-50V-C0G -> MLCC-100nF-50V-X7R-0603
- CEXA4: renamed from CLDE; value 22uF -> 47pF; footprint traction:C_1210_3225Metric -> traction:C_0603_1608Metric; MPN MLCC-22uF-25V-X7R-1210 -> MLCC-47pF-50V-C0G-0603
- CEXD: renamed from CLDEC; value 270pF -> 4.7uF; footprint traction:C_0603_1608Metric -> traction:C_1206_3216Metric; MPN MLCC-270pF-50V-C0G-0603 -> MLCC-4.7uF-25V-X7R
- CEXM: renamed from DEXN; value PMEG4050EP-Q -> 220pF; footprint traction:D_SOD-128 -> traction:C_0603_1608Metric; symbol traction-r1:D_21 -> traction-r1:C; MPN PMEG4050EP-Q -> MLCC-220pF-50V-C0G
- CFLTD: renamed from CLAT2; value 100nF -> 3.3nF; MPN MLCC-100nF-16V -> MLCC-3.3nF-50V-C0G
- CFLTF: renamed from CSCH; value 100nF -> 100pF; MPN MLCC-100nF-16V -> MLCC-100pF-16V
- CFLTF2: renamed from CSCH2; value 100nF -> 100pF; MPN MLCC-100nF-16V -> MLCC-100pF-16V
- CIGN: renamed from RIGN1; value 5.1k -> 100nF; footprint traction:R_0603_1608Metric -> traction:C_0603_1608Metric; symbol traction-r1:R -> traction-r1:C; MPN R0603-5k1 -> MLCC-100nF-50V
- CIGNS: renamed from RIGN2; value 10k -> 100nF; footprint traction:R_0603_1608Metric -> traction:C_0603_1608Metric; symbol traction-r1:R -> traction-r1:C; MPN R0603-10k -> MLCC-CLASS
- CILK: renamed from RILK3; value 10k -> 2.2nF; footprint traction:R_0603_1608Metric -> traction:C_0603_1608Metric; symbol traction-r1:R -> traction-r1:C; MPN R0603-10k -> MLCC-2.2nF-50V
- CLAT: renamed from RASCP; value 10k -> 100nF; footprint traction:R_0603_1608Metric -> traction:C_0603_1608Metric; symbol traction-r1:R -> traction-r1:C; MPN R0603-10k -> MLCC-100nF-16V
- CLDE: renamed from DEXP; value PMEG4050EP-Q -> 22uF; footprint traction:D_SOD-128 -> traction:C_1210_3225Metric; symbol traction-r1:D_21 -> traction-r1:C; MPN PMEG4050EP-Q -> MLCC-22uF-25V-X7R-1210
- CLDEC: renamed from FEXN; value MF-MSMF020/33X -> 270pF; footprint traction:Fuse_1812_4532Metric -> traction:C_0603_1608Metric; symbol traction-r1:F -> traction-r1:C; MPN MF-MSMF020/33X -> MLCC-270pF-50V-C0G-0603
- CLVC1: renamed from CLVSM; value 100nF -> 4.7uF; footprint traction:C_0603_1608Metric -> traction:C_1206_3216Metric; MPN MLCC-100nF-50V -> MLCC-4.7uF-50V
- CLVC2: renamed from DREVC; value STPS5L60S -> 22uF; footprint traction:D_SMC -> traction:C_1210_3225Metric; symbol traction-r1:D_21 -> traction-r1:C; LCSC C140620 -> CLASS; MPN STPS5L60S -> MLCC-22uF-50V
- CLVC3: renamed from DTVSC; value TPSMC33A-VR -> 100uF; footprint traction:D_SMC -> traction:CP_Elec_10x10.5; symbol traction-r1:D_21 -> traction-r1:CP; MPN TPSMC33A-VR -> EEH-ZC1H101P
- CLVSM: renamed from DTVSC2; value TPSMC18A-VR -> 100nF; footprint traction:D_SMC -> traction:C_0603_1608Metric; symbol traction-r1:D_21 -> traction-r1:C; MPN TPSMC18A-VR -> MLCC-100nF-50V
- CMT1F: renamed from FMT2; value 0438.375WRA -> 47nF; footprint traction:Fuse_0603_1608Metric -> traction:C_0603_1608Metric; symbol traction-r1:F -> traction-r1:C; MPN 0438.375WRA -> MLCC-47nF-25V
- CMT2F: renamed from RMT1P; value 10k -> 47nF; footprint traction:R_0603_1608Metric -> traction:C_0603_1608Metric; symbol traction-r1:R -> traction-r1:C; MPN R0603-CLASS -> MLCC-47nF-25V
- COF1: renamed from ROF2; value 1k -> 100nF; footprint traction:R_0603_1608Metric -> traction:C_0603_1608Metric; symbol traction-r1:R -> traction-r1:C; MPN R0603-CLASS -> MLCC-CLASS
- COR1: renamed from RILK1; value 10k -> 100nF; footprint traction:R_0603_1608Metric -> traction:C_0603_1608Metric; symbol traction-r1:R -> traction-r1:C; MPN R0603-10k -> MLCC-CLASS
- COR2: renamed from RILK2; value 10k -> 100nF; footprint traction:R_0603_1608Metric -> traction:C_0603_1608Metric; symbol traction-r1:R -> traction-r1:C; MPN R0603-10k -> MLCC-CLASS
- CR2R1: renamed from CV25; value 220nF -> 1uF; MPN MLCC-220nF-10V-X7R -> MLCC-1uF-10V-X7R-0603
- CR2R2: renamed from CYA; value 12pF -> 100nF; MPN MLCC-12pF-50V -> MLCC-100nF-50V-X7R-0603
- CRST: renamed from QLVS; value DMP6023LEQ-13 -> 100pF; footprint traction:SOT-223 -> traction:C_0603_1608Metric; symbol traction-r1:DMP6023LEQ-13 -> traction-r1:C; MPN DMP6023LEQ-13 -> MLCC-100pF-16V
- CSB1: renamed from CSB3B; MPN MLCC-22uF-10V-X7R-0805 -> MLCC-22uF-16V-X7R-0805
- CSB2: renamed from CSB4; value 10uF -> 22uF; MPN MLCC-10uF-10V-X7R-0805 -> MLCC-22uF-16V-X7R-0805
- CSB3: renamed from CSB5; value 1uF -> 22uF; MPN MLCC-1uF-16V-X7R-0805 -> MLCC-22uF-10V-X7R-0805
- CSB3B: renamed from CSB6; value 4.7uF -> 22uF; MPN MLCC-4.7uF-10V-X7R-0805 -> MLCC-22uF-10V-X7R-0805
- CSB4: renamed from CSB7; MPN MLCC-10uF-16V-X7R-0805 -> MLCC-10uF-10V-X7R-0805
- CSB5: renamed from CSB8; value 10uF -> 1uF; MPN MLCC-10uF-16V-X7R-0805 -> MLCC-1uF-16V-X7R-0805
- CSB6: renamed from CVBOS; MPN MLCC-4.7uF-25V-X7R-0805 -> MLCC-4.7uF-10V-X7R-0805
- CSB7: renamed from CVDIG; value 1uF -> 10uF; footprint traction:C_0603_1608Metric -> traction:C_0805_2012Metric; MPN MLCC-1uF-10V-X7R-0603 -> MLCC-10uF-16V-X7R-0805
- CSB8: renamed from DBAT; value BAT46ZFILM -> 10uF; footprint traction:D_SOD-123 -> traction:C_0805_2012Metric; symbol traction-r1:D_21 -> traction-r1:C; LCSC C283255 -> CLASS; MPN BAT46ZFILM -> MLCC-10uF-16V-X7R-0805
- CSCH: renamed from DCLR; value BAT46ZFILM -> 100nF; footprint traction:D_SOD-123 -> traction:C_0603_1608Metric; symbol traction-r1:D_21 -> traction-r1:C; LCSC C283255 -> CLASS; MPN BAT46ZFILM -> MLCC-100nF-16V
- CSCH2: renamed from DFLT1; value BAT46ZFILM -> 100nF; footprint traction:D_SOD-123 -> traction:C_0603_1608Metric; symbol traction-r1:D_21 -> traction-r1:C; LCSC C283255 -> CLASS; MPN BAT46ZFILM -> MLCC-100nF-16V
- CSCH3: renamed from DFLT2; value BAT46ZFILM -> 100nF; footprint traction:D_SOD-123 -> traction:C_0603_1608Metric; symbol traction-r1:D_21 -> traction-r1:C; LCSC C283255 -> CLASS; MPN BAT46ZFILM -> MLCC-100nF-16V
- CSINA1: renamed from CSIND; value 47pF -> 22pF; MPN MLCC-47pF-50V-C0G-0603 -> MLCC-22pF-50V-C0G-0603
- CSINA2: renamed from CSINF1; value 22pF -> 220pF; MPN MLCC-22pF-50V-C0G-0603 -> MLCC-220pF-50V-C0G-0603
- CSIND: renamed from RSIN1; value 12k -> 47pF; footprint traction:R_0603_1608Metric -> traction:C_0603_1608Metric; symbol traction-r1:R -> traction-r1:C; MPN R0603-CLASS -> MLCC-47pF-50V-C0G-0603
- CSINF1: renamed from RSIN2; value 12k -> 22pF; footprint traction:R_0603_1608Metric -> traction:C_0603_1608Metric; symbol traction-r1:R -> traction-r1:C; MPN R0603-CLASS -> MLCC-22pF-50V-C0G-0603
- CSINF2: renamed from RSINF1; value 12k -> 22pF; footprint traction:R_0603_1608Metric -> traction:C_0603_1608Metric; symbol traction-r1:R -> traction-r1:C; MPN R0603-CLASS -> MLCC-22pF-50V-C0G-0603
- CSNUF: renamed from RSNUP; value 5.1k -> 47nF; footprint traction:R_0603_1608Metric -> traction:C_0603_1608Metric; symbol traction-r1:R -> traction-r1:C; MPN R0603-5k1-1% -> MLCC-47nF-25V
- CSNVF: renamed from RSNVP; value 5.1k -> 47nF; footprint traction:R_0603_1608Metric -> traction:C_0603_1608Metric; symbol traction-r1:R -> traction-r1:C; MPN R0603-5k1-1% -> MLCC-47nF-25V
- CSNWF: renamed from RSNWP; value 5.1k -> 47nF; footprint traction:R_0603_1608Metric -> traction:C_0603_1608Metric; symbol traction-r1:R -> traction-r1:C; MPN R0603-5k1-1% -> MLCC-47nF-25V
- CTAMBF: renamed from RTAMBP; value 10k -> 47nF; footprint traction:R_0603_1608Metric -> traction:C_0603_1608Metric; symbol traction-r1:R -> traction-r1:C; MPN R0603-10k-1% -> MLCC-47nF-25V
- CTHSF: renamed from RTHS; value 10k -> 47nF; footprint traction:R_0603_1608Metric -> traction:C_0603_1608Metric; symbol traction-r1:R -> traction-r1:C; MPN NTC-10k-0603 -> MLCC-47nF-25V
- CUB1: renamed from CUS2; value 4.7nF -> 3.3nF; MPN MLCC-4.7nF-50V -> MLCC-3.3nF-50V
- CUB2: renamed from LUB; value BLM21PG221SH1D -> 100nF; footprint traction:L_0805_2012Metric -> traction:C_0603_1608Metric; symbol traction-r1:L -> traction-r1:C; MPN BLM21PG221SH1D -> MLCC-100nF-25V
- CUS1: renamed from RUB0; value 100k -> 47nF; footprint traction:R_0603_1608Metric -> traction:C_0603_1608Metric; symbol traction-r1:R -> traction-r1:C; MPN R0603-100k -> MLCC-47nF-25V
- CUS2: renamed from RUB1; value 100R -> 4.7nF; footprint traction:R_0603_1608Metric -> traction:C_0603_1608Metric; symbol traction-r1:R -> traction-r1:C; MPN R0603-100R -> MLCC-4.7nF-50V
- CV25: renamed from CYB; value 12pF -> 220nF; MPN MLCC-12pF-50V -> MLCC-220nF-10V-X7R
- CVB1: renamed from CVS2; value 4.7nF -> 3.3nF; MPN MLCC-4.7nF-50V -> MLCC-3.3nF-50V
- CVB2: renamed from LVB; value BLM21PG221SH1D -> 100nF; footprint traction:L_0805_2012Metric -> traction:C_0603_1608Metric; symbol traction-r1:L -> traction-r1:C; MPN BLM21PG221SH1D -> MLCC-100nF-25V
- CVBOS: renamed from LCOR; value XAL4020-222MEC -> 4.7uF; footprint traction:L_Coilcraft_XAL4020-XXX -> traction:C_0805_2012Metric; symbol traction-r1:L -> traction-r1:C; MPN XAL4020-222MEC -> MLCC-4.7uF-25V-X7R-0805
- CVD1: renamed from RVD1A; value 10k -> 100pF; footprint traction:R_0603_1608Metric -> traction:C_0603_1608Metric; symbol traction-r1:R -> traction-r1:C; MPN R0603-10k-0.1% -> MLCC-100pF-50V-C0G-0603
- CVD2: renamed from RVD2C; value 10k -> 100pF; footprint traction:R_0603_1608Metric -> traction:C_0603_1608Metric; symbol traction-r1:R -> traction-r1:C; MPN R0603-10k-0.1% -> MLCC-100pF-50V-C0G-0603
- CVDIG: renamed from LSBC; value XAL4040-103MEC -> 1uF; footprint traction:L_Coilcraft_XAL4040-XXX -> traction:C_0603_1608Metric; symbol traction-r1:L -> traction-r1:C; MPN XAL4040-103MEC -> MLCC-1uF-10V-X7R-0603
- CVM1: renamed from RVM2; value 24k -> 220nF; footprint traction:R_0603_1608Metric -> traction:C_0603_1608Metric; symbol traction-r1:R -> traction-r1:C; MPN R0603-24k-1% -> MLCC-220nF-16V-X7R-0603
- CVM2: renamed from RVM3; value 24k -> 220nF; footprint traction:R_0603_1608Metric -> traction:C_0603_1608Metric; symbol traction-r1:R -> traction-r1:C; MPN R0603-24k-1% -> MLCC-220nF-16V-X7R-0603
- CVS1: renamed from RVB0; value 100k -> 47nF; footprint traction:R_0603_1608Metric -> traction:C_0603_1608Metric; symbol traction-r1:R -> traction-r1:C; MPN R0603-100k -> MLCC-47nF-25V
- CVS2: renamed from RVB1; value 100R -> 4.7nF; footprint traction:R_0603_1608Metric -> traction:C_0603_1608Metric; symbol traction-r1:R -> traction-r1:C; MPN R0603-100R -> MLCC-4.7nF-50V
- CWB1: renamed from CWS2; value 4.7nF -> 3.3nF; MPN MLCC-4.7nF-50V -> MLCC-3.3nF-50V
- CWB2: renamed from LWB; value BLM21PG221SH1D -> 100nF; footprint traction:L_0805_2012Metric -> traction:C_0603_1608Metric; symbol traction-r1:L -> traction-r1:C; MPN BLM21PG221SH1D -> MLCC-100nF-25V
- CWS1: renamed from RWB0; value 100k -> 47nF; footprint traction:R_0603_1608Metric -> traction:C_0603_1608Metric; symbol traction-r1:R -> traction-r1:C; MPN R0603-100k -> MLCC-47nF-25V
- CWS2: renamed from RWB1; value 100R -> 4.7nF; footprint traction:R_0603_1608Metric -> traction:C_0603_1608Metric; symbol traction-r1:R -> traction-r1:C; MPN R0603-100R -> MLCC-4.7nF-50V
- CYA: renamed from RMRST; value 10k -> 12pF; footprint traction:R_0603_1608Metric -> traction:C_0603_1608Metric; symbol traction-r1:R -> traction-r1:C; MPN R0603-10k -> MLCC-12pF-50V
- CYB: renamed from Y1; value CX3225GA40000D0PTVCC -> 12pF; footprint traction:Kyocera_CX3225GA_2Pad -> traction:C_0603_1608Metric; symbol traction-r1:Y -> traction-r1:C; LCSC C6009848 -> CLASS; MPN CX3225GA40000D0PTVCC -> MLCC-12pF-50V
- DBAT: renamed from RAGT; value 0R -> BAT46ZFILM; footprint traction:R_0805_2012Metric -> traction:D_SOD-123; symbol traction-r1:R -> traction-r1:D_21; LCSC CLASS -> C283255; MPN R0805-0R-CLASS -> BAT46ZFILM
- DCLR: renamed from RDRB; value 10k -> BAT46ZFILM; footprint traction:R_0603_1608Metric -> traction:D_SOD-123; symbol traction-r1:R -> traction-r1:D_21; LCSC CLASS -> C283255; MPN R0603-10k -> BAT46ZFILM
- DCOSP: renamed from CCOSA3; value 22pF -> PESD2IVN24-T; footprint traction:C_0603_1608Metric -> traction:SOT-23-3; symbol traction-r1:C -> traction-r1:PESD2IVN24-T; LCSC CLASS -> C406047; MPN MLCC-22pF-50V-C0G-0603 -> PESD2IVN24-T
- DEXN: renamed from FEXP; value MF-MSMF020/33X -> PMEG4050EP-Q; footprint traction:Fuse_1812_4532Metric -> traction:D_SOD-128; symbol traction-r1:F -> traction-r1:D_21; MPN MF-MSMF020/33X -> PMEG4050EP-Q
- DEXP: renamed from REXA1; value 3k -> PMEG4050EP-Q; footprint traction:R_0603_1608Metric -> traction:D_SOD-128; symbol traction-r1:R -> traction-r1:D_21; MPN R0603-CLASS -> PMEG4050EP-Q
- DFLT1: renamed from RENP1; value 5.1k -> BAT46ZFILM; footprint traction:R_0603_1608Metric -> traction:D_SOD-123; symbol traction-r1:R -> traction-r1:D_21; LCSC CLASS -> C283255; MPN R0603-5k1 -> BAT46ZFILM
- DFLT2: renamed from RFCB; value 100k -> BAT46ZFILM; footprint traction:R_0603_1608Metric -> traction:D_SOD-123; symbol traction-r1:R -> traction-r1:D_21; LCSC CLASS -> C283255; MPN R0603-100k -> BAT46ZFILM
- DFO: renamed from RFS1; value 1k -> BAT46ZFILM; footprint traction:R_0603_1608Metric -> traction:D_SOD-123; symbol traction-r1:R -> traction-r1:D_21; LCSC CLASS -> C283255; MPN R0603-1k -> BAT46ZFILM
- DIGN: renamed from RIGNS1; value 47k -> US1M; footprint traction:R_0603_1608Metric -> traction:D_SMA; symbol traction-r1:R -> traction-r1:D_21; LCSC CLASS -> C412437; MPN R0603-CLASS -> US1M
- DREVC: renamed from FLVC; value 0680L5000-05 -> STPS5L60S; footprint traction:Bel_0680L_2410 -> traction:D_SMC; symbol traction-r1:F -> traction-r1:D_21; LCSC CLASS -> C140620; MPN 0680L5000-05 -> STPS5L60S
- DSINP: renamed from CSINA3; value 22pF -> PESD2IVN24-T; footprint traction:C_0603_1608Metric -> traction:SOT-23-3; symbol traction-r1:C -> traction-r1:PESD2IVN24-T; LCSC CLASS -> C406047; MPN MLCC-22pF-50V-C0G-0603 -> PESD2IVN24-T
- DTVSC: renamed from FVBH; value MF-LSMF300/24X-2 -> TPSMC33A-VR; footprint traction:Fuse_2920_7451Metric -> traction:D_SMC; symbol traction-r1:F -> traction-r1:D_21; LCSC C719172 -> CLASS; MPN MF-LSMF300/24X-2 -> TPSMC33A-VR
- DTVSC2: renamed from FVBL; value MF-LSMF300/24X-2 -> TPSMC18A-VR; footprint traction:Fuse_2920_7451Metric -> traction:D_SMC; symbol traction-r1:F -> traction-r1:D_21; LCSC C719172 -> CLASS; MPN MF-LSMF300/24X-2 -> TPSMC18A-VR
- FEXN: renamed from REXA2; value 10k -> MF-MSMF020/33X; footprint traction:R_0603_1608Metric -> traction:Fuse_1812_4532Metric; symbol traction-r1:R -> traction-r1:F; MPN R0603-CLASS -> MF-MSMF020/33X
- FEXP: renamed from REXA3; value 10k -> MF-MSMF020/33X; footprint traction:R_0603_1608Metric -> traction:Fuse_1812_4532Metric; symbol traction-r1:R -> traction-r1:F; MPN R0603-CLASS -> MF-MSMF020/33X
- FLVC: renamed from LFC; value BLM31PG121SH1L -> 0680L5000-05; footprint traction:L_1206_3216Metric -> traction:Bel_0680L_2410; symbol traction-r1:L -> traction-r1:F; MPN BLM31PG121SH1L -> 0680L5000-05
- FMT1: renamed from RMT1S; value 1k -> 0438.375WRA; footprint traction:R_0603_1608Metric -> traction:Fuse_0603_1608Metric; symbol traction-r1:R -> traction-r1:F; MPN R0603-CLASS -> 0438.375WRA
- FMT2: renamed from RMT2P; value 10k -> 0438.375WRA; footprint traction:R_0603_1608Metric -> traction:Fuse_0603_1608Metric; symbol traction-r1:R -> traction-r1:F; MPN R0603-CLASS -> 0438.375WRA
- FVBH: renamed from RLVSD; value 4.7k -> MF-LSMF300/24X-2; footprint traction:R_0603_1608Metric -> traction:Fuse_2920_7451Metric; symbol traction-r1:R -> traction-r1:F; LCSC CLASS -> C719172; MPN R0603-4k7 -> MF-LSMF300/24X-2
- FVBL: renamed from RLVSG; value 10k -> MF-LSMF300/24X-2; footprint traction:R_0603_1608Metric -> traction:Fuse_2920_7451Metric; symbol traction-r1:R -> traction-r1:F; LCSC CLASS -> C719172; MPN R0603-10k -> MF-LSMF300/24X-2
- FVS1: renamed from LVS3; value MMZ1608B471CTDH5 -> MF-MSMF010/60X; footprint traction:L_0603_1608Metric -> traction:Fuse_1812_4532Metric; symbol traction-r1:L -> traction-r1:F; MPN MMZ1608B471CTDH5 -> MF-MSMF010/60X
- JICC: renamed from RCPD2; value 10k -> IPL1-120-01-L-D-K; footprint traction:R_0603_1608Metric -> traction:Samtec_IPL1-120_2x20; symbol traction-r1:R -> traction-r1:IPL1-120-01-L-D-K; MPN R0603-10k -> IPL1-120-01-L-D-K
- JLEM: renamed from USNSW; value HC5FW900-S -> T2M-105-01-L-D-TH-WT; footprint (none) -> traction:PinHeader_2x05_P2.00mm_Vertical; symbol traction-r1:HC5FW900-S -> traction-r1:T2M-105-01-L-D-TH-WT; MPN HC5FW900-S -> T2M-105-01-L-D-TH-WT
- JSWD: renamed from QLVN; value 2N7002 -> FTSH-105-01-L-DV-K; footprint traction:SOT-23-3 -> traction:Samtec_FTSH-105-01-L-DV-K; symbol traction-r1:2N7002 -> traction-r1:FTSH-105-01-L-DV-K; LCSC C8545 -> CLASS; MPN 2N7002 -> FTSH-105-01-L-DV-K
- JVEH: renamed from LVS2; value MMZ1608B471CTDH5 -> TE 770669-1 (AMPSEAL 23); footprint traction:L_0603_1608Metric -> traction:TE_770669-1; symbol traction-r1:L -> traction-r1:TE_770669-1__AMPSEAL_23_; MPN MMZ1608B471CTDH5 -> TE 770669-1 (AMPSEAL 23)
- LCAN1: renamed from CCAN1; value 1uF -> ACT45B-101-2P-TL003; footprint traction:C_0603_1608Metric -> traction:TDK_ACT45B; symbol traction-r1:C -> traction-r1:ACT45B-101-2P-TL003; MPN MLCC-1uF-25V -> ACT45B-101-2P-TL003
- LCAN2: renamed from CCAN2; value 1uF -> ACT45B-101-2P-TL003; footprint traction:C_0603_1608Metric -> traction:TDK_ACT45B; symbol traction-r1:C -> traction-r1:ACT45B-101-2P-TL003; MPN MLCC-1uF-25V -> ACT45B-101-2P-TL003
- LCOR: renamed from RDBG; value 10k -> XAL4020-222MEC; footprint traction:R_0603_1608Metric -> traction:L_Coilcraft_XAL4020-XXX; symbol traction-r1:R -> traction-r1:L; MPN R0603-CLASS -> XAL4020-222MEC
- LFC: renamed from RLVSM; value 1k -> BLM31PG121SH1L; footprint traction:R_0603_1608Metric -> traction:L_1206_3216Metric; symbol traction-r1:R -> traction-r1:L; MPN R0603-1k -> BLM31PG121SH1L
- LSBC: renamed from RSB1; value 52.3k -> XAL4040-103MEC; footprint traction:R_0603_1608Metric -> traction:L_Coilcraft_XAL4040-XXX; symbol traction-r1:R -> traction-r1:L; MPN R0603-CLASS -> XAL4040-103MEC
- LUB: renamed from RUB2; value 100R -> BLM21PG221SH1D; footprint traction:R_0603_1608Metric -> traction:L_0805_2012Metric; symbol traction-r1:R -> traction-r1:L; MPN R0603-100R -> BLM21PG221SH1D
- LVB: renamed from RVB2; value 100R -> BLM21PG221SH1D; footprint traction:R_0603_1608Metric -> traction:L_0805_2012Metric; symbol traction-r1:R -> traction-r1:L; MPN R0603-100R -> BLM21PG221SH1D
- LVS2: renamed from JICC; value IPL1-120-01-L-D-K -> MMZ1608B471CTDH5; footprint traction:Samtec_IPL1-120_2x20 -> traction:L_0603_1608Metric; symbol traction-r1:IPL1-120-01-L-D-K -> traction-r1:L; MPN IPL1-120-01-L-D-K -> MMZ1608B471CTDH5
- LVS3: renamed from RCPD0; value 10k -> MMZ1608B471CTDH5; footprint traction:R_0603_1608Metric -> traction:L_0603_1608Metric; symbol traction-r1:R -> traction-r1:L; MPN R0603-10k -> MMZ1608B471CTDH5
- LVS4: renamed from RCPD1; value 10k -> MMZ1608B471CTDH5; footprint traction:R_0603_1608Metric -> traction:L_0603_1608Metric; symbol traction-r1:R -> traction-r1:L; MPN R0603-10k -> MMZ1608B471CTDH5
- LWB: renamed from RWB2; value 100R -> BLM21PG221SH1D; footprint traction:R_0603_1608Metric -> traction:L_0805_2012Metric; symbol traction-r1:R -> traction-r1:L; MPN R0603-100R -> BLM21PG221SH1D
- QBAL: renamed from CBTC; value 47nF -> SQ2310ES; footprint traction:C_0603_1608Metric -> traction:SOT-23-3; symbol traction-r1:C -> traction-r1:SQ2310ES; MPN MLCC-47nF-50V-X7R-0603 -> SQ2310ES
- QLVN: renamed from CLVC2; value 22uF -> 2N7002; footprint traction:C_1210_3225Metric -> traction:SOT-23-3; symbol traction-r1:C -> traction-r1:2N7002; LCSC CLASS -> C8545; MPN MLCC-22uF-50V -> 2N7002
- QLVS: renamed from CLVC3; value 100uF -> DMP6023LEQ-13; footprint traction:CP_Elec_10x10.5 -> traction:SOT-223; symbol traction-r1:CP -> traction-r1:DMP6023LEQ-13; MPN EEH-ZC1H101P -> DMP6023LEQ-13
- RAGT: renamed from RSB2; value 10k -> 0R; footprint traction:R_0603_1608Metric -> traction:R_0805_2012Metric; MPN R0603-CLASS -> R0805-0R-CLASS
- RASCP: renamed from RFS3; value 1k -> 10k; MPN R0603-1k -> R0603-10k
- RBOOT: renamed from CLVC1; value 4.7uF -> 10k; footprint traction:C_1206_3216Metric -> traction:R_0603_1608Metric; symbol traction-r1:C -> traction-r1:R; MPN MLCC-4.7uF-50V -> R0603-10k
- RCOS2: renamed from RCOSR1; value 120R -> 12k; MPN R0603-120R -> R0603-CLASS
- RCOSF1: renamed from RCOSR2; value 120R -> 12k; MPN R0603-120R -> R0603-CLASS
- RCOSF2: renamed from JLEM; value T2M-105-01-L-D-TH-WT -> 12k; footprint traction:PinHeader_2x05_P2.00mm_Vertical -> traction:R_0603_1608Metric; symbol traction-r1:T2M-105-01-L-D-TH-WT -> traction-r1:R; MPN T2M-105-01-L-D-TH-WT -> R0603-CLASS
- RCOSR1: renamed from USNSU; value HC5FW900-S -> 120R; footprint (none) -> traction:R_0603_1608Metric; symbol traction-r1:HC5FW900-S -> traction-r1:R; MPN HC5FW900-S -> R0603-120R
- RCOSR2: renamed from USNSV; value HC5FW900-S -> 120R; footprint (none) -> traction:R_0603_1608Metric; symbol traction-r1:HC5FW900-S -> traction-r1:R; MPN HC5FW900-S -> R0603-120R
- RCPD1: renamed from RHWP; MPN R0603-10k-1% -> R0603-10k
- RCT1A: renamed from TVSC2; value PESD2IVN24-T -> 60.4R; footprint traction:SOT-23-3 -> traction:R_0603_1608Metric; symbol traction-r1:PESD2IVN24-T -> traction-r1:R; LCSC C406047 -> CLASS; MPN PESD2IVN24-T -> R0603-60R4-1%
- RCT1B: renamed from UCAN2; value TCAN1042HGVDRQ1 -> 60.4R; footprint traction:SOIC-8_3.9x4.9mm_P1.27mm -> traction:R_0603_1608Metric; symbol traction-r1:TCAN1042HGVDRQ1 -> traction-r1:R; LCSC C132550 -> CLASS; MPN TCAN1042HGVDRQ1 -> R0603-60R4-1%
- RCT2A: renamed from FVS1; value MF-MSMF010/60X -> 60.4R; footprint traction:Fuse_1812_4532Metric -> traction:R_0603_1608Metric; symbol traction-r1:F -> traction-r1:R; MPN MF-MSMF010/60X -> R0603-60R4-1%
- RCT2B: renamed from LVS1; value MMZ1608B471CTDH5 -> 60.4R; footprint traction:L_0603_1608Metric -> traction:R_0603_1608Metric; symbol traction-r1:L -> traction-r1:R; MPN MMZ1608B471CTDH5 -> R0603-60R4-1%
- RDBG: renamed from RSB3; value 220R -> 10k
- RENP1: renamed from RFLTD; value 10k -> 5.1k; MPN R0603-10k -> R0603-5k1
- REXA1: renamed from REXA4; value 28k -> 3k
- REXA2: renamed from REXB1; value 24k -> 10k
- REXA3: renamed from REXB2; value 24k -> 10k
- REXA4: renamed from REXB3; value 24k -> 28k
- REXB2: renamed from REXM1; value 18k -> 24k; MPN R0603-18k-1% -> R0603-CLASS
- REXB3: renamed from REXM2; value 42.2k -> 24k; MPN R0603-42k2-1% -> R0603-CLASS
- REXB4: renamed from REXM3; value 18k -> 24k; MPN R0603-18k-1% -> R0603-CLASS
- REXM1: renamed from REXM4; value 84.5k -> 18k; MPN R0603-84k5-1% -> R0603-18k-1%
- REXM2: renamed from RLDE1; value 38.3k -> 42.2k; MPN R0603-CLASS -> R0603-42k2-1%
- REXM3: renamed from RLDE2; value 10k -> 18k; MPN R0603-CLASS -> R0603-18k-1%
- REXM4: renamed from RSDN; value 10k -> 84.5k; MPN R0603-CLASS -> R0603-84k5-1%
- RFCB: renamed from RFLTP1; value 5.1k -> 100k; MPN R0603-5k1 -> R0603-100k
- RFLTC: renamed from RFLTP2; value 5.1k -> 10k; MPN R0603-5k1 -> R0603-10k
- RFLTP1: renamed from RLAT2; value 10k -> 5.1k; MPN R0603-10k -> R0603-5k1
- RFLTP2: renamed from RQDM; value 10k -> 5.1k; MPN R0603-10k -> R0603-5k1
- RFS1: renamed from RFS4; footprint traction:R_1206_3216Metric -> traction:R_0603_1608Metric; MPN ESR18EZPF1001 -> R0603-1k
- RFS3: renamed from ZSET; value BZT52-B5V6 -> 1k; footprint traction:D_SOD-123 -> traction:R_0603_1608Metric; symbol traction-r1:D_21 -> traction-r1:R; MPN BZT52-B5V6 -> R0603-1k
- RFS4: renamed from UOR1; value 74LVC1G32GW-Q100 -> 1k; footprint traction:SOT-353_SC-70-5 -> traction:R_1206_3216Metric; symbol traction-r1:74LVC1G32GW-Q100 -> traction-r1:R; LCSC C548334 -> CLASS; MPN 74LVC1G32GW-Q100 -> ESR18EZPF1001
- RGPD: renamed from RRDB; value 100k -> 10k; MPN R0603-100k -> R0603-10k
- RIGN1: renamed from RIGNS2; value 10k -> 5.1k; MPN R0603-CLASS -> R0603-5k1
- RIGN2: renamed from UAND1; value 74LVC1G11GW-Q100 -> 10k; footprint traction:SOT-363_SC-70-6 -> traction:R_0603_1608Metric; symbol traction-r1:74LVC1G11GW-Q100 -> traction-r1:R; LCSC C548242 -> CLASS; MPN 74LVC1G11GW-Q100 -> R0603-10k
- RIGNS1: renamed from UAND2; value 74LVC1G11GW-Q100 -> 47k; footprint traction:SOT-363_SC-70-6 -> traction:R_0603_1608Metric; symbol traction-r1:74LVC1G11GW-Q100 -> traction-r1:R; LCSC C548242 -> CLASS; MPN 74LVC1G11GW-Q100 -> R0603-CLASS
- RIGNS2: renamed from ULAT2; value 74LVC1G74DC-Q100 -> 10k; footprint traction:VSSOP-8_2.3x2mm_P0.5mm -> traction:R_0603_1608Metric; symbol traction-r1:74LVC1G74DC-Q100 -> traction-r1:R; MPN 74LVC1G74DC-Q100 -> R0603-CLASS
- RILK2: renamed from UVMB1; value OPA348AQDBVRQ1 -> 10k; footprint traction:SOT-23-5 -> traction:R_0603_1608Metric; symbol traction-r1:OPA348AQDBVRQ1 -> traction-r1:R; LCSC C2877787 -> CLASS; MPN OPA348AQDBVRQ1 -> R0603-10k
- RILK3: renamed from UVMB2; value OPA348AQDBVRQ1 -> 10k; footprint traction:SOT-23-5 -> traction:R_0603_1608Metric; symbol traction-r1:OPA348AQDBVRQ1 -> traction-r1:R; LCSC C2877787 -> CLASS; MPN OPA348AQDBVRQ1 -> R0603-10k
- RILK4: renamed from CVM1; value 220nF -> 10k; footprint traction:C_0603_1608Metric -> traction:R_0603_1608Metric; symbol traction-r1:C -> traction-r1:R; MPN MLCC-220nF-16V-X7R-0603 -> R0603-10k
- RLAT1: renamed from UOR2; value 74LVC1G32GW-Q100 -> 10k; footprint traction:SOT-353_SC-70-5 -> traction:R_0603_1608Metric; symbol traction-r1:74LVC1G32GW-Q100 -> traction-r1:R; LCSC C548334 -> CLASS; MPN 74LVC1G32GW-Q100 -> R0603-10k
- RLAT2: renamed from RRDYP1; value 5.1k -> 10k; MPN R0603-5k1 -> R0603-10k
- RLDE1: renamed from RSXN; value 2.2R -> 38.3k; footprint traction:R_1206_3216Metric -> traction:R_0603_1608Metric; MPN ESR18EZPF2R20 -> R0603-CLASS
- RLDE2: renamed from RSXP; value 2.2R -> 10k; footprint traction:R_1206_3216Metric -> traction:R_0603_1608Metric; MPN ESR18EZPF2R20 -> R0603-CLASS
- RLVSD: renamed from ZLVS; value BZT52-C15 -> 4.7k; footprint traction:D_SOD-123 -> traction:R_0603_1608Metric; symbol traction-r1:D_21 -> traction-r1:R; MPN BZT52-C15 -> R0603-4k7
- RLVSG: renamed from QBAL; value SQ2310ES -> 10k; footprint traction:SOT-23-3 -> traction:R_0603_1608Metric; symbol traction-r1:SQ2310ES -> traction-r1:R; MPN SQ2310ES -> R0603-10k
- RLVSM: renamed from USBC; value FS2633D -> 1k; footprint traction:FS26_HLQFP48 -> traction:R_0603_1608Metric; symbol traction-r1:FS2633D -> traction-r1:R; MPN FS2633D -> R0603-1k
- RMRST: renamed from JSWD; value FTSH-105-01-L-DV-K -> 10k; footprint traction:PinHeader_2x05_P1.27mm_Vertical -> traction:R_0603_1608Metric; symbol traction-r1:FTSH-105-01-L-DV-K -> traction-r1:R; MPN FTSH-105-01-L-DV-K -> R0603-10k
- RMT1P: renamed from RMT2S; value 1k -> 10k
- RMT1S: renamed from TVSM1; value SMAJ5.0A -> 1k; footprint traction:D_SMA -> traction:R_0603_1608Metric; symbol traction-r1:D_21 -> traction-r1:R; MPN SMAJ5.0A -> R0603-CLASS
- RMT2P: renamed from TVSM2; value SMAJ5.0A -> 10k; footprint traction:D_SMA -> traction:R_0603_1608Metric; symbol traction-r1:D_21 -> traction-r1:R; MPN SMAJ5.0A -> R0603-CLASS
- renumbered CCOSF2 to CCOSA3, CSCH3 to CLAT2, CSINF2 to CSINA3, LVS4 to LVS1, RFS2 to RARB, RCOSF2 to RCOS1, RCPD3 to RCPD0, RFLTC to RDRB, REXB4 to REXB1, RGPD to RFLTD, RLAT1 to RFS2, RILK4 to RILK1, RSCH to RRDB, RSINF2 to RSIN1, RVD1D to RVD1A, RVD2A to RVD1D, RVD2D to RVD2A, RVM4 to RVM1
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Connections:
- net AGND: now also CCOSA1.2, CCOSA3.2, CEXD.2, CIGNS.2, CLDE.2, CMT1F.2, CMT2F.2, CR2R1.2, CR2R2.2, CSINA1.2, CSINA3.2, CSNUF.2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; no longer CCT2.10 (MT1R), CCT2.12 (MT2R), CEXA1.2, DBAT.1, DCOSP.2, DSINP.2, JLEM.5 (E1), JLEM.7 (E3), JLEM.8 (E4), LVS2.3 (P3_AGND), RCOSF2.10 (G3), RCOSF2.3 (G1)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
- net AMUXO: now also RSB3.1, USBC.29 (AMUX); no longer RDBG.1, RLVSM.29 (AMUX)
- net ASC_CLR_M: now also RFS3.1; no longer RASCP.1
- net ASC_CLR_N: now also RFS3.2, RLAT1.2, ULAT.6 (CLR_N); no longer RASCP.2, RFS2.2, RV5GP.6 (CLR_N)
- net ASC_CMD: now also JICC.15 (P15_ASC_CMD), RARB.1, UASCG.4 (Y); no longer CASCG.1, LVS2.15 (P15_ASC_CMD), RSCH.4 (Y)
- net ASC_CMD_RB: now also RARB.2; no longer CASCG.2
- net ASC_Q: now also RASCP.1, UASCG.2 (A), ULAT.5 (Q); no longer CLAT.1, RSCH.2 (A), RV5GP.5 (Q)
- net ASC_REQ: now also RCPD1.1, ULAT.1 (CLK); no longer LVS4.1, RV5GP.1 (CLK)
- net ASC_SET_B: now also ULAT.7 (PRE_N), USCH2.5 (Y2); no longer RV5GP.7 (PRE_N), UAND2.5 (Y2)
- net ASC_SET_N: now also RFS1.2, RFS2.2, USCH2.3 (A2), ZSET.1; no longer DFO.2, RARB.2, RFS3.1, UAND2.3 (A2)
- net BATSNS: now also DBAT.1, USBC.48 (BATSENSE); no longer CSB8.1, RLVSM.48 (BATSENSE)
- net BCTRL: now also CBAL.1, QBAL.1 (G); no longer RLVSG.1 (G), ZLVS.1
- net CAN0_RX: now also UCAN1.4 (RXD); no longer TVSM2.4 (RXD)
- net CAN0_TX: now also UCAN1.1 (TXD); no longer TVSM2.1 (TXD)
- net CAN1_RX: now also UCAN2.4 (RXD); no longer RCT1B.4 (RXD)
- net CAN1_TX: now also UCAN2.1 (TXD); no longer RCT1B.1 (TXD)
- net CANH1: now also LCAN1.4 (A2), LVS1.2, TVSC1.1 (A); no longer RCT2B.2, RMT2S.4 (A2), TVSM1.1 (A)
- net CANH1_T: now also LCAN1.1 (A1), RCT1A.1, UCAN1.7 (CANH); no longer RMT2S.1 (A1), TVSM2.7 (CANH), UCAN1.1
- net CANH2: now also LCAN2.4 (A2), LVS3.2, TVSC2.1 (A); no longer CCT1.4 (A2), FVS1.2, RCT1A.1 (A)
- net CANH2_T: now also LCAN2.1 (A1), RCT2A.1, UCAN2.7 (CANH); no longer CCT1.1 (A1), RCT1B.7 (CANH), UCAN2.1
- net CANL1: now also LCAN1.3 (B2), LVS2.2, TVSC1.2 (B); no longer JVEH.2, RMT2S.3 (B2), TVSM1.2 (B)
- net CANL1_T: now also LCAN1.2 (B1), RCT1B.2, UCAN1.6 (CANL); no longer CCAN1.2, RMT2S.2 (B1), TVSM2.6 (CANL)
- net CANL2: now also LCAN2.3 (B2), LVS4.2, TVSC2.2 (B); no longer CCT1.3 (B2), LVS1.2, RCT1A.2 (B)
- net CANL2_T: now also LCAN2.2 (B1), RCT2B.2, UCAN2.6 (CANL); no longer CCAN2.2, CCT1.2 (B1), RCT1B.6 (CANL)
- net CANS1: now also CCT1.1, RCT1A.2, RCT1B.1; no longer CCAN1.1, TVSC1.1, UCAN1.2
- net CANS2: now also CCT2.1, RCT2A.2, RCT2B.1; no longer CCAN2.1, TVSC2.1, UCAN2.2
- net CORBT: now also CBTC.1, USBC.33 (CORE_BT); no longer QBAL.1, RLVSM.33 (CORE_BT)
- net COSF_N: now also CCOSD.2, CCOSF2.1, DCOSP.2 (B), RCOSF2.2, RCOSR2.1; no longer CCOSA1.2, CCOSA3.1, RCOS1.2, RCOSF1.1, RSINF2.2 (B)
- net COSF_P: now also CCOSD.1, CCOSF1.1, DCOSP.1 (A), RCOSF1.2, RCOSR1.1; no longer CCOSA1.1, CCOSA2.1, CCOSF2.2, RCOS2.1, RSINF2.1 (A)
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Other:
- note added: "rev A.22 - 26 sections - 304 components"
- note removed: "rev A.21 - 26 sections - 301 components"
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
Commit message: Rev A.23: round 24 — four rechecks of 4ed0101 (F240–F244): the SDADC reference on its supply node, acquisition freshness, the map's flux slope and the ripple limiter's exact bounds, the temperature latch, the V_DC expiry
Hardware (F240, no new part): the S32K39 data sheet's SDADC table (Rev. 3 Table 38, in our archive and our own
extracted-parameters file) requires VREFP within ±25 mV of AVDD; the round-23 disposition had judged the general +100 mV
note and called the figure absent while the references sat on the FS26 VREF, matched to the SDADC-supply LDO only within
±1 %. Every non-R2R reference group (E6/H6 SAR, E10/F13 SDADC) is now on V5A itself with VDDA_SDADC and VDD_HV_A (NXP's
GEN3 arrangement); the ratiometric loads (HW_ID and offset dividers, the seven NTC pull-ups) moved with the reference; the
R2R ladder keeps the FS26 VREF as its isolated supply through the 10 Ω branch (CR2R1 330 nF, 37 kHz); CSB5 2.2 µF holds
the FS26 window alone (1.36–2.92 µF effective); the absolute SAR scale re-budgeted at the LDO2's ±1.75 %; ERC locks, pin
freeze, manifest, handoff §4.11 island rule (≤ 20 mΩ from E12 to any VREFH ball), VR-34 closed by design, IR-26, QP-TH-06.
Pipeline at A.23: ERC 981/0/0, verify 158/18/0, sim 23/6/0, Marine 87/23/0, 21 pages / 2065 pins, KiCad proof PASS, PDFs
and BOMs regenerated (₹72,983 unchanged). The handoff §6 gives every open pre-layout decision a provisional default.

Firmware (TI_FW_ID 0x0A0F0016, CAL layout 4, 191 fields / 92 CAL rows, 82 DTCs): F241 a stopped slow ADC channel stayed
valid forever (the caller discarded the acquisition stamp) → a three-state contract new/held/expired for every slow-list
input with cal_temp_hold_ms and DTC_ADC_SLOW_STALE, every slow consumer audited (V5GD/VOFS, IGN, INTRLOK_N, VSUP, HW_ID);
F242 the inductance map must keep a positive flux slope (≥ 0.25 × L0 below every breakpoint) and the ripple limiter bounds
every piece of its interval in closed form (breakpoints alone shown insufficient by a 20 000-m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
Parts:
- CR2R1: value 1uF -> 330nF; MPN MLCC-1uF-10V-X7R-0603 -> MLCC-330nF-16V-X7R-0603
- CSB5: value 1uF -> 2.2uF; MPN MLCC-1uF-16V-X7R-0805 -> MLCC-2.2uF-16V-X7R-0805
Connections:
- net V5A: now also CMA1.1, CMA2.1, RHWP.1, RMT1P.1, RMT2P.1, ROF1.1, RSNUP.1, RSNVP.1, RSNWP.1, RTAMBP.1, RTHSP.1, UMCU.E10 (E10_VREFH_SDADC_01), UMCU.E6 (E6_VREFH_SAR_456), UMCU.F13 (F13_VREFH_SDADC_23), UMCU.H6 (H6_VREFH_SAR_0123)
- net VREF5: no longer CMA1.1, CMA2.1, RHWP.1, RMT1P.1, RMT2P.1, ROF1.1, RSNUP.1, RSNVP.1, RSNWP.1, RTAMBP.1, RTHSP.1, UMCU.E10 (E10_VREFH_SDADC_01), UMCU.E6 (E6_VREFH_SAR_456), UMCU.F13 (F13_VREFH_SDADC_23), UMCU.H6 (H6_VREFH_SAR_0123)
Other:
- note added: "rev A.23 - 26 sections - 304 components"
- note removed: "rev A.22 - 26 sections - 304 components"
Changed lines of the file:
@@
 Title "Traction Inverter — Control Card (S32K396 + FS26, ASIL D)"
 Date "2026-09-23"
-Rev "A.22"
+Rev "A.23"
 Comp "Traction Inverter 220 kW pk - Control card (LV), sheet 4 of 4"
 Comment1 "Inverter = Power board + Cap bank busbar + bolt-on Discharge board (all HV) + Control card (LV); safe state holds with any link lost"
@@
 VEHICLE-IF   -   1 section
 Text Notes 40810 15050 0    60   ~ 0
-rev A.22   -   26 sections   -   304 components
+rev A.23   -   26 sections   -   304 components
 Wire Notes Line
 	40750 16000 45200 16000
@@
 	3200 5100 3000 5100
 Text Label 3000 5100 2    45   ~ 0
-VREF5
+V5A
 Wire Wire Line
 	3200 5200 3000 5200
@@
 	3200 5600 3000 5600
 Text Label 3000 5600 2    45   ~ 0
-VREF5
+V5A
 Wire Wire Line
 	3200 5700 3000 5700
@@
 	3200 6100 3000 6100
 Text Label 3000 6100 2    45   ~ 0
-VREF5
+V5A
 Wire Wire Line
 	3200 6200 3000 6200
@@
 	4900 1400 5100 1400
 Text Label 5100 1400 0    45   ~ 0
-VREF5
+V5A
 Wire Wire Line
 	4900 1500 5100 1500
@@
 	6100 2750 5900 2750
 Text Label 5900 2750 2    45   ~ 0
-VREF5
+V5A
 Wire Wire Line
 	6600 2750 6800 2750
@@
 	6100 3150 5900 3150
 Text Label 5900 3150 2    45   ~ 0
-VREF5
+V5A
 Wire Wire Line
 	6600 3150 6800 3150
@@
 P 9450 1150
 F 0 "CR2R1" H 9450 990 50  0000 C CNN
-F 1 "1uF" H 9450 1320 50  0000 C CNN
+F 1 "330nF" H 9450 1320 50  0000 C CNN
 F 2 "traction:C_0603_1608Metric" H 9450 1150 50  0001 C CNN
 F 3 "~" H 9450 1150 50  0001 C CNN
 F 4 "CLASS" H 9450 1150 50  0001 C CNN "LCSC"
-F 5 "MLCC-1uF-10V-X7R-0603" H 9450 1150 50  0001 C CNN "MPN"
+F 5 "MLCC-330nF-16V-X7R-0603" H 9450 1150 50  0001 C CNN "MPN"
 	1    9450 1150
 	1    0    0    -1
@@
 P 19300 6900
 F 0 "CSB5" H 19300 6740 50  0000 C CNN
-F 1 "1uF" H 19300 7070 50  0000 C CNN
+F 1 "2.2uF" H 19300 7070 50  0000 C CNN
 F 2 "traction:C_0805_2012Metric" H 19300 6900 50  0001 C CNN
 F 3 "~" H 19300 6900 50  0001 C CNN
 F 4 "CLASS" H 19300 6900 50  0001 C CNN "LCSC"
-F 5 "MLCC-1uF-16V-X7R-0805" H 19300 6900 50  0001 C CNN "MPN"
+F 5 "MLCC-2.2uF-16V-X7R-0805" H 19300 6900 50  0001 C CNN "MPN"
 	1    19300 6900
 	1    0    0    -1
@@
 	5700 24150 5500 24150
 Text Label 5500 24150 2    45   ~ 0
-VREF5
+V5A
 Wire Wire Line
 	6200 24150 6400 24150
@@
 	33250 10400 33050 10400
 Text Label 33050 10400 2    45   ~ 0
-VREF5
+V5A
 Wire Wire Line
 	33750 10400 33950 10400
@@
 	33250 11200 33050 11200
 Text Label 33050 11200 2    45   ~ 0
-VREF5
+V5A
 Wire Wire Line
 	33750 11200 33950 11200
@@
 	33250 12000 33050 12000
 Text Label 33050 12000 2    45   ~ 0
-VREF5
+V5A
 Wire Wire Line
 	33750 12000 33950 12000
@@
 	34050 15350 33850 15350
 Text Label 33850 15350 2    45   ~ 0
-VREF5
+V5A
 Wire Wire Line
 	34550 15350 34750 15350
@@
 	34050 16150 33850 16150
 Text Label 33850 16150 2    45   ~ 0
-VREF5
+V5A
 Wire Wire Line
 	34550 16150 34750 16150
@@
 	18050 20050 17850 20050
 Text Label 17850 20050 2    45   ~ 0
-VREF5
+V5A
 Wire Wire Line
 	18550 20050 18750 20050
@@
 	20100 20050 19900 20050
 Text Label 19900 20050 2    45   ~ 0
-VREF5
+V5A
 Wire Wire Line
 	20600 20050 20800 20050
@@
 	45600 8750 45400 8750
 Text Label 45400 8750 2    45   ~ 0
-VREF5
+V5A
 Wire Wire Line
 	46100 8750 46300 8750
