File: kicad5/traction-native/traction-power.sch (KiCad schematic (older format))
At the start: 324 parts, among them U5LB NCV4276CDT50RKG, U5LC NCV4276CDT50RKG

Commit message: Rev A.16: round 17 — gap closure (F174-F189) + round 16 rev A.15 (F167-F173): every gap closed, upgraded or numbered
Round 16 (rev A.15, three rechecks of 32214be): exciter MFB gain 24 k -> 28 k with the amplitude
planes (setpoint 7.2 V pp at the monitor), unidirectional exciter TVS, /33X hold 0.07 A, firmware
acquisition contracts (phase triplets, resolver frame age, coherent SDADC frames); BOM furnished
(spec-class capacitors, drawn-size gate in bom-gen, last placeholders bound with archived sheets).

Round 17 (rev A.16, "close all gaps" / "feel free to upgrade"):
- Hardware: DEXP/DEXN PMEG4050EP-Q rated back-drive diversion (closes the ALM2402 OPEN row);
  exciter TVS -> SMDJ8.5A-HRA (3 kW, AEC-Q101, same pad); fault rows split single fault (PASS
  at any source impedance) vs load-dump-coincident double event; LV entry re-designed as
  LET-THROUGH for ISO 16750-2 test B (TPSMC33A-VR/TPSMC18A-VR anti-series pair at the pin ahead
  of the reverse Schottky, TPSMC33CA-VR on the power board, CLVC3 100 uF hybrid polymer, FLVC
  5 A fuse, DIGN US1M, ULDO15 D2PAK) — pulse 1 was avalanching DREVC, the 2023 26 V jump start
  opened the old TVS, the polyfuse was undersized at 9 V; RFS4 -> ESR18 1206.
- Stale/unsourced rows recomputed: cold-crank excitation, PTC hold (IR-13), discharge resistor
  no-flame statement, hall reference drift, ASC command-path collapse.
- KiCad: a KiCad 9/10 set (kicad/traction, Traction-Inverter-KiCad-modern.zip) proved by
  kicad-cli netlist export on every board with mutation tests; KiCad 10 cannot resolve the KiCad 5
  legacy symbols; the proof exposed harness pins numbered P1-P40 and the SMDJ drawn as a resistor
  in the legacy generator — fixed; sym-lib-table + cache library in both legacy sets.
- Firmware: all 35 open contract items closed (FW-08 zero-current decision, FW-31 liveness,
  FW-32 UDS service-lock routine, FW-33 supply-overvoltage supervision), FS26 watchdog answer
  3.0 ms -> 2.0 ms, ASC-exit release wait CAL, 39-row silicon/RM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
Parts:
- CB15C: MPN MLCC-CLASS -> MLCC-470pF-50V-C0G-0603
- CB15I: footprint C1210 -> C1206; MPN MLCC-10uF-50V -> MLCC-10uF-50V-X7R-1206
- CB15S: MPN MLCC-CLASS -> MLCC-47nF-50V-X7R-0603
- CFHCF, CFLCF: MPN MLCC-CLASS -> MLCC-47pF-50V-C0G-0603
- CFHCO, CFLCO: MPN MLCC-CLASS -> MLCC-22nF-50V-X7R-0603
- CFHCT, CFLCT: MPN MLCC-CLASS -> MLCC-680pF-50V-C0G-0603
- CFHSI, CFLSI: MPN MLCC-CLASS -> MLCC-100pF-50V-C0G-0603
- CLD15: footprint C0603 -> C1210; MPN MLCC-CLASS -> MLCC-22uF-25V-X7R-1210
- CLDC: MPN MLCC-CLASS -> MLCC-220pF-50V-C0G-0603
- CPET: footprint C0603 -> disc, 10 mm pitch (FilmBoxFP(10) land); MPN MLCC-CLASS -> VY2472M49Y5US6TV0
- DTVH, DTVL: value TPSMC24CA-VR -> TPSMC33CA-VR; LCSC C1975284 -> CLASS; MPN TPSMC24CA-VR -> TPSMC33CA-VR
- JDIS: value HDR-1x4-2.54 -> IPL1-104-01-L-S-K; footprint HDR1x4 -> IPL1-104 (1x4 2.54 mm THT); symbol traction-r1:HDR-1x4-2.54 -> traction-r1:IPL1-104-01-L-S-K; MPN HDR-1x4-2.54 -> IPL1-104-01-L-S-K
- JHVIL: value HDR-1x2-2.54 -> IPL1-102-01-L-S-K; footprint HDR1x2 -> IPL1-102 (1x2 2.54 mm THT); MPN HDR-1x2-2.54 -> IPL1-102-01-L-S-K
- LFH1, LFL1: value FB-120R-3A -> BLM31PG121SH1L; MPN FB-120R-3A -> BLM31PG121SH1L
- RPET: footprint R0603 -> R1206; MPN R0603-CLASS -> R1206-1M-CLASS
- ULDO15: value NCV4276CDTADJRKG -> NCV4276CDSADJR4G; footprint DPAK5 -> D2PAK5; symbol traction-r1:NCV4276CDTADJRKG -> traction-r1:NCV4276CDSADJR4G; MPN NCV4276CDTADJRKG -> NCV4276CDSADJR4G
Other:
- note added: "rev A.16 - 24 sections - 324 components"
- note removed: "rev A.14 - 24 sections - 324 components"
- moved on the sheet: CB15C, CB15CC, CB15I, CB15S, CLD15, CLDC, RB15C, RB15Q, RLD1, RLD2, UB15, ULDO15

Commit message: Rev A.17: round 18 — three rechecks of 4425af9 (F190-F198): diversion diodes on the amplifier node (loop passes RSX), diode cell cathode = pin 1 on all 35 diodes, exciter TVS/PTC rows at worst corners + ECU-asleep sustained short (WARN rows, layout rule, QP-RX-04 2b gate), anti-surge RSX, NCV4276C reverse current = QP-RX-05 gate + VR-33, IR-16/IR-42, firmware FW-34..36 (sample freshness, cadence-locked resolver frames, latency sign) + three self-found instances
Co-Authored-By: Claude Fable 5.1 <noreply@anthropic.com>
Parts:
- DASCR, DB15, DFHA, DFHFS, DFHG, DFHSN, DFHVZ, DFLA, DFLFS, DFLG, DFLSN, DFLVZ, DRH, DRL, DTVH, DTVL, DTVSH, DUHR, DUHS1, DUHS2, DUHZ1, DUHZ2, DULR, DULS1, DULS2, DULZ1, DULZ2, DUTP, DVHR, DVHS1, DVHS2, DVHZ1, DVHZ2, DVLR, DVLS1, DVLS2, DVLZ1, DVLZ2, DVTP, DWHR, DWHS1, DWHS2, DWHZ1, DWHZ2, DWLR, DWLS1, DWLS2, DWLZ1, DWLZ2, DWTP, ZASC, ZFHG, ZFHSN, ZFLG, ZFLSN, ZUHV, ZULV, ZVHV, ZVLV, ZWHV, ZWLV: symbol traction-r1:D -> traction-r1:D_21
Connections:
- net ASCVO: now also DASCR.1; no longer DASCR.2
- net ASC_DRV: now also DASCR.2, ZASC.1; no longer DASCR.1, ZASC.2
- net B15SW: now also DB15.2; no longer DB15.1
- net DCN: now also ZASC.2; no longer ZASC.1
- net DGND: now also DFHVZ.2, DFLVZ.2, DTVH.2, DTVL.2, DTVSH.2; no longer DFHVZ.1, DFLVZ.1, DTVH.1, DTVL.1, DTVSH.1
- net DS1_UH: now also DUHS1.2; no longer DUHS1.1
- net DS1_UL: now also DULS1.2; no longer DULS1.1
- net DS1_VH: now also DVHS1.2; no longer DVHS1.1
- net DS1_VL: now also DVLS1.2; no longer DVLS1.1
- net DS1_WH: now also DWHS1.2; no longer DWHS1.1
- net DS1_WL: now also DWLS1.2; no longer DWLS1.1
- net DS2_UH: now also DUHS1.1, DUHS2.2; no longer DUHS1.2, DUHS2.1
- net DS2_UL: now also DULS1.1, DULS2.2; no longer DULS1.2, DULS2.1
- net DS2_VH: now also DVHS1.1, DVHS2.2; no longer DVHS1.2, DVHS2.1
- net DS2_VL: now also DVLS1.1, DVLS2.2; no longer DVLS1.2, DVLS2.1
- net DS2_WH: now also DWHS1.1, DWHS2.2; no longer DWHS1.2, DWHS2.1
- net DS2_WL: now also DWLS1.1, DWLS2.2; no longer DWLS1.2, DWLS2.1
- net DSH_U: now also DUHS2.1; no longer DUHS2.2
- net DSH_V: now also DVHS2.1; no longer DVHS2.2
- net DSH_W: now also DWHS2.1; no longer DWHS2.2
- net FAX_H: now also DFHA.2, DFHFS.2; no longer DFHA.1, DFHFS.1
- net FAX_L: now also DFLA.2, DFLFS.2; no longer DFLA.1, DFLFS.1
- net FCL_H: now also DFHSN.1, ZFHSN.1; no longer DFHSN.2, ZFHSN.2
- net FCL_L: now also DFLSN.1, ZFLSN.1; no longer DFLSN.2, ZFLSN.2
- net FCS_H: now also ZFHG.2; no longer ZFHG.1
- net FCS_L: now also ZFLG.2; no longer ZFLG.1
- net FDR_H: now also DFHG.1; no longer DFHG.2
- net FDR_L: now also DFLG.1; no longer DFLG.2
- net FFD_H: now also DFHFS.1; no longer DFHFS.2
- net FFD_L: now also DFLFS.1; no longer DFLFS.2
- net FGO_H: now also DFHG.2; no longer DFHG.1
- net FGO_L: now also DFLG.2; no longer DFLG.1
- net FG_H: now also ZFHG.1; no longer ZFHG.2
- net FG_L: now also ZFLG.1; no longer ZFLG.2
- net FHO: now also DRH.2; no longer DRH.1
- net FLO: now also DRL.2; no longer DRL.1
- net FSW_H: now also DFHSN.2; no longer DFHSN.1
- net FSW_L: now also DFLSN.2; no longer DFLSN.1
- net FVCC_H: now also DFHA.1, DFHVZ.1; no longer DFHA.2, DFHVZ.2
- net FVCC_L: now also DFLA.1, DFLVZ.1; no longer DFLA.2, DFLVZ.2
- net G_UH: now also DUHZ1.1; no longer DUHZ1.2
- net G_UL: now also DULZ1.1; no longer DULZ1.2
- net G_VH: now also DVHZ1.1; no longer DVHZ1.2
- net G_VL: now also DVLZ1.1; no longer DVLZ1.2
- net G_WH: now also DWHZ1.1; no longer DWHZ1.2
- net G_WL: now also DWLZ1.1; no longer DWLZ1.2
- net HVIL_B: now also DTVSH.1; no longer DTVSH.2
- net KS_UH: now also DUHZ2.1, ZUHV.1; no longer DUHZ2.2, ZUHV.2
- net KS_UL: now also DULZ2.1, ZULV.1; no longer DULZ2.2, ZULV.2
- net KS_VH: now also DVHZ2.1, ZVHV.1; no longer DVHZ2.2, ZVHV.2
- net KS_VL: now also DVLZ2.1, ZVLV.1; no longer DVLZ2.2, ZVLV.2
- net KS_WH: now also DWHZ2.1, ZWHV.1; no longer DWHZ2.2, ZWHV.2
- net KS_WL: now also DWLZ2.1, ZWLV.1; no longer DWLZ2.2, ZWLV.2
- net NRH: now also DRH.1, DTVH.1; no longer DRH.2, DTVH.2
- net NRL: now also DRL.1, DTVL.1; no longer DRL.2, DTVL.2
- net PHU: now also DULS2.1; no longer DULS2.2
- net PHV: now also DVLS2.1; no longer DVLS2.2
- net PHW: now also DWLS2.1; no longer DWLS2.2
- net TMOD_U: now also DUTP.2; no longer DUTP.1
- net TMOD_V: now also DVTP.2; no longer DVTP.1
- net TMOD_W: now also DWTP.2; no longer DWTP.1
- net V12H: now also ZFHSN.2; no longer ZFHSN.1
- net V12L: now also ZFLSN.2; no longer ZFLSN.1
- net V15B: now also DB15.1; no longer DB15.2
- net V5GD: now also DUTP.1, DVTP.1, DWTP.1; no longer DUTP.2, DVTP.2, DWTP.2
- net VCC_UH: now also DUHR.1; no longer DUHR.2
- net VCC_UL: now also DULR.1; no longer DULR.2
- net VCC_VH: now also DVHR.1; no longer DVHR.2
- net VCC_VL: now also DVLR.1; no longer DVLR.2
- net VCC_WH: now also DWHR.1; no longer DWHR.2
- net VCC_WL: now also DWLR.1; no longer DWLR.2
- net VEE_UH: now also ZUHV.2; no longer ZUHV.1
- net VEE_UL: now also ZULV.2; no longer ZULV.1
- net VEE_VH: now also ZVHV.2; no longer ZVHV.1
- net VEE_VL: now also ZVLV.2; no longer ZVLV.1
- net VEE_WH: now also ZWHV.2; no longer ZWHV.1
- net VEE_WL: now also ZWLV.2; no longer ZWLV.1
- net W_UH_A: now also DUHR.2; no longer DUHR.1
- net W_UL_A: now also DULR.2; no longer DULR.1
- net W_VH_A: now also DVHR.2; no longer DVHR.1
- net W_VL_A: now also DVLR.2; no longer DVLR.1
- net W_WH_A: now also DWHR.2; no longer DWHR.1
- net W_WL_A: now also DWLR.2; no longer DWLR.1
- net ZK_UH: now also DUHZ1.2, DUHZ2.2; no longer DUHZ1.1, DUHZ2.1
- net ZK_UL: now also DULZ1.2, DULZ2.2; no longer DULZ1.1, DULZ2.1
- net ZK_VH: now also DVHZ1.2, DVHZ2.2; no longer DVHZ1.1, DVHZ2.1
- net ZK_VL: now also DVLZ1.2, DVLZ2.2; no longer DVLZ1.1, DVLZ2.1
- net ZK_WH: now also DWHZ1.2, DWHZ2.2; no longer DWHZ1.1, DWHZ2.1
- net ZK_WL: now also DWLZ1.2, DWLZ2.2; no longer DWLZ1.1, DWLZ2.1
Other:
- note added: "rev A.17 - 24 sections - 324 components"
- note removed: "rev A.16 - 24 sections - 324 components"
Changed lines of the file:
@@
 Title "Traction Inverter 220 kW — Power board (3x EconoDUAL 3 SiC)"
 Date "2026-09-23"
-Rev "A.16"
+Rev "A.17"
 Comp "Traction Inverter 220 kW pk - Power (HV), sheet 1 of 4"
 Comment1 "Inverter = Power board + Cap bank busbar + bolt-on Discharge board (all HV) + Control card (LV); safe state holds with any link lost"
@@
 DC-LINK   -   1 section
 Text Notes 29160 24850 0    60   ~ 0
-rev A.16   -   24 sections   -   324 components
+rev A.17   -   24 sections   -   324 components
 Wire Notes Line
 	9100 28000 17750 28000
@@
 DC-INPUT / HVIL
 $Comp
-L traction-r1:D DTVSH
+L traction-r1:D_21 DTVSH
 U 1 1 5E000008
 P 6300 1150
@@
 TMOD_RTN
 $Comp
-L traction-r1:D DUTP
+L traction-r1:D_21 DUTP
 U 1 1 5E000010
 P 11250 2750
@@
 KS_UH
 $Comp
-L traction-r1:D DUHR
+L traction-r1:D_21 DUHR
 U 1 1 5E00001A
 P 5400 8900
@@
 VCC_UH
 $Comp
-L traction-r1:D DUHS1
+L traction-r1:D_21 DUHS1
 U 1 1 5E00001B
 P 1750 11850
@@
 DS2_UH
 $Comp
-L traction-r1:D DUHS2
+L traction-r1:D_21 DUHS2
 U 1 1 5E00001C
 P 1750 12250
@@
 VCC_UH
 $Comp
-L traction-r1:D DUHZ1
+L traction-r1:D_21 DUHZ1
 U 1 1 5E00001E
 P 3800 10900
@@
 G_UH
 $Comp
-L traction-r1:D DUHZ2
+L traction-r1:D_21 DUHZ2
 U 1 1 5E00001F
 P 3800 11300
@@
 KS_UH
 $Comp
-L traction-r1:D ZUHV
+L traction-r1:D_21 ZUHV
 U 1 1 5E000027
 P 5400 9300
@@
 KS_UL
 $Comp
-L traction-r1:D DULR
+L traction-r1:D_21 DULR
 U 1 1 5E00002F
 P 5300 14400
@@
 VCC_UL
 $Comp
-L traction-r1:D DULS1
+L traction-r1:D_21 DULS1
 U 1 1 5E000030
 P 1700 17350
@@
 DS2_UL
 $Comp
-L traction-r1:D DULS2
+L traction-r1:D_21 DULS2
 U 1 1 5E000031
 P 1700 17750
@@
 VCC_UL
 $Comp
-L traction-r1:D DULZ1
+L traction-r1:D_21 DULZ1
 U 1 1 5E000033
 P 3700 16400
@@
 G_UL
 $Comp
-L traction-r1:D DULZ2
+L traction-r1:D_21 DULZ2
 U 1 1 5E000034
 P 3700 16800
@@
 KS_UL
 $Comp
-L traction-r1:D ZULV
+L traction-r1:D_21 ZULV
 U 1 1 5E00003D
 P 5300 14800
@@
 TMOD_RTN
 $Comp
-L traction-r1:D DVTP
+L traction-r1:D_21 DVTP
 U 1 1 5E000041
 P 11250 17000
@@
 KS_VH
 $Comp
-L traction-r1:D DVHR
+L traction-r1:D_21 DVHR
 U 1 1 5E00004B
 P 13400 4400
@@
 VCC_VH
 $Comp
-L traction-r1:D DVHS1
+L traction-r1:D_21 DVHS1
 U 1 1 5E00004C
 P 9750 7350
@@
 DS2_VH
 $Comp
-L traction-r1:D DVHS2
+L traction-r1:D_21 DVHS2
 U 1 1 5E00004D
 P 9750 7750
@@
 VCC_VH
 $Comp
-L traction-r1:D DVHZ1
+L traction-r1:D_21 DVHZ1
 U 1 1 5E00004F
 P 11800 6400
@@
 G_VH
 $Comp
-L traction-r1:D DVHZ2
+L traction-r1:D_21 DVHZ2
 U 1 1 5E000050
 P 11800 6800
@@
 KS_VH
 $Comp
-L traction-r1:D ZVHV
+L traction-r1:D_21 ZVHV
 U 1 1 5E000058
 P 13400 4800
@@
 KS_VL
 $Comp
-L traction-r1:D DVLR
+L traction-r1:D_21 DVLR
 U 1 1 5E000060
 P 13300 9900
@@
 VCC_VL
 $Comp
-L traction-r1:D DVLS1
+L traction-r1:D_21 DVLS1
 U 1 1 5E000061
 P 9700 12850
@@
 DS2_VL
 $Comp
-L traction-r1:D DVLS2
+L traction-r1:D_21 DVLS2
 U 1 1 5E000062
 P 9700 13250
@@
 VCC_VL
 $Comp
-L traction-r1:D DVLZ1
+L traction-r1:D_21 DVLZ1
 U 1 1 5E000064
 P 11700 11900
@@
 G_VL
 $Comp
-L traction-r1:D DVLZ2
+L traction-r1:D_21 DVLZ2
 U 1 1 5E000065
 P 11700 12300
@@
 KS_VL
 $Comp
-L traction-r1:D ZVLV
+L traction-r1:D_21 ZVLV
 U 1 1 5E00006E
 P 13300 10300
@@
 TMOD_RTN
 $Comp
-L traction-r1:D DWTP
+L traction-r1:D_21 DWTP
 U 1 1 5E000072
 P 23250 8250
@@
 KS_WH
 $Comp
-L traction-r1:D DWHR
+L traction-r1:D_21 DWHR
 U 1 1 5E00007C
 P 17400 15400
@@
 VCC_WH
 $Comp
-L traction-r1:D DWHS1
+L traction-r1:D_21 DWHS1
 U 1 1 5E00007D
 P 13750 18350
@@
 DS2_WH
 $Comp
-L traction-r1:D DWHS2
+L traction-r1:D_21 DWHS2
 U 1 1 5E00007E
 P 13750 18750
@@
 VCC_WH
 $Comp
-L traction-r1:D DWHZ1
+L traction-r1:D_21 DWHZ1
 U 1 1 5E000080
 P 15800 17400
@@
 G_WH
 $Comp
-L traction-r1:D DWHZ2
+L traction-r1:D_21 DWHZ2
 U 1 1 5E000081
 P 15800 17800
@@
 KS_WH
 $Comp
-L traction-r1:D ZWHV
+L traction-r1:D_21 ZWHV
 U 1 1 5E000089
 P 17400 15800
@@
 KS_WL
 $Comp
-L traction-r1:D DWLR
+L traction-r1:D_21 DWLR
 U 1 1 5E000091
 P 25300 1150
@@
 VCC_WL
 $Comp
-L traction-r1:D DWLS1
+L traction-r1:D_21 DWLS1
 U 1 1 5E000092
 P 21700 4100
@@
 DS2_WL
 $Comp
-L traction-r1:D DWLS2
+L traction-r1:D_21 DWLS2
 U 1 1 5E000093
 P 21700 4500
@@
 VCC_WL
 $Comp
-L traction-r1:D DWLZ1
+L traction-r1:D_21 DWLZ1
 U 1 1 5E000095
 P 23700 3150
@@
 G_WL
 $Comp
-L traction-r1:D DWLZ2
+L traction-r1:D_21 DWLZ2
 U 1 1 5E000096
 P 23700 3550
@@
 KS_WL
 $Comp
-L traction-r1:D ZWLV
+L traction-r1:D_21 ZWLV
 U 1 1 5E00009F
 P 25300 1550
@@
 DGND
 $Comp
-L traction-r1:D DFHA
+L traction-r1:D_21 DFHA
 U 1 1 5E0000AF
 P 6350 22200
@@
 FVCC_H
 $Comp
-L traction-r1:D DFHFS
+L traction-r1:D_21 DFHFS
 U 1 1 5E0000B0
 P 10200 20300
@@
 FFD_H
 $Comp
-L traction-r1:D DFHG
+L traction-r1:D_21 DFHG
 U 1 1 5E0000B1
 P 2400 23550
@@
 FDR_H
 $Comp
-L traction-r1:D DFHSN
+L traction-r1:D_21 DFHSN
 U 1 1 5E0000B2
 P 4350 22850
@@
 FCL_H
 $Comp
-L traction-r1:D DFHVZ
+L traction-r1:D_21 DFHVZ
 U 1 1 5E0000B3
 P 6350 23000
@@
 FVCC_H
 $Comp
-L traction-r1:D ZFHG
+L traction-r1:D_21 ZFHG
 U 1 1 5E0000C0
 P 2400 23950
@@
 FG_H
 $Comp
-L traction-r1:D ZFHSN
+L traction-r1:D_21 ZFHSN
 U 1 1 5E0000C1
 P 10200 21100
@@
 DGND
 $Comp
-L traction-r1:D DFLA
+L traction-r1:D_21 DFLA
 U 1 1 5E0000D1
 P 18350 23200
@@
 FVCC_L
 $Comp
-L traction-r1:D DFLFS
+L traction-r1:D_21 DFLFS
 U 1 1 5E0000D2
 P 22200 21300
@@
 FFD_L
 $Comp
-L traction-r1:D DFLG
+L traction-r1:D_21 DFLG
 U 1 1 5E0000D3
 P 14400 24550
@@
 FDR_L
 $Comp
-L traction-r1:D DFLSN
+L traction-r1:D_21 DFLSN
 U 1 1 5E0000D4
 P 16350 23850
@@
 FCL_L
 $Comp
-L traction-r1:D DFLVZ
+L traction-r1:D_21 DFLVZ
 U 1 1 5E0000D5
 P 18350 24000
@@
 FVCC_L
 $Comp
-L traction-r1:D ZFLG
+L traction-r1:D_21 ZFLG
 U 1 1 5E0000E2
 P 14400 24950
@@
 FG_L
 $Comp
-L traction-r1:D ZFLSN
+L traction-r1:D_21 ZFLSN
 U 1 1 5E0000E3
 P 22200 22100
@@
 DCN
 $Comp
-L traction-r1:D DASCR
+L traction-r1:D_21 DASCR
 U 1 1 5E00010D
 P 34350 1550
@@
 DCN
 $Comp
-L traction-r1:D ZASC
+L traction-r1:D_21 ZASC
 U 1 1 5E000115
 P 34350 1950
@@
 DGND
 $Comp
-L traction-r1:D DRH
+L traction-r1:D_21 DRH
 U 1 1 5E000118
 P 30350 14300
@@
 NRH
 $Comp
-L traction-r1:D DTVH
+L traction-r1:D_21 DTVH
 U 1 1 5E000119
 P 30350 14700
@@
 DGND
 $Comp
-L traction-r1:D DRL
+L traction-r1:D_21 DRL
 U 1 1 5E00011E
 P 34350 14300
@@
 NRL
 $Comp
-L traction-r1:D DTVL
+L traction-r1:D_21 DTVL
 U 1 1 5E00011F
 P 34350 14700
@@
 V15VA
 $Comp
-L traction-r1:D DB15
+L traction-r1:D_21 DB15
 U 1 1 5E000130
 P 32250 8550

Commit message: Rev A.18: round 19 — three rechecks of e315bf1 (F199-F204): PTC-current row at every permitted voltage (IR-16 0.08/0.14/0.37/0.26 Ω), ≥8 A TVS energy an explicit assumption + QP-RX-04 release criterion, window criterion fixed, exciter TVS → SMDJ7.0A-HRA (coupled island holds the 7.0 V class at a parked 12 V battery / the Marine rail), shared exciter-fault model run for the Marine port (QP-MA-11, kit-loom rule), FW-35 rewritten on an SWG-anchored time origin with clock-derived resync and bounded restart
Co-Authored-By: Claude Fable 5.1 <noreply@anthropic.com>
Other:
- note added: "rev A.18 - 24 sections - 324 components"
- note removed: "rev A.17 - 24 sections - 324 components"
Changed lines of the file:
@@
 Title "Traction Inverter 220 kW — Power board (3x EconoDUAL 3 SiC)"
 Date "2026-09-23"
-Rev "A.17"
+Rev "A.18"
 Comp "Traction Inverter 220 kW pk - Power (HV), sheet 1 of 4"
 Comment1 "Inverter = Power board + Cap bank busbar + bolt-on Discharge board (all HV) + Control card (LV); safe state holds with any link lost"
@@
 DC-LINK   -   1 section
 Text Notes 29160 24850 0    60   ~ 0
-rev A.17   -   24 sections   -   324 components
+rev A.18   -   24 sections   -   324 components
 Wire Notes Line
 	9100 28000 17750 28000

Commit message: Rev A.19: round 20 — three rechecks of 00f6252 (F205-F207): TVS alternate to the 7.0 V class + lock, 4XX discharge alternate 470→220 Ω + lock, T-05/T-06 firmware ID, 8.5 V-era figures re-derived at the IR-16 allocations
Co-Authored-By: Claude Fable 5.1 <noreply@anthropic.com>
Other:
- note added: "rev A.19 - 24 sections - 324 components"
- note removed: "rev A.18 - 24 sections - 324 components"
Changed lines of the file:
@@
 Title "Traction Inverter 220 kW — Power board (3x EconoDUAL 3 SiC)"
 Date "2026-09-23"
-Rev "A.18"
+Rev "A.19"
 Comp "Traction Inverter 220 kW pk - Power (HV), sheet 1 of 4"
 Comment1 "Inverter = Power board + Cap bank busbar + bolt-on Discharge board (all HV) + Control card (LV); safe state holds with any link lost"
@@
 DC-LINK   -   1 section
 Text Notes 29160 24850 0    60   ~ 0
-rev A.18   -   24 sections   -   324 components
+rev A.19   -   24 sections   -   324 components
 Wire Notes Line
 	9100 28000 17750 28000

Commit message: Rev A.20: round 21 — three rechecks of 551c405 (F208): stale 0.29 Ω in gate ㉘ and the QP-RX-04 fixture instruction → 0.37 Ω, last 8.5 V-era figures aligned, Marine sweep cross-references at the current values
Co-Authored-By: Claude Fable 5.1 <noreply@anthropic.com>
Other:
- note added: "rev A.20 - 24 sections - 324 components"
- note removed: "rev A.19 - 24 sections - 324 components"
Changed lines of the file:
@@
 Title "Traction Inverter 220 kW — Power board (3x EconoDUAL 3 SiC)"
 Date "2026-09-23"
-Rev "A.19"
+Rev "A.20"
 Comp "Traction Inverter 220 kW pk - Power (HV), sheet 1 of 4"
 Comment1 "Inverter = Power board + Cap bank busbar + bolt-on Discharge board (all HV) + Control card (LV); safe state holds with any link lost"
@@
 DC-LINK   -   1 section
 Text Notes 29160 24850 0    60   ~ 0
-rev A.19   -   24 sections   -   324 components
+rev A.20   -   24 sections   -   324 components
 Wire Notes Line
 	9100 28000 17750 28000
