File: kicad5/traction-native/traction-power.sch (KiCad schematic (older format))
At the start: 324 parts, among them U5LB NCV4276CDT50RKG, U5LC NCV4276CDT50RKG

Commit message: Rev A.21: round 22 — three rechecks of 0ff44d9 (F209) + the layout handoff (F210–F213): every KiCad symbol bound to a footprint in a shipped traction.pretty (45 verbatim KiCad-10 patterns + 18 datasheet-drawn), fp-lib-table and per-board projects in all sets, pad-per-pin KiCad proof; NCV4276C 5-lead lands, ALM2402/TPS55340 thermal-pad pins, 2-pad crystal; QP §0.2 baseline and stale IDs; docs/layout-handoff.md
Co-Authored-By: Claude Fable 5.1 <noreply@anthropic.com>
Parts:
- C5B1, C5C1, C5G2, C5LB2, C5LC2, CASCI1, CASCI2, CB15I, CFHSN, CFLSN, CLVH1, CLVH2, CLVL1, CLVL2, CUHB2, CUHE1, CUHV1, CULB2, CULE1, CULV1, CVHB2, CVHE1, CVHV1, CVLB2, CVLE1, CVLV1, CWHB2, CWHE1, CWHV1, CWLB2, CWLE1, CWLV1: footprint C1206 -> traction:C_1206_3216Metric
- C5B2, C5C2, CASC, CASCD, CASCF, CASCIB, CB15C, CB15CC, CB15S, CFHCF, CFHCO, CFHCT, CFHFS, CFHSI, CFHVR, CFLCF, CFLCO, CFLCT, CFLFS, CFLSI, CFLVR, CLDC, CUHB1, CUHBL, CUHIN, CULB1, CULBL, CULIN, CUTF, CVBDF, CVDDF, CVHB1, CVHBL, CVHIN, CVLB1, CVLBL, CVLIN, CVTF, CWHB1, CWHBL, CWHIN, CWLB1, CWLBL, CWLIN, CWTF: footprint C0603 -> traction:C_0603_1608Metric
- C5G1, C5LB1, C5LC1: footprint C0805 -> traction:C_0805_2012Metric
- CASCO, CB15O1, CB15O2, CFHA, CFLA, CLD15: footprint C1210 -> traction:C_1210_3225Metric
- CPET: footprint disc, 10 mm pitch (FilmBoxFP(10) land) -> traction:C_Disc_D12.5mm_W5.0mm_P10.00mm
- CUSN, CVSN, CWSN: footprint FilmP27.5 -> traction:C_Rect_L31.5mm_W17.0mm_P27.50mm_MKS4
- CY1, CY2: footprint DiscP10 -> traction:C_Disc_D16.0mm_W5.0mm_P10.00mm
- DASCR, DFHFS, DFLFS, DTVSH, DUTP, DVTP, DWTP: footprint SOD323 -> traction:D_SOD-323
- DB15, DFHA, DFHSN, DFLA, DFLSN, DUHR, DUHS1, DUHS2, DULR, DULS1, DULS2, DVHR, DVHS1, DVHS2, DVLR, DVLS1, DVLS2, DWHR, DWHS1, DWHS2, DWLR, DWLS1, DWLS2, ZFHSN, ZFLSN: footprint SMA -> traction:D_SMA
- DFHG, DFLG: footprint SOD123 -> traction:D_SOD-123F
- DFHVZ, DFLVZ, DUHZ1, DUHZ2, DULZ1, DULZ2, DVHZ1, DVHZ2, DVLZ1, DVLZ2, DWHZ1, DWHZ2, DWLZ1, DWLZ2, ZASC, ZFHG, ZFLG, ZUHV, ZULV, ZVHV, ZVLV, ZWHV, ZWLV: footprint SOD123 -> traction:D_SOD-123
- DRH, DRL: footprint SMA-flat -> traction:NRVBAF360T3G_SMA-FL
- DTVH, DTVL: footprint SMC -> traction:D_SMC
- DUHSB, DULSB, DVHSB, DVLSB, DWHSB, DWLSB, QFHE1, QFHE2, QFLE1, QFLE2: footprint SOT23 -> traction:SOT-23-3
- FH1, FL1: footprint PTC2920 -> traction:Fuse_2920_7451Metric
- JDIS: footprint IPL1-104 (1x4 2.54 mm THT) -> traction:Samtec_IPL1-104_1x04
- JHVIL: footprint IPL1-102 (1x2 2.54 mm THT) -> traction:Samtec_IPL1-102_1x02
- JHVN, JHVP, JMU, JMV, JMW: footprint StudM8 -> traction:MountingHole_8.4mm_M8_Pad
- JIC: footprint HDR2x20-2.54 -> traction:Samtec_IPL1-120_2x20
- JPE: footprint StudM6 -> traction:MountingHole_6.4mm_M6_Pad
- LB15: footprint XAL4040 -> traction:L_Coilcraft_XAL4040-XXX
- LFH1, LFL1: footprint FB1206 -> traction:L_1206_3216Metric
- MODU, MODV, MODW: footprint EconoDUAL3 -> traction:EconoDUAL3
- PS5B, PS5C, UUHG, UULG, UVHG, UVLG, UWHG, UWLG: footprint SOIC16W -> traction:SOIC-16W_7.5x10.3mm_P1.27mm
- PSASC: footprint DWN36 -> traction:UCC14141-Q1_DWN36
- QFH, QFL: footprint LFPAK56 -> traction:LFPAK56
- R5LB, R5LC, RUHOFF, RUHON, RULOFF, RULON, RVHOFF, RVHON, RVLOFF, RVLON, RWHOFF, RWHON, RWLOFF, RWLON: footprint R2512 -> traction:R_2512_6332Metric
- RASCE1, RASCE2, RASCF1, RASCF2, RASCG, RASCL, RASCPD, RB15C, RB15F1, RB15F2, RB15Q, RFHEN, RFHFB1, RFHFB2, RFHFS, RFHG, RFHGO, RFHGS, RFHRT, RFHSI, RFLEN, RFLFB1, RFLFB2, RFLFS, RFLG, RFLGO, RFLGS, RFLRT, RFLSI, RGDLE, RHVL1, RHVL2, RHWID, RLD1, RLD2, RPD0, RPD1, RPD10, RPD2, RPD3, RPD4, RPD5, RPD6, RPD7, RPD8, RPD9, RULAS, RUTS, RVBDL, RVDDL, RVLAS, RVTS, RWLAS, RWTS: footprint R0603 -> traction:R_0603_1608Metric
- RFHCS, RFLCS: footprint R1210 -> traction:R_1210_3225Metric
- RFHSN, RFLSN, RUHBL, RUHDS, RUHGS, RUHMC, RULBL, RULDS, RULGS, RULMC, RVHBL, RVHDS, RVHGS, RVHMC, RVLBL, RVLDS, RVLGS, RVLMC, RWHBL, RWHDS, RWHGS, RWHMC, RWLBL, RWLDS, RWLGS, RWLMC: footprint R0805 -> traction:R_0805_2012Metric
- RFHST, RFLST, RPET, RUHPD, RULPD, RVBD1, RVBD2, RVBD3, RVBD4, RVBD5, RVBD6, RVDD1, RVDD2, RVDD3, RVDD4, RVDD5, RVDD6, RVHPD, RVLPD, RWHPD, RWLPD: footprint R1206 -> traction:R_1206_3216Metric
- TFH1, TFH2, TFH3, TFL1, TFL2, TFL3: footprint XfmrEE12 -> traction:VGT12EEM-200S1A4
- U5LB, U5LC, UGDL: footprint DPAK -> traction:TO-252-5_TabPin3
- UASC: footprint SMD8W -> traction:VOW3120_SMD8W
- UB15: footprint WQFN16 -> traction:WQFN-16-1EP_3x3mm_P0.5mm_EP1.68x1.68mm
- UFH, UFL: footprint SOP8 -> traction:SOIC-8_3.9x4.9mm_P1.27mm
- UIVB, UIVDC: footprint SOIC8W -> traction:AMC1311B_DWV8
- ULDO15: footprint D2PAK5 -> traction:TO-263-5_TabPin3
Connections:
- net B15CO: now also UB15.7 (COMP)
- net B15FB: now also UB15.8 (FB)
- net B15FQ: now also UB15.9 (FREQ)
- net B15SS: now also UB15.4 (SS)
- net B15SW: now also UB15.1 (SW1), UB15.15 (SW2), UB15.16 (SW3)
- net DGND: now also UB15.10 (NC1), UB15.11 (PGND1), UB15.12 (PGND2), UB15.13 (PGND3), UB15.14 (NC2), UB15.17 (PAD), UB15.5 (SYNC), UB15.6 (AGND)
- net V12L: now also UB15.2 (VIN1), UB15.3 (EN)
Other:
- note added: "rev A.21 - 24 sections - 324 components"
- note removed: "rev A.20 - 24 sections - 324 components"
- moved on the sheet: CB15C, CB15CC, CB15I, CB15O1, CB15O2, CB15S, CLD15, CLDC, DB15, LB15, RB15C, RB15F1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

Commit message: Rev A.22: round 23 — rechecks of 452de85 (F214–F220), the VESC program (FW-38…FW-46, Traction Tool in Qt) and the "why not done" extension (F221–F239)
Hardware: the R2R reference isolated at ball A9 (RR2R 10 Ω + 1 µF + 100 nF, S32K39 DS note 8), the SWD header on its
surface-mount Samtec land with a mounting-technology lock in the library generator, the footprint library declared
KiCad 10.0.6+ and no longer mirrored into the KiCad 5 sets; the BOM intro follows the SKU; a VREFH window row and VR-34/35.

Firmware (TI_FW_ID 0x0A0F0015, CAL layout 4, 190 fields / 91 CAL rows, 80 DTCs): FW-37 joint torque solve with a
postcondition; the VESC gap closure — FW-38 signed field update (Ed25519, anti-rollback, ISO-TP), FW-39 interlocked motor
self-commissioning, FW-40 UDS diagnostics (0x19/0x22/0x2A/0x14 over ISO 15765-2), FW-41 fault-triggered waveform capture,
FW-42 overspeed, FW-43 run-time statistics, FW-44 key-on offset adoption, FW-45 saturation-dependent inductance tables
with gain scheduling, FW-46 cogging feed-forward; twelve defects found by the closed-loop simulator bridge (F221–F232),
the 64-bit divide out of every ISR path with a link-time guard, the UDS escape single frame accepted by every service,
the root of trust reported (DID 0xFD23), the boot record, motor data and active maps as DIDs; 421 tests / 4937 checks /
0 failed on the host (-O1, -O2, ASan/UBSan, -ffp-contract=off) and on the Cortex-M7 under QEMU with the target compiler
(make qemu-test, T-59); make target-check 63 markers, make target-size with the divide guard.

Traction Tool (tool/): Qt 6 / C++17 Widgets + Qwt, offline; pages Dashboard, Live plots, Controls, Commissioning,
Parameters, Faults & alerts, Analysis, Terminal, Firmware; transports simulator bridge (tool/bridge, the real firmware
against a plant), log replay, CAN (QCanBus with ISO-TP both ways, proved against the firmware over the virtualcan bus);
the signed update end to end over both transports; the commissioning routines, the map sw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
Other:
- note added: "rev A.22 - 24 sections - 324 components"
- note removed: "rev A.21 - 24 sections - 324 components"
Changed lines of the file:
@@
 Title "Traction Inverter 220 kW — Power board (3x EconoDUAL 3 SiC)"
 Date "2026-09-23"
-Rev "A.21"
+Rev "A.22"
 Comp "Traction Inverter 220 kW pk - Power (HV), sheet 1 of 4"
 Comment1 "Inverter = Power board + Cap bank busbar + bolt-on Discharge board (all HV) + Control card (LV); safe state holds with any link lost"
@@
 DC-LINK   -   1 section
 Text Notes 29160 24850 0    60   ~ 0
-rev A.21   -   24 sections   -   324 components
+rev A.22   -   24 sections   -   324 components
 Wire Notes Line
 	9100 28000 17750 28000

Commit message: Rev A.23: round 24 — four rechecks of 4ed0101 (F240–F244): the SDADC reference on its supply node, acquisition freshness, the map's flux slope and the ripple limiter's exact bounds, the temperature latch, the V_DC expiry
Hardware (F240, no new part): the S32K39 data sheet's SDADC table (Rev. 3 Table 38, in our archive and our own
extracted-parameters file) requires VREFP within ±25 mV of AVDD; the round-23 disposition had judged the general +100 mV
note and called the figure absent while the references sat on the FS26 VREF, matched to the SDADC-supply LDO only within
±1 %. Every non-R2R reference group (E6/H6 SAR, E10/F13 SDADC) is now on V5A itself with VDDA_SDADC and VDD_HV_A (NXP's
GEN3 arrangement); the ratiometric loads (HW_ID and offset dividers, the seven NTC pull-ups) moved with the reference; the
R2R ladder keeps the FS26 VREF as its isolated supply through the 10 Ω branch (CR2R1 330 nF, 37 kHz); CSB5 2.2 µF holds
the FS26 window alone (1.36–2.92 µF effective); the absolute SAR scale re-budgeted at the LDO2's ±1.75 %; ERC locks, pin
freeze, manifest, handoff §4.11 island rule (≤ 20 mΩ from E12 to any VREFH ball), VR-34 closed by design, IR-26, QP-TH-06.
Pipeline at A.23: ERC 981/0/0, verify 158/18/0, sim 23/6/0, Marine 87/23/0, 21 pages / 2065 pins, KiCad proof PASS, PDFs
and BOMs regenerated (₹72,983 unchanged). The handoff §6 gives every open pre-layout decision a provisional default.

Firmware (TI_FW_ID 0x0A0F0016, CAL layout 4, 191 fields / 92 CAL rows, 82 DTCs): F241 a stopped slow ADC channel stayed
valid forever (the caller discarded the acquisition stamp) → a three-state contract new/held/expired for every slow-list
input with cal_temp_hold_ms and DTC_ADC_SLOW_STALE, every slow consumer audited (V5GD/VOFS, IGN, INTRLOK_N, VSUP, HW_ID);
F242 the inductance map must keep a positive flux slope (≥ 0.25 × L0 below every breakpoint) and the ripple limiter bounds
every piece of its interval in closed form (breakpoints alone shown insufficient by a 20 000-m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
Other:
- note added: "rev A.23 - 24 sections - 324 components"
- note removed: "rev A.22 - 24 sections - 324 components"
Changed lines of the file:
@@
 Title "Traction Inverter 220 kW — Power board (3x EconoDUAL 3 SiC)"
 Date "2026-09-23"
-Rev "A.22"
+Rev "A.23"
 Comp "Traction Inverter 220 kW pk - Power (HV), sheet 1 of 4"
 Comment1 "Inverter = Power board + Cap bank busbar + bolt-on Discharge board (all HV) + Control card (LV); safe state holds with any link lost"
@@
 DC-LINK   -   1 section
 Text Notes 29160 24850 0    60   ~ 0
-rev A.22   -   24 sections   -   324 components
+rev A.23   -   24 sections   -   324 components
 Wire Notes Line
 	9100 28000 17750 28000
